Commit message: modified path in models

File: arm/xacro/full_arm_motor.urdf.xacro (robot description, xacro)
@@ -4,9 +4,9 @@
        xmlns:xacro="http://www.ros.org/wiki/xacro"
        name="full_arm_motor">
-  <include filename="$(find sr_hand)/model/arm_urdf/base/shadowarm_base.urdf.xacro" />
-  <include filename="$(find sr_hand)/model/arm_urdf/trunk/shadowarm_trunk.urdf.xacro" />
-  <include filename="$(find sr_hand)/model/arm_urdf/upper_arm/shadowarm_upperarm.urdf.xacro" />
-  <include filename="$(find sr_hand)/model/arm_urdf/lower_arm/shadowarm_lowerarm.urdf.xacro" />
-  <include filename="$(find sr_hand)/model/arm_urdf/hand_support/shadowarm_handsupport_motor.urdf.xacro" />
+  <include filename="$(find sr_description)/arm/xacro/base/shadowarm_base.urdf.xacro" />
+  <include filename="$(find sr_description)/arm/xacro/trunk/shadowarm_trunk.urdf.xacro" />
+  <include filename="$(find sr_description)/arm/xacro/upper_arm/shadowarm_upperarm.urdf.xacro" />
+  <include filename="$(find sr_description)/arm/xacro/lower_arm/shadowarm_lowerarm.urdf.xacro" />
+  <include filename="$(find sr_description)/arm/xacro/hand_support/shadowarm_handsupport_motor.urdf.xacro" />
   <xacro:macro name="sr_arm_motor">
     <xacro:shadowarm_base>

File: arm/xacro/full_arm_motor_with_kinect.urdf.xacro (robot description, xacro)
@@ -4,10 +4,10 @@
        xmlns:xacro="http://www.ros.org/wiki/xacro"
        name="full_arm_motor">
-  <include filename="$(find sr_hand)/model/arm_urdf/base/shadowarm_base.urdf.xacro" />
-  <include filename="$(find sr_hand)/model/arm_urdf/trunk/shadowarm_trunk.urdf.xacro" />
-  <include filename="$(find sr_hand)/model/arm_urdf/upper_arm/shadowarm_upperarm.urdf.xacro" />
-  <include filename="$(find sr_hand)/model/arm_urdf/lower_arm/shadowarm_lowerarm.urdf.xacro" />
-  <include filename="$(find sr_hand)/model/arm_urdf/hand_support/shadowarm_handsupport_motor.urdf.xacro" />
-  <include filename="$(find sr_hand)/model/kinect/shadowarm_kinect.urdf.xacro" />
+  <include filename="$(find sr_description)/arm/xacro/base/shadowarm_base.urdf.xacro" />
+  <include filename="$(find sr_description)/arm/xacro/trunk/shadowarm_trunk.urdf.xacro" />
+  <include filename="$(find sr_description)/arm/xacro/upper_arm/shadowarm_upperarm.urdf.xacro" />
+  <include filename="$(find sr_description)/arm/xacro/lower_arm/shadowarm_lowerarm.urdf.xacro" />
+  <include filename="$(find sr_description)/arm/xacro/hand_support/shadowarm_handsupport_motor.urdf.xacro" />
+  <include filename="$(find sr_description)/other/xacro/kinect/shadowarm_kinect.urdf.xacro" />
   <xacro:macro name="sr_arm_motor">
     <xacro:shadowarm_base>

File: arm/xacro/full_arm_muscle.urdf.xacro (robot description, xacro)
@@ -4,9 +4,9 @@
        xmlns:xacro="http://www.ros.org/wiki/xacro"
        name="full_arm_muscle">
-  <include filename="$(find sr_hand)/model/arm_urdf/base/shadowarm_base.urdf.xacro" />
-  <include filename="$(find sr_hand)/model/arm_urdf/trunk/shadowarm_trunk.urdf.xacro" />
-  <include filename="$(find sr_hand)/model/arm_urdf/upper_arm/shadowarm_upperarm.urdf.xacro" />
-  <include filename="$(find sr_hand)/model/arm_urdf/lower_arm/shadowarm_lowerarm.urdf.xacro" />
-  <include filename="$(find sr_hand)/model/arm_urdf/hand_support/shadowarm_handsupport_muscle.urdf.xacro" />
+  <include filename="$(find sr_description)/arm/xacro/base/shadowarm_base.urdf.xacro" />
+  <include filename="$(find sr_description)/arm/xacro/trunk/shadowarm_trunk.urdf.xacro" />
+  <include filename="$(find sr_description)/arm/xacro/upper_arm/shadowarm_upperarm.urdf.xacro" />
+  <include filename="$(find sr_description)/arm/xacro/lower_arm/shadowarm_lowerarm.urdf.xacro" />
+  <include filename="$(find sr_description)/arm/xacro/hand_support/shadowarm_handsupport_muscle.urdf.xacro" />
   <xacro:macro name="sr_arm_muscle">
     <xacro:shadowarm_base>

File: arm/xacro/hand_support/shadowarm_handsupport_motor.urdf.xacro (robot description, xacro)
@@ -1,4 +1,4 @@
 <robot xmlns:xacro="http://www.ros.org/wiki/xacro">
-  <include filename="$(find sr_hand)/model/arm_urdf/hand_support/shadowarm_handsupport_motor.transmission.xacro" />
+  <include filename="$(find sr_description)/arm/xacro/hand_support/shadowarm_handsupport_motor.transmission.xacro" />
   <xacro:macro name="shadowarm_handsupport_motor" params="parent">
     <link name="shadowarm_handsupport_motor">
@@ -11,5 +11,5 @@
 	<origin xyz="0 0 -0.04" rpy="0 0 0"/>
 	<geometry name="shadowarm_handsupport_visual">
-	  <mesh filename="package://sr_hand/model/meshes/arm/elbow_rotate_motor.dae" scale="0.001 0.001 0.001" />
+	  <mesh filename="package://sr_description/arm/model/elbow_rotate_motor.dae" scale="0.001 0.001 0.001" />
 	</geometry>
 	<material name="LightGrey" />

File: arm/xacro/hand_support/shadowarm_handsupport_muscle.urdf.xacro (robot description, xacro)
@@ -1,4 +1,4 @@
 <robot xmlns:xacro="http://www.ros.org/wiki/xacro">
-  <include filename="$(find sr_hand)/model/arm_urdf/hand_support/shadowarm_handsupport_muscle.transmission.xacro" />
+  <include filename="$(find sr_description)/arm/xacro/hand_support/shadowarm_handsupport_muscle.transmission.xacro" />
   <xacro:macro name="shadowarm_handsupport_muscle" params="parent">
     <link name="shadowarm_handsupport_muscle">
@@ -11,5 +11,5 @@
 	<origin xyz="0 0 -0.04" rpy="${M_PI/2} 0 0"/>
 	<geometry name="shadowarm_handsupport_visual">
-	  <mesh filename="package://sr_hand/model/meshes/arm/elbow_rotate_muscle.mesh" scale="0.001 0.001 0.001" />
+	  <mesh filename="package://sr_description/arm/model/elbow_rotate_muscle.mesh" scale="0.001 0.001 0.001" />
 	</geometry>
 	<material name="LightGrey" />

File: hand/xacro/finger/classic_finger.urdf.xacro (robot description, xacro)
@@ -1,7 +1,7 @@
 <robot xmlns:xacro="http://www.ros.org/wiki/xacro">
-  <include filename="$(find sr_hand)/model/hand_urdf/finger/knuckle/knuckle.urdf.xacro" />
-  <include filename="$(find sr_hand)/model/hand_urdf/finger/proximal/proximal.urdf.xacro" />
-  <include filename="$(find sr_hand)/model/hand_urdf/finger/middle/middle.urdf.xacro" />
-  <include filename="$(find sr_hand)/model/hand_urdf/finger/distal/distal.urdf.xacro" />
+  <include filename="$(find sr_description/hand/xacro/finger/knuckle/knuckle.urdf.xacro" />
+  <include filename="$(find sr_description/hand/xacro/finger/proximal/proximal.urdf.xacro" />
+  <include filename="$(find sr_description/hand/xacro/finger/middle/middle.urdf.xacro" />
+  <include filename="$(find sr_description/hand/xacro/finger/distal/distal.urdf.xacro" />
   <xacro:macro name="finger" params="link_prefix joint_prefix parent *origin *axis">
     <xacro:knuckle link_prefix="${link_prefix}" joint_prefix="${joint_prefix}" parent="${parent}" >

File: hand/xacro/finger/classic_finger_biotac.urdf.xacro (robot description, xacro)
@@ -1,7 +1,7 @@
 <robot xmlns:xacro="http://www.ros.org/wiki/xacro">
-  <include filename="$(find sr_hand)/model/hand_urdf/finger/knuckle/knuckle.urdf.xacro" />
-  <include filename="$(find sr_hand)/model/hand_urdf/finger/proximal/proximal.urdf.xacro" />
-  <include filename="$(find sr_hand)/model/hand_urdf/finger/middle/middle.urdf.xacro" />
-  <include filename="$(find sr_hand)/model/hand_urdf/finger/distal/distal_biotac.urdf.xacro" />
+  <include filename="$(find sr_description/hand/xacro/finger/knuckle/knuckle.urdf.xacro" />
+  <include filename="$(find sr_description/hand/xacro/finger/proximal/proximal.urdf.xacro" />
+  <include filename="$(find sr_description/hand/xacro/finger/middle/middle.urdf.xacro" />
+  <include filename="$(find sr_description/hand/xacro/finger/distal/distal_biotac.urdf.xacro" />
   <xacro:macro name="finger" params="link_prefix joint_prefix parent *origin *axis">
     <xacro:knuckle link_prefix="${link_prefix}" joint_prefix="${joint_prefix}" parent="${parent}" >

File: hand/xacro/finger/classic_finger_ellipsoid.urdf.xacro (robot description, xacro)
@@ -1,7 +1,7 @@
 <robot xmlns:xacro="http://www.ros.org/wiki/xacro">
-  <include filename="$(find sr_hand)/model/hand_urdf/finger/knuckle/knuckle.urdf.xacro" />
-  <include filename="$(find sr_hand)/model/hand_urdf/finger/proximal/proximal.urdf.xacro" />
-  <include filename="$(find sr_hand)/model/hand_urdf/finger/middle/middle.urdf.xacro" />
-  <include filename="$(find sr_hand)/model/hand_urdf/finger/distal/distal_ellipsoid.urdf.xacro" />
+  <include filename="$(find sr_description/hand/xacro/finger/knuckle/knuckle.urdf.xacro" />
+  <include filename="$(find sr_description/hand/xacro/finger/proximal/proximal.urdf.xacro" />
+  <include filename="$(find sr_description/hand/xacro/finger/middle/middle.urdf.xacro" />
+  <include filename="$(find sr_description/hand/xacro/finger/distal/distal_ellipsoid.urdf.xacro" />
   <xacro:macro name="finger" params="link_prefix joint_prefix parent *origin *axis">
     <xacro:knuckle link_prefix="${link_prefix}" joint_prefix="${joint_prefix}" parent="${parent}" >

File: hand/xacro/finger/distal/distal.urdf.xacro (robot description, xacro)
@@ -6,5 +6,5 @@
        xmlns:body="http://playerstage.sourceforge.net/gazebo/xmlschema/#body"
        xmlns:geom="http://playerstage.sourceforge.net/gazebo/xmlschema/#geom">
-  <include filename="$(find sr_hand)/model/hand_urdf/finger/distal/distal.transmission.xacro" />
+  <include filename="$(find sr_description/hand/xacro/finger/distal/distal.transmission.xacro" />
   <xacro:macro name="distal" params="link_prefix joint_prefix parent">
     <link name="${link_prefix}distal">
@@ -18,5 +18,5 @@
 	<origin xyz="0 0 0" rpy="0 0 0" />
 	<geometry name="distal_visual">
-      <mesh filename="package://sr_hand/model/meshes/F1.dae" scale="0.001 0.001 0.001" />
+      <mesh filename="package://sr_description/hand/model/F1.dae" scale="0.001 0.001 0.001" />
       </geometry>
       <material name="Grey" />
@@ -25,5 +25,5 @@
 	<origin xyz="0 0 0" rpy="0 0 0" />
 	<geometry name="distal_collision_geom">
-	 <mesh filename="package://sr_hand/model/meshes/F1.dae" scale="0.001 0.001 0.001" />
+	 <mesh filename="package://sr_description/hand/model/F1.dae" scale="0.001 0.001 0.001" />
 	</geometry>
       </collision>

File: hand/xacro/finger/distal/distal_biotac.urdf.xacro (robot description, xacro)
@@ -6,5 +6,5 @@
        xmlns:body="http://playerstage.sourceforge.net/gazebo/xmlschema/#body"
        xmlns:geom="http://playerstage.sourceforge.net/gazebo/xmlschema/#geom">
-  <include filename="$(find sr_hand)/model/hand_urdf/finger/distal/distal.transmission.xacro" />
+  <include filename="$(find sr_description/hand/xacro/finger/distal/distal.transmission.xacro" />
   <xacro:macro name="distal" params="link_prefix joint_prefix parent">
     <link name="${link_prefix}distal">
@@ -18,5 +18,5 @@
 	<origin xyz="0 0 0" rpy="0 0 0" />
 	<geometry name="distal_visual">
-      <mesh filename="package://sr_hand/model/meshes/F1.mesh" scale="0.001 0.001 0.001" />
+      <mesh filename="package://sr_description/hand/model/F1.mesh" scale="0.001 0.001 0.001" />
       </geometry>
       <material name="Grey" />
@@ -25,5 +25,5 @@
 	<origin xyz="0 0 0" rpy="0 0 0" />
 	<geometry name="distal_collision_geom">
-	  <mesh filename="package://sr_hand/model/meshes/F1.mesh" scale="0.001 0.001 0.001" />
+	  <mesh filename="package://sr_description/hand/model/F1.mesh" scale="0.001 0.001 0.001" />
 	</geometry>
       </collision>

File: hand/xacro/finger/distal/distal_ellipsoid.urdf.xacro (robot description, xacro)
@@ -6,5 +6,5 @@
        xmlns:body="http://playerstage.sourceforge.net/gazebo/xmlschema/#body"
        xmlns:geom="http://playerstage.sourceforge.net/gazebo/xmlschema/#geom">
-  <include filename="$(find sr_hand)/model/hand_urdf/finger/distal/distal.transmission.xacro" />
+  <include filename="$(find sr_description/hand/xacro/finger/distal/distal.transmission.xacro" />
   <xacro:macro name="distal" params="link_prefix joint_prefix parent">
     <link name="${link_prefix}distal">
@@ -18,5 +18,5 @@
 	<origin xyz="0 0 0" rpy="0 0 0" />
 	<geometry name="distal_visual">
-	  <mesh filename="package://sr_hand/model/meshes/distal_ellipsoid.dae" scale="0.001 0.001 0.001" />
+	  <mesh filename="package://sr_description/hand/model/distal_ellipsoid.dae" scale="0.001 0.001 0.001" />
 	</geometry>
 	<material name="Grey" />
@@ -25,5 +25,5 @@
 	   <origin xyz="0 0 0" rpy="0 0 0" />
 	   <geometry name="nano17">
-	   <mesh filename="package://sr_hand/model/meshes/nano17.dae" scale="0.001 0.001 0.001" />
+	   <mesh filename="package://sr_description/hand/model/nano17.dae" scale="0.001 0.001 0.001" />
 	   </geometry>
 	   <material name="Grey" />
@@ -32,5 +32,5 @@
         <origin xyz="0 0 0" rpy="0 0 0" />
         <geometry name="distal_collision_geom">
-          <mesh filename="package://sr_hand/model/meshes/distal_ellipsoid.dae" scale="0.001 0.001 0.001" />
+          <mesh filename="package://sr_description/hand/model/distal_ellipsoid.dae" scale="0.001 0.001 0.001" />
         </geometry>
       </collision>

File: hand/xacro/finger/knuckle/knuckle.urdf.xacro (robot description, xacro)
@@ -6,5 +6,5 @@
        xmlns:body="http://playerstage.sourceforge.net/gazebo/xmlschema/#body"
        xmlns:geom="http://playerstage.sourceforge.net/gazebo/xmlschema/#geom">
-  <include filename="$(find sr_hand)/model/hand_urdf/finger/knuckle/knuckle.transmission.xacro" />
+  <include filename="$(find sr_description/hand/xacro/finger/knuckle/knuckle.transmission.xacro" />
   <xacro:macro name="knuckle" params="link_prefix joint_prefix parent *origin">
     <link name="${link_prefix}knuckle">
@@ -19,5 +19,5 @@
 	<origin xyz="0 0 0.0005" rpy="0 0 0" />
 	<geometry name="knuckle_visual">
-      <mesh filename="package://sr_hand/model/meshes/knuckle.dae" scale="0.001 0.001 0.001" />
+      <mesh filename="package://sr_description/hand/model/knuckle.dae" scale="0.001 0.001 0.001" />
       </geometry>
       <material name="LightGrey" />

File: hand/xacro/finger/lfmetacarpal/lfmetacarpal.urdf.xacro (robot description, xacro)
@@ -6,5 +6,5 @@
        xmlns:body="http://playerstage.sourceforge.net/gazebo/xmlschema/#body"
        xmlns:geom="http://playerstage.sourceforge.net/gazebo/xmlschema/#geom">
-  <include filename="$(find sr_hand)/model/hand_urdf/finger/lfmetacarpal/lfmetacarpal.transmission.xacro" />
+  <include filename="$(find sr_description/hand/xacro/finger/lfmetacarpal/lfmetacarpal.transmission.xacro" />
   <!-- Right Handed -->
   <xacro:macro name="lfmetacarpal" params="parent">
@@ -27,5 +27,5 @@
         <origin xyz="0 0 0" rpy="0 0 0" />
         <geometry name="lfmetacarpal_visual">
-          <mesh filename="package://sr_hand/model/meshes/${mesh}" scale="0.001 0.001 0.001" />
+          <mesh filename="package://sr_description/hand/model/${mesh}" scale="0.001 0.001 0.001" />
         </geometry>
         <material name="Grey" />

File: hand/xacro/finger/little_finger.urdf.xacro (robot description, xacro)
@@ -6,9 +6,9 @@
        xmlns:body="http://playerstage.sourceforge.net/gazebo/xmlschema/#body"
        xmlns:geom="http://playerstage.sourceforge.net/gazebo/xmlschema/#geom">
-  <include filename="$(find sr_hand)/model/hand_urdf/finger/knuckle/knuckle.urdf.xacro" />
-  <include filename="$(find sr_hand)/model/hand_urdf/finger/proximal/proximal.urdf.xacro" />
-  <include filename="$(find sr_hand)/model/hand_urdf/finger/middle/middle.urdf.xacro" />
-  <include filename="$(find sr_hand)/model/hand_urdf/finger/distal/distal.urdf.xacro" />
-  <include filename="$(find sr_hand)/model/hand_urdf/finger/lfmetacarpal/lfmetacarpal.urdf.xacro" />
+  <include filename="$(find sr_description/hand/xacro/finger/knuckle/knuckle.urdf.xacro" />
+  <include filename="$(find sr_description/hand/xacro/finger/proximal/proximal.urdf.xacro" />
+  <include filename="$(find sr_description/hand/xacro/finger/middle/middle.urdf.xacro" />
+  <include filename="$(find sr_description/hand/xacro/finger/distal/distal.urdf.xacro" />
+  <include filename="$(find sr_description/hand/xacro/finger/lfmetacarpal/lfmetacarpal.urdf.xacro" />
   <!-- Right Handed -->
   <xacro:macro name="little_finger" params="link_prefix joint_prefix parent">
@@ -34,5 +34,5 @@
         <origin xyz="0 0 0" rpy="0 0 0" />
         <geometry name="knuckle_visual">
-          <mesh filename="package://sr_hand/model/meshes/knuckle.dae" scale="0.001 0.001 0.001" />
+          <mesh filename="package://sr_description/hand/model/knuckle.dae" scale="0.001 0.001 0.001" />
         </geometry>
         <material name="LightGrey" />

File: hand/xacro/finger/little_finger_biotac.urdf.xacro (robot description, xacro)
@@ -6,9 +6,9 @@
        xmlns:body="http://playerstage.sourceforge.net/gazebo/xmlschema/#body"
        xmlns:geom="http://playerstage.sourceforge.net/gazebo/xmlschema/#geom">
-  <include filename="$(find sr_hand)/model/hand_urdf/finger/knuckle/knuckle.urdf.xacro" />
-  <include filename="$(find sr_hand)/model/hand_urdf/finger/proximal/proximal.urdf.xacro" />
-  <include filename="$(find sr_hand)/model/hand_urdf/finger/middle/middle.urdf.xacro" />
-  <include filename="$(find sr_hand)/model/hand_urdf/finger/distal/distal_biotac.urdf.xacro" />
-  <include filename="$(find sr_hand)/model/hand_urdf/finger/lfmetacarpal/lfmetacarpal.urdf.xacro" />
+  <include filename="$(find sr_description/hand/xacro/finger/knuckle/knuckle.urdf.xacro" />
+  <include filename="$(find sr_description/hand/xacro/finger/proximal/proximal.urdf.xacro" />
+  <include filename="$(find sr_description/hand/xacro/finger/middle/middle.urdf.xacro" />
+  <include filename="$(find sr_description/hand/xacro/finger/distal/distal_biotac.urdf.xacro" />
+  <include filename="$(find sr_description/hand/xacro/finger/lfmetacarpal/lfmetacarpal.urdf.xacro" />
   <!-- Right Handed -->
   <xacro:macro name="little_finger" params="link_prefix joint_prefix parent">
@@ -34,5 +34,5 @@
         <origin xyz="0 0 0" rpy="0 0 0" />
         <geometry name="knuckle_visual">
-          <mesh filename="package://sr_hand/model/meshes/knuckle.dae" scale="0.001 0.001 0.001" />
+          <mesh filename="package://sr_description/hand/model/knuckle.dae" scale="0.001 0.001 0.001" />
         </geometry>
         <material name="LightGrey" />

File: hand/xacro/finger/little_finger_ellipsoid.urdf.xacro (robot description, xacro)
@@ -6,9 +6,9 @@
        xmlns:body="http://playerstage.sourceforge.net/gazebo/xmlschema/#body"
        xmlns:geom="http://playerstage.sourceforge.net/gazebo/xmlschema/#geom">
-  <include filename="$(find sr_hand)/model/hand_urdf/finger/knuckle/knuckle.urdf.xacro" />
-  <include filename="$(find sr_hand)/model/hand_urdf/finger/proximal/proximal.urdf.xacro" />
-  <include filename="$(find sr_hand)/model/hand_urdf/finger/middle/middle.urdf.xacro" />
-  <include filename="$(find sr_hand)/model/hand_urdf/finger/distal/distal_ellipsoid.urdf.xacro" />
-  <include filename="$(find sr_hand)/model/hand_urdf/finger/lfmetacarpal/lfmetacarpal.urdf.xacro" />
+  <include filename="$(find sr_description/hand/xacro/finger/knuckle/knuckle.urdf.xacro" />
+  <include filename="$(find sr_description/hand/xacro/finger/proximal/proximal.urdf.xacro" />
+  <include filename="$(find sr_description/hand/xacro/finger/middle/middle.urdf.xacro" />
+  <include filename="$(find sr_description/hand/xacro/finger/distal/distal_ellipsoid.urdf.xacro" />
+  <include filename="$(find sr_description/hand/xacro/finger/lfmetacarpal/lfmetacarpal.urdf.xacro" />
   <xacro:macro name="little_finger" params="link_prefix joint_prefix parent">
     <xacro:lfmetacarpal parent="${parent}" >
@@ -24,5 +24,5 @@
 	<origin xyz="0 0 0" rpy="0 0 0" />
 	<geometry name="knuckle_visual">
-      <mesh filename="package://sr_hand/model/meshes/knuckle.dae" scale="0.001 0.001 0.001" />
+      <mesh filename="package://sr_description/hand/model/knuckle.dae" scale="0.001 0.001 0.001" />
       </geometry>
       <material name="LightGrey" />

File: hand/xacro/finger/middle/middle.urdf.xacro (robot description, xacro)
@@ -6,5 +6,5 @@
        xmlns:body="http://playerstage.sourceforge.net/gazebo/xmlschema/#body"
        xmlns:geom="http://playerstage.sourceforge.net/gazebo/xmlschema/#geom">
-  <include filename="$(find sr_hand)/model/hand_urdf/finger/middle/middle.transmission.xacro" />
+  <include filename="$(find sr_description/hand/xacro/finger/middle/middle.transmission.xacro" />
   <xacro:macro name="middle" params="link_prefix joint_prefix parent">
     <link name="${link_prefix}middle">
@@ -18,5 +18,5 @@
 	<origin xyz="0 0 0" rpy="0 0 0" />
 	<geometry name="middle_visual">
-      <mesh filename="package://sr_hand/model/meshes/F2.dae" scale="0.001 0.001 0.001" />
+      <mesh filename="package://sr_description/hand/model/F2.dae" scale="0.001 0.001 0.001" />
       </geometry>
       <material name="Grey" />

File: hand/xacro/finger/proximal/proximal.urdf.xacro (robot description, xacro)
@@ -6,5 +6,5 @@
        xmlns:body="http://playerstage.sourceforge.net/gazebo/xmlschema/#body"
        xmlns:geom="http://playerstage.sourceforge.net/gazebo/xmlschema/#geom">
-  <include filename="$(find sr_hand)/model/hand_urdf/finger/proximal/proximal.transmission.xacro" />
+  <include filename="$(find sr_description/hand/xacro/finger/proximal/proximal.transmission.xacro" />
   <xacro:macro name="proximal" params="link_prefix joint_prefix parent">
     <link name="${link_prefix}proximal">
@@ -18,5 +18,5 @@
 	<origin xyz="0 0 0" rpy="0 0 0" />
 	<geometry name="proximal_visual">
-      <mesh filename="package://sr_hand/model/meshes/F3.dae" scale="0.001 0.001 0.001" />
+      <mesh filename="package://sr_description/hand/model/F3.dae" scale="0.001 0.001 0.001" />
       </geometry>
       <material name="Grey" />

File: hand/xacro/full_hand_motor.urdf.xacro (robot description, xacro)
@@ -3,10 +3,10 @@
        xmlns:interface="http://playerstage.sourceforge.net/gazebo/xmlschema/#interface"
        xmlns:xacro="http://www.ros.org/wiki/xacro">
-  <include filename="$(find sr_hand)/model/hand_urdf/forearm/forearm_motor.urdf.xacro" />
-  <include filename="$(find sr_hand)/model/hand_urdf/wrist/wrist.urdf.xacro" />
-  <include filename="$(find sr_hand)/model/hand_urdf/palm/palm.urdf.xacro" />
-  <include filename="$(find sr_hand)/model/hand_urdf/finger/classic_finger.urdf.xacro" />
-  <include filename="$(find sr_hand)/model/hand_urdf/finger/little_finger.urdf.xacro" />
-  <include filename="$(find sr_hand)/model/hand_urdf/thumb/thumb.urdf.xacro" />
+  <include filename="$(find sr_description/hand/xacro/forearm/forearm_motor.urdf.xacro" />
+  <include filename="$(find sr_description/hand/xacro/wrist/wrist.urdf.xacro" />
+  <include filename="$(find sr_description/hand/xacro/palm/palm.urdf.xacro" />
+  <include filename="$(find sr_description/hand/xacro/finger/classic_finger.urdf.xacro" />
+  <include filename="$(find sr_description/hand/xacro/finger/little_finger.urdf.xacro" />
+  <include filename="$(find sr_description/hand/xacro/thumb/thumb.urdf.xacro" />
   <!-- Right Hand -->
   <xacro:macro name="shadowhand_motor">
