Commit message: modified path in models

File: hand/xacro/full_hand_motor_biotac.urdf.xacro (robot description, xacro)
@@ -3,10 +3,10 @@
        xmlns:interface="http://playerstage.sourceforge.net/gazebo/xmlschema/#interface"
        xmlns:xacro="http://www.ros.org/wiki/xacro">
-  <include filename="$(find sr_hand)/model/hand_urdf/forearm/forearm_motor.urdf.xacro" />
-  <include filename="$(find sr_hand)/model/hand_urdf/wrist/wrist.urdf.xacro" />
-  <include filename="$(find sr_hand)/model/hand_urdf/palm/palm.urdf.xacro" />
-  <include filename="$(find sr_hand)/model/hand_urdf/finger/classic_finger_biotac.urdf.xacro" />
-  <include filename="$(find sr_hand)/model/hand_urdf/finger/little_finger_biotac.urdf.xacro" />
-  <include filename="$(find sr_hand)/model/hand_urdf/thumb/thumb_biotac.urdf.xacro" />
+  <include filename="$(find sr_description/hand/xacro/forearm/forearm_motor.urdf.xacro" />
+  <include filename="$(find sr_description/hand/xacro/wrist/wrist.urdf.xacro" />
+  <include filename="$(find sr_description/hand/xacro/palm/palm.urdf.xacro" />
+  <include filename="$(find sr_description/hand/xacro/finger/classic_finger_biotac.urdf.xacro" />
+  <include filename="$(find sr_description/hand/xacro/finger/little_finger_biotac.urdf.xacro" />
+  <include filename="$(find sr_description/hand/xacro/thumb/thumb_biotac.urdf.xacro" />
   <!-- Right Hand -->
   <xacro:macro name="shadowhand_motor">
