Commit message: unified srh_motor.launch and srh_muscle.launch in the same file -> renamed forearm_muscle and forearm_motor to forearm only

File: hand/xacro/forearm/forearm_motor.urdf.xacro (robot description, xacro)
@@ -1,6 +1,6 @@
 <robot xmlns:xacro="http://ros.org/wiki/xacro">
   <property name="M_PI" value="3.1415926535897931" />
-  <xacro:macro name="forearm_motor">
-    <link name="forearm_motor">
+  <xacro:macro name="forearm">
+    <link name="forearm">
       <inertial>
 	<origin xyz="0 0 0.09" rpy="0 0 0"/>
@@ -22,5 +22,5 @@
       </collision>
     </link>
-    <gazebo reference="forearm_motor">
+    <gazebo reference="forearm">
       <material>Gazebo/Grey</material>
       <selfCollide>true</selfCollide>

File: hand/xacro/forearm/forearm_muscle.urdf.xacro (robot description, xacro)
@@ -1,6 +1,6 @@
 <robot xmlns:xacro="http://ros.org/wiki/xacro">
   <property name="M_PI" value="3.1415926535897931" />
-  <xacro:macro name="forearm_muscle">
-    <link name="forearm_muscle">
+  <xacro:macro name="forearm">
+    <link name="forearm">
       <inertial>
 	<origin xyz="0 0 0.175" />
@@ -11,5 +11,5 @@
 	<origin xyz="0 0 0" rpy="${M_PI} 0 0" />
 	<geometry name="shadow_forearm_geom">
-	  <mesh filename="package://sr_hand/model/meshes/forearm_muscle.mesh" scale="0.016 0.016 0.016" />
+	  <mesh filename="package://sr_description/hand/model/forearm_muscle.mesh" scale="0.016 0.016 0.016" />
 	</geometry>
 	<material name="Grey" />
@@ -22,5 +22,5 @@
       </collision>
     </link>
-    <gazebo reference="forearm_muscle">
+    <gazebo reference="forearm">
       <material>Gazebo/Grey</material>
       <selfCollide>true</selfCollide>

File: hand/xacro/full_hand_motor.urdf.xacro (robot description, xacro)
@@ -11,7 +11,7 @@
   <!-- Right Hand -->
   <xacro:macro name="shadowhand_motor">
-    <xacro:forearm_motor>
-    </xacro:forearm_motor>
-    <xacro:wrist parent="forearm_motor">
+    <xacro:forearm>
+    </xacro:forearm>
+    <xacro:wrist parent="forearm">
       <origin xyz="0 -0.010 0.213" rpy="0 0 0" />
     </xacro:wrist>
@@ -37,7 +37,7 @@
   <!-- Left Hand -->
   <xacro:macro name="shadowhand_left_motor">
-    <xacro:forearm_motor>
-    </xacro:forearm_motor>
-    <xacro:wrist_left parent="forearm_motor">
+    <xacro:forearm>
+    </xacro:forearm>
+    <xacro:wrist_left parent="forearm">
       <origin xyz="0 -0.010 0.213" rpy="0 0 0" />
     </xacro:wrist_left>

File: hand/xacro/full_hand_motor_biotac.urdf.xacro (robot description, xacro)
@@ -11,7 +11,7 @@
   <!-- Right Hand -->
   <xacro:macro name="shadowhand_motor">
-    <xacro:forearm_motor>
-    </xacro:forearm_motor>
-    <xacro:wrist parent="forearm_motor">
+    <xacro:forearm>
+    </xacro:forearm>
+    <xacro:wrist parent="forearm">
       <origin xyz="0 -0.010 0.213" rpy="0 0 0" />
     </xacro:wrist>
@@ -37,7 +37,7 @@
   <!-- Left Hand -->
   <xacro:macro name="shadowhand_left_motor">
-    <xacro:forearm_motor>
-    </xacro:forearm_motor>
-    <xacro:wrist_left parent="forearm_motor">
+    <xacro:forearm>
+    </xacro:forearm>
+    <xacro:wrist_left parent="forearm">
       <origin xyz="0 -0.010 0.213" rpy="0 0 0" />
     </xacro:wrist_left>

File: hand/xacro/full_hand_motor_ellipsoid.urdf.xacro (robot description, xacro)
@@ -10,7 +10,7 @@
   <include filename="$(find sr_description)/hand/xacro/thumb/thumb_ellipsoid.urdf.xacro" />
   <xacro:macro name="shadowhand_motor">
-    <xacro:forearm_motor>
-    </xacro:forearm_motor>
-    <xacro:wrist parent="forearm_motor">
+    <xacro:forearm>
+    </xacro:forearm>
+    <xacro:wrist parent="forearm">
       <origin xyz="0 -0.010 0.213" rpy="0 0 0" />
     </xacro:wrist>

File: hand/xacro/full_hand_muscle.urdf.xacro (robot description, xacro)
@@ -11,7 +11,7 @@
   <!-- Right Hand -->
   <xacro:macro name="shadowhand_muscle">
-    <xacro:forearm_muscle>
-    </xacro:forearm_muscle>
-    <xacro:wrist parent="forearm_muscle">
+    <xacro:forearm>
+    </xacro:forearm>
+    <xacro:wrist parent="forearm">
       <origin xyz="0 0 0.396" rpy="0 0 0" />
     </xacro:wrist>
@@ -37,7 +37,7 @@
   <!-- Left Hand -->
   <xacro:macro name="shadowhand_left_muscle">
-    <xacro:forearm_muscle>
-    </xacro:forearm_muscle>
-    <xacro:wrist_left parent="forearm_muscle">
+    <xacro:forearm>
+    </xacro:forearm>
+    <xacro:wrist_left parent="forearm">
       <origin xyz="0 0 0.396" rpy="0 0 0" />
     </xacro:wrist_left>

File: hand/xacro/one_finger_unit_motor.urdf.xacro (robot description, xacro)
@@ -6,6 +6,6 @@
   <include filename="$(find sr_description)/hand/xacro/finger/classic_finger.urdf.xacro" />
   <xacro:macro name="shadowhand_motor">
-    <xacro:forearm_motor>
-    </xacro:forearm_motor>
+    <xacro:forearm>
+    </xacro:forearm>
     <link name="dummy_palm">
       <inertial>
@@ -30,9 +30,9 @@
     </link>
     <joint name="forearm_to_dummy" type="fixed">
-      <parent link="forearm_motor"/>
+      <parent link="forearm"/>
       <child link="dummy_palm"/>
       <origin xyz="0.011 0.010 0.22" rpy="0 0 3.14"/>
     </joint>
-    <!-- mfknuckle is at [0.011 -0.01 0.346] from the bottom of forearm_motor -->
+    <!-- mfknuckle is at [0.011 -0.01 0.346] from the bottom of forearm -->
     <xacro:finger link_prefix="mf" joint_prefix="MF" parent="dummy_palm">
       <origin xyz="0.0 0 0.116" rpy="0 0 0" />

File: hand/xacro/three_finger_unit_motor.urdf.xacro (robot description, xacro)
@@ -10,7 +10,7 @@
   <!-- Right Hand -->
   <xacro:macro name="shadowhand_motor">
-    <xacro:forearm_motor>
-    </xacro:forearm_motor>
-    <xacro:wrist parent="forearm_motor">
+    <xacro:forearm>
+    </xacro:forearm>
+    <xacro:wrist parent="forearm">
       <origin xyz="0 -0.010 0.213" rpy="0 0 0" />
     </xacro:wrist>
@@ -30,7 +30,7 @@
   <!-- Left Hand -->
   <xacro:macro name="shadowhand_left_motor">
-    <xacro:forearm_motor>
-    </xacro:forearm_motor>
-    <xacro:wrist_left parent="forearm_motor">
+    <xacro:forearm>
+    </xacro:forearm>
+    <xacro:wrist_left parent="forearm">
       <origin xyz="0 -0.010 0.213" rpy="0 0 0" />
     </xacro:wrist_left>

File: robots/arm_and_hand_motor.urdf.xacro (robot description, xacro)
@@ -15,5 +15,5 @@
   <joint name="arm_link" type="fixed">
     <parent link="shadowarm_handsupport_motor"/>
-    <child link="forearm_motor"/>
+    <child link="forearm"/>
     <origin xyz="0 0 0" rpy="0 0 ${2.35619449}" />
   </joint>

File: robots/arm_and_hand_motor_ellipsoid.urdf.xacro (robot description, xacro)
@@ -15,5 +15,5 @@
   <joint name="arm_link" type="fixed">
     <parent link="shadowarm_handsupport_motor"/>
-    <child link="forearm_motor"/>
+    <child link="forearm"/>
     <origin xyz="0 0 0" rpy="0 0 ${2.35619449}" />
   </joint>

File: robots/arm_and_hand_motor_three_finger.urdf.xacro (robot description, xacro)
@@ -15,5 +15,5 @@
   <joint name="arm_link" type="fixed">
     <parent link="shadowarm_handsupport_motor"/>
-    <child link="forearm_motor"/>
+    <child link="forearm"/>
     <origin xyz="0 0 0" rpy="0 0 ${2.35619449}" />
   </joint>

File: robots/arm_and_hand_muscle.urdf.xacro (robot description, xacro)
@@ -15,5 +15,5 @@
   <joint name="arm_link" type="fixed">
     <parent link="shadowarm_handsupport_muscle"/>
-    <child link="forearm_muscle"/>
+    <child link="forearm"/>
     <origin xyz="0 0 0" rpy="0 0 ${M_PI}" />
   </joint>

File: robots/arm_and_sr_one_finger_motor.urdf.xacro (robot description, xacro)
@@ -15,5 +15,5 @@
   <joint name="arm_link" type="revolute">
     <parent link="shadowarm_handsupport_motor"/>
-    <child link="forearm_motor"/>
+    <child link="forearm"/>
     <origin xyz="0 0 0" rpy="0 0 ${M_PI}" />
     <axis xyz="0 -1 0" />

File: robots/desk_arm_and_hand_motor.urdf.xacro (robot description, xacro)
@@ -15,5 +15,5 @@
   <joint name="arm_link" type="revolute">
     <parent link="shadowarm_handsupport_motor"/>
-    <child link="forearm_motor"/>
+    <child link="forearm"/>
     <origin xyz="0 0 0" rpy="0 0 ${M_PI}" />
     <axis xyz="0 -1 0" />
