Commit message: biotac model

File: hand/xacro/finger/classic_finger_biotac.urdf.xacro (robot description, xacro)
@@ -2,6 +2,5 @@
   <include filename="$(find sr_description)/hand/xacro/finger/knuckle/knuckle.urdf.xacro" />
   <include filename="$(find sr_description)/hand/xacro/finger/proximal/proximal.urdf.xacro" />
-  <include filename="$(find sr_description)/hand/xacro/finger/middle/middle.urdf.xacro" />
-  <include filename="$(find sr_description)/hand/xacro/finger/distal/distal_biotac.urdf.xacro" />
+  <include filename="$(find sr_description)/hand/xacro/finger/biotac/biotac.urdf.xacro" />
   <xacro:macro name="finger" params="link_prefix joint_prefix parent *origin *axis">
     <xacro:knuckle link_prefix="${link_prefix}" joint_prefix="${joint_prefix}" parent="${parent}" >
@@ -11,8 +10,6 @@
     <xacro:proximal link_prefix="${link_prefix}" joint_prefix="${joint_prefix}" parent="${link_prefix}knuckle" >
     </xacro:proximal>
-    <xacro:middle link_prefix="${link_prefix}" joint_prefix="${joint_prefix}" parent="${link_prefix}proximal" >
-    </xacro:middle>
-    <xacro:distal link_prefix="${link_prefix}" joint_prefix="${joint_prefix}" parent="${link_prefix}middle" >
-    </xacro:distal>
+    <xacro:biotac_middle link_prefix="${link_prefix}" joint_prefix="${joint_prefix}" parent="${link_prefix}proximal">
+    </xacro:biotac_middle>
   </xacro:macro>
 </robot>

File: hand/xacro/finger/little_finger_biotac.urdf.xacro (robot description, xacro)
@@ -6,9 +6,8 @@
        xmlns:body="http://playerstage.sourceforge.net/gazebo/xmlschema/#body"
        xmlns:geom="http://playerstage.sourceforge.net/gazebo/xmlschema/#geom">
+  <include filename="$(find sr_description)/hand/xacro/finger/lfmetacarpal/lfmetacarpal.urdf.xacro" />
   <include filename="$(find sr_description)/hand/xacro/finger/knuckle/knuckle.urdf.xacro" />
   <include filename="$(find sr_description)/hand/xacro/finger/proximal/proximal.urdf.xacro" />
-  <include filename="$(find sr_description)/hand/xacro/finger/middle/middle.urdf.xacro" />
-  <include filename="$(find sr_description)/hand/xacro/finger/distal/distal_biotac.urdf.xacro" />
-  <include filename="$(find sr_description)/hand/xacro/finger/lfmetacarpal/lfmetacarpal.urdf.xacro" />
+  <include filename="$(find sr_description)/hand/xacro/finger/biotac/biotac.urdf.xacro" />
   <!-- Right Handed -->
   <xacro:macro name="little_finger" params="link_prefix joint_prefix parent">
@@ -76,8 +75,6 @@
     <xacro:proximal link_prefix="${link_prefix}" joint_prefix="${joint_prefix}" parent="${link_prefix}knuckle">
     </xacro:proximal>
-    <xacro:middle link_prefix="${link_prefix}" joint_prefix="${joint_prefix}" parent="${link_prefix}proximal">
-    </xacro:middle>
-    <xacro:distal link_prefix="${link_prefix}" joint_prefix="${joint_prefix}" parent="${link_prefix}middle">
-    </xacro:distal>
+    <xacro:biotac_middle link_prefix="${link_prefix}" joint_prefix="${joint_prefix}" parent="${link_prefix}proximal">
+    </xacro:biotac_middle>
   </xacro:macro>
 </robot>

File: hand/xacro/forearm/forearm_muscle.urdf.xacro (robot description, xacro)
@@ -4,12 +4,12 @@
     <link name="forearm">
       <inertial>
-	<origin xyz="0 0 0.175" />
+	<origin xyz="0 0 0" />
 	<mass value="3.0" />
 	<inertia  ixx="0.00735" ixy="0.0"  ixz="0.0"  iyy="0.00735"  iyz="0.0"  izz="0.0343" />
       </inertial>
       <visual>
-	<origin xyz="0 0 0" rpy="${M_PI} 0 0" />
+	<origin xyz="0 0 0" rpy="0 0 0" />
 	<geometry name="shadow_forearm_geom">
-	  <mesh filename="package://sr_description/hand/model/forearm_muscle.mesh" scale="0.016 0.016 0.016" />
+	  <mesh filename="package://sr_description/hand/model/forearm_muscle.dae" scale="0.016 0.016 0.016" />
 	</geometry>
 	<material name="Grey" />

File: hand/xacro/thumb/thumb_biotac.urdf.xacro (robot description, xacro)
@@ -3,6 +3,5 @@
   <include filename="$(find sr_description)/hand/xacro/thumb/thproximal.urdf.xacro" />
   <include filename="$(find sr_description)/hand/xacro/thumb/thhub.urdf.xacro" />
-  <include filename="$(find sr_description)/hand/xacro/thumb/thmiddle.urdf.xacro" />
-  <include filename="$(find sr_description)/hand/xacro/thumb/thdistal_biotac.urdf.xacro" />
+  <include filename="$(find sr_description)/hand/xacro/thumb/thbiotac.urdf.xacro" />
   <!-- Right Hand -->
   <xacro:macro name="thumb" params="parent">
@@ -26,8 +25,6 @@
     <xacro:thhub parent="thproximal">
     </xacro:thhub>
-    <xacro:thmiddle parent="thhub">
-    </xacro:thmiddle>
-    <xacro:thdistal parent="thmiddle">
-    </xacro:thdistal>
+    <xacro:thbiotac parent="thhub"> <!-- fnh: note: also includes thtip link -->
+    </xacro:thbiotac>
   </xacro:macro>
 </robot>

File: materials.urdf.xacro (robot description, xacro)
@@ -6,4 +6,7 @@
   <material name="Green">
     <color rgba="0.0 0.8 0.0 1.0"/>
+  </material>
+  <material name="BiotacGreen">
+    <color rgba="0.31 0.85 0.42 1.0"/>
   </material>
   <material name="Grey">

File: robots/shadowhand_motor_biotac.urdf.xacro (robot description, xacro)
@@ -7,4 +7,7 @@
   <include filename="$(find sr_description)/hand/xacro/full_hand_motor_biotac.urdf.xacro" />
   <include filename="$(find sr_description)/other/xacro/gazebo/gazebo.urdf.xacro" />
+<!-- C6 hand with BioTAC sensor
+  (C) 2012 fnh, hendrich@informatik.uni-hamburg.de
+-->
   <xacro:shadowhand_motor>
   </xacro:shadowhand_motor>
