Commit message: Fixed full_hand_motor_biotac

File: hand/xacro/finger/little_finger_biotac.urdf.xacro (robot description, xacro)
@@ -7,75 +7,20 @@
        xmlns:geom="http://playerstage.sourceforge.net/gazebo/xmlschema/#geom">
   <include filename="$(find sr_description)/hand/xacro/finger/lfmetacarpal/lfmetacarpal.urdf.xacro" />
-  <include filename="$(find sr_description)/hand/xacro/finger/knuckle/knuckle.urdf.xacro" />
-  <include filename="$(find sr_description)/hand/xacro/finger/proximal/proximal.urdf.xacro" />
-  <include filename="$(find sr_description)/hand/xacro/finger/biotac/biotac.urdf.xacro" />
+  <include filename="$(find sr_description)/hand/xacro/finger/classic_finger_biotac.urdf.xacro" />
   <!-- Right Handed -->
   <xacro:macro name="little_finger" params="link_prefix joint_prefix parent">
     <xacro:lfmetacarpal parent="${parent}" />
-    <xacro:little_finger_common link_prefix="${link_prefix}" joint_prefix="${joint_prefix}" parent="${parent}" />
+    <xacro:finger_biotac link_prefix="${link_prefix}" joint_prefix="${joint_prefix}" parent="lfmetacarpal">
+      <origin xyz="0 0 0.06579" rpy="0 0 0" />
+      <axis xyz="0 1 0" />
+    </xacro:finger_biotac>
   </xacro:macro>
   <!-- Left Handed -->
   <xacro:macro name="little_finger_left" params="link_prefix joint_prefix parent">
     <xacro:lfmetacarpal_left parent="${parent}" />
-    <xacro:little_finger_common link_prefix="${link_prefix}" joint_prefix="${joint_prefix}" parent="${parent}" />
-  </xacro:macro>
-  <!-- Common bits for left handed and right handed little fingers. For use in
-  macros above to generate little_finger and little_finger_left.
-  DO NOT use out side of here ie treat as a private macro -->
-  <xacro:macro name="little_finger_common" params="link_prefix joint_prefix parent">
-    <link name="lfknuckle">
-      <inertial>
-        <origin xyz="0 0 0.0" rpy="0 0 0" />
-        <mass value="0.008" />
-        <inertia ixx="0.1" ixy="0.0" ixz="0.0" iyy="0.1" iyz="0.0" izz="0.1" />
-      </inertial>
-      <visual>
-        <origin xyz="0 0 0" rpy="0 0 0" />
-        <geometry name="lfknuckle_visual">
-          <mesh filename="package://sr_description/hand/model/knuckle.dae" scale="0.001 0.001 0.001" />
-        </geometry>
-        <material name="LightGrey" />
-      </visual>
-      <collision>
-        <origin xyz="0 0 0" rpy="0 0 0" />
-        <geometry name="lfknuckle_collision_geom">
-          <box size="0.005 0.005 0.005" />
-        </geometry>
-      </collision>
-    </link>
-    <gazebo reference="lfknuckle">
-      <sensor type="contact" name="lfknuckle_contact_sensor">
-        <update_rate>100.0</update_rate>
-        <contact>
-          <collision>lfknuckle_collision_geom</collision>
-        </contact>
-        <plugin name="lfknuckle_gazebo_ros_bumper_controller" filename="libgazebo_ros_bumper.so">
-          <alwaysOn>true</alwaysOn>
-          <frameName>lfknuckle</frameName>
-          <updateRate>100.0</updateRate>
-          <bumperTopicName>lfknuckle_bumper</bumperTopicName>
-        </plugin>
-      </sensor>
-      <material>Gazebo/Grey</material>
-    </gazebo>
-    <joint name="LFJ4" type="revolute">
-      <parent link="lfmetacarpal" />
-      <child link="lfknuckle" />
+    <xacro:finger_biotac link_prefix="${link_prefix}" joint_prefix="${joint_prefix}" parent="lfmetacarpal">
       <origin xyz="0 0 0.06579" rpy="0 0 0" />
-      <axis xyz="0 1 0" />
-      <limit lower="-0.3491" upper="0.3491" effort="10" velocity="1.0" />
-      <dynamics damping="50.5" />
-    </joint>
-    <transmission type="sr_mechanism_model/SimpleTransmission" name="lfknuckle_transmission">
-      <actuator name="LFJ4" />
-      <joint name="LFJ4" />
-      <mechanicalReduction>1</mechanicalReduction>
-      <motorTorqueConstant>1</motorTorqueConstant>
-      <pulsesPerRevolution>90000</pulsesPerRevolution>
-    </transmission>
-    <xacro:proximal link_prefix="${link_prefix}" joint_prefix="${joint_prefix}" parent="${link_prefix}knuckle">
-    </xacro:proximal>
-    <xacro:biotac_middle link_prefix="${link_prefix}" joint_prefix="${joint_prefix}" parent="${link_prefix}proximal">
-    </xacro:biotac_middle>
+      <axis xyz="0 -1 0" />
+    </xacro:finger_biotac>
   </xacro:macro>
 </robot>

File: hand/xacro/full_hand_motor_3_biotacs.urdf.xacro (robot description, xacro)
@@ -7,5 +7,6 @@
   <include filename="$(find sr_description)/hand/xacro/palm/palm.urdf.xacro" />
   <include filename="$(find sr_description)/hand/xacro/finger/classic_finger_biotac.urdf.xacro" />
-  <include filename="$(find sr_description)/hand/xacro/finger/little_finger_biotac.urdf.xacro" />
+  <include filename="$(find sr_description)/hand/xacro/finger/classic_finger.urdf.xacro" />
+  <include filename="$(find sr_description)/hand/xacro/finger/little_finger.urdf.xacro" />
   <include filename="$(find sr_description)/hand/xacro/thumb/thumb_biotac.urdf.xacro" />
   <!-- Right Hand -->
@@ -26,8 +27,8 @@
       <axis xyz="0 -1 0" />
     </xacro:finger_biotac>
-    <xacro:finger_biotac link_prefix="rf" joint_prefix="RF" parent="palm">
+    <xacro:finger link_prefix="rf" joint_prefix="RF" parent="palm">
       <origin xyz="-0.011 0 0.095" rpy="0 0 0" />
       <axis xyz="0 1 0" />
-    </xacro:finger_biotac>
+    </xacro:finger>
     <xacro:little_finger link_prefix="lf" joint_prefix="LF" parent="palm">
     </xacro:little_finger>
@@ -44,16 +45,16 @@
     <xacro:palm_left parent="wrist">
     </xacro:palm_left>
-    <xacro:finger_biotac link_prefix="ff" joint_prefix="FF" parent="palm">
+    <xacro:finger link_prefix="ff" joint_prefix="FF" parent="palm">
       <origin xyz="-0.033 0 0.095" rpy="0 0 0" />
       <axis xyz="0 -1 0" />
-    </xacro:finger_biotac>
-    <xacro:finger_biotac link_prefix="mf" joint_prefix="MF" parent="palm">
+    </xacro:finger>
+    <xacro:finger link_prefix="mf" joint_prefix="MF" parent="palm">
       <origin xyz="-0.011 0 0.099" rpy="0 0 0" />
       <axis xyz="0 -1 0" />
-    </xacro:finger_biotac>
-    <xacro:finger_biotac link_prefix="rf" joint_prefix="RF" parent="palm">
+    </xacro:finger>
+    <xacro:finger link_prefix="rf" joint_prefix="RF" parent="palm">
       <origin xyz="0.011 0 0.095" rpy="0 0 0" />
       <axis xyz="0 1 0" />
-    </xacro:finger_biotac>
+    </xacro:finger>
     <xacro:little_finger_left link_prefix="lf" joint_prefix="LF" parent="palm">
     </xacro:little_finger_left>
