Commit message: better mesh, fixed forearm length for muscle hand: 409.6 instead of 396

File: hand/xacro/full_hand_muscle.urdf.xacro (robot description, xacro)
@@ -14,5 +14,5 @@
     </xacro:forearm>
     <xacro:wrist parent="forearm">
-      <origin xyz="0 0 0.396" rpy="0 0 0" />
+      <origin xyz="0 0 0.4096" rpy="0 0 0" />
     </xacro:wrist>
     <xacro:palm parent="wrist">

File: hand/xacro/full_hand_muscle_biotac.urdf.xacro (robot description, xacro)
@@ -14,5 +14,5 @@
     </xacro:forearm>
     <xacro:wrist parent="forearm">
-      <origin xyz="0 0.0 0.396" rpy="0 0 0" />
+      <origin xyz="0 0.0 0.4096" rpy="0 0 0" />
     </xacro:wrist>
     <xacro:palm parent="wrist">

Commit message: added a disk below the muscle hand when it's on its own to reflect real hand

File: hand/xacro/full_hand_muscle.urdf.xacro (robot description, xacro)
@@ -40,5 +40,5 @@
     </xacro:forearm>
     <xacro:wrist_left parent="forearm">
-      <origin xyz="0 0 0.396" rpy="0 0 0" />
+      <origin xyz="0 0 0.4096" rpy="0 0 0" />
     </xacro:wrist_left>
     <xacro:palm_left parent="wrist">

File: hand/xacro/full_hand_muscle_biotac.urdf.xacro (robot description, xacro)
@@ -40,5 +40,5 @@
     </xacro:forearm>
     <xacro:wrist_left parent="forearm">
-      <origin xyz="0 0 0.396" rpy="0 0 0" />
+      <origin xyz="0 0 0.4096" rpy="0 0 0" />
     </xacro:wrist_left>
     <xacro:palm_left parent="wrist">
