Commit message: Changes in joint ranges to match the real limits

File: hand/xacro/thumb/thbiotac.urdf.xacro (robot description, xacro)
@@ -55,5 +55,5 @@
       <origin xyz="0 0 0.01" rpy="0 0 0" /> <!-- FIXME: z offset is too large -->
       <axis xyz="0 -1 0" />
-      <limit lower="-0.5237" upper="0.5237" effort="10"
+      <limit lower="-0.6981" upper="0.6981" effort="10"
       velocity="1.0" />
       <dynamics damping="50.5"/>
