Commit message: Changes in joint ranges to match the real limits. Ported this commit from development as a patch, as we can't merge both branches at the moment (no time).

File: hand/xacro/finger/knuckle/knuckle.urdf.xacro (robot description, xacro)
@@ -51,5 +51,5 @@
       <insert_block name="origin" />
       <insert_block name="axis"/>
-      <limit lower="-0.43633231299858238" upper="0.43633231299858238"
+      <limit lower="-0.3491" upper="0.3491"
       effort="10" velocity="1.0"/>
       <dynamics damping="50.5"/>

File: hand/xacro/finger/little_finger_biotac.urdf.xacro (robot description, xacro)
@@ -64,5 +64,5 @@
       <origin xyz="0 0 0.06579" rpy="0 0 0" />
       <axis xyz="0 1 0" />
-      <limit lower="-0.43633231299858238" upper="0.43633231299858238" effort="10" velocity="1.0" />
+      <limit lower="-0.3491" upper="0.3491" effort="10" velocity="1.0" />
       <dynamics damping="50.5" />
     </joint>

File: hand/xacro/finger/little_finger_ellipsoid.urdf.xacro (robot description, xacro)
@@ -55,5 +55,5 @@
       <origin xyz="0 0 0.06579" rpy="0 0 0" />
       <axis xyz="0 1 0" />
-      <limit lower="-0.43633231299858238" upper="0.43633231299858238"
+      <limit lower="-0.3491" upper="0.3491"
       effort="10" velocity="1.0"/>
       <dynamics damping="50.5"/>

File: hand/xacro/palm/palm.urdf.xacro (robot description, xacro)
@@ -58,5 +58,5 @@
       <origin xyz="0 0 0.034" rpy="0 0 0" />
       <axis xyz="1 0 0" />
-      <limit lower="-0.78539816339744828" upper="0.6108652381980153"
+      <limit lower="-0.7854" upper="0.5236"
       effort="5" velocity="1.0"/>
       <dynamics damping="100.5"/>

File: hand/xacro/thumb/thbiotac.urdf.xacro (robot description, xacro)
@@ -56,5 +56,5 @@
       <origin xyz="0 0 0.01" rpy="0 0 0" /> <!-- FIXME: z offset is too large -->
       <axis xyz="0 -1 0" />
-      <limit lower="-0.5237" upper="0.5237" effort="10"
+      <limit lower="-0.6981" upper="0.6981" effort="10"
       velocity="1.0" />
       <dynamics damping="50.5"/>

File: hand/xacro/thumb/thmiddle.urdf.xacro (robot description, xacro)
@@ -51,5 +51,5 @@
       <origin xyz="0 0 0" rpy="0 0 0" />
       <axis xyz="0 -1 0" />
-      <limit lower="-0.5237" upper="0.5237" effort="10"
+      <limit lower="-0.6981" upper="0.6981" effort="10"
       velocity="1.0" />
       <dynamics damping="50.5"/>
