Commit message: Correction of the lfmetacarpal range. It was 40 deg, it must be 45.

File: hand/xacro/finger/lfmetacarpal/lfmetacarpal.urdf.xacro (robot description, xacro)
@@ -58,5 +58,5 @@
       <origin xyz="${reflect*-0.033} 0 0.02071" rpy="0 0 0" />
       <axis xyz="0.573576436 0 ${reflect*0.819152044}" />
-      <limit lower="0" upper="0.69813170079773179" effort="10"
+      <limit lower="0" upper="0.7854" effort="10"
       velocity="1.0" />
       <dynamics damping="50.5"/>
