Commit message: higher effort limits for the arm - now moving

File: arm/xacro/lower_arm/shadowarm_lowerarm.urdf.xacro (robot description, xacro)
@@ -32,5 +32,5 @@
       <axis xyz="0 -1 0" />
       <limit lower="0.52" upper="2.09439510239"
-      effort="10" velocity="1.0"/>
+      effort="100" velocity="1.0"/>
       <dynamics damping="50.5"/>
     </joint>

File: arm/xacro/trunk/shadowarm_trunk.urdf.xacro (robot description, xacro)
@@ -32,5 +32,5 @@
       <axis xyz="0 0 1" />
       <limit lower="-${M_PI/4}" upper="${M_PI/2}"
-      effort="10" velocity="1.0"/>
+      effort="100" velocity="1.0"/>
       <dynamics damping="200.5"/>
     </joint>

File: arm/xacro/upper_arm/shadowarm_upperarm.urdf.xacro (robot description, xacro)
@@ -31,5 +31,5 @@
       <origin xyz="0 -0.134 0.5305" rpy="0 -${M_PI} 0.0" /> <!-- yaw=-0.026 -->
       <axis xyz="0 -1 0" />
-      <limit lower="0" upper="${M_PI/2}" effort="10" velocity="1.0"/>
+      <limit lower="0" upper="${M_PI/2}" effort="100" velocity="1.0"/>
       <dynamics damping="50.5"/>
     </joint>
