Commit message: modified paths, added test for xacro files

File: arm/xacro/base/shadowarm_base.urdf.xacro (robot description, xacro)
@@ -2,5 +2,4 @@
 <property name="M_PI" value="3.1415926535897931" />
 <xacro:macro name="shadowarm_base">
-  <link name="world" />
   <link name="shadowarm_base">
     <inertial>
@@ -12,5 +11,5 @@
       <origin xyz="0 0 0" rpy="0 0 0"/>
       <geometry name="shadowarm_base_visual">
-        <mesh filename="package://sr_hand/model/meshes/arm/arm_base.dae" scale="0.001 0.001 0.001" />
+        <mesh filename="package://sr_description/arm/model/arm_base.dae" scale="0.001 0.001 0.001" />
       </geometry>
       <material name="LightGrey" />

File: hand/xacro/finger/classic_finger.urdf.xacro (robot description, xacro)
@@ -1,7 +1,7 @@
 <robot xmlns:xacro="http://www.ros.org/wiki/xacro">
-  <include filename="$(find sr_description/hand/xacro/finger/knuckle/knuckle.urdf.xacro" />
-  <include filename="$(find sr_description/hand/xacro/finger/proximal/proximal.urdf.xacro" />
-  <include filename="$(find sr_description/hand/xacro/finger/middle/middle.urdf.xacro" />
-  <include filename="$(find sr_description/hand/xacro/finger/distal/distal.urdf.xacro" />
+  <include filename="$(find sr_description)/hand/xacro/finger/knuckle/knuckle.urdf.xacro" />
+  <include filename="$(find sr_description)/hand/xacro/finger/proximal/proximal.urdf.xacro" />
+  <include filename="$(find sr_description)/hand/xacro/finger/middle/middle.urdf.xacro" />
+  <include filename="$(find sr_description)/hand/xacro/finger/distal/distal.urdf.xacro" />
   <xacro:macro name="finger" params="link_prefix joint_prefix parent *origin *axis">
     <xacro:knuckle link_prefix="${link_prefix}" joint_prefix="${joint_prefix}" parent="${parent}" >

File: hand/xacro/finger/classic_finger_biotac.urdf.xacro (robot description, xacro)
@@ -1,7 +1,7 @@
 <robot xmlns:xacro="http://www.ros.org/wiki/xacro">
-  <include filename="$(find sr_description/hand/xacro/finger/knuckle/knuckle.urdf.xacro" />
-  <include filename="$(find sr_description/hand/xacro/finger/proximal/proximal.urdf.xacro" />
-  <include filename="$(find sr_description/hand/xacro/finger/middle/middle.urdf.xacro" />
-  <include filename="$(find sr_description/hand/xacro/finger/distal/distal_biotac.urdf.xacro" />
+  <include filename="$(find sr_description)/hand/xacro/finger/knuckle/knuckle.urdf.xacro" />
+  <include filename="$(find sr_description)/hand/xacro/finger/proximal/proximal.urdf.xacro" />
+  <include filename="$(find sr_description)/hand/xacro/finger/middle/middle.urdf.xacro" />
+  <include filename="$(find sr_description)/hand/xacro/finger/distal/distal_biotac.urdf.xacro" />
   <xacro:macro name="finger" params="link_prefix joint_prefix parent *origin *axis">
     <xacro:knuckle link_prefix="${link_prefix}" joint_prefix="${joint_prefix}" parent="${parent}" >

File: hand/xacro/finger/classic_finger_ellipsoid.urdf.xacro (robot description, xacro)
@@ -1,7 +1,7 @@
 <robot xmlns:xacro="http://www.ros.org/wiki/xacro">
-  <include filename="$(find sr_description/hand/xacro/finger/knuckle/knuckle.urdf.xacro" />
-  <include filename="$(find sr_description/hand/xacro/finger/proximal/proximal.urdf.xacro" />
-  <include filename="$(find sr_description/hand/xacro/finger/middle/middle.urdf.xacro" />
-  <include filename="$(find sr_description/hand/xacro/finger/distal/distal_ellipsoid.urdf.xacro" />
+  <include filename="$(find sr_description)/hand/xacro/finger/knuckle/knuckle.urdf.xacro" />
+  <include filename="$(find sr_description)/hand/xacro/finger/proximal/proximal.urdf.xacro" />
+  <include filename="$(find sr_description)/hand/xacro/finger/middle/middle.urdf.xacro" />
+  <include filename="$(find sr_description)/hand/xacro/finger/distal/distal_ellipsoid.urdf.xacro" />
   <xacro:macro name="finger" params="link_prefix joint_prefix parent *origin *axis">
     <xacro:knuckle link_prefix="${link_prefix}" joint_prefix="${joint_prefix}" parent="${parent}" >

File: hand/xacro/finger/distal/distal.urdf.xacro (robot description, xacro)
@@ -6,5 +6,5 @@
        xmlns:body="http://playerstage.sourceforge.net/gazebo/xmlschema/#body"
        xmlns:geom="http://playerstage.sourceforge.net/gazebo/xmlschema/#geom">
-  <include filename="$(find sr_description/hand/xacro/finger/distal/distal.transmission.xacro" />
+  <include filename="$(find sr_description)/hand/xacro/finger/distal/distal.transmission.xacro" />
   <xacro:macro name="distal" params="link_prefix joint_prefix parent">
     <link name="${link_prefix}distal">

File: hand/xacro/finger/distal/distal_biotac.urdf.xacro (robot description, xacro)
@@ -6,5 +6,5 @@
        xmlns:body="http://playerstage.sourceforge.net/gazebo/xmlschema/#body"
        xmlns:geom="http://playerstage.sourceforge.net/gazebo/xmlschema/#geom">
-  <include filename="$(find sr_description/hand/xacro/finger/distal/distal.transmission.xacro" />
+  <include filename="$(find sr_description)/hand/xacro/finger/distal/distal.transmission.xacro" />
   <xacro:macro name="distal" params="link_prefix joint_prefix parent">
     <link name="${link_prefix}distal">

File: hand/xacro/finger/distal/distal_ellipsoid.urdf.xacro (robot description, xacro)
@@ -6,5 +6,5 @@
        xmlns:body="http://playerstage.sourceforge.net/gazebo/xmlschema/#body"
        xmlns:geom="http://playerstage.sourceforge.net/gazebo/xmlschema/#geom">
-  <include filename="$(find sr_description/hand/xacro/finger/distal/distal.transmission.xacro" />
+  <include filename="$(find sr_description)/hand/xacro/finger/distal/distal.transmission.xacro" />
   <xacro:macro name="distal" params="link_prefix joint_prefix parent">
     <link name="${link_prefix}distal">

File: hand/xacro/finger/knuckle/knuckle.urdf.xacro (robot description, xacro)
@@ -6,5 +6,5 @@
        xmlns:body="http://playerstage.sourceforge.net/gazebo/xmlschema/#body"
        xmlns:geom="http://playerstage.sourceforge.net/gazebo/xmlschema/#geom">
-  <include filename="$(find sr_description/hand/xacro/finger/knuckle/knuckle.transmission.xacro" />
+  <include filename="$(find sr_description)/hand/xacro/finger/knuckle/knuckle.transmission.xacro" />
   <xacro:macro name="knuckle" params="link_prefix joint_prefix parent *origin">
     <link name="${link_prefix}knuckle">

File: hand/xacro/finger/lfmetacarpal/lfmetacarpal.urdf.xacro (robot description, xacro)
@@ -6,5 +6,5 @@
        xmlns:body="http://playerstage.sourceforge.net/gazebo/xmlschema/#body"
        xmlns:geom="http://playerstage.sourceforge.net/gazebo/xmlschema/#geom">
-  <include filename="$(find sr_description/hand/xacro/finger/lfmetacarpal/lfmetacarpal.transmission.xacro" />
+  <include filename="$(find sr_description)/hand/xacro/finger/lfmetacarpal/lfmetacarpal.transmission.xacro" />
   <!-- Right Handed -->
   <xacro:macro name="lfmetacarpal" params="parent">

File: hand/xacro/finger/little_finger.urdf.xacro (robot description, xacro)
@@ -6,9 +6,9 @@
        xmlns:body="http://playerstage.sourceforge.net/gazebo/xmlschema/#body"
        xmlns:geom="http://playerstage.sourceforge.net/gazebo/xmlschema/#geom">
-  <include filename="$(find sr_description/hand/xacro/finger/knuckle/knuckle.urdf.xacro" />
-  <include filename="$(find sr_description/hand/xacro/finger/proximal/proximal.urdf.xacro" />
-  <include filename="$(find sr_description/hand/xacro/finger/middle/middle.urdf.xacro" />
-  <include filename="$(find sr_description/hand/xacro/finger/distal/distal.urdf.xacro" />
-  <include filename="$(find sr_description/hand/xacro/finger/lfmetacarpal/lfmetacarpal.urdf.xacro" />
+  <include filename="$(find sr_description)/hand/xacro/finger/knuckle/knuckle.urdf.xacro" />
+  <include filename="$(find sr_description)/hand/xacro/finger/proximal/proximal.urdf.xacro" />
+  <include filename="$(find sr_description)/hand/xacro/finger/middle/middle.urdf.xacro" />
+  <include filename="$(find sr_description)/hand/xacro/finger/distal/distal.urdf.xacro" />
+  <include filename="$(find sr_description)/hand/xacro/finger/lfmetacarpal/lfmetacarpal.urdf.xacro" />
   <!-- Right Handed -->
   <xacro:macro name="little_finger" params="link_prefix joint_prefix parent">

File: hand/xacro/finger/little_finger_biotac.urdf.xacro (robot description, xacro)
@@ -6,9 +6,9 @@
        xmlns:body="http://playerstage.sourceforge.net/gazebo/xmlschema/#body"
        xmlns:geom="http://playerstage.sourceforge.net/gazebo/xmlschema/#geom">
-  <include filename="$(find sr_description/hand/xacro/finger/knuckle/knuckle.urdf.xacro" />
-  <include filename="$(find sr_description/hand/xacro/finger/proximal/proximal.urdf.xacro" />
-  <include filename="$(find sr_description/hand/xacro/finger/middle/middle.urdf.xacro" />
-  <include filename="$(find sr_description/hand/xacro/finger/distal/distal_biotac.urdf.xacro" />
-  <include filename="$(find sr_description/hand/xacro/finger/lfmetacarpal/lfmetacarpal.urdf.xacro" />
+  <include filename="$(find sr_description)/hand/xacro/finger/knuckle/knuckle.urdf.xacro" />
+  <include filename="$(find sr_description)/hand/xacro/finger/proximal/proximal.urdf.xacro" />
+  <include filename="$(find sr_description)/hand/xacro/finger/middle/middle.urdf.xacro" />
+  <include filename="$(find sr_description)/hand/xacro/finger/distal/distal_biotac.urdf.xacro" />
+  <include filename="$(find sr_description)/hand/xacro/finger/lfmetacarpal/lfmetacarpal.urdf.xacro" />
   <!-- Right Handed -->
   <xacro:macro name="little_finger" params="link_prefix joint_prefix parent">

File: hand/xacro/finger/little_finger_ellipsoid.urdf.xacro (robot description, xacro)
@@ -6,9 +6,9 @@
        xmlns:body="http://playerstage.sourceforge.net/gazebo/xmlschema/#body"
        xmlns:geom="http://playerstage.sourceforge.net/gazebo/xmlschema/#geom">
-  <include filename="$(find sr_description/hand/xacro/finger/knuckle/knuckle.urdf.xacro" />
-  <include filename="$(find sr_description/hand/xacro/finger/proximal/proximal.urdf.xacro" />
-  <include filename="$(find sr_description/hand/xacro/finger/middle/middle.urdf.xacro" />
-  <include filename="$(find sr_description/hand/xacro/finger/distal/distal_ellipsoid.urdf.xacro" />
-  <include filename="$(find sr_description/hand/xacro/finger/lfmetacarpal/lfmetacarpal.urdf.xacro" />
+  <include filename="$(find sr_description)/hand/xacro/finger/knuckle/knuckle.urdf.xacro" />
+  <include filename="$(find sr_description)/hand/xacro/finger/proximal/proximal.urdf.xacro" />
+  <include filename="$(find sr_description)/hand/xacro/finger/middle/middle.urdf.xacro" />
+  <include filename="$(find sr_description)/hand/xacro/finger/distal/distal_ellipsoid.urdf.xacro" />
+  <include filename="$(find sr_description)/hand/xacro/finger/lfmetacarpal/lfmetacarpal.urdf.xacro" />
   <xacro:macro name="little_finger" params="link_prefix joint_prefix parent">
     <xacro:lfmetacarpal parent="${parent}" >

File: hand/xacro/finger/middle/middle.urdf.xacro (robot description, xacro)
@@ -6,5 +6,5 @@
        xmlns:body="http://playerstage.sourceforge.net/gazebo/xmlschema/#body"
        xmlns:geom="http://playerstage.sourceforge.net/gazebo/xmlschema/#geom">
-  <include filename="$(find sr_description/hand/xacro/finger/middle/middle.transmission.xacro" />
+  <include filename="$(find sr_description)/hand/xacro/finger/middle/middle.transmission.xacro" />
   <xacro:macro name="middle" params="link_prefix joint_prefix parent">
     <link name="${link_prefix}middle">

File: hand/xacro/finger/proximal/proximal.urdf.xacro (robot description, xacro)
@@ -6,5 +6,5 @@
        xmlns:body="http://playerstage.sourceforge.net/gazebo/xmlschema/#body"
        xmlns:geom="http://playerstage.sourceforge.net/gazebo/xmlschema/#geom">
-  <include filename="$(find sr_description/hand/xacro/finger/proximal/proximal.transmission.xacro" />
+  <include filename="$(find sr_description)/hand/xacro/finger/proximal/proximal.transmission.xacro" />
   <xacro:macro name="proximal" params="link_prefix joint_prefix parent">
     <link name="${link_prefix}proximal">

File: hand/xacro/forearm/forearm_motor.urdf.xacro (robot description, xacro)
@@ -11,5 +11,5 @@
 	<origin xyz="0 0 0" rpy="0 0 0" />
 	<geometry name="shadow_forearm_geom">
-	  <mesh filename="package://sr_hand/model/meshes/forearm.dae" scale="0.001 0.001 0.001"/>
+	  <mesh filename="package://sr_description/hand/model/forearm.dae" scale="0.001 0.001 0.001"/>
 	</geometry>
 	<material name="Grey" />

File: hand/xacro/full_hand_motor.urdf.xacro (robot description, xacro)
@@ -3,10 +3,10 @@
        xmlns:interface="http://playerstage.sourceforge.net/gazebo/xmlschema/#interface"
        xmlns:xacro="http://www.ros.org/wiki/xacro">
-  <include filename="$(find sr_description/hand/xacro/forearm/forearm_motor.urdf.xacro" />
-  <include filename="$(find sr_description/hand/xacro/wrist/wrist.urdf.xacro" />
-  <include filename="$(find sr_description/hand/xacro/palm/palm.urdf.xacro" />
-  <include filename="$(find sr_description/hand/xacro/finger/classic_finger.urdf.xacro" />
-  <include filename="$(find sr_description/hand/xacro/finger/little_finger.urdf.xacro" />
-  <include filename="$(find sr_description/hand/xacro/thumb/thumb.urdf.xacro" />
+  <include filename="$(find sr_description)/hand/xacro/forearm/forearm_motor.urdf.xacro" />
+  <include filename="$(find sr_description)/hand/xacro/wrist/wrist.urdf.xacro" />
+  <include filename="$(find sr_description)/hand/xacro/palm/palm.urdf.xacro" />
+  <include filename="$(find sr_description)/hand/xacro/finger/classic_finger.urdf.xacro" />
+  <include filename="$(find sr_description)/hand/xacro/finger/little_finger.urdf.xacro" />
+  <include filename="$(find sr_description)/hand/xacro/thumb/thumb.urdf.xacro" />
   <!-- Right Hand -->
   <xacro:macro name="shadowhand_motor">

File: hand/xacro/full_hand_motor_biotac.urdf.xacro (robot description, xacro)
@@ -3,10 +3,10 @@
        xmlns:interface="http://playerstage.sourceforge.net/gazebo/xmlschema/#interface"
        xmlns:xacro="http://www.ros.org/wiki/xacro">
-  <include filename="$(find sr_description/hand/xacro/forearm/forearm_motor.urdf.xacro" />
-  <include filename="$(find sr_description/hand/xacro/wrist/wrist.urdf.xacro" />
-  <include filename="$(find sr_description/hand/xacro/palm/palm.urdf.xacro" />
-  <include filename="$(find sr_description/hand/xacro/finger/classic_finger_biotac.urdf.xacro" />
-  <include filename="$(find sr_description/hand/xacro/finger/little_finger_biotac.urdf.xacro" />
-  <include filename="$(find sr_description/hand/xacro/thumb/thumb_biotac.urdf.xacro" />
+  <include filename="$(find sr_description)/hand/xacro/forearm/forearm_motor.urdf.xacro" />
+  <include filename="$(find sr_description)/hand/xacro/wrist/wrist.urdf.xacro" />
+  <include filename="$(find sr_description)/hand/xacro/palm/palm.urdf.xacro" />
+  <include filename="$(find sr_description)/hand/xacro/finger/classic_finger_biotac.urdf.xacro" />
+  <include filename="$(find sr_description)/hand/xacro/finger/little_finger_biotac.urdf.xacro" />
+  <include filename="$(find sr_description)/hand/xacro/thumb/thumb_biotac.urdf.xacro" />
   <!-- Right Hand -->
   <xacro:macro name="shadowhand_motor">

File: hand/xacro/full_hand_motor_ellipsoid.urdf.xacro (robot description, xacro)
@@ -3,10 +3,10 @@
        xmlns:interface="http://playerstage.sourceforge.net/gazebo/xmlschema/#interface"
        xmlns:xacro="http://www.ros.org/wiki/xacro">
-  <include filename="$(find sr_description/hand/xacro/forearm/forearm_motor.urdf.xacro" />
-  <include filename="$(find sr_description/hand/xacro/wrist/wrist.urdf.xacro" />
-  <include filename="$(find sr_description/hand/xacro/palm/palm.urdf.xacro" />
-  <include filename="$(find sr_description/hand/xacro/finger/classic_finger_ellipsoid.urdf.xacro" />
-  <include filename="$(find sr_description/hand/xacro/finger/little_finger_ellipsoid.urdf.xacro" />
-  <include filename="$(find sr_description/hand/xacro/thumb/thumb_ellipsoid.urdf.xacro" />
+  <include filename="$(find sr_description)/hand/xacro/forearm/forearm_motor.urdf.xacro" />
+  <include filename="$(find sr_description)/hand/xacro/wrist/wrist.urdf.xacro" />
+  <include filename="$(find sr_description)/hand/xacro/palm/palm.urdf.xacro" />
+  <include filename="$(find sr_description)/hand/xacro/finger/classic_finger_ellipsoid.urdf.xacro" />
+  <include filename="$(find sr_description)/hand/xacro/finger/little_finger_ellipsoid.urdf.xacro" />
+  <include filename="$(find sr_description)/hand/xacro/thumb/thumb_ellipsoid.urdf.xacro" />
   <xacro:macro name="shadowhand_motor">
     <xacro:forearm_motor>

File: hand/xacro/full_hand_muscle.urdf.xacro (robot description, xacro)
@@ -3,10 +3,10 @@
        xmlns:interface="http://playerstage.sourceforge.net/gazebo/xmlschema/#interface"
        xmlns:xacro="http://www.ros.org/wiki/xacro">
-  <include filename="$(find sr_description/hand/xacro/forearm/forearm_muscle.urdf.xacro" />
-  <include filename="$(find sr_description/hand/xacro/wrist/wrist.urdf.xacro" />
-  <include filename="$(find sr_description/hand/xacro/palm/palm.urdf.xacro" />
-  <include filename="$(find sr_description/hand/xacro/finger/classic_finger.urdf.xacro" />
-  <include filename="$(find sr_description/hand/xacro/finger/little_finger.urdf.xacro" />
-  <include filename="$(find sr_description/hand/xacro/thumb/thumb.urdf.xacro" />
+  <include filename="$(find sr_description)/hand/xacro/forearm/forearm_muscle.urdf.xacro" />
+  <include filename="$(find sr_description)/hand/xacro/wrist/wrist.urdf.xacro" />
+  <include filename="$(find sr_description)/hand/xacro/palm/palm.urdf.xacro" />
+  <include filename="$(find sr_description)/hand/xacro/finger/classic_finger.urdf.xacro" />
+  <include filename="$(find sr_description)/hand/xacro/finger/little_finger.urdf.xacro" />
+  <include filename="$(find sr_description)/hand/xacro/thumb/thumb.urdf.xacro" />
   <!-- Right Hand -->
   <xacro:macro name="shadowhand_muscle">

File: hand/xacro/one_finger_unit_motor.urdf.xacro (robot description, xacro)
@@ -3,6 +3,6 @@
        xmlns:interface="http://playerstage.sourceforge.net/gazebo/xmlschema/#interface"
        xmlns:xacro="http://www.ros.org/wiki/xacro">
-  <include filename="$(find sr_description/hand/xacro/forearm/forearm_motor.urdf.xacro" />
-  <include filename="$(find sr_description/hand/xacro/finger/classic_finger.urdf.xacro" />
+  <include filename="$(find sr_description)/hand/xacro/forearm/forearm_motor.urdf.xacro" />
+  <include filename="$(find sr_description)/hand/xacro/finger/classic_finger.urdf.xacro" />
   <xacro:macro name="shadowhand_motor">
     <xacro:forearm_motor>
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