Commit message: Modified urdf to spawn arm support separately Removed desk from all the arm urdfs Corrected selfCollide flags to have coherent and logical status (arm is never self collides but fingers do) Corrected static transforms to use /world Removed any reference to /desk_suppport when not needed Removed any reference to /base_link or /fixed

File: arm/xacro/base/shadowarm_base.urdf.xacro (robot description, xacro)
@@ -24,5 +24,5 @@
   <gazebo reference="shadowarm_base">
     <material>Gazebo/Grey</material>
-    <selfCollide>true</selfCollide>
+    <selfCollide>false</selfCollide>
   </gazebo>
 </xacro:macro>

File: arm/xacro/hand_support/shadowarm_handsupport_motor.urdf.xacro (robot description, xacro)
@@ -24,5 +24,5 @@
     <gazebo reference="shadowarm_handsupport">
       <material>Gazebo/Grey</material>
-      <selfCollide>true</selfCollide>
+      <selfCollide>false</selfCollide>
     </gazebo>
     <joint name="ElbowJRotate" type="revolute">

File: arm/xacro/hand_support/shadowarm_handsupport_muscle.urdf.xacro (robot description, xacro)
@@ -24,5 +24,5 @@
     <gazebo reference="shadowarm_handsupport">
       <material>Gazebo/Grey</material>
-      <selfCollide>true</selfCollide>
+      <selfCollide>false</selfCollide>
     </gazebo>
     <joint name="ElbowJRotate" type="revolute">

File: arm/xacro/lower_arm/shadowarm_lowerarm.urdf.xacro (robot description, xacro)
@@ -24,5 +24,5 @@
     <gazebo reference="shadowarm_lowerarm">
 	<material>Gazebo/Grey</material>
-	<selfCollide>true</selfCollide>
+	<selfCollide>false</selfCollide>
     </gazebo>
     <joint name="ElbowJSwing" type="revolute">

File: arm/xacro/trunk/shadowarm_trunk.urdf.xacro (robot description, xacro)
@@ -24,5 +24,5 @@
       <gazebo reference="shadowarm_trunk">
 	<material>Gazebo/Grey</material>
-	<selfCollide>true</selfCollide>
+	<selfCollide>false</selfCollide>
       </gazebo>
     <joint name="ShoulderJRotate" type="revolute">

File: arm/xacro/upper_arm/shadowarm_upperarm.urdf.xacro (robot description, xacro)
@@ -24,5 +24,5 @@
     <gazebo reference="shadowarm_upperarm">
       <material>Gazebo/Grey</material>
-      <selfCollide>true</selfCollide>
+      <selfCollide>false</selfCollide>
     </gazebo>
     <joint name="ShoulderJSwing" type="revolute">

File: hand/xacro/finger/distal/distal.urdf.xacro (robot description, xacro)
@@ -46,5 +46,5 @@
       <kd  value="1.0" />
       <material>Gazebo/Grey</material>
-      <selfCollide>false</selfCollide>
+      <selfCollide>true</selfCollide>
     </gazebo>
     <joint name="${joint_prefix}J1" type="revolute">

File: hand/xacro/finger/distal/distal_ellipsoid.urdf.xacro (robot description, xacro)
@@ -53,5 +53,5 @@
       <kd  value="1.0" />
       <material>Gazebo/Grey</material>
-      <selfCollide>false</selfCollide>
+      <selfCollide>true</selfCollide>
     </gazebo>
     <joint name="${joint_prefix}J1" type="revolute">

File: hand/xacro/finger/middle/middle.urdf.xacro (robot description, xacro)
@@ -42,4 +42,5 @@
       </sensor:contact>
       <material>Gazebo/Grey</material>
+      <selfCollide>true</selfCollide>
     </gazebo>
     <joint name="${joint_prefix}J2" type="revolute">

File: hand/xacro/finger/proximal/proximal.urdf.xacro (robot description, xacro)
@@ -42,4 +42,5 @@
       </sensor:contact>
       <material>Gazebo/Grey</material>
+      <selfCollide>true</selfCollide>
     </gazebo>
     <joint name="${joint_prefix}J3" type="revolute">

File: hand/xacro/forearm/forearm_motor.urdf.xacro (robot description, xacro)
@@ -24,5 +24,5 @@
     <gazebo reference="forearm">
       <material>Gazebo/Grey</material>
-      <selfCollide>true</selfCollide>
+      <selfCollide>false</selfCollide>
     </gazebo>
   </xacro:macro>

File: hand/xacro/forearm/forearm_muscle.urdf.xacro (robot description, xacro)
@@ -24,5 +24,5 @@
     <gazebo reference="forearm">
       <material>Gazebo/Grey</material>
-      <selfCollide>true</selfCollide>
+      <selfCollide>false</selfCollide>
     </gazebo>
   </xacro:macro>

File: hand/xacro/thumb/thdistal.urdf.xacro (robot description, xacro)
@@ -49,5 +49,5 @@
       <kd  value="1.0" />
       <material>Gazebo/Grey</material>
-      <selfCollide>false</selfCollide>
+      <selfCollide>true</selfCollide>
     </gazebo>
     <joint name="THJ1" type="revolute">

File: hand/xacro/thumb/thdistal_ellipsoid.urdf.xacro (robot description, xacro)
@@ -48,5 +48,5 @@
       <kd  value="1.0" />
       <material>Gazebo/Grey</material>
-      <selfCollide>false</selfCollide>
+      <selfCollide>true</selfCollide>
     </gazebo>
     <joint name="THJ1" type="revolute">

File: hand/xacro/wrist/wrist.urdf.xacro (robot description, xacro)
@@ -39,5 +39,5 @@
     <gazebo reference="wrist">
       <material>PR2/Grey2</material>
-      <selfCollide>true</selfCollide>
+      <selfCollide>false</selfCollide>
     </gazebo>
     <joint name="WRJ2" type="revolute">

File: other/xacro/desk/desk.urdf.xacro (robot description, xacro)
@@ -1,8 +1,9 @@
 <robot name="desk" xmlns:body="http://playerstage.sourceforge.net/gazebo/xmlschema/#body" xmlns:geom="http://playerstage.sourceforge.net/gazebo/xmlschema/#geom" xmlns:interface="http://playerstage.sourceforge.net/gazebo/xmlschema/#interface" xmlns:joint="http://playerstage.sourceforge.net/gazebo/xmlschema/#slider" xmlns:xacro="http://ros.org/wiki/xacro">
   <xacro:macro name="desk">
+  <link name="world"/>
   <link name="desk_pillar">
     <inertial>
       <origin xyz="0 0 0.5"/>
-      <mass value="1000.0"/>
+      <mass value="10.0"/>
       <inertia ixx="1.0" ixy="0.0" ixz="0.0" iyy="1.0" iyz="0.0" izz="1.0"/>
     </inertial>
@@ -10,5 +11,5 @@
       <origin rpy="0 0 0" xyz="0 0 0.51"/>
       <geometry name="desk_visual">
-        <cylinder length="0.98" radius="0.1"/>
+        <cylinder length="0.97" radius="0.1"/>
       </geometry>
       <material name="Green"/>
@@ -17,5 +18,5 @@
       <origin rpy="0 0 0" xyz="0 0 0.51"/>
       <geometry name="desk_collision">
-        <cylinder length=".98" radius="0.1"/>
+        <cylinder length=".97" radius="0.05"/>
       </geometry>
     </collision>
@@ -23,14 +24,10 @@
   <gazebo reference="desk_pillar">
     <material>Gazebo/Green</material>
-    <mu1>1000.0</mu1>
-    <mu2>1000.0</mu2>
-    <kp>10000000.0</kp>
-    <kd>1.0</kd>
-    <selfCollide>true</selfCollide>
+    <selfCollide>false</selfCollide>
   </gazebo>
   <link name="desk_support">
     <inertial>
       <origin xyz="0 0 0"/>
-      <mass value="1000.0"/>
+      <mass value="10.0"/>
       <inertia ixx="1.0" ixy="0.0" ixz="0.0" iyy="1.0" iyz="0.0" izz="1.0"/>
     </inertial>
@@ -45,5 +42,5 @@
       <origin rpy="0 0 0" xyz="0 0 0.01"/>
       <geometry name="desk_s_collision">
-        <cylinder length="0.02" radius="1.0"/>
+        <cylinder length="0.002" radius="0.01"/>
       </geometry>
     </collision>
@@ -51,14 +48,15 @@
   <gazebo reference="desk_support">
     <material>Gazebo/Green</material>
-    <mu1>1000.0</mu1>
-    <mu2>1000.0</mu2>
-    <kp>10000000.0</kp>
-    <kd>1.0</kd>
-    <selfCollide>true</selfCollide>
+    <selfCollide>false</selfCollide>
   </gazebo>
   <joint name="desk_joint" type="fixed">
     <parent link="desk_support"/>
     <child link="desk_pillar"/>
-    <origin rpy="0 0 0" xyz="0 0 0.02"/>
+    <origin rpy="0 0 0" xyz="0 0 0"/>
+  </joint>
+  <joint name="desk_to_world_joint" type="fixed">
+    <parent link="world"/>
+    <child link="desk_support"/>
+    <origin rpy="0 0 0" xyz="0 0 0"/>
   </joint>
   </xacro:macro>

File: robots/arm_and_hand_motor.urdf.xacro (robot description, xacro)
@@ -4,8 +4,7 @@
   <include filename="$(find sr_description)/hand/xacro/full_hand_motor.urdf.xacro" />
   <include filename="$(find sr_description)/other/xacro/gazebo/gazebo.urdf.xacro" />
-  <include filename="$(find sr_description)/other/xacro/desk/desk.urdf.xacro" />
-  <xacro:desk/>
-  <joint name="arm_to_desk_fixed" type="fixed">
-    <parent link="desk_pillar"/>
+  <link name="world" />
+  <joint name="arm_to_world_fixed" type="fixed">
+    <parent link="world"/>
     <child link="shadowarm_base"/>
     <origin rpy="0 0 0" xyz="0 0 1.0"/>

File: robots/arm_and_hand_motor_ellipsoid.urdf.xacro (robot description, xacro)
@@ -4,8 +4,7 @@
   <include filename="$(find sr_description)/hand/xacro/full_hand_motor_ellipsoid.urdf.xacro" />
   <include filename="$(find sr_description)/other/xacro/gazebo/gazebo.urdf.xacro" />
-  <include filename="$(find sr_description)/other/xacro/desk/desk.urdf.xacro" />
-  <xacro:desk/>
-  <joint name="arm_to_desk_fixed" type="fixed">
-    <parent link="desk_pillar"/>
+  <link name="world" />
+  <joint name="arm_to_world_fixed" type="fixed">
+    <parent link="world"/>
     <child link="shadowarm_base"/>
     <origin rpy="0 0 0" xyz="0 0 1.0"/>

File: robots/arm_and_hand_motor_three_finger.urdf.xacro (robot description, xacro)
@@ -4,8 +4,7 @@
   <include filename="$(find sr_description)/hand/xacro/three_finger_unit_motor.urdf.xacro" />
   <include filename="$(find sr_description)/other/xacro/gazebo/gazebo.urdf.xacro" />
-  <include filename="$(find sr_description)/other/xacro/desk/desk.urdf.xacro" />
-  <xacro:desk/>
-  <joint name="arm_to_desk_fixed" type="fixed">
-    <parent link="desk_pillar"/>
+  <link name="world" />
+  <joint name="arm_to_world_fixed" type="fixed">
+    <parent link="world"/>
     <child link="shadowarm_base"/>
     <origin rpy="0 0 0" xyz="0 0 1.0"/>

File: robots/arm_and_hand_muscle.urdf.xacro (robot description, xacro)
@@ -4,8 +4,7 @@
   <include filename="$(find sr_description)/hand/xacro/full_hand_muscle.urdf.xacro" />
   <include filename="$(find sr_description)/other/xacro/gazebo/gazebo.urdf.xacro" />
-  <include filename="$(find sr_description)/other/xacro/desk/desk.urdf.xacro" />
-  <xacro:desk/>
-  <joint name="arm_to_desk_fixed" type="fixed">
-    <parent link="desk_pillar"/>
+  <link name="world" />
+  <joint name="arm_to_world_fixed" type="fixed">
+    <parent link="world"/>
     <child link="shadowarm_base"/>
     <origin rpy="0 0 0" xyz="0 0 1.0"/>
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
Commit message: Fixed the arm model for the latest gazebo 1.9.3 update...

File: arm/xacro/base/shadowarm_base.urdf.xacro (robot description, xacro)
@@ -2,28 +2,29 @@
 <property name="M_PI" value="3.1415926535897931" />
 <xacro:macro name="shadowarm_base">
-  <link name="shadowarm_base">
-    <inertial>
-      <origin xyz="0 0 0" rpy="0 0 0"/>
-      <mass value="0.4" />
-      <inertia  ixx="1.0" ixy="0.0"  ixz="0.0"  iyy="0.0"  iyz="0.0"  izz="0.0" />
-    </inertial>
-    <visual>
-      <origin xyz="0 0 0" rpy="0 0 0"/>
-      <geometry name="shadowarm_base_visual">
-        <mesh filename="package://sr_description/arm/model/arm_base.dae" scale="0.001 0.001 0.001" />
-      </geometry>
-      <material name="LightGrey" />
-    </visual>
-    <collision>
-      <origin xyz="0 0 0.005" rpy="0 0 0" />
-      <geometry name="shadowarm_base_collision">
-        <box size="0.03 0.03 0.01"/>
-      </geometry>
-    </collision>
-  </link>
-  <gazebo reference="shadowarm_base">
-    <material>Gazebo/Grey</material>
-    <selfCollide>false</selfCollide>
-  </gazebo>
+    <link name="shadowarm_base">
+      <inertial>
+	<origin xyz="0 0 0.0" rpy="0 0 0" />
+	<mass value="0.4" />
+	<inertia  ixx="0.1" ixy="0.0"  ixz="0.0"  iyy="0.1"  iyz="0.0"
+	izz="0.0" />
+      </inertial>
+      <visual>
+	<origin xyz="0 0 0" rpy="0 0 0" />
+	<geometry name="shadowarm_visual">
+          <mesh filename="package://sr_description/arm/model/arm_base.dae" scale="0.001 0.001 0.001" />
+        </geometry>
+        <material name="Grey" />
+      </visual>
+      <collision>
+	<origin xyz="0 0 0.0" rpy="0 0 0" />
+	<geometry name="shadowarm_collision_geom">
+          <mesh filename="package://sr_description/arm/model/arm_base.dae" scale="0.001 0.001 0.001" />
+	</geometry>
+      </collision>
+    </link>
+    <gazebo reference="shadowarm_base">
+      <material>Gazebo/Grey</material>
+      <selfCollide>true</selfCollide>
+    </gazebo>
 </xacro:macro>
 </robot>

File: arm/xacro/lower_arm/shadowarm_lowerarm.urdf.xacro (robot description, xacro)
@@ -3,26 +3,27 @@
   <xacro:macro name="shadowarm_lowerarm" params="parent">
     <link name="shadowarm_lowerarm">
-	<inertial>
-	  <origin xyz="0.08 0 0.0625" rpy="0 0 0" />
-	  <mass value="1.7" />
-	  <inertia  ixx="1.0" ixy="0.0"  ixz="0.0"  iyy="0.0"  iyz="0.0"  izz="0.0" />
-	</inertial>
-	<visual>
-	  <origin xyz="0.03 0 0.036" rpy="0 0 0"/>
-	  <geometry name="shadowarm_lowerarm_visual">
-	    <mesh filename="package://sr_description/arm/model/elbow_flex.dae" scale="0.001 0.001 0.001" />
-	  </geometry>
-	  <material name="Grey" />
-	</visual>
-	<collision>
-	  <origin xyz="0.08 0 0.0625" rpy="0 0 0"/>
-	  <geometry name="shadowarm_lowerarm_collision">
-	    <box size="0.03 0.03 0.10"/>
-	  </geometry>
-	</collision>
+      <inertial>
+	<origin xyz="0 0 0.0" rpy="0 0 0" />
+	<mass value="0.5" />
+	<inertia  ixx="0.1" ixy="0.0"  ixz="0.0"  iyy="0.1"  iyz="0.0"
+	izz="0.0" />
+      </inertial>
+      <visual>
+	<origin xyz="0 0 0" rpy="0 0 0" />
+	<geometry name="shadowarm_visual">
+          <mesh filename="package://sr_description/arm/model/elbow_flex.dae" scale="0.001 0.001 0.001" />
+        </geometry>
+        <material name="Grey" />
+      </visual>
+      <collision>
+	<origin xyz="0 0 0.0" rpy="0 0 0" />
+	<geometry name="shadowarm_collision_geom">
+          <mesh filename="package://sr_description/arm/model/elbow_flex.dae" scale="0.001 0.001 0.001" />
+	</geometry>
+      </collision>
     </link>
     <gazebo reference="shadowarm_lowerarm">
-	<material>Gazebo/Grey</material>
-	<selfCollide>false</selfCollide>
+      <material>Gazebo/Grey</material>
+      <selfCollide>true</selfCollide>
     </gazebo>
     <joint name="ElbowJSwing" type="revolute">
@@ -32,6 +33,6 @@
       <axis xyz="0 -1 0" />
       <limit lower="0.52" upper="2.09439510239"
-      effort="100" velocity="1.0"/>
-      <dynamics damping="50.5"/>
+             effort="100" velocity="1.0"/>
+      <dynamics damping="200.5"/>
     </joint>
     <xacro:shadowarm_lowerarm_transmission />

File: arm/xacro/trunk/shadowarm_trunk.urdf.xacro (robot description, xacro)
@@ -3,27 +3,28 @@
   <xacro:macro name="shadowarm_trunk" params="parent">
     <link name="shadowarm_trunk">
-	<inertial>
-	  <origin xyz="0 0 0.26525" rpy="0 0 0" />
-	  <mass value="10" />
-	  <inertia  ixx="1.47" ixy="0.0"  ixz="0.0"  iyy="1.47"  iyz="0.0"  izz="2.4" />
-	</inertial>
-	<visual>
-	  <origin xyz="0 0 0.005" rpy="0 0 0" />
-	  <geometry name="shadowarm_trunk_visual">
-	    <mesh filename="package://sr_description/arm/model/arm_trunk.dae" scale="0.001 0.001 0.001" />
-	  </geometry>
-	  <material name="Grey" />
-	</visual>
-	<collision>
-	  <origin xyz="0 0 0.26525" rpy="0 0 0"/>
-	  <geometry name="shadowarm_trunk_collision">
-	    <box size="0.03 0.03 0.52"/>
-	  </geometry>
-	</collision>
-      </link>
-      <gazebo reference="shadowarm_trunk">
-	<material>Gazebo/Grey</material>
-	<selfCollide>false</selfCollide>
-      </gazebo>
+      <inertial>
+	<origin xyz="0 0 0.0" rpy="0 0 0" />
+	<mass value="0.5" />
+	<inertia  ixx="0.1" ixy="0.0"  ixz="0.0"  iyy="0.1"  iyz="0.0"
+	izz="0.0" />
+      </inertial>
+      <visual>
+	<origin xyz="0 0 0" rpy="0 0 0" />
+	<geometry name="shadowarm_visual">
+          <mesh filename="package://sr_description/arm/model/arm_trunk.dae" scale="0.001 0.001 0.001" />
+        </geometry>
+        <material name="Grey" />
+      </visual>
+      <collision>
+	<origin xyz="0 0 0.0" rpy="0 0 0" />
+	<geometry name="shadowarm_collision_geom">
+          <mesh filename="package://sr_description/arm/model/arm_trunk.dae" scale="0.001 0.001 0.001" />
+	</geometry>
+      </collision>
+    </link>
+    <gazebo reference="shadowarm_trunk">
+      <material>Gazebo/Grey</material>
+      <selfCollide>true</selfCollide>
+    </gazebo>
     <joint name="ShoulderJRotate" type="revolute">
       <parent link="${parent}"/>

File: arm/xacro/upper_arm/shadowarm_upperarm.urdf.xacro (robot description, xacro)
@@ -4,19 +4,20 @@
     <link name="shadowarm_upperarm">
       <inertial>
-	<origin xyz="0 0 0.1845" rpy="0 0 0" />
-	<mass value="2" />
-	<inertia  ixx="0.5" ixy="0.0"  ixz="0.0"  iyy="0.5"  iyz="0.0"  izz="0.1" />
+	<origin xyz="0 0 0.0" rpy="0 0 0" />
+	<mass value="0.5" />
+	<inertia  ixx="0.1" ixy="0.0"  ixz="0.0"  iyy="0.1"  iyz="0.0"
+	izz="0.0" />
       </inertial>
       <visual>
-	<origin xyz="0 0.067 0" rpy="0 0 0" />
-	<geometry name="shadowarm_upperarm_visual">
-	  <mesh filename="package://sr_description/arm/model/upper_arm.dae" scale="0.001 0.001 0.001" />
-	</geometry>
-	<material name="Grey" />
+	<origin xyz="0 0 0" rpy="0 0 0" />
+	<geometry name="shadowarm_visual">
+          <mesh filename="package://sr_description/arm/model/upper_arm.dae" scale="0.001 0.001 0.001" />
+        </geometry>
+        <material name="Grey" />
       </visual>
       <collision>
-	<origin xyz="0 0 0.1845" rpy="0 -${M_PI} 0"/>
-	<geometry name="shadowarm_upperarm_collision">
-	  <box size="0.03 0.03 0.369"/>
+	<origin xyz="0 0 0.0" rpy="0 0 0" />
+	<geometry name="shadowarm_collision_geom">
+          <mesh filename="package://sr_description/arm/model/upper_arm.dae" scale="0.001 0.001 0.001" />
 	</geometry>
       </collision>
@@ -24,5 +25,5 @@
     <gazebo reference="shadowarm_upperarm">
       <material>Gazebo/Grey</material>
-      <selfCollide>false</selfCollide>
+      <selfCollide>true</selfCollide>
     </gazebo>
     <joint name="ShoulderJSwing" type="revolute">
@@ -32,5 +33,5 @@
       <axis xyz="0 -1 0" />
       <limit lower="0" upper="${M_PI/2}" effort="100" velocity="1.0"/>
-      <dynamics damping="50.5"/>
+      <dynamics damping="200.5"/>
     </joint>
     <xacro:shadowarm_upperarm_transmission />
