Commit message: Tab and whitespace cleanup.

File: arm/xacro/base/shadowarm_base.urdf.xacro (robot description, xacro)
@@ -2,29 +2,28 @@
 <property name="M_PI" value="3.1415926535897931" />
 <xacro:macro name="shadowarm_base">
-    <link name="shadowarm_base">
-      <inertial>
-	<origin xyz="0 0 0.0" rpy="0 0 0" />
-	<mass value="0.4" />
-	<inertia  ixx="0.1" ixy="0.0"  ixz="0.0"  iyy="0.1"  iyz="0.0"
-	izz="0.0" />
-      </inertial>
-      <visual>
-	<origin xyz="0 0 0" rpy="0 0 0" />
-	<geometry name="shadowarm_visual">
-          <mesh filename="package://sr_description/arm/model/arm_base.dae" scale="0.001 0.001 0.001" />
-        </geometry>
-        <material name="Grey" />
-      </visual>
-      <collision>
-	<origin xyz="0 0 0.0" rpy="0 0 0" />
-	<geometry name="shadowarm_collision_geom">
-          <mesh filename="package://sr_description/arm/model/arm_base.dae" scale="0.001 0.001 0.001" />
-	</geometry>
-      </collision>
-    </link>
-    <gazebo reference="shadowarm_base">
-      <material>Gazebo/Grey</material>
-      <selfCollide>true</selfCollide>
-    </gazebo>
+  <link name="shadowarm_base">
+    <inertial>
+      <origin xyz="0 0 0.0" rpy="0 0 0" />
+      <mass value="0.4" />
+      <inertia  ixx="0.1" ixy="0.0"  ixz="0.0"  iyy="0.1"  iyz="0.0" izz="0.0" />
+    </inertial>
+    <visual>
+      <origin xyz="0 0 0" rpy="0 0 0" />
+      <geometry name="shadowarm_visual">
+        <mesh filename="package://sr_description/arm/model/arm_base.dae" scale="0.001 0.001 0.001" />
+      </geometry>
+      <material name="Grey" />
+    </visual>
+    <collision>
+      <origin xyz="0 0 0.0" rpy="0 0 0" />
+      <geometry name="shadowarm_collision_geom">
+        <mesh filename="package://sr_description/arm/model/arm_base.dae" scale="0.001 0.001 0.001" />
+      </geometry>
+    </collision>
+  </link>
+  <gazebo reference="shadowarm_base">
+    <material>Gazebo/Grey</material>
+    <selfCollide>true</selfCollide>
+  </gazebo>
 </xacro:macro>
 </robot>

File: arm/xacro/lower_arm/shadowarm_lowerarm.urdf.xacro (robot description, xacro)
@@ -4,12 +4,11 @@
     <link name="shadowarm_lowerarm">
       <inertial>
-	<origin xyz="0 0 0.0" rpy="0 0 0" />
-	<mass value="0.5" />
-	<inertia  ixx="0.1" ixy="0.0"  ixz="0.0"  iyy="0.1"  iyz="0.0"
-	izz="0.0" />
+        <origin xyz="0 0 0.0" rpy="0 0 0" />
+        <mass value="0.5" />
+        <inertia  ixx="0.1" ixy="0.0"  ixz="0.0"  iyy="0.1"  iyz="0.0" izz="0.0" />
       </inertial>
       <visual>
-	<origin xyz="0 0 0" rpy="0 0 0" />
-	<geometry name="shadowarm_visual">
+        <origin xyz="0 0 0" rpy="0 0 0" />
+        <geometry name="shadowarm_visual">
           <mesh filename="package://sr_description/arm/model/elbow_flex.dae" scale="0.001 0.001 0.001" />
         </geometry>
@@ -17,8 +16,8 @@
       </visual>
       <collision>
-	<origin xyz="0 0 0.0" rpy="0 0 0" />
-	<geometry name="shadowarm_collision_geom">
+        <origin xyz="0 0 0.0" rpy="0 0 0" />
+        <geometry name="shadowarm_collision_geom">
           <mesh filename="package://sr_description/arm/model/elbow_flex.dae" scale="0.001 0.001 0.001" />
-	</geometry>
+        </geometry>
       </collision>
     </link>
@@ -32,6 +31,5 @@
       <origin xyz="0 0 0.369" rpy="0 0 0" />
       <axis xyz="0 -1 0" />
-      <limit lower="0.52" upper="2.09439510239"
-             effort="100" velocity="1.0"/>
+      <limit lower="0.52" upper="2.09439510239" effort="100" velocity="1.0"/>
       <dynamics damping="200.5"/>
     </joint>

File: arm/xacro/trunk/shadowarm_trunk.urdf.xacro (robot description, xacro)
@@ -4,12 +4,11 @@
     <link name="shadowarm_trunk">
       <inertial>
-	<origin xyz="0 0 0.0" rpy="0 0 0" />
-	<mass value="0.5" />
-	<inertia  ixx="0.1" ixy="0.0"  ixz="0.0"  iyy="0.1"  iyz="0.0"
-	izz="0.0" />
+        <origin xyz="0 0 0.0" rpy="0 0 0" />
+        <mass value="0.5" />
+        <inertia  ixx="0.1" ixy="0.0"  ixz="0.0"  iyy="0.1"  iyz="0.0" izz="0.0" />
       </inertial>
       <visual>
-	<origin xyz="0 0 0" rpy="0 0 0" />
-	<geometry name="shadowarm_visual">
+        <origin xyz="0 0 0" rpy="0 0 0" />
+        <geometry name="shadowarm_visual">
           <mesh filename="package://sr_description/arm/model/arm_trunk.dae" scale="0.001 0.001 0.001" />
         </geometry>
@@ -17,8 +16,8 @@
       </visual>
       <collision>
-	<origin xyz="0 0 0.0" rpy="0 0 0" />
-	<geometry name="shadowarm_collision_geom">
+        <origin xyz="0 0 0.0" rpy="0 0 0" />
+        <geometry name="shadowarm_collision_geom">
           <mesh filename="package://sr_description/arm/model/arm_trunk.dae" scale="0.001 0.001 0.001" />
-	</geometry>
+        </geometry>
       </collision>
     </link>

File: arm/xacro/upper_arm/shadowarm_upperarm.urdf.xacro (robot description, xacro)
@@ -4,12 +4,11 @@
     <link name="shadowarm_upperarm">
       <inertial>
-	<origin xyz="0 0 0.0" rpy="0 0 0" />
-	<mass value="0.5" />
-	<inertia  ixx="0.1" ixy="0.0"  ixz="0.0"  iyy="0.1"  iyz="0.0"
-	izz="0.0" />
+        <origin xyz="0 0 0.0" rpy="0 0 0" />
+        <mass value="0.5" />
+        <inertia  ixx="0.1" ixy="0.0"  ixz="0.0"  iyy="0.1"  iyz="0.0" izz="0.0" />
       </inertial>
       <visual>
-	<origin xyz="0 0 0" rpy="0 0 0" />
-	<geometry name="shadowarm_visual">
+        <origin xyz="0 0 0" rpy="0 0 0" />
+        <geometry name="shadowarm_visual">
           <mesh filename="package://sr_description/arm/model/upper_arm.dae" scale="0.001 0.001 0.001" />
         </geometry>
@@ -17,8 +16,8 @@
       </visual>
       <collision>
-	<origin xyz="0 0 0.0" rpy="0 0 0" />
-	<geometry name="shadowarm_collision_geom">
+        <origin xyz="0 0 0.0" rpy="0 0 0" />
+        <geometry name="shadowarm_collision_geom">
           <mesh filename="package://sr_description/arm/model/upper_arm.dae" scale="0.001 0.001 0.001" />
-	</geometry>
+        </geometry>
       </collision>
     </link>

Commit message: fixing the bad offsets, removing self collisions for the arm

File: arm/xacro/base/shadowarm_base.urdf.xacro (robot description, xacro)
@@ -25,5 +25,5 @@
     <gazebo reference="shadowarm_base">
       <material>Gazebo/Grey</material>
-      <selfCollide>true</selfCollide>
+      <selfCollide>false</selfCollide>
     </gazebo>
 </xacro:macro>

File: arm/xacro/lower_arm/shadowarm_lowerarm.urdf.xacro (robot description, xacro)
@@ -4,5 +4,5 @@
     <link name="shadowarm_lowerarm">
       <inertial>
-	<origin xyz="0 0 0.0" rpy="0 0 0" />
+	<origin xyz="0 0 0" rpy="0 0 0" />
 	<mass value="0.5" />
 	<inertia  ixx="0.1" ixy="0.0"  ixz="0.0"  iyy="0.1"  iyz="0.0"
@@ -10,5 +10,5 @@
       </inertial>
       <visual>
-	<origin xyz="0 0 0" rpy="0 0 0" />
+	<origin xyz="0.03 0 0.036" rpy="0 0 0" />
 	<geometry name="shadowarm_visual">
           <mesh filename="package://sr_description/arm/model/elbow_flex.dae" scale="0.001 0.001 0.001" />
@@ -17,5 +17,5 @@
       </visual>
       <collision>
-	<origin xyz="0 0 0.0" rpy="0 0 0" />
+	<origin xyz="0.03 0 0.036" rpy="0 0 0" />
 	<geometry name="shadowarm_collision_geom">
           <mesh filename="package://sr_description/arm/model/elbow_flex.dae" scale="0.001 0.001 0.001" />
@@ -25,5 +25,5 @@
     <gazebo reference="shadowarm_lowerarm">
       <material>Gazebo/Grey</material>
-      <selfCollide>true</selfCollide>
+      <selfCollide>false</selfCollide>
     </gazebo>
     <joint name="ElbowJSwing" type="revolute">

File: arm/xacro/trunk/shadowarm_trunk.urdf.xacro (robot description, xacro)
@@ -10,5 +10,5 @@
       </inertial>
       <visual>
-	<origin xyz="0 0 0" rpy="0 0 0" />
+	<origin xyz="0 0 0.005" rpy="0 0 0" />
 	<geometry name="shadowarm_visual">
           <mesh filename="package://sr_description/arm/model/arm_trunk.dae" scale="0.001 0.001 0.001" />
@@ -17,5 +17,5 @@
       </visual>
       <collision>
-	<origin xyz="0 0 0.0" rpy="0 0 0" />
+	<origin xyz="0 0 0.005" rpy="0 0 0" />
 	<geometry name="shadowarm_collision_geom">
           <mesh filename="package://sr_description/arm/model/arm_trunk.dae" scale="0.001 0.001 0.001" />
@@ -25,5 +25,5 @@
     <gazebo reference="shadowarm_trunk">
       <material>Gazebo/Grey</material>
-      <selfCollide>true</selfCollide>
+      <selfCollide>false</selfCollide>
     </gazebo>
     <joint name="ShoulderJRotate" type="revolute">

File: arm/xacro/upper_arm/shadowarm_upperarm.urdf.xacro (robot description, xacro)
@@ -10,5 +10,5 @@
       </inertial>
       <visual>
-	<origin xyz="0 0 0" rpy="0 0 0" />
+	<origin xyz="0 0.067 0" rpy="0 0 0" />
 	<geometry name="shadowarm_visual">
           <mesh filename="package://sr_description/arm/model/upper_arm.dae" scale="0.001 0.001 0.001" />
@@ -17,5 +17,5 @@
       </visual>
       <collision>
-	<origin xyz="0 0 0.0" rpy="0 0 0" />
+	<origin xyz="0 0.067 0" rpy="0 0 0" />
 	<geometry name="shadowarm_collision_geom">
           <mesh filename="package://sr_description/arm/model/upper_arm.dae" scale="0.001 0.001 0.001" />
@@ -25,5 +25,5 @@
     <gazebo reference="shadowarm_upperarm">
       <material>Gazebo/Grey</material>
-      <selfCollide>true</selfCollide>
+      <selfCollide>false</selfCollide>
     </gazebo>
     <joint name="ShoulderJSwing" type="revolute">
