Commit message: Modified the biotac hand model to have the biotacs for FFJ2, MFJ2 and thumb

File: hand/xacro/finger/biotac/biotac.urdf.xacro (robot description, xacro)
@@ -17,5 +17,5 @@
         <origin xyz="0 0 0" rpy="0 0 1.571" />
         <geometry name="adapter_visual">
-          <mesh filename="package://sr_description/hand/model/biotacs/F2_biotac_adapter.stl" scale="0.001 0.001 0.001" />
+          <mesh filename="package://sr_description/hand/model/biotacs/biotac_decimated.dae" scale="0.001 0.001 0.001" />
         </geometry>
         <material name="LightGrey" />

File: hand/xacro/finger/classic_finger_biotac.urdf.xacro (robot description, xacro)
@@ -3,5 +3,5 @@
   <include filename="$(find sr_description)/hand/xacro/finger/proximal/proximal.urdf.xacro" />
   <include filename="$(find sr_description)/hand/xacro/finger/biotac/biotac.urdf.xacro" />
-  <xacro:macro name="finger" params="link_prefix joint_prefix parent *origin *axis">
+  <xacro:macro name="finger_biotac" params="link_prefix joint_prefix parent *origin *axis">
     <xacro:knuckle link_prefix="${link_prefix}" joint_prefix="${joint_prefix}" parent="${parent}" >
       <insert_block name="origin" />

File: hand/xacro/full_hand_motor_biotac.urdf.xacro (robot description, xacro)
@@ -7,5 +7,6 @@
   <include filename="$(find sr_description)/hand/xacro/palm/palm.urdf.xacro" />
   <include filename="$(find sr_description)/hand/xacro/finger/classic_finger_biotac.urdf.xacro" />
-  <include filename="$(find sr_description)/hand/xacro/finger/little_finger_biotac.urdf.xacro" />
+  <include filename="$(find sr_description)/hand/xacro/finger/classic_finger.urdf.xacro" />
+  <include filename="$(find sr_description)/hand/xacro/finger/little_finger.urdf.xacro" />
   <include filename="$(find sr_description)/hand/xacro/thumb/thumb_biotac.urdf.xacro" />
   <!-- Right Hand -->
@@ -18,12 +19,12 @@
     <xacro:palm parent="wrist">
     </xacro:palm>
-    <xacro:finger link_prefix="ff" joint_prefix="FF" parent="palm">
+    <xacro:finger_biotac link_prefix="ff" joint_prefix="FF" parent="palm">
       <origin xyz="0.033 0 0.095" rpy="0 0 0" />
       <axis xyz="0 -1 0" />
-    </xacro:finger>
-    <xacro:finger link_prefix="mf" joint_prefix="MF" parent="palm">
+    </xacro:finger_biotac>
+    <xacro:finger_biotac link_prefix="mf" joint_prefix="MF" parent="palm">
       <origin xyz="0.011 0 0.099" rpy="0 0 0" />
       <axis xyz="0 -1 0" />
-    </xacro:finger>
+    </xacro:finger_biotac>
     <xacro:finger link_prefix="rf" joint_prefix="RF" parent="palm">
       <origin xyz="-0.011 0 0.095" rpy="0 0 0" />

Commit message: modified the other models to get rid of outdated sensor: syntax

File: hand/xacro/finger/biotac/biotac.urdf.xacro (robot description, xacro)
@@ -16,5 +16,5 @@
       <visual>
         <origin xyz="0 0 0" rpy="0 0 1.571" />
-        <geometry name="adapter_visual">
+        <geometry name="${link_prefix}adapter_visual">
           <mesh filename="package://sr_description/hand/model/biotacs/F2_biotac_adapter.stl" scale="0.001 0.001 0.001" />
         </geometry>
@@ -23,5 +23,5 @@
       <collision>
         <origin xyz="0 0 0.0125" rpy="0 0 0" />
-        <geometry name="adapter_collision_geom">
+        <geometry name="${link_prefix}adapter_collision_geom">
           <box size="0.008 0.008 0.03" />
         </geometry>
@@ -29,19 +29,16 @@
     </link>
     <gazebo reference="${link_prefix}adapter">
-<!--
-      <sensor:contact name="${link_prefix}adapter_contact_sensor">
-        <geom>${link_prefix}adapter_collision_geom</geom>
-        <updateRate>100.0</updateRate>
-        <controller:gazebo_ros_bumper
-            name="${link_prefix}adapter_gazebo_ros_bumper_controller"
-            plugin="libgazebo_ros_bumper.so">
+      <sensor type="contact" name="${link_prefix}adapter_contact_sensor">
+        <update_rate>100.0</update_rate>
+        <contact>
+          <collision>${link_prefix}adapter_collision_geom</collision>
+        </contact>
+        <plugin name="${link_prefix}adapter_gazebo_ros_bumper_controller" filename="libgazebo_ros_bumper.so">
           <alwaysOn>true</alwaysOn>
+          <frameName>${link_prefix}adapter</frameName>
           <updateRate>100.0</updateRate>
-          <frameName>${link_prefix}adapter</frameName>
           <bumperTopicName>${link_prefix}adapter_bumper</bumperTopicName>
-          <interface:bumper name="${link_prefix}adapter_gazebo_ros_bumper_iface" />
-        </controller:gazebo_ros_bumper>
-      </sensor:contact>
--->
+        </plugin>
+      </sensor>
       <material name="LightGrey"/>
     </gazebo>
@@ -79,5 +76,5 @@
       <visual>
         <origin xyz="0 0 0" rpy="0 0 0" />
-        <geometry name="biotac_visual">
+        <geometry name="${link_prefix}biotac_visual">
           <!-- <mesh filename="package://sr_description/hand/model/biotacs/biotac.stl" scale="0.0254 0.0254 0.0254" /> -->
           <mesh filename="package://sr_description/hand/model/biotacs/biotac_decimated.dae" scale="0.0254 0.0254 0.0254" />
@@ -93,19 +90,16 @@
     </link>
     <gazebo reference="${link_prefix}biotac">
-<!--
-      <sensor:contact name="${link_prefix}adapter_contact_sensor">
-        <geom>${link_prefix}biotac_collision_geom</geom>
-        <updateRate>100.0</updateRate>
-        <controller:gazebo_ros_bumper
-            name="${link_prefix}biotac_gazebo_ros_bumper_controller"
-            plugin="libgazebo_ros_bumper.so">
+      <sensor type="contact" name="${link_prefix}biotac_contact_sensor">
+        <update_rate>100.0</update_rate>
+        <contact>
+          <collision>${link_prefix}biotac_collision_geom</collision>
+        </contact>
+        <plugin name="${link_prefix}biotac_gazebo_ros_bumper_controller" filename="libgazebo_ros_bumper.so">
           <alwaysOn>true</alwaysOn>
+          <frameName>${link_prefix}biotac</frameName>
           <updateRate>100.0</updateRate>
-          <frameName>${link_prefix}biotac</frameName>
           <bumperTopicName>${link_prefix}biotac_bumper</bumperTopicName>
-          <interface:bumper name="${link_prefix}biotac_gazebo_ros_bumper_iface" />
-        </controller:gazebo_ros_bumper>
-      </sensor:contact>
--->
+        </plugin>
+      </sensor>
       <material name="BiotacGreen"/>
     </gazebo>

File: hand/xacro/finger/distal/distal_biotac.urdf.xacro (robot description, xacro)
@@ -17,5 +17,5 @@
       <visual>
 	<origin xyz="0 0 0" rpy="0 0 0" />
-	<geometry name="distal_visual">
+	<geometry name="${link_prefix}distal_visual">
       <mesh filename="package://sr_description/hand/model/F1.mesh" scale="0.001 0.001 0.001" />
       </geometry>
@@ -24,5 +24,5 @@
       <collision>
 	<origin xyz="0 0 0" rpy="0 0 0" />
-	<geometry name="distal_collision_geom">
+	<geometry name="${link_prefix}distal_collision_geom">
 	  <mesh filename="package://sr_description/hand/model/F1.mesh" scale="0.001 0.001 0.001" />
 	</geometry>
@@ -30,15 +30,16 @@
     </link>
     <gazebo reference="${link_prefix}distal">
-      <sensor:contact name="${link_prefix}distal_contact_sensor">
-        <geom>${link_prefix}distal_geom</geom>
-        <updateRate>100.0</updateRate>
-        <controller:gazebo_ros_bumper name="${link_prefix}distal_gazebo_ros_bumper_controller" plugin="libgazebo_ros_bumper.so">
+      <sensor type="contact" name="${link_prefix}distal_contact_sensor">
+        <update_rate>100.0</update_rate>
+        <contact>
+          <collision>${link_prefix}distal_collision_geom</collision>
+        </contact>
+        <plugin name="${link_prefix}distal_gazebo_ros_bumper_controller" filename="libgazebo_ros_bumper.so">
           <alwaysOn>true</alwaysOn>
+          <frameName>${link_prefix}distal</frameName>
           <updateRate>100.0</updateRate>
-          <frameName>${link_prefix}distal</frameName>
           <bumperTopicName>${link_prefix}distal_bumper</bumperTopicName>
-          <interface:bumper name="${link_prefix}distal_gazebo_ros_bumper_iface" />
-        </controller:gazebo_ros_bumper>
-      </sensor:contact>
+        </plugin>
+      </sensor>
       <material>Gazebo/Grey</material>
     </gazebo>

File: hand/xacro/finger/distal/distal_ellipsoid.urdf.xacro (robot description, xacro)
@@ -17,5 +17,5 @@
       <visual>
 	<origin xyz="0 0 0" rpy="0 0 0" />
-	<geometry name="distal_visual">
+	<geometry name="${link_prefix}distal_visual">
 	  <mesh filename="package://sr_description/hand/model/distal_ellipsoid.dae" scale="0.001 0.001 0.001" />
 	</geometry>
@@ -31,5 +31,5 @@
       <collision>
         <origin xyz="0 0 0" rpy="0 0 0" />
-        <geometry name="distal_collision_geom">
+        <geometry name="${link_prefix}distal_collision_geom">
           <mesh filename="package://sr_description/hand/model/distal_ellipsoid.dae" scale="0.001 0.001 0.001" />
         </geometry>
@@ -37,15 +37,16 @@
     </link>
     <gazebo reference="${link_prefix}distal">
-      <sensor:contact name="${link_prefix}distal_contact_sensor">
-        <geom>${link_prefix}distal_geom</geom>
-        <updateRate>100.0</updateRate>
-        <controller:gazebo_ros_bumper name="${link_prefix}distal_gazebo_ros_bumper_controller" plugin="libgazebo_ros_bumper.so">
+      <sensor type="contact" name="${link_prefix}distal_contact_sensor">
+        <update_rate>100.0</update_rate>
+        <contact>
+          <collision>${link_prefix}distal_collision_geom</collision>
+        </contact>
+        <plugin name="${link_prefix}distal_gazebo_ros_bumper_controller" filename="libgazebo_ros_bumper.so">
           <alwaysOn>true</alwaysOn>
+          <frameName>${link_prefix}distal</frameName>
           <updateRate>100.0</updateRate>
-          <frameName>${link_prefix}distal</frameName>
           <bumperTopicName>${link_prefix}distal_bumper</bumperTopicName>
-          <interface:bumper name="${link_prefix}distal_gazebo_ros_bumper_iface" />
-        </controller:gazebo_ros_bumper>
-      </sensor:contact>
+        </plugin>
+      </sensor>
       <mu1 value="500.0" />
       <mu2 value="500.0" />

File: hand/xacro/finger/little_finger_biotac.urdf.xacro (robot description, xacro)
@@ -32,5 +32,5 @@
       <visual>
         <origin xyz="0 0 0" rpy="0 0 0" />
-        <geometry name="knuckle_visual">
+        <geometry name="lfknuckle_visual">
           <mesh filename="package://sr_description/hand/model/knuckle.dae" scale="0.001 0.001 0.001" />
         </geometry>
@@ -39,5 +39,5 @@
       <collision>
         <origin xyz="0 0 0" rpy="0 0 0" />
-        <geometry name="knuckle_collision_geom">
+        <geometry name="lfknuckle_collision_geom">
           <box size="0.005 0.005 0.005" />
         </geometry>
@@ -45,16 +45,17 @@
     </link>
     <gazebo reference="lfknuckle">
-      <sensor:contact name="lfknuckle_contact_sensor">
-        <geom>lfknuckle_geom</geom>
-        <updateRate>100.0</updateRate>
-        <controller:gazebo_ros_bumper name="lfknuckle_gazebo_ros_bumper_controller" plugin="libgazebo_ros_bumper.so">
+      <sensor type="contact" name="lfknuckle_contact_sensor">
+        <update_rate>100.0</update_rate>
+        <contact>
+          <collision>lfknuckle_collision_geom</collision>
+        </contact>
+        <plugin name="lfknuckle_gazebo_ros_bumper_controller" filename="libgazebo_ros_bumper.so">
           <alwaysOn>true</alwaysOn>
+          <frameName>lfknuckle</frameName>
           <updateRate>100.0</updateRate>
-          <frameName>lfknuckle</frameName>
           <bumperTopicName>lfknuckle_bumper</bumperTopicName>
-          <interface:bumper name="lfknuckle_gazebo_ros_bumper_iface" />
-        </controller:gazebo_ros_bumper>
-      </sensor:contact>
-      <material>PR2/Grey2</material>
+        </plugin>
+      </sensor>
+      <material>Gazebo/Grey</material>
     </gazebo>
     <joint name="LFJ4" type="revolute">

File: hand/xacro/finger/little_finger_ellipsoid.urdf.xacro (robot description, xacro)
@@ -36,16 +36,17 @@
     </link>
     <gazebo reference="lfknuckle">
-      <sensor:contact name="lfknuckle_contact_sensor">
-        <geom>lfknuckle_geom</geom>
-       <updateRate>100.0</updateRate>
-        <controller:gazebo_ros_bumper name="lfknuckle_gazebo_ros_bumper_controller" plugin="libgazebo_ros_bumper.so">
+      <sensor type="contact" name="lfknuckle_contact_sensor">
+        <update_rate>100.0</update_rate>
+        <contact>
+          <collision>lfknuckle_collision_geom</collision>
+        </contact>
+        <plugin name="lfknuckle_gazebo_ros_bumper_controller" filename="libgazebo_ros_bumper.so">
           <alwaysOn>true</alwaysOn>
+          <frameName>lfknuckle</frameName>
           <updateRate>100.0</updateRate>
-          <frameName>lfknuckle</frameName>
           <bumperTopicName>lfknuckle_bumper</bumperTopicName>
-          <interface:bumper name="lfknuckle_gazebo_ros_bumper_iface" />
-        </controller:gazebo_ros_bumper>
-      </sensor:contact>
-      <material>PR2/Grey2</material>
+        </plugin>
+      </sensor>
+      <material>Gazebo/Grey</material>
     </gazebo>
     <joint name="LFJ4" type="revolute">

File: hand/xacro/thumb/thbiotac.urdf.xacro (robot description, xacro)
@@ -104,5 +104,5 @@
       </visual>
       <collision>
-        <geometry name="$th_biotac_collision_geom">
+        <geometry name="th_biotac_collision_geom">
           <!-- <box size="0.001 0.001 0.001" /> -->
           <!-- <mesh filename="package://sr_description/hand/model/biotacs/biotac-v5.stl" scale="0.0254 0.0254 0.0254" /> -->
@@ -112,19 +112,16 @@
     </link>
     <gazebo reference="thbiotac">
-<!--
-      <sensor:contact name="th_adapter_contact_sensor">
-        <geom>th_biotac_collision_geom</geom>
-        <updateRate>100.0</updateRate>
-        <controller:gazebo_ros_bumper
-            name="th_biotac_gazebo_ros_bumper_controller"
-            plugin="libgazebo_ros_bumper.so">
+      <sensor type="contact" name="thbiotac_contact_sensor">
+        <update_rate>100.0</update_rate>
+        <contact>
+          <collision>thbiotac_collision_geom</collision>
+        </contact>
+        <plugin name="thbiotac_gazebo_ros_bumper_controller" filename="libgazebo_ros_bumper.so">
           <alwaysOn>true</alwaysOn>
+          <frameName>thbiotac</frameName>
           <updateRate>100.0</updateRate>
-          <frameName>thbiotac</frameName>
-          <bumperTopicName>th_biotac_bumper</bumperTopicName>
-          <interface:bumper name="$th_biotac_gazebo_ros_bumper_iface" />
-        </controller:gazebo_ros_bumper>
-      </sensor:contact>
--->
+          <bumperTopicName>thbiotac_bumper</bumperTopicName>
+        </plugin>
+      </sensor>
       <material name="BiotacGreen"/>
     </gazebo>
