Commit message: better position pids

File: hand/xacro/finger/biotac/biotac.urdf.xacro (robot description, xacro)
@@ -48,7 +48,7 @@
       <origin xyz="0 0 0.045" rpy="0 0 0" />
       <axis xyz="1 0 0" />
-      <limit lower="0" upper="${M_PI/2}" effort="10"
-      velocity="1.0" />
-      <dynamics damping="50.5"/>
+      <limit lower="0" upper="${M_PI/2}" effort="1000.0"
+      velocity="10.0" />
+      <dynamics damping="10.0"/>
     </joint>
     <link name="${link_prefix}_J1_dummy">
@@ -64,6 +64,6 @@
       <origin xyz="0 0 0.02" rpy="0 0 0" />
       <axis xyz="1 0 0" />
-      <limit lower="${20*M_PI/180}" upper="${20.1*M_PI/180}" effort="10" velocity="0.1" />
-      <dynamics damping="50.5"/>
+      <limit lower="${20*M_PI/180}" upper="${20.1*M_PI/180}" effort="1000.0" velocity="10.0" />
+      <dynamics damping="10.0"/>
     </joint>
     <xacro:middle_transmission />

File: hand/xacro/finger/biotac/edc_muscle_biotac.urdf.xacro (robot description, xacro)
@@ -48,7 +48,7 @@
       <origin xyz="0 0 0.045" rpy="0 0 0" />
       <axis xyz="1 0 0" />
-      <limit lower="0" upper="${M_PI/2}" effort="10"
-      velocity="1.0" />
-      <dynamics damping="50.5"/>
+      <limit lower="0" upper="${M_PI/2}" effort="1000.0"
+      velocity="10.0" />
+      <dynamics damping="10.0"/>
     </joint>
     <link name="${link_prefix}_J1_dummy">
@@ -64,6 +64,6 @@
       <origin xyz="0 0 0.02" rpy="0 0 0" />
       <axis xyz="1 0 0" />
-      <limit lower="${20*M_PI/180}" upper="${20.1*M_PI/180}" effort="10" velocity="0.1" />
-      <dynamics damping="50.5"/>
+      <limit lower="${20*M_PI/180}" upper="${20.1*M_PI/180}" effort="1000.0" velocity="10.0" />
+      <dynamics damping="10.0"/>
     </joint>
     <xacro:middle_transmission />

File: hand/xacro/finger/distal/distal.urdf.xacro (robot description, xacro)
@@ -54,7 +54,7 @@
       <origin xyz="0 0 0.025" rpy="0 0 0" />
       <axis xyz="1 0 0" />
-      <limit lower="0" upper="${M_PI/2}" effort="10"
-      velocity="1.0" />
-      <dynamics damping="50.5"/>
+      <limit lower="0" upper="${M_PI/2}" effort="1000.0"
+      velocity="10.0" />
+      <dynamics damping="10.0"/>
     </joint>
     <link name="${link_prefix}tip">

File: hand/xacro/finger/distal/distal_biotac.urdf.xacro (robot description, xacro)
@@ -49,7 +49,7 @@
       <origin xyz="0 0 0.025" rpy="0 0 0" />
       <axis xyz="1 0 0" />
-      <limit lower="0.34906585" upper="0.34906585" effort="10"
-      velocity="1.0" />
-      <dynamics damping="50.5"/>
+      <limit lower="0.34906585" upper="0.34906585" effort="1000.0"
+      velocity="10.0" />
+      <dynamics damping="10.0"/>
     </joint>
 <!--

File: hand/xacro/finger/distal/distal_ellipsoid.urdf.xacro (robot description, xacro)
@@ -61,7 +61,7 @@
       <origin xyz="0 0 0.025" rpy="0 0 0" />
       <axis xyz="1 0 0" />
-      <limit lower="0" upper="${M_PI/2}" effort="10"
-	     velocity="1.0" />
-      <dynamics damping="50.5"/>
+      <limit lower="0" upper="${M_PI/2}" effort="1000.0"
+	     velocity="10.0" />
+      <dynamics damping="10.0"/>
     </joint>
     <link name="${link_prefix}tip">

File: hand/xacro/finger/knuckle/edc_muscle_knuckle.urdf.xacro (robot description, xacro)
@@ -52,6 +52,6 @@
       <insert_block name="axis"/>
       <limit lower="-0.43633231299858238" upper="0.43633231299858238"
-      effort="10" velocity="1.0"/>
-      <dynamics damping="50.5"/>
+      effort="1000.0" velocity="10.0"/>
+      <dynamics damping="10.0"/>
     </joint>
     <xacro:knuckle_transmission />

File: hand/xacro/finger/knuckle/knuckle.urdf.xacro (robot description, xacro)
@@ -52,6 +52,6 @@
       <insert_block name="axis"/>
       <limit lower="-0.3491" upper="0.3491"
-      effort="10" velocity="1.0"/>
-      <dynamics damping="50.5"/>
+      effort="1000.0" velocity="10.0"/>
+      <dynamics damping="10.0"/>
     </joint>
     <xacro:knuckle_transmission />

File: hand/xacro/finger/lfmetacarpal/edc_muscle_lfmetacarpal.urdf.xacro (robot description, xacro)
@@ -58,7 +58,7 @@
       <origin xyz="${reflect*-0.033} 0 0.02071" rpy="0 0 0" />
       <axis xyz="0.573576436 0 ${reflect*0.819152044}" />
-      <limit lower="0" upper="0.69813170079773179" effort="10"
-      velocity="1.0" />
-      <dynamics damping="50.5"/>
+      <limit lower="0" upper="0.69813170079773179" effort="1000.0"
+      velocity="10.0" />
+      <dynamics damping="10.0"/>
     </joint>
     <xacro:lfmetacarpal_transmission />

File: hand/xacro/finger/lfmetacarpal/lfmetacarpal.urdf.xacro (robot description, xacro)
@@ -58,7 +58,7 @@
       <origin xyz="${reflect*-0.033} 0 0.02071" rpy="0 0 0" />
       <axis xyz="0.573576436 0 ${reflect*0.819152044}" />
-      <limit lower="0" upper="0.785398163" effort="10"
-      velocity="1.0" />
-      <dynamics damping="50.5"/>
+      <limit lower="0" upper="0.785398163" effort="1000.0"
+      velocity="10.0" />
+      <dynamics damping="10.0"/>
     </joint>
     <xacro:lfmetacarpal_transmission />

File: hand/xacro/finger/little_finger_ellipsoid.urdf.xacro (robot description, xacro)
@@ -56,6 +56,6 @@
       <axis xyz="0 1 0" />
       <limit lower="-0.3491" upper="0.3491"
-      effort="10" velocity="1.0"/>
-      <dynamics damping="50.5"/>
+      effort="1000.0" velocity="10.0"/>
+      <dynamics damping="10.0"/>
     </joint>
     <transmission type="sr_mechanism_model/SimpleTransmission" name="lfknuckle_transmission">

File: hand/xacro/finger/middle/middle.urdf.xacro (robot description, xacro)
@@ -50,7 +50,7 @@
       <origin xyz="0 0 0.045" rpy="0 0 0" />
       <axis xyz="1 0 0" />
-      <limit lower="0" upper="${M_PI/2}" effort="10"
-      velocity="1.0" />
-      <dynamics damping="50.5"/>
+      <limit lower="0" upper="${M_PI/2}" effort="1000.0"
+      velocity="10.0" />
+      <dynamics damping="10.0"/>
     </joint>
     <xacro:middle_transmission />

File: hand/xacro/finger/proximal/edc_muscle_proximal.urdf.xacro (robot description, xacro)
@@ -50,7 +50,7 @@
       <origin xyz="0 0 0" rpy="0 0 0" />
       <axis xyz="1 0 0" />
-      <limit lower="0" upper="${M_PI/2}" effort="10"
-      velocity="1.0"/>
-      <dynamics damping="50.5"/>
+      <limit lower="0" upper="${M_PI/2}" effort="1000.0"
+      velocity="10.0"/>
+      <dynamics damping="10.0"/>
     </joint>
     <xacro:proximal_transmission />

File: hand/xacro/finger/proximal/proximal.urdf.xacro (robot description, xacro)
@@ -50,7 +50,7 @@
       <origin xyz="0 0 0" rpy="0 0 0" />
       <axis xyz="1 0 0" />
-      <limit lower="0" upper="${M_PI/2}" effort="10"
-      velocity="1.0"/>
-      <dynamics damping="50.5"/>
+      <limit lower="0" upper="${M_PI/2}" effort="1000.0"
+      velocity="10.0"/>
+      <dynamics damping="10.0"/>
     </joint>
     <xacro:proximal_transmission />

File: hand/xacro/palm/edc_muscle_palm.urdf.xacro (robot description, xacro)
@@ -59,6 +59,6 @@
       <axis xyz="1 0 0" />
       <limit lower="-0.78539816339744828" upper="0.6108652381980153"
-      effort="5" velocity="1.0"/>
-      <dynamics damping="100.5"/>
+      effort="1000.0" velocity="10.0"/>
+      <dynamics damping="30.0"/>
     </joint>
     <xacro:shadowhand_palm_transmission />

File: hand/xacro/palm/palm.urdf.xacro (robot description, xacro)
@@ -59,6 +59,6 @@
       <axis xyz="1 0 0" />
       <limit lower="-0.7854" upper="0.5236"
-      effort="5" velocity="1.0"/>
-      <dynamics damping="100.5"/>
+      effort="1000.0" velocity="10.0"/>
+      <dynamics damping="30.0"/>
     </joint>
     <xacro:shadowhand_palm_transmission />

File: hand/xacro/thumb/edc_muscle_thbase.urdf.xacro (robot description, xacro)
@@ -61,7 +61,7 @@
       <origin xyz="${reflect*0.034} -0.0085 0.029" rpy="0 ${M_PI/4} ${joint_yaw}" />
       <axis xyz="0 0 ${reflect*-1}" />
-      <limit lower="-1.047" upper="1.047" effort="10"
-      velocity="1.0" />
-      <dynamics damping="50.5"/>
+      <limit lower="-1.047" upper="1.047" effort="1000.0"
+      velocity="10.0" />
+      <dynamics damping="10.0"/>
     </joint>
     <xacro:thbase_transmission />

File: hand/xacro/thumb/edc_muscle_thbiotac.urdf.xacro (robot description, xacro)
@@ -56,7 +56,7 @@
       <origin xyz="0 0 0.01" rpy="0 0 0" /> <!-- FIXME: z offset is too large -->
       <axis xyz="0 -1 0" />
-      <limit lower="-0.5237" upper="0.5237" effort="10"
-      velocity="1.0" />
-      <dynamics damping="50.5"/>
+      <limit lower="-0.5237" upper="0.5237" effort="1000.0"
+      velocity="10.0" />
+      <dynamics damping="10.0"/>
     </joint>
     <transmission type="sr_mechanism_model/SimpleTransmissionForMuscle" name="thmiddle_transmission">
@@ -79,6 +79,6 @@
       <origin xyz="0 0 0.02" rpy="0 0 0" />
       <axis xyz="1 0 0" />
-      <limit lower="${20*M_PI/180}" upper="${20.1*M_PI/180}" effort="10" velocity="0.1" />
-      <dynamics damping="50.5"/>
+      <limit lower="${20*M_PI/180}" upper="${20.1*M_PI/180}" effort="1000.0" velocity="10.0" />
+      <dynamics damping="10.0"/>
     </joint>
     <transmission type="sr_mechanism_model/SimpleTransmissionForMuscle" name="thdistal_transmission">

File: hand/xacro/thumb/edc_muscle_thhub.urdf.xacro (robot description, xacro)
@@ -51,7 +51,7 @@
       <origin xyz="0 0 0.038" rpy="0 0 0" />
       <axis xyz="1 0 0" />
-      <limit lower="-0.2618" upper="0.2618" effort="10"
-      velocity="1.0" />
-      <dynamics damping="50.5"/>
+      <limit lower="-0.2618" upper="0.2618" effort="1000.0"
+      velocity="10.0" />
+      <dynamics damping="10.0"/>
     </joint>
     <xacro:thhub_transmission />

File: hand/xacro/thumb/edc_muscle_thproximal.urdf.xacro (robot description, xacro)
@@ -60,7 +60,7 @@
       <origin xyz="0 0 0" rpy="0 0 0" />
       <axis xyz="${reflect*1} 0 0" />
-      <limit lower="0" upper="1.309" effort="10"
-      velocity="1.0" />
-      <dynamics damping="50.5"/>
+      <limit lower="0" upper="1.309" effort="1000.0"
+      velocity="10.0" />
+      <dynamics damping="10.0"/>
     </joint>
     <xacro:thproximal_transmission />

File: hand/xacro/thumb/thbase.urdf.xacro (robot description, xacro)
@@ -61,7 +61,7 @@
       <origin xyz="${reflect*0.034} -0.0085 0.029" rpy="0 ${M_PI/4} ${joint_yaw}" />
       <axis xyz="0 0 ${reflect*-1}" />
-      <limit lower="-1.047" upper="1.047" effort="10"
-      velocity="1.0" />
-      <dynamics damping="50.5"/>
+      <limit lower="-1.047" upper="1.047" effort="1000.0"
+      velocity="10.0" />
+      <dynamics damping="10.0"/>
     </joint>
     <xacro:thbase_transmission />
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