Commit message: all joints in transmissions tagged just joint

File: hand/xacro/finger/biotac/biotac.transmission.xacro (robot description, xacro)
@@ -11,6 +11,6 @@
     <transmission type="sr_mechanism_model/J0Transmission" name="${link_prefix}middle_transmission">
       <actuator name="${joint_prefix}J0" />
-      <joint1 name="${joint_prefix}J1" />
-      <joint2 name="${joint_prefix}J2" />
+      <joint name="${joint_prefix}J1" />
+      <joint name="${joint_prefix}J2" />
     </transmission>
   </xacro:macro>

File: hand/xacro/finger/biotac/edc_muscle_biotac.transmission.xacro (robot description, xacro)
@@ -11,6 +11,6 @@
     <transmission type="sr_mechanism_model/J0TransmissionForMuscle" name="${link_prefix}middle_transmission">
       <actuator name="${joint_prefix}J0" />
-      <joint1 name="${joint_prefix}J1" />
-      <joint2 name="${joint_prefix}J2" />
+      <joint name="${joint_prefix}J1" />
+      <joint name="${joint_prefix}J2" />
     </transmission>
   </xacro:macro>

File: hand/xacro/finger/middle/middle.transmission.xacro (robot description, xacro)
@@ -7,6 +7,6 @@
     <transmission type="sr_mechanism_model/J0Transmission" name="${link_prefix}middle_transmission">
       <actuator name="${joint_prefix}J0" />
-      <joint1 name="${joint_prefix}J1" />
-      <joint2 name="${joint_prefix}J2" />
+      <joint name="${joint_prefix}J1" />
+      <joint name="${joint_prefix}J2" />
     </transmission>
   </xacro:macro>
