Commit message: merged arm muscle and motor launch into sr_arm.launch

File: arm/xacro/hand_support/shadowarm_handsupport_motor.urdf.xacro (robot description, xacro)
@@ -2,5 +2,5 @@
   <include filename="$(find sr_description)/arm/xacro/hand_support/shadowarm_handsupport_motor.transmission.xacro" />
   <xacro:macro name="shadowarm_handsupport_motor" params="parent">
-    <link name="shadowarm_handsupport_motor">
+    <link name="shadowarm_handsupport">
       <inertial>
 	<origin xyz="0 0 0" rpy="0 0 0" />
@@ -22,5 +22,5 @@
       </collision>
     </link>
-    <gazebo reference="shadowarm_handsupport_motor">
+    <gazebo reference="shadowarm_handsupport">
       <material>Gazebo/Grey</material>
       <selfCollide>true</selfCollide>
@@ -28,5 +28,5 @@
     <joint name="ElbowJRotate" type="revolute">
       <parent link="${parent}"/>
-      <child link="shadowarm_handsupport_motor"/>
+      <child link="shadowarm_handsupport"/>
       <origin xyz="0.08 0 0.125" rpy="0.0 0 0" />
       <axis xyz="0 0 -1" />

File: arm/xacro/hand_support/shadowarm_handsupport_muscle.urdf.xacro (robot description, xacro)
@@ -2,5 +2,5 @@
   <include filename="$(find sr_description)/arm/xacro/hand_support/shadowarm_handsupport_muscle.transmission.xacro" />
   <xacro:macro name="shadowarm_handsupport_muscle" params="parent">
-    <link name="shadowarm_handsupport_muscle">
+    <link name="shadowarm_handsupport">
       <inertial>
 	<origin xyz="0 0 0" rpy="0 0 0" />
@@ -22,5 +22,5 @@
       </collision>
     </link>
-    <gazebo reference="shadowarm_handsupport_muscle">
+    <gazebo reference="shadowarm_handsupport">
       <material>Gazebo/Grey</material>
       <selfCollide>true</selfCollide>
@@ -28,5 +28,5 @@
     <joint name="ElbowJRotate" type="revolute">
       <parent link="${parent}"/>
-      <child link="shadowarm_handsupport_muscle"/>
+      <child link="shadowarm_handsupport"/>
       <origin xyz="0.08 0 0.131" rpy="0 0 0" />
       <axis xyz="0 0 -1" />

File: robots/arm_and_hand_motor.urdf.xacro (robot description, xacro)
@@ -14,5 +14,5 @@
   </xacro:sr_arm_motor>
   <joint name="arm_link" type="fixed">
-    <parent link="shadowarm_handsupport_motor"/>
+    <parent link="shadowarm_handsupport"/>
     <child link="forearm"/>
     <origin xyz="0 0 0" rpy="0 0 ${2.35619449}" />

File: robots/arm_and_hand_motor_ellipsoid.urdf.xacro (robot description, xacro)
@@ -14,5 +14,5 @@
   </xacro:sr_arm_motor>
   <joint name="arm_link" type="fixed">
-    <parent link="shadowarm_handsupport_motor"/>
+    <parent link="shadowarm_handsupport"/>
     <child link="forearm"/>
     <origin xyz="0 0 0" rpy="0 0 ${2.35619449}" />

File: robots/arm_and_hand_motor_three_finger.urdf.xacro (robot description, xacro)
@@ -14,5 +14,5 @@
   </xacro:sr_arm_motor>
   <joint name="arm_link" type="fixed">
-    <parent link="shadowarm_handsupport_motor"/>
+    <parent link="shadowarm_handsupport"/>
     <child link="forearm"/>
     <origin xyz="0 0 0" rpy="0 0 ${2.35619449}" />

File: robots/arm_and_hand_muscle.urdf.xacro (robot description, xacro)
@@ -14,5 +14,5 @@
   </xacro:sr_arm_muscle>
   <joint name="arm_link" type="fixed">
-    <parent link="shadowarm_handsupport_muscle"/>
+    <parent link="shadowarm_handsupport"/>
     <child link="forearm"/>
     <origin xyz="0 0 0" rpy="0 0 ${M_PI}" />

File: robots/arm_and_sr_one_finger_motor.urdf.xacro (robot description, xacro)
@@ -14,5 +14,5 @@
   </xacro:sr_arm_motor>
   <joint name="arm_link" type="revolute">
-    <parent link="shadowarm_handsupport_motor"/>
+    <parent link="shadowarm_handsupport"/>
     <child link="forearm"/>
     <origin xyz="0 0 0" rpy="0 0 ${M_PI}" />

File: robots/desk_arm_and_hand_motor.urdf.xacro (robot description, xacro)
@@ -14,5 +14,5 @@
   </xacro:sr_arm_motor>
   <joint name="arm_link" type="revolute">
-    <parent link="shadowarm_handsupport_motor"/>
+    <parent link="shadowarm_handsupport"/>
     <child link="forearm"/>
     <origin xyz="0 0 0" rpy="0 0 ${M_PI}" />

Commit message: better arm reaction in gazebo

File: arm/xacro/hand_support/shadowarm_handsupport_motor.urdf.xacro (robot description, xacro)
@@ -32,6 +32,6 @@
       <axis xyz="0 0 -1" />
       <limit lower="-${M_PI/2}" upper="${M_PI/2}"
-      effort="10" velocity="1.0"/>
-      <dynamics damping="10.5"/>
+      effort="1000.0" velocity="10.0"/>
+      <dynamics damping="30.0"/>
     </joint>
     <xacro:shadowarm_handsupport_motor_transmission />

File: arm/xacro/hand_support/shadowarm_handsupport_muscle.urdf.xacro (robot description, xacro)
@@ -32,6 +32,6 @@
       <axis xyz="0 0 -1" />
       <limit lower="-${M_PI/2}" upper="${M_PI/2}"
-      effort="10" velocity="1.0"/>
-      <dynamics damping="10.5"/>
+      effort="1000.0" velocity="10.0"/>
+      <dynamics damping="20.0"/>
     </joint>
     <xacro:shadowarm_handsupport_muscle_transmission />

File: arm/xacro/lower_arm/shadowarm_lowerarm.urdf.xacro (robot description, xacro)
@@ -32,6 +32,6 @@
       <origin xyz="0 0 0.369" rpy="0 0 0" />
       <axis xyz="0 -1 0" />
-      <limit lower="0.52" upper="2.09439510239" effort="100" velocity="1.0"/>
-      <dynamics damping="200.5"/>
+      <limit lower="0.52" upper="2.09439510239" effort="1000.0" velocity="10.0"/>
+      <dynamics damping="20.0"/>
     </joint>
     <xacro:shadowarm_lowerarm_transmission />

File: arm/xacro/trunk/shadowarm_trunk.urdf.xacro (robot description, xacro)
@@ -32,6 +32,6 @@
       <axis xyz="0 0 1" />
       <limit lower="-${M_PI/4}" upper="${M_PI/2}"
-      effort="100" velocity="1.0"/>
-      <dynamics damping="200.5"/>
+      effort="1000.0" velocity="10.0"/>
+      <dynamics damping="30.0"/>
     </joint>
     <xacro:shadowarm_trunk_transmission />

File: arm/xacro/upper_arm/shadowarm_upperarm.urdf.xacro (robot description, xacro)
@@ -31,6 +31,6 @@
       <origin xyz="0 -0.134 0.5305" rpy="0 -${M_PI} 0.0" /> <!-- yaw=-0.026 -->
       <axis xyz="0 -1 0" />
-      <limit lower="0" upper="${M_PI/2}" effort="100" velocity="1.0"/>
-      <dynamics damping="200.5"/>
+      <limit lower="0" upper="${M_PI/2}" effort="1000.0" velocity="10.0"/>
+      <dynamics damping="30.0"/>
     </joint>
     <xacro:shadowarm_upperarm_transmission />
