Commit message: latest changes

File: arm/xacro/hand_support/shadowarm_handsupport_motor.transmission.xacro (robot description, xacro)
@@ -5,11 +5,11 @@
        xmlns:xacro="http://ros.org/wiki/xacro">
   <xacro:macro name="shadowarm_handsupport_motor_transmission">
-    <transmission type="sr_mechanism_model/SimpleTransmission" name="forearm_rotation_transmission">
-      <actuator name="forearm_rotation" />
-      <joint name="ElbowJRotate" />
-      <mechanicalReduction>1</mechanicalReduction>
-      <motorTorqueConstant>1</motorTorqueConstant>
-      <pulsesPerRevolution>90000</pulsesPerRevolution>
-    </transmission>
+    <transmission name="forearm_rotation_transmission">
+	  <type>sr_mechanism_model/SimpleTransmission</type>
+	  <joint name="ElbowJRotate"/>
+	  <actuator name="forearm_rotation">
+	    <hardwareInterface>Robot</hardwareInterface>
+	  </actuator>
+	</transmission>
   </xacro:macro>
 </robot>

File: arm/xacro/hand_support/shadowarm_handsupport_muscle.transmission.xacro (robot description, xacro)
@@ -5,11 +5,11 @@
        xmlns:xacro="http://ros.org/wiki/xacro">
   <xacro:macro name="shadowarm_handsupport_muscle_transmission">
-    <transmission type="sr_mechanism_model/SimpleTransmission" name="forearm_rotation_transmission">
-      <actuator name="forearm_rotation" />
-      <joint name="ElbowJRotate" />
-      <mechanicalReduction>1</mechanicalReduction>
-      <motorTorqueConstant>1</motorTorqueConstant>
-      <pulsesPerRevolution>90000</pulsesPerRevolution>
-    </transmission>
+    <transmission name="forearm_rotation_transmission">
+	  <type>sr_mechanism_model/SimpleTransmission</type>
+	  <joint name="ElbowJRotate"/>
+	  <actuator name="forearm_rotation">
+	    <hardwareInterface>Robot</hardwareInterface>
+	  </actuator>
+	</transmission>
   </xacro:macro>
 </robot>

File: arm/xacro/lower_arm/shadowarm_lowerarm.transmission.xacro (robot description, xacro)
@@ -5,11 +5,11 @@
        xmlns:xacro="http://ros.org/wiki/xacro">
   <xacro:macro name="shadowarm_lowerarm_transmission">
-    <transmission type="sr_mechanism_model/SimpleTransmission" name="elbow_abduction_transmission">
-      <actuator name="elbow_abduction" />
-      <joint name="ElbowJSwing" />
-      <mechanicalReduction>1</mechanicalReduction>
-      <motorTorqueConstant>1</motorTorqueConstant>
-      <pulsesPerRevolution>90000</pulsesPerRevolution>
-    </transmission>
+    <transmission name="elbow_abduction_transmission">
+	  <type>sr_mechanism_model/SimpleTransmission</type>
+	  <joint name="ElbowJSwing"/>
+	  <actuator name="elbow_abduction">
+	    <hardwareInterface>Robot</hardwareInterface>
+	  </actuator>
+	</transmission>
   </xacro:macro>
 </robot>

File: arm/xacro/trunk/shadowarm_trunk.transmission.xacro (robot description, xacro)
@@ -5,11 +5,11 @@
        xmlns:xacro="http://ros.org/wiki/xacro">
   <xacro:macro name="shadowarm_trunk_transmission">
-    <transmission type="sr_mechanism_model/SimpleTransmission" name="trunk_rotation_transmission">
-      <actuator name="trunk_rotation" />
-      <joint name="ShoulderJRotate" />
-      <mechanicalReduction>1</mechanicalReduction>
-      <motorTorqueConstant>1</motorTorqueConstant>
-      <pulsesPerRevolution>90000</pulsesPerRevolution>
-    </transmission>
+    <transmission name="trunk_rotation_transmission">
+	  <type>sr_mechanism_model/SimpleTransmission</type>
+	  <joint name="ShoulderJRotate"/>
+	  <actuator name="trunk_rotation">
+	    <hardwareInterface>Robot</hardwareInterface>
+	  </actuator>
+	</transmission>
   </xacro:macro>
 </robot>

File: arm/xacro/upper_arm/shadowarm_upperarm.transmission.xacro (robot description, xacro)
@@ -5,11 +5,11 @@
        xmlns:xacro="http://ros.org/wiki/xacro">
   <xacro:macro name="shadowarm_upperarm_transmission">
-    <transmission type="sr_mechanism_model/SimpleTransmission" name="shoulder_rotation_transmission">
-      <actuator name="shoulder_rotation" />
-      <joint name="ShoulderJSwing" />
-      <mechanicalReduction>1</mechanicalReduction>
-      <motorTorqueConstant>1</motorTorqueConstant>
-      <pulsesPerRevolution>90000</pulsesPerRevolution>
-    </transmission>
+    <transmission name="shoulder_rotation_transmission">
+	  <type>sr_mechanism_model/SimpleTransmission</type>
+	  <joint name="ShoulderJSwing"/>
+	  <actuator name="shoulder_rotation">
+	    <hardwareInterface>Robot</hardwareInterface>
+	  </actuator>
+	</transmission>
   </xacro:macro>
 </robot>

File: hand/xacro/finger/biotac/biotac.transmission.xacro (robot description, xacro)
@@ -9,12 +9,12 @@
        even if the actual BioTAC hand doesn't even have J1.
   -->
-    <transmission type="sr_mechanism_model/J0Transmission" name="${link_prefix}middle_transmission">
-      <actuator name="${joint_prefix}J0" />
+    <transmission name="${link_prefix}middle_transmission">
+	  <type>sr_mechanism_model/J0Transmission</type>
       <joint1 name="${joint_prefix}J1" />
       <joint2 name="${joint_prefix}J2" />
-      <mechanicalReduction>1</mechanicalReduction>
-      <motorTorqueConstant>1</motorTorqueConstant>
-      <pulsesPerRevolution>90000</pulsesPerRevolution>
-    </transmission>
+	  <actuator name="${joint_prefix}J0">
+	    <hardwareInterface>Robot</hardwareInterface>
+	  </actuator>
+	</transmission>
   </xacro:macro>
 </robot>

File: hand/xacro/finger/biotac/edc_muscle_biotac.transmission.xacro (robot description, xacro)
@@ -9,12 +9,12 @@
        even if the actual BioTAC hand doesn't even have J1.
   -->
-    <transmission type="sr_mechanism_model/J0TransmissionForMuscle" name="${link_prefix}middle_transmission">
-      <actuator name="${joint_prefix}J0" />
+    <transmission name="${link_prefix}middle_transmission">
+	  <type>sr_mechanism_model/J0TransmissionForMuscle</type>
       <joint1 name="${joint_prefix}J1" />
       <joint2 name="${joint_prefix}J2" />
-      <mechanicalReduction>1</mechanicalReduction>
-      <motorTorqueConstant>1</motorTorqueConstant>
-      <pulsesPerRevolution>90000</pulsesPerRevolution>
-    </transmission>
+      <actuator name="${joint_prefix}J0">
+	    <hardwareInterface>Robot</hardwareInterface>
+	  </actuator>
+	</transmission>
   </xacro:macro>
 </robot>

File: hand/xacro/finger/distal/distal.transmission.xacro (robot description, xacro)
@@ -5,11 +5,11 @@
        xmlns:xacro="http://ros.org/wiki/xacro">
   <xacro:macro name="distal_transmission">
-    <transmission type="sr_mechanism_model/SimpleTransmission" name="${link_prefix}distal_transmission">
-      <actuator name="${joint_prefix}J1" />
-      <joint name="${joint_prefix}J1" />
-      <mechanicalReduction>1</mechanicalReduction>
-      <motorTorqueConstant>1</motorTorqueConstant>
-      <pulsesPerRevolution>90000</pulsesPerRevolution>
-    </transmission>
+    <transmission name="${link_prefix}distal_transmission">
+	  <type>sr_mechanism_model/SimpleTransmission</type>
+	  <joint name="${joint_prefix}J1" />
+	  <actuator name="${joint_prefix}J1">
+	    <hardwareInterface>Robot</hardwareInterface>
+	  </actuator>
+	</transmission>
   </xacro:macro>
 </robot>

File: hand/xacro/finger/knuckle/edc_muscle_knuckle.transmission.xacro (robot description, xacro)
@@ -5,11 +5,11 @@
        xmlns:xacro="http://ros.org/wiki/xacro">
   <xacro:macro name="knuckle_transmission">
-    <transmission type="sr_mechanism_model/SimpleTransmissionForMuscle" name="${link_prefix}knuckle_transmission">
-      <actuator name="${joint_prefix}J4" />
-      <joint name="${joint_prefix}J4" />
-      <mechanicalReduction>1</mechanicalReduction>
-      <motorTorqueConstant>1</motorTorqueConstant>
-      <pulsesPerRevolution>90000</pulsesPerRevolution>
-    </transmission>
+    <transmission name="${link_prefix}knuckle_transmission">
+	  <type>sr_mechanism_model/SimpleTransmissionForMuscle</type>
+	  <joint name="${joint_prefix}J4" />
+	  <actuator name="${joint_prefix}J4">
+	    <hardwareInterface>Robot</hardwareInterface>
+	  </actuator>
+	</transmission>
   </xacro:macro>
 </robot>

File: hand/xacro/finger/knuckle/knuckle.transmission.xacro (robot description, xacro)
@@ -5,10 +5,10 @@
        xmlns:xacro="http://ros.org/wiki/xacro">
   <xacro:macro name="knuckle_transmission">
-    <transmission type="sr_mechanism_model/SimpleTransmission" name="${link_prefix}knuckle_transmission">
-      <actuator name="${joint_prefix}J4" />
+    <transmission name="${link_prefix}knuckle_transmission">
+      <type>sr_mechanism_model/SimpleTransmission</type>
       <joint name="${joint_prefix}J4" />
-      <mechanicalReduction>1</mechanicalReduction>
-      <motorTorqueConstant>1</motorTorqueConstant>
-      <pulsesPerRevolution>90000</pulsesPerRevolution>
+	  <actuator name="${joint_prefix}J4">
+	  	<hardwareInterface>Robot</hardwareInterface>
+	  </actuator>
     </transmission>
   </xacro:macro>

File: hand/xacro/finger/lfmetacarpal/edc_muscle_lfmetacarpal.transmission.xacro (robot description, xacro)
@@ -5,10 +5,10 @@
        xmlns:xacro="http://ros.org/wiki/xacro">
   <xacro:macro name="lfmetacarpal_transmission">
-    <transmission type="sr_mechanism_model/SimpleTransmissionForMuscle" name="lfmetacarpal_transmission">
-      <actuator name="LFJ5" />
-      <joint name="LFJ5" />
-      <mechanicalReduction>1</mechanicalReduction>
-      <motorTorqueConstant>1</motorTorqueConstant>
-      <pulsesPerRevolution>90000</pulsesPerRevolution>
+    <transmission name="lfmetacarpal_transmission">
+      <type>sr_mechanism_model/SimpleTransmissionForMuscle</type>
+      <joint name="LFJ5"/>
+      <actuator name="LFJ5">
+    	<hardwareInterface>Robot</hardwareInterface>
+	  </actuator>
     </transmission>
   </xacro:macro>

File: hand/xacro/finger/lfmetacarpal/lfmetacarpal.transmission.xacro (robot description, xacro)
@@ -5,10 +5,10 @@
        xmlns:xacro="http://ros.org/wiki/xacro">
   <xacro:macro name="lfmetacarpal_transmission">
-    <transmission type="sr_mechanism_model/SimpleTransmission" name="lfmetacarpal_transmission">
-      <actuator name="LFJ5" />
-      <joint name="LFJ5" />
-      <mechanicalReduction>1</mechanicalReduction>
-      <motorTorqueConstant>1</motorTorqueConstant>
-      <pulsesPerRevolution>90000</pulsesPerRevolution>
+    <transmission name="lfmetacarpal_transmission">
+      <type>sr_mechanism_model/SimpleTransmission</type>
+      <joint name="LFJ5"/>
+	  <actuator name="LFJ5">
+	  	<hardwareInterface>Robot</hardwareInterface>
+	  </actuator>
     </transmission>
   </xacro:macro>

File: hand/xacro/finger/little_finger_ellipsoid.urdf.xacro (robot description, xacro)
@@ -60,11 +60,11 @@
       <dynamics damping="10.0"/>
     </joint>
-    <transmission type="sr_mechanism_model/SimpleTransmission" name="lfknuckle_transmission">
-      <actuator name="LFJ4" />
-      <joint name="LFJ4" />
-      <mechanicalReduction>1</mechanicalReduction>
-      <motorTorqueConstant>1</motorTorqueConstant>
-      <pulsesPerRevolution>90000</pulsesPerRevolution>
-    </transmission>
+    <transmission name="lfknuckle_transmission">
+	  <type>sr_mechanism_model/SimpleTransmission</type>
+	  <joint name="LFJ4"/>
+	  <actuator name="LFJ4">
+	    <hardwareInterface>Robot</hardwareInterface>
+	  </actuator>
+	</transmission>
     <xacro:proximal link_prefix="${link_prefix}" joint_prefix="${joint_prefix}" parent="${link_prefix}knuckle" >
     </xacro:proximal>

File: hand/xacro/finger/middle/middle.transmission.xacro (robot description, xacro)
@@ -5,12 +5,12 @@
        xmlns:xacro="http://ros.org/wiki/xacro">
   <xacro:macro name="middle_transmission">
-    <transmission type="sr_mechanism_model/J0Transmission" name="${link_prefix}middle_transmission">
-      <actuator name="${joint_prefix}J0" />
-      <joint1 name="${joint_prefix}J1" />
-      <joint2 name="${joint_prefix}J2" />
-      <mechanicalReduction>1</mechanicalReduction>
-      <motorTorqueConstant>1</motorTorqueConstant>
-      <pulsesPerRevolution>90000</pulsesPerRevolution>
-    </transmission>
+    <transmission name="${link_prefix}middle_transmission">
+      <type>sr_mechanism_model/J0Transmission</type>
+      <joint1 name="${joint_prefix}J1"/>
+      <joint2 name="${joint_prefix}J2"/>
+      <actuator name="${joint_prefix}J0">
+	    <hardwareInterface>Robot</hardwareInterface>
+	  </actuator>
+	</transmission>
   </xacro:macro>
 </robot>

File: hand/xacro/finger/proximal/edc_muscle_proximal.transmission.xacro (robot description, xacro)
@@ -5,11 +5,11 @@
        xmlns:xacro="http://ros.org/wiki/xacro">
   <xacro:macro name="proximal_transmission">
-    <transmission type="sr_mechanism_model/SimpleTransmissionForMuscle" name="${link_prefix}proximal_transmission">
-      <actuator name="${joint_prefix}J3" />
-      <joint name="${joint_prefix}J3" />
-      <mechanicalReduction>1</mechanicalReduction>
-      <motorTorqueConstant>1</motorTorqueConstant>
-      <pulsesPerRevolution>90000</pulsesPerRevolution>
-    </transmission>
+    <transmission name="${link_prefix}proximal_transmission">
+      <type>sr_mechanism_model/SimpleTransmissionForMuscle</type>
+      <joint name="${joint_prefix}J3"/>
+	  <actuator name="${joint_prefix}J3">
+	  	<hardwareInterface>Robot</hardwareInterface>
+	  </actuator>
+	</transmission>
   </xacro:macro>
 </robot>

File: hand/xacro/finger/proximal/proximal.transmission.xacro (robot description, xacro)
@@ -5,11 +5,11 @@
        xmlns:xacro="http://ros.org/wiki/xacro">
   <xacro:macro name="proximal_transmission">
-    <transmission type="sr_mechanism_model/SimpleTransmission" name="${link_prefix}proximal_transmission">
-      <actuator name="${joint_prefix}J3" />
-      <joint name="${joint_prefix}J3" />
-      <mechanicalReduction>1</mechanicalReduction>
-      <motorTorqueConstant>1</motorTorqueConstant>
-      <pulsesPerRevolution>90000</pulsesPerRevolution>
-    </transmission>
+    <transmission name="${link_prefix}proximal_transmission">
+      <type>sr_mechanism_model/SimpleTransmission</type>
+      <joint name="${joint_prefix}J3"/>
+	  <actuator name="${joint_prefix}J3">
+        <hardwareInterface>Robot</hardwareInterface>
+	  </actuator>
+	</transmission>
   </xacro:macro>
 </robot>

File: hand/xacro/palm/edc_muscle_palm.transmission.xacro (robot description, xacro)
@@ -5,11 +5,11 @@
        xmlns:xacro="http://ros.org/wiki/xacro">
   <xacro:macro name="shadowhand_palm_transmission">
-    <transmission type="sr_mechanism_model/SimpleTransmissionForMuscle" name="palm_transmission">
-      <actuator name="WRJ1" />
-      <joint name="WRJ1" />
-      <mechanicalReduction>1</mechanicalReduction>
-      <motorTorqueConstant>1</motorTorqueConstant>
-      <pulsesPerRevolution>90000</pulsesPerRevolution>
-    </transmission>
+    <transmission name="palm_transmission">
+	  <type>sr_mechanism_model/SimpleTransmissionForMuscle</type>
+	  <joint name="WRJ1"/>
+	  <actuator name="WRJ1">
+	    <hardwareInterface>Robot</hardwareInterface>
+	  </actuator>
+	</transmission>
   </xacro:macro>
 </robot>

File: hand/xacro/palm/palm.transmission.xacro (robot description, xacro)
@@ -5,11 +5,11 @@
        xmlns:xacro="http://ros.org/wiki/xacro">
   <xacro:macro name="shadowhand_palm_transmission">
-    <transmission type="sr_mechanism_model/SimpleTransmission" name="palm_transmission">
-      <actuator name="WRJ1" />
-      <joint name="WRJ1" />
-      <mechanicalReduction>1</mechanicalReduction>
-      <motorTorqueConstant>1</motorTorqueConstant>
-      <pulsesPerRevolution>90000</pulsesPerRevolution>
-    </transmission>
+    <transmission name="palm_transmission">
+	  <type>sr_mechanism_model/SimpleTransmission</type>
+	  <joint name="WRJ1"/>
+	  <actuator name="WRJ1">
+	    <hardwareInterface>Robot</hardwareInterface>
+	  </actuator>
+	</transmission>
   </xacro:macro>
 </robot>

File: hand/xacro/thumb/edc_muscle_thbase.transmission.xacro (robot description, xacro)
@@ -5,11 +5,11 @@
        xmlns:xacro="http://ros.org/wiki/xacro">
   <xacro:macro name="thbase_transmission">
-    <transmission type="sr_mechanism_model/SimpleTransmissionForMuscle" name="thbase_transmission">
-      <actuator name="THJ5" />
-      <joint name="THJ5" />
-      <mechanicalReduction>1</mechanicalReduction>
-      <motorTorqueConstant>1</motorTorqueConstant>
-      <pulsesPerRevolution>90000</pulsesPerRevolution>
-    </transmission>
+    <transmission name="thbase_transmission">
+	  <type>sr_mechanism_model/SimpleTransmissionForMuscle</type>
+	  <joint name="THJ5"/>
+	  <actuator name="THJ5">
+	    <hardwareInterface>Robot</hardwareInterface>
+	  </actuator>
+	</transmission>
   </xacro:macro>
 </robot>

File: hand/xacro/thumb/edc_muscle_thbiotac.urdf.xacro (robot description, xacro)
@@ -61,11 +61,11 @@
       <dynamics damping="10.0"/>
     </joint>
-    <transmission type="sr_mechanism_model/SimpleTransmissionForMuscle" name="thmiddle_transmission">
-      <actuator name="THJ2" />
-      <joint name="THJ2" />
-      <mechanicalReduction>1</mechanicalReduction>
-      <motorTorqueConstant>1</motorTorqueConstant>
-      <pulsesPerRevolution>90000</pulsesPerRevolution>
-    </transmission>
+    <transmission name="thmiddle_transmission">
+	  <type>sr_mechanism_model/SimpleTransmissionForMuscle</type>
+	  <joint name="THJ2"/>
+	  <actuator name="THJ2">
+	    <hardwareInterface>Robot</hardwareInterface>
+	  </actuator>
+	</transmission>
     <link name="thbiotac_J1_dummy">
       <inertial>
@@ -83,11 +83,11 @@
       <dynamics damping="10.0"/>
     </joint>
-    <transmission type="sr_mechanism_model/SimpleTransmissionForMuscle" name="thdistal_transmission">
-      <actuator name="THJ1" />
-      <joint name="THJ1" />
-      <mechanicalReduction>1</mechanicalReduction>
-      <motorTorqueConstant>1</motorTorqueConstant>
-      <pulsesPerRevolution>90000</pulsesPerRevolution>
-    </transmission>
+    <transmission name="thdistal_transmission">
+	  <type>sr_mechanism_model/SimpleTransmissionForMuscle</type>
+	  <joint name="THJ1"/>
+	  <actuator name="THJ1">
+	    <hardwareInterface>Robot</hardwareInterface>
+	  </actuator>
+	</transmission>
     <link name="thbiotac">
       <inertial>
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