Commit message: updated sensor urdf the hand is now spawning in gazebo

File: hand/xacro/finger/distal/distal.urdf.xacro (robot description, xacro)
@@ -17,5 +17,5 @@
       <visual>
 	<origin xyz="0 0 0" rpy="0 0 0" />
-	<geometry name="distal_visual">
+	<geometry name="${link_prefix}distal_visual">
       <mesh filename="package://sr_description/hand/model/F1.dae" scale="0.001 0.001 0.001" />
       </geometry>
@@ -24,5 +24,5 @@
       <collision>
 	<origin xyz="0 0 0" rpy="0 0 0" />
-	<geometry name="distal_collision_geom">
+	<geometry name="${link_prefix}distal_collision_geom">
 	 <mesh filename="package://sr_description/hand/model/F1.dae" scale="0.001 0.001 0.001" />
 	</geometry>
@@ -30,15 +30,16 @@
     </link>
     <gazebo reference="${link_prefix}distal">
-      <sensor:contact name="${link_prefix}distal_contact_sensor">
-        <geom>${link_prefix}distal_geom</geom>
-        <updateRate>100.0</updateRate>
-        <controller:gazebo_ros_bumper name="${link_prefix}distal_gazebo_ros_bumper_controller" plugin="libgazebo_ros_bumper.so">
+      <sensor type="contact" name="${link_prefix}distal_contact_sensor">
+        <update_rate>100.0</update_rate>
+        <contact>
+          <collision>${link_prefix}distal_collision_geom</collision>
+        </contact>
+        <plugin name="${link_prefix}distal_gazebo_ros_bumper_controller" filename="libgazebo_ros_bumper.so">
           <alwaysOn>true</alwaysOn>
+          <frameName>${link_prefix}distal</frameName>
           <updateRate>100.0</updateRate>
-          <frameName>${link_prefix}distal</frameName>
           <bumperTopicName>${link_prefix}distal_bumper</bumperTopicName>
-          <interface:bumper name="${link_prefix}distal_gazebo_ros_bumper_iface" />
-        </controller:gazebo_ros_bumper>
-      </sensor:contact>
+        </plugin>
+      </sensor>
       <mu1 value="500.0" />
       <mu2 value="500.0" />

File: hand/xacro/finger/knuckle/knuckle.urdf.xacro (robot description, xacro)
@@ -18,5 +18,5 @@
       <visual>
 	<origin xyz="0 0 0.0005" rpy="0 0 0" />
-	<geometry name="knuckle_visual">
+	<geometry name="${link_prefix}knuckle_visual">
       <mesh filename="package://sr_description/hand/model/knuckle.dae" scale="0.001 0.001 0.001" />
       </geometry>
@@ -25,5 +25,5 @@
       <collision>
 	<origin xyz="0 0 0" rpy="0 0 0" />
-	<geometry name="knuckle_collision_geom">
+	<geometry name="${link_prefix}knuckle_collision_geom">
 	  <box size="0.005 0.005 0.005" />
 	</geometry>
@@ -31,16 +31,17 @@
     </link>
     <gazebo reference="${link_prefix}knuckle">
-      <sensor:contact name="${link_prefix}knuckle_contact_sensor">
-        <geom>${link_prefix}knuckle_geom</geom>
-       <updateRate>100.0</updateRate>
-        <controller:gazebo_ros_bumper name="${link_prefix}knuckle_gazebo_ros_bumper_controller" plugin="libgazebo_ros_bumper.so">
+      <sensor type="contact" name="${link_prefix}knuckle_contact_sensor">
+        <update_rate>100.0</update_rate>
+        <contact>
+          <collision>${link_prefix}knuckle_collision_geom</collision>
+        </contact>
+        <plugin name="${link_prefix}knuckle_gazebo_ros_bumper_controller" filename="libgazebo_ros_bumper.so">
           <alwaysOn>true</alwaysOn>
+          <frameName>${link_prefix}knuckle</frameName>
           <updateRate>100.0</updateRate>
-          <frameName>${link_prefix}knuckle</frameName>
           <bumperTopicName>${link_prefix}knuckle_bumper</bumperTopicName>
-          <interface:bumper name="${link_prefix}knuckle_gazebo_ros_bumper_iface" />
-        </controller:gazebo_ros_bumper>
-      </sensor:contact>
-      <material>PR2/Grey2</material>
+        </plugin>
+      </sensor>
+      <material>Gazebo/Grey</material>
     </gazebo>
     <joint name="${joint_prefix}J4" type="revolute">

File: hand/xacro/finger/lfmetacarpal/lfmetacarpal.urdf.xacro (robot description, xacro)
@@ -39,15 +39,16 @@
     </link>
     <gazebo reference="lfmetacarpal">
-      <sensor:contact name="lfmetacarpal_contact_sensor">
-        <geom>lfmetacarpal_geom</geom>
-       <updateRate>100.0</updateRate>
-        <controller:gazebo_ros_bumper name="lfmetacarpal_gazebo_ros_bumper_controller" plugin="libgazebo_ros_bumper.so">
+      <sensor type="contact" name="lfmetacarpal_contact_sensor">
+        <update_rate>100.0</update_rate>
+        <contact>
+          <collision>lfmetacarpal_collision_geom</collision>
+        </contact>
+        <plugin name="lfmetacarpal_gazebo_ros_bumper_controller" filename="libgazebo_ros_bumper.so">
           <alwaysOn>true</alwaysOn>
+          <frameName>lfmetacarpal</frameName>
           <updateRate>100.0</updateRate>
-          <frameName>lfmetacarpal</frameName>
           <bumperTopicName>lfmetacarpal_bumper</bumperTopicName>
-          <interface:bumper name="lfmetacarpal_gazebo_ros_bumper_iface" />
-        </controller:gazebo_ros_bumper>
-      </sensor:contact>
+        </plugin>
+      </sensor>
       <material>Gazebo/Grey</material>
     </gazebo>

File: hand/xacro/finger/little_finger.urdf.xacro (robot description, xacro)
@@ -46,16 +46,17 @@
     </link>
     <gazebo reference="lfknuckle">
-      <sensor:contact name="lfknuckle_contact_sensor">
-        <geom>lfknuckle_geom</geom>
-        <updateRate>100.0</updateRate>
-        <controller:gazebo_ros_bumper name="lfknuckle_gazebo_ros_bumper_controller" plugin="libgazebo_ros_bumper.so">
+      <sensor type="contact" name="lfknuckle_contact_sensor">
+        <update_rate>100.0</update_rate>
+        <contact>
+          <collision>lfknuckle_collision_geom</collision>
+        </contact>
+        <plugin name="lfknuckle_gazebo_ros_bumper_controller" filename="libgazebo_ros_bumper.so">
           <alwaysOn>true</alwaysOn>
+          <frameName>lfknuckle</frameName>
           <updateRate>100.0</updateRate>
-          <frameName>lfknuckle</frameName>
           <bumperTopicName>lfknuckle_bumper</bumperTopicName>
-          <interface:bumper name="lfknuckle_gazebo_ros_bumper_iface" />
-        </controller:gazebo_ros_bumper>
-      </sensor:contact>
-      <material>PR2/Grey2</material>
+        </plugin>
+      </sensor>
+      <material>Gazebo/Grey</material>
     </gazebo>
     <joint name="LFJ4" type="revolute">

File: hand/xacro/finger/middle/middle.urdf.xacro (robot description, xacro)
@@ -17,5 +17,5 @@
       <visual>
 	<origin xyz="0 0 0" rpy="0 0 0" />
-	<geometry name="middle_visual">
+	<geometry name="${link_prefix}middle_visual">
       <mesh filename="package://sr_description/hand/model/F2.dae" scale="0.001 0.001 0.001" />
       </geometry>
@@ -24,5 +24,5 @@
       <collision>
 	<origin xyz="0 0 0.0125" rpy="0 0 0" />
-	<geometry name="middle_collision_geom">
+	<geometry name="${link_prefix}middle_collision_geom">
 	  <box size="0.008 0.008 0.015" />
 	</geometry>
@@ -30,15 +30,16 @@
     </link>
     <gazebo reference="${link_prefix}middle">
-      <sensor:contact name="${link_prefix}middle_contact_sensor">
-        <geom>${link_prefix}middle_geom</geom>
-       <updateRate>100.0</updateRate>
-        <controller:gazebo_ros_bumper name="${link_prefix}middle_gazebo_ros_bumper_controller" plugin="libgazebo_ros_bumper.so">
+      <sensor type="contact" name="${link_prefix}middle_contact_sensor">
+        <update_rate>100.0</update_rate>
+        <contact>
+          <collision>${link_prefix}middle_collision_geom</collision>
+        </contact>
+        <plugin name="${link_prefix}middle_gazebo_ros_bumper_controller" filename="libgazebo_ros_bumper.so">
           <alwaysOn>true</alwaysOn>
+          <frameName>${link_prefix}middle</frameName>
           <updateRate>100.0</updateRate>
-          <frameName>${link_prefix}middle</frameName>
           <bumperTopicName>${link_prefix}middle_bumper</bumperTopicName>
-          <interface:bumper name="${link_prefix}middle_gazebo_ros_bumper_iface" />
-        </controller:gazebo_ros_bumper>
-      </sensor:contact>
+        </plugin>
+      </sensor>
       <material>Gazebo/Grey</material>
       <selfCollide>true</selfCollide>

File: hand/xacro/finger/proximal/proximal.urdf.xacro (robot description, xacro)
@@ -30,15 +30,16 @@
     </link>
     <gazebo reference="${link_prefix}proximal">
-      <sensor:contact name="${link_prefix}proximal_contact_sensor">
-        <geom>${link_prefix}proximal_geom</geom>
-       <updateRate>100.0</updateRate>
-        <controller:gazebo_ros_bumper name="${link_prefix}proximal_gazebo_ros_bumper_controller" plugin="libgazebo_ros_bumper.so">
+      <sensor type="contact" name="${link_prefix}proximal_contact_sensor">
+        <update_rate>100.0</update_rate>
+        <contact>
+          <collision>${link_prefix}proximal_collision_geom</collision>
+        </contact>
+        <plugin name="${link_prefix}proximal_gazebo_ros_bumper_controller" filename="libgazebo_ros_bumper.so">
           <alwaysOn>true</alwaysOn>
+          <frameName>${link_prefix}proximal</frameName>
           <updateRate>100.0</updateRate>
-          <frameName>${link_prefix}proximal</frameName>
           <bumperTopicName>${link_prefix}proximal_bumper</bumperTopicName>
-          <interface:bumper name="${link_prefix}proximal_gazebo_ros_bumper_iface" />
-        </controller:gazebo_ros_bumper>
-      </sensor:contact>
+        </plugin>
+      </sensor>
       <material>Gazebo/Grey</material>
       <selfCollide>true</selfCollide>

File: hand/xacro/palm/palm.urdf.xacro (robot description, xacro)
@@ -39,15 +39,16 @@
     </link>
     <gazebo reference="palm">
-      <sensor:contact name="palm_contact_sensor">
-       <geom>palm_geom</geom>
-       <updateRate>100.0</updateRate>
-       <controller:gazebo_ros_bumper name="palm_gazebo_ros_bumper_controller" plugin="libgazebo_ros_bumper.so">
+      <sensor type="contact" name="palm_contact_sensor">
+        <update_rate>100.0</update_rate>
+        <contact>
+          <collision>palm_collision_geom</collision>
+        </contact>
+        <plugin name="palm_gazebo_ros_bumper_controller" filename="libgazebo_ros_bumper.so">
           <alwaysOn>true</alwaysOn>
+          <frameName>palm</frameName>
           <updateRate>100.0</updateRate>
-          <frameName>palm</frameName>
           <bumperTopicName>palm_bumper</bumperTopicName>
-          <interface:bumper name="palm_gazebo_ros_bumper_iface" />
-       </controller:gazebo_ros_bumper>
-      </sensor:contact>
+        </plugin>
+      </sensor>
       <material>Gazebo/Grey</material>
     </gazebo>

File: hand/xacro/thumb/thbase.urdf.xacro (robot description, xacro)
@@ -42,15 +42,16 @@
     </link>
     <gazebo reference="thbase">
-      <sensor:contact name="thbase_contact_sensor">
-        <geom>thbase_geom</geom>
-       <updateRate>100.0</updateRate>
-        <controller:gazebo_ros_bumper name="thbase_gazebo_ros_bumper_controller" plugin="libgazebo_ros_bumper.so">
+      <sensor type="contact" name="thbase_contact_sensor">
+        <update_rate>100.0</update_rate>
+        <contact>
+          <collision>thbase_collision_geom</collision>
+        </contact>
+        <plugin name="thbase_gazebo_ros_bumper_controller" filename="libgazebo_ros_bumper.so">
           <alwaysOn>true</alwaysOn>
+          <frameName>thbase</frameName>
           <updateRate>100.0</updateRate>
-          <frameName>thbase</frameName>
           <bumperTopicName>thbase_bumper</bumperTopicName>
-          <interface:bumper name="thbase_gazebo_ros_bumper_iface" />
-        </controller:gazebo_ros_bumper>
-      </sensor:contact>
+        </plugin>
+      </sensor>
       <material>Gazebo/Grey</material>
     </gazebo>

File: hand/xacro/thumb/thbiotac.urdf.xacro (robot description, xacro)
@@ -37,16 +37,17 @@
     </link>
     <gazebo reference="thmiddle">
-      <sensor:contact name="thmiddle_contact_sensor">
-        <geom>thmiddle_geom</geom>
-       <updateRate>100.0</updateRate>
-        <controller:gazebo_ros_bumper name="thmiddle_gazebo_ros_bumper_controller" plugin="libgazebo_ros_bumper.so">
+      <sensor type="contact" name="thmiddle_contact_sensor">
+        <update_rate>100.0</update_rate>
+        <contact>
+          <collision>thmiddle_collision_geom</collision>
+        </contact>
+        <plugin name="thmiddle_gazebo_ros_bumper_controller" filename="libgazebo_ros_bumper.so">
           <alwaysOn>true</alwaysOn>
+          <frameName>thmiddle</frameName>
           <updateRate>100.0</updateRate>
-          <frameName>thmiddle</frameName>
           <bumperTopicName>thmiddle_bumper</bumperTopicName>
-          <interface:bumper name="thmiddle_gazebo_ros_bumper_iface" />
-        </controller:gazebo_ros_bumper>
-      </sensor:contact>
-      <material name="Grey"/>
+        </plugin>
+      </sensor>
+      <material>Gazebo/Grey</material>
     </gazebo>
     <joint name="THJ2" type="revolute">

File: hand/xacro/thumb/thdistal.urdf.xacro (robot description, xacro)
@@ -33,15 +33,17 @@
     </link>
     <gazebo reference="thdistal">
-      <sensor:contact name="thdistal_contact_sensor">
-        <geom>thdistal_geom</geom>
-	<updateRate>100.0</updateRate>
-        <controller:gazebo_ros_bumper name="thdistal_gazebo_ros_bumper_controller" plugin="libgazebo_ros_bumper.so">
+      <sensor type="contact" name="thdistal_contact_sensor">
+        <update_rate>100.0</update_rate>
+        <contact>
+          <collision>thdistal_collision_geom</collision>
+        </contact>
+        <plugin name="thdistal_gazebo_ros_bumper_controller" filename="libgazebo_ros_bumper.so">
           <alwaysOn>true</alwaysOn>
+          <frameName>thdistal</frameName>
           <updateRate>100.0</updateRate>
-          <frameName>thdistal</frameName>
           <bumperTopicName>thdistal_bumper</bumperTopicName>
-          <interface:bumper name="thdistal_gazebo_ros_bumper_iface" />
-        </controller:gazebo_ros_bumper>
-      </sensor:contact>
+        </plugin>
+      </sensor>
+      <material>Gazebo/Grey</material>
       <mu1 value="500.0" />
       <mu2 value="500.0" />

File: hand/xacro/thumb/thdistal_ellipsoid.urdf.xacro (robot description, xacro)
@@ -20,5 +20,5 @@
 	  <mesh filename="package://sr_description/hand/model/distal_ellipsoid.dae" scale="0.001 0.001 0.001" />
 	</geometry>
-	<material name="shadow_thmiddle_material">
+	<material name="shadow_thdistal_material">
 	  <color rgba="0.2 0.2 0.2 1.0"/>
 	</material>
@@ -26,5 +26,5 @@
       <collision>
 	<origin xyz="0 0.002 0.0025" rpy="0 0 0 " />
-	<geometry name="thmiddle_collision_geom">
+	<geometry name="thdistal_collision_geom">
 	  <mesh filename="package://sr_description/hand/model/distal_ellipsoid.dae" scale="0.001 0.001 0.001" />
 	</geometry>
@@ -32,15 +32,18 @@
     </link>
     <gazebo reference="thdistal">
-      <sensor:contact name="thdistal_contact_sensor">
-        <geom>thdistal_geom</geom>
-	<updateRate>100.0</updateRate>
-        <controller:gazebo_ros_bumper name="thdistal_gazebo_ros_bumper_controller" plugin="libgazebo_ros_bumper.so">
+      <sensor type="contact" name="thdistal_contact_sensor">
+        <update_rate>100.0</update_rate>
+        <contact>
+          <collision>thdistal_collision_geom</collision>
+        </contact>
+        <plugin name="thdistal_gazebo_ros_bumper_controller" filename="libgazebo_ros_bumper.so">
           <alwaysOn>true</alwaysOn>
+          <frameName>thdistal</frameName>
           <updateRate>100.0</updateRate>
-          <frameName>thdistal</frameName>
           <bumperTopicName>thdistal_bumper</bumperTopicName>
-          <interface:bumper name="thdistal_gazebo_ros_bumper_iface" />
-        </controller:gazebo_ros_bumper>
-      </sensor:contact>
+        </plugin>
+      </sensor>
+      <material>Gazebo/Grey</material>
+    </gazebo>
       <mu1 value="500.0" />
       <mu2 value="500.0" />

File: hand/xacro/thumb/thhub.urdf.xacro (robot description, xacro)
@@ -32,15 +32,16 @@
     </link>
     <gazebo reference="thhub">
-      <sensor:contact name="thhub_contact_sensor">
-        <geom>thhub_geom</geom>
-       <updateRate>100.0</updateRate>
-        <controller:gazebo_ros_bumper name="thhub_gazebo_ros_bumper_controller" plugin="libgazebo_ros_bumper.so">
+      <sensor type="contact" name="thhub_contact_sensor">
+        <update_rate>100.0</update_rate>
+        <contact>
+          <collision>thhub_collision_geom</collision>
+        </contact>
+        <plugin name="thhub_gazebo_ros_bumper_controller" filename="libgazebo_ros_bumper.so">
           <alwaysOn>true</alwaysOn>
+          <frameName>thhub</frameName>
           <updateRate>100.0</updateRate>
-          <frameName>thhub</frameName>
           <bumperTopicName>thhub_bumper</bumperTopicName>
-          <interface:bumper name="thhub_gazebo_ros_bumper_iface" />
-        </controller:gazebo_ros_bumper>
-      </sensor:contact>
+        </plugin>
+      </sensor>
       <material>Gazebo/Grey</material>
     </gazebo>

File: hand/xacro/thumb/thmiddle.urdf.xacro (robot description, xacro)
@@ -32,15 +32,16 @@
     </link>
     <gazebo reference="thmiddle">
-      <sensor:contact name="thmiddle_contact_sensor">
-        <geom>thmiddle_geom</geom>
-       <updateRate>100.0</updateRate>
-        <controller:gazebo_ros_bumper name="thmiddle_gazebo_ros_bumper_controller" plugin="libgazebo_ros_bumper.so">
+      <sensor type="contact" name="thmiddle_contact_sensor">
+        <update_rate>100.0</update_rate>
+        <contact>
+          <collision>thmiddle_collision_geom</collision>
+        </contact>
+        <plugin name="thmiddle_gazebo_ros_bumper_controller" filename="libgazebo_ros_bumper.so">
           <alwaysOn>true</alwaysOn>
+          <frameName>thmiddle</frameName>
           <updateRate>100.0</updateRate>
-          <frameName>thmiddle</frameName>
           <bumperTopicName>thmiddle_bumper</bumperTopicName>
-          <interface:bumper name="thmiddle_gazebo_ros_bumper_iface" />
-        </controller:gazebo_ros_bumper>
-      </sensor:contact>
+        </plugin>
+      </sensor>
       <material>Gazebo/Grey</material>
     </gazebo>

File: hand/xacro/thumb/thproximal.urdf.xacro (robot description, xacro)
@@ -41,15 +41,16 @@
     </link>
     <gazebo reference="thproximal">
-      <sensor:contact name="thproximal_contact_sensor">
-        <geom>thproximal_geom</geom>
-       <updateRate>100.0</updateRate>
-        <controller:gazebo_ros_bumper name="thproximal_gazebo_ros_bumper_controller" plugin="libgazebo_ros_bumper.so">
+      <sensor type="contact" name="thproximal_contact_sensor">
+        <update_rate>100.0</update_rate>
+        <contact>
+          <collision>thproximal_collision_geom</collision>
+        </contact>
+        <plugin name="thproximal_gazebo_ros_bumper_controller" filename="libgazebo_ros_bumper.so">
           <alwaysOn>true</alwaysOn>
+          <frameName>thproximal</frameName>
           <updateRate>100.0</updateRate>
-          <frameName>thproximal</frameName>
           <bumperTopicName>thproximal_bumper</bumperTopicName>
-          <interface:bumper name="thproximal_gazebo_ros_bumper_iface" />
-        </controller:gazebo_ros_bumper>
-      </sensor:contact>
+        </plugin>
+      </sensor>
       <material>Gazebo/Grey</material>
     </gazebo>

Commit message: fixing the tactiles for the finger tips

File: hand/xacro/finger/distal/distal.urdf.xacro (robot description, xacro)
@@ -30,22 +30,18 @@
     </link>
     <gazebo reference="${link_prefix}distal">
-      <sensor type="contact" name="${link_prefix}distal_contact_sensor">
-        <update_rate>100.0</update_rate>
+      <sensor type="contact" name="${link_prefix}distal_contact" >
+        <always_on>1</always_on>
+        <update_rate>1000.0</update_rate>
         <contact>
-          <collision>${link_prefix}distal_collision_geom</collision>
+          <collision>${link_prefix}distal_collision</collision>
+          <topic>${link_prefix}distal_collision</topic>
         </contact>
         <plugin name="${link_prefix}distal_gazebo_ros_bumper_controller" filename="libgazebo_ros_bumper.so">
-          <alwaysOn>true</alwaysOn>
-          <frameName>${link_prefix}distal</frameName>
           <updateRate>100.0</updateRate>
-          <bumperTopicName>${link_prefix}distal_bumper</bumperTopicName>
+	  <frameName>${link_prefix}distal</frameName>
+	  <bumperTopicName>/rh/contacts/${link_prefix}</bumperTopicName>
         </plugin>
       </sensor>
-      <mu1 value="500.0" />
-      <mu2 value="500.0" />
-      <kp  value="10000000.0" />
-      <kd  value="1.0" />
       <material>Gazebo/Grey</material>
-      <selfCollide>true</selfCollide>
     </gazebo>
     <joint name="${joint_prefix}J1" type="revolute">
@@ -59,8 +55,8 @@
     </joint>
     <link name="${link_prefix}tip">
-			<inertial>
-				<mass value="0.001" />
-				<inertia  ixx="0.0" ixy="0.0"  ixz="0.0"  iyy="0.0"  iyz="0.0" izz="0.0" />
-  		</inertial>
+      <inertial>
+	<mass value="0.001" />
+	<inertia  ixx="0.0" ixy="0.0"  ixz="0.0"  iyy="0.0"  iyz="0.0" izz="0.0" />
+      </inertial>
     </link>
     <joint name="${joint_prefix}tip" type="fixed">

Commit message: fixed all tactiles

File: hand/xacro/finger/distal/distal.urdf.xacro (robot description, xacro)
@@ -40,8 +40,8 @@
           <updateRate>100.0</updateRate>
 	  <frameName>${link_prefix}distal</frameName>
-	  <bumperTopicName>/rh/contacts/${link_prefix}</bumperTopicName>
+	  <bumperTopicName>contacts/${link_prefix}/distal</bumperTopicName>
         </plugin>
       </sensor>
-      <material>Gazebo/Grey</material>
+      <material>LightGrey</material>
     </gazebo>
     <joint name="${joint_prefix}J1" type="revolute">
