Commit message: fixing urdfs with missing prefix

File: sr_description/robots/arm_and_hand_motor.urdf.xacro (robot description, xacro)
@@ -13,5 +13,5 @@
   <joint name="arm_link" type="fixed">
     <parent link="shadowarm_handsupport" />
-    <child link="forearm" />
+    <child link="rh_forearm" />
     <origin xyz="0 0 0" rpy="0 0 ${2.35619449}" />
   </joint>

File: sr_description/robots/arm_and_hand_motor_biotac.urdf.xacro (robot description, xacro)
@@ -13,5 +13,5 @@
   <joint name="arm_link" type="fixed">
     <parent link="shadowarm_handsupport" />
-    <child link="forearm" />
+    <child link="rh_forearm" />
     <origin xyz="0 0 0" rpy="0 0 ${2.35619449}" />
   </joint>

File: sr_description/robots/arm_and_hand_motor_ellipsoid.urdf.xacro (robot description, xacro)
@@ -13,5 +13,5 @@
   <joint name="arm_link" type="fixed">
     <parent link="shadowarm_handsupport" />
-    <child link="forearm" />
+    <child link="rh_forearm" />
     <origin xyz="0 0 0" rpy="0 0 ${2.35619449}" />
   </joint>

File: sr_description/robots/arm_and_hand_motor_three_finger.urdf.xacro (robot description, xacro)
@@ -13,5 +13,5 @@
   <joint name="arm_link" type="fixed">
     <parent link="shadowarm_handsupport" />
-    <child link="forearm" />
+    <child link="rh_forearm" />
     <origin xyz="0 0 0" rpy="0 0 ${2.35619449}" />
   </joint>

File: sr_description/robots/arm_and_hand_muscle.urdf.xacro (robot description, xacro)
@@ -13,5 +13,5 @@
   <joint name="arm_link" type="fixed">
     <parent link="shadowarm_handsupport" />
-    <child link="forearm" />
+    <child link="rh_forearm" />
     <origin xyz="0 0 0" rpy="0 0 ${M_PI}" />
   </joint>

File: sr_description/robots/arm_and_hand_muscle_biotac.urdf.xacro (robot description, xacro)
@@ -13,5 +13,5 @@
   <joint name="arm_link" type="fixed">
     <parent link="shadowarm_handsupport" />
-    <child link="forearm" />
+    <child link="rh_forearm" />
     <origin xyz="0 0 0" rpy="0 0 ${M_PI}" />
   </joint>

File: sr_description/robots/arm_and_sr_one_finger_motor.urdf.xacro (robot description, xacro)
@@ -13,5 +13,5 @@
   <joint name="arm_link" type="revolute">
     <parent link="shadowarm_handsupport" />
-    <child link="forearm" />
+    <child link="rh_forearm" />
     <origin xyz="0 0 0" rpy="0 0 ${M_PI}" />
     <axis xyz="0 -1 0" />

File: sr_description/robots/desk_arm_and_hand_motor.urdf.xacro (robot description, xacro)
@@ -13,5 +13,5 @@
   <joint name="arm_link" type="revolute">
     <parent link="shadowarm_handsupport" />
-    <child link="forearm" />
+    <child link="rh_forearm" />
     <origin xyz="0 0 0" rpy="0 0 ${M_PI}" />
     <axis xyz="0 -1 0" />

File: sr_description/robots/shadowhand_edc_muscle.urdf.xacro (robot description, xacro)
@@ -9,5 +9,5 @@
   <xacro:shadowhand muscletrans="true" muscle="true" bio="false" bt_sp="false"
   ubi="false" eli="false" reflect="1.0" prefix="rh_" />
-  <link name="forearm_disk">
+  <link name="rh_forearm_disk">
     <inertial>
       <origin xyz="0 0 0" />
@@ -18,5 +18,5 @@
     <visual>
       <origin xyz="0 0 0" rpy="0 0 0" />
-      <geometry name="forearm_disk_geom">
+      <geometry name="rh_forearm_disk_geom">
         <mesh filename="package://sr_description/hand/model/forearm_muscle_disk.dae"
         scale="1.0 1.0 1.0" />
@@ -26,16 +26,16 @@
     <collision>
       <origin xyz="0 0 0.175" rpy="0 0 0" />
-      <geometry name="forearm_disk_collision">
+      <geometry name="rh_forearm_disk_collision">
         <cylinder radius="0.07" length="0.004" />
       </geometry>
     </collision>
   </link>
-  <gazebo reference="forearm_disk">
+  <gazebo reference="rh_forearm_disk">
     <material>Gazebo/Grey</material>
     <selfCollide>false</selfCollide>
   </gazebo>
-  <joint name="forearm_disk_to_forearm" type="fixed">
-    <parent link="forearm_disk" />
-    <child link="forearm" />
+  <joint name="rh_forearm_disk_to_forearm" type="fixed">
+    <parent link="rh_forearm_disk" />
+    <child link="rh_forearm" />
     <origin xyz="0 0 0.004" rpy="0 0 0" />
   </joint>

File: sr_description/robots/shadowhand_edc_muscle_biotac.urdf.xacro (robot description, xacro)
@@ -12,5 +12,5 @@
   <xacro:shadowhand muscletrans="true" muscle="true" bio="true" bt_sp="false"
   ubi="false" eli="false" reflect="1.0" prefix="rh_" />
-  <link name="forearm_disk">
+  <link name="rh_forearm_disk">
     <inertial>
       <origin xyz="0 0 0" />
@@ -21,5 +21,5 @@
     <visual>
       <origin xyz="0 0 0" rpy="0 0 0" />
-      <geometry name="forearm_disk_geom">
+      <geometry name="rh_forearm_disk_geom">
         <mesh filename="package://sr_description/hand/model/forearm_muscle_disk.dae"
         scale="1.0 1.0 1.0" />
@@ -29,16 +29,16 @@
     <collision>
       <origin xyz="0 0 0.175" rpy="0 0 0" />
-      <geometry name="forearm_disk_collision">
+      <geometry name="rh_forearm_disk_collision">
         <cylinder radius="0.07" length="0.004" />
       </geometry>
     </collision>
   </link>
-  <gazebo reference="forearm_disk">
+  <gazebo reference="rh_forearm_disk">
     <material>Gazebo/Grey</material>
     <selfCollide>false</selfCollide>
   </gazebo>
-  <joint name="forearm_disk_to_forearm" type="fixed">
-    <parent link="forearm_disk" />
-    <child link="forearm" />
+  <joint name="rh_forearm_disk_to_rh_forearm" type="fixed">
+    <parent link="rh_forearm_disk" />
+    <child link="rh_forearm" />
     <origin xyz="0 0 0.004" rpy="0 0 0" />
   </joint>

File: sr_description/robots/shadowhand_left_edc_muscle.urdf.xacro (robot description, xacro)
@@ -9,5 +9,5 @@
   <xacro:shadowhand muscletrans="true" muscle="true" bio="false" bt_sp="false"
   ubi="false" eli="false" reflect="-1.0" prefix="lh_" />
-  <link name="forearm_disk">
+  <link name="lh_forearm_disk">
     <inertial>
       <origin xyz="0 0 0" />
@@ -18,5 +18,5 @@
     <visual>
       <origin xyz="0 0 0" rpy="0 0 0" />
-      <geometry name="forearm_disk_geom">
+      <geometry name="lh_forearm_disk_geom">
         <mesh filename="package://sr_description/hand/model/forearm_muscle_disk.dae"
         scale="1.0 1.0 1.0" />
@@ -26,16 +26,16 @@
     <collision>
       <origin xyz="0 0 0.175" rpy="0 0 0" />
-      <geometry name="forearm_disk_collision">
+      <geometry name="lh_forearm_disk_collision">
         <cylinder radius="0.07" length="0.004" />
       </geometry>
     </collision>
   </link>
-  <gazebo reference="forearm_disk">
+  <gazebo reference="lh_forearm_disk">
     <material>Gazebo/Grey</material>
     <selfCollide>false</selfCollide>
   </gazebo>
-  <joint name="forearm_disk_to_forearm" type="fixed">
-    <parent link="forearm_disk" />
-    <child link="forearm" />
+  <joint name="lh_forearm_disk_to_lh_forearm" type="fixed">
+    <parent link="lh_forearm_disk" />
+    <child link="lh_forearm" />
     <origin xyz="0 0 0.004" rpy="0 0 0" />
   </joint>

File: sr_description/robots/shadowhand_left_muscle.urdf.xacro (robot description, xacro)
@@ -9,5 +9,5 @@
   <xacro:shadowhand muscletrans="false" muscle="true" bio="false" bt_sp="false"
   ubi="false" eli="false" reflect="-1.0" prefix="lh_" />
-  <link name="forearm_disk">
+  <link name="lh_forearm_disk">
     <inertial>
       <origin xyz="0 0 0" />
@@ -18,5 +18,5 @@
     <visual>
       <origin xyz="0 0 0" rpy="0 0 0" />
-      <geometry name="forearm_disk_geom">
+      <geometry name="lh_forearm_disk_geom">
         <mesh filename="package://sr_description/hand/model/forearm_muscle_disk.dae"
         scale="1.0 1.0 1.0" />
@@ -26,16 +26,16 @@
     <collision>
       <origin xyz="0 0 0.175" rpy="0 0 0" />
-      <geometry name="forearm_disk_collision">
+      <geometry name="lh_forearm_disk_collision">
         <cylinder radius="0.07" length="0.004" />
       </geometry>
     </collision>
   </link>
-  <gazebo reference="forearm_disk">
+  <gazebo reference="lh_forearm_disk">
     <material>Gazebo/Grey</material>
     <selfCollide>false</selfCollide>
   </gazebo>
-  <joint name="forearm_disk_to_forearm" type="fixed">
-    <parent link="forearm_disk" />
-    <child link="forearm" />
+  <joint name="lh_forearm_disk_to_lh_forearm" type="fixed">
+    <parent link="lh_forearm_disk" />
+    <child link="lh_forearm" />
     <origin xyz="0 0 0.004" rpy="0 0 0" />
   </joint>

File: sr_description/robots/shadowhand_muscle.urdf.xacro (robot description, xacro)
@@ -9,5 +9,5 @@
   <xacro:shadowhand muscletrans="false" muscle="true" bio="false" bt_sp="false"
   ubi="false" eli="false" reflect="1.0" prefix="rh_" />
-  <link name="forearm_disk">
+  <link name="rh_forearm_disk">
     <inertial>
       <origin xyz="0 0 0" />
@@ -18,5 +18,5 @@
     <visual>
       <origin xyz="0 0 0" rpy="0 0 0" />
-      <geometry name="forearm_disk_geom">
+      <geometry name="rh_forearm_disk_geom">
         <mesh filename="package://sr_description/hand/model/forearm_muscle_disk.dae"
         scale="1.0 1.0 1.0" />
@@ -26,16 +26,16 @@
     <collision>
       <origin xyz="0 0 0.175" rpy="0 0 0" />
-      <geometry name="forearm_disk_collision">
+      <geometry name="rh_forearm_disk_collision">
         <cylinder radius="0.07" length="0.004" />
       </geometry>
     </collision>
   </link>
-  <gazebo reference="forearm_disk">
+  <gazebo reference="rh_forearm_disk">
     <material>Gazebo/Grey</material>
     <selfCollide>false</selfCollide>
   </gazebo>
-  <joint name="forearm_disk_to_forearm" type="fixed">
-    <parent link="forearm_disk" />
-    <child link="forearm" />
+  <joint name="rh_forearm_disk_to_rh_forearm" type="fixed">
+    <parent link="rh_forearm_disk" />
+    <child link="rh_forearm" />
     <origin xyz="0 0 0.004" rpy="0 0 0" />
   </joint>

File: sr_description/robots/shadowhand_muscle_biotac.urdf.xacro (robot description, xacro)
@@ -12,5 +12,5 @@
   <xacro:shadowhand muscletrans="false" muscle="true" bio="true" bt_sp="false"
   ubi="false" eli="false" reflect="1.0" prefix="rh_" />
-  <link name="forearm_disk">
+  <link name="rh_forearm_disk">
     <inertial>
       <origin xyz="0 0 0" />
@@ -21,5 +21,5 @@
     <visual>
       <origin xyz="0 0 0" rpy="0 0 0" />
-      <geometry name="forearm_disk_geom">
+      <geometry name="rh_forearm_disk_geom">
         <mesh filename="package://sr_description/hand/model/forearm_muscle_disk.dae"
         scale="1.0 1.0 1.0" />
@@ -29,16 +29,16 @@
     <collision>
       <origin xyz="0 0 0.175" rpy="0 0 0" />
-      <geometry name="forearm_disk_collision">
+      <geometry name="rh_forearm_disk_collision">
         <cylinder radius="0.07" length="0.004" />
       </geometry>
     </collision>
   </link>
-  <gazebo reference="forearm_disk">
+  <gazebo reference="rh_forearm_disk">
     <material>Gazebo/Grey</material>
     <selfCollide>false</selfCollide>
   </gazebo>
-  <joint name="forearm_disk_to_forearm" type="fixed">
-    <parent link="forearm_disk" />
-    <child link="forearm" />
+  <joint name="rh_forearm_disk_to_rh_forearm" type="fixed">
+    <parent link="rh_forearm_disk" />
+    <child link="rh_forearm" />
     <origin xyz="0 0 0.004" rpy="0 0 0" />
   </joint>
