Commit message: Adding separation to launch file

File: sr_description/robots/bimanual_shadowhand_motor_plus.urdf.xacro (robot description, xacro)
@@ -5,4 +5,5 @@
   <xacro:include filename="$(find sr_description)/other/xacro/gazebo/gazebo.urdf.xacro" />
   <link name="world" />
+  <xacro:arg name="arm_x_separation" default="1.5"/>
   <joint name="world_joint" type="fixed">
     <parent link="world" />
@@ -15,5 +16,5 @@
     <parent link="rh_forearm" />
     <child link="lh_forearm" />
-    <origin xyz="0.4 0.0 0.0" rpy="0.0 0.0 0.0" />
+    <origin xyz="$(arg arm_x_separation) 0.0 0.0" rpy="0.0 0.0 0.0" />
   </joint>
   <xacro:shadowhand muscletrans="false" muscle="false" hand_type="hand_e_plus" bio="false" bt_sp="false"

Commit message: Adding files

File: sr_description/robots/bimanual_shadowhand_motor_plus.urdf.xacro (robot description, xacro)
@@ -5,4 +5,5 @@
   <xacro:include filename="$(find sr_description)/other/xacro/gazebo/gazebo.urdf.xacro" />
   <link name="world" />
+  <xacro:arg name="arm_x_separation" default="-0.4"/>
   <joint name="world_joint" type="fixed">
     <parent link="world" />
@@ -15,5 +16,5 @@
     <parent link="rh_forearm" />
     <child link="lh_forearm" />
-    <origin xyz="0.4 0.0 0.0" rpy="0.0 0.0 0.0" />
+    <origin xyz="$(arg arm_x_separation) 0.0 0.0" rpy="0.0 0.0 0.0" />
   </joint>
   <xacro:shadowhand muscletrans="false" muscle="false" hand_type="hand_e_plus" bio="false" bt_sp="false"
