Commit message: refactoring

File: sr_description/robots/sr_hand_bimanual.urdf.xacro (robot description, xacro)
@@ -8,18 +8,18 @@
   <xacro:include filename="$(find sr_description)/other/xacro/gazebo.urdf.xacro"/>
   <xacro:arg name="arm_x_separation" default="-0.4"/>
-  <xacro:arg name="hand_type_right" default="hand_e"/>
-  <xacro:arg name="hand_version_right" default="E3M5"/>
-  <xacro:arg name="fingers_right" default="all"/>
-  <xacro:arg name="tip_sensors_right" default="pst"/>
-  <xacro:arg name="mid_sensors_right" default="none"/>
-  <xacro:arg name="prox_sensors_right" default="none"/>
-  <xacro:arg name="palm_sensor_right" default="none"/>
-  <xacro:arg name="hand_type_left" default="hand_e"/>
-  <xacro:arg name="hand_version_left" default="E3M5"/>
-  <xacro:arg name="fingers_left" default="all"/>
-  <xacro:arg name="tip_sensors_left" default="pst"/>
-  <xacro:arg name="mid_sensors_left" default="none"/>
-  <xacro:arg name="prox_sensors_left" default="none"/>
-  <xacro:arg name="palm_sensor_left" default="none"/>
+  <xacro:arg name="right_hand_type" default="hand_e"/>
+  <xacro:arg name="right_hand_version" default="E3M5"/>
+  <xacro:arg name="right_fingers" default="all"/>
+  <xacro:arg name="right_tip_sensors" default="pst"/>
+  <xacro:arg name="right_mid_sensors" default="none"/>
+  <xacro:arg name="right_prox_sensors" default="none"/>
+  <xacro:arg name="right_palm_sensor" default="none"/>
+  <xacro:arg name="left_hand_type" default="hand_e"/>
+  <xacro:arg name="left_hand_version" default="E3M5"/>
+  <xacro:arg name="left_fingers" default="all"/>
+  <xacro:arg name="left_tip_sensors" default="pst"/>
+  <xacro:arg name="left_mid_sensors" default="none"/>
+  <xacro:arg name="left_prox_sensors" default="none"/>
+  <xacro:arg name="left_palm_sensor" default="none"/>
   <link name="world" />
   <joint name="world_joint" type="fixed">
@@ -28,14 +28,14 @@
     <origin xyz="0.0 0.0 0.0" rpy="0.0 0.0 0.0" />
   </joint>
-  <xacro:sr_hand hand_type="$(arg hand_type_right)" hand_version="$(arg hand_version_right)" side="right"
-                 fingers="$(arg fingers_right)" tip_sensors="$(arg tip_sensors_right)" mid_sensors="$(arg mid_sensors_right)"
-                 prox_sensors="$(arg prox_sensors_right)" palm_sensor="$(arg palm_sensor_right)"/>
-  <joint name="right_hand_to_left_hand" type="fixed">
+  <xacro:sr_hand side="right" hand_type="$(arg right_hand_type)" hand_version="$(arg right_hand_version)"
+                 fingers="$(arg right_fingers)" tip_sensors="$(arg right_tip_sensors)" mid_sensors="$(arg right_mid_sensors)"
+                 prox_sensors="$(arg right_prox_sensors)" palm_sensor="$(arg right_palm_sensor)"/>
+  <joint name="right_hand_to_hand" type="fixed">
     <parent link="rh_forearm" />
     <child link="lh_forearm" />
     <origin xyz="$(arg arm_x_separation) 0.0 0.0" rpy="0.0 0.0 0.0" />
   </joint>
-  <xacro:sr_hand hand_type="$(arg hand_type_left)" hand_version="$(arg hand_version_left)" side="left"
-                 fingers="$(arg fingers_left)" tip_sensors="$(arg tip_sensors_left)" mid_sensors="$(arg mid_sensors_left)"
-                 prox_sensors="$(arg prox_sensors_left)" palm_sensor="$(arg palm_sensor_left)"/>
+  <xacro:sr_hand side="left" hand_type="$(arg left_hand_type)" hand_version="$(arg left_hand_version)"
+                 fingers="$(arg left_fingers)" tip_sensors="$(arg left_tip_sensors)" mid_sensors="$(arg left_mid_sensors)"
+                 prox_sensors="$(arg left_prox_sensors)" palm_sensor="$(arg left_palm_sensor)"/>
 </robot>

Commit message: according to review

File: sr_description/robots/sr_hand_bimanual.urdf.xacro (robot description, xacro)
@@ -34,5 +34,5 @@
                  fingers="$(arg left_fingers)" tip_sensors="$(arg left_tip_sensors)" mid_sensors="$(arg left_mid_sensors)"
                  prox_sensors="$(arg left_prox_sensors)" palm_sensor="$(arg left_palm_sensor)"/>
-  <joint name="right_hand_to_hand" type="fixed">
+  <joint name="right_hand_to_left_hand" type="fixed">
     <parent link="rh_forearm" />
     <child link="lh_forearm" />
