Commit message: Fixed arm controllers to use standard gazebo ros control lib

File: sr_description/arm/xacro/full_arm_motor.urdf.xacro (robot description, xacro)
@@ -1,3 +1,3 @@
-<robot xmlns:sensor="http://playerstage.sourceforge.net/gazebo/xmlschema/#sensor"
+  <robot xmlns:sensor="http://playerstage.sourceforge.net/gazebo/xmlschema/#sensor"
 xmlns:controller="http://playerstage.sourceforge.net/gazebo/xmlschema/#controller"
 xmlns:interface="http://playerstage.sourceforge.net/gazebo/xmlschema/#interface"
@@ -18,4 +18,8 @@
     <xacro:shadowarm_handsupport_motor parent="shadowarm_lowerarm">
     </xacro:shadowarm_handsupport_motor>
+    <gazebo>
+      <plugin name="gazebo_ros_control" filename="libgazebo_ros_control.so">
+      </plugin>
+    </gazebo>
   </xacro:macro>
 </robot>

File: sr_description/arm/xacro/hand_support/shadowarm_handsupport_motor.transmission.xacro (robot description, xacro)
@@ -5,8 +5,12 @@
        xmlns:xacro="http://www.ros.org/wiki/xacro">
   <xacro:macro name="shadowarm_handsupport_motor_transmission">
-    <transmission type="sr_mechanism_model/SimpleTransmission" name="forearm_rotation_transmission">
-      <actuator name="forearm_rotation" />
-      <joint name="ElbowJRotate" />
-      <mechanicalReduction>1</mechanicalReduction>
+    <transmission name="forearm_rotation_transmission">
+      <type>sr_mechanism_model/SimpleTransmission</type>
+      <actuator name="forearm_rotation">
+        <mechanicalReduction>1</mechanicalReduction>
+      </actuator>
+      <joint name="ElbowJRotate">
+        <hardwareInterface>EffortJointInterface</hardwareInterface>
+      </joint>
     </transmission>
   </xacro:macro>

File: sr_description/arm/xacro/hand_support/shadowarm_handsupport_muscle.transmission.xacro (robot description, xacro)
@@ -5,8 +5,12 @@
        xmlns:xacro="http://www.ros.org/wiki/xacro">
   <xacro:macro name="shadowarm_handsupport_muscle_transmission">
-    <transmission type="sr_mechanism_model/SimpleTransmission" name="forearm_rotation_transmission">
-      <actuator name="forearm_rotation" />
-      <joint name="ElbowJRotate" />
-      <mechanicalReduction>1</mechanicalReduction>
+    <transmission name="forearm_rotation_transmission">
+      <type>sr_mechanism_model/SimpleTransmission</type>
+      <actuator name="forearm_rotation">
+        <mechanicalReduction>1</mechanicalReduction>
+      </actuator>
+      <joint name="ElbowJRotate">
+        <hardwareInterface>EffortJointInterface</hardwareInterface>
+      </joint>
     </transmission>
   </xacro:macro>

File: sr_description/arm/xacro/lower_arm/shadowarm_lowerarm.transmission.xacro (robot description, xacro)
@@ -5,8 +5,12 @@
        xmlns:xacro="http://www.ros.org/wiki/xacro">
   <xacro:macro name="shadowarm_lowerarm_transmission">
-    <transmission type="sr_mechanism_model/SimpleTransmission" name="elbow_abduction_transmission">
-      <actuator name="elbow_abduction" />
-      <joint name="ElbowJSwing" />
-      <mechanicalReduction>1</mechanicalReduction>
+    <transmission name="elbow_abduction_transmission">
+      <type>sr_mechanism_model/SimpleTransmission</type>
+      <actuator name="elbow_abduction">
+        <mechanicalReduction>1</mechanicalReduction>
+      </actuator>
+      <joint name="ElbowJSwing">
+        <hardwareInterface>EffortJointInterface</hardwareInterface>
+      </joint>
     </transmission>
   </xacro:macro>

File: sr_description/arm/xacro/trunk/shadowarm_trunk.transmission.xacro (robot description, xacro)
@@ -5,8 +5,12 @@
        xmlns:xacro="http://www.ros.org/wiki/xacro">
   <xacro:macro name="shadowarm_trunk_transmission">
-    <transmission type="sr_mechanism_model/SimpleTransmission" name="trunk_rotation_transmission">
-      <actuator name="trunk_rotation" />
-      <joint name="ShoulderJRotate" />
-      <mechanicalReduction>1</mechanicalReduction>
+    <transmission name="trunk_rotation_transmission">
+      <type>sr_mechanism_model/SimpleTransmission</type>
+      <actuator name="trunk_rotation">
+        <mechanicalReduction>1</mechanicalReduction>
+      </actuator>
+      <joint name="ShoulderJRotate">
+        <hardwareInterface>EffortJointInterface</hardwareInterface>
+      </joint>
     </transmission>
   </xacro:macro>

File: sr_description/arm/xacro/upper_arm/shadowarm_upperarm.transmission.xacro (robot description, xacro)
@@ -5,8 +5,12 @@
        xmlns:xacro="http://www.ros.org/wiki/xacro">
   <xacro:macro name="shadowarm_upperarm_transmission">
-    <transmission type="sr_mechanism_model/SimpleTransmission" name="shoulder_rotation_transmission">
-      <actuator name="shoulder_rotation" />
-      <joint name="ShoulderJSwing" />
-      <mechanicalReduction>1</mechanicalReduction>
+    <transmission name="shoulder_rotation_transmission">
+      <type>sr_mechanism_model/SimpleTransmission</type>
+      <actuator name="shoulder_rotation">
+        <mechanicalReduction>1</mechanicalReduction>
+      </actuator>
+      <joint name="ShoulderJSwing">
+        <hardwareInterface>EffortJointInterface</hardwareInterface>
+      </joint>
     </transmission>
   </xacro:macro>

File: sr_description/robots/sr_arm_motor.urdf.xacro (robot description, xacro)
@@ -5,5 +5,5 @@
   <xacro:include filename="$(find sr_description)/materials.urdf.xacro" />
   <xacro:include filename="$(find sr_description)/arm/xacro/full_arm_motor.urdf.xacro" />
-  <xacro:include filename="$(find sr_description)/other/xacro/gazebo/gazebo.urdf.xacro" />
+  <!--xacro:include filename="$(find sr_description)/other/xacro/gazebo/gazebo.urdf.xacro" /-->
   <link name="world" />
   <joint name="arm_to_world_fixed" type="fixed">
