Commit message: added manipulator link and joint to the palm

File: sr_description/hand/xacro/palm/palm.urdf.xacro (robot description, xacro)
@@ -87,4 +87,17 @@
       </collision>
     </link>
+    <joint name="${prefix}ee_fixed_joint" type="fixed">
+      <parent link="${prefix}palm" />
+      <child link = "${prefix}manipulator" />
+      <origin xyz="0.0 0.0 0.05" rpy="0.0 0.0 0.0" />
+    </joint>
+    <link name="${prefix}manipulator">
+      <collision>
+        <geometry>
+          <box size="0.001 0.001 0.001"/>
+        </geometry>
+        <origin rpy="0 0 0" xyz="-0.001 0 0"/>
+      </collision>
+    </link>
     <joint name="${prefix}WRJ1" type="revolute">
       <parent link="${parent}" />

Commit message: Removing collision

File: sr_description/hand/xacro/palm/palm.urdf.xacro (robot description, xacro)
@@ -92,12 +92,5 @@
       <origin xyz="0.0 0.0 0.05" rpy="0.0 0.0 0.0" />
     </joint>
-    <link name="${prefix}manipulator">
-      <collision>
-        <geometry>
-          <box size="0.001 0.001 0.001"/>
-        </geometry>
-        <origin rpy="0 0 0" xyz="-0.001 0 0"/>
-      </collision>
-    </link>
+    <link name="${prefix}manipulator" />
     <joint name="${prefix}WRJ1" type="revolute">
       <parent link="${parent}" />
