Commit message: added manipulator to palm lite

File: sr_description/hand/xacro/palm/palm_lite.urdf.xacro (robot description, xacro)
@@ -79,4 +79,17 @@
       </collision>
     </link>
+    <joint name="${prefix}ee_fixed_joint" type="fixed">
+      <parent link="${prefix}palm" />
+      <child link = "${prefix}manipulator" />
+      <origin xyz="0.0 0.0 0.05" rpy="0.0 0.0 0.0" />
+    </joint>
+    <link name="${prefix}manipulator">
+      <collision>
+        <geometry>
+          <box size="0.001 0.001 0.001"/>
+        </geometry>
+        <origin rpy="0 0 0" xyz="-0.001 0 0"/>
+      </collision>
+    </link>
     <!-- No wrist joints in a Lite palm -->
     <!-- extensions -->

Commit message: Removing collision for hand lite also

File: sr_description/hand/xacro/palm/palm_lite.urdf.xacro (robot description, xacro)
@@ -84,12 +84,5 @@
       <origin xyz="0.0 0.0 0.05" rpy="0.0 0.0 0.0" />
     </joint>
-    <link name="${prefix}manipulator">
-      <collision>
-        <geometry>
-          <box size="0.001 0.001 0.001"/>
-        </geometry>
-        <origin rpy="0 0 0" xyz="-0.001 0 0"/>
-      </collision>
-    </link>
+    <link name="${prefix}manipulator" />
     <!-- No wrist joints in a Lite palm -->
     <!-- extensions -->
