Commit message: add a child element called imu, to be compatible with SensorParser, and avoid xacro breaking by renaming macro to imu_sensor

File: sr_description/hand/xacro/palm/imu.urdf.xacro (robot description, xacro)
@@ -1,4 +1,4 @@
 <robot xmlns:xacro="http://www.ros.org/wiki/xacro" name="shadowhand_motor">
-  <xacro:macro name="imu" params="prefix">
+  <xacro:macro name="imu_sensor" params="prefix">
     <link name="${prefix}imu"/>
     <joint name="${prefix}palm_to_imu" type="fixed">
@@ -10,4 +10,5 @@
       <parent link="${prefix}imu"/>
       <origin xyz="0 0 0" rpy="0 0 0"/>
+      <imu />
     </sensor>
   </xacro:macro>
