Commit message: New hand E mujoco PID values based on Gazebo values.

File: sr_description/mujoco_models/urdfs/shadowhand_motor.urdf (robot description, URDF)
Before this commit: robot shadowhand_motor, 33 links, 32 joints
Joints:
- joint rh_FFJ1: limit lower=0 upper=1.57079632679 effort=2 velocity=2.0 -> lower=0 upper=1.57079632679 effort=1.0 velocity=2.0
- joint rh_FFJ2: limit lower=0 upper=1.57079632679 effort=2 velocity=2.0 -> lower=0 upper=1.57079632679 effort=1.0 velocity=2.0
- joint rh_FFJ3: limit lower=0 upper=1.57079632679 effort=2 velocity=2.0 -> lower=0 upper=1.57079632679 effort=1.0 velocity=2.0
- joint rh_FFJ4: limit lower=-0.349065850399 upper=0.349065850399 effort=2 velocity=2.0 -> lower=-0.349065850399 upper=0.349065850399 effort=1.0 velocity=2.0
- joint rh_LFJ1: limit lower=0 upper=1.57079632679 effort=2 velocity=2.0 -> lower=0 upper=1.57079632679 effort=1.0 velocity=2.0
- joint rh_LFJ2: limit lower=0 upper=1.57079632679 effort=2 velocity=2.0 -> lower=0 upper=1.57079632679 effort=1.0 velocity=2.0
- joint rh_LFJ3: limit lower=0 upper=1.57079632679 effort=2 velocity=2.0 -> lower=0 upper=1.57079632679 effort=1.0 velocity=2.0
- joint rh_LFJ4: limit lower=-0.349065850399 upper=0.349065850399 effort=2 velocity=2.0 -> lower=-0.349065850399 upper=0.349065850399 effort=1.0 velocity=2.0
- joint rh_LFJ5: limit lower=0 upper=0.785398163397 effort=2 velocity=2.0 -> lower=0 upper=0.785398163397 effort=1.0 velocity=2.0
- joint rh_MFJ1: limit lower=0 upper=1.57079632679 effort=2 velocity=2.0 -> lower=0 upper=1.57079632679 effort=1.0 velocity=2.0
- joint rh_MFJ2: limit lower=0 upper=1.57079632679 effort=2 velocity=2.0 -> lower=0 upper=1.57079632679 effort=1.0 velocity=2.0
- joint rh_MFJ3: limit lower=0 upper=1.57079632679 effort=2 velocity=2.0 -> lower=0 upper=1.57079632679 effort=1.0 velocity=2.0
- joint rh_MFJ4: limit lower=-0.349065850399 upper=0.349065850399 effort=2 velocity=2.0 -> lower=-0.349065850399 upper=0.349065850399 effort=1.0 velocity=2.0
- joint rh_RFJ1: limit lower=0 upper=1.57079632679 effort=2 velocity=2.0 -> lower=0 upper=1.57079632679 effort=1.0 velocity=2.0
- joint rh_RFJ2: limit lower=0 upper=1.57079632679 effort=2 velocity=2.0 -> lower=0 upper=1.57079632679 effort=1.0 velocity=2.0
- joint rh_RFJ3: limit lower=0 upper=1.57079632679 effort=2 velocity=2.0 -> lower=0 upper=1.57079632679 effort=1.0 velocity=2.0
- joint rh_RFJ4: limit lower=-0.349065850399 upper=0.349065850399 effort=2 velocity=2.0 -> lower=-0.349065850399 upper=0.349065850399 effort=1.0 velocity=2.0
- joint rh_THJ2: limit lower=-0.698131700798 upper=0.698131700798 effort=2.0 velocity=2.0 -> lower=-0.698131700798 upper=0.698131700798 effort=1.0 velocity=2.0
- joint rh_THJ3: limit lower=-0.209439510239 upper=0.209439510239 effort=2.0 velocity=4.0 -> lower=-0.209439510239 upper=0.209439510239 effort=1.0 velocity=4.0
- joint rh_THJ4: limit lower=0.0 upper=1.2217304764 effort=3 velocity=4.0 -> lower=0.0 upper=1.2217304764 effort=2.0 velocity=4.0
- joint rh_THJ5: limit lower=-1.0471975512 upper=1.0471975512 effort=5.0 velocity=4.0 -> lower=-1.0471975512 upper=1.0471975512 effort=3.0 velocity=4.0
- joint rh_WRJ1: limit lower=-0.698131700798 upper=0.488692190558 effort=30 velocity=2.0 -> lower=-0.698131700798 upper=0.488692190558 effort=5.0 velocity=2.0
- joint rh_WRJ2: limit lower=-0.523598775598 upper=0.174532925199 effort=10 velocity=2.0 -> lower=-0.523598775598 upper=0.174532925199 effort=10.0 velocity=2.0

Commit message: Working and PID tuned Hand E and Hand E plus.

File: sr_description/mujoco_models/urdfs/shadowhand_motor.urdf (robot description, URDF)
Before this commit: robot shadowhand_motor, 33 links, 32 joints
Joints:
- joint rh_FFJ1: limit lower=0 upper=1.57079632679 effort=1.0 velocity=2.0 -> lower=0 upper=1.57079632679 effort=4.0 velocity=2.0
- joint rh_FFJ2: limit lower=0 upper=1.57079632679 effort=1.0 velocity=2.0 -> lower=0 upper=1.57079632679 effort=4.0 velocity=2.0
- joint rh_FFJ3: limit lower=0 upper=1.57079632679 effort=1.0 velocity=2.0 -> lower=0 upper=1.57079632679 effort=4.0 velocity=2.0
- joint rh_FFJ4: limit lower=-0.349065850399 upper=0.349065850399 effort=1.0 velocity=2.0 -> lower=-0.349065850399 upper=0.349065850399 effort=4.0 velocity=2.0
- joint rh_LFJ1: limit lower=0 upper=1.57079632679 effort=1.0 velocity=2.0 -> lower=0 upper=1.57079632679 effort=4.0 velocity=2.0
- joint rh_LFJ2: limit lower=0 upper=1.57079632679 effort=1.0 velocity=2.0 -> lower=0 upper=1.57079632679 effort=4.0 velocity=2.0
- joint rh_LFJ3: limit lower=0 upper=1.57079632679 effort=1.0 velocity=2.0 -> lower=0 upper=1.57079632679 effort=4.0 velocity=2.0
- joint rh_LFJ4: limit lower=-0.349065850399 upper=0.349065850399 effort=1.0 velocity=2.0 -> lower=-0.349065850399 upper=0.349065850399 effort=4.0 velocity=2.0
- joint rh_LFJ5: limit lower=0 upper=0.785398163397 effort=1.0 velocity=2.0 -> lower=0 upper=0.785398163397 effort=4.0 velocity=2.0
- joint rh_MFJ1: limit lower=0 upper=1.57079632679 effort=1.0 velocity=2.0 -> lower=0 upper=1.57079632679 effort=4.0 velocity=2.0
- joint rh_MFJ2: limit lower=0 upper=1.57079632679 effort=1.0 velocity=2.0 -> lower=0 upper=1.57079632679 effort=4.0 velocity=2.0
- joint rh_MFJ3: limit lower=0 upper=1.57079632679 effort=1.0 velocity=2.0 -> lower=0 upper=1.57079632679 effort=4.0 velocity=2.0
- joint rh_MFJ4: limit lower=-0.349065850399 upper=0.349065850399 effort=1.0 velocity=2.0 -> lower=-0.349065850399 upper=0.349065850399 effort=4.0 velocity=2.0
- joint rh_RFJ1: limit lower=0 upper=1.57079632679 effort=1.0 velocity=2.0 -> lower=0 upper=1.57079632679 effort=4.0 velocity=2.0
- joint rh_RFJ2: limit lower=0 upper=1.57079632679 effort=1.0 velocity=2.0 -> lower=0 upper=1.57079632679 effort=4.0 velocity=2.0
- joint rh_RFJ3: limit lower=0 upper=1.57079632679 effort=1.0 velocity=2.0 -> lower=0 upper=1.57079632679 effort=4.0 velocity=2.0
- joint rh_RFJ4: limit lower=-0.349065850399 upper=0.349065850399 effort=1.0 velocity=2.0 -> lower=-0.349065850399 upper=0.349065850399 effort=4.0 velocity=2.0
- joint rh_THJ1: limit lower=0 upper=1.57079632679 effort=1.0 velocity=4.0 -> lower=0 upper=1.57079632679 effort=4.0 velocity=4.0
- joint rh_THJ2: limit lower=-0.698131700798 upper=0.698131700798 effort=1.0 velocity=2.0 -> lower=-0.698131700798 upper=0.698131700798 effort=4.0 velocity=2.0
- joint rh_THJ3: limit lower=-0.209439510239 upper=0.209439510239 effort=1.0 velocity=4.0 -> lower=-0.209439510239 upper=0.209439510239 effort=4.0 velocity=4.0
- joint rh_THJ4: limit lower=0.0 upper=1.2217304764 effort=2.0 velocity=4.0 -> lower=0.0 upper=1.2217304764 effort=4.0 velocity=4.0
- joint rh_THJ5: limit lower=-1.0471975512 upper=1.0471975512 effort=3.0 velocity=4.0 -> lower=-1.0471975512 upper=1.0471975512 effort=4.0 velocity=4.0

File: sr_description/mujoco_models/urdfs/shadowhand_motor_plus.urdf (robot description, URDF)
Before this commit: robot shadowhand_motor, 33 links, 32 joints
Joints:
- joint rh_FFJ1: limit lower=0 upper=1.57079632679 effort=1.0 velocity=2.0 -> lower=0 upper=1.57079632679 effort=4.0 velocity=2.0
- joint rh_FFJ2: limit lower=0 upper=1.57079632679 effort=1.0 velocity=2.0 -> lower=0 upper=1.57079632679 effort=4.0 velocity=2.0
- joint rh_FFJ3: limit lower=0 upper=1.57079632679 effort=1.0 velocity=2.0 -> lower=0 upper=1.57079632679 effort=4.0 velocity=2.0
- joint rh_FFJ4: limit lower=-0.349065850399 upper=0.349065850399 effort=1.0 velocity=2.0 -> lower=-0.349065850399 upper=0.349065850399 effort=4.0 velocity=2.0
- joint rh_LFJ1: limit lower=0 upper=1.57079632679 effort=1.0 velocity=2.0 -> lower=0 upper=1.57079632679 effort=4.0 velocity=2.0
- joint rh_LFJ2: limit lower=0 upper=1.57079632679 effort=1.0 velocity=2.0 -> lower=0 upper=1.57079632679 effort=4.0 velocity=2.0
- joint rh_LFJ3: limit lower=0 upper=1.57079632679 effort=1.0 velocity=2.0 -> lower=0 upper=1.57079632679 effort=4.0 velocity=2.0
- joint rh_LFJ4: limit lower=-0.349065850399 upper=0.349065850399 effort=1.0 velocity=2.0 -> lower=-0.349065850399 upper=0.349065850399 effort=4.0 velocity=2.0
- joint rh_LFJ5: limit lower=0 upper=0.785398163397 effort=1.0 velocity=2.0 -> lower=0 upper=0.785398163397 effort=4.0 velocity=2.0
- joint rh_MFJ1: limit lower=0 upper=1.57079632679 effort=1.0 velocity=2.0 -> lower=0 upper=1.57079632679 effort=4.0 velocity=2.0
- joint rh_MFJ2: limit lower=0 upper=1.57079632679 effort=1.0 velocity=2.0 -> lower=0 upper=1.57079632679 effort=4.0 velocity=2.0
- joint rh_MFJ3: limit lower=0 upper=1.57079632679 effort=1.0 velocity=2.0 -> lower=0 upper=1.57079632679 effort=4.0 velocity=2.0
- joint rh_MFJ4: limit lower=-0.349065850399 upper=0.349065850399 effort=1.0 velocity=2.0 -> lower=-0.349065850399 upper=0.349065850399 effort=4.0 velocity=2.0
- joint rh_RFJ1: limit lower=0 upper=1.57079632679 effort=1.0 velocity=2.0 -> lower=0 upper=1.57079632679 effort=4.0 velocity=2.0
- joint rh_RFJ2: limit lower=0 upper=1.57079632679 effort=1.0 velocity=2.0 -> lower=0 upper=1.57079632679 effort=4.0 velocity=2.0
- joint rh_RFJ3: limit lower=0 upper=1.57079632679 effort=1.0 velocity=2.0 -> lower=0 upper=1.57079632679 effort=4.0 velocity=2.0
- joint rh_RFJ4: limit lower=-0.349065850399 upper=0.349065850399 effort=1.0 velocity=2.0 -> lower=-0.349065850399 upper=0.349065850399 effort=4.0 velocity=2.0
- joint rh_THJ1: limit lower=0 upper=1.57079632679 effort=1.0 velocity=4.0 -> lower=0 upper=1.57079632679 effort=4.0 velocity=4.0
- joint rh_THJ2: limit lower=-0.698131700798 upper=0.698131700798 effort=1.0 velocity=2.0 -> lower=-0.698131700798 upper=0.698131700798 effort=4.0 velocity=2.0
- joint rh_THJ3: limit lower=-0.209439510239 upper=0.209439510239 effort=1.0 velocity=4.0 -> lower=-0.209439510239 upper=0.209439510239 effort=4.0 velocity=4.0
- joint rh_THJ4: limit lower=0.0 upper=1.2217304764 effort=2.0 velocity=4.0 -> lower=0.0 upper=1.2217304764 effort=4.0 velocity=4.0
- joint rh_THJ5: limit lower=-1.0471975512 upper=1.0471975512 effort=3.0 velocity=4.0 -> lower=-1.0471975512 upper=1.0471975512 effort=4.0 velocity=4.0
