Commit message: ur fix

File: sr_description/mujoco_models/urdfs/ur10.urdf (robot description, URDF)
Before this commit: robot ursr, 11 links, 10 joints
Links:
- removed link ra_ee_link
- added link ra_flange; collision box size=0.01 0.01 0.01
Joints:
- joint ra_ee_fixed_joint: child ra_ee_link -> ra_flange

File: sr_description/mujoco_models/urdfs/ur10_hand.urdf (robot description, URDF)
Before this commit: robot ur10srh, 43 links, 42 joints
Links:
- removed link ra_ee_link
- added link ra_flange; collision box size=0.01 0.01 0.01
Joints:
- joint ra_arm_to_hand: parent ra_ee_link -> ra_flange
- joint ra_ee_fixed_joint: child ra_ee_link -> ra_flange
