Commit message: adding element to xacro

File: sr_description/hand/xacro/forearm/forearm_lite.urdf.xacro (robot description, xacro)
@@ -39,4 +39,16 @@
         </xacro:unless>
       </collision>
+      <visual>
+        <origin rpy="0 1.57 -1.52" xyz="0.0 -0.012 0.01"/>
+        <geometry name="${prefix}cable_extr_collision">
+          <mesh filename="package://sr_description/hand/model/cable_collistion_mesh.stl" scale="1 1 1" />
+        </geometry>
+      </visual>
+      <collision>
+        <origin rpy="0 1.57 -1.52" xyz="0.0 -0.012 0.01"/>
+        <geometry name="${prefix}cable_extr_visualisation">
+          <mesh filename="package://sr_description/hand/model/cable_collistion_mesh.stl" scale="1 1 1" />
+        </geometry>
+      </collision>
     </link>
   </xacro:macro>
