Commit message: Add fix joint with the world and forearm. Improved the dimentions of the collision box of the lite hands

File: sr_description/hand/xacro/forearm/forearm.urdf.xacro (robot description, xacro)
@@ -35,5 +35,4 @@
           <geometry name="${prefix}forearm_collision">
             <cylinder radius="0.07" length="0.184"/>
-            <!--<box size="0.140 0.140 0.184" />-->
           </geometry>
         </xacro:unless>

File: sr_description/hand/xacro/forearm/forearm_lite.urdf.xacro (robot description, xacro)
@@ -33,7 +33,7 @@
         </xacro:if>
         <xacro:unless value="${muscle}">
-          <origin xyz="0 0 0.0775" rpy="0 0 0" />
+          <origin xyz="0 0 0.065" rpy="0 0 0" />
           <geometry name="${prefix}forearm_collision">
-            <box size="0.109 0.120 0.155" />
+            <box size="0.120 0.109 0.130" />
           </geometry>
         </xacro:unless>

File: sr_description/robots/shadowhand_extra_lite.urdf.xacro (robot description, xacro)
@@ -7,4 +7,11 @@
   <xacro:include filename="$(find sr_description)/hand/xacro/hand_lite.urdf.xacro" />
   <xacro:include filename="$(find sr_description)/other/xacro/gazebo/gazebo.urdf.xacro" />
+  <!-- hand with cylindrical base drifts in gazebo, attach it to the world -->
+  <link name="world" />
+  <joint name="rh_world_joint" type="fixed">
+    <parent link="world" />
+    <child link="rh_forearm" />
+    <origin xyz="0.0 0.0 0.0" rpy="0.0 0.0 0.0" />
+  </joint>
   <xacro:shadowhand muscletrans="false" muscle="false" bio="false" bt_sp="false"
   ubi="false" eli="false" reflect="1.0" prefix="rh_" extra_lite="true"/>

File: sr_description/robots/shadowhand_lite.urdf.xacro (robot description, xacro)
@@ -7,4 +7,11 @@
   <xacro:include filename="$(find sr_description)/hand/xacro/hand_lite.urdf.xacro" />
   <xacro:include filename="$(find sr_description)/other/xacro/gazebo/gazebo.urdf.xacro" />
+  <!-- hand with cylindrical base drifts in gazebo, attach it to the world -->
+  <link name="world" />
+  <joint name="rh_world_joint" type="fixed">
+    <parent link="world" />
+    <child link="rh_forearm" />
+    <origin xyz="0.0 0.0 0.0" rpy="0.0 0.0 0.0" />
+  </joint>
   <xacro:shadowhand muscletrans="false" muscle="false" bio="false" bt_sp="false"
   ubi="false" eli="false" reflect="1.0" prefix="rh_" extra_lite="false"/>

Commit message: Added meshes for hand_e_plus and also modified the xacros to load them

File: sr_description/hand/xacro/forearm/forearm.urdf.xacro (robot description, xacro)
@@ -1,6 +1,17 @@
 <robot xmlns:xacro="http://www.ros.org/wiki/xacro">
   <!-- muscle is true for muscle hand or false for motor hand -->
+  <!-- hand_type can be either hand_e (default) or hand_e_plus -->
   <!-- prefix can be anything but usually is "r_" or  "l_" for right and left hands distinction -->
-  <xacro:macro name="forearm" params="muscle prefix">
+  <xacro:macro name="dark_grey" >
+    <material name="dark_grey">
+      <color rgba="0.21961 0.21961 0.21961 1.0" />
+    </material>
+  </xacro:macro>
+  <xacro:macro name="light_grey" >
+    <material name="light_grey">
+      <color rgba="0.90000 0.90000 0.90000 1.0" />
+    </material>
+  </xacro:macro>
+  <xacro:macro name="forearm" params="muscle hand_type:='hand_e' prefix">
     <link name="${prefix}forearm">
       <inertial>
@@ -10,18 +21,47 @@
         iyz="0.0" izz="0.00744" />
       </inertial>
-      <visual>
-        <origin xyz="0 0 0" rpy="0 0 0" />
-        <geometry name="${prefix}forearm_visual">
-          <xacro:if value="${muscle}">
-            <mesh filename="package://sr_description/hand/model/forearm_muscle.dae"
-            scale="1.0 1.0 1.0" />
-          </xacro:if>
-          <xacro:unless value="${muscle}">
-            <mesh filename="package://sr_description/hand/model/forearm.dae"
-            scale="0.001 0.001 0.001" />
-          </xacro:unless>
-        </geometry>
-        <material name="Grey" />
-      </visual>
+      <xacro:if value="${muscle}">
+        <visual>
+          <origin xyz="0 0 0" rpy="0 0 0" />
+          <geometry name="${prefix}forearm_visual">
+            <mesh filename="package://sr_description/hand/model/forearm_muscle.dae" scale="1.0 1.0 1.0" />
+          </geometry>
+          <material name="Grey" />
+        </visual>
+      </xacro:if>
+      <xacro:unless value="${muscle}">
+        <xacro:if value="${hand_type == 'hand_e'}">
+          <visual>
+            <origin xyz="0 0 0" rpy="0 0 0" />
+            <geometry name="${prefix}forearm_visual">
+              <mesh filename="package://sr_description/hand/model/forearm.dae" scale="0.001 0.001 0.001" />
+            </geometry>
+            <material name="light_grey" />
+          </visual>
+        </xacro:if>
+        <xacro:if value="${hand_type == 'hand_e_plus'}">
+          <visual>
+            <origin xyz="0 0 0" rpy="0 0 0" />
+            <geometry name="${prefix}forearm_visual">
+              <mesh filename="package://sr_description/hand/model/forearm_visual_elbow_plate_plus.stl" scale="0.001 0.001 0.001" />
+            </geometry>
+            <xacro:light_grey/>
+          </visual>
+          <visual>
+            <origin xyz="0 0 0.015" rpy="0 0 0" />
+            <geometry>
+              <mesh filename="package://sr_description/hand/model/forearm_visual_shells_plus.stl" scale="0.001 0.001 0.001" />
+            </geometry>
+            <xacro:dark_grey/>
+          </visual>
+          <visual>
+            <origin xyz="0 0 0.1829" rpy="0 0 0" />
+            <geometry>
+              <mesh filename="package://sr_description/hand/model/forearm_visual_wrist_yaw_plus.stl" scale="0.001 0.001 0.001" />
+            </geometry>
+            <xacro:light_grey/>
+          </visual>
+        </xacro:if>
+      </xacro:unless>
       <collision>
         <xacro:if value="${muscle}">
@@ -30,10 +70,21 @@
             <cylinder radius="0.075" length="0.37" />
           </geometry>
+          <xacro:dark_grey/>
         </xacro:if>
         <xacro:unless value="${muscle}">
-          <origin xyz="0 0 0.092" rpy="0 0 0" />
-          <geometry name="${prefix}forearm_collision">
-            <cylinder radius="0.07" length="0.184"/>
-          </geometry>
+          <xacro:if value="${hand_type == 'hand_e'}">
+            <origin xyz="0 0 0.092" rpy="0 0 0" />
+            <geometry name="${prefix}forearm_collision">
+              <cylinder radius="0.07" length="0.184"/>
+            </geometry>
+            <xacro:dark_grey/>
+          </xacro:if>
+          <xacro:if value="${hand_type == 'hand_e_plus'}">
+            <origin xyz="0 0 0" rpy="0 0 0" />
+            <geometry name="${prefix}forearm_collision">
+              <mesh filename="package://sr_description/hand/model/forearm_collision_plus.stl" scale="0.001 0.001 0.001" />
+            </geometry>
+            <xacro:dark_grey/>
+          </xacro:if>
         </xacro:unless>
       </collision>
@@ -57,4 +108,9 @@
       <selfCollide>false</selfCollide>
     </gazebo>
+    <xacro:if value="${hand_type == 'hand_e_plus'}">
+      <gazebo reference="${prefix}forearm">
+        <material>Gazebo/DarkGrey</material>
+      </gazebo>
+    </xacro:if>
   </xacro:macro>
 </robot>

File: sr_description/hand/xacro/full_hand.urdf.xacro (robot description, xacro)
@@ -19,7 +19,8 @@
   <!-- lf is true if we want a little finger, false otherwise -->
   <xacro:macro name="shadowhand"
-  params="muscletrans muscle bio bt_sp ubi eli reflect prefix lf">
+  params="muscletrans muscle hand_type:='hand_e' bio bt_sp ubi eli reflect prefix lf">
+    <!--xacro:property name="hand_type" value="hand_e"/-->
     <!-- Forearm -->
-    <xacro:forearm muscle="${muscle}" prefix="${prefix}" />
+    <xacro:forearm muscle="${muscle}" hand_type="${hand_type}" prefix="${prefix}" />
     <!-- Wrist -->
     <xacro:if value="${muscle}">

File: sr_description/robots/shadowhand_left_motor.urdf.xacro (robot description, xacro)
@@ -14,5 +14,5 @@
     <origin xyz="0.0 0.0 0.0" rpy="0.0 0.0 0.0" />
   </joint>
-  <xacro:shadowhand muscletrans="false" muscle="false" bio="false" bt_sp="false"
-  ubi="false" eli="false" reflect="-1.0" prefix="lh_" lf="true" />
+  <xacro:shadowhand muscletrans="false" muscle="false" hand_type="hand_e" bio="false" bt_sp="false"
+                    ubi="false" eli="false" reflect="-1.0" prefix="lh_" lf="true" />
 </robot>

File: sr_description/robots/shadowhand_left_motor_plus.urdf.xacro (robot description, xacro)
@@ -9,10 +9,10 @@
     <!-- hand with cylindrical base drifts in gazebo, attach it to the world -->
     <link name="world" />
-    <joint name="rh_world_joint" type="fixed">
+    <joint name="lh_world_joint" type="fixed">
       <parent link="world" />
-      <child link="rh_forearm" />
+      <child link="lh_forearm" />
       <origin xyz="0.0 0.0 0.0" rpy="0.0 0.0 0.0" />
     </joint>
-    <xacro:shadowhand muscletrans="false" muscle="false" hand_type="hand_e" bio="false" bt_sp="false"
-                      ubi="false" eli="false" reflect="1.0" prefix="rh_" lf="true" />
+    <xacro:shadowhand muscletrans="false" muscle="false" hand_type="hand_e_plus" bio="false" bt_sp="false"
+                      ubi="false" eli="false" reflect="-1.0" prefix="lh_" lf="true" />
 </robot>

File: sr_description/robots/shadowhand_motor_plus.urdf.xacro (robot description, xacro)
@@ -14,5 +14,5 @@
       <origin xyz="0.0 0.0 0.0" rpy="0.0 0.0 0.0" />
     </joint>
-    <xacro:shadowhand muscletrans="false" muscle="false" hand_type="hand_e" bio="false" bt_sp="false"
+    <xacro:shadowhand muscletrans="false" muscle="false" hand_type="hand_e_plus" bio="false" bt_sp="false"
                       ubi="false" eli="false" reflect="1.0" prefix="rh_" lf="true" />
 </robot>

Commit message: added the offset to wrist yaw and fixed mesh

File: sr_description/hand/xacro/forearm/forearm.urdf.xacro (robot description, xacro)
@@ -56,5 +56,5 @@
           </visual>
           <visual>
-            <origin xyz="0 0 0.1829" rpy="0 0 0" />
+            <origin xyz="0 -0.010 0.1829" rpy="0 0 0" />
             <geometry>
               <mesh filename="package://sr_description/hand/model/forearm_visual_wrist_yaw_plus.stl" scale="0.001 0.001 0.001" />

Commit message: Changing stl by dae for visual

File: sr_description/hand/xacro/forearm/forearm.urdf.xacro (robot description, xacro)
@@ -44,21 +44,7 @@
             <origin xyz="0 0 0" rpy="0 0 0" />
             <geometry name="${prefix}forearm_visual">
-              <mesh filename="package://sr_description/hand/model/forearm_visual_elbow_plate_plus.stl" scale="0.001 0.001 0.001" />
+              <mesh filename="package://sr_description/hand/model/forearm_visual_plus.dae" scale="0.001 0.001 0.001" />
             </geometry>
-            <xacro:light_grey/>
-          </visual>
-          <visual>
-            <origin xyz="0 0 0.015" rpy="0 0 0" />
-            <geometry>
-              <mesh filename="package://sr_description/hand/model/forearm_visual_shells_plus.stl" scale="0.001 0.001 0.001" />
-            </geometry>
-            <xacro:dark_grey/>
-          </visual>
-          <visual>
-            <origin xyz="0 -0.010 0.1829" rpy="0 0 0" />
-            <geometry>
-              <mesh filename="package://sr_description/hand/model/forearm_visual_wrist_yaw_plus.stl" scale="0.001 0.001 0.001" />
-            </geometry>
-            <xacro:light_grey/>
+            <material name="light_grey" />
           </visual>
         </xacro:if>
@@ -108,9 +94,4 @@
       <selfCollide>false</selfCollide>
     </gazebo>
-    <xacro:if value="${hand_type == 'hand_e_plus'}">
-      <gazebo reference="${prefix}forearm">
-        <material>Gazebo/DarkGrey</material>
-      </gazebo>
-    </xacro:if>
   </xacro:macro>
 </robot>

Commit message: Add mesh and visual and collision part to the urdf

File: sr_description/hand/xacro/forearm/forearm.urdf.xacro (robot description, xacro)
@@ -90,4 +90,16 @@
         </xacro:unless>
       </collision>
+      <visual>
+        <origin rpy="0 1.57 -1.52" xyz="0.0 0 0.015"/>
+        <geometry name="${prefix}cable_extr_collision">
+          <mesh filename="package://sr_description/hand/model/cable_collistion_mesh.stl" scale="1 1 1" />
+        </geometry>
+      </visual>
+      <collision>
+        <origin rpy="0 1.57 -1.52" xyz="0.0 0 0.015"/>
+        <geometry name="${prefix}cable_extr_visualisation">
+          <mesh filename="package://sr_description/hand/model/cable_collistion_mesh.stl" scale="1 1 1" />
+        </geometry>
+      </collision>
     </link>
     <gazebo reference="${prefix}forearm">

Commit message: modify position slightly

File: sr_description/hand/xacro/forearm/forearm.urdf.xacro (robot description, xacro)
@@ -91,5 +91,5 @@
       </collision>
       <visual>
-        <origin rpy="0 1.57 -1.52" xyz="0.0 0 0.015"/>
+        <origin rpy="0 1.57 -1.52" xyz="0.0 0 0.01"/>
         <geometry name="${prefix}cable_extr_collision">
           <mesh filename="package://sr_description/hand/model/cable_collistion_mesh.stl" scale="1 1 1" />
@@ -97,5 +97,5 @@
       </visual>
       <collision>
-        <origin rpy="0 1.57 -1.52" xyz="0.0 0 0.015"/>
+        <origin rpy="0 1.57 -1.52" xyz="0.0 0 0.01"/>
         <geometry name="${prefix}cable_extr_visualisation">
           <mesh filename="package://sr_description/hand/model/cable_collistion_mesh.stl" scale="1 1 1" />

Commit message: kind of ready

File: sr_description/hand/xacro/forearm/forearm.urdf.xacro (robot description, xacro)
@@ -91,5 +91,5 @@
       </collision>
       <visual>
-        <origin rpy="0 1.57 -1.52" xyz="0.0 0 0.01"/>
+        <origin rpy="0 1.57 -1.52" xyz="0.0 0.073 0.0"/>
         <geometry name="${prefix}cable_extr_collision">
           <mesh filename="package://sr_description/hand/model/cable_collistion_mesh.stl" scale="1 1 1" />
@@ -97,5 +97,5 @@
       </visual>
       <collision>
-        <origin rpy="0 1.57 -1.52" xyz="0.0 0 0.01"/>
+        <origin rpy="0 1.57 -1.52" xyz="0.0 0.073 0.0"/>
         <geometry name="${prefix}cable_extr_visualisation">
           <mesh filename="package://sr_description/hand/model/cable_collistion_mesh.stl" scale="1 1 1" />

File: sr_description/hand/xacro/forearm/forearm_lite.urdf.xacro (robot description, xacro)
@@ -40,5 +40,5 @@
       </collision>
       <visual>
-        <origin rpy="0 1.57 -1.52" xyz="0.0 -0.012 0.01"/>
+        <origin rpy="0 1.57 -1.52" xyz="0.0 0.061 0.0"/>
         <geometry name="${prefix}cable_extr_collision">
           <mesh filename="package://sr_description/hand/model/cable_collistion_mesh.stl" scale="1 1 1" />
@@ -46,5 +46,5 @@
       </visual>
       <collision>
-        <origin rpy="0 1.57 -1.52" xyz="0.0 -0.012 0.01"/>
+        <origin rpy="0 1.57 -1.52" xyz="0.0 0.061 0.0"/>
         <geometry name="${prefix}cable_extr_visualisation">
           <mesh filename="package://sr_description/hand/model/cable_collistion_mesh.stl" scale="1 1 1" />

Commit message: ready

File: sr_description/hand/xacro/forearm/forearm.urdf.xacro (robot description, xacro)
@@ -91,13 +91,13 @@
       </collision>
       <visual>
-        <origin rpy="0 1.57 -1.52" xyz="0.0 0.073 0.0"/>
+        <origin rpy="0 -1.57 -1.52" xyz="0.0 0.067 0.0045"/>
         <geometry name="${prefix}cable_extr_collision">
-          <mesh filename="package://sr_description/hand/model/cable_collistion_mesh.stl" scale="1 1 1" />
+          <mesh filename="package://sr_description/hand/model/cable_collision_mesh.stl" scale="1 1 1" />
         </geometry>
       </visual>
       <collision>
-        <origin rpy="0 1.57 -1.52" xyz="0.0 0.073 0.0"/>
+        <origin rpy="0 -1.57 -1.52" xyz="0.0 0.067 0.0045"/>
         <geometry name="${prefix}cable_extr_visualisation">
-          <mesh filename="package://sr_description/hand/model/cable_collistion_mesh.stl" scale="1 1 1" />
+          <mesh filename="package://sr_description/hand/model/cable_collision_mesh.stl" scale="1 1 1" />
         </geometry>
       </collision>

File: sr_description/hand/xacro/forearm/forearm_lite.urdf.xacro (robot description, xacro)
@@ -40,13 +40,13 @@
       </collision>
       <visual>
-        <origin rpy="0 1.57 -1.52" xyz="0.0 0.061 0.0"/>
+        <origin rpy="0 -1.57 -1.52" xyz="0.0 0.055 0.0"/>
         <geometry name="${prefix}cable_extr_collision">
-          <mesh filename="package://sr_description/hand/model/cable_collistion_mesh.stl" scale="1 1 1" />
+          <mesh filename="package://sr_description/hand/model/cable_collision_mesh.stl" scale="1 1 1" />
         </geometry>
       </visual>
       <collision>
-        <origin rpy="0 1.57 -1.52" xyz="0.0 0.061 0.0"/>
+        <origin rpy="0 -1.57 -1.52" xyz="0.0 0.055 0.0"/>
         <geometry name="${prefix}cable_extr_visualisation">
-          <mesh filename="package://sr_description/hand/model/cable_collistion_mesh.stl" scale="1 1 1" />
+          <mesh filename="package://sr_description/hand/model/cable_collision_mesh.stl" scale="1 1 1" />
         </geometry>
       </collision>

Commit message: minor change

File: sr_description/hand/xacro/forearm/forearm.urdf.xacro (robot description, xacro)
@@ -91,5 +91,5 @@
       </collision>
       <visual>
-        <origin rpy="0 -1.57 -1.52" xyz="0.0 0.067 0.0045"/>
+        <origin rpy="0 -1.57 -1.57" xyz="0.0 0.067 0.0045"/>
         <geometry name="${prefix}cable_extr_collision">
           <mesh filename="package://sr_description/hand/model/cable_collision_mesh.stl" scale="1 1 1" />
@@ -97,5 +97,5 @@
       </visual>
       <collision>
-        <origin rpy="0 -1.57 -1.52" xyz="0.0 0.067 0.0045"/>
+        <origin rpy="0 -1.57 -1.57" xyz="0.0 0.067 0.0045"/>
         <geometry name="${prefix}cable_extr_visualisation">
           <mesh filename="package://sr_description/hand/model/cable_collision_mesh.stl" scale="1 1 1" />

File: sr_description/hand/xacro/forearm/forearm_lite.urdf.xacro (robot description, xacro)
@@ -40,5 +40,5 @@
       </collision>
       <visual>
-        <origin rpy="0 -1.57 -1.52" xyz="0.0 0.055 0.0"/>
+        <origin rpy="0 -1.57 -1.57" xyz="0.0 0.055 0.0"/>
         <geometry name="${prefix}cable_extr_collision">
           <mesh filename="package://sr_description/hand/model/cable_collision_mesh.stl" scale="1 1 1" />
@@ -46,5 +46,5 @@
       </visual>
       <collision>
-        <origin rpy="0 -1.57 -1.52" xyz="0.0 0.055 0.0"/>
+        <origin rpy="0 -1.57 -1.57" xyz="0.0 0.055 0.0"/>
         <geometry name="${prefix}cable_extr_visualisation">
           <mesh filename="package://sr_description/hand/model/cable_collision_mesh.stl" scale="1 1 1" />

Commit message: collision only with ut10

File: sr_description/hand/xacro/forearm/forearm.urdf.xacro (robot description, xacro)
@@ -13,5 +13,5 @@
     </material>
   </xacro:macro>
-  <xacro:macro name="forearm" params="muscle hand_type:='hand_e' prefix">
+  <xacro:macro name="forearm" params="muscle hand_type:='hand_e' prefix cable_collision:='false'">
     <link name="${prefix}forearm">
       <inertial>
@@ -90,16 +90,18 @@
         </xacro:unless>
       </collision>
-      <visual>
-        <origin rpy="0 -1.57 -1.57" xyz="0.0 0.067 0.0045"/>
-        <geometry name="${prefix}cable_extr_collision">
-          <mesh filename="package://sr_description/hand/model/cable_collision_mesh.stl" scale="1 1 1" />
-        </geometry>
-      </visual>
-      <collision>
-        <origin rpy="0 -1.57 -1.57" xyz="0.0 0.067 0.0045"/>
-        <geometry name="${prefix}cable_extr_visualisation">
-          <mesh filename="package://sr_description/hand/model/cable_collision_mesh.stl" scale="1 1 1" />
-        </geometry>
-      </collision>
+      <xacro:if value="${cable_collision}">
+        <visual>
+          <origin rpy="0 -1.57 -1.57" xyz="0.0 0.067 0.0045"/>
+          <geometry name="${prefix}cable_extr_collision">
+            <mesh filename="package://sr_description/hand/model/cable_collision_mesh.stl" scale="1 1 1" />
+          </geometry>
+        </visual>
+        <collision>
+          <origin rpy="0 -1.57 -1.57" xyz="0.0 0.067 0.0045"/>
+          <geometry name="${prefix}cable_extr_visualisation">
+            <mesh filename="package://sr_description/hand/model/cable_collision_mesh.stl" scale="1 1 1" />
+          </geometry>
+        </collision>
+      </xacro:if>
     </link>
     <gazebo reference="${prefix}forearm">

File: sr_description/hand/xacro/forearm/forearm_lite.urdf.xacro (robot description, xacro)
@@ -2,5 +2,5 @@
   <!-- muscle is true for muscle hand or false for motor hand -->
   <!-- prefix can be anything but usually is "r_" or  "l_" for right and left hands distinction -->
-  <xacro:macro name="forearm" params="muscle prefix">
+  <xacro:macro name="forearm" params="muscle prefix cable_collision:='false'">
     <link name="${prefix}forearm">
       <inertial>
@@ -39,16 +39,18 @@
         </xacro:unless>
       </collision>
-      <visual>
-        <origin rpy="0 -1.57 -1.57" xyz="0.0 0.055 0.0"/>
-        <geometry name="${prefix}cable_extr_collision">
-          <mesh filename="package://sr_description/hand/model/cable_collision_mesh.stl" scale="1 1 1" />
-        </geometry>
-      </visual>
-      <collision>
-        <origin rpy="0 -1.57 -1.57" xyz="0.0 0.055 0.0"/>
-        <geometry name="${prefix}cable_extr_visualisation">
-          <mesh filename="package://sr_description/hand/model/cable_collision_mesh.stl" scale="1 1 1" />
-        </geometry>
-      </collision>
+      <xacro:if value="${cable_collision}">
+        <visual>
+          <origin rpy="0 -1.57 -1.57" xyz="0.0 0.055 0.0"/>
+          <geometry name="${prefix}cable_extr_collision">
+            <mesh filename="package://sr_description/hand/model/cable_collision_mesh.stl" scale="1 1 1" />
+          </geometry>
+        </visual>
+        <collision>
+          <origin rpy="0 -1.57 -1.57" xyz="0.0 0.055 0.0"/>
+          <geometry name="${prefix}cable_extr_visualisation">
+            <mesh filename="package://sr_description/hand/model/cable_collision_mesh.stl" scale="1 1 1" />
+          </geometry>
+        </collision>
+      </xacro:if>
     </link>
   </xacro:macro>

File: sr_description/hand/xacro/full_hand.urdf.xacro (robot description, xacro)
@@ -19,8 +19,8 @@
   <!-- lf is true if we want a little finger, false otherwise -->
   <xacro:macro name="shadowhand"
-  params="muscletrans muscle hand_type:='hand_e' bio bt_sp ubi eli reflect prefix lf">
+  params="muscletrans muscle hand_type:='hand_e' bio bt_sp ubi eli reflect prefix lf cable_collision:='false'">
     <!--xacro:property name="hand_type" value="hand_e"/-->
     <!-- Forearm -->
-    <xacro:forearm muscle="${muscle}" hand_type="${hand_type}" prefix="${prefix}" />
+    <xacro:forearm muscle="${muscle}" hand_type="${hand_type}" prefix="${prefix}" cable_collision="${cable_collision}"/>
     <!-- Wrist -->
     <xacro:if value="${muscle}">
