Commit message: changing name to cable_mesh

File: sr_description/hand/xacro/forearm/forearm.urdf.xacro (robot description, xacro)
@@ -13,5 +13,5 @@
     </material>
   </xacro:macro>
-  <xacro:macro name="forearm" params="muscle hand_type:='hand_e' prefix cable_collision:='false'">
+  <xacro:macro name="forearm" params="muscle hand_type:='hand_e' prefix cable_mesh:='false'">
     <link name="${prefix}forearm">
       <inertial>
@@ -90,5 +90,5 @@
         </xacro:unless>
       </collision>
-      <xacro:if value="${cable_collision}">
+      <xacro:if value="${cable_mesh}">
         <visual>
           <origin rpy="0 -1.57 -1.57" xyz="0.0 0.067 0.0045"/>

File: sr_description/hand/xacro/forearm/forearm_lite.urdf.xacro (robot description, xacro)
@@ -2,5 +2,5 @@
   <!-- muscle is true for muscle hand or false for motor hand -->
   <!-- prefix can be anything but usually is "r_" or  "l_" for right and left hands distinction -->
-  <xacro:macro name="forearm" params="muscle prefix cable_collision:='false'">
+  <xacro:macro name="forearm" params="muscle prefix cable_mesh:='false'">
     <link name="${prefix}forearm">
       <inertial>
@@ -39,5 +39,5 @@
         </xacro:unless>
       </collision>
-      <xacro:if value="${cable_collision}">
+      <xacro:if value="${cable_mesh}">
         <visual>
           <origin rpy="0 -1.57 -1.57" xyz="0.0 0.055 0.0"/>

File: sr_description/hand/xacro/full_hand.urdf.xacro (robot description, xacro)
@@ -19,8 +19,8 @@
   <!-- lf is true if we want a little finger, false otherwise -->
   <xacro:macro name="shadowhand"
-  params="muscletrans muscle hand_type:='hand_e' bio bt_sp ubi eli reflect prefix lf cable_collision:='false'">
+  params="muscletrans muscle hand_type:='hand_e' bio bt_sp ubi eli reflect prefix lf cable_mesh:='false'">
     <!--xacro:property name="hand_type" value="hand_e"/-->
     <!-- Forearm -->
-    <xacro:forearm muscle="${muscle}" hand_type="${hand_type}" prefix="${prefix}" cable_collision="${cable_collision}"/>
+    <xacro:forearm muscle="${muscle}" hand_type="${hand_type}" prefix="${prefix}" cable_mesh="${cable_mesh}"/>
     <!-- Wrist -->
     <xacro:if value="${muscle}">

File: sr_description/hand/xacro/hand_lite.urdf.xacro (robot description, xacro)
@@ -18,7 +18,7 @@
   <!-- prefix can be anything but usually is "r_" or  "l_" for right and left hands distinction -->
   <xacro:macro name="shadowhand"
-  params="muscletrans muscle bio bt_sp ubi eli reflect prefix extra_lite  cable_collision:='false'">
+  params="muscletrans muscle bio bt_sp ubi eli reflect prefix extra_lite  cable_mesh:='false'">
     <!-- Forearm -->
-    <xacro:forearm muscle="${muscle}" prefix="${prefix}" cable_collision="${cable_collision}"/>
+    <xacro:forearm muscle="${muscle}" prefix="${prefix}" cable_mesh="${cable_mesh}"/>
     <!-- Wrist -->
     <!-- Completely fixed on the lite hand. Bent back at 40 degrees -->

Commit message: fixing according to rev

File: sr_description/hand/xacro/forearm/forearm.urdf.xacro (robot description, xacro)
@@ -93,5 +93,5 @@
         <visual>
           <origin rpy="0 -1.57 -1.57" xyz="0.0 0.067 0.0045"/>
-          <geometry name="${prefix}cable_extr_collision">
+          <geometry name="${prefix}cable_extr_visualisation">
             <mesh filename="package://sr_description/hand/model/cable_collision_mesh.stl" scale="1 1 1" />
           </geometry>
@@ -99,5 +99,5 @@
         <collision>
           <origin rpy="0 -1.57 -1.57" xyz="0.0 0.067 0.0045"/>
-          <geometry name="${prefix}cable_extr_visualisation">
+          <geometry name="${prefix}cable_extr_collision">
             <mesh filename="package://sr_description/hand/model/cable_collision_mesh.stl" scale="1 1 1" />
           </geometry>

File: sr_description/hand/xacro/forearm/forearm_lite.urdf.xacro (robot description, xacro)
@@ -42,5 +42,5 @@
         <visual>
           <origin rpy="0 -1.57 -1.57" xyz="0.0 0.055 0.0"/>
-          <geometry name="${prefix}cable_extr_collision">
+          <geometry name="${prefix}cable_extr_visualisation">
             <mesh filename="package://sr_description/hand/model/cable_collision_mesh.stl" scale="1 1 1" />
           </geometry>
@@ -48,5 +48,5 @@
         <collision>
           <origin rpy="0 -1.57 -1.57" xyz="0.0 0.055 0.0"/>
-          <geometry name="${prefix}cable_extr_visualisation">
+          <geometry name="${prefix}cable_extr_collision">
             <mesh filename="package://sr_description/hand/model/cable_collision_mesh.stl" scale="1 1 1" />
           </geometry>
