Commit message: Added mucle hand

File: sr_description/hand/xacro/forearm/forearm_c.urdf.xacro (robot description, xacro)
@@ -21,5 +21,5 @@
         <origin xyz="0 0 0" rpy="0 0 0" />
         <geometry name="${prefix}forearm_visual">
-          <mesh filename="package://sr_description/meshes/products/hand_m/C6M2/forearm.dae" scale="1.0 1.0 1.0" />
+          <mesh filename="package://sr_description/meshes/products/${hand_type}/${hand_version}/forearm_${hand_version}.dae"/>
         </geometry>
         <material name="Grey" />

File: sr_description/hand/xacro/hand.urdf.xacro (robot description, xacro)
@@ -22,8 +22,8 @@
        <xacro:sr_hand_g />
     </xacro:if>
-    <!--xacro:if value="${hand_type == 'hand_c'}">
+    <xacro:if value="${hand_type == 'hand_c'}">
        <xacro:include filename="$(find sr_description)/hand/xacro/hand_c.urdf.xacro" />
        <xacro:sr_hand_c />
-    </xacro:if-->
+    </xacro:if>
   </xacro:macro>
 </robot>

File: sr_description/hand/xacro/hand_c.urdf.xacro (robot description, xacro)
@@ -1,7 +1,4 @@
-<robot xmlns:sensor="http://playerstage.sourceforge.net/gazebo/xmlschema/#sensor"
-       xmlns:controller="http://playerstage.sourceforge.net/gazebo/xmlschema/#controller"
-       xmlns:interface="http://playerstage.sourceforge.net/gazebo/xmlschema/#interface"
-       xmlns:xacro="http://www.ros.org/wiki/xacro">
-  <xacro:include filename="$(find sr_description)/hand/xacro/forearm/forearm_e.urdf.xacro" />
+<robot xmlns:xacro="http://www.ros.org/wiki/xacro">
+  <xacro:include filename="$(find sr_description)/hand/xacro/forearm/forearm_c.urdf.xacro" />
   <xacro:include filename="$(find sr_description)/hand/xacro/wrist/wrist.urdf.xacro" />
   <xacro:include filename="$(find sr_description)/hand/xacro/palm/palm_e.urdf.xacro" />
@@ -14,8 +11,8 @@
   <!-- prox_sensors: plain or dict-like string specifying the proximal (tactile) sensors -->
   <!-- palm_sensor: specifies the palm tactile sensor -->
-  <xacro:macro name="sr_hand_e" params="hand_version:=^ reflect:=^ prefix:=^ fingers:=^|all tip_sensors:=^|pst
+  <xacro:macro name="sr_hand_c" params="hand_version:=^ reflect:=^ prefix:=^ fingers:=^|all tip_sensors:=^|pst
                prox_sensors:=^|none mid_sensors:=^|none palm_sensor:=^|none">
     <!-- Unify hand type parameter -->
-    <xacro:property name="hand_type" value="hand_e" />
+    <xacro:property name="hand_type" value="hand_c" />
     <xacro:include filename="$(find sr_description)/hand/xacro/process_hand_type_parameter.xacro" />
     <!-- Process fingers parameter, also handling deprecated lf -->
@@ -28,5 +25,5 @@
     <!-- Wrist -->
     <xacro:wrist parent="${prefix}forearm">
-      <origin xyz="0 -0.010 0.21301" rpy="0 0 0" />
+      <origin xyz="0 0 0.4096" rpy="0 0 0" />
     </xacro:wrist>
     <!-- Palm -->

File: sr_description/hand/xacro/process_hand_type_parameter.xacro (robot description, xacro)
@@ -24,3 +24,6 @@
 		<xacro:property name="hand_type" value="G" />
 	</xacro:if>
+	<xacro:if value="${hand_type.lower() == 'hand_c'}">
+		<xacro:property name="hand_type" value="C" />
+	</xacro:if>
 </robot>
