Commit message: Added mounting plates for hand e and hand g (#137)
* added mounting plate

* exported and added

* added temporal mount for hand g

* added argument

* Changing arm to mounting plate

* Changing arm to mounting plate

* Fixing coordinates

* Fixing coordinates

* Fixing coordinates

* Fixing coordinates

* Fixing coordinates

* Fixing coordinates

* Fixing coordinates

* Fixing coordinates

* Rename ur_hand_g_mounting_plate.dae to mounting_plate_G1M5.dae

* Changing hand g to make it compatible

* Changing hand g to make it compatible

* Update forearm_g.urdf.xacro

* Update forearm_g.urdf.xacro

* Update forearm_g.urdf.xacro

* Update forearm_g.urdf.xacro

* Update forearm_g.urdf.xacro

* Fixing forearm files

* Fixing mounting plate for hand E

* Fixing mounting plate for hand E

* Fixing mounting plate for hand E

* Fixing mounting plate for hand E

* Fixing mounting plate for hand E

* Fixing mounting plate for hand E

* Fixing mounting plate for hand E

* Fixing mounting plate for hand E

* Fixing mounting plate for hand E

* Fixing mounting plate for hand E

* Fixing mounting plate for hand E

* Added color to mounting plate meshes

* validate boolean mounting plate var

* Update process_hand_type_version_side_parameters.xacro

Co-authored-by: Beatriz Leon <beatriz@shadowrobot.com>

File: sr_description/hand/xacro/forearm/forearm_e.urdf.xacro (robot description, xacro)
@@ -10,5 +10,11 @@
     </material>
   </xacro:macro>
-  <xacro:macro name="forearm" params="hand_type:=^ hand_version:=^ prefix:=^">
+  <xacro:if value="${mounting_plate}">
+    <xacro:property name="mounting_plate_offset" value="0.006" />
+  </xacro:if>
+  <xacro:unless value="${mounting_plate}">
+    <xacro:property name="mounting_plate_offset" value="0.0" />
+  </xacro:unless>
+  <xacro:macro name="forearm" params="hand_type:=^ hand_version:=^ prefix:=^ mounting_plate:=^">
     <link name="${prefix}forearm">
       <inertial>
@@ -18,5 +24,5 @@
       </inertial>
       <visual>
-        <origin xyz="0 0 0" rpy="0 0 0" />
+        <origin xyz="0 0 ${mounting_plate_offset}" rpy="0 0 0" />
         <geometry name="${prefix}forearm_visual">
           <mesh filename="package://sr_description/meshes/components/forearm/forearm_${hand_version}.dae" scale="0.001 0.001 0.001" />
@@ -25,5 +31,5 @@
       </visual>
       <collision>
-        <origin xyz="0 0 0" rpy="0 0 0" />
+        <origin xyz="0 0 ${mounting_plate_offset}" rpy="0 0 0" />
         <geometry name="${prefix}forearm_collision">
           <mesh filename="package://sr_description/meshes/components/forearm/forearm_collision_${hand_version}.dae" scale="0.001 0.001 0.001" />
@@ -32,9 +38,24 @@
       <!-- wrist mount -->
       <collision>
-        <origin xyz="0 -0.01 0.181" rpy="0 0.78 0" />
+        <origin xyz="0 -0.01 ${0.181+mounting_plate_offset}" rpy="0 0.78 0" />
         <geometry>
           <box size="0.07 0.07 0.07" />
         </geometry>
       </collision>
+      <!-- mounting plate in case the hand is attached to an arm -->
+      <xacro:if value="${mounting_plate}">
+        <visual>
+          <origin xyz="0 0 0" rpy="0 0 0" />
+          <geometry name="${prefix}mounting_plate">
+            <mesh filename="package://sr_description/meshes/components/mounting_plate/mounting_plate_${hand_version}.dae" scale="0.001 0.001 0.001" />
+          </geometry>
+        </visual>
+        <collision>
+          <origin xyz="0 0 0.002" rpy="0 0 0" />
+          <geometry>
+            <cylinder radius="0.0675" length="0.008" />
+          </geometry>
+        </collision>
+      </xacro:if>
       <!-- TODO: Make a decision on whether to add the connector or not -->
       <!--visual>
@@ -43,11 +64,5 @@
           <mesh filename="package://sr_description/meshes/components/cable_connector/cable_connector_base_${hand_version}.dae" scale="0.001 0.001 0.001" />
         </geometry>
-      </visual>
-      <collision>
-        <origin rpy="0 -1.57 -1.57" xyz="0.0 0.067 0.0045"/>
-        <geometry name="${prefix}cable_extr_collision">
-          <mesh filename="package://sr_description/meshes/components/cable_connector/cable_connector_base_${hand_version}.dae" scale="0.001 0.001 0.001" />
-        </geometry>
-      </collision-->
+      </visual-->
     </link>
     <gazebo reference="${prefix}forearm">

File: sr_description/hand/xacro/forearm/forearm_g.urdf.xacro (robot description, xacro)
@@ -1,4 +1,10 @@
 <robot xmlns:xacro="http://www.ros.org/wiki/xacro">
-  <xacro:macro name="forearm" params="hand_type:=^ prefix:=^">
+  <xacro:if value="${mounting_plate}">
+    <xacro:property name="mounting_plate_offset" value="0.005" />
+  </xacro:if>
+  <xacro:unless value="${mounting_plate}">
+    <xacro:property name="mounting_plate_offset" value="0.0" />
+  </xacro:unless>
+  <xacro:macro name="forearm" params="hand_type:=^ hand_version:=^ prefix:=^ mounting_plate:=^">
     <link name="${prefix}forearm">
       <inertial>
@@ -6,9 +12,8 @@
         <!-- TODO: This is a rough estimate. Total hand is 2359g -->
         <mass value="1.8" />
-        <inertia ixx="0.108" ixy="0.0" ixz="0.0" iyy="0.108"
-        iyz="0.0" izz="0.054" />
+        <inertia ixx="0.108" ixy="0.0" ixz="0.0" iyy="0.108" iyz="0.0" izz="0.054" />
       </inertial>
       <visual>
-        <origin xyz="0 0 0" rpy="0 0 ${pi/2}" />
+        <origin xyz="0 0 ${mounting_plate_offset}" rpy="0 0 ${pi/2}" />
         <geometry name="${prefix}forearm_visual">
           <mesh filename="package://sr_description/meshes/components/forearm/forearm_${hand_version}.dae" scale="1.0 1.0 1.0" />
@@ -17,23 +22,28 @@
       </visual>
       <collision>
-        <origin xyz="0 0 0.065" rpy="0 0 0" />
+        <origin xyz="0 0 ${0.065+mounting_plate_offset}" rpy="0 0 0" />
         <geometry name="${prefix}forearm_collision">
           <box size="0.120 0.109 0.130" />
         </geometry>
       </collision>
-      <!-- TODO: Make a decision on whether to add the connector or not -->
-      <!--visual>
-        <origin rpy="0 -1.57 -1.57" xyz="0.0 0.055 0.0"/>
-        <geometry name="${prefix}cable_extr_visualisation">
-          <mesh filename="package://sr_description/meshes/components/cable_connector/cable_connector_base_${hand_version}.dae" scale="1 1 1" />
-        </geometry>
-      </visual>
-      <collision>
-        <origin rpy="0 -1.57 -1.57" xyz="0.0 0.055 0.0"/>
-        <geometry name="${prefix}cable_extr_collision">
-          <mesh filename="package://sr_description/components/cable_connector/cable_connector_base_${hand_version}.dae" scale="1 1 1" />
-        </geometry>
-      </collision-->
+      <!-- mounting plate in case the hand is attached to an arm -->
+      <xacro:if value="${mounting_plate}">
+        <visual>
+          <origin xyz="0 0 0" rpy="0 0 0" />
+          <geometry name="${prefix}mounting_plate">
+            <mesh filename="package://sr_description/meshes/components/mounting_plate/mounting_plate_${hand_version}.dae" scale="0.001 0.001 0.001" />
+          </geometry>
+        </visual>
+        <collision>
+          <origin xyz="0 0 0.002" rpy="0 0 0" />
+          <geometry>
+            <box size="0.120 0.109 0.006" />
+          </geometry>
+        </collision>
+      </xacro:if>
     </link>
+    <gazebo reference="${prefix}forearm">
+      <selfCollide>false</selfCollide>
+    </gazebo>
   </xacro:macro>
 </robot>

File: sr_description/hand/xacro/hand.urdf.xacro (robot description, xacro)
@@ -3,5 +3,5 @@
        xmlns:controller="http://playerstage.sourceforge.net/gazebo/xmlschema/#controller"
        xmlns:interface="http://playerstage.sourceforge.net/gazebo/xmlschema/#interface">
-  <xacro:macro name="sr_hand" params="hand_type hand_version side fingers tip_sensors prox_sensors mid_sensors palm_sensor">
+  <xacro:macro name="sr_hand" params="hand_type hand_version side fingers tip_sensors prox_sensors mid_sensors palm_sensor mounting_plate">
     <!-- Process hand type, version and side parameters -->
     <xacro:include filename="$(find sr_description)/hand/xacro/process_hand_type_version_side_parameters.xacro" />

File: sr_description/hand/xacro/hand_e.urdf.xacro (robot description, xacro)
@@ -14,5 +14,5 @@
   <!-- palm_sensor: specifies the palm tactile sensor -->
   <xacro:macro name="sr_hand_e" params="hand_version:=^ reflect:=^ prefix:=^ fingers:=^|all tip_sensors:=^|pst
-               prox_sensors:=^|none mid_sensors:=^|none palm_sensor:=^|none">
+               prox_sensors:=^|none mid_sensors:=^|none palm_sensor:=^|none mounting_plate:=^|false">
     <!-- Process fingers parameter -->
     <xacro:property name="_all_finger_tokens_" value="${python.set('th ff mf rf lf'.split())}" />

File: sr_description/hand/xacro/process_hand_type_version_side_parameters.xacro (robot description, xacro)
@@ -4,13 +4,17 @@
 	<xacro:property name="allowed_hand_versions" value="${python.set('E3M5 E2M3 C6M2 G1M5'.split())}"/>
         <xacro:property name="allowed_sides" value="${python.set('right left'.split())}"/>
+        <xacro:property name="allowed_mounting_plate" value="${python.set([False, True])}"/>
 	<!-- Validate hand type -->
 	<xacro:validate_tokens tokens="${python.set([hand_type])}" valid="${allowed_hand_types}" name="hand type specifier" />
 	<!-- Validate hand version -->
 	<xacro:validate_tokens tokens="${python.set([hand_version])}" valid="${allowed_hand_versions}" name="hand version specifier" />
+        <!-- Validate hand version corresponds to hand type -->
+	<xacro:unless value="${hand_type.lower()[-1] == hand_version.lower()[0]}">
+        	${xacro.error("Parameter 'hand_type' ("+hand_type+") doesn't comply with 'hand_version' ("+hand_version+")")}
+        </xacro:unless>
 	<!-- Validate side -->
 	<xacro:validate_tokens tokens="${python.set([side])}" valid="${allowed_sides}" name="hand side specifier" />
-	<xacro:unless value="${hand_type.lower()[-1] == hand_version.lower()[0]}">
-            ${xacro.error("Parameter 'hand_type' ("+hand_type+") doesn't comply with 'hand_version' ("+hand_version+")")}
-        </xacro:unless>
+        <!-- Validate mounting plate options -->
+        <xacro:validate_tokens tokens="${python.set([mounting_plate])}" valid="${allowed_mounting_plate}" name="hand mounting_plate specifier" />
 	<!-- Normalize hand_type to be lower case -->
 	<xacro:property name="hand_type" value="${hand_type.lower()}" lazy_eval="false" />

File: sr_description/robots/sr_hand.urdf.xacro (robot description, xacro)
@@ -15,4 +15,5 @@
   <xacro:arg name="prox_sensors" default="none"/>
   <xacro:arg name="palm_sensor" default="none"/>
+  <xacro:arg name="mounting_plate" default="false"/>
   <link name="world" />
   <xacro:if value="${'$(arg side)' == 'right'}">
@@ -32,4 +33,4 @@
   <xacro:sr_hand hand_type="$(arg hand_type)" hand_version="$(arg hand_version)" side="$(arg side)"
                  fingers="$(arg fingers)" tip_sensors="$(arg tip_sensors)" mid_sensors="$(arg mid_sensors)"
-                 prox_sensors="$(arg prox_sensors)" palm_sensor="$(arg palm_sensor)"/>
+                 prox_sensors="$(arg prox_sensors)" palm_sensor="$(arg palm_sensor)" mounting_plate="$(arg mounting_plate)"/>
 </robot>

File: sr_description/robots/sr_hand_bimanual.urdf.xacro (robot description, xacro)
@@ -15,4 +15,5 @@
   <xacro:arg name="right_prox_sensors" default="none"/>
   <xacro:arg name="right_palm_sensor" default="none"/>
+  <xacro:arg name="right_mounting_plate" default="false"/>
   <xacro:arg name="left_hand_type" default="hand_e"/>
   <xacro:arg name="left_hand_version" default="E3M5"/>
@@ -22,4 +23,5 @@
   <xacro:arg name="left_prox_sensors" default="none"/>
   <xacro:arg name="left_palm_sensor" default="none"/>
+  <xacro:arg name="left_mounting_plate" default="false"/>
   <link name="world" />
   <joint name="world_joint" type="fixed">
@@ -30,8 +32,8 @@
   <xacro:sr_hand side="right" hand_type="$(arg right_hand_type)" hand_version="$(arg right_hand_version)"
                  fingers="$(arg right_fingers)" tip_sensors="$(arg right_tip_sensors)" mid_sensors="$(arg right_mid_sensors)"
-                 prox_sensors="$(arg right_prox_sensors)" palm_sensor="$(arg right_palm_sensor)"/>
+                 prox_sensors="$(arg right_prox_sensors)" palm_sensor="$(arg right_palm_sensor)" mounting_plate="$(arg right_mounting_plate)"/>
   <xacro:sr_hand side="left" hand_type="$(arg left_hand_type)" hand_version="$(arg left_hand_version)"
                  fingers="$(arg left_fingers)" tip_sensors="$(arg left_tip_sensors)" mid_sensors="$(arg left_mid_sensors)"
-                 prox_sensors="$(arg left_prox_sensors)" palm_sensor="$(arg left_palm_sensor)"/>
+                 prox_sensors="$(arg left_prox_sensors)" palm_sensor="$(arg left_palm_sensor)" mounting_plate="$(arg left_mounting_plate)"/>
   <joint name="right_hand_to_left_hand" type="fixed">
     <parent link="rh_forearm" />
