Commit message: extend j3 urdf limit (tested)

File: sr_description/hand/xacro/finger/proximal/proximal.urdf.xacro (robot description, xacro)
@@ -42,5 +42,5 @@
       <origin xyz="0 0 0" rpy="0 0 0" />
       <axis xyz="1 0 0" />
-      <limit lower="0" upper="${M_PI/2}" effort="2"
+      <limit lower="-0.2618" upper="${M_PI/2}" effort="2"
       velocity="2.0" />
       <dynamics damping="0.1" />

File: sr_description/hand/xacro/thumb/thdistal.urdf.xacro (robot description, xacro)
@@ -192,5 +192,5 @@
         <origin xyz="0 0 0.032" rpy="0 0 ${-M_PI/2}" />
         <axis xyz="1 0 0" />
-        <limit lower="0" upper="${90.0*M_PI/180}" effort="1.0"
+        <limit lower="-0.2618" upper="${90.0*M_PI/180}" effort="1.0"
         velocity="4.0" />
         <dynamics damping="0.2" />

Commit message: Update sr_description/hand/xacro/finger/proximal/proximal.urdf.xacro
Co-Authored-By: Beatriz Leon <beatriz@shadowrobot.com>

File: sr_description/hand/xacro/finger/proximal/proximal.urdf.xacro (robot description, xacro)
@@ -42,5 +42,5 @@
       <origin xyz="0 0 0" rpy="0 0 0" />
       <axis xyz="1 0 0" />
-      <limit lower="-0.2618" upper="${M_PI/2}" effort="2"
+      <limit lower="-${15.0*M_PI/180}" upper="${M_PI/2}" effort="2"
       velocity="2.0" />
       <dynamics damping="0.1" />
