Commit message: Changing M_PI to pi - lint check fix

File: sr_description/arm/xacro/base/shadowarm_base.urdf.xacro (robot description, xacro)
@@ -1,4 +1,4 @@
 <robot xmlns:xacro="http://www.ros.org/wiki/xacro">
-  <xacro:property name="M_PI" value="3.1415926535897931" />
+  <xacro:property name="pi" value="3.1415926535897931" />
   <xacro:macro name="shadowarm_base">
     <link name="shadowarm_base">

File: sr_description/hand/xacro/ff_biotac_hand.urdf.xacro (robot description, xacro)
@@ -8,5 +8,5 @@
   <xacro:include filename="$(find sr_description)/hand/xacro/finger/fingers.urdf.xacro" />
   <xacro:include filename="$(find sr_description)/hand/xacro/thumb/thumb.urdf.xacro" />
-  <xacro:property name="M_PI" value="3.1415926535897931" />
+  <xacro:property name="pi" value="3.1415926535897931" />
   <!-- muscletrans is true for muscle transmission to be used, false to use motor transmission -->
   <!-- muscle is true for muscle hand or false for motor hand -->

File: sr_description/hand/xacro/finger/biotac/biotac.urdf.xacro (robot description, xacro)
@@ -61,5 +61,5 @@
       <origin xyz="0 0 0.045" rpy="0 0 0" />
       <axis xyz="1 0 0" />
-      <limit lower="0" upper="${M_PI/2}" effort="2.0"
+      <limit lower="0" upper="${pi/2}" effort="2.0"
       velocity="2.0" />
       <dynamics damping="0.1" />
@@ -82,5 +82,5 @@
       <origin xyz="0 0 0.02" rpy="0 0 0" />
       <axis xyz="1 0 0" />
-      <limit lower="${20*M_PI/180}" upper="${20.1*M_PI/180}"
+      <limit lower="${20*pi/180}" upper="${20.1*pi/180}"
       effort="0.0" velocity="2.0" />
       <dynamics damping="0.5" />

File: sr_description/hand/xacro/finger/distal/distal.urdf.xacro (robot description, xacro)
@@ -106,10 +106,10 @@
         <xacro:if value="${bio}">
           <!-- biotac fixed distal joint -->
-          <limit lower="${20/180*M_PI}" upper="${20/180*M_PI}"
+          <limit lower="${20/180*pi}" upper="${20/180*pi}"
           effort="10" velocity="2.0" />
         </xacro:if>
         <xacro:unless value="${bio}">
           <!-- standard distal joint -->
-          <limit lower="0" upper="${M_PI/2}" effort="2"
+          <limit lower="0" upper="${pi/2}" effort="2"
           velocity="2.0" />
         </xacro:unless>

File: sr_description/hand/xacro/finger/knuckle/knuckle.urdf.xacro (robot description, xacro)
@@ -43,5 +43,5 @@
       <xacro:insert_block name="origin" />
       <xacro:insert_block name="axis" />
-      <limit lower="${-20/180*M_PI}" upper="${20/180*M_PI}"
+      <limit lower="${-20/180*pi}" upper="${20/180*pi}"
       effort="2" velocity="2.0" />
       <dynamics damping="0.1" />

File: sr_description/hand/xacro/finger/lfmetacarpal/lfmetacarpal.urdf.xacro (robot description, xacro)
@@ -41,5 +41,5 @@
       <origin xyz="${reflect*-0.033} 0 0.02071" rpy="0 0 0" />
       <axis xyz="0.573576436 0 ${reflect*0.819152044}" />
-      <limit lower="0" upper="${45/180*M_PI}" effort="2"
+      <limit lower="0" upper="${45/180*pi}" effort="2"
       velocity="2.0" />
       <dynamics damping="0.1" />

File: sr_description/hand/xacro/finger/middle/middle.urdf.xacro (robot description, xacro)
@@ -54,5 +54,5 @@
       <origin xyz="0 0 0.045" rpy="0 0 0" />
       <axis xyz="1 0 0" />
-      <limit lower="0" upper="${M_PI/2}" effort="2"
+      <limit lower="0" upper="${pi/2}" effort="2"
       velocity="2.0" />
       <dynamics damping="0.1" />

File: sr_description/hand/xacro/finger/proximal/proximal.urdf.xacro (robot description, xacro)
@@ -42,5 +42,5 @@
       <origin xyz="0 0 0" rpy="0 0 0" />
       <axis xyz="1 0 0" />
-      <limit lower="-${15.0*M_PI/180}" upper="${M_PI/2}" effort="2"
+      <limit lower="-${15.0*pi/180}" upper="${pi/2}" effort="2"
       velocity="2.0" />
       <dynamics damping="0.1" />

File: sr_description/hand/xacro/forearm/forearm_lite.urdf.xacro (robot description, xacro)
@@ -13,5 +13,5 @@
       </inertial>
       <visual>
-        <origin xyz="0 0 0" rpy="0 0 ${M_PI/2}" />
+        <origin xyz="0 0 0" rpy="0 0 ${pi/2}" />
         <geometry name="${prefix}forearm_visual">
           <xacro:if value="${muscle}">

File: sr_description/hand/xacro/full_hand.urdf.xacro (robot description, xacro)
@@ -8,5 +8,5 @@
   <xacro:include filename="$(find sr_description)/hand/xacro/finger/fingers.urdf.xacro" />
   <xacro:include filename="$(find sr_description)/hand/xacro/thumb/thumb.urdf.xacro" />
-  <xacro:property name="M_PI" value="3.1415926535897931" />
+  <xacro:property name="pi" value="3.1415926535897931" />
   <!-- muscletrans is true for muscle transmission to be used, false to use motor transmission -->
   <!-- muscle is true for muscle hand or false for motor hand -->

File: sr_description/hand/xacro/hand_E_no_mf_rf.urdf.xacro (robot description, xacro)
@@ -8,5 +8,5 @@
   <xacro:include filename="$(find sr_description)/hand/xacro/finger/fingers.urdf.xacro" />
   <xacro:include filename="$(find sr_description)/hand/xacro/thumb/thumb.urdf.xacro" />
-  <xacro:property name="M_PI" value="3.1415926535897931" />
+  <xacro:property name="pi" value="3.1415926535897931" />
   <!-- muscletrans is true for muscle transmission to be used, false to use motor transmission -->
   <!-- muscle is true for muscle hand or false for motor hand -->

File: sr_description/hand/xacro/hand_lite.urdf.xacro (robot description, xacro)
@@ -8,5 +8,5 @@
   <xacro:include filename="$(find sr_description)/hand/xacro/finger/fingers.urdf.xacro" />
   <xacro:include filename="$(find sr_description)/hand/xacro/thumb/thumb.urdf.xacro" />
-  <xacro:property name="M_PI" value="3.1415926535897931" />
+  <xacro:property name="pi" value="3.1415926535897931" />
   <!-- muscletrans is true for muscle transmission to be used, false to use motor transmission -->
   <!-- muscle is true for muscle hand or false for motor hand -->
@@ -26,5 +26,5 @@
       <parent link="${prefix}forearm" />
       <child link="${prefix}palm" />
-      <origin xyz="0 -0.015 0.149" rpy="-${40*M_PI/180} 0 0" />
+      <origin xyz="0 -0.015 0.149" rpy="-${40*pi/180} 0 0" />
       <axis xyz="0 ${reflect} 0" />
     </joint>

File: sr_description/hand/xacro/one_finger_unit.urdf.xacro (robot description, xacro)
@@ -5,5 +5,5 @@
   <xacro:include filename="$(find sr_description)/hand/xacro/forearm/forearm.urdf.xacro" />
   <xacro:include filename="$(find sr_description)/hand/xacro/finger/fingers.urdf.xacro" />
-  <xacro:property name="M_PI" value="3.1415926535897931" />
+  <xacro:property name="pi" value="3.1415926535897931" />
   <!-- muscletrans is true for muscle transmission to be used, false to use motor transmission -->
   <!-- muscle is true for muscle hand or false for motor hand -->
@@ -44,5 +44,5 @@
       <child link="${prefix}palm" />
       <origin xyz="${reflect*0.011} 0.010 0.22"
-      rpy="0 0 ${M_PI}" />
+      rpy="0 0 ${pi}" />
     </joint>
     <!-- mfknuckle is at [0.011 -0.01 0.346] from the bottom of forearm -->

File: sr_description/hand/xacro/palm/palm.urdf.xacro (robot description, xacro)
@@ -99,5 +99,5 @@
       <origin xyz="0 0 0.034" rpy="0 0 0" />
       <axis xyz="1 0 0" />
-      <limit lower="${-40/180*M_PI}" upper="${28/180*M_PI}"
+      <limit lower="${-40/180*pi}" upper="${28/180*pi}"
       effort="30" velocity="2.0" />
       <dynamics damping="0.1" />

File: sr_description/hand/xacro/th_ff_rf_ellipsoid_hand.urdf.xacro (robot description, xacro)
@@ -8,5 +8,5 @@
   <xacro:include filename="$(find sr_description)/hand/xacro/finger/fingers.urdf.xacro" />
   <xacro:include filename="$(find sr_description)/hand/xacro/thumb/thumb.urdf.xacro" />
-  <xacro:property name="M_PI" value="3.1415926535897931" />
+  <xacro:property name="pi" value="3.1415926535897931" />
   <!-- muscletrans is true for muscle transmission to be used, false to use motor transmission -->
   <!-- muscle is true for muscle hand or false for motor hand -->

File: sr_description/hand/xacro/three_biotac_fingers_hand.urdf.xacro (robot description, xacro)
@@ -8,5 +8,5 @@
   <xacro:include filename="$(find sr_description)/hand/xacro/finger/fingers.urdf.xacro" />
   <xacro:include filename="$(find sr_description)/hand/xacro/thumb/thumb.urdf.xacro" />
-  <xacro:property name="M_PI" value="3.1415926535897931" />
+  <xacro:property name="pi" value="3.1415926535897931" />
   <!-- muscletrans is true for muscle transmission to be used, false to use motor transmission -->
   <!-- muscle is true for muscle hand or false for motor hand -->

File: sr_description/hand/xacro/three_fingers_hand.urdf.xacro (robot description, xacro)
@@ -8,5 +8,5 @@
   <xacro:include filename="$(find sr_description)/hand/xacro/finger/fingers.urdf.xacro" />
   <xacro:include filename="$(find sr_description)/hand/xacro/thumb/thumb.urdf.xacro" />
-  <xacro:property name="M_PI" value="3.1415926535897931" />
+  <xacro:property name="pi" value="3.1415926535897931" />
   <!-- muscletrans is true for muscle transmission to be used, false to use motor transmission -->
   <!-- muscle is true for muscle hand or false for motor hand -->

File: sr_description/hand/xacro/three_fingers_hand_RF.urdf.xacro (robot description, xacro)
@@ -8,5 +8,5 @@
   <xacro:include filename="$(find sr_description)/hand/xacro/finger/fingers.urdf.xacro" />
   <xacro:include filename="$(find sr_description)/hand/xacro/thumb/thumb.urdf.xacro" />
-  <xacro:property name="M_PI" value="3.1415926535897931" />
+  <xacro:property name="pi" value="3.1415926535897931" />
   <!-- muscletrans is true for muscle transmission to be used, false to use motor transmission -->
   <!-- muscle is true for muscle hand or false for motor hand -->

File: sr_description/hand/xacro/thumb/thbase.urdf.xacro (robot description, xacro)
@@ -40,7 +40,7 @@
       <child link="${prefix}thbase" />
       <origin xyz="${reflect*0.034} -0.0085 0.029"
-      rpy="0 ${M_PI/4} ${M_PI/2-reflect*M_PI/2}" />
+      rpy="0 ${pi/4} ${pi/2-reflect*pi/2}" />
       <axis xyz="0 0 ${reflect*-1}" />
-      <limit lower="${-60/180*M_PI}" upper="${60/180*M_PI}"
+      <limit lower="${-60/180*pi}" upper="${60/180*pi}"
       effort="5.0" velocity="4.0" />
       <dynamics damping="0.2" />

File: sr_description/hand/xacro/thumb/thdistal.urdf.xacro (robot description, xacro)
@@ -30,7 +30,7 @@
         <parent link="${parent}" />
         <child link="${prefix}thdistal_J1_dummy" />
-        <origin xyz="0 0 0.02" rpy="0 0 ${-M_PI/2}" />
+        <origin xyz="0 0 0.02" rpy="0 0 ${-pi/2}" />
         <axis xyz="1 0 0" />
-        <limit lower="${20*M_PI/180}" upper="${20.1*M_PI/180}"
+        <limit lower="${20*pi/180}" upper="${20.1*pi/180}"
         effort="0.0" velocity="2.0" />
         <dynamics damping="0.5" />
@@ -42,5 +42,5 @@
       <link name="${prefix}thdistal">
         <inertial>
-          <origin xyz="-0.009 0.0 0.035" rpy="0 0 ${-M_PI/2}" />
+          <origin xyz="-0.009 0.0 0.035" rpy="0 0 ${-pi/2}" />
           <!-- approximated only FIXME -->
           <mass value="0.008" />
@@ -89,5 +89,5 @@
         <parent link="${prefix}thmiddle" />
         <child link="${prefix}thdistal" />
-        <origin xyz="0 0.0 0.01" rpy="0 0 ${-M_PI/2}" />
+        <origin xyz="0 0.0 0.01" rpy="0 0 ${-pi/2}" />
       </joint>
       <!-- extra link to imaginary sphere in fingertip for FK/IK calculations -->
@@ -190,7 +190,7 @@
         <parent link="${parent}" />
         <child link="${prefix}thdistal" />
-        <origin xyz="0 0 0.032" rpy="0 0 ${-M_PI/2}" />
+        <origin xyz="0 0 0.032" rpy="0 0 ${-pi/2}" />
         <axis xyz="1 0 0" />
-        <limit lower="-${15.0*M_PI/180}" upper="${90.0*M_PI/180}" effort="1.0"
+        <limit lower="-${15.0*pi/180}" upper="${90.0*pi/180}" effort="1.0"
         velocity="4.0" />
         <dynamics damping="0.2" />
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