Commit message: Improved xacro for modularity and to permit sensor selection
Use modern xacro to simplify URDF generation for more hands and more
types of sensors. Also permits to deactivate gazebo sensors
Maintained backward compatibility of old parameters
Use python pi

File: sr_description/hand/xacro/finger/middle/middle.gazebo.xacro (robot description, xacro)
@@ -1,7 +1,8 @@
 <?xml version="1.0"?>
 <robot xmlns:xacro="http://www.ros.org/wiki/xacro">
-  <xacro:macro name="middle_gazebo" params="prefix link_prefix">
-  <!-- prefix can be anything but usually is "r_" or  "l_" for right and left hands distinction -->
-  <gazebo reference="${prefix}${link_prefix}middle">
+  <xacro:macro name="middle_gazebo" params="prefix:=^ link_prefix:=^ mid_sensor:=^|std">
+    <!-- prefix can be anything but usually is "r_" or  "l_" for right and left hands distinction -->
+    <gazebo reference="${prefix}${link_prefix}middle">
+      <xacro:unless value="${'none' in mid_sensor}">
       <sensor type="contact" name="${prefix}${link_prefix}middle_contact">
         <always_on>1</always_on>
@@ -18,4 +19,5 @@
         </plugin>
       </sensor>
+      </xacro:unless>
       <selfCollide>true</selfCollide>
     </gazebo>

File: sr_description/other/xacro/kinect/shadowarm_kinect.urdf.xacro (robot description, xacro)
@@ -1,11 +1,10 @@
 <robot xmlns:xacro="http://www.ros.org/wiki/xacro">
-  <xacro:property name="M_PI" value="3.1415926535" />
   <xacro:include filename="$(find sr_description)/other/xacro/kinect/gazebo_kinect.urdf.xacro" />
   <xacro:macro name="shadowarm_side_kinect" params="parent">
     <joint name="base_camera_joint" type="fixed">
       <!--        <origin xyz="0.00724 0.153 0.4405"
-          rpy="-${M_PI/2} 0.5236 -0.2618" /> -->
+          rpy="-${pi/2} 0.5236 -0.2618" /> -->
       <origin xyz="0.01216 0.1713 0.433"
-      rpy="-${M_PI/2} ${M_PI/4} -${M_PI/12}" />
+      rpy="-${pi/2} ${pi/4} -${pi/12}" />
       <parent link="${parent}" />
       <child link="camera_link" />
@@ -45,5 +44,5 @@
     </link>
     <joint name="camera_depth_optical_joint" type="fixed">
-      <origin xyz="0 0 0" rpy="${-M_PI/2} 0 ${-M_PI/2}" />
+      <origin xyz="0 0 0" rpy="${-pi/2} 0 ${-pi/2}" />
       <parent link="camera_depth_frame" />
       <child link="camera_depth_optical_frame" />
@@ -71,5 +70,5 @@
     </link>
     <joint name="camera_rgb_optical_joint" type="fixed">
-      <origin xyz="0 0 0" rpy="${-M_PI/2} 0 ${-M_PI/2}" />
+      <origin xyz="0 0 0" rpy="${-pi/2} 0 ${-pi/2}" />
       <parent link="camera_rgb_frame" />
       <child link="camera_rgb_optical_frame" />
