Commit message: Fixed deprecated .mesh

File: sr_description/arm/xacro/hand_support/shadowarm_handsupport_muscle.urdf.xacro (robot description, xacro)
@@ -10,7 +10,7 @@
       </inertial>
       <visual>
-        <origin xyz="0 0 -0.04" rpy="${M_PI/2} 0 0" />
+        <origin xyz="0 0 -0.04" rpy="0 0 0" />
         <geometry name="shadowarm_handsupport_visual">
-          <mesh filename="package://sr_description/arm/model/elbow_rotate_muscle.mesh"
+          <mesh filename="package://sr_description/arm/model/elbow_rotate_muscle.dae"
           scale="0.001 0.001 0.001" />
         </geometry>
