Commit message: pi fixes

File: sr_description/arm/xacro/hand_support/shadowarm_handsupport_motor.urdf.xacro (robot description, xacro)
@@ -33,5 +33,5 @@
       <origin xyz="0.08 0 0.125" rpy="0.0 0 0" />
       <axis xyz="0 0 -1" />
-      <limit lower="-${pi/2}" upper="${pi/2}" effort="30"
+      <limit lower="-${M_PI/2}" upper="${M_PI/2}" effort="30"
       velocity="1.0" />
       <dynamics damping="5.5" />

File: sr_description/arm/xacro/hand_support/shadowarm_handsupport_muscle.urdf.xacro (robot description, xacro)
@@ -10,5 +10,5 @@
       </inertial>
       <visual>
-        <origin xyz="0 0 -0.04" rpy="${pi/2} 0 0" />
+        <origin xyz="0 0 -0.04" rpy="${M_PI/2} 0 0" />
         <geometry name="shadowarm_handsupport_visual">
           <mesh filename="package://sr_description/arm/model/elbow_rotate_muscle.mesh"
@@ -33,5 +33,5 @@
       <origin xyz="0.08 0 0.131" rpy="0 0 0" />
       <axis xyz="0 0 -1" />
-      <limit lower="-${pi/2}" upper="${pi/2}" effort="30"
+      <limit lower="-${M_PI/2}" upper="${M_PI/2}" effort="30"
       velocity="1.0" />
       <dynamics damping="5.5" />

File: sr_description/arm/xacro/trunk/shadowarm_trunk.urdf.xacro (robot description, xacro)
@@ -32,5 +32,5 @@
       <origin xyz="0 0 0.01" rpy="0.0 0.0 0.0" />
       <axis xyz="0 0 1" />
-      <limit lower="-${pi/4}" upper="${pi/2}" effort="70"
+      <limit lower="-${M_PI/4}" upper="${M_PI/2}" effort="70"
       velocity="1.0" />
       <dynamics damping="5.5" />

File: sr_description/arm/xacro/upper_arm/shadowarm_upperarm.urdf.xacro (robot description, xacro)
@@ -18,5 +18,5 @@
       </visual>
       <collision>
-        <origin xyz="0 0 0.16" rpy="0 -${pi} 0" />
+        <origin xyz="0 0 0.16" rpy="0 -${M_PI} 0" />
         <geometry name="shadowarm_upperarm_collision">
           <box size="0.170 0.133 0.470" />
@@ -30,8 +30,8 @@
       <parent link="${parent}" />
       <child link="shadowarm_upperarm" />
-      <origin xyz="0 -0.134 0.5305" rpy="0 -${pi} 0.0" />
+      <origin xyz="0 -0.134 0.5305" rpy="0 -${M_PI} 0.0" />
       <!-- yaw=-0.026 -->
       <axis xyz="0 -1 0" />
-      <limit lower="0" upper="${pi/2}" effort="100"
+      <limit lower="0" upper="${M_PI/2}" effort="100"
       velocity="1.0" />
       <dynamics damping="5.3" />

File: sr_description/hand/xacro/finger/biotac/biotac.urdf.xacro (robot description, xacro)
@@ -61,5 +61,5 @@
       <origin xyz="0 0 0.045" rpy="0 0 0" />
       <axis xyz="1 0 0" />
-      <limit lower="0" upper="${pi/2}" effort="2.0"
+      <limit lower="0" upper="${M_PI/2}" effort="2.0"
       velocity="2.0" />
       <dynamics damping="0.1" />

File: sr_description/hand/xacro/finger/distal/distal.urdf.xacro (robot description, xacro)
@@ -111,5 +111,5 @@
         <xacro:unless value="${bio}">
           <!-- standard distal joint -->
-          <limit lower="0" upper="${pi/2}" effort="2"
+          <limit lower="0" upper="${M_PI/2}" effort="2"
           velocity="2.0" />
         </xacro:unless>

File: sr_description/hand/xacro/finger/middle/middle.urdf.xacro (robot description, xacro)
@@ -54,5 +54,5 @@
       <origin xyz="0 0 0.045" rpy="0 0 0" />
       <axis xyz="1 0 0" />
-      <limit lower="0" upper="${pi/2}" effort="2"
+      <limit lower="0" upper="${M_PI/2}" effort="2"
       velocity="2.0" />
       <dynamics damping="0.1" />

File: sr_description/hand/xacro/finger/proximal/proximal.urdf.xacro (robot description, xacro)
@@ -42,5 +42,5 @@
       <origin xyz="0 0 0" rpy="0 0 0" />
       <axis xyz="1 0 0" />
-      <limit lower="-${15.0*pi/180}" upper="${pi/2}" effort="2"
+      <limit lower="-${15.0*pi/180}" upper="${M_PI/2}" effort="2"
       velocity="2.0" />
       <dynamics damping="0.1" />

File: sr_description/hand/xacro/forearm/forearm_lite.urdf.xacro (robot description, xacro)
@@ -13,5 +13,5 @@
       </inertial>
       <visual>
-        <origin xyz="0 0 0" rpy="0 0 ${pi/2}" />
+        <origin xyz="0 0 0" rpy="0 0 ${M_PI/2}" />
         <geometry name="${prefix}forearm_visual">
           <xacro:if value="${muscle}">

File: sr_description/hand/xacro/one_finger_unit.urdf.xacro (robot description, xacro)
@@ -44,5 +44,5 @@
       <child link="${prefix}palm" />
       <origin xyz="${reflect*0.011} 0.010 0.22"
-      rpy="0 0 ${pi}" />
+      rpy="0 0 ${M_PI}" />
     </joint>
     <!-- mfknuckle is at [0.011 -0.01 0.346] from the bottom of forearm -->

File: sr_description/hand/xacro/thumb/thbase.urdf.xacro (robot description, xacro)
@@ -40,5 +40,5 @@
       <child link="${prefix}thbase" />
       <origin xyz="${reflect*0.034} -0.0085 0.029"
-      rpy="0 ${pi/4} ${pi/2-reflect*pi/2}" />
+      rpy="0 ${M_PI/4} ${M_PI/2-reflect*pi/2}" />
       <axis xyz="0 0 ${reflect*-1}" />
       <limit lower="${-60/180*pi}" upper="${60/180*pi}"

File: sr_description/other/xacro/kinect/shadowarm_kinect.urdf.xacro (robot description, xacro)
@@ -5,7 +5,7 @@
     <joint name="base_camera_joint" type="fixed">
       <!--        <origin xyz="0.00724 0.153 0.4405"
-          rpy="-${pi/2} 0.5236 -0.2618" /> -->
+          rpy="-${M_PI/2} 0.5236 -0.2618" /> -->
       <origin xyz="0.01216 0.1713 0.433"
-      rpy="-${pi/2} ${pi/4} -${pi/12}" />
+      rpy="-${M_PI/2} ${M_PI/4} -${M_PI/12}" />
       <parent link="${parent}" />
       <child link="camera_link" />

File: sr_description/robots/arm_and_hand_muscle.urdf.xacro (robot description, xacro)
@@ -14,5 +14,5 @@
     <parent link="shadowarm_handsupport" />
     <child link="rh_forearm" />
-    <origin xyz="0 0 0" rpy="0 0 ${pi}" />
+    <origin xyz="0 0 0" rpy="0 0 ${M_PI}" />
   </joint>
   <xacro:shadowhand muscletrans="false" muscle="true" bio="false" bt_sp="false"

File: sr_description/robots/arm_and_hand_muscle_biotac.urdf.xacro (robot description, xacro)
@@ -14,5 +14,5 @@
     <parent link="shadowarm_handsupport" />
     <child link="rh_forearm" />
-    <origin xyz="0 0 0" rpy="0 0 ${pi}" />
+    <origin xyz="0 0 0" rpy="0 0 ${M_PI}" />
   </joint>
   <xacro:shadowhand muscletrans="false" muscle="true" bio="true" bt_sp="false"

File: sr_description/robots/arm_and_sr_one_finger_motor.urdf.xacro (robot description, xacro)
@@ -14,5 +14,5 @@
     <parent link="shadowarm_handsupport" />
     <child link="rh_forearm" />
-    <origin xyz="0 0 0" rpy="0 0 ${pi}" />
+    <origin xyz="0 0 0" rpy="0 0 ${M_PI}" />
     <axis xyz="0 -1 0" />
     <limit lower="0" upper="0" effort="10" velocity="1.0" />

File: sr_description/robots/desk_arm_and_hand_motor.urdf.xacro (robot description, xacro)
@@ -14,5 +14,5 @@
     <parent link="shadowarm_handsupport" />
     <child link="rh_forearm" />
-    <origin xyz="0 0 0" rpy="0 0 ${pi}" />
+    <origin xyz="0 0 0" rpy="0 0 ${M_PI}" />
     <axis xyz="0 -1 0" />
     <limit lower="0" upper="0" effort="10" velocity="1.0" />
