Commit message: adding hand extra lite model

File: sr_description/hand/xacro/hand_lite.urdf.xacro (robot description, xacro)
@@ -18,5 +18,5 @@
   <!-- prefix can be anything but usually is "r_" or  "l_" for right and left hands distinction -->
   <xacro:macro name="shadowhand"
-  params="muscletrans muscle bio bt_sp ubi eli reflect prefix">
+  params="muscletrans muscle bio bt_sp ubi eli reflect prefix extra_lite">
     <!-- Forearm -->
     <xacro:forearm muscle="${muscle}" prefix="${prefix}" />
@@ -41,11 +41,13 @@
     </xacro:finger>
     <!-- Middle Finger -->
-    <xacro:finger muscletrans="${muscletrans}" lf="false"
-    bio="${bio}" bt_sp="${bt_sp}" ubi="${ubi}" eli="${eli}" prefix="${prefix}"
-    reflect="${reflect}" link_prefix="mf" joint_prefix="MF"
-    parent="${prefix}palm">
-      <origin xyz="${reflect*0.011} 0 0.099" rpy="0 0 0" />
-      <axis xyz="0 ${-1*reflect} 0" />
-    </xacro:finger>
+    <xacro:unless value="${extra_lite}">
+      <xacro:finger muscletrans="${muscletrans}" lf="false"
+		    bio="${bio}" bt_sp="${bt_sp}" ubi="${ubi}" eli="${eli}" prefix="${prefix}"
+		    reflect="${reflect}" link_prefix="mf" joint_prefix="MF"
+		    parent="${prefix}palm">
+	<origin xyz="${reflect*0.011} 0 0.099" rpy="0 0 0" />
+	<axis xyz="0 ${-1*reflect} 0" />
+      </xacro:finger>
+    </xacro:unless>
     <!-- Ring Finger -->
     <xacro:finger muscletrans="${muscletrans}" lf="false"

File: sr_description/robots/shadowhand_extra_lite.urdf.xacro (robot description, xacro)
@@ -8,4 +8,4 @@
   <xacro:include filename="$(find sr_description)/other/xacro/gazebo/gazebo.urdf.xacro" />
   <xacro:shadowhand muscletrans="false" muscle="false" bio="false" bt_sp="false"
-  ubi="false" eli="false" reflect="1.0" prefix="rh_" extra_lite="false"/>
+  ubi="false" eli="false" reflect="1.0" prefix="rh_" extra_lite="true"/>
 </robot>

Commit message: another fix

File: sr_description/hand/xacro/hand_lite.urdf.xacro (robot description, xacro)
@@ -8,5 +8,4 @@
   <xacro:include filename="$(find sr_description)/hand/xacro/finger/fingers.urdf.xacro" />
   <xacro:include filename="$(find sr_description)/hand/xacro/thumb/thumb.urdf.xacro" />
-  <xacro:property name="pi" value="3.1415926535897931" />
   <!-- muscletrans is true for muscle transmission to be used, false to use motor transmission -->
   <!-- muscle is true for muscle hand or false for motor hand -->
