Commit message: Fix backward compatibility
- Restore deleted files required by compatibility test
- Fix use of deprecated properties
- Fix use of deprecated parameters
- Undo unrelated changes w.r.t. upstream
- Fix extra_lite hands: it is missing MF not FF

File: sr_description/hand/xacro/backward_compat.urdf.xacro (robot description, xacro)
@@ -1,36 +1,29 @@
 <robot xmlns:xacro="http://www.ros.org/wiki/xacro">
   <!-- for backward compatibility define new params from old ones -->
-  <xacro:property name="old_tip_sensor" value="${(1 if bio==True else 0) + (1 if bt_sp==True else 0) + (1 if eli==True else 0)}"/>
-  <!-- if old parameters are used, valid only if sum is 1 -->
-  <xacro:if value="${old_tip_sensor==1}">
-    <xacro:if value="${bio}">
-      <xacro:property name="palm_sensor" value="std"/>
-      <xacro:property name="prox_sensor" value="${[std, std, std, std ,std]}"/>
-      <xacro:property name="mid_sensor" value="${[bio, bio, bio, bio ,bio]}"/>
-      <xacro:property name="tip_sensor" value="${[bio, bio, bio, bio ,bio]}"/>
-    </xacro:if>
-    <xacro:if value="${bt_sp}">
-      <xacro:property name="palm_sensor" value="std"/>
-      <xacro:property name="prox_sensor" value="${[std, std, std, std ,std]}"/>
-      <xacro:property name="mid_sensor" value="${[std, std, std, std ,std]}"/>
-      <xacro:property name="tip_sensor" value="${[bt_sp, bt_sp, bt_sp, bt_sp ,bt_sp]}"/>
-    </xacro:if>
-    <xacro:if value="${eli}">
-      <xacro:property name="palm_sensor" value="std"/>
-      <xacro:property name="prox_sensor" value="${[std, std, std, std ,std]}"/>
-      <xacro:property name="mid_sensor" value="${[std, std, std, std ,std]}"/>
-      <xacro:property name="tip_sensor" value="${[eli, eli, eli, eli ,eli]}"/>
-    </xacro:if>
+  <xacro:if value="${bio}">
+    <xacro:property name="palm_sensor" value="std" />
+    <xacro:property name="prox_sensors" value="${['std', 'std', 'std', 'std', 'std']}" />
+    <xacro:property name="mid_sensors" value="${['bio', 'bio', 'bio', 'bio', 'bio']}" />
+    <xacro:property name="tip_sensors" value="${['bio', 'bio', 'bio', 'bio', 'bio']}" />
+  </xacro:if>
+  <xacro:if value="${bt_sp}">
+    <xacro:property name="palm_sensor" value="std" />
+    <xacro:property name="prox_sensors" value="${['std', 'std', 'std', 'std', 'std']}" />
+    <xacro:property name="mid_sensors" value="${['std', 'std', 'std', 'std', 'std']}" />
+    <xacro:property name="tip_sensors" value="${['bt_sp', 'bt_sp', 'bt_sp', 'bt_sp', 'bt_sp']}" />
+  </xacro:if>
+  <xacro:if value="${eli}">
+    <xacro:property name="palm_sensor" value="std" />
+    <xacro:property name="prox_sensors" value="${['std', 'std', 'std', 'std', 'std']}" />
+    <xacro:property name="mid_sensors" value="${['std', 'std', 'std', 'std', 'std']}" />
+    <xacro:property name="tip_sensors" value="${['eli', 'eli', 'eli', 'eli', 'eli']}" />
   </xacro:if>
   <xacro:if value="${muscle}">
     <xacro:if value="${muscletrans}">
-      <xacro:property name="hand_type" value="hand_mt"/>
+      <xacro:property name="hand_type" value="hand_mt" />
     </xacro:if>
     <xacro:unless value="${muscletrans}">
-      <xacro:property name="hand_type" value="hand_m"/>
+      <xacro:property name="hand_type" value="hand_m" />
     </xacro:unless>
   </xacro:if>
-  <xacro:unless value="${lf}">
-    <xacro:property name="fingers" value="${[1,1,1,1,0]}"/>
-  </xacro:unless>
 </robot>

File: sr_description/hand/xacro/ff_biotac_hand.urdf.xacro (robot description, xacro)
@@ -1,11 +1,3 @@
-<robot xmlns:sensor="http://playerstage.sourceforge.net/gazebo/xmlschema/#sensor"
-xmlns:controller="http://playerstage.sourceforge.net/gazebo/xmlschema/#controller"
-xmlns:interface="http://playerstage.sourceforge.net/gazebo/xmlschema/#interface"
-xmlns:xacro="http://www.ros.org/wiki/xacro">
-  <xacro:include filename="$(find sr_description)/hand/xacro/forearm/forearm.urdf.xacro" />
-  <xacro:include filename="$(find sr_description)/hand/xacro/wrist/wrist.urdf.xacro" />
-  <xacro:include filename="$(find sr_description)/hand/xacro/palm/palm.urdf.xacro" />
-  <xacro:include filename="$(find sr_description)/hand/xacro/finger/fingers.urdf.xacro" />
-  <xacro:include filename="$(find sr_description)/hand/xacro/thumb/thumb.urdf.xacro" />
+<robot xmlns:xacro="http://www.ros.org/wiki/xacro">
   <!-- muscletrans is true for muscle transmission to be used, false to use motor transmission -->
   <!-- muscle is true for muscle hand or false for motor hand -->
@@ -16,54 +8,13 @@
   <!-- prefix can be anything but usually is "r_" or  "l_" for right and left hands distinction -->
   <xacro:macro name="shadowhand" params="muscletrans muscle bio bt_sp eli reflect prefix">
-    <!-- Forearm -->
-    <xacro:forearm muscle="${muscle}" prefix="${prefix}" />
-    <!-- Wrist -->
-    <xacro:if value="${muscle}">
-      <xacro:wrist muscletrans="${muscletrans}" prefix="${prefix}"
-      reflect="${reflect}" parent="${prefix}forearm">
-        <origin xyz="0 0 0.4096" rpy="0 0 0" />
-      </xacro:wrist>
-    </xacro:if>
-    <xacro:unless value="${muscle}">
-      <xacro:wrist muscletrans="false" prefix="${prefix}"
-      reflect="${reflect}" parent="${prefix}forearm">
-        <origin xyz="0 -0.010 0.213" rpy="0 0 0" />
-      </xacro:wrist>
-    </xacro:unless>
-    <!-- Palm -->
-    <xacro:palm muscletrans="${muscletrans}" prefix="${prefix}"
-    reflect="${reflect}" parent="${prefix}wrist" />
-    <!-- First Finger Biotac -->
-    <xacro:finger muscletrans="${muscletrans}" lf="false" bio="true" bt_sp="false" eli="false" prefix="${prefix}"
-    reflect="${reflect}" link_prefix="ff" joint_prefix="FF"
-    parent="${prefix}palm">
-      <origin xyz="${reflect*0.033} 0 0.095" rpy="0 0 0" />
-      <axis xyz="0 ${-1*reflect} 0" />
-    </xacro:finger>
-    <!-- Middle Finger -->
-    <xacro:finger muscletrans="${muscletrans}" lf="false" bio="${bio}" bt_sp="false" eli="${eli}" prefix="${prefix}"
-    reflect="${reflect}" link_prefix="mf" joint_prefix="MF"
-    parent="${prefix}palm">
-      <origin xyz="${reflect*0.011} 0 0.099" rpy="0 0 0" />
-      <axis xyz="0 ${-1*reflect} 0" />
-    </xacro:finger>
-    <!-- Ring Finger -->
-    <xacro:finger muscletrans="${muscletrans}" lf="false" bio="${bio}" bt_sp="${bt_sp}" eli="${eli}" prefix="${prefix}"
-    reflect="${reflect}" link_prefix="rf" joint_prefix="RF"
-    parent="${prefix}palm">
-      <origin xyz="${reflect*-0.011} 0 0.095" rpy="0 0 0" />
-      <axis xyz="0 ${reflect} 0" />
-    </xacro:finger>
-    <!-- Little Finger  -->
-    <xacro:finger muscletrans="${muscletrans}" lf="true" bio="${bio}" bt_sp="${bt_sp}" eli="${eli}" prefix="${prefix}"
-    reflect="${reflect}" link_prefix="lf" joint_prefix="LF"
-    parent="${prefix}palm">
-      <origin xyz="0 0 0.06579" rpy="0 0 0" />
-      <axis xyz="0 ${reflect} 0" />
-    </xacro:finger>
-    <!-- Thumb Biotac -->
-    <xacro:thumb muscletrans="${muscletrans}" bio="${bio}" bt_sp="${bt_sp}" eli="${eli}" prefix="${prefix}"
-    reflect="${reflect}" is_lite="0" parent="${prefix}palm">
-    </xacro:thumb>
+    <!-- Ensure tip_sensors is defined before usage below -->
+    <xacro:property name="tip_sensors" default="${5 * ['std']}" />
+    <!-- translate old parameters to new ones, eventually updating tip_sensors -->
+    <xacro:include filename="$(find sr_description)/hand/xacro/backward_compat.urdf.xacro" />
+    <!-- forward to generic macro -->
+    <xacro:include filename="$(find sr_description)/hand/xacro/full_hand.urdf.xacro" />
+    <!-- Enforce BioTac on First Finger -->
+    <xacro:shadowhand fingers="${5 * [1]}" reflect="${reflect}" prefix="${prefix}"
+    tip_sensors="${[tip_sensors[0]] + ['bio'] + tip_sensors[2:]}"/>
   </xacro:macro>
 </robot>

File: sr_description/hand/xacro/finger/distal/distal.urdf.xacro (robot description, xacro)
@@ -42,5 +42,5 @@
           </xacro:if>
         </geometry>
-        <material name="Grey" />
+        <!-- <material name="Grey" /> -->
       </visual>
       <collision>
@@ -72,14 +72,7 @@
         <origin xyz="0 0 0.025" rpy="0 0 0" />
         <axis xyz="1 0 0" />
-        <xacro:if value="${bio}">
-          <!-- biotac fixed distal joint -->
-          <limit lower="${20/180*pi}" upper="${20/180*pi}"
-          effort="10" velocity="2.0" />
-        </xacro:if>
-        <xacro:unless value="${bio}">
-          <!-- standard distal joint -->
-          <limit lower="0" upper="${pi/2}" effort="2"
-          velocity="2.0" />
-        </xacro:unless>
+        <!-- standard distal joint -->
+        <limit lower="0" upper="${pi/2}" effort="2"
+        velocity="2.0" />
         <dynamics damping="0.1" />
       </joint>

File: sr_description/hand/xacro/full_hand.urdf.xacro (robot description, xacro)
@@ -1,6 +1,3 @@
-<robot xmlns:sensor="http://playerstage.sourceforge.net/gazebo/xmlschema/#sensor"
-xmlns:controller="http://playerstage.sourceforge.net/gazebo/xmlschema/#controller"
-xmlns:interface="http://playerstage.sourceforge.net/gazebo/xmlschema/#interface"
-xmlns:xacro="http://www.ros.org/wiki/xacro">
+<robot xmlns:sensor="http://playerstage.sourceforge.net/gazebo/xmlschema/#sensor" xmlns:controller="http://playerstage.sourceforge.net/gazebo/xmlschema/#controller" xmlns:interface="http://playerstage.sourceforge.net/gazebo/xmlschema/#interface" xmlns:xacro="http://www.ros.org/wiki/xacro">
   <xacro:include filename="$(find sr_description)/hand/xacro/forearm/forearm.urdf.xacro" />
   <xacro:include filename="$(find sr_description)/hand/xacro/wrist/wrist.urdf.xacro" />
@@ -8,6 +5,12 @@
   <xacro:include filename="$(find sr_description)/hand/xacro/finger/fingers.urdf.xacro" />
   <xacro:include filename="$(find sr_description)/hand/xacro/thumb/thumb.urdf.xacro" />
-  <!-- hand_type describes the hand type, hand_e, hand_e_plus, hand_m (muscle) -->
-  <!-- fingers describes which fingers are present, [th, ff, mf, rf, lf], default [1, 1, 1, 1, 1] -->
+  <!-- hand_type can be: hand_e, hand_e_plus, hand_m (muscle), hand_mt (muscletrans) -->
+  <!-- fingers: dict specifying available fingers, default: dict(th=1, ff=1, mf=1, rf=1, lf=1) -->
+  <!-- tip_sensors: dict specifying the fingertip (tactile) sensors per finger: std, none, bio, bt_sp, eli -->
+  <!-- mid_sensors: dict specifying the middle-phalange (tactile) sensors per finger: std, none, bio -->
+  <!-- prox_sensors: dict specifying the proximal (tactile) sensors per finger: std, none -->
+  <!-- palm_sensor: specifies the palm tactile sensor: std, none -->
+  <!-- reflect is either 1 (for right hand) or -1 (for left hand) -->
+  <!-- prefix can be anything but usually is "r_" or  "l_" for right and left hands distinction -->
   <!-- muscletrans (deprecated) is true for muscle transmission to be used, false to use motor transmission -->
   <!-- muscle (deprecated) is true for muscle hand or false for motor hand -->
@@ -15,15 +18,8 @@
   <!-- bt_sp (deprecated) is true for BT_SP finger or false for standard finger -->
   <!-- eli (deprecated) is true for ellipsoid fingertip or false for standard finger -->
-  <!-- tip_sensors vector that describes the sensor std, none, bio, bt_sp, eli -->
-  <!-- mid_sensors vector that describes the sensor std, none, bio -->
-  <!-- prox_sensors vector that describes the sensor std, none -->
-  <!-- palm_sensor describes the sensor std, none -->
-  <!-- reflect is either 1 (for right hand) or -1 (for left hand) -->
-  <!-- prefix can be anything but usually is "r_" or  "l_" for right and left hands distinction -->
   <!-- lf (deprecated) is true if we want a little finger, false otherwise -->
-  <xacro:macro name="shadowhand" params="hand_type:='hand_e' reflect prefix cable_mesh:=False
-          fingers:=${[1,1,1,1,1]} tip_sensors:=${['std','std','std','std','std']} prox_sensors:=${['std','std','std','std','std']}
-          mid_sensors:=${['std','std','std','std','std']} palm_sensor:=std
-          muscletrans:=False muscle:=False lf:=True bio:=False bt_sp:=False eli:=False">
+  <xacro:macro name="shadowhand" params="hand_type:='hand_e' reflect prefix cable_mesh:=False fingers:=${[1,1,1,1,1]}
+          tip_sensors:=${5 * ['std']} mid_sensors:=${5 * ['std']} prox_sensors:=${5 * ['std']} palm_sensor:=std
+          muscletrans:=^|False muscle:=^|False lf:=^|True bio:=^|False bt_sp:=^|False eli:=^|False">
     <!-- handle deprecated parameters -->
     <xacro:include filename="$(find sr_description)/hand/xacro/backward_compat.urdf.xacro" />
@@ -45,7 +41,5 @@
     <!-- First Finger -->
     <xacro:if value="${fingers[1] == 1}">
-      <xacro:finger link_prefix="ff" joint_prefix="FF" tip_sensor="${tip_sensors[1]}"
-                    prox_sensor="${prox_sensors[1]}" mid_sensor="${mid_sensors[1]}"
-                    parent="${prefix}palm">
+      <xacro:finger link_prefix="ff" joint_prefix="FF" tip_sensor="${tip_sensors[1]}" prox_sensor="${prox_sensors[1]}" mid_sensor="${mid_sensors[1]}" parent="${prefix}palm">
         <origin xyz="${reflect*0.033} 0 0.095" rpy="0 0 0" />
         <axis xyz="0 ${-1*reflect} 0" />
@@ -54,7 +48,5 @@
     <!-- Middle Finger -->
     <xacro:if value="${fingers[2] == 1}">
-      <xacro:finger link_prefix="mf" joint_prefix="MF" tip_sensor="${tip_sensors[2]}"
-                    prox_sensor="${prox_sensors[2]}" mid_sensor="${mid_sensors[2]}"
-                    parent="${prefix}palm">
+      <xacro:finger link_prefix="mf" joint_prefix="MF" tip_sensor="${tip_sensors[2]}" prox_sensor="${prox_sensors[2]}" mid_sensor="${mid_sensors[2]}" parent="${prefix}palm">
         <origin xyz="${reflect*0.011} 0 0.099" rpy="0 0 0" />
         <axis xyz="0 ${-1*reflect} 0" />
@@ -63,7 +55,5 @@
     <!-- Ring Finger -->
     <xacro:if value="${fingers[3] == 1}">
-      <xacro:finger link_prefix="rf" joint_prefix="RF" tip_sensor="${tip_sensors[3]}"
-                    prox_sensor="${prox_sensors[3]}" mid_sensor="${mid_sensors[3]}"
-                    parent="${prefix}palm">
+      <xacro:finger link_prefix="rf" joint_prefix="RF" tip_sensor="${tip_sensors[3]}" prox_sensor="${prox_sensors[3]}" mid_sensor="${mid_sensors[3]}" parent="${prefix}palm">
         <origin xyz="${reflect*-0.011} 0 0.095" rpy="0 0 0" />
         <axis xyz="0 ${reflect} 0" />
@@ -71,8 +61,6 @@
     </xacro:if>
     <!-- Little Finger  -->
-    <xacro:if value="${fingers[4] == 1}">
-      <xacro:finger link_prefix="lf" joint_prefix="LF" tip_sensor="${tip_sensors[4]}"
-                    prox_sensor="${prox_sensors[4]}" mid_sensor="${mid_sensors[4]}"
-                    parent="${prefix}palm">
+    <xacro:if value="${fingers[4] == 1 and lf}">
+      <xacro:finger link_prefix="lf" joint_prefix="LF" tip_sensor="${tip_sensors[4]}" prox_sensor="${prox_sensors[4]}" mid_sensor="${mid_sensors[4]}" parent="${prefix}palm">
         <origin xyz="0 0 0.06579" rpy="0 0 0" />
         <axis xyz="0 ${reflect} 0" />
@@ -81,6 +69,5 @@
     <!-- Thumb  -->
     <xacro:if value="${fingers[0] == 1}">
-      <xacro:thumb is_lite="0" parent="${prefix}palm" tip_sensor="${tip_sensors[0]}"
-                   prox_sensor="${prox_sensors[0]}" mid_sensor="${mid_sensors[0]}" />
+      <xacro:thumb is_lite="0" parent="${prefix}palm" tip_sensor="${tip_sensors[0]}" prox_sensor="${prox_sensors[0]}" mid_sensor="${mid_sensors[0]}" />
     </xacro:if>
   </xacro:macro>

File: sr_description/hand/xacro/hand_E_no_mf_rf.urdf.xacro (robot description, xacro)
@@ -1,11 +1,3 @@
-<robot xmlns:sensor="http://playerstage.sourceforge.net/gazebo/xmlschema/#sensor"
-xmlns:controller="http://playerstage.sourceforge.net/gazebo/xmlschema/#controller"
-xmlns:interface="http://playerstage.sourceforge.net/gazebo/xmlschema/#interface"
-xmlns:xacro="http://www.ros.org/wiki/xacro">
-  <xacro:include filename="$(find sr_description)/hand/xacro/forearm/forearm.urdf.xacro" />
-  <xacro:include filename="$(find sr_description)/hand/xacro/wrist/wrist.urdf.xacro" />
-  <xacro:include filename="$(find sr_description)/hand/xacro/palm/palm.urdf.xacro" />
-  <xacro:include filename="$(find sr_description)/hand/xacro/finger/fingers.urdf.xacro" />
-  <xacro:include filename="$(find sr_description)/hand/xacro/thumb/thumb.urdf.xacro" />
+<robot xmlns:xacro="http://www.ros.org/wiki/xacro">
   <!-- muscletrans is true for muscle transmission to be used, false to use motor transmission -->
   <!-- muscle is true for muscle hand or false for motor hand -->
@@ -17,42 +9,7 @@
   <!-- lf is true if we want a little finger, false otherwise -->
   <xacro:macro name="shadowhand" params="muscletrans muscle bio bt_sp eli reflect prefix lf">
-    <!-- Forearm -->
-    <xacro:forearm muscle="${muscle}" prefix="${prefix}" />
-    <!-- Wrist -->
-    <xacro:if value="${muscle}">
-      <xacro:wrist muscletrans="${muscletrans}" prefix="${prefix}"
-      reflect="${reflect}" parent="${prefix}forearm">
-        <origin xyz="0 0 0.4096" rpy="0 0 0" />
-      </xacro:wrist>
-    </xacro:if>
-    <xacro:unless value="${muscle}">
-      <xacro:wrist muscletrans="false" prefix="${prefix}"
-      reflect="${reflect}" parent="${prefix}forearm">
-        <origin xyz="0 -0.010 0.213" rpy="0 0 0" />
-      </xacro:wrist>
-    </xacro:unless>
-    <!-- Palm -->
-    <xacro:palm muscletrans="${muscletrans}" prefix="${prefix}"
-    reflect="${reflect}" parent="${prefix}wrist" />
-    <!-- First Finger -->
-    <xacro:finger muscletrans="${muscletrans}" lf="false" bio="${bio}" bt_sp="${bt_sp}" eli="${eli}" prefix="${prefix}"
-    reflect="${reflect}" link_prefix="ff" joint_prefix="FF"
-    parent="${prefix}palm">
-      <origin xyz="${reflect*0.033} 0 0.095" rpy="0 0 0" />
-      <axis xyz="0 ${-1*reflect} 0" />
-    </xacro:finger>
-    <!-- Little Finger  -->
-    <xacro:if value="${lf}">
-      <xacro:finger muscletrans="${muscletrans}" lf="true" bio="${bio}" bt_sp="${bt_sp}" eli="${eli}" prefix="${prefix}"
-      reflect="${reflect}" link_prefix="lf" joint_prefix="LF"
-      parent="${prefix}palm">
-        <origin xyz="0 0 0.06579" rpy="0 0 0" />
-        <axis xyz="0 ${reflect} 0" />
-      </xacro:finger>
-    </xacro:if>
-    <!-- Thumb  -->
-    <xacro:thumb muscletrans="${muscletrans}" bio="${bio}" bt_sp="${bt_sp}" eli="${eli}" prefix="${prefix}"
-    reflect="${reflect}" is_lite="0" parent="${prefix}palm">
-    </xacro:thumb>
+    <!-- forward to generic macro -->
+    <xacro:include filename="$(find sr_description)/hand/xacro/full_hand.urdf.xacro" />
+    <xacro:shadowhand fingers="${[1, 1, 0, 0, 1 if lf else 0]}" reflect="${reflect}" prefix="${prefix}" />
   </xacro:macro>
 </robot>

File: sr_description/hand/xacro/hand_lite.urdf.xacro (robot description, xacro)
@@ -8,6 +8,13 @@
   <xacro:include filename="$(find sr_description)/hand/xacro/finger/fingers.urdf.xacro" />
   <xacro:include filename="$(find sr_description)/hand/xacro/thumb/thumb.urdf.xacro" />
-  <!-- hand_type describes the hand type, hand_e, hand_e_plus, hand_m (muscle) -->
-  <!-- extra_lite (deprecated) describes if the hand is extra_lite -->
+  <!-- hand_type can be: hand_e, hand_e_plus, hand_m (muscle), hand_mt (muscletrans) -->
+  <!-- fingers: dict specifying available fingers, default: dict(th=1, ff=1, mf=1, rf=1, lf=1) -->
+  <!-- tip_sensors: dict specifying the fingertip (tactile) sensors per finger: std, none, bio, bt_sp, eli -->
+  <!-- mid_sensors: dict specifying the middle-phalange (tactile) sensors per finger: std, none, bio -->
+  <!-- prox_sensors: dict specifying the proximal (tactile) sensors per finger: std, none -->
+  <!-- palm_sensor: specifies the palm tactile sensor: std, none -->
+  <!-- reflect is either 1 (for right hand) or -1 (for left hand) -->
+  <!-- prefix can be anything but usually is "r_" or  "l_" for right and left hands distinction -->
+  <!-- extra_lite (deprecated) describes if the hand is extra_lite, i.e. without MF -->
   <!-- muscletrans (deprecated) is true for muscle transmission to be used, false to use motor transmission -->
   <!-- muscle (deprecated) is true for muscle hand or false for motor hand -->
@@ -15,18 +22,11 @@
   <!-- bt_sp (deprecated) is true for BT_SP finger or false for standard finger -->
   <!-- eli (deprecated) is true for ellipsoid fingertip or false for standard finger -->
-  <!-- tip_sensors vector that describes the sensor std, none, bio, bt_sp, eli -->
-  <!-- mid_sensors vector that describes the sensor std, none, bio -->
-  <!-- prox_sensors vector that describes the sensor std, none -->
-  <!-- palm_sensor describes the sensor none, bumper -->
-  <!-- reflect is either 1 (for right hand) or -1 (for left hand) -->
-  <!-- prefix can be anything but usually is "r_" or  "l_" for right and left hands distinction -->
-  <xacro:macro name="shadowhand" params="hand_type:='hand_e' reflect prefix cable_mesh:=False
-          fingers:=${[1,1,1,1]} tip_sensors:=${['std','std','std','std']} prox_sensors:=${['std','std','std','std']}
-          mid_sensors:=${['std','std','std','std']} palm_sensor:=std
-          muscletrans:=False muscle:=False lf:=True extra_lite:=False bio:=False bt_sp:=False eli:=False">
+  <xacro:macro name="shadowhand" params="hand_type:='hand_e' reflect prefix cable_mesh:=False fingers:=${[1,1,1,1]}
+          tip_sensors:=${4 * ['std']} mid_sensors:=${4 * ['std']} prox_sensors:=${4 * ['std']} palm_sensor:=std
+          extra_lite:=^|False muscletrans:=^|False muscle:=^|False bio:=^|False bt_sp:=^|False eli:=^|False">
     <!-- handle deprecated parameters -->
     <xacro:include filename="$(find sr_description)/hand/xacro/backward_compat.urdf.xacro" />
     <xacro:if value="${extra_lite}">
-      <xacro:property name="fingers" value="${[1,0,1,1]}"/>
+      <xacro:property name="fingers" value="${[1,1,0,1]}" />
     </xacro:if>
     <!-- Forearm -->
