Commit message: Fix backward compatibility
- Restore deleted files required by compatibility test
- Fix use of deprecated properties
- Fix use of deprecated parameters
- Undo unrelated changes w.r.t. upstream
- Fix extra_lite hands: it is missing MF not FF

File: sr_description/hand/xacro/th_ff_rf_ellipsoid_hand.urdf.xacro (robot description, xacro)
@@ -1,11 +1,3 @@
-<robot xmlns:sensor="http://playerstage.sourceforge.net/gazebo/xmlschema/#sensor"
-xmlns:controller="http://playerstage.sourceforge.net/gazebo/xmlschema/#controller"
-xmlns:interface="http://playerstage.sourceforge.net/gazebo/xmlschema/#interface"
-xmlns:xacro="http://www.ros.org/wiki/xacro">
-  <xacro:include filename="$(find sr_description)/hand/xacro/forearm/forearm.urdf.xacro" />
-  <xacro:include filename="$(find sr_description)/hand/xacro/wrist/wrist.urdf.xacro" />
-  <xacro:include filename="$(find sr_description)/hand/xacro/palm/palm.urdf.xacro" />
-  <xacro:include filename="$(find sr_description)/hand/xacro/finger/fingers.urdf.xacro" />
-  <xacro:include filename="$(find sr_description)/hand/xacro/thumb/thumb.urdf.xacro" />
+<robot xmlns:xacro="http://www.ros.org/wiki/xacro">
   <!-- muscletrans is true for muscle transmission to be used, false to use motor transmission -->
   <!-- muscle is true for muscle hand or false for motor hand -->
@@ -16,53 +8,13 @@
   <!-- prefix can be anything but usually is "r_" or  "l_" for right and left hands distinction -->
   <xacro:macro name="shadowhand" params="muscletrans muscle bio bt_sp eli reflect prefix">
-    <!-- Forearm -->
-    <xacro:forearm muscle="${muscle}" prefix="${prefix}" />
-    <!-- Wrist -->
-    <xacro:if value="${muscle}">
-      <xacro:wrist muscletrans="${muscletrans}" prefix="${prefix}"
-      reflect="${reflect}" parent="${prefix}forearm">
-        <origin xyz="0 0 0.4096" rpy="0 0 0" />
-      </xacro:wrist>
-    </xacro:if>
-    <xacro:unless value="${muscle}">
-      <xacro:wrist muscletrans="false" prefix="${prefix}"
-      reflect="${reflect}" parent="${prefix}forearm">
-        <origin xyz="0 -0.010 0.213" rpy="0 0 0" />
-      </xacro:wrist>
-    </xacro:unless>
-    <!-- Palm -->
-    <xacro:palm muscletrans="${muscletrans}" prefix="${prefix}"
-    reflect="${reflect}" parent="${prefix}wrist" />
-    <!-- First Finger Biotac -->
-    <xacro:finger muscletrans="${muscletrans}" lf="false" bio="false" bt_sp="false" eli="true" prefix="${prefix}"
-    reflect="${reflect}" link_prefix="ff" joint_prefix="FF"
-    parent="${prefix}palm">
-      <origin xyz="${reflect*0.033} 0 0.095" rpy="0 0 0" />
-      <axis xyz="0 ${-1*reflect} 0" />
-    </xacro:finger>
-    <!-- Middle Finger -->
-    <xacro:finger muscletrans="${muscletrans}" lf="false" bio="${bio}" bt_sp="${bt_sp}" eli="${eli}" prefix="${prefix}"
-    reflect="${reflect}" link_prefix="mf" joint_prefix="MF"
-    parent="${prefix}palm">
-      <origin xyz="${reflect*0.011} 0 0.099" rpy="0 0 0" />
-      <axis xyz="0 ${-1*reflect} 0" />
-    </xacro:finger>
-    <!-- Ring Finger -->
-    <xacro:finger muscletrans="${muscletrans}" lf="false" bio="false" bt_sp="false" eli="true" prefix="${prefix}"
-    reflect="${reflect}" link_prefix="rf" joint_prefix="RF"
-    parent="${prefix}palm">
-      <origin xyz="${reflect*-0.011} 0 0.095" rpy="0 0 0" />
-      <axis xyz="0 ${reflect} 0" />
-    </xacro:finger>
-    <!-- Little Finger  -->
-    <xacro:finger muscletrans="${muscletrans}" lf="true" bio="${bio}" bt_sp="${bt_sp}" eli="${eli}" prefix="${prefix}"
-    reflect="${reflect}" link_prefix="lf" joint_prefix="LF"
-    parent="${prefix}palm">
-      <origin xyz="0 0 0.06579" rpy="0 0 0" />
-      <axis xyz="0 ${reflect} 0" />
-    </xacro:finger>
-    <!-- Thumb Biotac -->
-    <xacro:thumb muscletrans="${muscletrans}" bio="false" bt_sp="false" eli="true" prefix="${prefix}" reflect="${reflect}"
-    is_lite="0" parent="${prefix}palm"></xacro:thumb>
+    <!-- Ensure tip_sensors is defined before usage below -->
+    <xacro:property name="tip_sensors" default="${5 * ['std']}" />
+    <!-- translate old parameters to new ones, eventually updating tip_sensors -->
+    <xacro:include filename="$(find sr_description)/hand/xacro/backward_compat.urdf.xacro" />
+    <!-- forward to generic macro -->
+    <xacro:include filename="$(find sr_description)/hand/xacro/full_hand.urdf.xacro" />
+    <!-- Enforce ellipsoid sensor on First and Ring Finger as well as Thumb -->
+    <xacro:shadowhand fingers="${5 * [1]}" reflect="${reflect}" prefix="${prefix}"
+    tip_sensors="${['eli', 'eli', tip_sensors[2], 'eli', tip_sensors[4]]}"/>
   </xacro:macro>
 </robot>

File: sr_description/hand/xacro/three_biotac_fingers_hand.urdf.xacro (robot description, xacro)
@@ -1,11 +1,3 @@
-<robot xmlns:sensor="http://playerstage.sourceforge.net/gazebo/xmlschema/#sensor"
-xmlns:controller="http://playerstage.sourceforge.net/gazebo/xmlschema/#controller"
-xmlns:interface="http://playerstage.sourceforge.net/gazebo/xmlschema/#interface"
-xmlns:xacro="http://www.ros.org/wiki/xacro">
-  <xacro:include filename="$(find sr_description)/hand/xacro/forearm/forearm.urdf.xacro" />
-  <xacro:include filename="$(find sr_description)/hand/xacro/wrist/wrist.urdf.xacro" />
-  <xacro:include filename="$(find sr_description)/hand/xacro/palm/palm.urdf.xacro" />
-  <xacro:include filename="$(find sr_description)/hand/xacro/finger/fingers.urdf.xacro" />
-  <xacro:include filename="$(find sr_description)/hand/xacro/thumb/thumb.urdf.xacro" />
+<robot xmlns:xacro="http://www.ros.org/wiki/xacro">
   <!-- muscletrans is true for muscle transmission to be used, false to use motor transmission -->
   <!-- muscle is true for muscle hand or false for motor hand -->
@@ -16,53 +8,9 @@
   <!-- prefix can be anything but usually is "r_" or  "l_" for right and left hands distinction -->
   <xacro:macro name="shadowhand" params="muscletrans muscle bio bt_sp eli reflect prefix">
-    <!-- Forearm -->
-    <xacro:forearm muscle="${muscle}" prefix="${prefix}" />
-    <!-- Wrist -->
-    <xacro:if value="${muscle}">
-      <xacro:wrist muscletrans="${muscletrans}" prefix="${prefix}"
-      reflect="${reflect}" parent="${prefix}forearm">
-        <origin xyz="0 0 0.4096" rpy="0 0 0" />
-      </xacro:wrist>
-    </xacro:if>
-    <xacro:unless value="${muscle}">
-      <xacro:wrist muscletrans="false" prefix="${prefix}"
-      reflect="${reflect}" parent="${prefix}forearm">
-        <origin xyz="0 -0.010 0.213" rpy="0 0 0" />
-      </xacro:wrist>
-    </xacro:unless>
-    <!-- Palm -->
-    <xacro:palm muscletrans="${muscletrans}" prefix="${prefix}"
-    reflect="${reflect}" parent="${prefix}wrist" />
-    <!-- First Finger Biotac -->
-    <xacro:finger muscletrans="${muscletrans}" lf="false" bio="true" bt_sp="false" eli="false" prefix="${prefix}"
-    reflect="${reflect}" link_prefix="ff" joint_prefix="FF"
-    parent="${prefix}palm">
-      <origin xyz="${reflect*0.033} 0 0.095" rpy="0 0 0" />
-      <axis xyz="0 ${-1*reflect} 0" />
-    </xacro:finger>
-    <!-- Middle Finger Biotac -->
-    <xacro:finger muscletrans="${muscletrans}" lf="false" bio="true" bt_sp="false" eli="false" prefix="${prefix}"
-    reflect="${reflect}" link_prefix="mf" joint_prefix="MF"
-    parent="${prefix}palm">
-      <origin xyz="${reflect*0.011} 0 0.099" rpy="0 0 0" />
-      <axis xyz="0 ${-1*reflect} 0" />
-    </xacro:finger>
-    <!-- Ring Finger -->
-    <xacro:finger muscletrans="${muscletrans}" lf="false" bio="false" bt_sp="false" eli="false" prefix="${prefix}"
-    reflect="${reflect}" link_prefix="rf" joint_prefix="RF"
-    parent="${prefix}palm">
-      <origin xyz="${reflect*-0.011} 0 0.095" rpy="0 0 0" />
-      <axis xyz="0 ${reflect} 0" />
-    </xacro:finger>
-    <!-- Little Finger  -->
-    <xacro:finger muscletrans="${muscletrans}" lf="true" bio="false" bt_sp="false" eli="false" prefix="${prefix}"
-    reflect="${reflect}" link_prefix="lf" joint_prefix="LF"
-    parent="${prefix}palm">
-      <origin xyz="0 0 0.06579" rpy="0 0 0" />
-      <axis xyz="0 ${reflect} 0" />
-    </xacro:finger>
-    <!-- Thumb Biotac -->
-    <xacro:thumb muscletrans="${muscletrans}" bio="true" bt_sp="false" eli="false" prefix="${prefix}" reflect="${reflect}"
-    is_lite="0" parent="${prefix}palm"></xacro:thumb>
+    <!-- forward to generic macro -->
+    <xacro:include filename="$(find sr_description)/hand/xacro/full_hand.urdf.xacro" />
+    <!-- BioTacs on First and Middle Finger as well as Thumb -->
+    <xacro:shadowhand reflect="${reflect}" prefix="${prefix}"
+    tip_sensors="${['bio', 'bio', 'bio', 'std', 'std']}"/>
   </xacro:macro>
 </robot>

File: sr_description/hand/xacro/three_fingers_hand.urdf.xacro (robot description, xacro)
@@ -1,11 +1,3 @@
-<robot xmlns:sensor="http://playerstage.sourceforge.net/gazebo/xmlschema/#sensor"
-xmlns:controller="http://playerstage.sourceforge.net/gazebo/xmlschema/#controller"
-xmlns:interface="http://playerstage.sourceforge.net/gazebo/xmlschema/#interface"
-xmlns:xacro="http://www.ros.org/wiki/xacro">
-  <xacro:include filename="$(find sr_description)/hand/xacro/forearm/forearm.urdf.xacro" />
-  <xacro:include filename="$(find sr_description)/hand/xacro/wrist/wrist.urdf.xacro" />
-  <xacro:include filename="$(find sr_description)/hand/xacro/palm/palm.urdf.xacro" />
-  <xacro:include filename="$(find sr_description)/hand/xacro/finger/fingers.urdf.xacro" />
-  <xacro:include filename="$(find sr_description)/hand/xacro/thumb/thumb.urdf.xacro" />
+<robot xmlns:xacro="http://www.ros.org/wiki/xacro">
   <!-- muscletrans is true for muscle transmission to be used, false to use motor transmission -->
   <!-- muscle is true for muscle hand or false for motor hand -->
@@ -16,40 +8,7 @@
   <!-- prefix can be anything but usually is "r_" or  "l_" for right and left hands distinction -->
   <xacro:macro name="shadowhand" params="muscletrans muscle bio bt_sp eli reflect prefix">
-    <!-- Forearm -->
-    <xacro:forearm muscle="${muscle}" prefix="${prefix}" />
-    <!-- Wrist -->
-    <xacro:if value="${muscle}">
-      <xacro:wrist muscletrans="${muscletrans}" prefix="${prefix}"
-      reflect="${reflect}" parent="${prefix}forearm">
-        <origin xyz="0 0 0.4096" rpy="0 0 0" />
-      </xacro:wrist>
-    </xacro:if>
-    <xacro:unless value="${muscle}">
-      <xacro:wrist muscletrans="${muscletrans}" prefix="${prefix}"
-      reflect="${reflect}" parent="${prefix}forearm">
-        <origin xyz="0 -0.010 0.213" rpy="0 0 0" />
-      </xacro:wrist>
-    </xacro:unless>
-    <!-- Palm -->
-    <xacro:palm muscletrans="${muscletrans}" prefix="${prefix}"
-    reflect="${reflect}" parent="${prefix}wrist" />
-    <!-- First Finger -->
-    <xacro:finger muscletrans="${muscletrans}" lf="false" bio="${bio}" bt_sp="${bt_sp}" eli="${eli}" prefix="${prefix}"
-    reflect="${reflect}" link_prefix="ff" joint_prefix="FF"
-    parent="${prefix}palm">
-      <origin xyz="${reflect*0.033} 0 0.095" rpy="0 0 0" />
-      <axis xyz="0 ${-1*reflect} 0" />
-    </xacro:finger>
-    <!-- Middle Finger -->
-    <xacro:finger muscletrans="${muscletrans}" lf="false" bio="${bio}" bt_sp="${bt_sp}" eli="${eli}" prefix="${prefix}"
-    reflect="${reflect}" link_prefix="mf" joint_prefix="MF"
-    parent="${prefix}palm">
-      <origin xyz="${reflect*0.011} 0 0.099" rpy="0 0 0" />
-      <axis xyz="0 ${-1*reflect} 0" />
-    </xacro:finger>
-    <!-- Thumb  -->
-    <xacro:thumb muscletrans="${muscletrans}" bio="${bio}" bt_sp="${bt_sp}" eli="${eli}" prefix="${prefix}"
-    reflect="${reflect}" is_lite="0" parent="${prefix}palm">
-    </xacro:thumb>
+    <!-- forward to generic macro -->
+    <xacro:include filename="$(find sr_description)/hand/xacro/full_hand.urdf.xacro" />
+    <xacro:shadowhand fingers="${[1,1,1,0,0]}" reflect="${reflect}" prefix="${prefix}" />
   </xacro:macro>
 </robot>

File: sr_description/hand/xacro/three_fingers_hand_RF.urdf.xacro (robot description, xacro)
@@ -1,11 +1,3 @@
-<robot xmlns:sensor="http://playerstage.sourceforge.net/gazebo/xmlschema/#sensor"
-xmlns:controller="http://playerstage.sourceforge.net/gazebo/xmlschema/#controller"
-xmlns:interface="http://playerstage.sourceforge.net/gazebo/xmlschema/#interface"
-xmlns:xacro="http://www.ros.org/wiki/xacro">
-  <xacro:include filename="$(find sr_description)/hand/xacro/forearm/forearm.urdf.xacro" />
-  <xacro:include filename="$(find sr_description)/hand/xacro/wrist/wrist.urdf.xacro" />
-  <xacro:include filename="$(find sr_description)/hand/xacro/palm/palm.urdf.xacro" />
-  <xacro:include filename="$(find sr_description)/hand/xacro/finger/fingers.urdf.xacro" />
-  <xacro:include filename="$(find sr_description)/hand/xacro/thumb/thumb.urdf.xacro" />
+<robot xmlns:xacro="http://www.ros.org/wiki/xacro">
   <!-- muscletrans is true for muscle transmission to be used, false to use motor transmission -->
   <!-- muscle is true for muscle hand or false for motor hand -->
@@ -16,40 +8,7 @@
   <!-- prefix can be anything but usually is "r_" or  "l_" for right and left hands distinction -->
   <xacro:macro name="shadowhand" params="muscletrans muscle bio bt_sp eli reflect prefix">
-    <!-- Forearm -->
-    <xacro:forearm muscle="${muscle}" prefix="${prefix}" />
-    <!-- Wrist -->
-    <xacro:if value="${muscle}">
-      <xacro:wrist muscletrans="${muscletrans}" prefix="${prefix}"
-      reflect="${reflect}" parent="${prefix}forearm">
-        <origin xyz="0 0 0.4096" rpy="0 0 0" />
-      </xacro:wrist>
-    </xacro:if>
-    <xacro:unless value="${muscle}">
-      <xacro:wrist muscletrans="${muscletrans}" prefix="${prefix}"
-      reflect="${reflect}" parent="${prefix}forearm">
-        <origin xyz="0 -0.010 0.213" rpy="0 0 0" />
-      </xacro:wrist>
-    </xacro:unless>
-    <!-- Palm -->
-    <xacro:palm muscletrans="${muscletrans}" prefix="${prefix}"
-    reflect="${reflect}" parent="${prefix}wrist" />
-    <!-- First Finger -->
-    <xacro:finger muscletrans="${muscletrans}" lf="false" bio="${bio}" bt_sp="${bt_sp}" eli="${eli}" prefix="${prefix}"
-    reflect="${reflect}" link_prefix="ff" joint_prefix="FF"
-    parent="${prefix}palm">
-      <origin xyz="${reflect*0.033} 0 0.095" rpy="0 0 0" />
-      <axis xyz="0 ${-1*reflect} 0" />
-    </xacro:finger>
-    <!-- Ring Finger -->
-    <xacro:finger muscletrans="${muscletrans}" lf="false" bio="${bio}" bt_sp="${bt_sp}" eli="${eli}" prefix="${prefix}"
-    reflect="${reflect}" link_prefix="rf" joint_prefix="RF"
-    parent="${prefix}palm">
-      <origin xyz="${reflect*-0.011} 0 0.095" rpy="0 0 0" />
-      <axis xyz="0 ${reflect} 0" />
-    </xacro:finger>
-    <!-- Thumb  -->
-    <xacro:thumb muscletrans="${muscletrans}" bio="${bio}" bt_sp="${bt_sp}" eli="${eli}" prefix="${prefix}"
-    reflect="${reflect}" is_lite="0" parent="${prefix}palm">
-    </xacro:thumb>
+    <!-- forward to generic macro -->
+    <xacro:include filename="$(find sr_description)/hand/xacro/full_hand.urdf.xacro" />
+    <xacro:shadowhand fingers="${[1, 1, 0, 1, 0]}" reflect="${reflect}" prefix="${prefix}" />
   </xacro:macro>
 </robot>

File: sr_description/hand/xacro/thumb/thumb.urdf.xacro (robot description, xacro)
@@ -14,4 +14,7 @@
   <xacro:macro name="thumb"
   params=" tip_sensor:=^|'std' mid_sensor:=^|'std' prox_sensor:=^|'std' reflect:=^ prefix:=^ parent is_lite">
+    <xacro:if value="${tip_sensor == 'bio'}">
+      <xacro:property name="mid_sensor" value="bio" />
+    </xacro:if>
     <!-- Base -->
     <xacro:thbase parent="${parent}" />

File: sr_description/robots/arm_and_sr_one_finger_motor.urdf.xacro (robot description, xacro)
@@ -19,5 +19,4 @@
     <dynamics damping="3.5" />
   </joint>
-  <xacro:shadowhand muscletrans="false" muscle="false" bio="false" bt_sp="false"
-  eli="false" reflect="1.0" prefix="rh_" />
+  <xacro:shadowhand reflect="1.0" prefix="rh_" />
 </robot>

File: sr_description/robots/sr_one_finger_motor.urdf.xacro (robot description, xacro)
@@ -14,5 +14,4 @@
     <origin xyz="0.0 0.0 0.0" rpy="0.0 0.0 0.0" />
   </joint>
-  <xacro:shadowhand muscletrans="false" muscle="false" bio="false" bt_sp="false"
-  eli="false" reflect="1.0" prefix="rh_" />
+  <xacro:shadowhand reflect="1.0" prefix="rh_" />
 </robot>

Commit message: Issue deprecation warning
Use python's None value as default to know whether old parameters were specified.

File: sr_description/hand/xacro/backward_compat.urdf.xacro (robot description, xacro)
@@ -1,3 +1,8 @@
 <robot xmlns:xacro="http://www.ros.org/wiki/xacro">
+  <xacro:property name="lf" default="${None}" />
+  <xacro:property name="extra_lite" default="${None}" />
+  <xacro:if value="${[p for p in [muscle, muscletrans, extra_lite, lf, bio, bt_sp, eli] if p is not None]}">
+    ${xacro.warning('Deprecated use of shadowhand macro: \nReplace parameters muscle, muscletrans, lf, extra_lite with hand_type and fingers\nand parameters bio, bt_sp, eli with [tip|mid|prox|palm]_sensors.')}
+  </xacro:if>
   <!-- for backward compatibility define new params from old ones -->
   <xacro:if value="${bio}">
@@ -27,3 +32,6 @@
     </xacro:unless>
   </xacro:if>
+  <xacro:if value="${lf is None}">
+    <xacro:property name="lf" value="True" />
+  </xacro:if>
 </robot>

File: sr_description/hand/xacro/full_hand.urdf.xacro (robot description, xacro)
@@ -21,5 +21,5 @@
   <xacro:macro name="shadowhand" params="hand_type:='hand_e' reflect prefix cable_mesh:=False fingers:=${[1,1,1,1,1]}
           tip_sensors:=${5 * ['std']} mid_sensors:=${5 * ['std']} prox_sensors:=${5 * ['std']} palm_sensor:=std
-          muscletrans:=^|False muscle:=^|False lf:=^|True bio:=^|False bt_sp:=^|False eli:=^|False">
+          muscletrans:=^|${None} muscle:=^|${None} lf:=^|${None} bio:=^|${None} bt_sp:=^|${None} eli:=^|${None}">
     <!-- handle deprecated parameters -->
     <xacro:include filename="$(find sr_description)/hand/xacro/backward_compat.urdf.xacro" />

File: sr_description/hand/xacro/hand_lite.urdf.xacro (robot description, xacro)
@@ -24,5 +24,5 @@
   <xacro:macro name="shadowhand" params="hand_type:='hand_e' reflect prefix cable_mesh:=False fingers:=${[1,1,1,1]}
           tip_sensors:=${4 * ['std']} mid_sensors:=${4 * ['std']} prox_sensors:=${4 * ['std']} palm_sensor:=std
-          extra_lite:=^|False muscletrans:=^|False muscle:=^|False bio:=^|False bt_sp:=^|False eli:=^|False">
+          extra_lite:=^|${None} muscletrans:=^|${None} muscle:=^|${None} bio:=^|${None} bt_sp:=^|${None} eli:=^|${None}">
     <!-- handle deprecated parameters -->
     <xacro:include filename="$(find sr_description)/hand/xacro/backward_compat.urdf.xacro" />

File: sr_description/hand/xacro/one_finger_unit.urdf.xacro (robot description, xacro)
@@ -20,5 +20,5 @@
   <xacro:macro name="shadowhand" params="hand_type:='hand_e' reflect prefix cable_mesh:=False
           tip_sensor:=std mid_sensor:=std prox_sensor:=std palm_sensor:=std
-          muscletrans:=False muscle:=False bio:=False bt_sp:=False eli:=False">
+          muscletrans:=${None} muscle:=${None} bio:=${None} bt_sp:=${None} eli:=${None}">
     <xacro:property name="tip_sensors" value="${5 * [tip_sensor]}" />
     <xacro:property name="mid_sensors" value="${5 * [mid_sensor]}" />
