Commit message: More readable hand_types: muscle, muscletrans, motor, motor+
- hand_mt -> muscletrans
- hand_m -> muscle, regexp: (["' ])hand_m -> $1muscle
- hand_e_plus -> motor+
- hand_e -> motor

File: sr_description/hand/xacro/backward_compat.urdf.xacro (robot description, xacro)
@@ -2,6 +2,6 @@
   <xacro:property name="lf" default="${None}" />
   <xacro:property name="extra_lite" default="${None}" />
-  <xacro:if value="${[p for p in [muscle, muscletrans, extra_lite, lf, bio, bt_sp, eli] if p is not None]}">
-    ${xacro.warning('Deprecated use of shadowhand macro: \nReplace parameters muscle, muscletrans, lf, extra_lite with hand_type and fingers\nand parameters bio, bt_sp, eli with [tip|mid|prox|palm]_sensors.')}
+  <xacro:if value="${[p for p in [extra_lite, lf, bio, bt_sp, eli] if p is not None]}">
+    ${xacro.warning('Deprecated use of shadowhand macro: \nReplace parameters lf, extra_lite with fingers\nand parameters bio, bt_sp, eli with [tip|mid|prox|palm]_sensors.')}
   </xacro:if>
   <!-- for backward compatibility define new params from old ones -->
@@ -24,12 +24,4 @@
     <xacro:property name="tip_sensors" value="${['eli', 'eli', 'eli', 'eli', 'eli']}" />
   </xacro:if>
-  <xacro:if value="${muscle}">
-    <xacro:if value="${muscletrans}">
-      <xacro:property name="hand_type" value="hand_mt" />
-    </xacro:if>
-    <xacro:unless value="${muscletrans}">
-      <xacro:property name="hand_type" value="hand_m" />
-    </xacro:unless>
-  </xacro:if>
   <xacro:if value="${lf is None}">
     <xacro:property name="lf" value="True" />

File: sr_description/hand/xacro/finger/distal/distal.transmission.xacro (robot description, xacro)
@@ -9,5 +9,5 @@
   <xacro:macro name="distal_transmission" params="hand_type:=^ prefix:=^ joint_prefix:=^ link_prefix:=^" >
    <!-- muscle hand -->
-    <xacro:if value="${hand_type == 'hand_mt'}">
+    <xacro:if value="${hand_type == 'muscletrans'}">
         <transmission name="${prefix}${link_prefix}distal_transmission">
             <type>sr_mechanism_model/SimpleTransmissionForMuscle</type>
@@ -22,5 +22,5 @@
     </xacro:if>
     <!-- motor hand -->
-    <xacro:unless value="${hand_type == 'hand_mt'}">
+    <xacro:unless value="${hand_type == 'muscletrans'}">
         <transmission name="${prefix}${link_prefix}distal_transmission">
             <type>sr_mechanism_model/SimpleTransmission</type>

File: sr_description/hand/xacro/finger/knuckle/knuckle.transmission.xacro (robot description, xacro)
@@ -9,5 +9,5 @@
     <xacro:macro name="knuckle_transmission" params="hand_type:=^ prefix:=^ joint_prefix:=^ link_prefix:=^">
         <!-- muscle hand -->
-        <xacro:if value="${hand_type == 'hand_mt'}">
+        <xacro:if value="${hand_type == 'muscletrans'}">
             <transmission name="${prefix}${link_prefix}knuckle_transmission">
                 <type>sr_mechanism_model/SimpleTransmissionForMuscle</type>
@@ -22,5 +22,5 @@
         </xacro:if>
         <!-- motor hand -->
-        <xacro:unless value="${hand_type == 'hand_mt'}">
+        <xacro:unless value="${hand_type == 'muscletrans'}">
             <transmission name="${prefix}${link_prefix}knuckle_transmission">
                 <type>sr_mechanism_model/SimpleTransmission</type>

File: sr_description/hand/xacro/finger/lfmetacarpal/lfmetacarpal.transmission.xacro (robot description, xacro)
@@ -7,5 +7,5 @@
     <xacro:macro name="lfmetacarpal_transmission" params="hand_type:=^ prefix:=^">
         <!-- muscle hand -->
-        <xacro:if value="${hand_type == 'hand_mt'}">
+        <xacro:if value="${hand_type == 'muscletrans'}">
             <transmission name="${prefix}lfmetacarpal_transmission">
                 <type>sr_mechanism_model/SimpleTransmissionForMuscle</type>
@@ -20,5 +20,5 @@
         </xacro:if>
         <!-- motor hand -->
-        <xacro:unless value="${hand_type == 'hand_mt'}">
+        <xacro:unless value="${hand_type == 'muscletrans'}">
             <transmission name="${prefix}lfmetacarpal_transmission">
                 <type>sr_mechanism_model/SimpleTransmission</type>

File: sr_description/hand/xacro/finger/middle/middle.transmission.xacro (robot description, xacro)
@@ -9,5 +9,5 @@
     <xacro:macro name="middle_transmission" params="hand_type:=^ prefix:=^ joint_prefix:=^ link_prefix:=^">
         <!-- muscle hand -->
-        <xacro:if value="${hand_type == 'hand_mt'}">
+        <xacro:if value="${hand_type == 'muscletrans'}">
             <transmission name="${prefix}${link_prefix}middle_transmission">
                 <type>sr_mechanism_model/J0TransmissionForMuscle</type>
@@ -27,5 +27,5 @@
         </xacro:if>
         <!-- motor hand -->
-        <xacro:unless value="${hand_type == 'hand_mt'}">
+        <xacro:unless value="${hand_type == 'muscletrans'}">
             <transmission name="${prefix}${link_prefix}middle_transmission">
                 <type>sr_mechanism_model/J0Transmission</type>

File: sr_description/hand/xacro/finger/proximal/proximal.transmission.xacro (robot description, xacro)
@@ -9,5 +9,5 @@
     <xacro:macro name="proximal_transmission" params="hand_type:=^ prefix:=^ joint_prefix:=^ link_prefix:=^">
         <!-- muscle hand -->
-        <xacro:if value="${hand_type == 'hand_mt'}">
+        <xacro:if value="${hand_type == 'muscletrans'}">
             <transmission name="${prefix}${link_prefix}proximal_transmission">
                 <type>sr_mechanism_model/SimpleTransmissionForMuscle</type>
@@ -22,5 +22,5 @@
         </xacro:if>
         <!-- motor hand -->
-        <xacro:unless value="${hand_type == 'hand_mt'}">
+        <xacro:unless value="${hand_type == 'muscletrans'}">
             <transmission name="${prefix}${link_prefix}proximal_transmission">
                 <type>sr_mechanism_model/SimpleTransmission</type>

File: sr_description/hand/xacro/forearm/forearm.urdf.xacro (robot description, xacro)
@@ -1,4 +1,4 @@
 <robot xmlns:xacro="http://www.ros.org/wiki/xacro">
-  <!-- hand_type can be either hand_e (default), hand_m, hand_e_plus -->
+  <!-- hand_type can be either motor (default), muscle, motor+ -->
   <!-- prefix can be anything but usually is "r_" or  "l_" for right and left hands distinction -->
   <!-- cable_mesh is set to true when cable collision should be taken into account -->
@@ -21,5 +21,5 @@
         iyz="0.0" izz="0.00744" />
       </inertial>
-      <xacro:if value="${hand_type.startswith('hand_m')}">
+      <xacro:if value="${hand_type.startswith('muscle')}">
         <visual>
           <origin xyz="0 0 0" rpy="0 0 0" />
@@ -30,6 +30,6 @@
         </visual>
       </xacro:if>
-      <xacro:unless value="${hand_type.startswith('hand_m')}">
-        <xacro:if value="${hand_type == 'hand_e'}">
+      <xacro:unless value="${hand_type.startswith('muscle')}">
+        <xacro:if value="${hand_type == 'motor'}">
           <visual>
             <origin xyz="0 0 0" rpy="0 0 0" />
@@ -40,5 +40,5 @@
           </visual>
         </xacro:if>
-        <xacro:if value="${hand_type == 'hand_e_plus'}">
+        <xacro:if value="${hand_type == 'motor+'}">
           <visual>
             <origin xyz="0 0 0" rpy="0 0 0" />
@@ -51,5 +51,5 @@
       </xacro:unless>
       <collision>
-        <xacro:if value="${hand_type.startswith('hand_m')}">
+        <xacro:if value="${hand_type.startswith('muscle')}">
           <origin xyz="0 0 0.185" rpy="0 0 0" />
           <geometry name="${prefix}forearm_collision">
@@ -58,6 +58,6 @@
           <xacro:dark_grey/>
         </xacro:if>
-        <xacro:unless value="${hand_type.startswith('hand_m')}">
-          <xacro:if value="${hand_type == 'hand_e'}">
+        <xacro:unless value="${hand_type.startswith('muscle')}">
+          <xacro:if value="${hand_type == 'motor'}">
             <origin xyz="0 0 0.092" rpy="0 0 0" />
             <geometry name="${prefix}forearm_collision">
@@ -66,5 +66,5 @@
             <xacro:dark_grey/>
           </xacro:if>
-          <xacro:if value="${hand_type == 'hand_e_plus'}">
+          <xacro:if value="${hand_type == 'motor+'}">
             <origin xyz="0 0 0" rpy="0 0 0" />
             <geometry name="${prefix}forearm_collision">
@@ -77,5 +77,5 @@
       <!-- wrist mount -->
       <collision>
-        <xacro:if value="${hand_type.startswith('hand_m')}">
+        <xacro:if value="${hand_type.startswith('muscle')}">
           <origin xyz="0 0 0.395" rpy="0 0 0" />
           <geometry>
@@ -83,5 +83,5 @@
           </geometry>
         </xacro:if>
-        <xacro:unless value="${hand_type.startswith('hand_m')}">
+        <xacro:unless value="${hand_type.startswith('muscle')}">
           <origin xyz="0 -0.01 0.181" rpy="0 0.78 0" />
           <geometry>

File: sr_description/hand/xacro/forearm/forearm_lite.urdf.xacro (robot description, xacro)
@@ -15,9 +15,9 @@
         <origin xyz="0 0 0" rpy="0 0 ${pi/2}" />
         <geometry name="${prefix}forearm_visual">
-          <xacro:if value="${hand_type == 'hand_m'}">
+          <xacro:if value="${hand_type == 'muscle'}">
             <mesh filename="package://sr_description/meshes/hand/forearm_lite.dae"
             scale="1.0 1.0 1.0" />
           </xacro:if>
-          <xacro:unless value="${hand_type == 'hand_m'}">
+          <xacro:unless value="${hand_type == 'muscle'}">
             <mesh filename="package://sr_description/meshes/hand/forearm_lite.dae"
             scale="1.0 1.0 1.0" />
@@ -27,5 +27,5 @@
       </visual>
       <collision>
-        <xacro:if value="${hand_type == 'hand_m'}">
+        <xacro:if value="${hand_type == 'muscle'}">
           <origin xyz="0 0 0.185" rpy="0 0 0" />
           <geometry name="${prefix}forearm_collision">
@@ -33,5 +33,5 @@
           </geometry>
         </xacro:if>
-        <xacro:unless value="${hand_type == 'hand_m'}">
+        <xacro:unless value="${hand_type == 'muscle'}">
           <origin xyz="0 0 0.065" rpy="0 0 0" />
           <geometry name="${prefix}forearm_collision">

File: sr_description/hand/xacro/full_hand.urdf.xacro (robot description, xacro)
@@ -5,5 +5,5 @@
   <xacro:include filename="$(find sr_description)/hand/xacro/finger/fingers.urdf.xacro" />
   <xacro:include filename="$(find sr_description)/hand/xacro/thumb/thumb.urdf.xacro" />
-  <!-- hand_type can be: hand_e, hand_e_plus, hand_m (muscle), hand_mt (muscletrans) -->
+  <!-- hand_type can be: motor, motor+, muscle (muscle), muscletrans (muscletrans) -->
   <!-- fingers: dict specifying available fingers, default: dict(th=1, ff=1, mf=1, rf=1, lf=1) -->
   <!-- tip_sensors: dict specifying the fingertip (tactile) sensors per finger: std, none, bio, bt_sp, eli -->
@@ -19,18 +19,19 @@
   <!-- eli (deprecated) is true for ellipsoid fingertip or false for standard finger -->
   <!-- lf (deprecated) is true if we want a little finger, false otherwise -->
-  <xacro:macro name="shadowhand" params="hand_type:='hand_e' reflect prefix cable_mesh:=False fingers:=${[1,1,1,1,1]}
+  <xacro:macro name="shadowhand" params="hand_type:='motor' reflect prefix cable_mesh:=False fingers:=${[1,1,1,1,1]}
           tip_sensors:=${5 * ['std']} mid_sensors:=${5 * ['std']} prox_sensors:=${5 * ['std']} palm_sensor:=std
           muscletrans:=^|${None} muscle:=^|${None} lf:=^|${None} bio:=^|${None} bt_sp:=^|${None} eli:=^|${None}">
-    <!-- handle deprecated parameters -->
+    <!-- Unify hand type parameter, also handling deprecated muscletrans, muscle -->
+    <xacro:include filename="$(find sr_description)/hand/xacro/process_hand_type_parameter.xacro" />
     <xacro:include filename="$(find sr_description)/hand/xacro/backward_compat.urdf.xacro" />
     <!-- Forearm -->
     <xacro:forearm />
     <!-- Wrist -->
-    <xacro:if value="${hand_type.startswith('hand_m')}">
+    <xacro:if value="${hand_type.startswith('muscle')}">
       <xacro:wrist parent="${prefix}forearm">
         <origin xyz="0 0 0.4096" rpy="0 0 0" />
       </xacro:wrist>
     </xacro:if>
-    <xacro:unless value="${hand_type.startswith('hand_m')}">
+    <xacro:unless value="${hand_type.startswith('muscle')}">
       <xacro:wrist parent="${prefix}forearm">
         <origin xyz="0 -0.010 0.213" rpy="0 0 0" />

File: sr_description/hand/xacro/hand_lite.urdf.xacro (robot description, xacro)
@@ -8,5 +8,5 @@
   <xacro:include filename="$(find sr_description)/hand/xacro/finger/fingers.urdf.xacro" />
   <xacro:include filename="$(find sr_description)/hand/xacro/thumb/thumb.urdf.xacro" />
-  <!-- hand_type can be: hand_e, hand_e_plus, hand_m (muscle), hand_mt (muscletrans) -->
+  <!-- hand_type can be: motor, motor+, muscle (muscle), muscletrans (muscletrans) -->
   <!-- fingers: dict specifying available fingers, default: dict(th=1, ff=1, mf=1, rf=1, lf=1) -->
   <!-- tip_sensors: dict specifying the fingertip (tactile) sensors per finger: std, none, bio, bt_sp, eli -->
@@ -22,8 +22,9 @@
   <!-- bt_sp (deprecated) is true for BT_SP finger or false for standard finger -->
   <!-- eli (deprecated) is true for ellipsoid fingertip or false for standard finger -->
-  <xacro:macro name="shadowhand" params="hand_type:='hand_e' reflect prefix cable_mesh:=False fingers:=${[1,1,1,1]}
+  <xacro:macro name="shadowhand" params="hand_type:='motor' reflect prefix cable_mesh:=False fingers:=${[1,1,1,1]}
           tip_sensors:=${4 * ['std']} mid_sensors:=${4 * ['std']} prox_sensors:=${4 * ['std']} palm_sensor:=std
           extra_lite:=^|${None} muscletrans:=^|${None} muscle:=^|${None} bio:=^|${None} bt_sp:=^|${None} eli:=^|${None}">
-    <!-- handle deprecated parameters -->
+    <!-- Unify hand type parameter, also handling deprecated muscletrans, muscle -->
+    <xacro:include filename="$(find sr_description)/hand/xacro/process_hand_type_parameter.xacro" />
     <xacro:include filename="$(find sr_description)/hand/xacro/backward_compat.urdf.xacro" />
     <xacro:if value="${extra_lite}">

File: sr_description/hand/xacro/one_finger_unit.urdf.xacro (robot description, xacro)
@@ -5,5 +5,5 @@
   <xacro:include filename="$(find sr_description)/hand/xacro/forearm/forearm.urdf.xacro" />
   <xacro:include filename="$(find sr_description)/hand/xacro/finger/fingers.urdf.xacro" />
-  <!-- hand_type describes the hand type, hand_e, hand_e_plus, hand_m (muscle) -->
+  <!-- hand_type describes the hand type, motor, motor+, muscle (muscle) -->
   <!-- muscletrans (deprecated) is true for muscle transmission to be used, false to use motor transmission -->
   <!-- muscle (deprecated) is true for muscle hand or false for motor hand -->
@@ -18,5 +18,5 @@
   <!-- reflect is either 1 (for right hand) or -1 (for left hand) -->
   <!-- prefix can be anything but usually is "r_" or  "l_" for right and left hands distinction -->
-  <xacro:macro name="shadowhand" params="hand_type:='hand_e' reflect prefix cable_mesh:=False
+  <xacro:macro name="shadowhand" params="hand_type:='motor' reflect prefix cable_mesh:=False
           tip_sensor:=std mid_sensor:=std prox_sensor:=std palm_sensor:=std
           muscletrans:=${None} muscle:=${None} bio:=${None} bt_sp:=${None} eli:=${None}">

File: sr_description/hand/xacro/palm/palm.transmission.xacro (robot description, xacro)
@@ -7,5 +7,5 @@
     <xacro:macro name="shadowhand_palm_transmission" params="hand_type:=^ prefix:=^">
         <!-- muscle hand -->
-        <xacro:if value="${hand_type == 'hand_mt'}">
+        <xacro:if value="${hand_type == 'muscletrans'}">
             <transmission name="${prefix}palm_transmission">
                 <type>sr_mechanism_model/SimpleTransmissionForMuscle</type>
@@ -20,5 +20,5 @@
         </xacro:if>
         <!-- motor hand -->
-        <xacro:unless value="${hand_type == 'hand_mt'}">
+        <xacro:unless value="${hand_type == 'muscletrans'}">
             <transmission name="${prefix}palm_transmission">
                 <type>sr_mechanism_model/SimpleTransmission</type>

File: sr_description/hand/xacro/thumb/thbase.transmission.xacro (robot description, xacro)
@@ -7,5 +7,5 @@
     <xacro:macro name="thbase_transmission" params="hand_type:=^ prefix:=^">
         <!-- muscle hand -->
-        <xacro:if value="${hand_type == 'hand_mt'}">
+        <xacro:if value="${hand_type == 'muscletrans'}">
             <transmission name="${prefix}thbase_transmission">
                 <type>sr_mechanism_model/SimpleTransmissionForMuscle</type>
@@ -20,5 +20,5 @@
         </xacro:if>
         <!-- motor hand -->
-        <xacro:unless value="${hand_type == 'hand_mt'}">
+        <xacro:unless value="${hand_type == 'muscletrans'}">
             <transmission name="${prefix}thbase_transmission">
                 <type>sr_mechanism_model/SimpleTransmission</type>

File: sr_description/hand/xacro/thumb/thdistal.transmission.xacro (robot description, xacro)
@@ -7,5 +7,5 @@
     <xacro:macro name="thdistal_transmission" params="hand_type:=^ prefix:=^">
         <!-- muscle hand -->
-        <xacro:if value="${hand_type == 'hand_mt'}">
+        <xacro:if value="${hand_type == 'muscletrans'}">
             <transmission name="${prefix}thdistal_transmission">
                 <type>sr_mechanism_model/SimpleTransmissionForMuscle</type>
@@ -20,5 +20,5 @@
         </xacro:if>
         <!-- motor hand -->
-        <xacro:unless value="${hand_type == 'hand_mt'}">
+        <xacro:unless value="${hand_type == 'muscletrans'}">
             <transmission name="${prefix}thdistal_transmission">
                 <type>sr_mechanism_model/SimpleTransmission</type>

File: sr_description/hand/xacro/thumb/thhub.transmission.xacro (robot description, xacro)
@@ -7,5 +7,5 @@
     <xacro:macro name="thhub_transmission" params="hand_type:=^ prefix:=^">
         <!-- muscle hand -->
-        <xacro:if value="${hand_type == 'hand_mt'}">
+        <xacro:if value="${hand_type == 'muscletrans'}">
             <transmission name="${prefix}thhub_transmission">
                 <type>sr_mechanism_model/SimpleTransmissionForMuscle</type>
@@ -20,5 +20,5 @@
         </xacro:if>
         <!-- motor hand -->
-        <xacro:unless value="${hand_type == 'hand_mt'}">
+        <xacro:unless value="${hand_type == 'muscletrans'}">
             <transmission name="${prefix}thhub_transmission">
                 <type>sr_mechanism_model/SimpleTransmission</type>

File: sr_description/hand/xacro/thumb/thmiddle.transmission.xacro (robot description, xacro)
@@ -7,5 +7,5 @@
     <xacro:macro name="thmiddle_transmission" params="hand_type:=^ prefix:=^">
         <!-- muscle hand -->
-        <xacro:if value="${hand_type == 'hand_mt'}">
+        <xacro:if value="${hand_type == 'muscletrans'}">
             <transmission name="${prefix}thmiddle_transmission">
                 <type>sr_mechanism_model/SimpleTransmissionForMuscle</type>
@@ -20,5 +20,5 @@
         </xacro:if>
         <!-- motor hand -->
-        <xacro:unless value="${hand_type == 'hand_mt'}">
+        <xacro:unless value="${hand_type == 'muscletrans'}">
             <transmission name="${prefix}thmiddle_transmission">
                 <type>sr_mechanism_model/SimpleTransmission</type>

File: sr_description/hand/xacro/thumb/thproximal.transmission.xacro (robot description, xacro)
@@ -7,5 +7,5 @@
     <xacro:macro name="thproximal_transmission" params="hand_type:=^ prefix:=^">
         <!-- muscle hand -->
-        <xacro:if value="${hand_type == 'hand_mt'}">
+        <xacro:if value="${hand_type == 'muscletrans'}">
             <transmission name="${prefix}thproximal_transmission">
                 <type>sr_mechanism_model/SimpleTransmissionForMuscle</type>
@@ -20,5 +20,5 @@
         </xacro:if>
         <!-- motor hand -->
-        <xacro:unless value="${hand_type == 'hand_mt'}">
+        <xacro:unless value="${hand_type == 'muscletrans'}">
             <transmission name="${prefix}thproximal_transmission">
                 <type>sr_mechanism_model/SimpleTransmission</type>

File: sr_description/hand/xacro/wrist/wrist.transmission.xacro (robot description, xacro)
@@ -7,5 +7,5 @@
     <xacro:macro name="shadowhand_wrist_transmission" params="hand_type:=^ prefix:=^">
         <!-- muscle hand -->
-        <xacro:if value="${hand_type == 'hand_mt'}">
+        <xacro:if value="${hand_type == 'muscletrans'}">
             <transmission name="${prefix}wrist_transmission">
                 <type>sr_mechanism_model/SimpleTransmissionForMuscle</type>
@@ -20,5 +20,5 @@
         </xacro:if>
         <!-- motor hand -->
-        <xacro:unless value="${hand_type == 'hand_mt'}">
+        <xacro:unless value="${hand_type == 'muscletrans'}">
             <transmission name="${prefix}wrist_transmission">
                 <type>sr_mechanism_model/SimpleTransmission</type>

File: sr_description/robots/arm_and_hand_motor.urdf.xacro (robot description, xacro)
@@ -16,4 +16,4 @@
     <origin xyz="0 0 0" rpy="0 0 ${2.35619449}" />
   </joint>
-  <xacro:shadowhand hand_type="hand_e" reflect="1.0" prefix="rh_" />
+  <xacro:shadowhand hand_type="motor" reflect="1.0" prefix="rh_" />
 </robot>

File: sr_description/robots/arm_and_hand_motor_biotac.urdf.xacro (robot description, xacro)
@@ -16,4 +16,4 @@
     <origin xyz="0 0 0" rpy="0 0 ${2.35619449}" />
   </joint>
-  <xacro:shadowhand hand_type="hand_e" tip_sensors="${['bio','bio','bio','bio','bio']}" reflect="1.0" prefix="rh_" />
+  <xacro:shadowhand hand_type="motor" tip_sensors="${['bio','bio','bio','bio','bio']}" reflect="1.0" prefix="rh_" />
 </robot>
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