Commit message: Fixed broken backward_compatibility
variable name was forgotten in the backward compat file, also hiding
typo mistakes from the xacro expansion due to lazy evaluation

File: sr_description/hand/xacro/backward_compat.urdf.xacro (robot description, xacro)
@@ -6,25 +6,25 @@
     <xacro:if value="${bio}">
       <xacro:property name="palm_sensor" value="std"/>
-      <xacro:property name="prox_sensor" value="${[std, std, std, std ,std]}"/>
-      <xacro:property name="mid_sensor" value="${[bio, bio, bio, bio ,bio]}"/>
-      <xacro:property name="tip_sensor" value="${[bio, bio, bio, bio ,bio]}"/>
+      <xacro:property name="prox_sensors" value="${['std','std','std','std','std']}"/>
+      <xacro:property name="mid_sensors" value="${['bio','bio','bio','bio','bio']}"/>
+      <xacro:property name="tip_sensors" value="${['bio','bio','bio','bio','bio']}"/>
     </xacro:if>
     <xacro:if value="${bt_sp}">
       <xacro:property name="palm_sensor" value="std"/>
-      <xacro:property name="prox_sensor" value="${[std, std, std, std ,std]}"/>
-      <xacro:property name="mid_sensor" value="${[std, std, std, std ,std]}"/>
-      <xacro:property name="tip_sensor" value="${[bt_sp, bt_sp, bt_sp, bt_sp ,bt_sp]}"/>
+      <xacro:property name="prox_sensors" value="${['std','std','std','std','std']}"/>
+      <xacro:property name="mid_sensors" value="${['std','std','std','std','std']}"/>
+      <xacro:property name="tip_sensors" value="${['bt_sp','bt_sp','bt_sp','bt_sp','bt_sp']}"/>
     </xacro:if>
     <xacro:if value="${ubi}">
       <xacro:property name="palm_sensor" value="ubi_fabric"/>
-      <xacro:property name="prox_sensor" value="${[ubi, ubi, ubi, ubi ,ubi]}"/>
-      <xacro:property name="mid_sensor" value="${[ubi, ubi, ubi, ubi ,ubi]}"/>
-      <xacro:property name="tip_sensor" value="${[ubi, ubi, ubi, ubi ,ubi]}"/>
+      <xacro:property name="prox_sensors" value="${['ubi','ubi,'ubi','ubi','ubi']}"/>
+      <xacro:property name="mid_sensors" value="${['ubi','ubi,'ubi','ubi','ubi']}"/>
+      <xacro:property name="tip_sensors" value="${['ubi','ubi,'ubi','ubi','ubi']}"/>
     </xacro:if>
     <xacro:if value="${eli}">
       <xacro:property name="palm_sensor" value="std"/>
-      <xacro:property name="prox_sensor" value="${[std, std, std, std ,std]}"/>
-      <xacro:property name="mid_sensor" value="${[std, std, std, std ,std]}"/>
-      <xacro:property name="tip_sensor" value="${[eli, eli, eli, eli ,eli]}"/>
+      <xacro:property name="prox_sensors" value="${['std','std','std','std','std']}"/>
+      <xacro:property name="mid_sensors" value="${['std','std','std','std','std']}"/>
+      <xacro:property name="tip_sensors" value="${['eli','eli','eli','eli','eli']}"/>
     </xacro:if>
   </xacro:if>

Commit message: Make fingers parameter a string

File: sr_description/hand/xacro/backward_compat.urdf.xacro (robot description, xacro)
@@ -1,7 +1,5 @@
 <robot xmlns:xacro="http://www.ros.org/wiki/xacro">
-  <xacro:property name="lf" default="${None}" />
-  <xacro:property name="extra_lite" default="${None}" />
-  <xacro:if value="${[p for p in [extra_lite, lf, bio, bt_sp, eli] if p is not None]}">
-    ${xacro.warning('Deprecated use of shadowhand macro: \nReplace parameters lf, extra_lite with fingers\nand parameters bio, bt_sp, eli with [tip|mid|prox|palm]_sensors.')}
+  <xacro:if value="${[p for p in [bio, bt_sp, eli] if p is not None]}">
+    ${xacro.warning('Deprecated use of shadowhand macro: Replace parameters bio, bt_sp, eli with [tip|mid|prox|palm]_sensors.')}
   </xacro:if>
   <!-- for backward compatibility define new params from old ones -->
@@ -24,6 +22,3 @@
     <xacro:property name="tip_sensors" value="${['eli', 'eli', 'eli', 'eli', 'eli']}" />
   </xacro:if>
-  <xacro:if value="${lf is None}">
-    <xacro:property name="lf" value="True" />
-  </xacro:if>
 </robot>

File: sr_description/hand/xacro/ff_biotac_hand.urdf.xacro (robot description, xacro)
@@ -17,5 +17,5 @@
     <xacro:include filename="$(find sr_description)/hand/xacro/full_hand.urdf.xacro" />
     <!-- Enforce BioTac on First Finger -->
-    <xacro:shadowhand fingers="${5 * [1]}" reflect="${reflect}" prefix="${prefix}"
+    <xacro:shadowhand fingers="all" reflect="${reflect}" prefix="${prefix}"
     tip_sensors="${[tip_sensors[0]] + ['bio'] + tip_sensors[2:]}"/>
   </xacro:macro>

File: sr_description/hand/xacro/full_hand.urdf.xacro (robot description, xacro)
@@ -6,5 +6,5 @@
   <xacro:include filename="$(find sr_description)/hand/xacro/thumb/thumb.urdf.xacro" />
   <!-- hand_type can be: motor, motor+, muscle (muscle), muscletrans (muscletrans) -->
-  <!-- fingers: dict specifying available fingers, default: dict(th=1, ff=1, mf=1, rf=1, lf=1) -->
+  <!-- fingers: list-like string specifying available fingers, default: 'th ff mf rf lf' -->
   <!-- tip_sensors: dict specifying the fingertip (tactile) sensors per finger: std, none, bio, bt_sp, eli -->
   <!-- mid_sensors: dict specifying the middle-phalange (tactile) sensors per finger: std, none, bio -->
@@ -19,9 +19,13 @@
   <!-- eli (deprecated) is true for ellipsoid fingertip or false for standard finger -->
   <!-- lf (deprecated) is true if we want a little finger, false otherwise -->
-  <xacro:macro name="shadowhand" params="hand_type:='motor' reflect prefix cable_mesh:=False fingers:=${[1,1,1,1,1]}
+  <xacro:macro name="shadowhand" params="hand_type:='motor' reflect prefix cable_mesh:=False fingers:=all
           tip_sensors:=${5 * ['std']} mid_sensors:=${5 * ['std']} prox_sensors:=${5 * ['std']} palm_sensor:=std
           muscletrans:=^|${None} muscle:=^|${None} lf:=^|${None} bio:=^|${None} bt_sp:=^|${None} eli:=^|${None}">
     <!-- Unify hand type parameter, also handling deprecated muscletrans, muscle -->
     <xacro:include filename="$(find sr_description)/hand/xacro/process_hand_type_parameter.xacro" />
+    <!-- Process fingers parameter, also handling deprecated lf -->
+    <xacro:property name="_all_finger_tokens_" value="${python.set('th ff mf rf lf'.split())}" />
+    <xacro:include filename="$(find sr_description)/hand/xacro/process_fingers_parameter.xacro" />
+    <!-- handle deprecated parameters -->
     <xacro:include filename="$(find sr_description)/hand/xacro/backward_compat.urdf.xacro" />
     <!-- Forearm -->
@@ -41,5 +45,5 @@
     <xacro:palm parent="${prefix}wrist" />
     <!-- First Finger -->
-    <xacro:if value="${fingers[1] == 1}">
+    <xacro:if value="${'ff' in fingers}">
       <xacro:finger link_prefix="ff" joint_prefix="FF" tip_sensor="${tip_sensors[1]}" prox_sensor="${prox_sensors[1]}" mid_sensor="${mid_sensors[1]}" parent="${prefix}palm">
         <origin xyz="${reflect*0.033} 0 0.095" rpy="0 0 0" />
@@ -48,5 +52,5 @@
     </xacro:if>
     <!-- Middle Finger -->
-    <xacro:if value="${fingers[2] == 1}">
+    <xacro:if value="${'mf' in fingers}">
       <xacro:finger link_prefix="mf" joint_prefix="MF" tip_sensor="${tip_sensors[2]}" prox_sensor="${prox_sensors[2]}" mid_sensor="${mid_sensors[2]}" parent="${prefix}palm">
         <origin xyz="${reflect*0.011} 0 0.099" rpy="0 0 0" />
@@ -55,5 +59,5 @@
     </xacro:if>
     <!-- Ring Finger -->
-    <xacro:if value="${fingers[3] == 1}">
+    <xacro:if value="${'rf' in fingers}">
       <xacro:finger link_prefix="rf" joint_prefix="RF" tip_sensor="${tip_sensors[3]}" prox_sensor="${prox_sensors[3]}" mid_sensor="${mid_sensors[3]}" parent="${prefix}palm">
         <origin xyz="${reflect*-0.011} 0 0.095" rpy="0 0 0" />
@@ -62,5 +66,5 @@
     </xacro:if>
     <!-- Little Finger  -->
-    <xacro:if value="${fingers[4] == 1 and lf}">
+    <xacro:if value="${'lf' in fingers}">
       <xacro:finger link_prefix="lf" joint_prefix="LF" tip_sensor="${tip_sensors[4]}" prox_sensor="${prox_sensors[4]}" mid_sensor="${mid_sensors[4]}" parent="${prefix}palm">
         <origin xyz="0 0 0.06579" rpy="0 0 0" />
@@ -69,5 +73,5 @@
     </xacro:if>
     <!-- Thumb  -->
-    <xacro:if value="${fingers[0] == 1}">
+    <xacro:if value="${'th' in fingers}">
       <xacro:thumb is_lite="0" parent="${prefix}palm" tip_sensor="${tip_sensors[0]}" prox_sensor="${prox_sensors[0]}" mid_sensor="${mid_sensors[0]}" />
     </xacro:if>

File: sr_description/hand/xacro/hand_E_no_mf_rf.urdf.xacro (robot description, xacro)
@@ -13,5 +13,5 @@
     <!-- forward to generic macro -->
     <xacro:include filename="$(find sr_description)/hand/xacro/full_hand.urdf.xacro" />
-    <xacro:shadowhand fingers="${[1, 1, 0, 0, 1 if lf else 0]}" reflect="${reflect}" prefix="${prefix}" />
+    <xacro:shadowhand fingers="th ff ${'lf' if lf else ''}" reflect="${reflect}" prefix="${prefix}" />
   </xacro:macro>
 </robot>

File: sr_description/hand/xacro/hand_lite.urdf.xacro (robot description, xacro)
@@ -9,5 +9,5 @@
   <xacro:include filename="$(find sr_description)/hand/xacro/thumb/thumb.urdf.xacro" />
   <!-- hand_type can be: motor, motor+, muscle (muscle), muscletrans (muscletrans) -->
-  <!-- fingers: dict specifying available fingers, default: dict(th=1, ff=1, mf=1, rf=1, lf=1) -->
+  <!-- fingers: list-like string specifying available fingers, default: 'th ff mf rf' -->
   <!-- tip_sensors: dict specifying the fingertip (tactile) sensors per finger: std, none, bio, bt_sp, eli -->
   <!-- mid_sensors: dict specifying the middle-phalange (tactile) sensors per finger: std, none, bio -->
@@ -22,13 +22,14 @@
   <!-- bt_sp (deprecated) is true for BT_SP finger or false for standard finger -->
   <!-- eli (deprecated) is true for ellipsoid fingertip or false for standard finger -->
-  <xacro:macro name="shadowhand" params="hand_type:='motor' reflect prefix cable_mesh:=False fingers:=${[1,1,1,1]}
+  <xacro:macro name="shadowhand" params="hand_type:='motor' reflect prefix cable_mesh:=False fingers:=all
           tip_sensors:=${4 * ['std']} mid_sensors:=${4 * ['std']} prox_sensors:=${4 * ['std']} palm_sensor:=std
           extra_lite:=^|${None} muscletrans:=^|${None} muscle:=^|${None} bio:=^|${None} bt_sp:=^|${None} eli:=^|${None}">
     <!-- Unify hand type parameter, also handling deprecated muscletrans, muscle -->
     <xacro:include filename="$(find sr_description)/hand/xacro/process_hand_type_parameter.xacro" />
+    <!-- Process fingers parameter, also handling deprecated extra_lite -->
+    <xacro:property name="_all_finger_tokens_" value="${python.set('th ff mf rf'.split())}" />
+    <xacro:include filename="$(find sr_description)/hand/xacro/process_fingers_parameter.xacro" />
+    <!-- handle deprecated parameters -->
     <xacro:include filename="$(find sr_description)/hand/xacro/backward_compat.urdf.xacro" />
-    <xacro:if value="${extra_lite}">
-      <xacro:property name="fingers" value="${[1,1,0,1]}" />
-    </xacro:if>
     <!-- Forearm -->
     <xacro:forearm />
@@ -44,5 +45,5 @@
     <xacro:palm parent="${prefix}wrist" />
     <!-- First Finger -->
-    <xacro:if value="${fingers[1] == 1}">
+    <xacro:if value="${'ff' in fingers}">
       <xacro:finger link_prefix="ff" joint_prefix="FF" tip_sensor="${tip_sensors[1]}"
                     prox_sensor="${prox_sensors[1]}" mid_sensor="${mid_sensors[1]}"
@@ -53,5 +54,5 @@
     </xacro:if>
     <!-- Middle Finger -->
-    <xacro:if value="${fingers[2] == 1}">
+    <xacro:if value="${'mf' in fingers}">
       <xacro:finger link_prefix="mf" joint_prefix="MF" tip_sensor="${tip_sensors[2]}"
                     prox_sensor="${prox_sensors[2]}" mid_sensor="${mid_sensors[2]}"
@@ -62,5 +63,5 @@
     </xacro:if>
     <!-- Ring Finger -->
-    <xacro:if value="${fingers[3] == 1}">
+    <xacro:if value="${'rf' in fingers}">
       <xacro:finger link_prefix="rf" joint_prefix="RF" tip_sensor="${tip_sensors[3]}"
                     prox_sensor="${prox_sensors[3]}" mid_sensor="${mid_sensors[3]}"
@@ -72,5 +73,5 @@
     <!-- No Little Finger on Lite hand -->
     <!-- Thumb  -->
-    <xacro:if value="${fingers[0] == 1}">
+    <xacro:if value="${'th' in fingers}">
       <xacro:thumb is_lite="1" parent="${prefix}palm" tip_sensor="${tip_sensors[0]}"
                    prox_sensor="${prox_sensors[0]}" mid_sensor="${mid_sensors[0]}" />

File: sr_description/hand/xacro/one_finger_unit.urdf.xacro (robot description, xacro)
@@ -21,4 +21,6 @@
           tip_sensor:=std mid_sensor:=std prox_sensor:=std palm_sensor:=std
           muscletrans:=${None} muscle:=${None} bio:=${None} bt_sp:=${None} eli:=${None}">
+    <!-- Unify hand type parameter, also handling deprecated muscletrans, muscle -->
+    <xacro:include filename="$(find sr_description)/hand/xacro/process_hand_type_parameter.xacro" />
     <xacro:property name="tip_sensors" value="${5 * [tip_sensor]}" />
     <xacro:property name="mid_sensors" value="${5 * [mid_sensor]}" />

File: sr_description/hand/xacro/th_ff_rf_ellipsoid_hand.urdf.xacro (robot description, xacro)
@@ -17,5 +17,5 @@
     <xacro:include filename="$(find sr_description)/hand/xacro/full_hand.urdf.xacro" />
     <!-- Enforce ellipsoid sensor on First and Ring Finger as well as Thumb -->
-    <xacro:shadowhand fingers="${5 * [1]}" reflect="${reflect}" prefix="${prefix}"
+    <xacro:shadowhand fingers="all" reflect="${reflect}" prefix="${prefix}"
     tip_sensors="${['eli', 'eli', tip_sensors[2], 'eli', tip_sensors[4]]}"/>
   </xacro:macro>

File: sr_description/hand/xacro/three_fingers_hand.urdf.xacro (robot description, xacro)
@@ -12,5 +12,5 @@
     <!-- forward to generic macro -->
     <xacro:include filename="$(find sr_description)/hand/xacro/full_hand.urdf.xacro" />
-    <xacro:shadowhand fingers="${[1,1,1,0,0]}" reflect="${reflect}" prefix="${prefix}" />
+    <xacro:shadowhand fingers="th ff mf" reflect="${reflect}" prefix="${prefix}" />
   </xacro:macro>
 </robot>

File: sr_description/hand/xacro/three_fingers_hand_RF.urdf.xacro (robot description, xacro)
@@ -12,5 +12,5 @@
     <!-- forward to generic macro -->
     <xacro:include filename="$(find sr_description)/hand/xacro/full_hand.urdf.xacro" />
-    <xacro:shadowhand fingers="${[1, 1, 0, 1, 0]}" reflect="${reflect}" prefix="${prefix}" />
+    <xacro:shadowhand fingers="th ff rf" reflect="${reflect}" prefix="${prefix}" />
   </xacro:macro>
 </robot>

File: sr_description/robots/arm_and_hand_motor_three_finger.urdf.xacro (robot description, xacro)
@@ -16,4 +16,4 @@
     <origin xyz="0 0 0" rpy="0 0 ${2.35619449}" />
   </joint>
-  <xacro:shadowhand hand_type="motor" fingers="${[1,1,1,0,0]}" reflect="1.0" prefix="rh_" />
+  <xacro:shadowhand hand_type="motor" fingers="th ff mf" reflect="1.0" prefix="rh_" />
 </robot>

File: sr_description/robots/bimanual_shadowhand_extra_lite.urdf.xacro (robot description, xacro)
@@ -11,5 +11,5 @@
     <origin xyz="0.0 0.0 0.0" rpy="0.0 0.0 0.0" />
   </joint>
-  <xacro:shadowhand hand_type="motor" fingers="${[1,1,0,1]}" reflect="1.0" prefix="rh_" />
+  <xacro:shadowhand hand_type="motor" fingers="th ff rf" reflect="1.0" prefix="rh_" />
   <joint name="right_hand_to_left_hand" type="fixed">
     <parent link="rh_forearm" />
@@ -17,4 +17,4 @@
     <origin xyz="$(arg arm_x_separation) 0.0 0.0" rpy="0.0 0.0 0.0" />
   </joint>
-  <xacro:shadowhand hand_type="motor" fingers="${[1,1,0,1]}" reflect="-1.0" prefix="lh_" />
+  <xacro:shadowhand hand_type="motor" fingers="th ff rf" reflect="-1.0" prefix="lh_" />
 </robot>

File: sr_description/robots/shadowhand_extra_lite.urdf.xacro (robot description, xacro)
@@ -14,4 +14,4 @@
     <origin xyz="0.0 0.0 0.0" rpy="0.0 0.0 0.0" />
   </joint>
-  <xacro:shadowhand hand_type="motor" fingers="${[1,1,0,1]}" reflect="1.0" prefix="rh_" />
+  <xacro:shadowhand hand_type="motor" fingers="th ff rf" reflect="1.0" prefix="rh_" />
 </robot>

File: sr_description/robots/shadowhand_left_extra_lite.urdf.xacro (robot description, xacro)
@@ -14,4 +14,4 @@
     <origin xyz="0.0 0.0 0.0" rpy="0.0 0.0 0.0" />
   </joint>
-  <xacro:shadowhand hand_type="motor" fingers="${[1,1,0,1]}" reflect="-1.0" prefix="lh_" />
+  <xacro:shadowhand hand_type="motor" fingers="th ff rf" reflect="-1.0" prefix="lh_" />
 </robot>

File: sr_description/robots/shadowhand_motor_no_lf.urdf.xacro (robot description, xacro)
@@ -14,4 +14,4 @@
       <origin xyz="0.0 0.0 0.0" rpy="0.0 0.0 0.0" />
     </joint>
-  <xacro:shadowhand hand_type="motor" fingers="${[1,1,1,1,0]}" reflect="1.0" prefix="rh_" />
+  <xacro:shadowhand hand_type="motor" fingers="th ff mf rf" reflect="1.0" prefix="rh_" />
 </robot>

File: sr_description/robots/shadowhand_motor_no_mf_rf_lf.urdf.xacro (robot description, xacro)
@@ -14,4 +14,4 @@
       <origin xyz="0.0 0.0 0.0" rpy="0.0 0.0 0.0" />
     </joint>
-  <xacro:shadowhand hand_type="motor" fingers="${[1,1,0,0,0]}" reflect="1.0" prefix="rh_" />
+  <xacro:shadowhand hand_type="motor" fingers="th ff" reflect="1.0" prefix="rh_" />
 </robot>

File: sr_description/robots/sr_three_finger_edc_muscle_biotac.urdf.xacro (robot description, xacro)
@@ -14,4 +14,4 @@
     <origin xyz="0.0 0.0 0.0" rpy="0.0 0.0 0.0" />
   </joint>
-  <xacro:shadowhand hand_type="muscletrans" fingers="${[1,1,1,0,0]}" tip_sensors="${['bio','bio','bio','std','std']}" reflect="1.0" prefix="rh_" />
+  <xacro:shadowhand hand_type="muscletrans" fingers="th ff mf" tip_sensors="${['bio','bio','bio','std','std']}" reflect="1.0" prefix="rh_" />
 </robot>

File: sr_description/robots/sr_three_finger_motor.urdf.xacro (robot description, xacro)
@@ -14,4 +14,4 @@
     <origin xyz="0.0 0.0 0.0" rpy="0.0 0.0 0.0" />
   </joint>
-  <xacro:shadowhand hand_type="motor" fingers="${[1,1,1,0,0]}" reflect="1.0" prefix="rh_" />
+  <xacro:shadowhand hand_type="motor" fingers="th ff mf" reflect="1.0" prefix="rh_" />
 </robot>

File: sr_description/robots/sr_three_finger_rf_motor.urdf.xacro (robot description, xacro)
@@ -14,4 +14,4 @@
     <origin xyz="0.0 0.0 0.0" rpy="0.0 0.0 0.0" />
   </joint>
-  <xacro:shadowhand hand_type="motor" fingers="${[1,1,0,1,0]}" reflect="1.0" prefix="rh_" />
+  <xacro:shadowhand hand_type="motor" fingers="th ff rf" reflect="1.0" prefix="rh_" />
 </robot>
