Commit message: Add lf parameter to full_hand. Create a hand E model with no lf

File: sr_description/hand/xacro/full_hand.urdf.xacro (robot description, xacro)
@@ -17,6 +17,7 @@
   <!-- reflect is either 1 (for right hand) or -1 (for left hand) -->
   <!-- prefix can be anything but usually is "r_" or  "l_" for right and left hands distinction -->
+  <!-- lf is true if we want a little finger, false otherwise -->
   <xacro:macro name="shadowhand"
-  params="muscletrans muscle bio bt_sp ubi eli reflect prefix">
+  params="muscletrans muscle bio bt_sp ubi eli reflect prefix lf">
     <!-- Forearm -->
     <xacro:forearm muscle="${muscle}" prefix="${prefix}" />
@@ -62,11 +63,13 @@
     </xacro:finger>
     <!-- Little Finger  -->
-    <xacro:finger muscletrans="${muscletrans}" lf="true"
-    bio="${bio}" bt_sp="${bt_sp}" ubi="${ubi}" eli="${eli}" prefix="${prefix}"
-    reflect="${reflect}" link_prefix="lf" joint_prefix="LF"
-    parent="${prefix}palm">
-      <origin xyz="0 0 0.06579" rpy="0 0 0" />
-      <axis xyz="0 ${reflect} 0" />
-    </xacro:finger>
+    <xacro:if value="${lf}">
+      <xacro:finger muscletrans="${muscletrans}" lf="true"
+      bio="${bio}" bt_sp="${bt_sp}" ubi="${ubi}" eli="${eli}" prefix="${prefix}"
+      reflect="${reflect}" link_prefix="lf" joint_prefix="LF"
+      parent="${prefix}palm">
+        <origin xyz="0 0 0.06579" rpy="0 0 0" />
+        <axis xyz="0 ${reflect} 0" />
+      </xacro:finger>
+    </xacro:if>
     <!-- Thumb  -->
     <xacro:thumb muscletrans="${muscletrans}" bio="${bio}" bt_sp="${bt_sp}"

File: sr_description/robots/arm_and_hand_motor.urdf.xacro (robot description, xacro)
@@ -17,4 +17,4 @@
   </joint>
   <xacro:shadowhand muscletrans="false" muscle="false" bio="false" bt_sp="false"
-  ubi="false" eli="false" reflect="1.0" prefix="rh_" />
+  ubi="false" eli="false" reflect="1.0" prefix="rh_" lf="true" />
 </robot>

File: sr_description/robots/arm_and_hand_motor_biotac.urdf.xacro (robot description, xacro)
@@ -17,4 +17,4 @@
   </joint>
   <xacro:shadowhand muscletrans="false" muscle="false" bio="true" bt_sp="false"
-  ubi="false" eli="false" reflect="1.0" prefix="rh_" />
+  ubi="false" eli="false" reflect="1.0" prefix="rh_" lf="true" />
 </robot>

File: sr_description/robots/arm_and_hand_motor_ellipsoid.urdf.xacro (robot description, xacro)
@@ -17,4 +17,4 @@
   </joint>
   <xacro:shadowhand muscletrans="false" muscle="false" bio="false" bt_sp="false"
-  ubi="false" eli="true" reflect="1.0" prefix="rh_" />
+  ubi="false" eli="true" reflect="1.0" prefix="rh_" lf="true" />
 </robot>

File: sr_description/robots/arm_and_hand_muscle.urdf.xacro (robot description, xacro)
@@ -17,4 +17,4 @@
   </joint>
   <xacro:shadowhand muscletrans="false" muscle="true" bio="false" bt_sp="false"
-  ubi="false" eli="false" reflect="1.0" prefix="rh_" />
+  ubi="false" eli="false" reflect="1.0" prefix="rh_" lf="true" />
 </robot>

File: sr_description/robots/arm_and_hand_muscle_biotac.urdf.xacro (robot description, xacro)
@@ -17,4 +17,4 @@
   </joint>
   <xacro:shadowhand muscletrans="false" muscle="true" bio="true" bt_sp="false"
-  ubi="false" eli="false" reflect="1.0" prefix="rh_" />
+  ubi="false" eli="false" reflect="1.0" prefix="rh_" lf="true" />
 </robot>

File: sr_description/robots/bimanual_shadowhand_motor.urdf.xacro (robot description, xacro)
@@ -11,5 +11,5 @@
   </joint>
   <xacro:shadowhand muscletrans="false" muscle="false" bio="false" bt_sp="false"
-  ubi="false" eli="false" reflect="1.0" prefix="rh_" />
+  ubi="false" eli="false" reflect="1.0" prefix="rh_" lf="true" />
   <joint name="right_hand_to_left_hand" type="fixed">
     <parent link="rh_forearm" />
@@ -18,4 +18,4 @@
   </joint>
   <xacro:shadowhand muscletrans="false" muscle="false" bio="false" bt_sp="false"
-  ubi="false" eli="false" reflect="-1.0" prefix="lh_" />
+  ubi="false" eli="false" reflect="-1.0" prefix="lh_" lf="true" />
 </robot>

File: sr_description/robots/desk_arm_and_hand_motor.urdf.xacro (robot description, xacro)
@@ -20,4 +20,4 @@
   </joint>
   <xacro:shadowhand muscletrans="false" muscle="false" bio="false" bt_sp="false"
-  ubi="false" eli="false" reflect="1.0" prefix="rh_" />
+  ubi="false" eli="false" reflect="1.0" prefix="rh_" lf="true" />
 </robot>

File: sr_description/robots/shadowhand_edc_muscle.urdf.xacro (robot description, xacro)
@@ -15,5 +15,5 @@
   </joint>
   <xacro:shadowhand muscletrans="true" muscle="true" bio="false" bt_sp="false"
-  ubi="false" eli="false" reflect="1.0" prefix="rh_" />
+  ubi="false" eli="false" reflect="1.0" prefix="rh_" lf="true" />
   <link name="rh_forearm_disk">
     <inertial>

File: sr_description/robots/shadowhand_edc_muscle_biotac.urdf.xacro (robot description, xacro)
@@ -18,5 +18,5 @@
 -->
   <xacro:shadowhand muscletrans="true" muscle="true" bio="true" bt_sp="false"
-  ubi="false" eli="false" reflect="1.0" prefix="rh_" />
+  ubi="false" eli="false" reflect="1.0" prefix="rh_" lf="true" />
   <link name="rh_forearm_disk">
     <inertial>

File: sr_description/robots/shadowhand_left_edc_muscle.urdf.xacro (robot description, xacro)
@@ -15,5 +15,5 @@
   </joint>
   <xacro:shadowhand muscletrans="true" muscle="true" bio="false" bt_sp="false"
-  ubi="false" eli="false" reflect="-1.0" prefix="lh_" />
+  ubi="false" eli="false" reflect="-1.0" prefix="lh_" lf="true" />
   <link name="lh_forearm_disk">
     <inertial>

File: sr_description/robots/shadowhand_left_motor.urdf.xacro (robot description, xacro)
@@ -15,4 +15,4 @@
   </joint>
   <xacro:shadowhand muscletrans="false" muscle="false" bio="false" bt_sp="false"
-  ubi="false" eli="false" reflect="-1.0" prefix="lh_" />
+  ubi="false" eli="false" reflect="-1.0" prefix="lh_" lf="true" />
 </robot>

File: sr_description/robots/shadowhand_left_motor_biotac.urdf.xacro (robot description, xacro)
@@ -15,4 +15,4 @@
   </joint>
   <xacro:shadowhand muscletrans="false" muscle="false" bio="true" bt_sp="false"
-  ubi="false" eli="false" reflect="-1.0" prefix="lh_" />
+  ubi="false" eli="false" reflect="-1.0" prefix="lh_" lf="true" />
 </robot>

File: sr_description/robots/shadowhand_left_muscle.urdf.xacro (robot description, xacro)
@@ -15,5 +15,5 @@
   </joint>
   <xacro:shadowhand muscletrans="false" muscle="true" bio="false" bt_sp="false"
-  ubi="false" eli="false" reflect="-1.0" prefix="lh_" />
+  ubi="false" eli="false" reflect="-1.0" prefix="lh_" lf="true" />
   <link name="lh_forearm_disk">
     <inertial>

File: sr_description/robots/shadowhand_motor_biotac.urdf.xacro (robot description, xacro)
@@ -18,4 +18,4 @@
 -->
   <xacro:shadowhand muscletrans="false" muscle="false" bio="true" bt_sp="false"
-  ubi="false" eli="false" reflect="1.0" prefix="rh_" />
+  ubi="false" eli="false" reflect="1.0" prefix="rh_" lf="true" />
 </robot>

File: sr_description/robots/shadowhand_motor_btsp.urdf.xacro (robot description, xacro)
@@ -15,4 +15,4 @@
   </joint>
   <xacro:shadowhand muscletrans="false" muscle="false" bio="false" bt_sp="true"
-  ubi="false" eli="false" reflect="1.0" prefix="rh_" />
+  ubi="false" eli="false" reflect="1.0" prefix="rh_" lf="true" />
 </robot>

File: sr_description/robots/shadowhand_motor_ellipsoid.urdf.xacro (robot description, xacro)
@@ -15,4 +15,4 @@
   </joint>
   <xacro:shadowhand muscletrans="false" muscle="false" bio="false" bt_sp="false"
-  ubi="false" eli="true" reflect="1.0" prefix="rh_" />
+  ubi="false" eli="true" reflect="1.0" prefix="rh_" lf="true" />
 </robot>

File: sr_description/robots/shadowhand_motor_no_lf.urdf.xacro (robot description, xacro)
@@ -15,4 +15,4 @@
     </joint>
     <xacro:shadowhand muscletrans="false" muscle="false" bio="false" bt_sp="false"
-                      ubi="false" eli="false" reflect="1.0" prefix="rh_" lf="true" />
+                      ubi="false" eli="false" reflect="1.0" prefix="rh_" lf="false" />
 </robot>

File: sr_description/robots/shadowhand_muscle.urdf.xacro (robot description, xacro)
@@ -15,5 +15,5 @@
   </joint>
   <xacro:shadowhand muscletrans="false" muscle="true" bio="false" bt_sp="false"
-  ubi="false" eli="false" reflect="1.0" prefix="rh_" />
+  ubi="false" eli="false" reflect="1.0" prefix="rh_" lf="true" />
   <link name="rh_forearm_disk">
     <inertial>

File: sr_description/robots/shadowhand_muscle_biotac.urdf.xacro (robot description, xacro)
@@ -18,5 +18,5 @@
   </joint>
   <xacro:shadowhand muscletrans="false" muscle="true" bio="true" bt_sp="false"
-  ubi="false" eli="false" reflect="1.0" prefix="rh_" />
+  ubi="false" eli="false" reflect="1.0" prefix="rh_" lf="true" />
   <link name="rh_forearm_disk">
     <inertial>
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
Commit message: Internally use dotified dict for *_sensors

File: sr_description/hand/xacro/full_hand.urdf.xacro (robot description, xacro)
@@ -46,5 +46,5 @@
     <!-- First Finger -->
     <xacro:if value="${'ff' in fingers}">
-      <xacro:finger link_prefix="ff" joint_prefix="FF" tip_sensor="${tip_sensors[1]}" prox_sensor="${prox_sensors[1]}" mid_sensor="${mid_sensors[1]}" parent="${prefix}palm">
+      <xacro:finger link_prefix="ff" joint_prefix="FF" tip_sensor="${tip_sensors.ff}" prox_sensor="${prox_sensors.ff}" mid_sensor="${mid_sensors.ff}" parent="${prefix}palm">
         <origin xyz="${reflect*0.033} 0 0.095" rpy="0 0 0" />
         <axis xyz="0 ${-1*reflect} 0" />
@@ -53,5 +53,5 @@
     <!-- Middle Finger -->
     <xacro:if value="${'mf' in fingers}">
-      <xacro:finger link_prefix="mf" joint_prefix="MF" tip_sensor="${tip_sensors[2]}" prox_sensor="${prox_sensors[2]}" mid_sensor="${mid_sensors[2]}" parent="${prefix}palm">
+      <xacro:finger link_prefix="mf" joint_prefix="MF" tip_sensor="${tip_sensors.mf}" prox_sensor="${prox_sensors.mf}" mid_sensor="${mid_sensors.mf}" parent="${prefix}palm">
         <origin xyz="${reflect*0.011} 0 0.099" rpy="0 0 0" />
         <axis xyz="0 ${-1*reflect} 0" />
@@ -60,5 +60,5 @@
     <!-- Ring Finger -->
     <xacro:if value="${'rf' in fingers}">
-      <xacro:finger link_prefix="rf" joint_prefix="RF" tip_sensor="${tip_sensors[3]}" prox_sensor="${prox_sensors[3]}" mid_sensor="${mid_sensors[3]}" parent="${prefix}palm">
+      <xacro:finger link_prefix="rf" joint_prefix="RF" tip_sensor="${tip_sensors.rf}" prox_sensor="${prox_sensors.rf}" mid_sensor="${mid_sensors.rf}" parent="${prefix}palm">
         <origin xyz="${reflect*-0.011} 0 0.095" rpy="0 0 0" />
         <axis xyz="0 ${reflect} 0" />
@@ -67,5 +67,5 @@
     <!-- Little Finger  -->
     <xacro:if value="${'lf' in fingers}">
-      <xacro:finger link_prefix="lf" joint_prefix="LF" tip_sensor="${tip_sensors[4]}" prox_sensor="${prox_sensors[4]}" mid_sensor="${mid_sensors[4]}" parent="${prefix}palm">
+      <xacro:finger link_prefix="lf" joint_prefix="LF" tip_sensor="${tip_sensors.lf}" prox_sensor="${prox_sensors.lf}" mid_sensor="${mid_sensors.lf}" parent="${prefix}palm">
         <origin xyz="0 0 0.06579" rpy="0 0 0" />
         <axis xyz="0 ${reflect} 0" />
@@ -74,5 +74,5 @@
     <!-- Thumb  -->
     <xacro:if value="${'th' in fingers}">
-      <xacro:thumb is_lite="0" parent="${prefix}palm" tip_sensor="${tip_sensors[0]}" prox_sensor="${prox_sensors[0]}" mid_sensor="${mid_sensors[0]}" />
+      <xacro:thumb is_lite="0" parent="${prefix}palm" tip_sensor="${tip_sensors.th}" prox_sensor="${prox_sensors.th}" mid_sensor="${mid_sensors.th}" />
     </xacro:if>
   </xacro:macro>

File: sr_description/hand/xacro/hand_lite.urdf.xacro (robot description, xacro)
@@ -46,6 +46,5 @@
     <!-- First Finger -->
     <xacro:if value="${'ff' in fingers}">
-      <xacro:finger link_prefix="ff" joint_prefix="FF" tip_sensor="${tip_sensors[1]}"
-                    prox_sensor="${prox_sensors[1]}" mid_sensor="${mid_sensors[1]}"
+      <xacro:finger link_prefix="ff" joint_prefix="FF" tip_sensor="${tip_sensors.ff}" prox_sensor="${prox_sensors.ff}" mid_sensor="${mid_sensors.ff}"
                     parent="${prefix}palm">
         <origin xyz="${reflect*0.033} 0 0.095" rpy="0 0 0" />
@@ -55,6 +54,5 @@
     <!-- Middle Finger -->
     <xacro:if value="${'mf' in fingers}">
-      <xacro:finger link_prefix="mf" joint_prefix="MF" tip_sensor="${tip_sensors[2]}"
-                    prox_sensor="${prox_sensors[2]}" mid_sensor="${mid_sensors[2]}"
+      <xacro:finger link_prefix="mf" joint_prefix="MF" tip_sensor="${tip_sensors.mf}" prox_sensor="${prox_sensors.mf}" mid_sensor="${mid_sensors.mf}"
                     parent="${prefix}palm">
         <origin xyz="${reflect*0.011} 0 0.099" rpy="0 0 0" />
@@ -64,6 +62,5 @@
     <!-- Ring Finger -->
     <xacro:if value="${'rf' in fingers}">
-      <xacro:finger link_prefix="rf" joint_prefix="RF" tip_sensor="${tip_sensors[3]}"
-                    prox_sensor="${prox_sensors[3]}" mid_sensor="${mid_sensors[3]}"
+      <xacro:finger link_prefix="rf" joint_prefix="RF" tip_sensor="${tip_sensors.rf}" prox_sensor="${prox_sensors.rf}" mid_sensor="${mid_sensors.rf}"
                     parent="${prefix}palm">
         <origin xyz="${reflect*-0.011} 0 0.095" rpy="0 0 0" />
@@ -74,6 +71,5 @@
     <!-- Thumb  -->
     <xacro:if value="${'th' in fingers}">
-      <xacro:thumb is_lite="1" parent="${prefix}palm" tip_sensor="${tip_sensors[0]}"
-                   prox_sensor="${prox_sensors[0]}" mid_sensor="${mid_sensors[0]}" />
+      <xacro:thumb is_lite="1" parent="${prefix}palm" tip_sensor="${tip_sensors.th}" prox_sensor="${prox_sensors.th}" mid_sensor="${mid_sensors.th}" />
     </xacro:if>
   </xacro:macro>

File: sr_description/hand/xacro/one_finger_unit.urdf.xacro (robot description, xacro)
@@ -62,6 +62,5 @@
     <!-- Middle Finger -->
     <!-- TODO: Check if offset is the same for muscle hand -->
-    <xacro:finger link_prefix="mf" joint_prefix="MF" tip_sensor="${tip_sensors[2]}"
-                  prox_sensor="${prox_sensors[2]}" mid_sensor="${mid_sensors[2]}"
+    <xacro:finger link_prefix="mf" joint_prefix="MF" tip_sensor="${tip_sensors.mf}" prox_sensor="${prox_sensors.mf}" mid_sensor="${mid_sensors.mf}"
                   parent="${prefix}palm">
       <origin xyz="0.0 0 0.116" rpy="0 0 0" />

File: sr_description/hand/xacro/process_sensor_parameters.xacro (robot description, xacro)
@@ -40,13 +40,17 @@
 		<!-- Finally, _tmp_ should become a list of (finger, sensor) pairs -->
 		<xacro:property name="_tmp_" value="${None}" />
+		<!-- Formatter for preferred dict-like string -->
+		<xacro:property name="_fmt_pair_" value="{f}={sensor}" />
 		<!-- Handle list input of single items -->
 		<xacro:if value="${_tmp_ is None and python.isinstance(value, list)}">
 			<!-- Transform into list of (finger,sensor) pairs -->
-			<xacro:property name="_tmp_" value="${python.zip(valid_finger_tokens, value)}" lazy_eval="false" />
+			<xacro:property name="_tmp_" value="${list(python.zip(valid_finger_tokens, value))}" lazy_eval="false" />
+			${xacro.warning('Deprecated specifier (list) used for ' + name + '. Replace with: ' + name + '="' + ' '.join([_fmt_pair_.format(f=k, sensor=v) for k,v in _tmp_]) + '"')}
 		</xacro:if>
 		<!-- Handle dict input -->
 		<xacro:if value="${_tmp_ is None and python.isinstance(value, dict)}">
 			<!-- Transform dict into list -->
-			<xacro:property name="_tmp_" value="${value.items()}" lazy_eval="false" />
+			<xacro:property name="_tmp_" value="${list(value.items())}" lazy_eval="false" />
+			${xacro.warning('Deprecated specifier (dict) used for ' + name + '. Replace with: ' + name + '="' + ' '.join([_fmt_pair_.format(f=k, sensor=v) for k,v in _tmp_]) + '"')}
 		</xacro:if>
 		<!-- Handle dict-like string: 'th=bio, ff=bio, mf=std, rf=std, lf=none' -->
@@ -72,8 +76,6 @@
 		<!-- Validate sensor tokens -->
 		<xacro:validate_tokens tokens="${_tmp_.values()}" valid="${valid_sensor_tokens}" name="tactile sensor specifier" />
-		<!-- Finally transform into desired type (a list) -->
-		<xacro:property name="${name}" value="${[v.lower() for k, v in _tmp_.items()]}" scope="parent" />
 		<!-- Finally transform into desired type (a dotified dict) -->
-		<xacro:property name="${name}_unused" value="${xacro.dotify(dict([(k.lower(), v.lower()) for k, v in _tmp_.items()]))}" scope="parent" />
+		<xacro:property name="${name}" value="${xacro.dotify(dict([(k.lower(), v.lower()) for k, v in _tmp_.items()]))}" scope="parent" />
 	</xacro:macro>
 	<xacro:transform_to_type name="tip_sensors" value="${tip_sensors}" />
