Commit message: Python 2.x compatibility
As xacro returns unicode objects from property evaluations
we cannot apply str.lower to them in Python 2.x
In Python 3.x str and unicode is essentially the same.

File: sr_description/hand/xacro/process_fingers_parameter.xacro (robot description, xacro)
@@ -8,5 +8,5 @@
 	</xacro:unless>
 	<!-- Normalize finger tokens to lower case -->
-	<xacro:property name="fingers" value="${list(map(str.lower, fingers))}" lazy_eval="false" />
+	<xacro:property name="fingers" value="${[f.lower() for f in fingers]}" lazy_eval="false" />
 	<!-- Validate for invalid finger tokens -->
 	<xacro:property name="_unknown_finger_tokens_" value="${python.set(fingers) - _all_finger_tokens_}" />
