Commit message: Remove redundant definition of pi
pi is available globally in xacro as python's math.pi

File: sr_description/hand/xacro/ff_biotac_hand.urdf.xacro (robot description, xacro)
@@ -8,5 +8,4 @@
   <xacro:include filename="$(find sr_description)/hand/xacro/finger/fingers.urdf.xacro" />
   <xacro:include filename="$(find sr_description)/hand/xacro/thumb/thumb.urdf.xacro" />
-  <xacro:property name="pi" value="3.1415926535897931" />
   <!-- muscletrans is true for muscle transmission to be used, false to use motor transmission -->
   <!-- muscle is true for muscle hand or false for motor hand -->

File: sr_description/hand/xacro/full_hand.urdf.xacro (robot description, xacro)
@@ -8,5 +8,4 @@
   <xacro:include filename="$(find sr_description)/hand/xacro/finger/fingers.urdf.xacro" />
   <xacro:include filename="$(find sr_description)/hand/xacro/thumb/thumb.urdf.xacro" />
-  <xacro:property name="pi" value="3.1415926535897931" />
   <!-- muscletrans is true for muscle transmission to be used, false to use motor transmission -->
   <!-- muscle is true for muscle hand or false for motor hand -->

File: sr_description/hand/xacro/hand_E_no_mf_rf.urdf.xacro (robot description, xacro)
@@ -8,5 +8,4 @@
   <xacro:include filename="$(find sr_description)/hand/xacro/finger/fingers.urdf.xacro" />
   <xacro:include filename="$(find sr_description)/hand/xacro/thumb/thumb.urdf.xacro" />
-  <xacro:property name="pi" value="3.1415926535897931" />
   <!-- muscletrans is true for muscle transmission to be used, false to use motor transmission -->
   <!-- muscle is true for muscle hand or false for motor hand -->

File: sr_description/hand/xacro/one_finger_unit.urdf.xacro (robot description, xacro)
@@ -5,5 +5,4 @@
   <xacro:include filename="$(find sr_description)/hand/xacro/forearm/forearm.urdf.xacro" />
   <xacro:include filename="$(find sr_description)/hand/xacro/finger/fingers.urdf.xacro" />
-  <xacro:property name="pi" value="3.1415926535897931" />
   <!-- muscletrans is true for muscle transmission to be used, false to use motor transmission -->
   <!-- muscle is true for muscle hand or false for motor hand -->

File: sr_description/hand/xacro/th_ff_rf_ellipsoid_hand.urdf.xacro (robot description, xacro)
@@ -8,5 +8,4 @@
   <xacro:include filename="$(find sr_description)/hand/xacro/finger/fingers.urdf.xacro" />
   <xacro:include filename="$(find sr_description)/hand/xacro/thumb/thumb.urdf.xacro" />
-  <xacro:property name="pi" value="3.1415926535897931" />
   <!-- muscletrans is true for muscle transmission to be used, false to use motor transmission -->
   <!-- muscle is true for muscle hand or false for motor hand -->

File: sr_description/hand/xacro/three_biotac_fingers_hand.urdf.xacro (robot description, xacro)
@@ -8,5 +8,4 @@
   <xacro:include filename="$(find sr_description)/hand/xacro/finger/fingers.urdf.xacro" />
   <xacro:include filename="$(find sr_description)/hand/xacro/thumb/thumb.urdf.xacro" />
-  <xacro:property name="pi" value="3.1415926535897931" />
   <!-- muscletrans is true for muscle transmission to be used, false to use motor transmission -->
   <!-- muscle is true for muscle hand or false for motor hand -->

File: sr_description/hand/xacro/three_fingers_hand.urdf.xacro (robot description, xacro)
@@ -8,5 +8,4 @@
   <xacro:include filename="$(find sr_description)/hand/xacro/finger/fingers.urdf.xacro" />
   <xacro:include filename="$(find sr_description)/hand/xacro/thumb/thumb.urdf.xacro" />
-  <xacro:property name="pi" value="3.1415926535897931" />
   <!-- muscletrans is true for muscle transmission to be used, false to use motor transmission -->
   <!-- muscle is true for muscle hand or false for motor hand -->

File: sr_description/hand/xacro/three_fingers_hand_RF.urdf.xacro (robot description, xacro)
@@ -8,5 +8,4 @@
   <xacro:include filename="$(find sr_description)/hand/xacro/finger/fingers.urdf.xacro" />
   <xacro:include filename="$(find sr_description)/hand/xacro/thumb/thumb.urdf.xacro" />
-  <xacro:property name="pi" value="3.1415926535897931" />
   <!-- muscletrans is true for muscle transmission to be used, false to use motor transmission -->
   <!-- muscle is true for muscle hand or false for motor hand -->

File: sr_description/other/xacro/kinect/shadowarm_kinect.urdf.xacro (robot description, xacro)
@@ -1,4 +1,3 @@
 <robot xmlns:xacro="http://www.ros.org/wiki/xacro">
-  <xacro:property name="pi" value="3.1415926535" />
   <xacro:include filename="$(find sr_description)/other/xacro/kinect/gazebo_kinect.urdf.xacro" />
   <xacro:macro name="shadowarm_side_kinect" params="parent">

Commit message: Simplify syntax for sensor specification
Use textual sensor specifications:
- tip_sensors=bio
- tip_sensors='th=bio, ff=bio, mf=std, rf=std, lf=none'
- tip_sensors='bio, bio, std, std, none'

- Rename backward_compat.urdf.xacro -> process_sensor_parameters.xacro
- Introduce macro validate_tokens

File: sr_description/hand/xacro/ff_biotac_hand.urdf.xacro (robot description, xacro)
@@ -10,8 +10,6 @@
     ${xacro.warning("The file ff_biotac_hand.urdf.xacro is deprecated", print_location=False)}
     ${xacro.warning("Use full_hand.urdf.xacro instead with tip_sensors=dict(ff='bio')")}
-    <!-- Ensure tip_sensors is defined before usage below -->
-    <xacro:property name="tip_sensors" default="${5 * ['std']}" />
-    <!-- translate old parameters to new ones, eventually updating tip_sensors -->
-    <xacro:include filename="$(find sr_description)/hand/xacro/backward_compat.urdf.xacro" />
+    <!-- translate old parameters to new ones, eventually initializing tip_sensors -->
+    <xacro:include filename="$(find sr_description)/hand/xacro/process_sensor_parameters.xacro" />
     <!-- forward to generic macro -->
     <xacro:include filename="$(find sr_description)/hand/xacro/full_hand.urdf.xacro" />

File: sr_description/hand/xacro/full_hand.urdf.xacro (robot description, xacro)
@@ -27,6 +27,6 @@
     <xacro:property name="_all_finger_tokens_" value="${python.set('th ff mf rf lf'.split())}" />
     <xacro:include filename="$(find sr_description)/hand/xacro/process_fingers_parameter.xacro" />
-    <!-- handle deprecated parameters -->
-    <xacro:include filename="$(find sr_description)/hand/xacro/backward_compat.urdf.xacro" />
+    <!-- Process sensor parameters -->
+    <xacro:include filename="$(find sr_description)/hand/xacro/process_sensor_parameters.xacro" />
     <!-- Forearm -->
     <xacro:forearm />

File: sr_description/hand/xacro/hand_lite.urdf.xacro (robot description, xacro)
@@ -30,6 +30,6 @@
     <xacro:property name="_all_finger_tokens_" value="${python.set('th ff mf rf'.split())}" />
     <xacro:include filename="$(find sr_description)/hand/xacro/process_fingers_parameter.xacro" />
-    <!-- handle deprecated parameters -->
-    <xacro:include filename="$(find sr_description)/hand/xacro/backward_compat.urdf.xacro" />
+    <!-- Process sensor parameters -->
+    <xacro:include filename="$(find sr_description)/hand/xacro/process_sensor_parameters.xacro" />
     <!-- Forearm -->
     <xacro:forearm />

File: sr_description/hand/xacro/one_finger_unit.urdf.xacro (robot description, xacro)
@@ -23,8 +23,10 @@
     <!-- Unify hand type parameter, also handling deprecated muscletrans, muscle -->
     <xacro:include filename="$(find sr_description)/hand/xacro/process_hand_type_parameter.xacro" />
-    <xacro:property name="tip_sensors" value="${5 * [tip_sensor]}" />
-    <xacro:property name="mid_sensors" value="${5 * [mid_sensor]}" />
-    <xacro:property name="prox_sensors" value="${5 * [prox_sensor]}" />
-    <xacro:include filename="$(find sr_description)/hand/xacro/backward_compat.urdf.xacro" />
+    <!-- Translate [tip|mid|prox]_sensor to plural form handled in process_sensor_parameters.xacro -->
+    <xacro:property name="tip_sensors" value="${tip_sensor}" />
+    <xacro:property name="mid_sensors" value="${mid_sensor}" />
+    <xacro:property name="prox_sensors" value="${prox_sensor}" />
+    <!-- Process sensor parameters -->
+    <xacro:include filename="$(find sr_description)/hand/xacro/process_sensor_parameters.xacro" />
     <!-- Forearm -->
     <xacro:forearm />

File: sr_description/hand/xacro/process_fingers_parameter.xacro (robot description, xacro)
@@ -1,3 +1,4 @@
 <robot xmlns:xacro="http://www.ros.org/wiki/xacro">
+	<xacro:include filename="$(find sr_description)/hand/xacro/validate_macros.xacro" />
 	<xacro:if value="${fingers.lower() == 'all'}">
 		<xacro:property name="fingers" value="${list(_all_finger_tokens_)}" />
@@ -9,7 +10,6 @@
 	<!-- Normalize finger tokens to lower case -->
 	<xacro:property name="fingers" value="${[f.lower() for f in fingers]}" lazy_eval="false" />
-	<!-- Validate for invalid finger tokens -->
-	<xacro:property name="_unknown_finger_tokens_" value="${python.set(fingers) - _all_finger_tokens_}" />
-	<xacro:if value="${_unknown_finger_tokens_}">${xacro.error('Unknown finger specifiers: ' + ', '.join(_unknown_finger_tokens_))}</xacro:if>
+	<!-- Validate finger tokens -->
+	<xacro:validate_tokens tokens="${fingers}" valid="${_all_finger_tokens_}" name="finger specifier" />
 	<!-- Handle deprecated lf parameter -->
 	<xacro:property name="lf" default="${None}" />

File: sr_description/hand/xacro/th_ff_rf_ellipsoid_hand.urdf.xacro (robot description, xacro)
@@ -13,5 +13,5 @@
     <xacro:property name="tip_sensors" default="${5 * ['std']}" />
     <!-- translate old parameters to new ones, eventually updating tip_sensors -->
-    <xacro:include filename="$(find sr_description)/hand/xacro/backward_compat.urdf.xacro" />
+    <xacro:include filename="$(find sr_description)/hand/xacro/process_sensor_parameters.xacro" />
     <!-- forward to generic macro -->
     <xacro:include filename="$(find sr_description)/hand/xacro/full_hand.urdf.xacro" />

Commit message: Apply new sensor specification

File: sr_description/hand/xacro/ff_biotac_hand.urdf.xacro (robot description, xacro)
@@ -9,5 +9,5 @@
   <xacro:macro name="shadowhand" params="muscletrans muscle bio bt_sp eli reflect prefix">
     ${xacro.warning("The file ff_biotac_hand.urdf.xacro is deprecated", print_location=False)}
-    ${xacro.warning("Use full_hand.urdf.xacro instead with tip_sensors=dict(ff='bio')")}
+    ${xacro.warning("Use full_hand.urdf.xacro instead with tip_sensors='ff=bio'")}
     <!-- translate old parameters to new ones, eventually initializing tip_sensors -->
     <xacro:include filename="$(find sr_description)/hand/xacro/process_sensor_parameters.xacro" />
@@ -16,5 +16,5 @@
     <!-- Enforce BioTac on First Finger -->
     <xacro:shadowhand fingers="all" reflect="${reflect}" prefix="${prefix}"
-    tip_sensors="${[tip_sensors[0]] + ['bio'] + tip_sensors[2:]}"/>
+    tip_sensors="${' '.join([k+'='+v for k, v in tip_sensors.items()] + ['ff=bio'])}"/>
   </xacro:macro>
 </robot>

File: sr_description/hand/xacro/full_hand.urdf.xacro (robot description, xacro)
@@ -7,7 +7,7 @@
   <!-- hand_type can be: motor, motor+, muscle (muscle), muscletrans (muscletrans) -->
   <!-- fingers: list-like string specifying available fingers, default: 'th ff mf rf lf' -->
-  <!-- tip_sensors: dict specifying the fingertip (tactile) sensors per finger: std, none, bio, bt_sp, eli -->
-  <!-- mid_sensors: dict specifying the middle-phalange (tactile) sensors per finger: std, none, bio -->
-  <!-- prox_sensors: dict specifying the proximal (tactile) sensors per finger: std, none -->
+  <!-- tip_sensors: plain or dict-like string specifying the fingertip (tactile) sensors: 'th=bio ff=bt_sp mf=eli rf=std, lf=none' -->
+  <!-- mid_sensors: plain or dict-like string specifying the middle-phalange (tactile) sensors -->
+  <!-- prox_sensors: plain or dict-like string specifying the proximal (tactile) sensors -->
   <!-- palm_sensor: specifies the palm tactile sensor: std, none -->
   <!-- reflect is either 1 (for right hand) or -1 (for left hand) -->
@@ -20,5 +20,5 @@
   <!-- lf (deprecated) is true if we want a little finger, false otherwise -->
   <xacro:macro name="shadowhand" params="hand_type:='motor' reflect prefix cable_mesh:=False fingers:=all
-          tip_sensors:=${5 * ['std']} mid_sensors:=${5 * ['std']} prox_sensors:=${5 * ['std']} palm_sensor:=std
+          tip_sensors:=std mid_sensors:=std prox_sensors:=std palm_sensor:=std
           muscletrans:=^|${None} muscle:=^|${None} lf:=^|${None} bio:=^|${None} bt_sp:=^|${None} eli:=^|${None}">
     <!-- Unify hand type parameter, also handling deprecated muscletrans, muscle -->

File: sr_description/hand/xacro/hand_lite.urdf.xacro (robot description, xacro)
@@ -10,7 +10,7 @@
   <!-- hand_type can be: motor, motor+, muscle (muscle), muscletrans (muscletrans) -->
   <!-- fingers: list-like string specifying available fingers, default: 'th ff mf rf' -->
-  <!-- tip_sensors: dict specifying the fingertip (tactile) sensors per finger: std, none, bio, bt_sp, eli -->
-  <!-- mid_sensors: dict specifying the middle-phalange (tactile) sensors per finger: std, none, bio -->
-  <!-- prox_sensors: dict specifying the proximal (tactile) sensors per finger: std, none -->
+  <!-- tip_sensors: plain or dict-like string specifying the fingertip (tactile) sensors: 'th=bio ff=bt_sp mf=eli rf=std, lf=none' -->
+  <!-- mid_sensors: plain or dict-like string specifying the middle-phalange (tactile) sensors -->
+  <!-- prox_sensors: plain or dict-like string specifying the proximal (tactile) sensors -->
   <!-- palm_sensor: specifies the palm tactile sensor: std, none -->
   <!-- reflect is either 1 (for right hand) or -1 (for left hand) -->
@@ -23,5 +23,5 @@
   <!-- eli (deprecated) is true for ellipsoid fingertip or false for standard finger -->
   <xacro:macro name="shadowhand" params="hand_type:='motor' reflect prefix cable_mesh:=False fingers:=all
-          tip_sensors:=${4 * ['std']} mid_sensors:=${4 * ['std']} prox_sensors:=${4 * ['std']} palm_sensor:=std
+          tip_sensors:=std mid_sensors:=std prox_sensors:=std palm_sensor:=std
           extra_lite:=^|${None} muscletrans:=^|${None} muscle:=^|${None} bio:=^|${None} bt_sp:=^|${None} eli:=^|${None}">
     <!-- Unify hand type parameter, also handling deprecated muscletrans, muscle -->

File: sr_description/hand/xacro/th_ff_rf_ellipsoid_hand.urdf.xacro (robot description, xacro)
@@ -9,8 +9,6 @@
   <xacro:macro name="shadowhand" params="muscletrans muscle bio bt_sp eli reflect prefix">
     ${xacro.warning("The file th_ff_rf_ellipsoid_hand.urdf.xacro is deprecated", print_location=False)}
-    ${xacro.warning("Use full_hand.urdf.xacro instead with tip_sensors=dict([(f, 'eli') for f in 'th ff rf'.split()])")}
-    <!-- Ensure tip_sensors is defined before usage below -->
-    <xacro:property name="tip_sensors" default="${5 * ['std']}" />
-    <!-- translate old parameters to new ones, eventually updating tip_sensors -->
+    ${xacro.warning("Use full_hand.urdf.xacro instead with tip_sensors='th=eli ff=eli rf=eli'")}
+    <!-- translate old parameters to new ones, eventually initializing tip_sensors -->
     <xacro:include filename="$(find sr_description)/hand/xacro/process_sensor_parameters.xacro" />
     <!-- forward to generic macro -->
@@ -18,5 +16,5 @@
     <!-- Enforce ellipsoid sensor on First and Ring Finger as well as Thumb -->
     <xacro:shadowhand fingers="all" reflect="${reflect}" prefix="${prefix}"
-    tip_sensors="${['eli', 'eli', tip_sensors[2], 'eli', tip_sensors[4]]}"/>
+    tip_sensors="${' '.join([k+'='+v for k, v in tip_sensors.items()] + ['ff=eli','rf=eli','th=eli'])}"/>
   </xacro:macro>
 </robot>

File: sr_description/hand/xacro/three_biotac_fingers_hand.urdf.xacro (robot description, xacro)
@@ -9,10 +9,9 @@
   <xacro:macro name="shadowhand" params="muscletrans muscle bio bt_sp eli reflect prefix">
     ${xacro.warning("The file three_biotac_fingers_hand.urdf.xacro is deprecated", print_location=False)}
-    ${xacro.warning("Use full_hand.urdf.xacro instead with tip_sensors=dict([(f, 'bio') for f in 'th ff mf'.split()])")}
+    ${xacro.warning("Use full_hand.urdf.xacro instead with tip_sensors='th=bio ff=bio mf=bio'")}
     <!-- forward to generic macro -->
     <xacro:include filename="$(find sr_description)/hand/xacro/full_hand.urdf.xacro" />
     <!-- BioTacs on First and Middle Finger as well as Thumb -->
-    <xacro:shadowhand reflect="${reflect}" prefix="${prefix}"
-    tip_sensors="${['bio', 'bio', 'bio', 'std', 'std']}"/>
+    <xacro:shadowhand reflect="${reflect}" prefix="${prefix}" tip_sensors="th=bio ff=bio mf=bio" />
   </xacro:macro>
 </robot>

File: sr_description/robots/arm_and_hand_motor_biotac.urdf.xacro (robot description, xacro)
@@ -16,4 +16,4 @@
     <origin xyz="0 0 0" rpy="0 0 ${2.35619449}" />
   </joint>
-  <xacro:shadowhand hand_type="motor" tip_sensors="${['bio','bio','bio','bio','bio']}" reflect="1.0" prefix="rh_" />
+  <xacro:shadowhand hand_type="motor" tip_sensors="bio" reflect="1.0" prefix="rh_" />
 </robot>

File: sr_description/robots/arm_and_hand_motor_ellipsoid.urdf.xacro (robot description, xacro)
@@ -16,4 +16,4 @@
     <origin xyz="0 0 0" rpy="0 0 ${2.35619449}" />
   </joint>
-  <xacro:shadowhand hand_type="motor" tip_sensors="${['eli','eli','eli','eli','eli']}" reflect="1.0" prefix="rh_" />
+  <xacro:shadowhand hand_type="motor" tip_sensors="eli" reflect="1.0" prefix="rh_" />
 </robot>

File: sr_description/robots/arm_and_hand_muscle_biotac.urdf.xacro (robot description, xacro)
@@ -16,4 +16,4 @@
     <origin xyz="0 0 0" rpy="0 0 ${pi}" />
   </joint>
-  <xacro:shadowhand hand_type="muscle" tip_sensors="${['bio','bio','bio','bio','bio']}" reflect="1.0" prefix="rh_" />
+  <xacro:shadowhand hand_type="muscle" tip_sensors="bio" reflect="1.0" prefix="rh_" />
 </robot>

File: sr_description/robots/bimanual_shadowhand_lite_btsp.urdf.xacro (robot description, xacro)
@@ -11,5 +11,5 @@
     <origin xyz="0.0 0.0 0.0" rpy="0.0 0.0 0.0" />
   </joint>
-  <xacro:shadowhand hand_type="motor" tip_sensors="${5 * ['bt_sp']}" reflect="1.0" prefix="rh_" />
+  <xacro:shadowhand hand_type="motor" tip_sensors="bt_sp" reflect="1.0" prefix="rh_" />
   <joint name="right_hand_to_left_hand" type="fixed">
     <parent link="rh_forearm" />
@@ -17,4 +17,4 @@
     <origin xyz="$(arg arm_x_separation) 0.0 0.0" rpy="0.0 0.0 0.0" />
   </joint>
-  <xacro:shadowhand hand_type="motor" tip_sensors="${5 * ['bt_sp']}" reflect="-1.0" prefix="lh_" />
+  <xacro:shadowhand hand_type="motor" tip_sensors="bt_sp" reflect="-1.0" prefix="lh_" />
 </robot>

File: sr_description/robots/bimanual_shadowhand_lite_right_btsp.urdf.xacro (robot description, xacro)
@@ -11,5 +11,5 @@
     <origin xyz="0.0 0.0 0.0" rpy="0.0 0.0 0.0" />
   </joint>
-  <xacro:shadowhand hand_type="motor" tip_sensors="${['bt_sp','bt_sp','bt_sp','bt_sp','bt_sp']}" reflect="1.0" prefix="rh_" />
+  <xacro:shadowhand hand_type="motor" tip_sensors="bt_sp" reflect="1.0" prefix="rh_" />
   <joint name="right_hand_to_left_hand" type="fixed">
     <parent link="rh_forearm" />

File: sr_description/robots/bimanual_shadowhand_motor_plus_right_biotac.urdf.xacro (robot description, xacro)
@@ -10,5 +10,5 @@
     <origin xyz="0.0 0.0 0.0" rpy="0.0 0.0 0.0" />
   </joint>
-  <xacro:shadowhand hand_type="motor+" tip_sensors="${['bt_sp','bt_sp','bt_sp','bt_sp','bt_sp']}" reflect="1.0" prefix="rh_" />
+  <xacro:shadowhand hand_type="motor+" tip_sensors="bt_sp" reflect="1.0" prefix="rh_" />
   <joint name="right_hand_to_left_hand" type="fixed">
     <parent link="rh_forearm" />

File: sr_description/robots/shadowhand_edc_muscle_biotac.urdf.xacro (robot description, xacro)
@@ -17,5 +17,5 @@
   (C) 2012 fnh, hendrich@informatik.uni-hamburg.de
 -->
-  <xacro:shadowhand hand_type="muscletrans" tip_sensors="${['bio','bio','bio','bio','bio']}" reflect="1.0" prefix="rh_" />
+  <xacro:shadowhand hand_type="muscletrans" tip_sensors="bio" reflect="1.0" prefix="rh_" />
   <link name="rh_forearm_disk">
     <inertial>

File: sr_description/robots/shadowhand_left_lite_btsp.urdf.xacro (robot description, xacro)
@@ -14,4 +14,4 @@
     <origin xyz="0.0 0.0 0.0" rpy="0.0 0.0 0.0" />
   </joint>
-  <xacro:shadowhand hand_type="motor" tip_sensors="${['bt_sp','bt_sp','bt_sp','bt_sp']}" reflect="-1.0" prefix="lh_" />
+  <xacro:shadowhand hand_type="motor" tip_sensors="bt_sp" reflect="-1.0" prefix="lh_" />
 </robot>

File: sr_description/robots/shadowhand_left_motor_biotac.urdf.xacro (robot description, xacro)
@@ -14,4 +14,4 @@
     <origin xyz="0.0 0.0 0.0" rpy="0.0 0.0 0.0" />
   </joint>
-  <xacro:shadowhand hand_type="motor" tip_sensors="${['bio','bio','bio','bio','bio']}" reflect="-1.0" prefix="lh_" />
+  <xacro:shadowhand hand_type="motor" tip_sensors="bio" reflect="-1.0" prefix="lh_" />
 </robot>

File: sr_description/robots/shadowhand_left_motor_plus_btsp.urdf.xacro (robot description, xacro)
@@ -14,4 +14,4 @@
       <origin xyz="0.0 0.0 0.0" rpy="0.0 0.0 0.0" />
     </joint>
-  <xacro:shadowhand hand_type="motor+" tip_sensors="${['bt_sp','bt_sp','bt_sp','bt_sp','bt_sp']}" reflect="-1.0" prefix="lh_" />
+  <xacro:shadowhand hand_type="motor+" tip_sensors="bt_sp" reflect="-1.0" prefix="lh_" />
 </robot>

File: sr_description/robots/shadowhand_lite_btsp.urdf.xacro (robot description, xacro)
@@ -14,4 +14,4 @@
     <origin xyz="0.0 0.0 0.0" rpy="0.0 0.0 0.0" />
   </joint>
-  <xacro:shadowhand hand_type="motor" tip_sensors="${['bt_sp','bt_sp','bt_sp','bt_sp']}" reflect="1.0" prefix="rh_" />
+  <xacro:shadowhand hand_type="motor" tip_sensors="bt_sp" reflect="1.0" prefix="rh_" />
 </robot>

File: sr_description/robots/shadowhand_motor_biotac.urdf.xacro (robot description, xacro)
@@ -14,7 +14,4 @@
     <origin xyz="0.0 0.0 0.0" rpy="0.0 0.0 0.0" />
   </joint>
-  <!-- C6 hand with BioTAC sensor
-  (C) 2012 fnh, hendrich@informatik.uni-hamburg.de
--->
-  <xacro:shadowhand hand_type="motor" tip_sensors="${['bio','bio','bio','bio','bio']}" reflect="1.0" prefix="rh_" />
+  <xacro:shadowhand hand_type="motor" tip_sensors="bio" reflect="1.0" prefix="rh_" />
 </robot>

File: sr_description/robots/shadowhand_motor_btsp.urdf.xacro (robot description, xacro)
@@ -14,4 +14,4 @@
     <origin xyz="0.0 0.0 0.0" rpy="0.0 0.0 0.0" />
   </joint>
-  <xacro:shadowhand hand_type="motor" tip_sensors="${['bt_sp','bt_sp','bt_sp','bt_sp','bt_sp']}" reflect="1.0" prefix="rh_" />
+  <xacro:shadowhand hand_type="motor" tip_sensors="bt_sp" reflect="1.0" prefix="rh_" />
 </robot>

File: sr_description/robots/shadowhand_motor_ellipsoid.urdf.xacro (robot description, xacro)
@@ -14,4 +14,4 @@
     <origin xyz="0.0 0.0 0.0" rpy="0.0 0.0 0.0" />
   </joint>
-  <xacro:shadowhand hand_type="motor" tip_sensors="${['eli','eli','eli','eli','eli']}" reflect="1.0" prefix="rh_" />
+  <xacro:shadowhand hand_type="motor" tip_sensors="eli" reflect="1.0" prefix="rh_" />
 </robot>

File: sr_description/robots/shadowhand_motor_ff_biotac.urdf.xacro (robot description, xacro)
@@ -14,4 +14,4 @@
       <origin xyz="0.0 0.0 0.0" rpy="0.0 0.0 0.0" />
     </joint>
-  <xacro:shadowhand hand_type="motor" tip_sensors="${['std','bio','std','std','std']}" reflect="1.0" prefix="rh_" />
+  <xacro:shadowhand hand_type="motor" tip_sensors="ff=bio" reflect="1.0" prefix="rh_" />
 </robot>
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