Commit message: Remove ubi params

File: sr_description/hand/xacro/ff_biotac_hand.urdf.xacro (robot description, xacro)
@@ -12,10 +12,8 @@
   <!-- bio is true for biotac finger or false for standard finger -->
   <!-- bt_sp is true for BT_SP finger or false for standard finger -->
-  <!-- ubi is true for ubi finger or false for standard finger -->
   <!-- eli is true for ellipsoid fingertip or false for standard finger -->
   <!-- reflect is either 1 (for right hand) or -1 (for left hand) -->
   <!-- prefix can be anything but usually is "r_" or  "l_" for right and left hands distinction -->
-  <xacro:macro name="shadowhand"
-  params="muscletrans muscle bio bt_sp ubi eli reflect prefix">
+  <xacro:macro name="shadowhand" params="muscletrans muscle bio bt_sp eli reflect prefix">
     <!-- Forearm -->
     <xacro:forearm muscle="${muscle}" prefix="${prefix}" />
@@ -37,6 +35,5 @@
     reflect="${reflect}" parent="${prefix}wrist" />
     <!-- First Finger Biotac -->
-    <xacro:finger muscletrans="${muscletrans}" lf="false"
-    bio="true" bt_sp="false" ubi="false" eli="false" prefix="${prefix}"
+    <xacro:finger muscletrans="${muscletrans}" lf="false" bio="true" bt_sp="false" eli="false" prefix="${prefix}"
     reflect="${reflect}" link_prefix="ff" joint_prefix="FF"
     parent="${prefix}palm">
@@ -45,6 +42,5 @@
     </xacro:finger>
     <!-- Middle Finger -->
-    <xacro:finger muscletrans="${muscletrans}" lf="false"
-    bio="${bio}" bt_sp="false" ubi="${ubi}" eli="${eli}" prefix="${prefix}"
+    <xacro:finger muscletrans="${muscletrans}" lf="false" bio="${bio}" bt_sp="false" eli="${eli}" prefix="${prefix}"
     reflect="${reflect}" link_prefix="mf" joint_prefix="MF"
     parent="${prefix}palm">
@@ -53,6 +49,5 @@
     </xacro:finger>
     <!-- Ring Finger -->
-    <xacro:finger muscletrans="${muscletrans}" lf="false"
-    bio="${bio}" bt_sp="${bt_sp}" ubi="${ubi}" eli="${eli}" prefix="${prefix}"
+    <xacro:finger muscletrans="${muscletrans}" lf="false" bio="${bio}" bt_sp="${bt_sp}" eli="${eli}" prefix="${prefix}"
     reflect="${reflect}" link_prefix="rf" joint_prefix="RF"
     parent="${prefix}palm">
@@ -61,6 +56,5 @@
     </xacro:finger>
     <!-- Little Finger  -->
-    <xacro:finger muscletrans="${muscletrans}" lf="true"
-    bio="${bio}" bt_sp="${bt_sp}" ubi="${ubi}" eli="${eli}" prefix="${prefix}"
+    <xacro:finger muscletrans="${muscletrans}" lf="true" bio="${bio}" bt_sp="${bt_sp}" eli="${eli}" prefix="${prefix}"
     reflect="${reflect}" link_prefix="lf" joint_prefix="LF"
     parent="${prefix}palm">
@@ -69,6 +63,5 @@
     </xacro:finger>
     <!-- Thumb Biotac -->
-    <xacro:thumb muscletrans="${muscletrans}" bio="${bio}" bt_sp="${bt_sp}"
-    ubi="${ubi}" eli="${eli}" prefix="${prefix}"
+    <xacro:thumb muscletrans="${muscletrans}" bio="${bio}" bt_sp="${bt_sp}" eli="${eli}" prefix="${prefix}"
     reflect="${reflect}" is_lite="0" parent="${prefix}palm">
     </xacro:thumb>

File: sr_description/hand/xacro/finger/distal/distal.urdf.xacro (robot description, xacro)
@@ -11,5 +11,4 @@
   <!-- bio is true for biotac finger or false for standard finger -->
   <!-- bt_sp is true for BT_SP finger or false for standard finger -->
-  <!-- ubi is true for ubi finger or false for standard finger -->
   <!-- eli is true for ellipsoid fingertip or false for standard finger -->
   <!-- prefix can be anything but usually is "r_" or  "l_" for right and left hands distinction -->
@@ -17,6 +16,5 @@
   <!-- joint_prefix prepends fingername to the joint names -->
   <!-- parent is the parent link for the joint -->
-  <xacro:macro name="distal"
-  params="muscle bio bt_sp ubi eli prefix link_prefix joint_prefix parent">
+  <xacro:macro name="distal" params="muscle bio bt_sp eli prefix link_prefix joint_prefix parent">
     <link name="${prefix}${link_prefix}distal">
       <inertial>

File: sr_description/hand/xacro/finger/fingers.urdf.xacro (robot description, xacro)
@@ -10,5 +10,4 @@
   <!-- bio is true for biotac finger or false for standard finger -->
   <!-- bt_sp is true for BT_SP finger or false for standard finger -->
-  <!-- ubi is true for ubi finger or false for standard finger -->
   <!-- eli is true for ellipsoid fingertip or false for standard finger -->
   <!-- reflect is either 1 (for right hand) or -1 (for left hand) -->
@@ -17,6 +16,5 @@
   <!-- joint_prefix prepends fingername to the joint names -->
   <!-- parent is the parent link for the first joint -->
-  <xacro:macro name="finger"
-  params="muscletrans lf bio bt_sp ubi eli reflect prefix link_prefix joint_prefix parent *origin *axis">
+  <xacro:macro name="finger" params="muscletrans lf bio bt_sp eli reflect prefix link_prefix joint_prefix parent *origin *axis">
     <!-- Little finger special case -->
     <xacro:if value="${lf}">
@@ -60,6 +58,5 @@
     <!-- only if finger is not biotac  -->
     <xacro:unless value="${bio}">
-      <xacro:distal muscle="${muscletrans}" bio="${bio}" bt_sp="${bt_sp}"
-      ubi="${ubi}" eli="${eli}" prefix="${prefix}"
+      <xacro:distal muscle="${muscletrans}" bio="${bio}" bt_sp="${bt_sp}" eli="${eli}" prefix="${prefix}"
       link_prefix="${link_prefix}" joint_prefix="${joint_prefix}"
       parent="${prefix}${link_prefix}middle"></xacro:distal>

File: sr_description/hand/xacro/full_hand.urdf.xacro (robot description, xacro)
@@ -12,11 +12,9 @@
   <!-- bio is true for biotac finger or false for standard finger -->
   <!-- bt_sp is true for BT_SP finger or false for standard finger -->
-  <!-- ubi is true for ubi finger or false for standard finger -->
   <!-- eli is true for ellipsoid fingertip or false for standard finger -->
   <!-- reflect is either 1 (for right hand) or -1 (for left hand) -->
   <!-- prefix can be anything but usually is "r_" or  "l_" for right and left hands distinction -->
   <!-- lf is true if we want a little finger, false otherwise -->
-  <xacro:macro name="shadowhand"
-  params="muscletrans muscle hand_type:='hand_e' bio bt_sp ubi eli reflect prefix lf cable_mesh:='false'">
+  <xacro:macro name="shadowhand" params="muscletrans muscle hand_type:='hand_e' bio bt_sp eli reflect prefix lf cable_mesh:='false'">
     <!--xacro:property name="hand_type" value="hand_e"/-->
     <!-- Forearm -->
@@ -39,6 +37,5 @@
     reflect="${reflect}" parent="${prefix}wrist" />
     <!-- First Finger -->
-    <xacro:finger muscletrans="${muscletrans}" lf="false"
-    bio="${bio}" bt_sp="${bt_sp}" ubi="${ubi}" eli="${eli}" prefix="${prefix}"
+    <xacro:finger muscletrans="${muscletrans}" lf="false" bio="${bio}" bt_sp="${bt_sp}" eli="${eli}" prefix="${prefix}"
     reflect="${reflect}" link_prefix="ff" joint_prefix="FF"
     parent="${prefix}palm">
@@ -47,6 +44,5 @@
     </xacro:finger>
     <!-- Middle Finger -->
-    <xacro:finger muscletrans="${muscletrans}" lf="false"
-    bio="${bio}" bt_sp="${bt_sp}" ubi="${ubi}" eli="${eli}" prefix="${prefix}"
+    <xacro:finger muscletrans="${muscletrans}" lf="false" bio="${bio}" bt_sp="${bt_sp}" eli="${eli}" prefix="${prefix}"
     reflect="${reflect}" link_prefix="mf" joint_prefix="MF"
     parent="${prefix}palm">
@@ -55,6 +51,5 @@
     </xacro:finger>
     <!-- Ring Finger -->
-    <xacro:finger muscletrans="${muscletrans}" lf="false"
-    bio="${bio}" bt_sp="${bt_sp}" ubi="${ubi}" eli="${eli}" prefix="${prefix}"
+    <xacro:finger muscletrans="${muscletrans}" lf="false" bio="${bio}" bt_sp="${bt_sp}" eli="${eli}" prefix="${prefix}"
     reflect="${reflect}" link_prefix="rf" joint_prefix="RF"
     parent="${prefix}palm">
@@ -64,6 +59,5 @@
     <!-- Little Finger  -->
     <xacro:if value="${lf}">
-      <xacro:finger muscletrans="${muscletrans}" lf="true"
-      bio="${bio}" bt_sp="${bt_sp}" ubi="${ubi}" eli="${eli}" prefix="${prefix}"
+      <xacro:finger muscletrans="${muscletrans}" lf="true" bio="${bio}" bt_sp="${bt_sp}" eli="${eli}" prefix="${prefix}"
       reflect="${reflect}" link_prefix="lf" joint_prefix="LF"
       parent="${prefix}palm">
@@ -73,6 +67,5 @@
     </xacro:if>
     <!-- Thumb  -->
-    <xacro:thumb muscletrans="${muscletrans}" bio="${bio}" bt_sp="${bt_sp}"
-    ubi="${ubi}" eli="${eli}" prefix="${prefix}"
+    <xacro:thumb muscletrans="${muscletrans}" bio="${bio}" bt_sp="${bt_sp}" eli="${eli}" prefix="${prefix}"
     reflect="${reflect}" is_lite="0" parent="${prefix}palm">
     </xacro:thumb>

File: sr_description/hand/xacro/hand_E_no_mf_rf.urdf.xacro (robot description, xacro)
@@ -12,11 +12,9 @@
   <!-- bio is true for biotac finger or false for standard finger -->
   <!-- bt_sp is true for BT_SP finger or false for standard finger -->
-  <!-- ubi is true for ubi finger or false for standard finger -->
   <!-- eli is true for ellipsoid fingertip or false for standard finger -->
   <!-- reflect is either 1 (for right hand) or -1 (for left hand) -->
   <!-- prefix can be anything but usually is "r_" or  "l_" for right and left hands distinction -->
   <!-- lf is true if we want a little finger, false otherwise -->
-  <xacro:macro name="shadowhand"
-  params="muscletrans muscle bio bt_sp ubi eli reflect prefix lf">
+  <xacro:macro name="shadowhand" params="muscletrans muscle bio bt_sp eli reflect prefix lf">
     <!-- Forearm -->
     <xacro:forearm muscle="${muscle}" prefix="${prefix}" />
@@ -38,6 +36,5 @@
     reflect="${reflect}" parent="${prefix}wrist" />
     <!-- First Finger -->
-    <xacro:finger muscletrans="${muscletrans}" lf="false"
-    bio="${bio}" bt_sp="${bt_sp}" ubi="${ubi}" eli="${eli}" prefix="${prefix}"
+    <xacro:finger muscletrans="${muscletrans}" lf="false" bio="${bio}" bt_sp="${bt_sp}" eli="${eli}" prefix="${prefix}"
     reflect="${reflect}" link_prefix="ff" joint_prefix="FF"
     parent="${prefix}palm">
@@ -47,6 +44,5 @@
     <!-- Little Finger  -->
     <xacro:if value="${lf}">
-      <xacro:finger muscletrans="${muscletrans}" lf="true"
-      bio="${bio}" bt_sp="${bt_sp}" ubi="${ubi}" eli="${eli}" prefix="${prefix}"
+      <xacro:finger muscletrans="${muscletrans}" lf="true" bio="${bio}" bt_sp="${bt_sp}" eli="${eli}" prefix="${prefix}"
       reflect="${reflect}" link_prefix="lf" joint_prefix="LF"
       parent="${prefix}palm">
@@ -56,6 +52,5 @@
     </xacro:if>
     <!-- Thumb  -->
-    <xacro:thumb muscletrans="${muscletrans}" bio="${bio}" bt_sp="${bt_sp}"
-    ubi="${ubi}" eli="${eli}" prefix="${prefix}"
+    <xacro:thumb muscletrans="${muscletrans}" bio="${bio}" bt_sp="${bt_sp}" eli="${eli}" prefix="${prefix}"
     reflect="${reflect}" is_lite="0" parent="${prefix}palm">
     </xacro:thumb>

File: sr_description/hand/xacro/hand_lite.urdf.xacro (robot description, xacro)
@@ -12,10 +12,8 @@
   <!-- bio is true for biotac finger or false for standard finger -->
   <!-- bt_sp is true for BT_SP finger or false for standard finger -->
-  <!-- ubi is true for ubi finger or false for standard finger -->
   <!-- eli is true for ellipsoid fingertip or false for standard finger -->
   <!-- reflect is either 1 (for right hand) or -1 (for left hand) -->
   <!-- prefix can be anything but usually is "r_" or  "l_" for right and left hands distinction -->
-  <xacro:macro name="shadowhand"
-  params="muscletrans muscle bio bt_sp ubi eli reflect prefix extra_lite  cable_mesh:='false'">
+  <xacro:macro name="shadowhand" params="muscletrans muscle bio bt_sp eli reflect prefix extra_lite  cable_mesh:='false'">
     <!-- Forearm -->
     <xacro:forearm muscle="${muscle}" prefix="${prefix}" cable_mesh="${cable_mesh}"/>
@@ -32,6 +30,5 @@
     reflect="${reflect}" parent="${prefix}wrist" />
     <!-- First Finger -->
-    <xacro:finger muscletrans="${muscletrans}" lf="false"
-    bio="${bio}" bt_sp="${bt_sp}" ubi="${ubi}" eli="${eli}" prefix="${prefix}"
+    <xacro:finger muscletrans="${muscletrans}" lf="false" bio="${bio}" bt_sp="${bt_sp}" eli="${eli}" prefix="${prefix}"
     reflect="${reflect}" link_prefix="ff" joint_prefix="FF"
     parent="${prefix}palm">
@@ -41,6 +38,5 @@
     <!-- Middle Finger -->
     <xacro:unless value="${extra_lite}">
-      <xacro:finger muscletrans="${muscletrans}" lf="false"
-		    bio="${bio}" bt_sp="${bt_sp}" ubi="${ubi}" eli="${eli}" prefix="${prefix}"
+      <xacro:finger muscletrans="${muscletrans}" lf="false" bio="${bio}" bt_sp="${bt_sp}" eli="${eli}" prefix="${prefix}"
 		    reflect="${reflect}" link_prefix="mf" joint_prefix="MF"
 		    parent="${prefix}palm">
@@ -50,6 +46,5 @@
     </xacro:unless>
     <!-- Ring Finger -->
-    <xacro:finger muscletrans="${muscletrans}" lf="false"
-    bio="${bio}" bt_sp="${bt_sp}" ubi="${ubi}" eli="${eli}" prefix="${prefix}"
+    <xacro:finger muscletrans="${muscletrans}" lf="false" bio="${bio}" bt_sp="${bt_sp}" eli="${eli}" prefix="${prefix}"
     reflect="${reflect}" link_prefix="rf" joint_prefix="RF"
     parent="${prefix}palm">
@@ -59,6 +54,5 @@
     <!-- No Little Finger on Lite hand -->
     <!-- Thumb  -->
-    <xacro:thumb muscletrans="${muscletrans}" bio="${bio}" bt_sp="${bt_sp}"
-    ubi="${ubi}" eli="${eli}" prefix="${prefix}"
+    <xacro:thumb muscletrans="${muscletrans}" bio="${bio}" bt_sp="${bt_sp}" eli="${eli}" prefix="${prefix}"
     reflect="${reflect}" is_lite="1" parent="${prefix}palm">
     </xacro:thumb>

File: sr_description/hand/xacro/one_finger_unit.urdf.xacro (robot description, xacro)
@@ -9,10 +9,8 @@
   <!-- bio is true for biotac finger or false for standard finger -->
   <!-- bt_sp is true for BT_SP finger or false for standard finger -->
-  <!-- ubi is true for ubi finger or false for standard finger -->
   <!-- eli is true for ellipsoid fingertip or false for standard finger -->
   <!-- reflect is either 1 (for right hand) or -1 (for left hand) -->
   <!-- prefix can be anything but usually is "r_" or  "l_" for right and left hands distinction -->
-  <xacro:macro name="shadowhand"
-  params="muscletrans muscle bio bt_sp ubi eli reflect prefix">
+  <xacro:macro name="shadowhand" params="muscletrans muscle bio bt_sp eli reflect prefix">
     <!-- Forearm -->
     <xacro:forearm muscle="${muscle}" prefix="${prefix}" />
@@ -48,6 +46,5 @@
     <!-- Middle Finger -->
     <!-- TODO: Check if offset is the same for muscle hand -->
-    <xacro:finger muscletrans="${muscletrans}" lf="false"
-    bio="${bio}" bt_sp="${bt_sp}" ubi="${ubi}" eli="${eli}" prefix="${prefix}"
+    <xacro:finger muscletrans="${muscletrans}" lf="false" bio="${bio}" bt_sp="${bt_sp}" eli="${eli}" prefix="${prefix}"
     reflect="${reflect}" link_prefix="mf" joint_prefix="MF"
     parent="${prefix}palm">

File: sr_description/hand/xacro/th_ff_rf_ellipsoid_hand.urdf.xacro (robot description, xacro)
@@ -12,10 +12,8 @@
   <!-- bio is true for biotac finger or false for standard finger -->
   <!-- bt_sp is true for BT_SP finger or false for standard finger -->
-  <!-- ubi is true for ubi finger or false for standard finger -->
   <!-- eli is true for ellipsoid fingertip or false for standard finger -->
   <!-- reflect is either 1 (for right hand) or -1 (for left hand) -->
   <!-- prefix can be anything but usually is "r_" or  "l_" for right and left hands distinction -->
-  <xacro:macro name="shadowhand"
-  params="muscletrans muscle bio bt_sp ubi eli reflect prefix">
+  <xacro:macro name="shadowhand" params="muscletrans muscle bio bt_sp eli reflect prefix">
     <!-- Forearm -->
     <xacro:forearm muscle="${muscle}" prefix="${prefix}" />
@@ -37,6 +35,5 @@
     reflect="${reflect}" parent="${prefix}wrist" />
     <!-- First Finger Biotac -->
-    <xacro:finger muscletrans="${muscletrans}" lf="false"
-    bio="false" bt_sp="false" ubi="false" eli="true" prefix="${prefix}"
+    <xacro:finger muscletrans="${muscletrans}" lf="false" bio="false" bt_sp="false" eli="true" prefix="${prefix}"
     reflect="${reflect}" link_prefix="ff" joint_prefix="FF"
     parent="${prefix}palm">
@@ -45,6 +42,5 @@
     </xacro:finger>
     <!-- Middle Finger -->
-    <xacro:finger muscletrans="${muscletrans}" lf="false"
-    bio="${bio}" bt_sp="${bt_sp}" ubi="${ubi}" eli="${eli}" prefix="${prefix}"
+    <xacro:finger muscletrans="${muscletrans}" lf="false" bio="${bio}" bt_sp="${bt_sp}" eli="${eli}" prefix="${prefix}"
     reflect="${reflect}" link_prefix="mf" joint_prefix="MF"
     parent="${prefix}palm">
@@ -53,6 +49,5 @@
     </xacro:finger>
     <!-- Ring Finger -->
-    <xacro:finger muscletrans="${muscletrans}" lf="false"
-    bio="false" bt_sp="false" ubi="false" eli="true" prefix="${prefix}"
+    <xacro:finger muscletrans="${muscletrans}" lf="false" bio="false" bt_sp="false" eli="true" prefix="${prefix}"
     reflect="${reflect}" link_prefix="rf" joint_prefix="RF"
     parent="${prefix}palm">
@@ -61,6 +56,5 @@
     </xacro:finger>
     <!-- Little Finger  -->
-    <xacro:finger muscletrans="${muscletrans}" lf="true"
-    bio="${bio}" bt_sp="${bt_sp}" ubi="${ubi}" eli="${eli}" prefix="${prefix}"
+    <xacro:finger muscletrans="${muscletrans}" lf="true" bio="${bio}" bt_sp="${bt_sp}" eli="${eli}" prefix="${prefix}"
     reflect="${reflect}" link_prefix="lf" joint_prefix="LF"
     parent="${prefix}palm">
@@ -69,6 +63,5 @@
     </xacro:finger>
     <!-- Thumb Biotac -->
-    <xacro:thumb muscletrans="${muscletrans}" bio="false" bt_sp="false"
-    ubi="false" eli="true" prefix="${prefix}" reflect="${reflect}"
+    <xacro:thumb muscletrans="${muscletrans}" bio="false" bt_sp="false" eli="true" prefix="${prefix}" reflect="${reflect}"
     is_lite="0" parent="${prefix}palm"></xacro:thumb>
   </xacro:macro>

File: sr_description/hand/xacro/three_biotac_fingers_hand.urdf.xacro (robot description, xacro)
@@ -12,10 +12,8 @@
   <!-- bio is true for biotac finger or false for standard finger -->
   <!-- bt_sp is true for BT_SP finger or false for standard finger -->
-  <!-- ubi is true for ubi finger or false for standard finger -->
   <!-- eli is true for ellipsoid fingertip or false for standard finger -->
   <!-- reflect is either 1 (for right hand) or -1 (for left hand) -->
   <!-- prefix can be anything but usually is "r_" or  "l_" for right and left hands distinction -->
-  <xacro:macro name="shadowhand"
-  params="muscletrans muscle bio bt_sp ubi eli reflect prefix">
+  <xacro:macro name="shadowhand" params="muscletrans muscle bio bt_sp eli reflect prefix">
     <!-- Forearm -->
     <xacro:forearm muscle="${muscle}" prefix="${prefix}" />
@@ -37,6 +35,5 @@
     reflect="${reflect}" parent="${prefix}wrist" />
     <!-- First Finger Biotac -->
-    <xacro:finger muscletrans="${muscletrans}" lf="false"
-    bio="true" bt_sp="false"  ubi="false" eli="false" prefix="${prefix}"
+    <xacro:finger muscletrans="${muscletrans}" lf="false" bio="true" bt_sp="false" eli="false" prefix="${prefix}"
     reflect="${reflect}" link_prefix="ff" joint_prefix="FF"
     parent="${prefix}palm">
@@ -45,6 +42,5 @@
     </xacro:finger>
     <!-- Middle Finger Biotac -->
-    <xacro:finger muscletrans="${muscletrans}" lf="false"
-    bio="true" bt_sp="false" ubi="false" eli="false" prefix="${prefix}"
+    <xacro:finger muscletrans="${muscletrans}" lf="false" bio="true" bt_sp="false" eli="false" prefix="${prefix}"
     reflect="${reflect}" link_prefix="mf" joint_prefix="MF"
     parent="${prefix}palm">
@@ -53,6 +49,5 @@
     </xacro:finger>
     <!-- Ring Finger -->
-    <xacro:finger muscletrans="${muscletrans}" lf="false"
-    bio="false" bt_sp="false" ubi="false" eli="false" prefix="${prefix}"
+    <xacro:finger muscletrans="${muscletrans}" lf="false" bio="false" bt_sp="false" eli="false" prefix="${prefix}"
     reflect="${reflect}" link_prefix="rf" joint_prefix="RF"
     parent="${prefix}palm">
@@ -61,6 +56,5 @@
     </xacro:finger>
     <!-- Little Finger  -->
-    <xacro:finger muscletrans="${muscletrans}" lf="true"
-    bio="false" bt_sp="false" ubi="false" eli="false" prefix="${prefix}"
+    <xacro:finger muscletrans="${muscletrans}" lf="true" bio="false" bt_sp="false" eli="false" prefix="${prefix}"
     reflect="${reflect}" link_prefix="lf" joint_prefix="LF"
     parent="${prefix}palm">
@@ -69,6 +63,5 @@
     </xacro:finger>
     <!-- Thumb Biotac -->
-    <xacro:thumb muscletrans="${muscletrans}" bio="true" bt_sp="false"
-    ubi="false" eli="false" prefix="${prefix}" reflect="${reflect}"
+    <xacro:thumb muscletrans="${muscletrans}" bio="true" bt_sp="false" eli="false" prefix="${prefix}" reflect="${reflect}"
     is_lite="0" parent="${prefix}palm"></xacro:thumb>
   </xacro:macro>

File: sr_description/hand/xacro/three_fingers_hand.urdf.xacro (robot description, xacro)
@@ -12,10 +12,8 @@
   <!-- bio is true for biotac finger or false for standard finger -->
   <!-- bt_sp is true for BT_SP finger or false for standard finger -->
-  <!-- ubi is true for ubi finger or false for standard finger -->
   <!-- eli is true for ellipsoid fingertip or false for standard finger -->
   <!-- reflect is either 1 (for right hand) or -1 (for left hand) -->
   <!-- prefix can be anything but usually is "r_" or  "l_" for right and left hands distinction -->
-  <xacro:macro name="shadowhand"
-  params="muscletrans muscle bio bt_sp ubi eli reflect prefix">
+  <xacro:macro name="shadowhand" params="muscletrans muscle bio bt_sp eli reflect prefix">
     <!-- Forearm -->
     <xacro:forearm muscle="${muscle}" prefix="${prefix}" />
@@ -37,6 +35,5 @@
     reflect="${reflect}" parent="${prefix}wrist" />
     <!-- First Finger -->
-    <xacro:finger muscletrans="${muscletrans}" lf="false"
-    bio="${bio}" bt_sp="${bt_sp}" ubi="${ubi}" eli="${eli}" prefix="${prefix}"
+    <xacro:finger muscletrans="${muscletrans}" lf="false" bio="${bio}" bt_sp="${bt_sp}" eli="${eli}" prefix="${prefix}"
     reflect="${reflect}" link_prefix="ff" joint_prefix="FF"
     parent="${prefix}palm">
@@ -45,6 +42,5 @@
     </xacro:finger>
     <!-- Middle Finger -->
-    <xacro:finger muscletrans="${muscletrans}" lf="false"
-    bio="${bio}" bt_sp="${bt_sp}" ubi="${ubi}" eli="${eli}" prefix="${prefix}"
+    <xacro:finger muscletrans="${muscletrans}" lf="false" bio="${bio}" bt_sp="${bt_sp}" eli="${eli}" prefix="${prefix}"
     reflect="${reflect}" link_prefix="mf" joint_prefix="MF"
     parent="${prefix}palm">
@@ -53,6 +49,5 @@
     </xacro:finger>
     <!-- Thumb  -->
-    <xacro:thumb muscletrans="${muscletrans}" bio="${bio}" bt_sp="${bt_sp}"
-    ubi="${ubi}" eli="${eli}" prefix="${prefix}"
+    <xacro:thumb muscletrans="${muscletrans}" bio="${bio}" bt_sp="${bt_sp}" eli="${eli}" prefix="${prefix}"
     reflect="${reflect}" is_lite="0" parent="${prefix}palm">
     </xacro:thumb>
