Commit message: Remove ubi params

File: sr_description/hand/xacro/three_fingers_hand_RF.urdf.xacro (robot description, xacro)
@@ -12,10 +12,8 @@
   <!-- bio is true for biotac finger or false for standard finger -->
   <!-- bt_sp is true for BT_SP finger or false for standard finger -->
-  <!-- ubi is true for ubi finger or false for standard finger -->
   <!-- eli is true for ellipsoid fingertip or false for standard finger -->
   <!-- reflect is either 1 (for right hand) or -1 (for left hand) -->
   <!-- prefix can be anything but usually is "r_" or  "l_" for right and left hands distinction -->
-  <xacro:macro name="shadowhand"
-  params="muscletrans muscle bio bt_sp ubi eli reflect prefix">
+  <xacro:macro name="shadowhand" params="muscletrans muscle bio bt_sp eli reflect prefix">
     <!-- Forearm -->
     <xacro:forearm muscle="${muscle}" prefix="${prefix}" />
@@ -37,6 +35,5 @@
     reflect="${reflect}" parent="${prefix}wrist" />
     <!-- First Finger -->
-    <xacro:finger muscletrans="${muscletrans}" lf="false"
-    bio="${bio}" bt_sp="${bt_sp}" ubi="${ubi}" eli="${eli}" prefix="${prefix}"
+    <xacro:finger muscletrans="${muscletrans}" lf="false" bio="${bio}" bt_sp="${bt_sp}" eli="${eli}" prefix="${prefix}"
     reflect="${reflect}" link_prefix="ff" joint_prefix="FF"
     parent="${prefix}palm">
@@ -45,6 +42,5 @@
     </xacro:finger>
     <!-- Ring Finger -->
-    <xacro:finger muscletrans="${muscletrans}" lf="false"
-    bio="${bio}" bt_sp="${bt_sp}" ubi="${ubi}" eli="${eli}" prefix="${prefix}"
+    <xacro:finger muscletrans="${muscletrans}" lf="false" bio="${bio}" bt_sp="${bt_sp}" eli="${eli}" prefix="${prefix}"
     reflect="${reflect}" link_prefix="rf" joint_prefix="RF"
     parent="${prefix}palm">
@@ -53,6 +49,5 @@
     </xacro:finger>
     <!-- Thumb  -->
-    <xacro:thumb muscletrans="${muscletrans}" bio="${bio}" bt_sp="${bt_sp}"
-    ubi="${ubi}" eli="${eli}" prefix="${prefix}"
+    <xacro:thumb muscletrans="${muscletrans}" bio="${bio}" bt_sp="${bt_sp}" eli="${eli}" prefix="${prefix}"
     reflect="${reflect}" is_lite="0" parent="${prefix}palm">
     </xacro:thumb>

File: sr_description/hand/xacro/thumb/thdistal.urdf.xacro (robot description, xacro)
@@ -11,10 +11,8 @@
   <!-- bio is true for biotac finger or false for standard finger -->
   <!-- bt_sp is true for BT_SP finger or false for standard finger -->
-  <!-- ubi is true for ubi finger or false for standard finger -->
   <!-- eli is true for ellipsoid fingertip or false for standard finger -->
   <!-- prefix can be anything but usually is "r_" or  "l_" for right and left hands distinction -->
   <!-- parent is the parent link for the first joint -->
-  <xacro:macro name="thdistal"
-  params="muscle bio bt_sp ubi eli prefix parent">
+  <xacro:macro name="thdistal" params="muscle bio bt_sp eli prefix parent">
     <xacro:if value="${bio}">
       <!--    BIOTAC -->

File: sr_description/hand/xacro/thumb/thumb.urdf.xacro (robot description, xacro)
@@ -8,5 +8,4 @@
   <!-- bio is true for biotac finger or false for standard finger -->
   <!-- bt_sp is true for BT_SP finger or false for standard finger -->
-  <!-- ubi is true for ubi finger or false for standard finger -->
   <!-- eli is true for ellipsoid fingertip or false for standard finger -->
   <!-- reflect is either 1 (for right hand) or -1 (for left hand) -->
@@ -14,6 +13,5 @@
   <!-- parent is the parent link for the first joint -->
   <!-- is_lite is this the lite hand, if so lock J3 -->
-  <xacro:macro name="thumb"
-  params="muscletrans bio bt_sp ubi eli reflect prefix parent is_lite">
+  <xacro:macro name="thumb" params="muscletrans bio bt_sp eli reflect prefix parent is_lite">
     <!-- Base -->
     <xacro:thbase muscle="${muscletrans}" prefix="${prefix}"
@@ -31,6 +29,5 @@
     prefix="${prefix}" parent="${prefix}thhub"></xacro:thmiddle>
     <!-- Distal -->
-    <xacro:thdistal muscle="${muscletrans}" bio="${bio}" bt_sp="${bt_sp}"
-    ubi="${ubi}" eli="${eli}" prefix="${prefix}"
+    <xacro:thdistal muscle="${muscletrans}" bio="${bio}" bt_sp="${bt_sp}" eli="${eli}" prefix="${prefix}"
     parent="${prefix}thmiddle"></xacro:thdistal>
   </xacro:macro>

File: sr_description/robots/arm_and_hand_motor.urdf.xacro (robot description, xacro)
@@ -16,5 +16,4 @@
     <origin xyz="0 0 0" rpy="0 0 ${2.35619449}" />
   </joint>
-  <xacro:shadowhand muscletrans="false" muscle="false" bio="false" bt_sp="false"
-  ubi="false" eli="false" reflect="1.0" prefix="rh_" lf="true" />
+  <xacro:shadowhand muscletrans="false" muscle="false" bio="false" bt_sp="false" eli="false" reflect="1.0" prefix="rh_" lf="true" />
 </robot>

File: sr_description/robots/arm_and_hand_motor_biotac.urdf.xacro (robot description, xacro)
@@ -16,5 +16,4 @@
     <origin xyz="0 0 0" rpy="0 0 ${2.35619449}" />
   </joint>
-  <xacro:shadowhand muscletrans="false" muscle="false" bio="true" bt_sp="false"
-  ubi="false" eli="false" reflect="1.0" prefix="rh_" lf="true" />
+  <xacro:shadowhand muscletrans="false" muscle="false" bio="true" bt_sp="false" eli="false" reflect="1.0" prefix="rh_" lf="true" />
 </robot>

File: sr_description/robots/arm_and_hand_motor_ellipsoid.urdf.xacro (robot description, xacro)
@@ -16,5 +16,4 @@
     <origin xyz="0 0 0" rpy="0 0 ${2.35619449}" />
   </joint>
-  <xacro:shadowhand muscletrans="false" muscle="false" bio="false" bt_sp="false"
-  ubi="false" eli="true" reflect="1.0" prefix="rh_" lf="true" />
+  <xacro:shadowhand muscletrans="false" muscle="false" bio="false" bt_sp="false" eli="true" reflect="1.0" prefix="rh_" lf="true" />
 </robot>

File: sr_description/robots/arm_and_hand_motor_three_finger.urdf.xacro (robot description, xacro)
@@ -16,5 +16,4 @@
     <origin xyz="0 0 0" rpy="0 0 ${2.35619449}" />
   </joint>
-  <xacro:shadowhand muscletrans="false" muscle="false" bio="false" bt_sp="false"
-  ubi="false" eli="false" reflect="1.0" prefix="rh_" />
+  <xacro:shadowhand muscletrans="false" muscle="false" bio="false" bt_sp="false" eli="false" reflect="1.0" prefix="rh_" />
 </robot>

File: sr_description/robots/arm_and_hand_muscle.urdf.xacro (robot description, xacro)
@@ -16,5 +16,4 @@
     <origin xyz="0 0 0" rpy="0 0 ${pi}" />
   </joint>
-  <xacro:shadowhand muscletrans="false" muscle="true" bio="false" bt_sp="false"
-  ubi="false" eli="false" reflect="1.0" prefix="rh_" lf="true" />
+  <xacro:shadowhand muscletrans="false" muscle="true" bio="false" bt_sp="false" eli="false" reflect="1.0" prefix="rh_" lf="true" />
 </robot>

File: sr_description/robots/arm_and_hand_muscle_biotac.urdf.xacro (robot description, xacro)
@@ -16,5 +16,4 @@
     <origin xyz="0 0 0" rpy="0 0 ${pi}" />
   </joint>
-  <xacro:shadowhand muscletrans="false" muscle="true" bio="true" bt_sp="false"
-  ubi="false" eli="false" reflect="1.0" prefix="rh_" lf="true" />
+  <xacro:shadowhand muscletrans="false" muscle="true" bio="true" bt_sp="false" eli="false" reflect="1.0" prefix="rh_" lf="true" />
 </robot>

File: sr_description/robots/arm_and_sr_one_finger_motor.urdf.xacro (robot description, xacro)
@@ -19,5 +19,4 @@
     <dynamics damping="3.5" />
   </joint>
-  <xacro:shadowhand muscletrans="false" muscle="false" bio="false" bt_sp="false"
-  ubi="false" eli="false" reflect="1.0" prefix="rh_" />
+  <xacro:shadowhand muscletrans="false" muscle="false" bio="false" bt_sp="false" eli="false" reflect="1.0" prefix="rh_" />
 </robot>
