Commit message: hand e working with versions and hand type

File: sr_description/hand/xacro/ff_biotac_hand.urdf.xacro (robot description, xacro)
@@ -9,5 +9,5 @@
   <xacro:macro name="shadowhand" params="muscletrans muscle bio bt_sp eli reflect prefix">
     ${xacro.warning("The file ff_biotac_hand.urdf.xacro is deprecated", print_location=False)}
-    ${xacro.warning("Use full_hand.urdf.xacro instead with tip_sensors='ff=bio'")}
+    ${xacro.warning("Use full_hand.urdf.xacro instead with tip_sensors='ff=bt_2p'")}
     <!-- translate old parameters to new ones, eventually initializing tip_sensors -->
     <xacro:include filename="$(find sr_description)/hand/xacro/process_sensor_parameters.xacro" />
@@ -16,5 +16,5 @@
     <!-- Enforce BioTac on First Finger -->
     <xacro:shadowhand fingers="all" reflect="${reflect}" prefix="${prefix}"
-    tip_sensors="${' '.join([k+'='+v for k, v in tip_sensors.items()] + ['ff=bio'])}"/>
+    tip_sensors="${' '.join([k+'='+v for k, v in tip_sensors.items()] + ['ff=bt_2p'])}"/>
   </xacro:macro>
 </robot>

File: sr_description/hand/xacro/finger/distal/distal.urdf.xacro (robot description, xacro)
@@ -8,5 +8,5 @@
   <xacro:include filename="$(find sr_description)/hand/xacro/finger/distal/distal.gazebo.xacro" />
   <xacro:include filename="$(find sr_description)/hand/xacro/finger/distal/distal.transmission.xacro" />
-  <!-- tip_sensor describes the sensor std, none, bio, bt_sp, eli -->
+  <!-- tip_sensor describes the sensor none, bt_2p, bt_sp, eli -->
   <!-- prefix can be anything but usually is "r_" or  "l_" for right and left hands distinction -->
   <!-- link_prefix prepends fingername to the link names -->
@@ -69,5 +69,5 @@
       </collision>
     </link>
-    <xacro:unless value="${tip_sensor == 'bio'}">
+    <xacro:unless value="${tip_sensor == 'bt_2p'}">
       <joint name="${prefix}${joint_prefix}J1" type="revolute">
         <parent link="${parent}" />

File: sr_description/hand/xacro/finger/fingers.urdf.xacro (robot description, xacro)
@@ -7,6 +7,6 @@
   <xacro:include filename="$(find sr_description)/hand/xacro/finger/biotac/biotac.urdf.xacro" />
   <!-- lf is true for little finger or false for standard finger -->
-  <!-- tip_sensor describes the sensor none, bio, bt_sp, eli -->
-  <!-- mid_sensor describes the sensor none, bio -->
+  <!-- tip_sensor describes the sensor none, bt_2p, bt_sp, eli -->
+  <!-- mid_sensor describes the sensor none, bt_2p -->
   <!-- prox_sensor describes the sensor none, standard -->
   <!-- reflect is either 1 (for right hand) or -1 (for left hand) -->
@@ -35,10 +35,10 @@
     <xacro:proximal parent="${prefix}${link_prefix}knuckle"></xacro:proximal>
     <!-- BioTac combines Middle + Distal -->
-    <xacro:if value="${tip_sensor == 'bio'}">
+    <xacro:if value="${tip_sensor == 'bt_2p'}">
       <xacro:biotac_middle parent="${prefix}${link_prefix}proximal">
       </xacro:biotac_middle>
     </xacro:if>
     <!-- Non-BioTac -->
-    <xacro:unless value="${tip_sensor == 'bio'}">
+    <xacro:unless value="${tip_sensor == 'bt_2p'}">
       <!-- Middle -->
       <xacro:middle parent="${prefix}${link_prefix}proximal"></xacro:middle>

File: sr_description/hand/xacro/finger/lfmetacarpal/lfmetacarpal.gazebo.xacro (robot description, xacro)
@@ -1,5 +1,5 @@
 <?xml version="1.0"?>
 <robot xmlns:xacro="http://www.ros.org/wiki/xacro">
-  <xacro:macro name="lfmetacarpal_gazebo" params="prefix:=^ palm_sensor:=^|std link_prefix">
+  <xacro:macro name="lfmetacarpal_gazebo" params="prefix:=^ palm_sensor:=^|none link_prefix">
     <!-- prefix can be anything but usually is "r_" or  "l_" for right and left hands distinction -->
     <gazebo reference="${prefix}lfmetacarpal">

File: sr_description/hand/xacro/finger/proximal/proximal.gazebo.xacro (robot description, xacro)
@@ -1,5 +1,5 @@
 <?xml version="1.0"?>
 <robot xmlns:xacro="http://www.ros.org/wiki/xacro">
-  <xacro:macro name="proximal_gazebo" params="prefix:=^ link_prefix:=^ prox_sensor:=^|std">
+  <xacro:macro name="proximal_gazebo" params="prefix:=^ link_prefix:=^ prox_sensor:=^|none">
     <!-- prefix can be anything but usually is "r_" or  "l_" for right and left hands distinction -->
     <gazebo reference="${prefix}${link_prefix}proximal">

File: sr_description/hand/xacro/full_hand.urdf.xacro (robot description, xacro)
@@ -1,11 +1,14 @@
-<robot xmlns:sensor="http://playerstage.sourceforge.net/gazebo/xmlschema/#sensor" xmlns:controller="http://playerstage.sourceforge.net/gazebo/xmlschema/#controller" xmlns:interface="http://playerstage.sourceforge.net/gazebo/xmlschema/#interface" xmlns:xacro="http://www.ros.org/wiki/xacro">
-  <xacro:include filename="$(find sr_description)/hand/xacro/forearm/forearm.urdf.xacro" />
+<robot xmlns:sensor="http://playerstage.sourceforge.net/gazebo/xmlschema/#sensor"
+       xmlns:controller="http://playerstage.sourceforge.net/gazebo/xmlschema/#controller"
+       xmlns:interface="http://playerstage.sourceforge.net/gazebo/xmlschema/#interface"
+       xmlns:xacro="http://www.ros.org/wiki/xacro">
+  <xacro:include filename="forearm_e.urdf.xacro" />
   <xacro:include filename="$(find sr_description)/hand/xacro/wrist/wrist.urdf.xacro" />
   <xacro:include filename="$(find sr_description)/hand/xacro/palm/palm.urdf.xacro" />
   <xacro:include filename="$(find sr_description)/hand/xacro/finger/fingers.urdf.xacro" />
   <xacro:include filename="$(find sr_description)/hand/xacro/thumb/thumb.urdf.xacro" />
-  <!-- hand_type can be: motor, motor+, muscle (muscle), muscletrans (muscletrans) -->
+  <!-- hand_type can be: E, G, muscle (muscle), muscletrans (muscletrans) -->
   <!-- fingers: list-like string specifying available fingers, default: 'th ff mf rf lf' -->
-  <!-- tip_sensors: plain or dict-like string specifying the fingertip (tactile) sensors: 'th=bio ff=bt_sp mf=eli rf=std, lf=none' -->
+  <!-- tip_sensors: plain or dict-like string specifying the fingertip (tactile) sensors: 'th=bt_2p ff=bt_sp mf=eli rf=none, lf=none' -->
   <!-- mid_sensors: plain or dict-like string specifying the middle-phalange (tactile) sensors -->
   <!-- prox_sensors: plain or dict-like string specifying the proximal (tactile) sensors -->
@@ -20,5 +23,5 @@
   <!-- lf (deprecated) is true if we want a little finger, false otherwise -->
   <xacro:macro name="shadowhand" params="hand_type:='motor' reflect prefix cable_mesh:=False fingers:=all
-          tip_sensors:=std mid_sensors:=std prox_sensors:=std palm_sensor:=std
+          tip_sensors:=pst mid_sensors:=none prox_sensors:=none palm_sensor:=none
           muscletrans:=^|${None} muscle:=^|${None} lf:=^|${None} bio:=^|${None} bt_sp:=^|${None} eli:=^|${None}">
     <!-- Unify hand type parameter, also handling deprecated muscletrans, muscle -->

File: sr_description/hand/xacro/hand_lite.urdf.xacro (robot description, xacro)
@@ -10,8 +10,8 @@
   <!-- hand_type can be: motor, motor+, muscle (muscle), muscletrans (muscletrans) -->
   <!-- fingers: list-like string specifying available fingers, default: 'th ff mf rf' -->
-  <!-- tip_sensors: plain or dict-like string specifying the fingertip (tactile) sensors: 'th=bio ff=bt_sp mf=eli rf=std, lf=none' -->
+  <!-- tip_sensors: plain or dict-like string specifying the fingertip (tactile) sensors: 'th=bt_2p ff=bt_sp mf=eli rf=none, lf=none' -->
   <!-- mid_sensors: plain or dict-like string specifying the middle-phalange (tactile) sensors -->
   <!-- prox_sensors: plain or dict-like string specifying the proximal (tactile) sensors -->
-  <!-- palm_sensor: specifies the palm tactile sensor: std, none -->
+  <!-- palm_sensor: specifies the palm tactile sensor: none -->
   <!-- reflect is either 1 (for right hand) or -1 (for left hand) -->
   <!-- prefix can be anything but usually is "r_" or  "l_" for right and left hands distinction -->
@@ -23,5 +23,5 @@
   <!-- eli (deprecated) is true for ellipsoid fingertip or false for standard finger -->
   <xacro:macro name="shadowhand" params="hand_type:='motor' reflect prefix cable_mesh:=False fingers:=all
-          tip_sensors:=std mid_sensors:=std prox_sensors:=std palm_sensor:=std
+          tip_sensors:=pst mid_sensors:=none prox_sensors:=none palm_sensor:=none
           extra_lite:=^|${None} muscletrans:=^|${None} muscle:=^|${None} bio:=^|${None} bt_sp:=^|${None} eli:=^|${None}">
     <!-- Unify hand type parameter, also handling deprecated muscletrans, muscle -->

File: sr_description/hand/xacro/one_finger_unit.urdf.xacro (robot description, xacro)
@@ -3,5 +3,5 @@
 xmlns:interface="http://playerstage.sourceforge.net/gazebo/xmlschema/#interface"
 xmlns:xacro="http://www.ros.org/wiki/xacro">
-  <xacro:include filename="$(find sr_description)/hand/xacro/forearm/forearm.urdf.xacro" />
+  <xacro:include filename="forearm_e.urdf.xacro" />
   <xacro:include filename="$(find sr_description)/hand/xacro/finger/fingers.urdf.xacro" />
   <!-- hand_type describes the hand type, motor, motor+, muscle (muscle) -->
@@ -12,6 +12,6 @@
   <!-- bt_sp (deprecated) is true for BT_SP finger or false for standard finger -->
   <!-- eli (deprecated) is true for ellipsoid fingertip or false for standard finger -->
-  <!-- tip_sensor describes the sensor none, bio, bt_sp, eli -->
-  <!-- mid_sensor describes the sensor none, bio -->
+  <!-- tip_sensor describes the sensor none, bt_2p, bt_sp, eli -->
+  <!-- mid_sensor describes the sensor none, bt_2p -->
   <!-- prox_sensor describes the sensor none, bumper -->
   <!-- palm_sensor describes the sensor none, bumper -->

File: sr_description/hand/xacro/palm/palm.urdf.xacro (robot description, xacro)
@@ -12,18 +12,15 @@
   <!-- reflect is either 1 (for right hand) or -1 (for left hand) -->
   <!-- parent is the parent link for the joint -->
-  <xacro:macro name="palm"
-  params="prefix:=^ reflect:=^ parent">
+  <xacro:macro name="palm" params="prefix:=^ reflect:=^ parent">
     <link name="${prefix}palm">
       <inertial>
         <origin xyz="0 0 0.035" rpy="0 0 0" />
         <mass value="0.3" />
-        <inertia ixx="0.0003581" ixy="0.0" ixz="0.0"
-        iyy="0.0005287" iyz="0.0" izz="0.000191" />
+        <inertia ixx="0.0003581" ixy="0.0" ixz="0.0" iyy="0.0005287" iyz="0.0" izz="0.000191" />
       </inertial>
       <visual>
         <origin xyz="0 0 0" rpy="0 0 0" />
         <geometry name="${prefix}palm_visual">
-          <mesh filename="package://sr_description/meshes/hand/palm.dae"
-          scale="${reflect*0.001} 0.001 0.001" />
+          <mesh filename="package://sr_description/meshes/hand/palm.dae" scale="${reflect*0.001} 0.001 0.001" />
         </geometry>
         <material name="Grey" />
@@ -36,6 +33,5 @@
       </collision>
       <collision>
-        <origin xyz="${-reflect*0.002} -0.0035 0.038"
-        rpy="0 0 0" />
+        <origin xyz="${-reflect*0.002} -0.0035 0.038" rpy="0 0 0" />
         <geometry>
           <box size="0.036 0.017 0.098" />
@@ -44,6 +40,5 @@
       <!-- palm complement below first finger -->
       <collision>
-        <origin xyz="${reflect*0.029} -0.0035 0.082"
-        rpy="0 0 0" />
+        <origin xyz="${reflect*0.029} -0.0035 0.082" rpy="0 0 0" />
         <geometry>
           <box size="0.026 0.017 0.010" />
@@ -51,6 +46,5 @@
       </collision>
       <collision>
-        <origin xyz="${reflect*0.0265} -0.001 0.070"
-        rpy="0.2 0 ${reflect*0.25}" />
+        <origin xyz="${reflect*0.0265} -0.001 0.070" rpy="0.2 0 ${reflect*0.25}" />
         <geometry>
           <box size="0.026 0.014 0.018" />
@@ -59,6 +53,5 @@
       <!-- thumb pulp side -->
       <collision>
-        <origin xyz="${reflect*0.0315} -0.0085 0.001"
-        rpy="0 0 0" />
+        <origin xyz="${reflect*0.0315} -0.0085 0.001" rpy="0 0 0" />
         <geometry>
           <box size="0.021 0.027 0.024" />
@@ -98,6 +91,5 @@
       <origin xyz="0 0 0.034" rpy="0 0 0" />
       <axis xyz="1 0 0" />
-      <limit lower="${-40/180*pi}" upper="${28/180*pi}"
-      effort="30" velocity="2.0" />
+      <limit lower="${-40/180*pi}" upper="${28/180*pi}" effort="30" velocity="2.0" />
       <dynamics damping="0.1" />
     </joint>

File: sr_description/hand/xacro/process_hand_type_parameter.xacro (robot description, xacro)
@@ -2,5 +2,5 @@
 <robot xmlns:xacro="http://www.ros.org/wiki/xacro">
 	<!-- Translate deprecated parameters 'muscle' and 'muscletrans' -->
-	<xacro:if value="${muscle}">
+	<!--xacro:if value="${muscle}">
 		<xacro:if value="${muscletrans}">
 			<xacro:property name="hand_type" value="muscletrans" />
@@ -11,16 +11,19 @@
 			${xacro.warning('Parameter "muscle" is deprecated. Please use hand_type="muscle" instead!')}
 		</xacro:unless>
-	</xacro:if>
+	</xacro:if-->
 	<!-- Unset deprecated parameters, now that we have translated them to hand_type -->
-	<xacro:property name="muscletrans" remove="true" />
-	<xacro:property name="muscle" remove="true" />
+	<!--xacro:property name="muscletrans" remove="true" />
+	<xacro:property name="muscle" remove="true" /-->
 	<!-- Normalize hand_type to be lower case -->
 	<xacro:property name="hand_type" value="${hand_type.lower()}" lazy_eval="false" />
 	<!-- Unify hand_type names, mapping hand_e -> motor, hand_e_plus -> motor+ -->
 	<xacro:if value="${hand_type.lower() == 'hand_e'}">
-		<xacro:property name="hand_type" value="motor" />
+		<xacro:property name="hand_type" value="E" />
 	</xacro:if>
-	<xacro:if value="${hand_type.lower() == 'hand_e_plus'}">
-		<xacro:property name="hand_type" value="motor+" />
+	<xacro:if value="${hand_type.lower() == 'hand_lite'}">
+		<xacro:property name="hand_type" value="G" />
+	</xacro:if>
+	<xacro:if value="${hand_type.lower() == 'hand_extra_lite'}">
+		<xacro:property name="hand_type" value="G-" />
 	</xacro:if>
 </robot>

File: sr_description/hand/xacro/process_sensor_parameters.xacro (robot description, xacro)
@@ -2,6 +2,6 @@
 	<xacro:include filename="$(find sr_description)/hand/xacro/validate_macros.xacro" />
 	<!-- Set defaults -->
-	<xacro:property name="default_tactile_sensor" default="std" />
-	<xacro:property name="tip_sensors" default="${default_tactile_sensor}" />
+	<xacro:property name="default_tactile_sensor" default="none" />
+	<xacro:property name="tip_sensors" default="${pst}" />
 	<xacro:property name="mid_sensors" default="${default_tactile_sensor}" />
 	<xacro:property name="prox_sensors" default="${default_tactile_sensor}" />
@@ -9,5 +9,5 @@
 	<!---->
 	<!-- Translate deprecated sensor parameters -->
-	<xacro:macro name="translate_from_deprecated" params="name value tip:=${None} mid:=std prox:=std palm:=std">
+	<xacro:macro name="translate_from_deprecated" params="name value tip:=${None} mid:=none prox:=none palm:=std">
 		<xacro:if value="${value}">
 			<xacro:if value="${tip is None}">

File: sr_description/hand/xacro/th_ff_rf_ellipsoid_hand.urdf.xacro (robot description, xacro)
@@ -7,5 +7,5 @@
   <!-- reflect is either 1 (for right hand) or -1 (for left hand) -->
   <!-- prefix can be anything but usually is "r_" or  "l_" for right and left hands distinction -->
-  <xacro:macro name="shadowhand" params="muscletrans muscle bio bt_sp eli reflect prefix">
+  <xacro:macro name="shadowhand" params="muscletrans muscle bt_2p bt_sp eli reflect prefix">
     ${xacro.warning("The file th_ff_rf_ellipsoid_hand.urdf.xacro is deprecated", print_location=False)}
     ${xacro.warning("Use full_hand.urdf.xacro instead with tip_sensors='th=eli ff=eli rf=eli'")}

File: sr_description/hand/xacro/three_biotac_fingers_hand.urdf.xacro (robot description, xacro)
@@ -9,9 +9,9 @@
   <xacro:macro name="shadowhand" params="muscletrans muscle bio bt_sp eli reflect prefix">
     ${xacro.warning("The file three_biotac_fingers_hand.urdf.xacro is deprecated", print_location=False)}
-    ${xacro.warning("Use full_hand.urdf.xacro instead with tip_sensors='th=bio ff=bio mf=bio'")}
+    ${xacro.warning("Use full_hand.urdf.xacro instead with tip_sensors='th=bt_2p ff=bt_2p mf=bt_2p'")}
     <!-- forward to generic macro -->
     <xacro:include filename="$(find sr_description)/hand/xacro/full_hand.urdf.xacro" />
     <!-- BioTacs on First and Middle Finger as well as Thumb -->
-    <xacro:shadowhand reflect="${reflect}" prefix="${prefix}" tip_sensors="th=bio ff=bio mf=bio" />
+    <xacro:shadowhand reflect="${reflect}" prefix="${prefix}" tip_sensors="th=bt_2p ff=bt_2p mf=bt_2p" />
   </xacro:macro>
 </robot>

File: sr_description/hand/xacro/thumb/thdistal.urdf.xacro (robot description, xacro)
@@ -8,10 +8,10 @@
   <xacro:include filename="$(find sr_description)/hand/xacro/thumb/thdistal.gazebo.xacro" />
   <xacro:include filename="$(find sr_description)/hand/xacro/thumb/thdistal.transmission.xacro" />
-  <!-- tip_sensor describes the sensor std, none, bio, bt_sp, eli -->
+  <!-- tip_sensor describes the sensor none, bt_2p, bt_sp, eli -->
   <!-- prefix can be anything but usually is "r_" or  "l_" for right and left hands distinction -->
   <!-- parent is the parent link for the first joint -->
   <xacro:macro name="thdistal"
     params="tip_sensor:=^|std prefix:=^ parent">
-    <xacro:if value="${tip_sensor == 'bio'}">
+    <xacro:if value="${tip_sensor == 'bt_2p'}">
       <!--    BIOTAC -->
       <link name="${prefix}thdistal_J1_dummy">
@@ -113,5 +113,5 @@
       </joint>
     </xacro:if>
-    <xacro:unless value="${tip_sensor == 'bio'}">
+    <xacro:unless value="${tip_sensor == 'bt_2p'}">
       <!-- common -->
       <link name="${prefix}thdistal">

File: sr_description/hand/xacro/thumb/thmiddle.urdf.xacro (robot description, xacro)
@@ -8,5 +8,5 @@
   <xacro:include filename="$(find sr_description)/hand/xacro/thumb/thmiddle.gazebo.xacro" />
   <xacro:include filename="$(find sr_description)/hand/xacro/thumb/thmiddle.transmission.xacro" />
-  <!-- mid_sensor can have value bio for specific middle anything else for standard finger -->
+  <!-- mid_sensor can have value bt_2p for specific middle anything else for standard finger -->
   <!-- prefix can be anything but usually is "r_" or  "l_" for right and left hands distinction -->
   <!-- parent is the parent link for the first joint -->
@@ -21,5 +21,5 @@
       <visual>
         <origin xyz="0 0 0" rpy="0 0 0" />
-        <xacro:if value="${mid_sensor == 'bio'}">
+        <xacro:if value="${mid_sensor == 'bt_2p'}">
           <geometry name="${prefix}thmiddle_visual">
             <mesh filename="package://sr_description/meshes/hand/biotacs/biotac_thumb_adapter.dae"
@@ -27,5 +27,5 @@
           </geometry>
         </xacro:if>
-        <xacro:unless value="${mid_sensor == 'bio'}">
+        <xacro:unless value="${mid_sensor == 'bt_2p'}">
           <geometry name="${prefix}thmiddle_visual">
             <mesh filename="package://sr_description/meshes/hand/TH2_z.dae"
@@ -38,5 +38,5 @@
       </visual>
       <collision>
-        <xacro:if value="${mid_sensor == 'bio'}">
+        <xacro:if value="${mid_sensor == 'bt_2p'}">
           <origin xyz="0 0 0.005" rpy="0 0 0" />
           <geometry name="${prefix}thmiddle_collision_geom">
@@ -44,5 +44,5 @@
           </geometry>
         </xacro:if>
-        <xacro:unless value="${mid_sensor == 'bio'}">
+        <xacro:unless value="${mid_sensor == 'bt_2p'}">
           <origin xyz="0 0 0.012" rpy="0 0 0" />
           <geometry name="${prefix}thmiddle_collision_geom">
@@ -51,5 +51,5 @@
         </xacro:unless>
       </collision>
-      <xacro:unless value="${mid_sensor == 'bio'}">
+      <xacro:unless value="${mid_sensor == 'bt_2p'}">
         <collision>
           <origin xyz="0 0 0.019" rpy="0 0 0" />
@@ -63,9 +63,9 @@
       <parent link="${parent}" />
       <child link="${prefix}thmiddle" />
-      <xacro:if value="${mid_sensor == 'bio'}">
+      <xacro:if value="${mid_sensor == 'bt_2p'}">
         <origin xyz="0 0 0.01" rpy="0 0 0" />
         <!-- FIXME: z offset is too large -->
       </xacro:if>
-      <xacro:unless value="${mid_sensor == 'bio'}">
+      <xacro:unless value="${mid_sensor == 'bt_2p'}">
         <origin xyz="0 0 0" rpy="0 0 0" />
       </xacro:unless>

File: sr_description/hand/xacro/thumb/thumb.urdf.xacro (robot description, xacro)
@@ -5,6 +5,6 @@
   <xacro:include filename="$(find sr_description)/hand/xacro/thumb/thmiddle.urdf.xacro" />
   <xacro:include filename="$(find sr_description)/hand/xacro/thumb/thdistal.urdf.xacro" />
-  <!-- tip_sensor describes the sensor none, bio, bt_sp, eli -->
-  <!-- mid_sensor describes the sensor none, bio -->
+  <!-- tip_sensor describes the sensor none, bt_2p, bt_sp, eli -->
+  <!-- mid_sensor describes the sensor none, bt_2p -->
   <!-- prox_sensor describes the sensor none, standard -->
   <!-- reflect is either 1 (for right hand) or -1 (for left hand) -->
@@ -14,6 +14,6 @@
   <xacro:macro name="thumb"
   params=" tip_sensor:=^|std mid_sensor:=^|std prox_sensor:=^|std reflect:=^ prefix:=^ parent is_lite">
-    <xacro:if value="${tip_sensor == 'bio'}">
-      <xacro:property name="mid_sensor" value="bio" />
+    <xacro:if value="${tip_sensor == 'bt_2p'}">
+      <xacro:property name="mid_sensor" value="bt_2p" />
     </xacro:if>
     <!-- Base -->

File: sr_description/robots/shadowhand_left_motor_biotac.urdf.xacro (robot description, xacro)
@@ -14,4 +14,4 @@
     <origin xyz="0.0 0.0 0.0" rpy="0.0 0.0 0.0" />
   </joint>
-  <xacro:shadowhand hand_type="motor" tip_sensors="bio" reflect="-1.0" prefix="lh_" />
+  <xacro:shadowhand hand_type="motor" tip_sensors="bt_2p" reflect="-1.0" prefix="lh_" />
 </robot>

File: sr_description/robots/shadowhand_motor.urdf.xacro (robot description, xacro)
@@ -14,4 +14,4 @@
       <origin xyz="0.0 0.0 0.0" rpy="0.0 0.0 0.0" />
     </joint>
-  <xacro:shadowhand hand_type="motor" reflect="1.0" prefix="rh_" />
+  <xacro:shadowhand hand_type="E" reflect="1.0" prefix="rh_" />
 </robot>

File: sr_description/robots/shadowhand_motor_biotac.urdf.xacro (robot description, xacro)
@@ -14,4 +14,4 @@
     <origin xyz="0.0 0.0 0.0" rpy="0.0 0.0 0.0" />
   </joint>
-  <xacro:shadowhand hand_type="motor" tip_sensors="bio" reflect="1.0" prefix="rh_" />
+  <xacro:shadowhand hand_type="motor" tip_sensors="bt_2p" reflect="1.0" prefix="rh_" />
 </robot>

File: sr_description/robots/shadowhand_motor_ff_biotac.urdf.xacro (robot description, xacro)
@@ -14,4 +14,4 @@
       <origin xyz="0.0 0.0 0.0" rpy="0.0 0.0 0.0" />
     </joint>
-  <xacro:shadowhand hand_type="motor" tip_sensors="ff=bio" reflect="1.0" prefix="rh_" />
+  <xacro:shadowhand hand_type="motor" tip_sensors="ff=bt_2p" reflect="1.0" prefix="rh_" />
 </robot>
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