Commit message: Replaced muscletrans with hand_c

File: sr_description/hand/xacro/ff_biotac_hand.urdf.xacro (robot description, xacro)
@@ -1,10 +1,3 @@
 <robot xmlns:xacro="http://www.ros.org/wiki/xacro">
-  <!-- muscletrans is true for muscle transmission to be used, false to use motor transmission -->
-  <!-- muscle is true for muscle hand or false for motor hand -->
-  <!-- bio is true for biotac finger or false for standard finger -->
-  <!-- bt_sp is true for BT_SP finger or false for standard finger -->
-  <!-- eli is true for ellipsoid fingertip or false for standard finger -->
-  <!-- reflect is either 1 (for right hand) or -1 (for left hand) -->
-  <!-- prefix can be anything but usually is "r_" or  "l_" for right and left hands distinction -->
   <xacro:macro name="shadowhand" params="muscletrans muscle bio bt_sp eli reflect prefix">
     ${xacro.warning("The file ff_biotac_hand.urdf.xacro is deprecated", print_location=False)}

File: sr_description/hand/xacro/finger/knuckle/knuckle.gazebo.xacro (robot description, xacro)
@@ -2,5 +2,4 @@
 <robot xmlns:xacro="http://www.ros.org/wiki/xacro">
   <xacro:macro name="knuckle_gazebo" params="prefix:=^ link_prefix:=^">
-    <!-- prefix can be anything but usually is "r_" or  "l_" for right and left hands distinction -->
     <gazebo reference="${prefix}${link_prefix}knuckle">
       <sensor type="contact" name="${prefix}${link_prefix}knuckle_contact">

File: sr_description/hand/xacro/finger/knuckle/knuckle.transmission.xacro (robot description, xacro)
@@ -4,10 +4,7 @@
        xmlns:interface="http://playerstage.sourceforge.net/gazebo/xmlschema/#interface"
        xmlns:xacro="http://www.ros.org/wiki/xacro">
-    <!-- prefix can be anything but usually is "r_" or  "l_" for right and left hands distinction -->
-    <!-- link_prefix prepends fingername to the link names -->
-    <!-- joint_prefix prepends fingername to the joint names -->
     <xacro:macro name="knuckle_transmission" params="hand_type:=^ prefix:=^ joint_prefix:=^ link_prefix:=^">
         <!-- muscle hand -->
-        <xacro:if value="${hand_type == 'muscletrans'}">
+        <xacro:if value="${hand_type == 'hand_c'}">
             <transmission name="${prefix}${link_prefix}knuckle_transmission">
                 <type>sr_mechanism_model/SimpleTransmissionForMuscle</type>
@@ -22,5 +19,5 @@
         </xacro:if>
         <!-- motor hand -->
-        <xacro:unless value="${hand_type == 'muscletrans'}">
+        <xacro:unless value="${hand_type == 'hand_c'}">
             <transmission name="${prefix}${link_prefix}knuckle_transmission">
                 <type>sr_mechanism_model/SimpleTransmission</type>

File: sr_description/hand/xacro/finger/knuckle/knuckle.urdf.xacro (robot description, xacro)
@@ -1,29 +1,22 @@
 <robot xmlns:xacro="http://www.ros.org/wiki/xacro"
-xmlns:sensor="http://playerstage.sourceforge.net/gazebo/xmlschema/#sensor"
-xmlns:controller="http://playerstage.sourceforge.net/gazebo/xmlschema/#controller"
-xmlns:joint="http://playerstage.sourceforge.net/gazebo/xmlschema/#slider"
-xmlns:interface="http://playerstage.sourceforge.net/gazebo/xmlschema/#interface"
-xmlns:body="http://playerstage.sourceforge.net/gazebo/xmlschema/#body"
-xmlns:geom="http://playerstage.sourceforge.net/gazebo/xmlschema/#geom">
+       xmlns:sensor="http://playerstage.sourceforge.net/gazebo/xmlschema/#sensor"
+       xmlns:controller="http://playerstage.sourceforge.net/gazebo/xmlschema/#controller"
+       xmlns:joint="http://playerstage.sourceforge.net/gazebo/xmlschema/#slider"
+       xmlns:interface="http://playerstage.sourceforge.net/gazebo/xmlschema/#interface"
+       xmlns:body="http://playerstage.sourceforge.net/gazebo/xmlschema/#body"
+       xmlns:geom="http://playerstage.sourceforge.net/gazebo/xmlschema/#geom">
   <xacro:include filename="$(find sr_description)/hand/xacro/finger/knuckle/knuckle.gazebo.xacro" />
   <xacro:include filename="$(find sr_description)/hand/xacro/finger/knuckle/knuckle.transmission.xacro" />
-  <!-- prefix can be anything but usually is "r_" or  "l_" for right and left hands distinction -->
-  <!-- link_prefix prepends fingername to the link names -->
-  <!-- joint_prefix prepends fingername to the joint names -->
-  <!-- parent is the parent link for the joint -->
-  <xacro:macro name="knuckle"
-  params="prefix:=^ link_prefix:=^ joint_prefix:=^ parent *origin">
+  <xacro:macro name="knuckle" params="prefix:=^ link_prefix:=^ joint_prefix:=^ parent *origin">
     <link name="${prefix}${link_prefix}knuckle">
       <inertial>
         <origin xyz="0 0 0" rpy="0 0 0" />
         <mass value="0.008" />
-        <inertia ixx="0.00000026" ixy="0.0" ixz="0.0"
-        iyy="0.00000026" iyz="0.0" izz="0.00000032" />
+        <inertia ixx="0.00000026" ixy="0.0" ixz="0.0" iyy="0.00000026" iyz="0.0" izz="0.00000032" />
       </inertial>
       <visual>
         <origin xyz="0 0 0.0005" rpy="0 0 0" />
         <geometry name="${prefix}${link_prefix}knuckle_visual">
-          <mesh filename="package://sr_description/meshes/hand/knuckle.dae"
-          scale="0.001 0.001 0.001" />
+          <mesh filename="package://sr_description/meshes/hand/knuckle.dae" scale="0.001 0.001 0.001" />
         </geometry>
         <material name="LightGrey" />
@@ -42,6 +35,5 @@
       <xacro:insert_block name="origin" />
       <xacro:insert_block name="axis" />
-      <limit lower="${-20/180*pi}" upper="${20/180*pi}"
-      effort="2" velocity="2.0" />
+      <limit lower="${-20/180*pi}" upper="${20/180*pi}" effort="2" velocity="2.0" />
       <dynamics damping="0.1" />
     </joint>

File: sr_description/hand/xacro/finger/lfmetacarpal/lfmetacarpal.gazebo.xacro (robot description, xacro)
@@ -2,5 +2,4 @@
 <robot xmlns:xacro="http://www.ros.org/wiki/xacro">
   <xacro:macro name="lfmetacarpal_gazebo" params="prefix:=^ palm_sensor:=^|none link_prefix">
-    <!-- prefix can be anything but usually is "r_" or  "l_" for right and left hands distinction -->
     <gazebo reference="${prefix}lfmetacarpal">
       <xacro:unless value="${'none' in palm_sensor}" >

File: sr_description/hand/xacro/finger/lfmetacarpal/lfmetacarpal.transmission.xacro (robot description, xacro)
@@ -4,8 +4,7 @@
        xmlns:interface="http://playerstage.sourceforge.net/gazebo/xmlschema/#interface"
        xmlns:xacro="http://www.ros.org/wiki/xacro">
-    <!-- prefix can be anything but usually is "r_" or  "l_" for right and left hands distinction -->
     <xacro:macro name="lfmetacarpal_transmission" params="hand_type:=^ prefix:=^">
         <!-- muscle hand -->
-        <xacro:if value="${hand_type == 'muscletrans'}">
+        <xacro:if value="${hand_type == 'hand_c'}">
             <transmission name="${prefix}lfmetacarpal_transmission">
                 <type>sr_mechanism_model/SimpleTransmissionForMuscle</type>
@@ -20,5 +19,5 @@
         </xacro:if>
         <!-- motor hand -->
-        <xacro:unless value="${hand_type == 'muscletrans'}">
+        <xacro:unless value="${hand_type == 'hand_c'}">
             <transmission name="${prefix}lfmetacarpal_transmission">
                 <type>sr_mechanism_model/SimpleTransmission</type>

File: sr_description/hand/xacro/finger/middle/middle.transmission.xacro (robot description, xacro)
@@ -4,10 +4,7 @@
        xmlns:interface="http://playerstage.sourceforge.net/gazebo/xmlschema/#interface"
        xmlns:xacro="http://www.ros.org/wiki/xacro">
-    <!-- prefix can be anything but usually is "r_" or  "l_" for right and left hands distinction -->
-    <!-- link_prefix prepends fingername to the link names -->
-    <!-- joint_prefix prepends fingername to the joint names -->
     <xacro:macro name="middle_transmission" params="hand_type:=^ prefix:=^ joint_prefix:=^ link_prefix:=^">
         <!-- muscle hand -->
-        <xacro:if value="${hand_type == 'muscletrans'}">
+        <xacro:if value="${hand_type == 'hand_c'}">
             <transmission name="${prefix}${link_prefix}middle_transmission">
                 <type>sr_mechanism_model/J0TransmissionForMuscle</type>
@@ -27,5 +24,5 @@
         </xacro:if>
         <!-- motor hand -->
-        <xacro:unless value="${hand_type == 'muscletrans'}">
+        <xacro:unless value="${hand_type == 'hand_c'}">
             <transmission name="${prefix}${link_prefix}middle_transmission">
                 <type>sr_mechanism_model/J0Transmission</type>

File: sr_description/hand/xacro/finger/proximal/proximal.gazebo.xacro (robot description, xacro)
@@ -2,5 +2,4 @@
 <robot xmlns:xacro="http://www.ros.org/wiki/xacro">
   <xacro:macro name="proximal_gazebo" params="prefix:=^ link_prefix:=^ prox_sensor:=^|none">
-    <!-- prefix can be anything but usually is "r_" or  "l_" for right and left hands distinction -->
     <gazebo reference="${prefix}${link_prefix}proximal">
       <xacro:unless value="${'none' in prox_sensor}" >

File: sr_description/hand/xacro/finger/proximal/proximal.transmission.xacro (robot description, xacro)
@@ -4,10 +4,7 @@
        xmlns:interface="http://playerstage.sourceforge.net/gazebo/xmlschema/#interface"
        xmlns:xacro="http://www.ros.org/wiki/xacro">
-    <!-- prefix can be anything but usually is "r_" or  "l_" for right and left hands distinction -->
-    <!-- link_prefix prepends fingername to the link names -->
-    <!-- joint_prefix prepends fingername to the joint names -->
     <xacro:macro name="proximal_transmission" params="hand_type:=^ prefix:=^ joint_prefix:=^ link_prefix:=^">
         <!-- muscle hand -->
-        <xacro:if value="${hand_type == 'muscletrans'}">
+        <xacro:if value="${hand_type == 'hand_c'}">
             <transmission name="${prefix}${link_prefix}proximal_transmission">
                 <type>sr_mechanism_model/SimpleTransmissionForMuscle</type>
@@ -22,5 +19,5 @@
         </xacro:if>
         <!-- motor hand -->
-        <xacro:unless value="${hand_type == 'muscletrans'}">
+        <xacro:unless value="${hand_type == 'hand_c'}">
             <transmission name="${prefix}${link_prefix}proximal_transmission">
                 <type>sr_mechanism_model/SimpleTransmission</type>

File: sr_description/hand/xacro/full_hand.urdf.xacro (robot description, xacro)
@@ -8,5 +8,5 @@
   <xacro:include filename="$(find sr_description)/hand/xacro/finger/fingers.urdf.xacro" />
   <xacro:include filename="$(find sr_description)/hand/xacro/thumb/thumb.urdf.xacro" />
-  <!-- hand_type can be: E, G, muscle (muscle), muscletrans (muscletrans) -->
+  <!-- hand_type can be: hand_e, hand_g, hand_c -->
   <!-- fingers: list-like string specifying available fingers, default: 'th ff mf rf lf' -->
   <!-- tip_sensors: plain or dict-like string specifying the fingertip (tactile) sensors: 'th=bt_2p ff=bt_sp mf=pst rf=pst, lf=pst' -->
@@ -22,5 +22,5 @@
   <!-- eli (deprecated) is true for ellipsoid fingertip or false for standard finger -->
   <!-- lf (deprecated) is true if we want a little finger, false otherwise -->
-  <xacro:macro name="shadowhand" params="hand_type:='motor' reflect prefix cable_mesh:=False fingers:=all
+  <xacro:macro name="shadowhand" params="hand_type:='hand_e' reflect prefix cable_mesh:=False fingers:=all
           tip_sensors:=pst mid_sensors:=none prox_sensors:=none palm_sensor:=none
           muscletrans:=^|${None} muscle:=^|${None} lf:=^|${None} bio:=^|${None} bt_sp:=^|${None} eli:=^|${None}">

File: sr_description/hand/xacro/hand_lite.urdf.xacro (robot description, xacro)
@@ -8,5 +8,5 @@
   <xacro:include filename="$(find sr_description)/hand/xacro/finger/fingers.urdf.xacro" />
   <xacro:include filename="$(find sr_description)/hand/xacro/thumb/thumb.urdf.xacro" />
-  <!-- hand_type can be: motor, motor+, muscle (muscle), muscletrans (muscletrans) -->
+  <!-- hand_type can be: hand_e, hand_g, hand_c -->
   <!-- fingers: list-like string specifying available fingers, default: 'th ff mf rf' -->
   <!-- tip_sensors: plain or dict-like string specifying the fingertip (tactile) sensors: 'th=bt_2p ff=bt_sp mf=pst rf=pst, lf=pst' -->

File: sr_description/hand/xacro/th_ff_rf_ellipsoid_hand.urdf.xacro (robot description, xacro)
@@ -1,10 +1,3 @@
 <robot xmlns:xacro="http://www.ros.org/wiki/xacro">
-  <!-- muscletrans is true for muscle transmission to be used, false to use motor transmission -->
-  <!-- muscle is true for muscle hand or false for motor hand -->
-  <!-- bio is true for biotac finger or false for standard finger -->
-  <!-- bt_sp is true for BT_SP finger or false for standard finger -->
-  <!-- eli is true for ellipsoid fingertip or false for standard finger -->
-  <!-- reflect is either 1 (for right hand) or -1 (for left hand) -->
-  <!-- prefix can be anything but usually is "r_" or  "l_" for right and left hands distinction -->
   <xacro:macro name="shadowhand" params="muscletrans muscle bt_2p bt_sp eli reflect prefix">
     ${xacro.warning("The file th_ff_rf_ellipsoid_hand.urdf.xacro is deprecated", print_location=False)}

File: sr_description/hand/xacro/three_biotac_fingers_hand.urdf.xacro (robot description, xacro)
@@ -1,10 +1,3 @@
 <robot xmlns:xacro="http://www.ros.org/wiki/xacro">
-  <!-- muscletrans is true for muscle transmission to be used, false to use motor transmission -->
-  <!-- muscle is true for muscle hand or false for motor hand -->
-  <!-- bio is true for biotac finger or false for standard finger -->
-  <!-- bt_sp is true for BT_SP finger or false for standard finger -->
-  <!-- eli is true for ellipsoid fingertip or false for standard finger -->
-  <!-- reflect is either 1 (for right hand) or -1 (for left hand) -->
-  <!-- prefix can be anything but usually is "r_" or  "l_" for right and left hands distinction -->
   <xacro:macro name="shadowhand" params="muscletrans muscle bio bt_sp eli reflect prefix">
     ${xacro.warning("The file three_biotac_fingers_hand.urdf.xacro is deprecated", print_location=False)}

File: sr_description/hand/xacro/three_fingers_hand.urdf.xacro (robot description, xacro)
@@ -1,10 +1,3 @@
 <robot xmlns:xacro="http://www.ros.org/wiki/xacro">
-  <!-- muscletrans is true for muscle transmission to be used, false to use motor transmission -->
-  <!-- muscle is true for muscle hand or false for motor hand -->
-  <!-- bio is true for biotac finger or false for standard finger -->
-  <!-- bt_sp is true for BT_SP finger or false for standard finger -->
-  <!-- eli is true for ellipsoid fingertip or false for standard finger -->
-  <!-- reflect is either 1 (for right hand) or -1 (for left hand) -->
-  <!-- prefix can be anything but usually is "r_" or  "l_" for right and left hands distinction -->
   <xacro:macro name="shadowhand" params="muscletrans muscle bio bt_sp eli reflect prefix">
     ${xacro.warning("The file three_fingers_hand.urdf.xacro is deprecated", print_location=False)}

File: sr_description/hand/xacro/three_fingers_hand_RF.urdf.xacro (robot description, xacro)
@@ -1,10 +1,3 @@
 <robot xmlns:xacro="http://www.ros.org/wiki/xacro">
-  <!-- muscletrans is true for muscle transmission to be used, false to use motor transmission -->
-  <!-- muscle is true for muscle hand or false for motor hand -->
-  <!-- bio is true for biotac finger or false for standard finger -->
-  <!-- bt_sp is true for BT_SP finger or false for standard finger -->
-  <!-- eli is true for ellipsoid fingertip or false for standard finger -->
-  <!-- reflect is either 1 (for right hand) or -1 (for left hand) -->
-  <!-- prefix can be anything but usually is "r_" or  "l_" for right and left hands distinction -->
   <xacro:macro name="shadowhand" params="muscletrans muscle bio bt_sp eli reflect prefix">
     ${xacro.warning("The file three_fingers_hand_RF.urdf.xacro is deprecated", print_location=False)}

File: sr_description/hand/xacro/thumb/thbase.gazebo.xacro (robot description, xacro)
@@ -2,5 +2,4 @@
 <robot xmlns:xacro="http://www.ros.org/wiki/xacro">
   <xacro:macro name="thbase_gazebo" params="prefix:=^">
-    <!-- prefix can be anything but usually is "r_" or  "l_" for right and left hands distinction -->
     <gazebo reference="${prefix}thbase">
       <sensor type="contact" name="${prefix}thbase_contact">

File: sr_description/hand/xacro/thumb/thbase.transmission.xacro (robot description, xacro)
@@ -4,8 +4,7 @@
        xmlns:interface="http://playerstage.sourceforge.net/gazebo/xmlschema/#interface"
        xmlns:xacro="http://www.ros.org/wiki/xacro">
-    <!-- prefix can be anything but usually is "r_" or  "l_" for right and left hands distinction -->
     <xacro:macro name="thbase_transmission" params="hand_type:=^ prefix:=^">
         <!-- muscle hand -->
-        <xacro:if value="${hand_type == 'muscletrans'}">
+        <xacro:if value="${hand_type == 'hand_c'}">
             <transmission name="${prefix}thbase_transmission">
                 <type>sr_mechanism_model/SimpleTransmissionForMuscle</type>
@@ -20,5 +19,5 @@
         </xacro:if>
         <!-- motor hand -->
-        <xacro:unless value="${hand_type == 'muscletrans'}">
+        <xacro:unless value="${hand_type == 'hand_c'}">
             <transmission name="${prefix}thbase_transmission">
                 <type>sr_mechanism_model/SimpleTransmission</type>

File: sr_description/hand/xacro/thumb/thdistal.transmission.xacro (robot description, xacro)
@@ -4,8 +4,7 @@
        xmlns:interface="http://playerstage.sourceforge.net/gazebo/xmlschema/#interface"
        xmlns:xacro="http://www.ros.org/wiki/xacro">
-    <!-- prefix can be anything but usually is "r_" or  "l_" for right and left hands distinction -->
     <xacro:macro name="thdistal_transmission" params="hand_type:=^ prefix:=^">
         <!-- muscle hand -->
-        <xacro:if value="${hand_type == 'muscletrans'}">
+        <xacro:if value="${hand_type == 'hand_c'}">
             <transmission name="${prefix}thdistal_transmission">
                 <type>sr_mechanism_model/SimpleTransmissionForMuscle</type>
@@ -20,5 +19,5 @@
         </xacro:if>
         <!-- motor hand -->
-        <xacro:unless value="${hand_type == 'muscletrans'}">
+        <xacro:unless value="${hand_type == 'hand_c'}">
             <transmission name="${prefix}thdistal_transmission">
                 <type>sr_mechanism_model/SimpleTransmission</type>

File: sr_description/hand/xacro/thumb/thhub.gazebo.xacro (robot description, xacro)
@@ -2,5 +2,4 @@
 <robot xmlns:xacro="http://www.ros.org/wiki/xacro">
   <xacro:macro name="thhub_gazebo" params="prefix:=^">
-    <!-- prefix can be anything but usually is "r_" or  "l_" for right and left hands distinction -->
     <gazebo reference="${prefix}thhub">
       <sensor type="contact" name="${prefix}thhub_contact">

File: sr_description/hand/xacro/thumb/thhub.transmission.xacro (robot description, xacro)
@@ -4,8 +4,7 @@
        xmlns:interface="http://playerstage.sourceforge.net/gazebo/xmlschema/#interface"
        xmlns:xacro="http://www.ros.org/wiki/xacro">
-    <!-- prefix can be anything but usually is "r_" or  "l_" for right and left hands distinction -->
     <xacro:macro name="thhub_transmission" params="hand_type:=^ prefix:=^">
         <!-- muscle hand -->
-        <xacro:if value="${hand_type == 'muscletrans'}">
+        <xacro:if value="${hand_type == 'hand_c'}">
             <transmission name="${prefix}thhub_transmission">
                 <type>sr_mechanism_model/SimpleTransmissionForMuscle</type>
@@ -20,5 +19,5 @@
         </xacro:if>
         <!-- motor hand -->
-        <xacro:unless value="${hand_type == 'muscletrans'}">
+        <xacro:unless value="${hand_type == 'hand_c'}">
             <transmission name="${prefix}thhub_transmission">
                 <type>sr_mechanism_model/SimpleTransmission</type>
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