Commit message: Updated validation xacro and small fixes

File: sr_description/hand/xacro/validate_xacro.xacro (robot description, xacro)
@@ -1,5 +1,5 @@
 <robot xmlns:xacro="http://www.ros.org/wiki/xacro">
 	<xacro:property name="allowed_hand_types" value="${python.list(['hand_e','hand_g','hand_c'])}"/>
-  <xacro:property name="allowed_hand_versions" value="${python.list(['E3M5','E2M3','C6M2'])}"/>
+  <xacro:property name="allowed_hand_versions" value="${python.list(['E3M5','E2M3','C6M2', 'G1M5'])}"/>
   <xacro:property name="allowed_sides" value="${python.list(['right','left'])}"/>
   <xacro:property name="allowed_fingers" value="${python.list(['th','ff','mf','rf','lf','all'])}"/>
@@ -13,6 +13,6 @@
     ${xacro.error("Parameter 'side' ("+side+") not within allowed values "+python.str(allowed_sides))}
   </xacro:unless>
-  <xacro:unless value="${python.len(python.set(python.list(fingers.split(',')))-python.set(allowed_fingers)) == 0}">
-    ${xacro.error("Parameter 'fingers' ("+python.str(python.set(python.list(fingers.split(',')))-python.set(allowed_fingers))+") not within allowed values "+python.str(allowed_fingers))}
+	<xacro:unless value="${hand_type.lower()[-1] == hand_version.lower()[0]}">
+    ${xacro.error("Parameter 'hand_type' ("+hand_type+") doesn't comply with 'hand_version' ("+hand_version+")")}
   </xacro:unless>
 </robot>
