Commit message: Fixed hand lite and extra lite

File: sr_description/hand/xacro/hand.urdf.xacro (robot description, xacro)
@@ -4,6 +4,5 @@
        xmlns:interface="http://playerstage.sourceforge.net/gazebo/xmlschema/#interface">
   <xacro:macro name="sr_hand"
-               params="hand_type:='hand_e' hand_version:='E3M5' side fingers tip_sensors prox_sensors mid_sensors
-                      palm_sensor">
+               params="hand_type hand_version side fingers tip_sensors prox_sensors mid_sensors palm_sensor">
     <xacro:if value="${side == 'right'}">
       <xacro:property name="reflect" value="1" />
@@ -15,15 +14,15 @@
     </xacro:if>
     <!-- Selecting hand according with hand_type -->
-    <xacro:if value="${hand_type.startswith('hand_e')}">
+    <xacro:if value="${hand_type == 'hand_e'}">
        <xacro:include filename="$(find sr_description)/hand/xacro/hand_e.urdf.xacro" />
        <xacro:sr_hand_e />
     </xacro:if>
-    <!--xacro:if value="${hand_version.startswith('G')}">
+    <xacro:if value="${hand_type == 'hand_g'}">
        <xacro:include filename="$(find sr_description)/hand/xacro/hand_g.urdf.xacro" />
        <xacro:sr_hand_g />
     </xacro:if>
-    <xacro:if value="${hand_version.startswith('C')}">
+    <!--xacro:if value="${hand_type == 'hand_c'}">
        <xacro:include filename="$(find sr_description)/hand/xacro/hand_c.urdf.xacro" />
-       <xacro:sr_hand_m />
+       <xacro:sr_hand_c />
     </xacro:if-->
   </xacro:macro>

File: sr_description/hand/xacro/hand_g.urdf.xacro (robot description, xacro)
@@ -14,5 +14,5 @@
   <!-- prox_sensors: plain or dict-like string specifying the proximal (tactile) sensors -->
   <!-- palm_sensor: specifies the palm tactile sensor -->
-  <xacro:macro name="sr_hand_e" params="hand_version:=^ reflect:=^ prefix:=^ fingers:=^|all tip_sensors:=^|pst
+  <xacro:macro name="sr_hand_g" params="hand_version:=^ reflect:=^ prefix:=^ fingers:=^|all tip_sensors:=^|pst
                prox_sensors:=^|none mid_sensors:=^|none palm_sensor:=^|none">
     <!-- Unify hand type parameter -->

File: sr_description/hand/xacro/palm/palm_g.urdf.xacro (robot description, xacro)
@@ -18,5 +18,5 @@
         <origin xyz="0 0 0" rpy="0 0 0" />
         <geometry name="${prefix}palm_visual">
-          <mesh filename="package://sr_description/meshes/products/${hand_type}/${hand_version}/palm_${hand_version}.stl"
+          <mesh filename="package://sr_description/meshes/products/${hand_type}/${hand_version}/palm_${hand_version}.dae"
           scale="${reflect*0.001} 0.001 0.001" />
         </geometry>

File: sr_description/hand/xacro/process_hand_type_parameter.xacro (robot description, xacro)
@@ -21,9 +21,6 @@
 		<xacro:property name="hand_type" value="E" />
 	</xacro:if>
-	<xacro:if value="${hand_type.lower() == 'hand_lite'}">
+	<xacro:if value="${hand_type.lower() == 'hand_g'}">
 		<xacro:property name="hand_type" value="G" />
 	</xacro:if>
-	<xacro:if value="${hand_type.lower() == 'hand_extra_lite'}">
-		<xacro:property name="hand_type" value="G-" />
-	</xacro:if>
 </robot>

File: sr_description/robots/sr_hand_only.urdf.xacro (robot description, xacro)
@@ -11,5 +11,5 @@
     <xacro:arg name="side" default="right"/>
     <xacro:arg name="fingers" default="all"/>
-    <xacro:arg name="tip_sensors" default="bt_sp"/>
+    <xacro:arg name="tip_sensors" default="pst"/>
     <xacro:arg name="mid_sensors" default="none"/>
     <xacro:arg name="prox_sensors" default="none"/>

Commit message: Fixed validation of parameters

File: sr_description/hand/xacro/hand.urdf.xacro (robot description, xacro)
@@ -5,5 +5,6 @@
   <xacro:macro name="sr_hand"
                params="hand_type hand_version side fingers tip_sensors prox_sensors mid_sensors palm_sensor">
-  <xacro:include filename="$(find sr_description)/hand/xacro/validate_xacro.xacro" />
+    <!-- Process hand type, version and side parameters -->
+    <xacro:include filename="$(find sr_description)/hand/xacro/process_hand_type_version_side_parameters.xacro" />
     <xacro:if value="${side == 'right'}">
       <xacro:property name="reflect" value="1" />
@@ -15,13 +16,13 @@
     </xacro:if>
     <!-- Selecting hand according with hand_type -->
-    <xacro:if value="${hand_type == 'hand_e'}">
+    <xacro:if value="${hand_type == 'E'}">
        <xacro:include filename="$(find sr_description)/hand/xacro/hand_e.urdf.xacro" />
        <xacro:sr_hand_e />
     </xacro:if>
-    <xacro:if value="${hand_type == 'hand_g'}">
+    <xacro:if value="${hand_type == 'G'}">
        <xacro:include filename="$(find sr_description)/hand/xacro/hand_g.urdf.xacro" />
        <xacro:sr_hand_g />
     </xacro:if>
-    <xacro:if value="${hand_type == 'hand_c'}">
+    <xacro:if value="${hand_type == 'C'}">
        <xacro:include filename="$(find sr_description)/hand/xacro/hand_c.urdf.xacro" />
        <xacro:sr_hand_c />

File: sr_description/hand/xacro/hand_c.urdf.xacro (robot description, xacro)
@@ -5,5 +5,4 @@
   <xacro:include filename="$(find sr_description)/hand/xacro/finger/fingers.urdf.xacro" />
   <xacro:include filename="$(find sr_description)/hand/xacro/thumb/thumb.urdf.xacro" />
-  <!-- hand_type can be: hand_e, hand_g, hand_c -->
   <!-- fingers: list-like string specifying available fingers, default: 'th ff mf rf' -->
   <!-- tip_sensors: plain or dict-like string specifying the fingertip (tactile) sensors: 'th=bt_2p ff=bt_sp mf=pst rf=pst, lf=pst' -->
@@ -13,8 +12,5 @@
   <xacro:macro name="sr_hand_c" params="hand_version:=^ reflect:=^ prefix:=^ fingers:=^|all tip_sensors:=^|pst
                prox_sensors:=^|none mid_sensors:=^|none palm_sensor:=^|none">
-    <!-- Unify hand type parameter -->
-    <xacro:property name="hand_type" value="hand_c" />
-    <xacro:include filename="$(find sr_description)/hand/xacro/process_hand_type_parameter.xacro" />
-    <!-- Process fingers parameter, also handling deprecated lf -->
+    <!-- Process fingers parameter -->
     <xacro:property name="_all_finger_tokens_" value="${python.set('th ff mf rf lf'.split())}" />
     <xacro:include filename="$(find sr_description)/hand/xacro/process_fingers_parameter.xacro" />

File: sr_description/hand/xacro/hand_e.urdf.xacro (robot description, xacro)
@@ -8,5 +8,4 @@
   <xacro:include filename="$(find sr_description)/hand/xacro/finger/fingers.urdf.xacro" />
   <xacro:include filename="$(find sr_description)/hand/xacro/thumb/thumb.urdf.xacro" />
-  <!-- hand_type can be: hand_e, hand_g, hand_c -->
   <!-- fingers: list-like string specifying available fingers, default: 'th ff mf rf' -->
   <!-- tip_sensors: plain or dict-like string specifying the fingertip (tactile) sensors: 'th=bt_2p ff=bt_sp mf=pst rf=pst, lf=pst' -->
@@ -16,8 +15,5 @@
   <xacro:macro name="sr_hand_e" params="hand_version:=^ reflect:=^ prefix:=^ fingers:=^|all tip_sensors:=^|pst
                prox_sensors:=^|none mid_sensors:=^|none palm_sensor:=^|none">
-    <!-- Unify hand type parameter -->
-    <xacro:property name="hand_type" value="hand_e" />
-    <xacro:include filename="$(find sr_description)/hand/xacro/process_hand_type_parameter.xacro" />
-    <!-- Process fingers parameter, also handling deprecated lf -->
+    <!-- Process fingers parameter -->
     <xacro:property name="_all_finger_tokens_" value="${python.set('th ff mf rf lf'.split())}" />
     <xacro:include filename="$(find sr_description)/hand/xacro/process_fingers_parameter.xacro" />

File: sr_description/hand/xacro/hand_g.urdf.xacro (robot description, xacro)
@@ -8,5 +8,4 @@
   <xacro:include filename="$(find sr_description)/hand/xacro/finger/fingers.urdf.xacro" />
   <xacro:include filename="$(find sr_description)/hand/xacro/thumb/thumb.urdf.xacro" />
-  <!-- hand_type can be: hand_e, hand_g, hand_c -->
   <!-- fingers: list-like string specifying available fingers, default: 'th ff mf rf' -->
   <!-- tip_sensors: plain or dict-like string specifying the fingertip (tactile) sensors: 'th=bt_2p ff=bt_sp mf=pst rf=pst, lf=pst' -->
@@ -16,8 +15,5 @@
   <xacro:macro name="sr_hand_g" params="hand_version:=^ reflect:=^ prefix:=^ fingers:=^|all tip_sensors:=^|pst
                prox_sensors:=^|none mid_sensors:=^|none palm_sensor:=^|none">
-    <!-- Unify hand type parameter -->
-    <xacro:property name="hand_type" value="hand_g" />
-    <xacro:include filename="$(find sr_description)/hand/xacro/process_hand_type_parameter.xacro" />
-    <!-- Process fingers parameter, also handling deprecated -->
+    <!-- Process fingers parameter -->
     <xacro:property name="_all_finger_tokens_" value="${python.set('th ff mf rf'.split())}" />
     <xacro:include filename="$(find sr_description)/hand/xacro/process_fingers_parameter.xacro" />

File: sr_description/hand/xacro/process_sensor_parameters.xacro (robot description, xacro)
@@ -7,5 +7,4 @@
 	<xacro:property name="prox_sensors" default="${default_tactile_sensor}" />
 	<xacro:property name="palm_sensor" default="${default_tactile_sensor}" />
-	<!---->
 	<!-- Translate deprecated sensor parameters -->
 	<xacro:macro name="translate_from_deprecated" params="name value tip:=${None} mid:=none prox:=none palm:=none">
@@ -32,5 +31,4 @@
 	<xacro:property name="eli" default="${None}" />
 	<xacro:translate_from_deprecated name="eli" value="${eli}" />
-	<!---->
 	<!-- Transform sensor parameter into proper type -->
 	<xacro:macro name="transform_to_type" params="name value default_tactile_sensor:=^|none

File: sr_description/hand/xacro/validate_macros.xacro (robot description, xacro)
@@ -3,5 +3,5 @@
 		<!-- Check that list of tokens is valid -->
 		<xacro:property name="_unknown_tokens_" value="${python.set(tokens) - python.set(valid)}" />
-		<xacro:if value="${_unknown_tokens_}">${xacro.error('Unknown '+name+': '+', '.join(_unknown_tokens_))}</xacro:if>
+		<xacro:if value="${_unknown_tokens_}">${xacro.error('Unknown '+name+': '+', '.join(_unknown_tokens_)+'. The set of available specifiers is: '+', '.join(valid))}</xacro:if>
 	</xacro:macro>
 </validate>

Commit message: Refactoring sr_description: adapted test and added more parameters validation (#124)
* Removing robots.old folder

* Lint fixes

* Fixing CMakeLists

* Removing whitespace

* Applying changes from https://github.com/ubi-agni/sr_common/pull/2

* Adapting tests to refactored sr_description

* Adding validation xacro

* Update process_hand_type_parameter.xacro

* Updated validation xacro and small fixes

* Update test_models.sh

* Fixed validation of parameters

* Fixing formtating and deleted unnecessary files

* Work in progress

* Removed unnecessary files

Co-authored-by: Beatriz Leon <beatriz@shadowrobot.com>

File: sr_description/hand/xacro/hand.urdf.xacro (robot description, xacro)
@@ -3,6 +3,7 @@
        xmlns:controller="http://playerstage.sourceforge.net/gazebo/xmlschema/#controller"
        xmlns:interface="http://playerstage.sourceforge.net/gazebo/xmlschema/#interface">
-  <xacro:macro name="sr_hand"
-               params="hand_type hand_version side fingers tip_sensors prox_sensors mid_sensors palm_sensor">
+  <xacro:macro name="sr_hand" params="hand_type hand_version side fingers tip_sensors prox_sensors mid_sensors palm_sensor">
+    <!-- Process hand type, version and side parameters -->
+    <xacro:include filename="$(find sr_description)/hand/xacro/process_hand_type_version_side_parameters.xacro" />
     <xacro:if value="${side == 'right'}">
       <xacro:property name="reflect" value="1" />
@@ -14,13 +15,13 @@
     </xacro:if>
     <!-- Selecting hand according with hand_type -->
-    <xacro:if value="${hand_type == 'hand_e'}">
+    <xacro:if value="${hand_type == 'E'}">
        <xacro:include filename="$(find sr_description)/hand/xacro/hand_e.urdf.xacro" />
        <xacro:sr_hand_e />
     </xacro:if>
-    <xacro:if value="${hand_type == 'hand_g'}">
+    <xacro:if value="${hand_type == 'G'}">
        <xacro:include filename="$(find sr_description)/hand/xacro/hand_g.urdf.xacro" />
        <xacro:sr_hand_g />
     </xacro:if>
-    <xacro:if value="${hand_type == 'hand_c'}">
+    <xacro:if value="${hand_type == 'C'}">
        <xacro:include filename="$(find sr_description)/hand/xacro/hand_c.urdf.xacro" />
        <xacro:sr_hand_c />
