Commit message: Replaced full_hand with hand xacro and updated hand_g

File: sr_description/hand/xacro/hand_e.urdf.xacro (robot description, xacro)
@@ -1,3 +1,6 @@
-<robot xmlns:xacro="http://www.ros.org/wiki/xacro">
+<robot xmlns:sensor="http://playerstage.sourceforge.net/gazebo/xmlschema/#sensor"
+       xmlns:controller="http://playerstage.sourceforge.net/gazebo/xmlschema/#controller"
+       xmlns:interface="http://playerstage.sourceforge.net/gazebo/xmlschema/#interface"
+       xmlns:xacro="http://www.ros.org/wiki/xacro">
   <xacro:include filename="$(find sr_description)/hand/xacro/forearm/forearm_e.urdf.xacro" />
   <xacro:include filename="$(find sr_description)/hand/xacro/wrist/wrist.urdf.xacro" />
@@ -5,7 +8,12 @@
   <xacro:include filename="$(find sr_description)/hand/xacro/finger/fingers.urdf.xacro" />
   <xacro:include filename="$(find sr_description)/hand/xacro/thumb/thumb.urdf.xacro" />
-  <xacro:macro name="sr_hand_e"
-               params="hand_version:=^ reflect:=^ prefix:=^ fingers:=^|all tip_sensors:=^|bt_sp prox_sensors:=^|none
-                      mid_sensors:=^|none palm_sensor:=^|none">
+  <!-- hand_type can be: hand_e, hand_g, hand_c -->
+  <!-- fingers: list-like string specifying available fingers, default: 'th ff mf rf' -->
+  <!-- tip_sensors: plain or dict-like string specifying the fingertip (tactile) sensors: 'th=bt_2p ff=bt_sp mf=pst rf=pst, lf=pst' -->
+  <!-- mid_sensors: plain or dict-like string specifying the middle-phalange (tactile) sensors -->
+  <!-- prox_sensors: plain or dict-like string specifying the proximal (tactile) sensors -->
+  <!-- palm_sensor: specifies the palm tactile sensor -->
+  <xacro:macro name="sr_hand_e" params="hand_version:=^ reflect:=^ prefix:=^ fingers:=^|all tip_sensors:=^|pst
+               prox_sensors:=^|none mid_sensors:=^|none palm_sensor:=^|none">
     <!-- Unify hand type parameter -->
     <xacro:property name="hand_type" value="hand_e" />

File: sr_description/hand/xacro/hand_g.urdf.xacro (robot description, xacro)
@@ -1,9 +1,9 @@
 <robot xmlns:sensor="http://playerstage.sourceforge.net/gazebo/xmlschema/#sensor"
-xmlns:controller="http://playerstage.sourceforge.net/gazebo/xmlschema/#controller"
-xmlns:interface="http://playerstage.sourceforge.net/gazebo/xmlschema/#interface"
-xmlns:xacro="http://www.ros.org/wiki/xacro">
-  <xacro:include filename="$(find sr_description)/hand/xacro/forearm/forearm_lite.urdf.xacro" />
+       xmlns:controller="http://playerstage.sourceforge.net/gazebo/xmlschema/#controller"
+       xmlns:interface="http://playerstage.sourceforge.net/gazebo/xmlschema/#interface"
+       xmlns:xacro="http://www.ros.org/wiki/xacro">
+  <xacro:include filename="$(find sr_description)/hand/xacro/forearm/forearm_g.urdf.xacro" />
   <xacro:include filename="$(find sr_description)/hand/xacro/wrist/wrist.urdf.xacro" />
-  <xacro:include filename="$(find sr_description)/hand/xacro/palm/palm_lite.urdf.xacro" />
+  <xacro:include filename="$(find sr_description)/hand/xacro/palm/palm_g.urdf.xacro" />
   <xacro:include filename="$(find sr_description)/hand/xacro/finger/fingers.urdf.xacro" />
   <xacro:include filename="$(find sr_description)/hand/xacro/thumb/thumb.urdf.xacro" />
@@ -14,18 +14,10 @@
   <!-- prox_sensors: plain or dict-like string specifying the proximal (tactile) sensors -->
   <!-- palm_sensor: specifies the palm tactile sensor -->
-  <!-- reflect is either 1 (for right hand) or -1 (for left hand) -->
-  <!-- prefix can be anything but usually is "r_" or  "l_" for right and left hands distinction -->
-  <!-- extra_lite (deprecated) describes if the hand is extra_lite, i.e. without MF -->
-  <!-- muscletrans (deprecated) is true for muscle transmission to be used, false to use motor transmission -->
-  <!-- muscle (deprecated) is true for muscle hand or false for motor hand -->
-  <!-- bio (deprecated) is true for biotac finger or false for standard finger -->
-  <!-- bt_sp (deprecated) is true for BT_SP finger or false for standard finger -->
-  <!-- eli (deprecated) is true for ellipsoid fingertip or false for standard finger -->
-  <xacro:macro name="shadowhand" params="hand_type:='motor' reflect prefix cable_mesh:=False fingers:=all
-          tip_sensors:=pst mid_sensors:=none prox_sensors:=none palm_sensor:=none
-          extra_lite:=^|${None} muscletrans:=^|${None} muscle:=^|${None} bio:=^|${None} bt_sp:=^|${None} eli:=^|${None}">
-    <!-- Unify hand type parameter, also handling deprecated muscletrans, muscle -->
+  <xacro:macro name="sr_hand_e" params="hand_version:=^ reflect:=^ prefix:=^ fingers:=^|all tip_sensors:=^|pst
+               prox_sensors:=^|none mid_sensors:=^|none palm_sensor:=^|none">
+    <!-- Unify hand type parameter -->
+    <xacro:property name="hand_type" value="hand_g" />
     <xacro:include filename="$(find sr_description)/hand/xacro/process_hand_type_parameter.xacro" />
-    <!-- Process fingers parameter, also handling deprecated extra_lite -->
+    <!-- Process fingers parameter, also handling deprecated -->
     <xacro:property name="_all_finger_tokens_" value="${python.set('th ff mf rf'.split())}" />
     <xacro:include filename="$(find sr_description)/hand/xacro/process_fingers_parameter.xacro" />

File: sr_description/hand/xacro/legacy/ff_biotac_hand.urdf.xacro (robot description, xacro)
@@ -2,11 +2,11 @@
   <xacro:macro name="shadowhand" params="muscletrans muscle bio bt_sp eli reflect prefix">
     ${xacro.warning("The file ff_biotac_hand.urdf.xacro is deprecated", print_location=False)}
-    ${xacro.warning("Use full_hand.urdf.xacro instead with tip_sensors='ff=bt_2p'")}
+    ${xacro.warning("Use hand.urdf.xacro instead with tip_sensors='ff=bt_2p'")}
     <!-- translate old parameters to new ones, eventually initializing tip_sensors -->
     <xacro:include filename="$(find sr_description)/hand/xacro/process_sensor_parameters.xacro" />
     <!-- forward to generic macro -->
-    <xacro:include filename="$(find sr_description)/hand/xacro/full_hand.urdf.xacro" />
+    <xacro:include filename="$(find sr_description)/hand/xacro/hand.urdf.xacro" />
     <!-- Enforce BioTac on First Finger -->
-    <xacro:shadowhand fingers="all" reflect="${reflect}" prefix="${prefix}"
+    <xacro:sr_hand fingers="all" reflect="${reflect}" prefix="${prefix}"
     tip_sensors="${' '.join([k+'='+v for k, v in tip_sensors.items()] + ['ff=bt_2p'])}"/>
   </xacro:macro>

File: sr_description/hand/xacro/legacy/hand_E_no_mf_rf.urdf.xacro (robot description, xacro)
@@ -10,8 +10,8 @@
   <xacro:macro name="shadowhand" params="muscletrans muscle bio bt_sp eli reflect prefix lf">
     ${xacro.warning("The file hand_E_no_mf_rf.urdf.xacro is deprecated", print_location=False)}
-    ${xacro.warning("Use full_hand.urdf.xacro instead with fingers='th ff lf'")}
+    ${xacro.warning("Use hand.urdf.xacro instead with fingers='th ff lf'")}
     <!-- forward to generic macro -->
-    <xacro:include filename="$(find sr_description)/hand/xacro/full_hand.urdf.xacro" />
-    <xacro:shadowhand fingers="th ff ${'lf' if lf else ''}" reflect="${reflect}" prefix="${prefix}" />
+    <xacro:include filename="$(find sr_description)/hand/xacro/hand.urdf.xacro" />
+    <xacro:sr_hand fingers="th ff ${'lf' if lf else ''}" reflect="${reflect}" prefix="${prefix}" />
   </xacro:macro>
 </robot>

File: sr_description/hand/xacro/legacy/th_ff_rf_ellipsoid_hand.urdf.xacro (robot description, xacro)
@@ -2,11 +2,11 @@
   <xacro:macro name="shadowhand" params="muscletrans muscle bt_2p bt_sp eli reflect prefix">
     ${xacro.warning("The file th_ff_rf_ellipsoid_hand.urdf.xacro is deprecated", print_location=False)}
-    ${xacro.warning("Use full_hand.urdf.xacro instead with tip_sensors='th=eli ff=eli rf=eli'")}
+    ${xacro.warning("Use hand.urdf.xacro instead with tip_sensors='th=eli ff=eli rf=eli'")}
     <!-- translate old parameters to new ones, eventually initializing tip_sensors -->
     <xacro:include filename="$(find sr_description)/hand/xacro/process_sensor_parameters.xacro" />
     <!-- forward to generic macro -->
-    <xacro:include filename="$(find sr_description)/hand/xacro/full_hand.urdf.xacro" />
+    <xacro:include filename="$(find sr_description)/hand/xacro/hand.urdf.xacro" />
     <!-- Enforce ellipsoid sensor on First and Ring Finger as well as Thumb -->
-    <xacro:shadowhand fingers="all" reflect="${reflect}" prefix="${prefix}"
+    <xacro:sr_hand fingers="all" reflect="${reflect}" prefix="${prefix}"
     tip_sensors="${' '.join([k+'='+v for k, v in tip_sensors.items()] + ['ff=eli','rf=eli','th=eli'])}"/>
   </xacro:macro>

File: sr_description/hand/xacro/legacy/three_biotac_fingers_hand.urdf.xacro (robot description, xacro)
@@ -2,9 +2,9 @@
   <xacro:macro name="shadowhand" params="muscletrans muscle bio bt_sp eli reflect prefix">
     ${xacro.warning("The file three_biotac_fingers_hand.urdf.xacro is deprecated", print_location=False)}
-    ${xacro.warning("Use full_hand.urdf.xacro instead with tip_sensors='th=bt_2p ff=bt_2p mf=bt_2p'")}
+    ${xacro.warning("Use hand.urdf.xacro instead with tip_sensors='th=bt_2p ff=bt_2p mf=bt_2p'")}
     <!-- forward to generic macro -->
-    <xacro:include filename="$(find sr_description)/hand/xacro/full_hand.urdf.xacro" />
+    <xacro:include filename="$(find sr_description)/hand/xacro/hand.urdf.xacro" />
     <!-- BioTacs on First and Middle Finger as well as Thumb -->
-    <xacro:shadowhand reflect="${reflect}" prefix="${prefix}" tip_sensors="th=bt_2p ff=bt_2p mf=bt_2p" />
+    <xacro:sr_hand reflect="${reflect}" prefix="${prefix}" tip_sensors="th=bt_2p ff=bt_2p mf=bt_2p" />
   </xacro:macro>
 </robot>

File: sr_description/hand/xacro/legacy/three_fingers_hand.urdf.xacro (robot description, xacro)
@@ -2,8 +2,8 @@
   <xacro:macro name="shadowhand" params="muscletrans muscle bio bt_sp eli reflect prefix">
     ${xacro.warning("The file three_fingers_hand.urdf.xacro is deprecated", print_location=False)}
-    ${xacro.warning("Use full_hand.urdf.xacro instead with fingers='th ff mf'")}
+    ${xacro.warning("Use hand.urdf.xacro instead with fingers='th ff mf'")}
     <!-- forward to generic macro -->
-    <xacro:include filename="$(find sr_description)/hand/xacro/full_hand.urdf.xacro" />
-    <xacro:shadowhand fingers="th ff mf" reflect="${reflect}" prefix="${prefix}" />
+    <xacro:include filename="$(find sr_description)/hand/xacro/hand.urdf.xacro" />
+    <xacro:sr_hand fingers="th ff mf" reflect="${reflect}" prefix="${prefix}" />
   </xacro:macro>
 </robot>

File: sr_description/hand/xacro/legacy/three_fingers_hand_RF.urdf.xacro (robot description, xacro)
@@ -2,8 +2,8 @@
   <xacro:macro name="shadowhand" params="muscletrans muscle bio bt_sp eli reflect prefix">
     ${xacro.warning("The file three_fingers_hand_RF.urdf.xacro is deprecated", print_location=False)}
-    ${xacro.warning("Use full_hand.urdf.xacro instead with fingers='th ff rf'")}
+    ${xacro.warning("Use hand.urdf.xacro instead with fingers='th ff rf'")}
     <!-- forward to generic macro -->
-    <xacro:include filename="$(find sr_description)/hand/xacro/full_hand.urdf.xacro" />
-    <xacro:shadowhand fingers="th ff rf" reflect="${reflect}" prefix="${prefix}" />
+    <xacro:include filename="$(find sr_description)/hand/xacro/hand.urdf.xacro" />
+    <xacro:sr_hand fingers="th ff rf" reflect="${reflect}" prefix="${prefix}" />
   </xacro:macro>
 </robot>

File: sr_description/robots/bimanual_shadowhand_extra_lite.urdf.xacro (robot description, xacro)
@@ -11,5 +11,5 @@
     <origin xyz="0.0 0.0 0.0" rpy="0.0 0.0 0.0" />
   </joint>
-  <xacro:shadowhand hand_type="motor" fingers="th ff rf" reflect="1.0" prefix="rh_" />
+  <xacro:sr_hand hand_type="motor" fingers="th ff rf" reflect="1.0" prefix="rh_" />
   <joint name="right_hand_to_left_hand" type="fixed">
     <parent link="rh_forearm" />
@@ -17,4 +17,4 @@
     <origin xyz="$(arg arm_x_separation) 0.0 0.0" rpy="0.0 0.0 0.0" />
   </joint>
-  <xacro:shadowhand hand_type="motor" fingers="th ff rf" reflect="-1.0" prefix="lh_" />
+  <xacro:sr_hand hand_type="motor" fingers="th ff rf" reflect="-1.0" prefix="lh_" />
 </robot>

File: sr_description/robots/bimanual_shadowhand_lite.urdf.xacro (robot description, xacro)
@@ -11,5 +11,5 @@
     <origin xyz="0.0 0.0 0.0" rpy="0.0 0.0 0.0" />
   </joint>
-  <xacro:shadowhand hand_type="motor" reflect="1.0" prefix="rh_" />
+  <xacro:sr_hand hand_type="motor" reflect="1.0" prefix="rh_" />
   <joint name="right_hand_to_left_hand" type="fixed">
     <parent link="rh_forearm" />
@@ -17,4 +17,4 @@
     <origin xyz="$(arg arm_x_separation) 0.0 0.0" rpy="0.0 0.0 0.0" />
   </joint>
-  <xacro:shadowhand hand_type="motor" reflect="-1.0" prefix="lh_" />
+  <xacro:sr_hand hand_type="motor" reflect="-1.0" prefix="lh_" />
 </robot>

File: sr_description/robots/bimanual_shadowhand_lite_btsp.urdf.xacro (robot description, xacro)
@@ -11,5 +11,5 @@
     <origin xyz="0.0 0.0 0.0" rpy="0.0 0.0 0.0" />
   </joint>
-  <xacro:shadowhand hand_type="motor" tip_sensors="bt_sp" reflect="1.0" prefix="rh_" />
+  <xacro:sr_hand hand_type="motor" tip_sensors="bt_sp" reflect="1.0" prefix="rh_" />
   <joint name="right_hand_to_left_hand" type="fixed">
     <parent link="rh_forearm" />
@@ -17,4 +17,4 @@
     <origin xyz="$(arg arm_x_separation) 0.0 0.0" rpy="0.0 0.0 0.0" />
   </joint>
-  <xacro:shadowhand hand_type="motor" tip_sensors="bt_sp" reflect="-1.0" prefix="lh_" />
+  <xacro:sr_hand hand_type="motor" tip_sensors="bt_sp" reflect="-1.0" prefix="lh_" />
 </robot>

File: sr_description/robots/bimanual_shadowhand_lite_right_btsp.urdf.xacro (robot description, xacro)
@@ -11,5 +11,5 @@
     <origin xyz="0.0 0.0 0.0" rpy="0.0 0.0 0.0" />
   </joint>
-  <xacro:shadowhand hand_type="motor" tip_sensors="bt_sp" reflect="1.0" prefix="rh_" />
+  <xacro:sr_hand hand_type="motor" tip_sensors="bt_sp" reflect="1.0" prefix="rh_" />
   <joint name="right_hand_to_left_hand" type="fixed">
     <parent link="rh_forearm" />
@@ -17,4 +17,4 @@
     <origin xyz="$(arg arm_x_separation) 0.0 0.0" rpy="0.0 0.0 0.0" />
   </joint>
-  <xacro:shadowhand hand_type="motor" reflect="-1.0" prefix="lh_" />
+  <xacro:sr_hand hand_type="motor" reflect="-1.0" prefix="lh_" />
 </robot>

File: sr_description/robots/bimanual_shadowhand_motor.urdf.xacro (robot description, xacro)
@@ -2,5 +2,5 @@
 name="bimanual_shadowhand_motor">
   <xacro:include filename="$(find sr_description)/materials.urdf.xacro" />
-  <xacro:include filename="$(find sr_description)/hand/xacro/full_hand.urdf.xacro" />
+  <xacro:include filename="$(find sr_description)/hand/xacro/hand.urdf.xacro" />
   <xacro:include filename="$(find sr_description)/other/xacro/gazebo/gazebo.urdf.xacro" />
   <link name="world" />
@@ -10,5 +10,5 @@
     <origin xyz="0.0 0.0 0.0" rpy="0.0 0.0 0.0" />
   </joint>
-  <xacro:shadowhand hand_type="motor" reflect="1.0" prefix="rh_" />
+  <xacro:sr_hand hand_type="motor" reflect="1.0" prefix="rh_" />
   <joint name="right_hand_to_left_hand" type="fixed">
     <parent link="rh_forearm" />
@@ -16,4 +16,4 @@
     <origin xyz="0.4 0.0 0.0" rpy="0.0 0.0 0.0" />
   </joint>
-  <xacro:shadowhand hand_type="motor" reflect="-1.0" prefix="lh_" />
+  <xacro:sr_hand hand_type="motor" reflect="-1.0" prefix="lh_" />
 </robot>

File: sr_description/robots/bimanual_shadowhand_motor_plus.urdf.xacro (robot description, xacro)
@@ -2,5 +2,5 @@
 name="bimanual_shadowhand_motor">
   <xacro:include filename="$(find sr_description)/materials.urdf.xacro" />
-  <xacro:include filename="$(find sr_description)/hand/xacro/full_hand.urdf.xacro" />
+  <xacro:include filename="$(find sr_description)/hand/xacro/hand.urdf.xacro" />
   <xacro:include filename="$(find sr_description)/other/xacro/gazebo/gazebo.urdf.xacro" />
   <link name="world" />
@@ -11,5 +11,5 @@
     <origin xyz="0.0 0.0 0.0" rpy="0.0 0.0 0.0" />
   </joint>
-  <xacro:shadowhand hand_type="motor+" reflect="1.0" prefix="rh_" />
+  <xacro:sr_hand hand_type="motor+" reflect="1.0" prefix="rh_" />
   <joint name="right_hand_to_left_hand" type="fixed">
     <parent link="rh_forearm" />
@@ -17,4 +17,4 @@
     <origin xyz="$(arg arm_x_separation) 0.0 0.0" rpy="0.0 0.0 0.0" />
   </joint>
-  <xacro:shadowhand hand_type="motor+" reflect="-1.0" prefix="lh_" />
+  <xacro:sr_hand hand_type="motor+" reflect="-1.0" prefix="lh_" />
 </robot>

File: sr_description/robots/bimanual_shadowhand_motor_plus_right_biotac.urdf.xacro (robot description, xacro)
@@ -2,5 +2,5 @@
 name="bimanual_shadowhand_motor">
   <xacro:include filename="$(find sr_description)/materials.urdf.xacro" />
-  <xacro:include filename="$(find sr_description)/hand/xacro/full_hand.urdf.xacro" />
+  <xacro:include filename="$(find sr_description)/hand/xacro/hand.urdf.xacro" />
   <xacro:include filename="$(find sr_description)/other/xacro/gazebo/gazebo.urdf.xacro" />
   <link name="world" />
@@ -10,5 +10,5 @@
     <origin xyz="0.0 0.0 0.0" rpy="0.0 0.0 0.0" />
   </joint>
-  <xacro:shadowhand hand_type="motor+" tip_sensors="bt_sp" reflect="1.0" prefix="rh_" />
+  <xacro:sr_hand hand_type="motor+" tip_sensors="bt_sp" reflect="1.0" prefix="rh_" />
   <joint name="right_hand_to_left_hand" type="fixed">
     <parent link="rh_forearm" />
@@ -16,4 +16,4 @@
     <origin xyz="0.4 0.0 0.0" rpy="0.0 0.0 0.0" />
   </joint>
-  <xacro:shadowhand hand_type="motor+" reflect="-1.0" prefix="lh_" />
+  <xacro:sr_hand hand_type="motor+" reflect="-1.0" prefix="lh_" />
 </robot>

File: sr_description/robots/shadowhand_extra_lite.urdf.xacro (robot description, xacro)
@@ -14,4 +14,4 @@
     <origin xyz="0.0 0.0 0.0" rpy="0.0 0.0 0.0" />
   </joint>
-  <xacro:shadowhand hand_type="motor" fingers="th ff rf" reflect="1.0" prefix="rh_" />
+  <xacro:sr_hand hand_type="motor" fingers="th ff rf" reflect="1.0" prefix="rh_" />
 </robot>

File: sr_description/robots/shadowhand_left_extra_lite.urdf.xacro (robot description, xacro)
@@ -14,4 +14,4 @@
     <origin xyz="0.0 0.0 0.0" rpy="0.0 0.0 0.0" />
   </joint>
-  <xacro:shadowhand hand_type="motor" fingers="th ff rf" reflect="-1.0" prefix="lh_" />
+  <xacro:sr_hand hand_type="motor" fingers="th ff rf" reflect="-1.0" prefix="lh_" />
 </robot>

File: sr_description/robots/shadowhand_left_lite.urdf.xacro (robot description, xacro)
@@ -14,4 +14,4 @@
     <origin xyz="0.0 0.0 0.0" rpy="0.0 0.0 0.0" />
   </joint>
-  <xacro:shadowhand hand_type="motor" reflect="-1.0" prefix="lh_" />
+  <xacro:sr_hand hand_type="motor" reflect="-1.0" prefix="lh_" />
 </robot>

File: sr_description/robots/shadowhand_left_lite_btsp.urdf.xacro (robot description, xacro)
@@ -14,4 +14,4 @@
     <origin xyz="0.0 0.0 0.0" rpy="0.0 0.0 0.0" />
   </joint>
-  <xacro:shadowhand hand_type="motor" tip_sensors="bt_sp" reflect="-1.0" prefix="lh_" />
+  <xacro:sr_hand hand_type="motor" tip_sensors="bt_sp" reflect="-1.0" prefix="lh_" />
 </robot>

File: sr_description/robots/shadowhand_left_motor.urdf.xacro (robot description, xacro)
@@ -5,5 +5,5 @@
 name="shadowhand_motor">
   <xacro:include filename="$(find sr_description)/materials.urdf.xacro" />
-  <xacro:include filename="$(find sr_description)/hand/xacro/full_hand.urdf.xacro" />
+  <xacro:include filename="$(find sr_description)/hand/xacro/hand.urdf.xacro" />
   <xacro:include filename="$(find sr_description)/other/xacro/gazebo/gazebo.urdf.xacro" />
   <!-- hand with cylindrical base drifts in gazebo, attach it to the world -->
@@ -14,4 +14,4 @@
     <origin xyz="0.0 0.0 0.0" rpy="0.0 0.0 0.0" />
   </joint>
-  <xacro:shadowhand hand_type="motor" reflect="-1.0" prefix="lh_" />
+  <xacro:sr_hand hand_type="motor" reflect="-1.0" prefix="lh_" />
 </robot>
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
Commit message: Fixing relative lfknuckle position (model was wrongly describing it 0.1mm closer to lfmetacarpal

File: sr_description/hand/xacro/hand_e.urdf.xacro (robot description, xacro)
@@ -80,5 +80,5 @@
       <xacro:finger link_prefix="lf" joint_prefix="LF" tip_sensor="${tip_sensors.lf}" prox_sensor="${prox_sensors.lf}"
                     mid_sensor="${mid_sensors.lf}" parent="${prefix}palm">
-        <origin xyz="${reflect*0.05389084} 0 0.03773727" rpy="0 ${reflect*0.9599} 0" />
+        <origin xyz="${reflect*0.05397275} 0 0.03779463" rpy="0 ${reflect*0.9599} 0" />
         <axis xyz="0 ${reflect} 0" />
       </xacro:finger>
