Commit message: Update process_hand_type_version_side_parameters.xacro

File: sr_description/hand/xacro/process_hand_type_version_side_parameters.xacro (robot description, xacro)
@@ -3,5 +3,5 @@
 	<xacro:property name="allowed_hand_types" value="${python.set('hand_e hand_g hand_c'.split())}" />
 	<xacro:property name="allowed_hand_versions" value="${python.set('E3M5 E2M3 C6M2 G1M5'.split())}"/>
-  <xacro:property name="allowed_sides" value="${python.set('right left'.split())}"/>
+        <xacro:property name="allowed_sides" value="${python.set('right left'.split())}"/>
 	<!-- Validate hand type -->
 	<xacro:validate_tokens tokens="${python.set([hand_type])}" valid="${allowed_hand_types}" name="hand type specifier" />
@@ -11,6 +11,6 @@
 	<xacro:validate_tokens tokens="${python.set([side])}" valid="${allowed_sides}" name="hand side specifier" />
 	<xacro:unless value="${hand_type.lower()[-1] == hand_version.lower()[0]}">
-    ${xacro.error("Parameter 'hand_type' ("+hand_type+") doesn't comply with 'hand_version' ("+hand_version+")")}
-  </xacro:unless>
+            ${xacro.error("Parameter 'hand_type' ("+hand_type+") doesn't comply with 'hand_version' ("+hand_version+")")}
+        </xacro:unless>
 	<!-- Normalize hand_type to be lower case -->
 	<xacro:property name="hand_type" value="${hand_type.lower()}" lazy_eval="false" />

Commit message: Changing arm to mounting plate

File: sr_description/hand/xacro/process_hand_type_version_side_parameters.xacro (robot description, xacro)
@@ -4,5 +4,5 @@
 	<xacro:property name="allowed_hand_versions" value="${python.set('E3M5 E2M3 C6M2 G1M5'.split())}"/>
     <xacro:property name="allowed_sides" value="${python.set('right left'.split())}"/>
-    <xacro:property name="allowed_mounting_plate" value="${python.set('false true'.split())}"/>
+    <!--xacro:property name="allowed_mounting_plate" value="${python.set('false true'.split())}"/-->
 	<!-- Validate hand type -->
 	<xacro:validate_tokens tokens="${python.set([hand_type])}" valid="${allowed_hand_types}" name="hand type specifier" />
@@ -16,5 +16,5 @@
 	<xacro:validate_tokens tokens="${python.set([side])}" valid="${allowed_sides}" name="hand side specifier" />
     <!-- Validate mounting plate options -->
-    <xacro:validate_tokens tokens="${python.set([mounting_plate])}" valid="${allowed_mounting_plate}" name="hand mounting_plate specifier" />
+    <!--xacro:validate_tokens tokens="${python.set([mounting_plate])}" valid="${allowed_mounting_plate}" name="hand mounting_plate specifier" /-->
 	<!-- Normalize hand_type to be lower case -->
 	<xacro:property name="hand_type" value="${hand_type.lower()}" lazy_eval="false" />

Commit message: validate boolean mounting plate var

File: sr_description/hand/xacro/process_hand_type_version_side_parameters.xacro (robot description, xacro)
@@ -4,5 +4,5 @@
 	<xacro:property name="allowed_hand_versions" value="${python.set('E3M5 E2M3 C6M2 G1M5'.split())}"/>
     <xacro:property name="allowed_sides" value="${python.set('right left'.split())}"/>
-    <!--xacro:property name="allowed_mounting_plate" value="${python.set('false true'.split())}"/-->
+    <xacro:property name="allowed_mounting_plate" value="${python.set([False, True])}"/>
 	<!-- Validate hand type -->
 	<xacro:validate_tokens tokens="${python.set([hand_type])}" valid="${allowed_hand_types}" name="hand type specifier" />
@@ -16,5 +16,5 @@
 	<xacro:validate_tokens tokens="${python.set([side])}" valid="${allowed_sides}" name="hand side specifier" />
     <!-- Validate mounting plate options -->
-    <!--xacro:validate_tokens tokens="${python.set([mounting_plate])}" valid="${allowed_mounting_plate}" name="hand mounting_plate specifier" /-->
+    <xacro:validate_tokens tokens="${python.set([mounting_plate])}" valid="${allowed_mounting_plate}" name="hand mounting_plate specifier" />
 	<!-- Normalize hand_type to be lower case -->
 	<xacro:property name="hand_type" value="${hand_type.lower()}" lazy_eval="false" />

Commit message: Update process_hand_type_version_side_parameters.xacro

File: sr_description/hand/xacro/process_hand_type_version_side_parameters.xacro (robot description, xacro)
@@ -3,18 +3,18 @@
 	<xacro:property name="allowed_hand_types" value="${python.set('hand_e hand_g hand_c'.split())}" />
 	<xacro:property name="allowed_hand_versions" value="${python.set('E3M5 E2M3 C6M2 G1M5'.split())}"/>
-    <xacro:property name="allowed_sides" value="${python.set('right left'.split())}"/>
-    <xacro:property name="allowed_mounting_plate" value="${python.set([False, True])}"/>
+        <xacro:property name="allowed_sides" value="${python.set('right left'.split())}"/>
+        <xacro:property name="allowed_mounting_plate" value="${python.set([False, True])}"/>
 	<!-- Validate hand type -->
 	<xacro:validate_tokens tokens="${python.set([hand_type])}" valid="${allowed_hand_types}" name="hand type specifier" />
 	<!-- Validate hand version -->
 	<xacro:validate_tokens tokens="${python.set([hand_version])}" valid="${allowed_hand_versions}" name="hand version specifier" />
-    <!-- Validate hand version corresponds to hand type -->
+        <!-- Validate hand version corresponds to hand type -->
 	<xacro:unless value="${hand_type.lower()[-1] == hand_version.lower()[0]}">
-        ${xacro.error("Parameter 'hand_type' ("+hand_type+") doesn't comply with 'hand_version' ("+hand_version+")")}
-    </xacro:unless>
+        	${xacro.error("Parameter 'hand_type' ("+hand_type+") doesn't comply with 'hand_version' ("+hand_version+")")}
+        </xacro:unless>
 	<!-- Validate side -->
 	<xacro:validate_tokens tokens="${python.set([side])}" valid="${allowed_sides}" name="hand side specifier" />
-    <!-- Validate mounting plate options -->
-    <xacro:validate_tokens tokens="${python.set([mounting_plate])}" valid="${allowed_mounting_plate}" name="hand mounting_plate specifier" />
+        <!-- Validate mounting plate options -->
+        <xacro:validate_tokens tokens="${python.set([mounting_plate])}" valid="${allowed_mounting_plate}" name="hand mounting_plate specifier" />
 	<!-- Normalize hand_type to be lower case -->
 	<xacro:property name="hand_type" value="${hand_type.lower()}" lazy_eval="false" />

Commit message: Adding E4 to the list of correct options

File: sr_description/hand/xacro/process_hand_type_version_side_parameters.xacro (robot description, xacro)
@@ -27,5 +27,5 @@
 	<xacro:include filename="$(find sr_description)/hand/xacro/validate_macros.xacro" />
 	<xacro:property name="allowed_hand_types" value="${python.set('hand_e hand_g hand_c'.split())}" />
-	<xacro:property name="allowed_hand_versions" value="${python.set('E3M5 E2M3 C6M2 G1M5'.split())}"/>
+	<xacro:property name="allowed_hand_versions" value="${python.set('E4 E3M5 E2M3 C6M2 G1M5'.split())}"/>
         <xacro:property name="allowed_sides" value="${python.set('right left'.split())}"/>
         <xacro:property name="allowed_mounting_plate" value="${python.set([False, True])}"/>

Commit message: Adding E4 to the list of correct options (#157)
* Adding E4 to the list of correct options

* Update process_hand_type_version_side_parameters.xacro

File: sr_description/hand/xacro/process_hand_type_version_side_parameters.xacro (robot description, xacro)
@@ -2,5 +2,5 @@
 <!--
  Software License Agreement (BSD License)
- Copyright © 2022 belongs to Shadow Robot Company Ltd.
+ Copyright © 2022-2023 belongs to Shadow Robot Company Ltd.
  All rights reserved.
  Redistribution and use in source and binary forms, with or without modification,
@@ -27,5 +27,5 @@
 	<xacro:include filename="$(find sr_description)/hand/xacro/validate_macros.xacro" />
 	<xacro:property name="allowed_hand_types" value="${python.set('hand_e hand_g hand_c'.split())}" />
-	<xacro:property name="allowed_hand_versions" value="${python.set('E3M5 E2M3 C6M2 G1M5'.split())}"/>
+	<xacro:property name="allowed_hand_versions" value="${python.set('E4 E3M5 E2M3 C6M2 G1M5'.split())}"/>
         <xacro:property name="allowed_sides" value="${python.set('right left'.split())}"/>
         <xacro:property name="allowed_mounting_plate" value="${python.set([False, True])}"/>
