Commit message: updating all transmissions to new type

File: sr_description/hand/xacro/finger/distal/distal.transmission.xacro (robot description, xacro)
@@ -11,17 +11,27 @@
    <!-- muscle hand -->
     <xacro:if value="${muscletrans}">
-      <transmission type="sr_mechanism_model/SimpleTransmissionForMuscle" name="${prefix}${link_prefix}distal_transmission">
-      <actuator name="${prefix}${joint_prefix}J1" />
-      <joint name="${prefix}${joint_prefix}J1" />
-      <mechanicalReduction>1</mechanicalReduction>
-      </transmission>
+        <transmission name="${prefix}${link_prefix}distal_transmission">
+            <type>sr_mechanism_model/SimpleTransmissionForMuscle</type>
+            <actuator name="${prefix}${joint_prefix}J1">
+                <mechanicalReduction>1</mechanicalReduction>
+            </actuator>
+            <joint name="${prefix}${joint_prefix}J1">
+                <hardwareInterface>EffortJointInterface</hardwareInterface>
+                <hardwareInterface>PositionJointInterface</hardwareInterface>
+            </joint>
+        </transmission>
     </xacro:if>
     <!-- motor hand -->
     <xacro:unless value="${muscletrans}">
-      <transmission type="sr_mechanism_model/SimpleTransmission" name="${prefix}${link_prefix}distal_transmission">
-      <actuator name="${prefix}${joint_prefix}J1" />
-      <joint name="${prefix}${joint_prefix}J1" />
-      <mechanicalReduction>1</mechanicalReduction>
-      </transmission>
+        <transmission name="${prefix}${link_prefix}distal_transmission">
+            <type>sr_mechanism_model/SimpleTransmission</type>
+            <actuator name="${prefix}${joint_prefix}J1">
+                <mechanicalReduction>1</mechanicalReduction>
+            </actuator>
+            <joint name="${prefix}${joint_prefix}J1">
+                <hardwareInterface>EffortJointInterface</hardwareInterface>
+                <hardwareInterface>PositionJointInterface</hardwareInterface>
+            </joint>
+        </transmission>
     </xacro:unless>
   </xacro:macro>

File: sr_description/hand/xacro/finger/knuckle/knuckle.transmission.xacro (robot description, xacro)
@@ -4,30 +4,35 @@
        xmlns:interface="http://playerstage.sourceforge.net/gazebo/xmlschema/#interface"
        xmlns:xacro="http://www.ros.org/wiki/xacro">
-  <!-- muscletrans is true for muscle transmission or false for motor transmission -->
-  <!-- prefix can be anything but usually is "r_" or  "l_" for right and left hands distinction -->
-  <!-- link_prefix prepends fingername to the link names -->
-  <!-- joint_prefix prepends fingername to the joint names -->
-  <xacro:macro name="knuckle_transmission" params="muscletrans prefix joint_prefix link_prefix" >
-   <!-- muscle hand -->
-    <xacro:if value="${muscletrans}">
-      <transmission type="sr_mechanism_model/SimpleTransmissionForMuscle" name="${prefix}${link_prefix}knuckle_transmission">
-      <actuator name="${prefix}${joint_prefix}J4" />
-      <joint name="${prefix}${joint_prefix}J4" />
-      <mechanicalReduction>1</mechanicalReduction>
-      </transmission>
-    </xacro:if>
-    <!-- motor hand -->
-    <xacro:unless value="${muscletrans}">
-      <transmission name="${prefix}${link_prefix}knuckle_transmission">
-        <type>sr_mechanism_model/SimpleTransmission</type>
-      <actuator name="${prefix}${joint_prefix}J4">
-        <mechanicalReduction>1</mechanicalReduction>
-      </actuator>
-      <joint name="${prefix}${joint_prefix}J4">
-        <hardwareInterface>EffortJointInterface</hardwareInterface>
-        <hardwareInterface>PositionJointInterface</hardwareInterface>
-      </joint>
-      </transmission>
-    </xacro:unless>
-  </xacro:macro>
+    <!-- muscletrans is true for muscle transmission or false for motor transmission -->
+    <!-- prefix can be anything but usually is "r_" or  "l_" for right and left hands distinction -->
+    <!-- link_prefix prepends fingername to the link names -->
+    <!-- joint_prefix prepends fingername to the joint names -->
+    <xacro:macro name="knuckle_transmission" params="muscletrans prefix joint_prefix link_prefix">
+        <!-- muscle hand -->
+        <xacro:if value="${muscletrans}">
+            <transmission name="${prefix}${link_prefix}knuckle_transmission">
+                <type>sr_mechanism_model/SimpleTransmissionForMuscle</type>
+                <actuator name="${prefix}${joint_prefix}J4">
+                    <mechanicalReduction>1</mechanicalReduction>
+                </actuator>
+                <joint name="${prefix}${joint_prefix}J4">
+                    <hardwareInterface>EffortJointInterface</hardwareInterface>
+                    <hardwareInterface>PositionJointInterface</hardwareInterface>
+                </joint>
+            </transmission>
+        </xacro:if>
+        <!-- motor hand -->
+        <xacro:unless value="${muscletrans}">
+            <transmission name="${prefix}${link_prefix}knuckle_transmission">
+                <type>sr_mechanism_model/SimpleTransmission</type>
+                <actuator name="${prefix}${joint_prefix}J4">
+                    <mechanicalReduction>1</mechanicalReduction>
+                </actuator>
+                <joint name="${prefix}${joint_prefix}J4">
+                    <hardwareInterface>EffortJointInterface</hardwareInterface>
+                    <hardwareInterface>PositionJointInterface</hardwareInterface>
+                </joint>
+            </transmission>
+        </xacro:unless>
+    </xacro:macro>
 </robot>

File: sr_description/hand/xacro/finger/lfmetacarpal/lfmetacarpal.transmission.xacro (robot description, xacro)
@@ -4,28 +4,33 @@
        xmlns:interface="http://playerstage.sourceforge.net/gazebo/xmlschema/#interface"
        xmlns:xacro="http://www.ros.org/wiki/xacro">
-  <!-- muscletrans is true for muscle transmission or false for motor transmission -->
-  <!-- prefix can be anything but usually is "r_" or  "l_" for right and left hands distinction -->
-  <xacro:macro name="lfmetacarpal_transmission" params="muscletrans prefix" >
-   <!-- muscle hand -->
-    <xacro:if value="${muscletrans}">
-      <transmission type="sr_mechanism_model/SimpleTransmissionForMuscle" name="${prefix}lfmetacarpal_transmission">
-      <actuator name="${prefix}LFJ5" />
-      <joint name="${prefix}LFJ5" />
-      <mechanicalReduction>1</mechanicalReduction>
-      </transmission>
-    </xacro:if>
-    <!-- motor hand -->
-    <xacro:unless value="${muscletrans}">
-      <transmission name="${prefix}lfmetacarpal_transmission">
-        <type>sr_mechanism_model/SimpleTransmission</type>
-      <actuator name="${prefix}LFJ5">
-        <mechanicalReduction>1</mechanicalReduction>
-      </actuator>
-      <joint name="${prefix}LFJ5">
-        <hardwareInterface>EffortJointInterface</hardwareInterface>
-        <hardwareInterface>PositionJointInterface</hardwareInterface>
-      </joint>
-      </transmission>
-    </xacro:unless>
-  </xacro:macro>
+    <!-- muscletrans is true for muscle transmission or false for motor transmission -->
+    <!-- prefix can be anything but usually is "r_" or  "l_" for right and left hands distinction -->
+    <xacro:macro name="lfmetacarpal_transmission" params="muscletrans prefix">
+        <!-- muscle hand -->
+        <xacro:if value="${muscletrans}">
+            <transmission name="${prefix}lfmetacarpal_transmission">
+                <type>sr_mechanism_model/SimpleTransmissionForMuscle</type>
+                <actuator name="${prefix}LFJ5">
+                    <mechanicalReduction>1</mechanicalReduction>
+                </actuator>
+                <joint name="${prefix}LFJ5">
+                    <hardwareInterface>EffortJointInterface</hardwareInterface>
+                    <hardwareInterface>PositionJointInterface</hardwareInterface>
+                </joint>
+            </transmission>
+        </xacro:if>
+        <!-- motor hand -->
+        <xacro:unless value="${muscletrans}">
+            <transmission name="${prefix}lfmetacarpal_transmission">
+                <type>sr_mechanism_model/SimpleTransmission</type>
+                <actuator name="${prefix}LFJ5">
+                    <mechanicalReduction>1</mechanicalReduction>
+                </actuator>
+                <joint name="${prefix}LFJ5">
+                    <hardwareInterface>EffortJointInterface</hardwareInterface>
+                    <hardwareInterface>PositionJointInterface</hardwareInterface>
+                </joint>
+            </transmission>
+        </xacro:unless>
+    </xacro:macro>
 </robot>

File: sr_description/hand/xacro/finger/middle/middle.transmission.xacro (robot description, xacro)
@@ -4,32 +4,41 @@
        xmlns:interface="http://playerstage.sourceforge.net/gazebo/xmlschema/#interface"
        xmlns:xacro="http://www.ros.org/wiki/xacro">
-  <!-- muscletrans is true for muscle transmission or false for motor transmission -->
-  <!-- prefix can be anything but usually is "r_" or  "l_" for right and left hands distinction -->
-  <!-- link_prefix prepends fingername to the link names -->
-  <!-- joint_prefix prepends fingername to the joint names -->
-  <xacro:macro name="middle_transmission" params="muscletrans prefix joint_prefix link_prefix" >
-   <!-- muscle hand -->
-    <xacro:if value="${muscletrans}">
-      <transmission type="sr_mechanism_model/J0TransmissionForMuscle" name="${prefix}${link_prefix}middle_transmission">
-      <actuator name="${prefix}${joint_prefix}J0" />
-      <joint name="${prefix}${joint_prefix}J1" />
-      <joint name="${prefix}${joint_prefix}J2" />
-      <mechanicalReduction>1</mechanicalReduction>
-      </transmission>
-    </xacro:if>
-    <!-- motor hand -->
-    <xacro:unless value="${muscletrans}">
-      <transmission name="${prefix}${link_prefix}middle_transmission">
-        <type>sr_mechanism_model/J0Transmission</type>
-        <actuator name="${prefix}${joint_prefix}J0">
-          <mechanicalReduction>1</mechanicalReduction>
-        </actuator>
-        <joint name="${prefix}${joint_prefix}J1">
-          <hardwareInterface>EffortJointInterface</hardwareInterface>
-          <hardwareInterface>PositionJointInterface</hardwareInterface>
-        </joint>
-        <secondJoint name="${prefix}${joint_prefix}J2" />
-      </transmission>
-    </xacro:unless>
-  </xacro:macro>
+    <!-- muscletrans is true for muscle transmission or false for motor transmission -->
+    <!-- prefix can be anything but usually is "r_" or  "l_" for right and left hands distinction -->
+    <!-- link_prefix prepends fingername to the link names -->
+    <!-- joint_prefix prepends fingername to the joint names -->
+    <xacro:macro name="middle_transmission" params="muscletrans prefix joint_prefix link_prefix">
+        <!-- muscle hand -->
+        <xacro:if value="${muscletrans}">
+            <transmission name="${prefix}${link_prefix}middle_transmission">
+                <type>sr_mechanism_model/J0TransmissionForMuscle</type>
+                <actuator name="${prefix}${joint_prefix}J0">
+                    <mechanicalReduction>1</mechanicalReduction>
+                </actuator>
+                <joint name="${prefix}${joint_prefix}J1">
+                    <hardwareInterface>EffortJointInterface</hardwareInterface>
+                    <hardwareInterface>PositionJointInterface</hardwareInterface>
+                </joint>
+                <joint name="${prefix}${joint_prefix}J2">
+                    <hardwareInterface>EffortJointInterface</hardwareInterface>
+                    <hardwareInterface>PositionJointInterface</hardwareInterface>
+                </joint>
+                <mechanicalReduction>1</mechanicalReduction>
+            </transmission>
+        </xacro:if>
+        <!-- motor hand -->
+        <xacro:unless value="${muscletrans}">
+            <transmission name="${prefix}${link_prefix}middle_transmission">
+                <type>sr_mechanism_model/J0Transmission</type>
+                <actuator name="${prefix}${joint_prefix}J0">
+                    <mechanicalReduction>1</mechanicalReduction>
+                </actuator>
+                <joint name="${prefix}${joint_prefix}J1">
+                    <hardwareInterface>EffortJointInterface</hardwareInterface>
+                    <hardwareInterface>PositionJointInterface</hardwareInterface>
+                </joint>
+                <secondJoint name="${prefix}${joint_prefix}J2"/>
+            </transmission>
+        </xacro:unless>
+    </xacro:macro>
 </robot>

File: sr_description/hand/xacro/finger/proximal/proximal.transmission.xacro (robot description, xacro)
@@ -4,30 +4,35 @@
        xmlns:interface="http://playerstage.sourceforge.net/gazebo/xmlschema/#interface"
        xmlns:xacro="http://www.ros.org/wiki/xacro">
-  <!-- muscletrans is true for muscle transmission or false for motor transmission -->
-  <!-- prefix can be anything but usually is "r_" or  "l_" for right and left hands distinction -->
-  <!-- link_prefix prepends fingername to the link names -->
-  <!-- joint_prefix prepends fingername to the joint names -->
-  <xacro:macro name="proximal_transmission" params="muscletrans prefix joint_prefix link_prefix" >
-   <!-- muscle hand -->
-    <xacro:if value="${muscletrans}">
-      <transmission type="sr_mechanism_model/SimpleTransmissionForMuscle" name="${prefix}${link_prefix}proximal_transmission">
-      <actuator name="${prefix}${joint_prefix}J3" />
-      <joint name="${prefix}${joint_prefix}J3" />
-      <mechanicalReduction>1</mechanicalReduction>
-      </transmission>
-    </xacro:if>
-    <!-- motor hand -->
-    <xacro:unless value="${muscletrans}">
-      <transmission name="${prefix}${link_prefix}proximal_transmission">
-        <type>sr_mechanism_model/SimpleTransmission</type>
-      <actuator name="${prefix}${joint_prefix}J3">
-        <mechanicalReduction>1</mechanicalReduction>
-      </actuator>
-      <joint name="${prefix}${joint_prefix}J3">
-        <hardwareInterface>EffortJointInterface</hardwareInterface>
-        <hardwareInterface>PositionJointInterface</hardwareInterface>
-      </joint>
-      </transmission>
-    </xacro:unless>
-  </xacro:macro>
+    <!-- muscletrans is true for muscle transmission or false for motor transmission -->
+    <!-- prefix can be anything but usually is "r_" or  "l_" for right and left hands distinction -->
+    <!-- link_prefix prepends fingername to the link names -->
+    <!-- joint_prefix prepends fingername to the joint names -->
+    <xacro:macro name="proximal_transmission" params="muscletrans prefix joint_prefix link_prefix">
+        <!-- muscle hand -->
+        <xacro:if value="${muscletrans}">
+            <transmission name="${prefix}${link_prefix}proximal_transmission">
+                <type>sr_mechanism_model/SimpleTransmissionForMuscle</type>
+                <actuator name="${prefix}${joint_prefix}J3">
+                    <mechanicalReduction>1</mechanicalReduction>
+                </actuator>
+                <joint name="${prefix}${joint_prefix}J3">
+                    <hardwareInterface>EffortJointInterface</hardwareInterface>
+                    <hardwareInterface>PositionJointInterface</hardwareInterface>
+                </joint>
+            </transmission>
+        </xacro:if>
+        <!-- motor hand -->
+        <xacro:unless value="${muscletrans}">
+            <transmission name="${prefix}${link_prefix}proximal_transmission">
+                <type>sr_mechanism_model/SimpleTransmission</type>
+                <actuator name="${prefix}${joint_prefix}J3">
+                    <mechanicalReduction>1</mechanicalReduction>
+                </actuator>
+                <joint name="${prefix}${joint_prefix}J3">
+                    <hardwareInterface>EffortJointInterface</hardwareInterface>
+                    <hardwareInterface>PositionJointInterface</hardwareInterface>
+                </joint>
+            </transmission>
+        </xacro:unless>
+    </xacro:macro>
 </robot>

File: sr_description/hand/xacro/palm/palm.transmission.xacro (robot description, xacro)
@@ -4,28 +4,33 @@
        xmlns:interface="http://playerstage.sourceforge.net/gazebo/xmlschema/#interface"
        xmlns:xacro="http://www.ros.org/wiki/xacro">
-  <!-- muscletrans is true for muscle transmission or false for motor transmission -->
-  <!-- prefix can be anything but usually is "r_" or  "l_" for right and left hands distinction -->
-  <xacro:macro name="shadowhand_palm_transmission" params="muscletrans prefix" >
-   <!-- muscle hand -->
-    <xacro:if value="${muscletrans}">
-      <transmission type="sr_mechanism_model/SimpleTransmissionForMuscle" name="${prefix}palm_transmission">
-      <actuator name="${prefix}WRJ1" />
-      <joint name="${prefix}WRJ1" />
-      <mechanicalReduction>1</mechanicalReduction>
-      </transmission>
-    </xacro:if>
-    <!-- motor hand -->
-    <xacro:unless value="${muscletrans}">
-      <transmission name="${prefix}palm_transmission">
-        <type>sr_mechanism_model/SimpleTransmission</type>
-        <actuator name="${prefix}WRJ1">
-          <mechanicalReduction>1</mechanicalReduction>
-        </actuator>
-        <joint name="${prefix}WRJ1">
-          <hardwareInterface>EffortJointInterface</hardwareInterface>
-          <hardwareInterface>PositionJointInterface</hardwareInterface>
-        </joint>
-      </transmission>
-    </xacro:unless>
-  </xacro:macro>
+    <!-- muscletrans is true for muscle transmission or false for motor transmission -->
+    <!-- prefix can be anything but usually is "r_" or  "l_" for right and left hands distinction -->
+    <xacro:macro name="shadowhand_palm_transmission" params="muscletrans prefix">
+        <!-- muscle hand -->
+        <xacro:if value="${muscletrans}">
+            <transmission name="${prefix}palm_transmission">
+                <type>sr_mechanism_model/SimpleTransmissionForMuscle</type>
+                <actuator name="${prefix}WRJ1">
+                    <mechanicalReduction>1</mechanicalReduction>
+                </actuator>
+                <joint name="${prefix}WRJ1">
+                    <hardwareInterface>EffortJointInterface</hardwareInterface>
+                    <hardwareInterface>PositionJointInterface</hardwareInterface>
+                </joint>
+            </transmission>
+        </xacro:if>
+        <!-- motor hand -->
+        <xacro:unless value="${muscletrans}">
+            <transmission name="${prefix}palm_transmission">
+                <type>sr_mechanism_model/SimpleTransmission</type>
+                <actuator name="${prefix}WRJ1">
+                    <mechanicalReduction>1</mechanicalReduction>
+                </actuator>
+                <joint name="${prefix}WRJ1">
+                    <hardwareInterface>EffortJointInterface</hardwareInterface>
+                    <hardwareInterface>PositionJointInterface</hardwareInterface>
+                </joint>
+            </transmission>
+        </xacro:unless>
+    </xacro:macro>
 </robot>

File: sr_description/hand/xacro/thumb/thbase.transmission.xacro (robot description, xacro)
@@ -4,28 +4,33 @@
        xmlns:interface="http://playerstage.sourceforge.net/gazebo/xmlschema/#interface"
        xmlns:xacro="http://www.ros.org/wiki/xacro">
-  <!-- muscletrans is true for muscle transmission or false for motor transmission -->
-  <!-- prefix can be anything but usually is "r_" or  "l_" for right and left hands distinction -->
-  <xacro:macro name="thbase_transmission" params="muscletrans prefix" >
-   <!-- muscle hand -->
-    <xacro:if value="${muscletrans}">
-      <transmission type="sr_mechanism_model/SimpleTransmissionForMuscle" name="${prefix}thbase_transmission">
-      <actuator name="${prefix}THJ5" />
-      <joint name="${prefix}THJ5" />
-      <mechanicalReduction>1</mechanicalReduction>
-      </transmission>
-    </xacro:if>
-    <!-- motor hand -->
-    <xacro:unless value="${muscletrans}">
-      <transmission name="${prefix}thbase_transmission">
-        <type>sr_mechanism_model/SimpleTransmission</type>
-        <actuator name="${prefix}THJ5">
-          <mechanicalReduction>1</mechanicalReduction>
-        </actuator>
-        <joint name="${prefix}THJ5">
-          <hardwareInterface>EffortJointInterface</hardwareInterface>
-          <hardwareInterface>PositionJointInterface</hardwareInterface>
-        </joint>
-      </transmission>
-    </xacro:unless>
-  </xacro:macro>
+    <!-- muscletrans is true for muscle transmission or false for motor transmission -->
+    <!-- prefix can be anything but usually is "r_" or  "l_" for right and left hands distinction -->
+    <xacro:macro name="thbase_transmission" params="muscletrans prefix">
+        <!-- muscle hand -->
+        <xacro:if value="${muscletrans}">
+            <transmission name="${prefix}thbase_transmission">
+                <type>sr_mechanism_model/SimpleTransmissionForMuscle</type>
+                <actuator name="${prefix}THJ5">
+                    <mechanicalReduction>1</mechanicalReduction>
+                </actuator>
+                <joint name="${prefix}THJ5">
+                    <hardwareInterface>EffortJointInterface</hardwareInterface>
+                    <hardwareInterface>PositionJointInterface</hardwareInterface>
+                </joint>
+            </transmission>
+        </xacro:if>
+        <!-- motor hand -->
+        <xacro:unless value="${muscletrans}">
+            <transmission name="${prefix}thbase_transmission">
+                <type>sr_mechanism_model/SimpleTransmission</type>
+                <actuator name="${prefix}THJ5">
+                    <mechanicalReduction>1</mechanicalReduction>
+                </actuator>
+                <joint name="${prefix}THJ5">
+                    <hardwareInterface>EffortJointInterface</hardwareInterface>
+                    <hardwareInterface>PositionJointInterface</hardwareInterface>
+                </joint>
+            </transmission>
+        </xacro:unless>
+    </xacro:macro>
 </robot>
