Commit message: updating all transmissions to new type

File: sr_description/hand/xacro/thumb/thdistal.transmission.xacro (robot description, xacro)
@@ -4,28 +4,33 @@
        xmlns:interface="http://playerstage.sourceforge.net/gazebo/xmlschema/#interface"
        xmlns:xacro="http://www.ros.org/wiki/xacro">
-  <!-- muscletrans is true for muscle transmission or false for motor transmission -->
-  <!-- prefix can be anything but usually is "r_" or  "l_" for right and left hands distinction -->
-  <xacro:macro name="thdistal_transmission" params="muscletrans prefix" >
-   <!-- muscle hand -->
-    <xacro:if value="${muscletrans}">
-      <transmission type="sr_mechanism_model/SimpleTransmissionForMuscle" name="${prefix}thdistal_transmission">
-      <actuator name="${prefix}THJ1" />
-      <joint name="${prefix}THJ1" />
-      <mechanicalReduction>1</mechanicalReduction>
-      </transmission>
-    </xacro:if>
-    <!-- motor hand -->
-    <xacro:unless value="${muscletrans}">
-      <transmission name="${prefix}thdistal_transmission">
-        <type>sr_mechanism_model/SimpleTransmission</type>
-        <actuator name="${prefix}THJ1">
-          <mechanicalReduction>1</mechanicalReduction>
-        </actuator>
-        <joint name="${prefix}THJ1">
-          <hardwareInterface>EffortJointInterface</hardwareInterface>
-          <hardwareInterface>PositionJointInterface</hardwareInterface>
-        </joint>
-      </transmission>
-    </xacro:unless>
-  </xacro:macro>
-  </robot>
+    <!-- muscletrans is true for muscle transmission or false for motor transmission -->
+    <!-- prefix can be anything but usually is "r_" or  "l_" for right and left hands distinction -->
+    <xacro:macro name="thdistal_transmission" params="muscletrans prefix">
+        <!-- muscle hand -->
+        <xacro:if value="${muscletrans}">
+            <transmission name="${prefix}thdistal_transmission">
+                <type>sr_mechanism_model/SimpleTransmissionForMuscle</type>
+                <actuator name="${prefix}THJ1">
+                    <mechanicalReduction>1</mechanicalReduction>
+                </actuator>
+                <joint name="${prefix}THJ1">
+                    <hardwareInterface>EffortJointInterface</hardwareInterface>
+                    <hardwareInterface>PositionJointInterface</hardwareInterface>
+                </joint>
+            </transmission>
+        </xacro:if>
+        <!-- motor hand -->
+        <xacro:unless value="${muscletrans}">
+            <transmission name="${prefix}thdistal_transmission">
+                <type>sr_mechanism_model/SimpleTransmission</type>
+                <actuator name="${prefix}THJ1">
+                    <mechanicalReduction>1</mechanicalReduction>
+                </actuator>
+                <joint name="${prefix}THJ1">
+                    <hardwareInterface>EffortJointInterface</hardwareInterface>
+                    <hardwareInterface>PositionJointInterface</hardwareInterface>
+                </joint>
+            </transmission>
+        </xacro:unless>
+    </xacro:macro>
+</robot>

File: sr_description/hand/xacro/thumb/thhub.transmission.xacro (robot description, xacro)
@@ -4,28 +4,33 @@
        xmlns:interface="http://playerstage.sourceforge.net/gazebo/xmlschema/#interface"
        xmlns:xacro="http://www.ros.org/wiki/xacro">
-  <!-- muscletrans is true for muscle transmission or false for motor transmission -->
-  <!-- prefix can be anything but usually is "r_" or  "l_" for right and left hands distinction -->
-  <xacro:macro name="thhub_transmission" params="muscletrans prefix" >
-   <!-- muscle hand -->
-    <xacro:if value="${muscletrans}">
-      <transmission type="sr_mechanism_model/SimpleTransmissionForMuscle" name="${prefix}thhub_transmission">
-      <actuator name="${prefix}THJ3" />
-      <joint name="${prefix}THJ3" />
-      <mechanicalReduction>1</mechanicalReduction>
-      </transmission>
-    </xacro:if>
-    <!-- motor hand -->
-    <xacro:unless value="${muscletrans}">
-      <transmission name="${prefix}thhub_transmission">
-        <type>sr_mechanism_model/SimpleTransmission</type>
-        <actuator name="${prefix}THJ3">
-          <mechanicalReduction>1</mechanicalReduction>
-        </actuator>
-        <joint name="${prefix}THJ3">
-          <hardwareInterface>EffortJointInterface</hardwareInterface>
-          <hardwareInterface>PositionJointInterface</hardwareInterface>
-        </joint>
-      </transmission>
-    </xacro:unless>
-  </xacro:macro>
+    <!-- muscletrans is true for muscle transmission or false for motor transmission -->
+    <!-- prefix can be anything but usually is "r_" or  "l_" for right and left hands distinction -->
+    <xacro:macro name="thhub_transmission" params="muscletrans prefix">
+        <!-- muscle hand -->
+        <xacro:if value="${muscletrans}">
+            <transmission name="${prefix}thhub_transmission">
+                <type>sr_mechanism_model/SimpleTransmissionForMuscle</type>
+                <actuator name="${prefix}THJ3">
+                    <mechanicalReduction>1</mechanicalReduction>
+                </actuator>
+                <joint name="${prefix}THJ3">
+                    <hardwareInterface>EffortJointInterface</hardwareInterface>
+                    <hardwareInterface>PositionJointInterface</hardwareInterface>
+                </joint>
+            </transmission>
+        </xacro:if>
+        <!-- motor hand -->
+        <xacro:unless value="${muscletrans}">
+            <transmission name="${prefix}thhub_transmission">
+                <type>sr_mechanism_model/SimpleTransmission</type>
+                <actuator name="${prefix}THJ3">
+                    <mechanicalReduction>1</mechanicalReduction>
+                </actuator>
+                <joint name="${prefix}THJ3">
+                    <hardwareInterface>EffortJointInterface</hardwareInterface>
+                    <hardwareInterface>PositionJointInterface</hardwareInterface>
+                </joint>
+            </transmission>
+        </xacro:unless>
+    </xacro:macro>
 </robot>

File: sr_description/hand/xacro/thumb/thmiddle.transmission.xacro (robot description, xacro)
@@ -4,28 +4,33 @@
        xmlns:interface="http://playerstage.sourceforge.net/gazebo/xmlschema/#interface"
        xmlns:xacro="http://www.ros.org/wiki/xacro">
-  <!-- muscletrans is true for muscle transmission or false for motor transmission -->
-  <!-- prefix can be anything but usually is "r_" or  "l_" for right and left hands distinction -->
-  <xacro:macro name="thmiddle_transmission" params="muscletrans prefix" >
-   <!-- muscle hand -->
-    <xacro:if value="${muscletrans}">
-      <transmission type="sr_mechanism_model/SimpleTransmissionForMuscle" name="${prefix}thmiddle_transmission">
-      <actuator name="${prefix}THJ2" />
-      <joint name="${prefix}THJ2" />
-      <mechanicalReduction>1</mechanicalReduction>
-      </transmission>
-    </xacro:if>
-    <!-- motor hand -->
-    <xacro:unless value="${muscletrans}">
-      <transmission name="${prefix}thmiddle_transmission">
-        <type>sr_mechanism_model/SimpleTransmission</type>
-        <actuator name="${prefix}THJ2">
-          <mechanicalReduction>1</mechanicalReduction>
-        </actuator>
-        <joint name="${prefix}THJ2">
-          <hardwareInterface>EffortJointInterface</hardwareInterface>
-          <hardwareInterface>PositionJointInterface</hardwareInterface>
-        </joint>
-      </transmission>
-    </xacro:unless>
-  </xacro:macro>
+    <!-- muscletrans is true for muscle transmission or false for motor transmission -->
+    <!-- prefix can be anything but usually is "r_" or  "l_" for right and left hands distinction -->
+    <xacro:macro name="thmiddle_transmission" params="muscletrans prefix">
+        <!-- muscle hand -->
+        <xacro:if value="${muscletrans}">
+            <transmission name="${prefix}thmiddle_transmission">
+                <type>sr_mechanism_model/SimpleTransmissionForMuscle</type>
+                <actuator name="${prefix}THJ2">
+                    <mechanicalReduction>1</mechanicalReduction>
+                </actuator>
+                <joint name="${prefix}THJ2">
+                    <hardwareInterface>EffortJointInterface</hardwareInterface>
+                    <hardwareInterface>PositionJointInterface</hardwareInterface>
+                </joint>
+            </transmission>
+        </xacro:if>
+        <!-- motor hand -->
+        <xacro:unless value="${muscletrans}">
+            <transmission name="${prefix}thmiddle_transmission">
+                <type>sr_mechanism_model/SimpleTransmission</type>
+                <actuator name="${prefix}THJ2">
+                    <mechanicalReduction>1</mechanicalReduction>
+                </actuator>
+                <joint name="${prefix}THJ2">
+                    <hardwareInterface>EffortJointInterface</hardwareInterface>
+                    <hardwareInterface>PositionJointInterface</hardwareInterface>
+                </joint>
+            </transmission>
+        </xacro:unless>
+    </xacro:macro>
 </robot>

File: sr_description/hand/xacro/thumb/thproximal.transmission.xacro (robot description, xacro)
@@ -4,28 +4,33 @@
        xmlns:interface="http://playerstage.sourceforge.net/gazebo/xmlschema/#interface"
        xmlns:xacro="http://www.ros.org/wiki/xacro">
-  <!-- muscletrans is true for muscle transmission or false for motor transmission -->
-  <!-- prefix can be anything but usually is "r_" or  "l_" for right and left hands distinction -->
-  <xacro:macro name="thproximal_transmission" params="muscletrans prefix" >
-   <!-- muscle hand -->
-    <xacro:if value="${muscletrans}">
-      <transmission type="sr_mechanism_model/SimpleTransmissionForMuscle" name="${prefix}thproximal_transmission">
-      <actuator name="${prefix}THJ4" />
-      <joint name="${prefix}THJ4" />
-      <mechanicalReduction>1</mechanicalReduction>
-      </transmission>
-    </xacro:if>
-    <!-- motor hand -->
-    <xacro:unless value="${muscletrans}">
-      <transmission name="${prefix}thproximal_transmission">
-        <type>sr_mechanism_model/SimpleTransmission</type>
-        <actuator name="${prefix}THJ4">
-          <mechanicalReduction>1</mechanicalReduction>
-        </actuator>
-        <joint name="${prefix}THJ4">
-          <hardwareInterface>EffortJointInterface</hardwareInterface>
-          <hardwareInterface>PositionJointInterface</hardwareInterface>
-        </joint>
-      </transmission>
-    </xacro:unless>
-  </xacro:macro>
+    <!-- muscletrans is true for muscle transmission or false for motor transmission -->
+    <!-- prefix can be anything but usually is "r_" or  "l_" for right and left hands distinction -->
+    <xacro:macro name="thproximal_transmission" params="muscletrans prefix">
+        <!-- muscle hand -->
+        <xacro:if value="${muscletrans}">
+            <transmission name="${prefix}thproximal_transmission">
+                <type>sr_mechanism_model/SimpleTransmissionForMuscle</type>
+                <actuator name="${prefix}THJ4">
+                    <mechanicalReduction>1</mechanicalReduction>
+                </actuator>
+                <joint name="${prefix}THJ4">
+                    <hardwareInterface>EffortJointInterface</hardwareInterface>
+                    <hardwareInterface>PositionJointInterface</hardwareInterface>
+                </joint>
+            </transmission>
+        </xacro:if>
+        <!-- motor hand -->
+        <xacro:unless value="${muscletrans}">
+            <transmission name="${prefix}thproximal_transmission">
+                <type>sr_mechanism_model/SimpleTransmission</type>
+                <actuator name="${prefix}THJ4">
+                    <mechanicalReduction>1</mechanicalReduction>
+                </actuator>
+                <joint name="${prefix}THJ4">
+                    <hardwareInterface>EffortJointInterface</hardwareInterface>
+                    <hardwareInterface>PositionJointInterface</hardwareInterface>
+                </joint>
+            </transmission>
+        </xacro:unless>
+    </xacro:macro>
 </robot>

File: sr_description/hand/xacro/wrist/wrist.transmission.xacro (robot description, xacro)
@@ -4,28 +4,33 @@
        xmlns:interface="http://playerstage.sourceforge.net/gazebo/xmlschema/#interface"
        xmlns:xacro="http://www.ros.org/wiki/xacro">
-  <!-- muscletrans is true for muscle transmission or false for motor transmission -->
-  <!-- prefix can be anything but usually is "r_" or  "l_" for right and left hands distinction -->
-  <xacro:macro name="shadowhand_wrist_transmission" params="muscletrans prefix" >
-    <!-- muscle hand -->
-    <xacro:if value="${muscletrans}">
-      <transmission type="sr_mechanism_model/SimpleTransmissionForMuscle" name="${prefix}wrist_transmission">
-        <actuator name="${prefix}WRJ2" />
-        <joint name="${prefix}WRJ2" />
-        <mechanicalReduction>1</mechanicalReduction>
-      </transmission>
-    </xacro:if>
-    <!-- motor hand -->
-    <xacro:unless value="${muscletrans}">
-      <transmission name="${prefix}wrist_transmission">
-        <type>sr_mechanism_model/SimpleTransmission</type>
-        <actuator name="${prefix}WRJ2">
-          <mechanicalReduction>1</mechanicalReduction>
-        </actuator>
-        <joint name="${prefix}WRJ2">
-          <hardwareInterface>EffortJointInterface</hardwareInterface>
-          <hardwareInterface>PositionJointInterface</hardwareInterface>
-        </joint>
-      </transmission>
-    </xacro:unless>
-  </xacro:macro>
+    <!-- muscletrans is true for muscle transmission or false for motor transmission -->
+    <!-- prefix can be anything but usually is "r_" or  "l_" for right and left hands distinction -->
+    <xacro:macro name="shadowhand_wrist_transmission" params="muscletrans prefix">
+        <!-- muscle hand -->
+        <xacro:if value="${muscletrans}">
+            <transmission name="${prefix}wrist_transmission">
+                <type>sr_mechanism_model/SimpleTransmissionForMuscle</type>
+                <actuator name="${prefix}WRJ2">
+                    <mechanicalReduction>1</mechanicalReduction>
+                </actuator>
+                <joint name="${prefix}WRJ2">
+                    <hardwareInterface>EffortJointInterface</hardwareInterface>
+                    <hardwareInterface>PositionJointInterface</hardwareInterface>
+                </joint>
+            </transmission>
+        </xacro:if>
+        <!-- motor hand -->
+        <xacro:unless value="${muscletrans}">
+            <transmission name="${prefix}wrist_transmission">
+                <type>sr_mechanism_model/SimpleTransmission</type>
+                <actuator name="${prefix}WRJ2">
+                    <mechanicalReduction>1</mechanicalReduction>
+                </actuator>
+                <joint name="${prefix}WRJ2">
+                    <hardwareInterface>EffortJointInterface</hardwareInterface>
+                    <hardwareInterface>PositionJointInterface</hardwareInterface>
+                </joint>
+            </transmission>
+        </xacro:unless>
+    </xacro:macro>
 </robot>

File: sr_description/robots/shadowhand_motor.urdf.xacro (robot description, xacro)
@@ -1,11 +1,11 @@
 <robot xmlns:sensor="http://playerstage.sourceforge.net/gazebo/xmlschema/#sensor"
-xmlns:controller="http://playerstage.sourceforge.net/gazebo/xmlschema/#controller"
-xmlns:interface="http://playerstage.sourceforge.net/gazebo/xmlschema/#interface"
-xmlns:xacro="http://www.ros.org/wiki/xacro"
-name="shadowhand_motor">
-  <xacro:include filename="$(find sr_description)/materials.urdf.xacro" />
-  <xacro:include filename="$(find sr_description)/hand/xacro/full_hand.urdf.xacro" />
-  <xacro:include filename="$(find sr_description)/other/xacro/gazebo/gazebo.urdf.xacro" />
-  <xacro:shadowhand muscletrans="false" muscle="false" bio="false" bt_sp="false"
-  ubi="false" eli="false" reflect="1.0" prefix="rh_" />
+       xmlns:controller="http://playerstage.sourceforge.net/gazebo/xmlschema/#controller"
+       xmlns:interface="http://playerstage.sourceforge.net/gazebo/xmlschema/#interface"
+       xmlns:xacro="http://www.ros.org/wiki/xacro"
+       name="shadowhand_motor">
+    <xacro:include filename="$(find sr_description)/materials.urdf.xacro"/>
+    <xacro:include filename="$(find sr_description)/hand/xacro/full_hand.urdf.xacro"/>
+    <xacro:include filename="$(find sr_description)/other/xacro/gazebo/gazebo.urdf.xacro"/>
+    <xacro:shadowhand muscletrans="false" muscle="false" bio="false" bt_sp="false"
+                      ubi="false" eli="false" reflect="1.0" prefix="rh_"/>
 </robot>

Commit message: fix depcrecation messages

File: sr_description/hand/xacro/finger/distal/distal.transmission.xacro (robot description, xacro)
@@ -17,6 +17,6 @@
             </actuator>
             <joint name="${prefix}${joint_prefix}J1">
-                <hardwareInterface>EffortJointInterface</hardwareInterface>
-                <hardwareInterface>PositionJointInterface</hardwareInterface>
+                <hardwareInterface>hardware_interface/EffortJointInterface</hardwareInterface>
+                <hardwareInterface>hardware_interface/PositionJointInterface</hardwareInterface>
             </joint>
         </transmission>

File: sr_description/hand/xacro/finger/knuckle/knuckle.transmission.xacro (robot description, xacro)
@@ -17,6 +17,6 @@
                 </actuator>
                 <joint name="${prefix}${joint_prefix}J4">
-                    <hardwareInterface>EffortJointInterface</hardwareInterface>
-                    <hardwareInterface>PositionJointInterface</hardwareInterface>
+                    <hardwareInterface>hardware_interface/EffortJointInterface</hardwareInterface>
+                    <hardwareInterface>hardware_interface/PositionJointInterface</hardwareInterface>
                 </joint>
             </transmission>
@@ -30,6 +30,6 @@
                 </actuator>
                 <joint name="${prefix}${joint_prefix}J4">
-                    <hardwareInterface>EffortJointInterface</hardwareInterface>
-                    <hardwareInterface>PositionJointInterface</hardwareInterface>
+                    <hardwareInterface>hardware_interface/EffortJointInterface</hardwareInterface>
+                    <hardwareInterface>hardware_interface/PositionJointInterface</hardwareInterface>
                 </joint>
             </transmission>

File: sr_description/hand/xacro/forearm/forearm.urdf.xacro (robot description, xacro)
@@ -9,6 +9,6 @@
     </material>
   </xacro:macro>
-  <xacro:macro name="light_grey" >
-    <material name="light_grey">
+  <xacro:macro name="grey" >
+    <material name="Grey">
       <color rgba="0.90000 0.90000 0.90000 1.0" />
     </material>
@@ -38,5 +38,5 @@
               <mesh filename="package://sr_description/meshes/hand/forearm.dae" scale="0.001 0.001 0.001" />
             </geometry>
-            <material name="light_grey" />
+            <material name="Grey" />
           </visual>
         </xacro:if>
@@ -47,5 +47,5 @@
               <mesh filename="package://sr_description/meshes/hand/forearm_visual_plus.dae" scale="0.001 0.001 0.001" />
             </geometry>
-            <material name="light_grey" />
+            <material name="Grey" />
           </visual>
         </xacro:if>

File: sr_description/hand/xacro/thumb/thhub.transmission.xacro (robot description, xacro)
@@ -15,6 +15,6 @@
                 </actuator>
                 <joint name="${prefix}THJ3">
-                    <hardwareInterface>EffortJointInterface</hardwareInterface>
-                    <hardwareInterface>PositionJointInterface</hardwareInterface>
+                    <hardwareInterface>hardware_interface/EffortJointInterface</hardwareInterface>
+                    <hardwareInterface>hardware_interface/PositionJointInterface</hardwareInterface>
                 </joint>
             </transmission>
@@ -28,6 +28,6 @@
                 </actuator>
                 <joint name="${prefix}THJ3">
-                    <hardwareInterface>EffortJointInterface</hardwareInterface>
-                    <hardwareInterface>PositionJointInterface</hardwareInterface>
+                    <hardwareInterface>hardware_interface/EffortJointInterface</hardwareInterface>
+                    <hardwareInterface>hardware_interface/PositionJointInterface</hardwareInterface>
                 </joint>
             </transmission>

File: sr_description/hand/xacro/thumb/thproximal.transmission.xacro (robot description, xacro)
@@ -15,6 +15,6 @@
                 </actuator>
                 <joint name="${prefix}THJ4">
-                    <hardwareInterface>EffortJointInterface</hardwareInterface>
-                    <hardwareInterface>PositionJointInterface</hardwareInterface>
+                    <hardwareInterface>hardware_interface/EffortJointInterface</hardwareInterface>
+                    <hardwareInterface>hardware_interface/PositionJointInterface</hardwareInterface>
                 </joint>
             </transmission>
@@ -28,6 +28,6 @@
                 </actuator>
                 <joint name="${prefix}THJ4">
-                    <hardwareInterface>EffortJointInterface</hardwareInterface>
-                    <hardwareInterface>PositionJointInterface</hardwareInterface>
+                    <hardwareInterface>hardware_interface/EffortJointInterface</hardwareInterface>
+                    <hardwareInterface>hardware_interface/PositionJointInterface</hardwareInterface>
                 </joint>
             </transmission>
