Commit message: Modify the tip frame so that it coincides with PSTs tip

File: sr_description/hand/xacro/finger/distal/distal.urdf.xacro (robot description, xacro)
@@ -130,5 +130,5 @@
         <parent link="${prefix}${link_prefix}distal" />
         <child link="${prefix}${link_prefix}tip" />
-        <origin xyz="0 0 0.026" rpy="0 0 0" />
+        <origin xyz="0 0 0.0295" rpy="0 0 0" />
       </joint>
     </xacro:unless>

File: sr_description/hand/xacro/thumb/thdistal.urdf.xacro (robot description, xacro)
@@ -49,5 +49,5 @@
         </inertial>
         <visual>
-          <origin xyz="0 0 0" rpy="0 0 0" />
+          <origin xyz="0 0 0.0022" rpy="0 0 0" />
           <geometry name="${prefix}th_distal_visual">
             <!-- <mesh filename="package://sr_description/hand/model/biotacs/biotac.stl" scale="0.0254 0.0254 0.0254" /> -->
@@ -210,5 +210,5 @@
         <parent link="${prefix}thdistal" />
         <child link="${prefix}thtip" />
-        <origin xyz="0 0 0.0275" rpy="0 0 0" />
+        <origin xyz="0 0 0.0350" rpy="0 0 0" />
       </joint>
       <xacro:thdistal_gazebo prefix="${prefix}" />

File: sr_description/mujoco_models/urdfs/shadowhand_motor_plus.urdf (robot description, URDF)
Before this commit: robot shadowhand_motor, 33 links, 32 joints
Joints:
- joint rh_FFtip: origin xyz=0 0 0.026 rpy=0 0 0 -> xyz=0 0 0.0295 rpy=0 0 0
- joint rh_LFtip: origin xyz=0 0 0.026 rpy=0 0 0 -> xyz=0 0 0.0295 rpy=0 0 0
- joint rh_MFtip: origin xyz=0 0 0.026 rpy=0 0 0 -> xyz=0 0 0.0295 rpy=0 0 0
- joint rh_RFtip: origin xyz=0 0 0.026 rpy=0 0 0 -> xyz=0 0 0.0295 rpy=0 0 0
- joint rh_thtip: origin xyz=0 0 0.0275 rpy=0 0 0 -> xyz=0 0 0.0350 rpy=0 0 0

Commit message: Adapt tips for biotac

File: sr_description/hand/xacro/finger/distal/distal.urdf.xacro (robot description, xacro)
@@ -130,5 +130,5 @@
         <parent link="${prefix}${link_prefix}distal" />
         <child link="${prefix}${link_prefix}tip" />
-        <origin xyz="0 0 0.0295" rpy="0 0 0" />
+        <origin xyz="0 0 0.034" rpy="0 0 0" />
       </joint>
     </xacro:unless>

File: sr_description/hand/xacro/thumb/thdistal.urdf.xacro (robot description, xacro)
@@ -127,5 +127,5 @@
         </inertial>
         <visual>
-          <origin xyz="0 0 0" rpy="0 0 0" />
+          <origin xyz="0 0 0.0022" rpy="0 0 0" />
           <geometry name="${prefix}thdistal_visual">
             <xacro:if value="${eli}">
@@ -158,5 +158,5 @@
         </visual>
         <collision>
-          <origin xyz="0 0 0" rpy="0 0 0" />
+          <origin xyz="0 0 0.0022" rpy="0 0 0" />
           <geometry name="${prefix}thmiddle_collision_geom">
             <xacro:if value="${eli}">

Commit message: More simplifications
- Simpify one_finger_unit.urdf.xacro
  There is only one finger. No need to pass *_sensors. A single one is sufficient.
  Also, a fingers parameter doesn't make sense.

- Reduce number of xacro:if in fingers.urdf.xacro

- Plain string default parameters don't need to be quoted

File: sr_description/hand/xacro/finger/distal/distal.urdf.xacro (robot description, xacro)
@@ -14,5 +14,5 @@
   <!-- parent is the parent link for the joint -->
   <xacro:macro name="distal"
-  params="prefix:=^ link_prefix:=^ joint_prefix:=^ tip_sensor:=^|'std' parent">
+  params="prefix:=^ link_prefix:=^ joint_prefix:=^ tip_sensor:=^|std parent">
     <link name="${prefix}${link_prefix}distal">
       <inertial>

File: sr_description/hand/xacro/finger/fingers.urdf.xacro (robot description, xacro)
@@ -16,5 +16,5 @@
   <!-- parent is the parent link for the first joint -->
   <xacro:macro name="finger"
-  params="tip_sensor:=^|'std' mid_sensor:=^|'std' prox_sensor:=^|'std' reflect:=^ prefix:=^ link_prefix joint_prefix parent *origin *axis">
+  params="tip_sensor:=^|std mid_sensor:=^|std prox_sensor:=^|std reflect:=^ prefix:=^ link_prefix joint_prefix parent *origin *axis">
     <!-- Little finger special case -->
     <xacro:if value="${'lf' in link_prefix}">
@@ -34,16 +34,14 @@
     <!-- Proximal -->
     <xacro:proximal parent="${prefix}${link_prefix}knuckle"></xacro:proximal>
-    <!-- Biotac Middle -->
+    <!-- BioTac combines Middle + Distal -->
     <xacro:if value="${'bio' in tip_sensor}">
       <xacro:biotac_middle parent="${prefix}${link_prefix}proximal">
       </xacro:biotac_middle>
     </xacro:if>
-    <!-- Standard Middle -->
+    <!-- Non-BioTac -->
     <xacro:unless value="${'bio' in tip_sensor}">
+      <!-- Middle -->
       <xacro:middle parent="${prefix}${link_prefix}proximal"></xacro:middle>
-    </xacro:unless>
-    <!-- Distal  -->
-    <!-- only if finger is not biotac  -->
-    <xacro:unless value="${'bio' in tip_sensor}">
+      <!-- Distal  -->
       <xacro:distal parent="${prefix}${link_prefix}middle"></xacro:distal>
     </xacro:unless>

File: sr_description/hand/xacro/one_finger_unit.urdf.xacro (robot description, xacro)
@@ -19,7 +19,9 @@
   <!-- prefix can be anything but usually is "r_" or  "l_" for right and left hands distinction -->
   <xacro:macro name="shadowhand" params="hand_type:='hand_e' reflect prefix cable_mesh:=False
-          fingers:=${[1,1,1,1]} tip_sensors:=${['std','std','std','std']} prox_sensors:=${['std','std','std','std']}
-          mid_sensors:=${['std','std','std','std']} palm_sensor:=std
-          muscletrans:=False muscle:=False lf:=True extra_lite:=False bio:=False bt_sp:=False eli:=False">
+          tip_sensor:=std mid_sensor:=std prox_sensor:=std palm_sensor:=std
+          muscletrans:=False muscle:=False bio:=False bt_sp:=False eli:=False">
+    <xacro:property name="tip_sensors" value="${5 * [tip_sensor]}" />
+    <xacro:property name="mid_sensors" value="${5 * [mid_sensor]}" />
+    <xacro:property name="prox_sensors" value="${5 * [prox_sensor]}" />
     <xacro:include filename="$(find sr_description)/hand/xacro/backward_compat.urdf.xacro" />
     <!-- Forearm -->
@@ -56,12 +58,10 @@
     <!-- Middle Finger -->
     <!-- TODO: Check if offset is the same for muscle hand -->
-    <xacro:if value="${fingers[2] == 1}">
-      <xacro:finger link_prefix="mf" joint_prefix="MF" tip_sensor="${tip_sensors[2]}"
-                    prox_sensor="${prox_sensors[2]}" mid_sensor="${mid_sensors[2]}"
-                    parent="${prefix}palm">
-        <origin xyz="0.0 0 0.116" rpy="0 0 0" />
-        <axis xyz="0 ${-1*reflect} 0" />
-      </xacro:finger>
-    </xacro:if>
+    <xacro:finger link_prefix="mf" joint_prefix="MF" tip_sensor="${tip_sensors[2]}"
+                  prox_sensor="${prox_sensors[2]}" mid_sensor="${mid_sensors[2]}"
+                  parent="${prefix}palm">
+      <origin xyz="0.0 0 0.116" rpy="0 0 0" />
+      <axis xyz="0 ${-1*reflect} 0" />
+    </xacro:finger>
   </xacro:macro>
 </robot>

File: sr_description/hand/xacro/thumb/thumb.urdf.xacro (robot description, xacro)
@@ -13,5 +13,5 @@
   <!-- is_lite is this the lite hand, if so lock J3 -->
   <xacro:macro name="thumb"
-  params=" tip_sensor:=^|'std' mid_sensor:=^|'std' prox_sensor:=^|'std' reflect:=^ prefix:=^ parent is_lite">
+  params=" tip_sensor:=^|std mid_sensor:=^|std prox_sensor:=^|std reflect:=^ prefix:=^ parent is_lite">
     <xacro:if value="${tip_sensor == 'bio'}">
       <xacro:property name="mid_sensor" value="bio" />

Commit message: Remove use of ubi param

File: sr_description/hand/xacro/finger/distal/distal.urdf.xacro (robot description, xacro)
@@ -29,10 +29,4 @@
         <origin xyz="0 0 0" rpy="0 0 0" />
         <geometry name="${prefix}${link_prefix}distal_visual">
-          <xacro:if value="${ubi}">
-            <!-- Ubi distal -->
-            <mesh filename="package://sr_description/meshes/hand/ubi_tactiles/ubi_tip_visual.dae"
-		  scale="0.001 0.001 0.001" />
-          </xacro:if>
-          <xacro:unless value="${ubi}">
             <xacro:if value="${eli}">
               <!-- Ellispoid distal  -->
@@ -58,5 +52,4 @@
               </xacro:unless>
             </xacro:unless>
-          </xacro:unless>
         </geometry>
         <!-- <material name="Grey" /> -->
@@ -65,10 +58,4 @@
         <origin xyz="0 0 0" rpy="0 0 0" />
         <geometry name="${prefix}${link_prefix}distal_collision_geom">
-          <xacro:if value="${ubi}">
-            <!-- Ubi distal -->
-            <mesh filename="package://sr_description/meshes/hand/ubi_tactiles/ubi_tip_collision.dae"
-            scale="0.001 0.001 0.001" />
-          </xacro:if>
-          <xacro:unless value="${ubi}">
             <xacro:if value="${eli}">
               <!-- Ellispoid distal  -->
@@ -94,5 +81,4 @@
               </xacro:unless>
             </xacro:unless>
-          </xacro:unless>
         </geometry>
       </collision>

File: sr_description/hand/xacro/thumb/thdistal.urdf.xacro (robot description, xacro)
@@ -135,10 +135,4 @@
             </xacro:if>
             <xacro:unless value="${eli}">
-              <xacro:if value="${ubi}">
-                <!-- Ubi distal -->
-                <mesh filename="package://sr_description/meshes/hand/TH1_z.dae"
-                      scale="0.001 0.001 0.001" />
-              </xacro:if>
-	      <xacro:unless value="${ubi}">
 		<xacro:if value="${bt_sp}">
 		  <!-- bt sp distal  -->
@@ -150,5 +144,4 @@
 			scale="0.001 0.001 0.001" />
 		</xacro:unless>
-	      </xacro:unless>
             </xacro:unless>
           </geometry>
@@ -166,10 +159,4 @@
             </xacro:if>
             <xacro:unless value="${eli}">
-              <xacro:if value="${ubi}">
-                <!-- Ubi distal -->
-                <mesh filename="package://sr_description/meshes/hand/TH1_z.dae"
-                scale="0.001 0.001 0.001" />
-              </xacro:if>
-              <xacro:unless value="${ubi}">
 		<xacro:if value="${bt_sp}">
 		  <!-- bt sp distal  -->
@@ -181,5 +168,4 @@
 			scale="0.001 0.001 0.001" />
 		</xacro:unless>
-              </xacro:unless>
             </xacro:unless>
             <!--      <box size="0.015 0.015 0.015" /> -->

Commit message: Simplify if-else clauses
Improve extensibility (adding more sensors) by emloying an exclusive-if-and-final-else
strategy, utilizing a helper variable. This way we avoid augmenting the list in the
'sensor in [...]' tests.

File: sr_description/hand/xacro/finger/distal/distal.urdf.xacro (robot description, xacro)
@@ -25,19 +25,20 @@
         <origin xyz="0 0 0" rpy="0 0 0" />
         <geometry name="${prefix}${link_prefix}distal_visual">
-          <xacro:unless value="${tip_sensor in ['bt_sp','eli']}">
+          <!-- Do we need to instantiate the standard distal? -->
+          <xacro:property name="standard" value="true" />
+          <xacro:if value="${tip_sensor == 'eli'}">
+            <!-- Ellispoid distal  -->
+            <mesh filename="package://sr_description/meshes/hand/ellipsoids/distal_ellipsoid_visual.dae"
+                  scale="0.001 0.001 0.001" />
+            <xacro:property name="standard" value="false" />
+          </xacro:if>
+          <xacro:if value="${tip_sensor == 'bt_sp'}">
+            <!-- bt_sp distal  -->
+            <mesh filename="package://sr_description/meshes/hand/biotacs/sp.dae" />
+            <xacro:property name="standard" value="false" />
+          </xacro:if>
+          <xacro:if value="${standard}">
             <!-- Standard distal  -->
-            <mesh filename="package://sr_description/meshes/hand/F1.dae"
-                  scale="0.001 0.001 0.001" />
-          </xacro:unless>
-          <xacro:if value="${tip_sensor in ['bt_sp','eli']}">
-            <xacro:if value="${tip_sensor == 'eli'}">
-              <!-- Ellispoid distal  -->
-              <mesh filename="package://sr_description/meshes/hand/ellipsoids/distal_ellipsoid_visual.dae"
-		    scale="0.001 0.001 0.001" />
-            </xacro:if>
-            <xacro:if value="${tip_sensor == 'bt_sp'}">
-              <!-- bt_sp distal  -->
-              <mesh filename="package://sr_description/meshes/hand/biotacs/sp.dae" />
-            </xacro:if>
+            <mesh filename="package://sr_description/meshes/hand/F1.dae" scale="0.001 0.001 0.001" />
           </xacro:if>
         </geometry>
@@ -47,20 +48,22 @@
         <origin xyz="0 0 0" rpy="0 0 0" />
         <geometry name="${prefix}${link_prefix}distal_collision_geom">
-          <xacro:if value="${tip_sensor in ['bt_sp','eli']}">
-            <xacro:if value="${tip_sensor == 'eli'}">
-              <!-- Ellispoid distal  -->
-              <mesh filename="package://sr_description/meshes/hand/ellipsoids/distal_ellipsoid.dae"
-                    scale="0.001 0.001 0.001" />
-            </xacro:if>
-            <xacro:if value="${tip_sensor == 'bt_sp'}">
-              <!-- bt_sp distal  -->
-              <mesh filename="package://sr_description/meshes/hand/biotacs/sp.dae" />
-            </xacro:if>
+          <!-- Do we need to instantiate the standard distal? -->
+          <xacro:property name="standard" value="true" />
+          <xacro:if value="${tip_sensor == 'eli'}">
+            <!-- Ellispoid distal  -->
+            <mesh filename="package://sr_description/meshes/hand/ellipsoids/distal_ellipsoid.dae"
+                  scale="0.001 0.001 0.001" />
+            <xacro:property name="standard" value="false" />
           </xacro:if>
-          <xacro:unless value="${tip_sensor in ['bt_sp','eli']}">
+          <xacro:if value="${tip_sensor == 'bt_sp'}">
+            <!-- bt_sp distal  -->
+            <mesh filename="package://sr_description/meshes/hand/biotacs/sp.dae" />
+            <xacro:property name="standard" value="false" />
+          </xacro:if>
+          <xacro:if value="${standard}">
             <!-- Standard distal  -->
             <mesh filename="package://sr_description/meshes/hand/F1.dae"
                   scale="0.001 0.001 0.001" />
-          </xacro:unless>
+          </xacro:if>
         </geometry>
       </collision>

File: sr_description/hand/xacro/thumb/thdistal.gazebo.xacro (robot description, xacro)
@@ -4,5 +4,5 @@
     <!-- prefix can be anything but usually is "r_" or  "l_" for right and left hands distinction -->
     <gazebo reference="${prefix}thdistal">
-     <xacro:unless value="${'none' in tip_sensor}" >
+      <xacro:unless value="${'none' in tip_sensor}" >
         <sensor type="contact" name="${prefix}thdistal_contact">
           <always_on>1</always_on>

File: sr_description/hand/xacro/thumb/thdistal.urdf.xacro (robot description, xacro)
@@ -125,17 +125,21 @@
           <origin xyz="0 0 0" rpy="0 0 0" />
           <geometry name="${prefix}thdistal_visual">
-            <xacro:unless value="${tip_sensor in ['bt_sp','eli']}">
+            <!-- Do we need to instantiate the standard distal? -->
+            <xacro:property name="standard" value="true" />
+            <xacro:if value="${tip_sensor == 'eli'}">
+              <!-- Ellispoid distal  -->
+              <mesh filename="package://sr_description/meshes/hand/ellipsoids/thdistal_ellipsoid_visual.dae"
+                    scale="0.001 0.001 0.001" />
+              <xacro:property name="standard" value="false" />
+            </xacro:if>
+            <xacro:if value="${tip_sensor == 'bt_sp'}">
+              <!-- bt sp distal  -->
+              <mesh filename="package://sr_description/meshes/hand/biotacs/sp.dae" />
+              <xacro:property name="standard" value="false" />
+            </xacro:if>
+            <xacro:if value="${standard}">
               <!-- Standard distal  -->
               <mesh filename="package://sr_description/meshes/hand/TH1_z.dae"
                     scale="0.001 0.001 0.001" />
-            </xacro:unless>
-            <xacro:if value="${tip_sensor == 'eli'}">
-              <!-- Ellispoid distal  -->
-              <mesh filename="package://sr_description/meshes/hand/ellipsoids/thdistal_ellipsoid_visual.dae"
-              scale="0.001 0.001 0.001" />
-            </xacro:if>
-            <xacro:if value="${tip_sensor == 'bt_sp'}">
-              <!-- bt sp distal  -->
-              <mesh filename="package://sr_description/meshes/hand/biotacs/sp.dae" />
             </xacro:if>
           </geometry>
@@ -147,17 +151,20 @@
           <origin xyz="0 0 0" rpy="0 0 0" />
           <geometry name="${prefix}thmiddle_collision_geom">
-            <xacro:unless value="${tip_sensor in ['bt_sp','eli']}">
-              <!-- Standard distal  -->
-              <mesh filename="package://sr_description/meshes/hand/TH1_z.dae"
-                    scale="0.001 0.001 0.001" />
-            </xacro:unless>
+            <!-- Do we need to instantiate the standard distal? -->
+            <xacro:property name="standard" value="true" />
             <xacro:if value="${tip_sensor == 'eli'}">
               <!-- Ellispoid distal  -->
               <mesh filename="package://sr_description/meshes/hand/ellipsoids/thdistal_ellipsoid.dae"
-              scale="0.001 0.001 0.001" />
+                    scale="0.001 0.001 0.001" />
+              <xacro:property name="standard" value="false" />
             </xacro:if>
             <xacro:if value="${tip_sensor == 'bt_sp'}">
               <!-- bt sp distal  -->
               <mesh filename="package://sr_description/meshes/hand/biotacs/sp.dae" />
+              <xacro:property name="standard" value="false" />
+            </xacro:if>
+            <xacro:if value="${standard}">
+              <!-- Standard distal  -->
+              <mesh filename="package://sr_description/meshes/hand/TH1_z.dae" scale="0.001 0.001 0.001" />
             </xacro:if>
             <!-- <box size="0.015 0.015 0.015" /> -->
