Commit message: Fixed Thumb plus a few issues from finger forearm and palm

File: sr_description/hand/xacro/finger/distal/distal.urdf.xacro (robot description, xacro)
@@ -25,8 +25,10 @@
         <geometry name="${prefix}${link_prefix}distal_visual">
           <xacro:if value="${tip_sensor == 'pst'}">
-            <mesh filename="package://sr_description/meshes/components/f_distal/pst/f_distal_pst.stl" scale="0.001 0.001 0.001" />
+            <mesh filename="package://sr_description/meshes/components/f_distal/pst/f_distal_pst.stl"
+                  scale="0.001 0.001 0.001" />
           </xacro:if>
           <xacro:if value="${tip_sensor == 'bt_sp'}">
-            <mesh filename="package://sr_description/meshes/components/f_distal/bt_sp/f_distal_bt_sp.stl" />
+            <mesh filename="package://sr_description/meshes/components/f_distal/bt_sp/f_distal_bt_sp.stl"
+                  scale="0.001 0.001 0.001" />
           </xacro:if>
           <xacro:if value="${tip_sensor == 'bt_2p'}">
@@ -39,8 +41,10 @@
         <geometry name="${prefix}${link_prefix}distal_collision_geom">
           <xacro:if value="${tip_sensor == 'pst'}">
-            <mesh filename="package://sr_description/meshes/components/f_distal/pst/f_distal_pst.stl" scale="0.001 0.001 0.001" />
+            <mesh filename="package://sr_description/meshes/components/f_distal/pst/f_distal_pst.stl"
+                  scale="0.001 0.001 0.001" />
           </xacro:if>
           <xacro:if value="${tip_sensor == 'bt_sp'}">
-            <mesh filename="package://sr_description/meshes/components/f_distal/bt_sp/f_distal_bt_sp.stl" />
+            <mesh filename="package://sr_description/meshes/components/f_distal/bt_sp/f_distal_bt_sp.stl"
+                  scale="0.001 0.001 0.001" />
           </xacro:if>
           <xacro:if value="${tip_sensor == 'bt_2p'}">

File: sr_description/hand/xacro/forearm/forearm_g.urdf.xacro (robot description, xacro)
@@ -1,4 +1,4 @@
 <robot xmlns:xacro="http://www.ros.org/wiki/xacro">
-  <xacro:macro name="forearm" params="hand_type:=^ prefix:=^ cable_mesh:=^">
+  <xacro:macro name="forearm" params="hand_type:=^ prefix:=^">
     <link name="${prefix}forearm">
       <inertial>

File: sr_description/hand/xacro/palm/palm_g.urdf.xacro (robot description, xacro)
@@ -8,5 +8,5 @@
   <xacro:include filename="$(find sr_description)/hand/xacro/palm/palm.gazebo.xacro" />
   <xacro:include filename="$(find sr_description)/hand/xacro/palm/imu.urdf.xacro" />
-  <xacro:macro name="palm" params="prefix:=^ reflect:=^ parent">
+  <xacro:macro name="palm" params="hand_type:=^ hand_version:=^ prefix:=^ reflect:=^ parent">
     <link name="${prefix}palm">
       <inertial>

File: sr_description/hand/xacro/thumb/thbase.urdf.xacro (robot description, xacro)
@@ -8,7 +8,4 @@
   <xacro:include filename="$(find sr_description)/hand/xacro/thumb/thbase.gazebo.xacro" />
   <xacro:include filename="$(find sr_description)/hand/xacro/thumb/thbase.transmission.xacro" />
-  <!-- reflect is either 1 (for right hand) or -1 (for left hand) -->
-  <!-- prefix can be anything but usually is "r_" or  "l_" for right and left hands distinction -->
-  <!-- parent is the parent link for the first joint -->
   <xacro:macro name="thbase" params="reflect:=^ prefix:=^ parent">
     <link name="${prefix}thbase">
@@ -38,5 +35,5 @@
       <parent link="${parent}" />
       <child link="${prefix}thbase" />
-      <origin xyz="${reflect*0.034} -0.0085 0.029"
+      <origin xyz="${reflect*0.034} -0.00858 0.029"
       rpy="0 ${pi/4} ${pi/2-reflect*pi/2}" />
       <axis xyz="0 0 ${reflect*-1}" />

File: sr_description/hand/xacro/thumb/thdistal.urdf.xacro (robot description, xacro)
@@ -10,5 +10,4 @@
   <xacro:macro name="thdistal" params="tip_sensor:=^|pst prefix:=^ parent">
     <xacro:if value="${tip_sensor == 'bt_2p'}">
-      <!--    BIOTAC -->
       <link name="${prefix}thdistal_J1_dummy">
         <inertial>
@@ -43,6 +42,5 @@
           <origin xyz="0 0 0" rpy="0 0 0" />
           <geometry name="${prefix}th_distal_visual">
-            <!-- <mesh filename="package://sr_description/meshes/hand/biotacs/biotac.stl" scale="0.0254 0.0254 0.0254" /> -->
-            <mesh filename="package://sr_description/meshes/hand/biotacs/biotac_decimated.dae"
+            <mesh filename="package://sr_description/meshes/components/th_distal/bt_2p/th_distal_bt_2p.dae"
             scale="0.0254 0.0254 0.0254" />
           </geometry>
@@ -51,7 +49,5 @@
         <collision>
           <geometry name="${prefix}th_distal_collision_geom">
-            <!-- <box size="0.001 0.001 0.001" /> -->
-            <!-- <mesh filename="package://sr_description/meshes/hand/biotacs/biotac-v5.stl" scale="0.0254 0.0254 0.0254" /> -->
-            <mesh filename="package://sr_description/meshes/hand/biotacs/biotac_decimated.dae"
+            <mesh filename="package://sr_description/meshes/components/th_distal/bt_2p/th_distal_bt_2p.dae"
             scale="0.0254 0.0254 0.0254" />
           </geometry>
@@ -84,5 +80,4 @@
       </joint>
       <!-- extra link to imaginary sphere in fingertip for FK/IK calculations -->
-      <!-- remove visual and collision once the correct position is found -->
       <link name="${prefix}thtip">
         <inertial>
@@ -92,9 +87,4 @@
           izz="0" />
         </inertial>
-        <!--visual>
-          <geometry>
-            <sphere radius="0.002" />
-          </geometry>
-        </visual-->
       </link>
       <gazebo reference="${prefix}thtip">
@@ -104,6 +94,5 @@
         <parent link="${prefix}thdistal_J1_dummy" />
         <child link="${prefix}thtip" />
-        <origin xyz="0.0 0.004 ${0.032}"
-        rpy="0 0 0" />
+        <origin xyz="0.0 0.004 ${0.032}" rpy="0 0 0" />
         <!-- approximated only FIXME -->
       </joint>
@@ -121,20 +110,14 @@
           <origin xyz="0 0 0" rpy="0 0 0" />
           <geometry name="${prefix}thdistal_visual">
-            <!-- Do we need to instantiate the standard distal? -->
-            <xacro:property name="standard" value="true" />
-            <xacro:if value="${tip_sensor == 'eli'}">
-              <!-- Ellispoid distal  -->
-              <mesh filename="package://sr_description/meshes/hand/ellipsoids/thdistal_ellipsoid_visual.dae"
+            <xacro:if value="${tip_sensor == 'pst'}">
+              <mesh filename="package://sr_description/meshes/components/th_distal/pst/th_distal_pst.stl"
                     scale="0.001 0.001 0.001" />
-              <xacro:property name="standard" value="false" />
             </xacro:if>
             <xacro:if value="${tip_sensor == 'bt_sp'}">
-              <!-- bt sp distal  -->
-              <mesh filename="package://sr_description/meshes/hand/biotacs/sp.dae" />
-              <xacro:property name="standard" value="false" />
+              <mesh filename="package://sr_description/meshes/components/th_distal/bt_sp/th_distal_bt_sp.stl"
+                    scale="0.001 0.001 0.001" />
             </xacro:if>
-            <xacro:if value="${standard}">
-              <!-- Standard distal  -->
-              <mesh filename="package://sr_description/meshes/hand/TH1_z.dae"
+            <xacro:if value="${tip_sensor == 'bt_2p'}">
+              <mesh filename="package://sr_description/meshes/components/th_distal/bt_2p/th_distal_bt_2p.dae"
                     scale="0.001 0.001 0.001" />
             </xacro:if>
@@ -147,22 +130,16 @@
           <origin xyz="0 0 0" rpy="0 0 0" />
           <geometry name="${prefix}thmiddle_collision_geom">
-            <!-- Do we need to instantiate the standard distal? -->
-            <xacro:property name="standard" value="true" />
-            <xacro:if value="${tip_sensor == 'eli'}">
-              <!-- Ellispoid distal  -->
-              <mesh filename="package://sr_description/meshes/hand/ellipsoids/thdistal_ellipsoid.dae"
+            <xacro:if value="${tip_sensor == 'pst'}">
+              <mesh filename="package://sr_description/meshes/components/th_distal/pst/th_distal_pst.stl"
                     scale="0.001 0.001 0.001" />
-              <xacro:property name="standard" value="false" />
             </xacro:if>
             <xacro:if value="${tip_sensor == 'bt_sp'}">
-              <!-- bt sp distal  -->
-              <mesh filename="package://sr_description/meshes/hand/biotacs/sp.dae" />
-              <xacro:property name="standard" value="false" />
+              <mesh filename="package://sr_description/meshes/components/th_distal/bt_sp/th_distal_bt_sp.stl"
+                    scale="0.001 0.001 0.001" />
             </xacro:if>
-            <xacro:if value="${standard}">
-              <!-- Standard distal  -->
-              <mesh filename="package://sr_description/meshes/hand/TH1_z.dae" scale="0.001 0.001 0.001" />
+            <xacro:if value="${tip_sensor == 'bt_2p'}">
+              <mesh filename="package://sr_description/meshes/components/th_distal/bt_2p/th_distal_bt_2p.dae"
+                    scale="0.001 0.001 0.001" />
             </xacro:if>
-            <!-- <box size="0.015 0.015 0.015" /> -->
           </geometry>
         </collision>

File: sr_description/hand/xacro/thumb/thhub.urdf.xacro (robot description, xacro)
@@ -8,7 +8,4 @@
   <xacro:include filename="$(find sr_description)/hand/xacro/thumb/thhub.gazebo.xacro" />
   <xacro:include filename="$(find sr_description)/hand/xacro/thumb/thhub.transmission.xacro" />
-  <!-- prefix can be anything but usually is "r_" or  "l_" for right and left hands distinction -->
-  <!-- parent is the parent link for the first joint -->
-  <!-- is_lite is this the lite hand, if so lock J3 -->
   <xacro:macro name="thhub" params="prefix:=^ parent:=^ is_lite">
     <link name="${prefix}thhub">

File: sr_description/hand/xacro/thumb/thmiddle.urdf.xacro (robot description, xacro)
@@ -8,6 +8,4 @@
   <xacro:include filename="$(find sr_description)/hand/xacro/thumb/thmiddle.gazebo.xacro" />
   <xacro:include filename="$(find sr_description)/hand/xacro/thumb/thmiddle.transmission.xacro" />
-  <!-- mid_sensor can have value bt_2p for specific middle anything else for standard finger -->
-  <!-- prefix can be anything but usually is "r_" or  "l_" for right and left hands distinction -->
   <!-- parent is the parent link for the first joint -->
   <xacro:macro name="thmiddle" params="mid_sensor:=^ prefix:=^ parent">
@@ -23,5 +21,5 @@
         <xacro:if value="${mid_sensor == 'bt_2p'}">
           <geometry name="${prefix}thmiddle_visual">
-            <mesh filename="package://sr_description/meshes/hand/biotacs/biotac_thumb_adapter.dae"
+            <mesh filename="package://sr_description/meshes/components/th_distal/bt_2p/th_distal_bt_2p_adapter.dae"
             scale="0.001 0.001 0.001" />
           </geometry>
@@ -29,5 +27,5 @@
         <xacro:unless value="${mid_sensor == 'bt_2p'}">
           <geometry name="${prefix}thmiddle_visual">
-            <mesh filename="package://sr_description/meshes/hand/TH2_z.dae"
+            <mesh filename="package://sr_description/meshes/products/${hand_type}/${hand_version}/th_middle_${hand_version}.dae"
             scale="0.001 0.001 0.001" />
           </geometry>
@@ -71,6 +69,5 @@
       </xacro:unless>
       <axis xyz="0 -1 0" />
-      <limit lower="${-40/180*pi}" upper="${40/180*pi}"
-      effort="2.0" velocity="2.0" />
+      <limit lower="${-40/180*pi}" upper="${40/180*pi}" effort="2.0" velocity="2.0" />
       <dynamics damping="0.1" />
     </joint>

File: sr_description/hand/xacro/thumb/thproximal.urdf.xacro (robot description, xacro)
@@ -8,20 +8,15 @@
   <xacro:include filename="$(find sr_description)/hand/xacro/thumb/thproximal.gazebo.xacro" />
   <xacro:include filename="$(find sr_description)/hand/xacro/thumb/thproximal.transmission.xacro" />
-  <!-- reflect is either 1 (for right hand) or -1 (for left hand) -->
-  <!-- prefix can be anything but usually is "r_" or  "l_" for right and left hands distinction -->
-  <!-- parent is the parent link for the first joint -->
-  <xacro:macro name="thproximal"
-  params="reflect:=^ prefix:=^ parent">
+  <xacro:macro name="thproximal" params="hand_type:=^ hand_version:=^ reflect:=^ prefix:=^ parent">
     <link name="${prefix}thproximal">
       <inertial>
         <mass value="0.040" />
         <origin xyz="0 0 0.019" rpy="0 0 0" />
-        <inertia ixx="0.0000136" ixy="0.0" ixz="0.0"
-        iyy="0.0000136" iyz="0.0" izz="0.00000313" />
+        <inertia ixx="0.0000136" ixy="0.0" ixz="0.0" iyy="0.0000136" iyz="0.0" izz="0.00000313" />
       </inertial>
       <visual>
         <origin xyz="0 0 0" rpy="0 0 0" />
         <geometry name="${prefix}thproximal_visual">
-          <mesh filename="package://sr_description/meshes/hand/TH3_z.dae"
+          <mesh filename="package://sr_description/meshes/products/${hand_type}/${hand_version}/th_proximal_${hand_version}.dae"
           scale="0.001 0.001 0.001" />
         </geometry>
@@ -42,6 +37,5 @@
       <origin xyz="0 0 0" rpy="0 0 0" />
       <axis xyz="${reflect} 0 0" />
-      <limit lower="0.0" upper="${70/180*pi}" effort="3"
-      velocity="4.0" />
+      <limit lower="0.0" upper="${70/180*pi}" effort="3" velocity="4.0" />
       <dynamics damping="0.2" />
     </joint>

File: sr_description/hand/xacro/thumb/thumb.urdf.xacro (robot description, xacro)
@@ -5,13 +5,5 @@
   <xacro:include filename="$(find sr_description)/hand/xacro/thumb/thmiddle.urdf.xacro" />
   <xacro:include filename="$(find sr_description)/hand/xacro/thumb/thdistal.urdf.xacro" />
-  <!-- tip_sensor describes the sensor -->
-  <!-- mid_sensor describes the sensor -->
-  <!-- prox_sensor describes the sensor -->
-  <!-- reflect is either 1 (for right hand) or -1 (for left hand) -->
-  <!-- prefix can be anything but usually is "r_" or  "l_" for right and left hands distinction -->
-  <!-- parent is the parent link for the first joint -->
-  <!-- is_lite is this the lite hand, if so lock J3 -->
-  <xacro:macro name="thumb"
-  params=" tip_sensor:=^|pst mid_sensor:=^|none prox_sensor:=^|none reflect:=^ prefix:=^ parent is_lite">
+  <xacro:macro name="thumb" params="hand_type:=^ hand_version:=^ tip_sensor:=^|pst mid_sensor:=^|none prox_sensor:=^|none reflect:=^ prefix:=^ parent is_lite">
     <xacro:if value="${tip_sensor == 'bt_2p'}">
       <xacro:property name="mid_sensor" value="bt_2p" />
