Commit message: Fixing formtating and deleted unnecessary files

File: sr_description/hand/xacro/finger/distal/distal.urdf.xacro (robot description, xacro)
@@ -1,16 +1,11 @@
 <robot xmlns:xacro="http://www.ros.org/wiki/xacro"
-xmlns:sensor="http://playerstage.sourceforge.net/gazebo/xmlschema/#sensor"
-xmlns:controller="http://playerstage.sourceforge.net/gazebo/xmlschema/#controller"
-xmlns:joint="http://playerstage.sourceforge.net/gazebo/xmlschema/#slider"
-xmlns:interface="http://playerstage.sourceforge.net/gazebo/xmlschema/#interface"
-xmlns:body="http://playerstage.sourceforge.net/gazebo/xmlschema/#body"
-xmlns:geom="http://playerstage.sourceforge.net/gazebo/xmlschema/#geom">
+       xmlns:sensor="http://playerstage.sourceforge.net/gazebo/xmlschema/#sensor"
+       xmlns:controller="http://playerstage.sourceforge.net/gazebo/xmlschema/#controller"
+       xmlns:joint="http://playerstage.sourceforge.net/gazebo/xmlschema/#slider"
+       xmlns:interface="http://playerstage.sourceforge.net/gazebo/xmlschema/#interface"
+       xmlns:body="http://playerstage.sourceforge.net/gazebo/xmlschema/#body"
+       xmlns:geom="http://playerstage.sourceforge.net/gazebo/xmlschema/#geom">
   <xacro:include filename="$(find sr_description)/hand/xacro/finger/distal/distal.gazebo.xacro" />
   <xacro:include filename="$(find sr_description)/hand/xacro/finger/distal/distal.transmission.xacro" />
-  <!-- tip_sensor describes the sensor bt_2p, bt_sp, pst -->
-  <!-- prefix can be anything but usually is "r_" or  "l_" for right and left hands distinction -->
-  <!-- link_prefix prepends fingername to the link names -->
-  <!-- joint_prefix prepends fingername to the joint names -->
-  <!-- parent is the parent link for the joint -->
   <xacro:macro name="distal" params="prefix:=^ link_prefix:=^ joint_prefix:=^ tip_sensor:=^|pst parent">
     <link name="${prefix}${link_prefix}distal">
@@ -18,6 +13,5 @@
         <mass value="0.012" />
         <origin xyz="0 0 0.012" />
-        <inertia ixx="0.00000094" ixy="0.0" ixz="0.0"
-		 iyy="0.0000011" iyz="0.0" izz="0.00000053" />
+        <inertia ixx="0.00000094" ixy="0.0" ixz="0.0" iyy="0.0000011" iyz="0.0" izz="0.00000053" />
       </inertial>
       <visual>
@@ -61,6 +55,5 @@
         <axis xyz="1 0 0" />
         <!-- standard distal joint -->
-        <limit lower="0" upper="${pi/2}" effort="2"
-        velocity="2.0" />
+        <limit lower="0" upper="${pi/2}" effort="2" velocity="2.0" />
         <dynamics damping="0.1" />
       </joint>
@@ -72,6 +65,5 @@
         <inertial>
           <mass value="0.001" />
-          <inertia ixx="0.0" ixy="0.0" ixz="0.0" iyy="0.0"
-          iyz="0.0" izz="0.0" />
+          <inertia ixx="0.0" ixy="0.0" ixz="0.0" iyy="0.0" iyz="0.0" izz="0.0" />
         </inertial>
       </link>

File: sr_description/hand/xacro/finger/lfmetacarpal/lfmetacarpal.urdf.xacro (robot description, xacro)
@@ -1,22 +1,17 @@
 <robot xmlns:xacro="http://www.ros.org/wiki/xacro"
-xmlns:sensor="http://playerstage.sourceforge.net/gazebo/xmlschema/#sensor"
-xmlns:controller="http://playerstage.sourceforge.net/gazebo/xmlschema/#controller"
-xmlns:joint="http://playerstage.sourceforge.net/gazebo/xmlschema/#slider"
-xmlns:interface="http://playerstage.sourceforge.net/gazebo/xmlschema/#interface"
-xmlns:body="http://playerstage.sourceforge.net/gazebo/xmlschema/#body"
-xmlns:geom="http://playerstage.sourceforge.net/gazebo/xmlschema/#geom">
+       xmlns:sensor="http://playerstage.sourceforge.net/gazebo/xmlschema/#sensor"
+       xmlns:controller="http://playerstage.sourceforge.net/gazebo/xmlschema/#controller"
+       xmlns:joint="http://playerstage.sourceforge.net/gazebo/xmlschema/#slider"
+       xmlns:interface="http://playerstage.sourceforge.net/gazebo/xmlschema/#interface"
+       xmlns:body="http://playerstage.sourceforge.net/gazebo/xmlschema/#body"
+       xmlns:geom="http://playerstage.sourceforge.net/gazebo/xmlschema/#geom">
   <xacro:include filename="$(find sr_description)/hand/xacro/finger/lfmetacarpal/lfmetacarpal.gazebo.xacro" />
   <xacro:include filename="$(find sr_description)/hand/xacro/finger/lfmetacarpal/lfmetacarpal.transmission.xacro" />
-  <!-- prefix can be anything but usually is "r_" or  "l_" for right and left hands distinction -->
-  <!-- reflect is either 1 (for right hand) or -1 (for left hand) -->
-  <!-- parent is the parent link for the joint -->
-  <xacro:macro name="lfmetacarpal"
-  params="prefix:=^ reflect:=^ parent">
+  <xacro:macro name="lfmetacarpal" params="prefix:=^ reflect:=^ parent">
     <link name="${prefix}lfmetacarpal">
       <inertial>
         <origin xyz="0 0 0.04" rpy="0 0 0" />
         <mass value="0.030" />
-        <inertia ixx="0.0000145" ixy="0.0" ixz="0.0"
-        iyy="0.00001638" iyz="0.0" izz="0.000004272" />
+        <inertia ixx="0.0000145" ixy="0.0" ixz="0.0" iyy="0.00001638" iyz="0.0" izz="0.000004272" />
       </inertial>
       <visual>
@@ -40,6 +35,5 @@
       <origin xyz="${reflect*-0.033} 0 0.02071" rpy="0 0 0" />
       <axis xyz="0.573576436 0 ${reflect*0.819152044}" />
-      <limit lower="0" upper="${45/180*pi}" effort="2"
-      velocity="2.0" />
+      <limit lower="0" upper="${45/180*pi}" effort="2" velocity="2.0" />
       <dynamics damping="0.1" />
     </joint>

File: sr_description/hand/xacro/finger/proximal/proximal.urdf.xacro (robot description, xacro)
@@ -1,9 +1,9 @@
 <robot xmlns:xacro="http://www.ros.org/wiki/xacro"
-xmlns:sensor="http://playerstage.sourceforge.net/gazebo/xmlschema/#sensor"
-xmlns:controller="http://playerstage.sourceforge.net/gazebo/xmlschema/#controller"
-xmlns:joint="http://playerstage.sourceforge.net/gazebo/xmlschema/#slider"
-xmlns:interface="http://playerstage.sourceforge.net/gazebo/xmlschema/#interface"
-xmlns:body="http://playerstage.sourceforge.net/gazebo/xmlschema/#body"
-xmlns:geom="http://playerstage.sourceforge.net/gazebo/xmlschema/#geom">
+       xmlns:sensor="http://playerstage.sourceforge.net/gazebo/xmlschema/#sensor"
+       xmlns:controller="http://playerstage.sourceforge.net/gazebo/xmlschema/#controller"
+       xmlns:joint="http://playerstage.sourceforge.net/gazebo/xmlschema/#slider"
+       xmlns:interface="http://playerstage.sourceforge.net/gazebo/xmlschema/#interface"
+       xmlns:body="http://playerstage.sourceforge.net/gazebo/xmlschema/#body"
+       xmlns:geom="http://playerstage.sourceforge.net/gazebo/xmlschema/#geom">
   <xacro:include filename="$(find sr_description)/hand/xacro/finger/proximal/proximal.gazebo.xacro" />
   <xacro:include filename="$(find sr_description)/hand/xacro/finger/proximal/proximal.transmission.xacro" />

File: sr_description/hand/xacro/forearm/forearm_c.urdf.xacro (robot description, xacro)
@@ -15,6 +15,5 @@
         <origin xyz="0 0 0.09" rpy="0 0 0" />
         <mass value="3.0" />
-        <inertia ixx="0.0138" ixy="0.0" ixz="0.0" iyy="0.0138"
-        iyz="0.0" izz="0.00744" />
+        <inertia ixx="0.0138" ixy="0.0" ixz="0.0" iyy="0.0138" iyz="0.0" izz="0.00744" />
       </inertial>
       <visual>

File: sr_description/hand/xacro/forearm/forearm_e.urdf.xacro (robot description, xacro)
@@ -15,6 +15,5 @@
         <origin xyz="0 0 0.09" rpy="0 0 0" />
         <mass value="3.0" />
-        <inertia ixx="0.0138" ixy="0.0" ixz="0.0" iyy="0.0138"
-        iyz="0.0" izz="0.00744" />
+        <inertia ixx="0.0138" ixy="0.0" ixz="0.0" iyy="0.0138" iyz="0.0" izz="0.00744" />
       </inertial>
       <visual>

File: sr_description/hand/xacro/hand.urdf.xacro (robot description, xacro)
@@ -3,6 +3,5 @@
        xmlns:controller="http://playerstage.sourceforge.net/gazebo/xmlschema/#controller"
        xmlns:interface="http://playerstage.sourceforge.net/gazebo/xmlschema/#interface">
-  <xacro:macro name="sr_hand"
-               params="hand_type hand_version side fingers tip_sensors prox_sensors mid_sensors palm_sensor">
+  <xacro:macro name="sr_hand" params="hand_type hand_version side fingers tip_sensors prox_sensors mid_sensors palm_sensor">
     <!-- Process hand type, version and side parameters -->
     <xacro:include filename="$(find sr_description)/hand/xacro/process_hand_type_version_side_parameters.xacro" />

File: sr_description/hand/xacro/thumb/thbase.urdf.xacro (robot description, xacro)
@@ -1,9 +1,9 @@
 <robot xmlns:xacro="http://www.ros.org/wiki/xacro"
-xmlns:sensor="http://playerstage.sourceforge.net/gazebo/xmlschema/#sensor"
-xmlns:controller="http://playerstage.sourceforge.net/gazebo/xmlschema/#controller"
-xmlns:joint="http://playerstage.sourceforge.net/gazebo/xmlschema/#slider"
-xmlns:interface="http://playerstage.sourceforge.net/gazebo/xmlschema/#interface"
-xmlns:body="http://playerstage.sourceforge.net/gazebo/xmlschema/#body"
-xmlns:geom="http://playerstage.sourceforge.net/gazebo/xmlschema/#geom">
+       xmlns:sensor="http://playerstage.sourceforge.net/gazebo/xmlschema/#sensor"
+       xmlns:controller="http://playerstage.sourceforge.net/gazebo/xmlschema/#controller"
+       xmlns:joint="http://playerstage.sourceforge.net/gazebo/xmlschema/#slider"
+       xmlns:interface="http://playerstage.sourceforge.net/gazebo/xmlschema/#interface"
+       xmlns:body="http://playerstage.sourceforge.net/gazebo/xmlschema/#body"
+       xmlns:geom="http://playerstage.sourceforge.net/gazebo/xmlschema/#geom">
   <xacro:include filename="$(find sr_description)/hand/xacro/thumb/thbase.gazebo.xacro" />
   <xacro:include filename="$(find sr_description)/hand/xacro/thumb/thbase.transmission.xacro" />
@@ -13,6 +13,5 @@
         <mass value="0.010" />
         <origin xyz="0 0 0" rpy="0 0 0" />
-        <inertia ixx="0.00000016" ixy="0.0" ixz="0.0"
-        iyy="0.00000016" iyz="0.0" izz="0.00000016" />
+        <inertia ixx="0.00000016" ixy="0.0" ixz="0.0" iyy="0.00000016" iyz="0.0" izz="0.00000016" />
       </inertial>
       <visual>
@@ -35,9 +34,7 @@
       <parent link="${parent}" />
       <child link="${prefix}thbase" />
-      <origin xyz="${reflect*0.034} -0.00858 0.029"
-      rpy="0 ${pi/4} ${pi/2-reflect*pi/2}" />
+      <origin xyz="${reflect*0.034} -0.00858 0.029" rpy="0 ${pi/4} ${pi/2-reflect*pi/2}" />
       <axis xyz="0 0 ${reflect*-1}" />
-      <limit lower="${-60/180*pi}" upper="${60/180*pi}"
-      effort="5.0" velocity="4.0" />
+      <limit lower="${-60/180*pi}" upper="${60/180*pi}" effort="5.0" velocity="4.0" />
       <dynamics damping="0.2" />
     </joint>

File: sr_description/hand/xacro/thumb/thdistal.urdf.xacro (robot description, xacro)
@@ -1,9 +1,9 @@
 <robot xmlns:xacro="http://www.ros.org/wiki/xacro"
-xmlns:sensor="http://playerstage.sourceforge.net/gazebo/xmlschema/#sensor"
-xmlns:controller="http://playerstage.sourceforge.net/gazebo/xmlschema/#controller"
-xmlns:joint="http://playerstage.sourceforge.net/gazebo/xmlschema/#slider"
-xmlns:interface="http://playerstage.sourceforge.net/gazebo/xmlschema/#interface"
-xmlns:body="http://playerstage.sourceforge.net/gazebo/xmlschema/#body"
-xmlns:geom="http://playerstage.sourceforge.net/gazebo/xmlschema/#geom">
+       xmlns:sensor="http://playerstage.sourceforge.net/gazebo/xmlschema/#sensor"
+       xmlns:controller="http://playerstage.sourceforge.net/gazebo/xmlschema/#controller"
+       xmlns:joint="http://playerstage.sourceforge.net/gazebo/xmlschema/#slider"
+       xmlns:interface="http://playerstage.sourceforge.net/gazebo/xmlschema/#interface"
+       xmlns:body="http://playerstage.sourceforge.net/gazebo/xmlschema/#body"
+       xmlns:geom="http://playerstage.sourceforge.net/gazebo/xmlschema/#geom">
   <xacro:include filename="$(find sr_description)/hand/xacro/thumb/thdistal.gazebo.xacro" />
   <xacro:include filename="$(find sr_description)/hand/xacro/thumb/thdistal.transmission.xacro" />
@@ -23,6 +23,5 @@
         <origin xyz="0 0 0.02" rpy="0 0 ${-pi/2}" />
         <axis xyz="1 0 0" />
-        <limit lower="${20*pi/180}" upper="${20.1*pi/180}"
-        effort="0.0" velocity="2.0" />
+        <limit lower="${20*pi/180}" upper="${20.1*pi/180}" effort="0.0" velocity="2.0" />
         <dynamics damping="0.5" />
       </joint>
@@ -36,6 +35,5 @@
           <!-- approximated only FIXME -->
           <mass value="0.008" />
-          <inertia ixx="0.0000011" ixy="0.0" ixz="0.0"
-          iyy="0.0000011" iyz="0.0" izz="0.0000005" />
+          <inertia ixx="0.0000011" ixy="0.0" ixz="0.0" iyy="0.0000011" iyz="0.0" izz="0.0000005" />
         </inertial>
         <visual>
@@ -62,11 +60,9 @@
             <topic>${prefix}thdistal_collision</topic>
           </contact>
-          <plugin name="${prefix}thdistal_gazebo_ros_bumper_controller"
-          filename="libgazebo_ros_bumper.so">
+          <plugin name="${prefix}thdistal_gazebo_ros_bumper_controller" filename="libgazebo_ros_bumper.so">
             <alwaysOn>true</alwaysOn>
             <frameName>${prefix}thdistal</frameName>
             <updateRate>100.0</updateRate>
-            <bumperTopicName>
-            contacts/${prefix}th/distal</bumperTopicName>
+            <bumperTopicName>contacts/${prefix}th/distal</bumperTopicName>
           </plugin>
         </sensor>
@@ -84,6 +80,5 @@
           <mass value="0.001" />
           <origin xyz="0 0 0" rpy="0 0 0" />
-          <inertia ixx="0" ixy="0" ixz="0" iyy="0" iyz="0"
-          izz="0" />
+          <inertia ixx="0" ixy="0" ixz="0" iyy="0" iyz="0" izz="0" />
         </inertial>
       </link>
@@ -104,6 +99,5 @@
           <mass value="0.016" />
           <origin xyz="0 0 0.01375" rpy="0 0 0" />
-          <inertia ixx="0.0000021" ixy="0.0" ixz="0.0"
-          iyy="0.0000022" iyz="0.0" izz="0.000001" />
+          <inertia ixx="0.0000021" ixy="0.0" ixz="0.0" iyy="0.0000022" iyz="0.0" izz="0.000001" />
         </inertial>
         <visual>
@@ -150,6 +144,5 @@
         <origin xyz="0 0 0.032" rpy="0 0 ${-pi/2}" />
         <axis xyz="1 0 0" />
-        <limit lower="-${15.0*pi/180}" upper="${90.0*pi/180}" effort="1.0"
-        velocity="4.0" />
+        <limit lower="-${15.0*pi/180}" upper="${90.0*pi/180}" effort="1.0" velocity="4.0" />
         <dynamics damping="0.2" />
       </joint>
@@ -161,6 +154,5 @@
         <inertial>
           <mass value="0.001" />
-          <inertia ixx="0.0" ixy="0.0" ixz="0.0" iyy="0.0"
-          iyz="0.0" izz="0.0" />
+          <inertia ixx="0.0" ixy="0.0" ixz="0.0" iyy="0.0" iyz="0.0" izz="0.0" />
         </inertial>
       </link>

File: sr_description/hand/xacro/thumb/thhub.urdf.xacro (robot description, xacro)
@@ -1,9 +1,9 @@
 <robot xmlns:xacro="http://www.ros.org/wiki/xacro"
-xmlns:sensor="http://playerstage.sourceforge.net/gazebo/xmlschema/#sensor"
-xmlns:controller="http://playerstage.sourceforge.net/gazebo/xmlschema/#controller"
-xmlns:joint="http://playerstage.sourceforge.net/gazebo/xmlschema/#slider"
-xmlns:interface="http://playerstage.sourceforge.net/gazebo/xmlschema/#interface"
-xmlns:body="http://playerstage.sourceforge.net/gazebo/xmlschema/#body"
-xmlns:geom="http://playerstage.sourceforge.net/gazebo/xmlschema/#geom">
+       xmlns:sensor="http://playerstage.sourceforge.net/gazebo/xmlschema/#sensor"
+       xmlns:controller="http://playerstage.sourceforge.net/gazebo/xmlschema/#controller"
+       xmlns:joint="http://playerstage.sourceforge.net/gazebo/xmlschema/#slider"
+       xmlns:interface="http://playerstage.sourceforge.net/gazebo/xmlschema/#interface"
+       xmlns:body="http://playerstage.sourceforge.net/gazebo/xmlschema/#body"
+       xmlns:geom="http://playerstage.sourceforge.net/gazebo/xmlschema/#geom">
   <xacro:include filename="$(find sr_description)/hand/xacro/thumb/thhub.gazebo.xacro" />
   <xacro:include filename="$(find sr_description)/hand/xacro/thumb/thhub.transmission.xacro" />
@@ -13,6 +13,5 @@
         <mass value="0.005" />
         <origin xyz="0 0 0" rpy="0 0 0" />
-        <inertia ixx="0.000001" ixy="0.0" ixz="0.0" iyy="0.000001"
-        iyz="0.0" izz="0.0000003" />
+        <inertia ixx="0.000001" ixy="0.0" ixz="0.0" iyy="0.000001" iyz="0.0" izz="0.0000003" />
       </inertial>
       <visual>
@@ -46,6 +45,5 @@
         <origin xyz="0 0 0.038" rpy="0 0 0" />
         <axis xyz="1 0 0" />
-        <limit lower="${-12/180*pi}" upper="${12/180*pi}"
-        effort="2.0" velocity="4.0" />
+        <limit lower="${-12/180*pi}" upper="${12/180*pi}" effort="2.0" velocity="4.0" />
         <dynamics damping="0.2" />
       </joint>

File: sr_description/hand/xacro/thumb/thmiddle.urdf.xacro (robot description, xacro)
@@ -1,9 +1,9 @@
 <robot xmlns:xacro="http://www.ros.org/wiki/xacro"
-xmlns:sensor="http://playerstage.sourceforge.net/gazebo/xmlschema/#sensor"
-xmlns:controller="http://playerstage.sourceforge.net/gazebo/xmlschema/#controller"
-xmlns:joint="http://playerstage.sourceforge.net/gazebo/xmlschema/#slider"
-xmlns:interface="http://playerstage.sourceforge.net/gazebo/xmlschema/#interface"
-xmlns:body="http://playerstage.sourceforge.net/gazebo/xmlschema/#body"
-xmlns:geom="http://playerstage.sourceforge.net/gazebo/xmlschema/#geom">
+       xmlns:sensor="http://playerstage.sourceforge.net/gazebo/xmlschema/#sensor"
+       xmlns:controller="http://playerstage.sourceforge.net/gazebo/xmlschema/#controller"
+       xmlns:joint="http://playerstage.sourceforge.net/gazebo/xmlschema/#slider"
+       xmlns:interface="http://playerstage.sourceforge.net/gazebo/xmlschema/#interface"
+       xmlns:body="http://playerstage.sourceforge.net/gazebo/xmlschema/#body"
+       xmlns:geom="http://playerstage.sourceforge.net/gazebo/xmlschema/#geom">
   <xacro:include filename="$(find sr_description)/hand/xacro/thumb/thmiddle.gazebo.xacro" />
   <xacro:include filename="$(find sr_description)/hand/xacro/thumb/thmiddle.transmission.xacro" />
@@ -14,6 +14,5 @@
         <mass value="0.020" />
         <origin xyz="0 0 0.016" rpy="0 0 0" />
-        <inertia ixx="0.0000051" ixy="0.0" ixz="0.0"
-        iyy="0.0000051" iyz="0.0" izz="0.00000121" />
+        <inertia ixx="0.0000051" ixy="0.0" ixz="0.0" iyy="0.0000051" iyz="0.0" izz="0.00000121" />
       </inertial>
       <visual>

File: sr_description/hand/xacro/thumb/thproximal.urdf.xacro (robot description, xacro)
@@ -1,9 +1,9 @@
 <robot xmlns:xacro="http://www.ros.org/wiki/xacro"
-xmlns:sensor="http://playerstage.sourceforge.net/gazebo/xmlschema/#sensor"
-xmlns:controller="http://playerstage.sourceforge.net/gazebo/xmlschema/#controller"
-xmlns:joint="http://playerstage.sourceforge.net/gazebo/xmlschema/#slider"
-xmlns:interface="http://playerstage.sourceforge.net/gazebo/xmlschema/#interface"
-xmlns:body="http://playerstage.sourceforge.net/gazebo/xmlschema/#body"
-xmlns:geom="http://playerstage.sourceforge.net/gazebo/xmlschema/#geom">
+       xmlns:sensor="http://playerstage.sourceforge.net/gazebo/xmlschema/#sensor"
+       xmlns:controller="http://playerstage.sourceforge.net/gazebo/xmlschema/#controller"
+       xmlns:joint="http://playerstage.sourceforge.net/gazebo/xmlschema/#slider"
+       xmlns:interface="http://playerstage.sourceforge.net/gazebo/xmlschema/#interface"
+       xmlns:body="http://playerstage.sourceforge.net/gazebo/xmlschema/#body"
+       xmlns:geom="http://playerstage.sourceforge.net/gazebo/xmlschema/#geom">
   <xacro:include filename="$(find sr_description)/hand/xacro/thumb/thproximal.gazebo.xacro" />
   <xacro:include filename="$(find sr_description)/hand/xacro/thumb/thproximal.transmission.xacro" />

File: sr_description/other/xacro/gazebo.urdf.xacro (robot description, xacro)
@@ -1,6 +1,6 @@
 <?xml version="1.0"?>
 <robot xmlns:sensor="http://playerstage.sourceforge.net/gazebo/xmlschema/#sensor"
-xmlns:controller="http://playerstage.sourceforge.net/gazebo/xmlschema/#controller"
-xmlns:interface="http://playerstage.sourceforge.net/gazebo/xmlschema/#interface">
+       xmlns:controller="http://playerstage.sourceforge.net/gazebo/xmlschema/#controller"
+       xmlns:interface="http://playerstage.sourceforge.net/gazebo/xmlschema/#interface">
   <gazebo>
     <plugin name="gazebo_ros_control" filename="libgazebo_ros_control.so">

File: sr_description/robots/sr_hand_bimanual.urdf.xacro (robot description, xacro)
@@ -3,5 +3,5 @@
        xmlns:controller="http://playerstage.sourceforge.net/gazebo/xmlschema/#controller"
        xmlns:interface="http://playerstage.sourceforge.net/gazebo/xmlschema/#interface"
-       name="bumanual_shadowhand_motor">
+       name="bimanual_shadowhand_motor">
   <xacro:include filename="$(find sr_description)/other/xacro/materials.urdf.xacro"/>
   <xacro:include filename="$(find sr_description)/hand/xacro/hand.urdf.xacro"/>

File: sr_description/test/test_process_fingers_parameter.xacro (robot description, xacro)
@@ -4,5 +4,5 @@
 		<xacro:property name="input" value="${fingers}" lazy_eval="false" />
 		<xacro:include filename="$(find sr_description)/hand/xacro/process_fingers_parameter.xacro" />
-	${input} ${msg} : ${fingers}
+		${input} ${msg} : ${fingers}
 	</xacro:macro>
 	<xacro:test />

Commit message: removing stl reference

File: sr_description/hand/xacro/finger/distal/distal.urdf.xacro (robot description, xacro)
@@ -19,5 +19,5 @@
         <geometry name="${prefix}${link_prefix}distal_visual">
           <xacro:if value="${tip_sensor == 'pst'}">
-            <mesh filename="package://sr_description/meshes/components/f_distal/pst/f_distal_pst.stl"
+            <mesh filename="package://sr_description/meshes/components/f_distal/pst/f_distal_pst.dae"
                   scale="0.001 0.001 0.001" />
           </xacro:if>
@@ -35,5 +35,5 @@
         <geometry name="${prefix}${link_prefix}distal_collision_geom">
           <xacro:if value="${tip_sensor == 'pst'}">
-            <mesh filename="package://sr_description/meshes/components/f_distal/pst/f_distal_pst.stl"
+            <mesh filename="package://sr_description/meshes/components/f_distal/pst/f_distal_pst.dae"
                   scale="0.001 0.001 0.001" />
           </xacro:if>
