Commit message: all changed to dae

File: sr_description/hand/xacro/finger/distal/distal.urdf.xacro (robot description, xacro)
@@ -23,5 +23,5 @@
           </xacro:if>
           <xacro:if value="${tip_sensor == 'bt_sp'}">
-            <mesh filename="package://sr_description/meshes/components/f_distal/bt_sp/f_distal_bt_sp.stl"
+            <mesh filename="package://sr_description/meshes/components/f_distal/bt_sp/f_distal_bt_sp.dae"
                   scale="0.001 0.001 0.001" />
           </xacro:if>
@@ -39,5 +39,5 @@
           </xacro:if>
           <xacro:if value="${tip_sensor == 'bt_sp'}">
-            <mesh filename="package://sr_description/meshes/components/f_distal/bt_sp/f_distal_bt_sp.stl"
+            <mesh filename="package://sr_description/meshes/components/f_distal/bt_sp/f_distal_bt_sp.dae"
                   scale="0.001 0.001 0.001" />
           </xacro:if>

File: sr_description/hand/xacro/forearm/forearm_e.urdf.xacro (robot description, xacro)
@@ -27,5 +27,5 @@
         <origin xyz="0 0 0" rpy="0 0 0" />
         <geometry name="${prefix}forearm_collision">
-          <mesh filename="package://sr_description/meshes/components/forearm/forearm_collision_${hand_version}.stl" scale="0.001 0.001 0.001" />
+          <mesh filename="package://sr_description/meshes/components/forearm/forearm_collision_${hand_version}.dae" scale="0.001 0.001 0.001" />
         </geometry>
       </collision>
@@ -41,5 +41,5 @@
         <origin rpy="0 -1.57 -1.57" xyz="0.0 0.067 0.0045"/>
         <geometry name="${prefix}cable_extr_visualisation">
-          <mesh filename="package://sr_description/meshes/components/cable_connector/cable_connector_base_${hand_version}.stl" scale="0.001 0.001 0.001" />
+          <mesh filename="package://sr_description/meshes/components/cable_connector/cable_connector_base_${hand_version}.dae" scale="0.001 0.001 0.001" />
         </geometry>
       </visual>
@@ -47,5 +47,5 @@
         <origin rpy="0 -1.57 -1.57" xyz="0.0 0.067 0.0045"/>
         <geometry name="${prefix}cable_extr_collision">
-          <mesh filename="package://sr_description/meshes/components/cable_connector/cable_connector_base_${hand_version}.stl" scale="0.001 0.001 0.001" />
+          <mesh filename="package://sr_description/meshes/components/cable_connector/cable_connector_base_${hand_version}.dae" scale="0.001 0.001 0.001" />
         </geometry>
       </collision-->

File: sr_description/hand/xacro/forearm/forearm_g.urdf.xacro (robot description, xacro)
@@ -26,5 +26,5 @@
         <origin rpy="0 -1.57 -1.57" xyz="0.0 0.055 0.0"/>
         <geometry name="${prefix}cable_extr_visualisation">
-          <mesh filename="package://sr_description/meshes/components/cable_connector/cable_connector_base_${hand_version}.stl" scale="1 1 1" />
+          <mesh filename="package://sr_description/meshes/components/cable_connector/cable_connector_base_${hand_version}.dae" scale="1 1 1" />
         </geometry>
       </visual>
@@ -32,5 +32,5 @@
         <origin rpy="0 -1.57 -1.57" xyz="0.0 0.055 0.0"/>
         <geometry name="${prefix}cable_extr_collision">
-          <mesh filename="package://sr_description/components/cable_connector/cable_connector_base_${hand_version}.stl" scale="1 1 1" />
+          <mesh filename="package://sr_description/components/cable_connector/cable_connector_base_${hand_version}.dae" scale="1 1 1" />
         </geometry>
       </collision-->

File: sr_description/hand/xacro/palm/palm_e.urdf.xacro (robot description, xacro)
@@ -19,5 +19,5 @@
         <origin xyz="0 0 0" rpy="0 0 0" />
         <geometry name="${prefix}palm_visual">
-          <mesh filename="package://sr_description/meshes/components/palm/palm_${hand_version}.stl"
+          <mesh filename="package://sr_description/meshes/components/palm/palm_${hand_version}.dae"
                 scale="${reflect*0.001} 0.001 0.001" />
         </geometry>

File: sr_description/hand/xacro/thumb/thdistal.urdf.xacro (robot description, xacro)
@@ -105,9 +105,9 @@
           <geometry name="${prefix}thdistal_visual">
             <xacro:if value="${tip_sensor == 'pst'}">
-              <mesh filename="package://sr_description/meshes/components/th_distal/pst/th_distal_pst.stl"
+              <mesh filename="package://sr_description/meshes/components/th_distal/pst/th_distal_pst.dae"
                     scale="0.001 0.001 0.001" />
             </xacro:if>
             <xacro:if value="${tip_sensor == 'bt_sp'}">
-              <mesh filename="package://sr_description/meshes/components/th_distal/bt_sp/th_distal_bt_sp.stl"
+              <mesh filename="package://sr_description/meshes/components/th_distal/bt_sp/th_distal_bt_sp.dae"
                     scale="0.001 0.001 0.001" />
             </xacro:if>
@@ -125,9 +125,9 @@
           <geometry name="${prefix}thmiddle_collision_geom">
             <xacro:if value="${tip_sensor == 'pst'}">
-              <mesh filename="package://sr_description/meshes/components/th_distal/pst/th_distal_pst.stl"
+              <mesh filename="package://sr_description/meshes/components/th_distal/pst/th_distal_pst.dae"
                     scale="0.001 0.001 0.001" />
             </xacro:if>
             <xacro:if value="${tip_sensor == 'bt_sp'}">
-              <mesh filename="package://sr_description/meshes/components/th_distal/bt_sp/th_distal_bt_sp.stl"
+              <mesh filename="package://sr_description/meshes/components/th_distal/bt_sp/th_distal_bt_sp.dae"
                     scale="0.001 0.001 0.001" />
             </xacro:if>

Commit message: Switching to new xacros (#130)
* F refactoring sr description multi (#126)

* Remove redundant definition of pi

pi is available globally in xacro as python's math.pi

* Delete unused meshes in ubi_tactiles

* Remove use of ubi param

* Remove ubi params

* Replace $(find xacro)/xacro -> xacro

* Remove deprecated --inorder option

* Fix missing xacro namespace prefixes

* Fix typo

* Improved xacro for modularity and to permit sensor selection

Modern xacro allows to automatically forward macro arguments when they are
defined with the arg:=^ syntax. Using this feature simplifies macro calling.

Also, instead of specifying hand attributes with an ever-growing set of
binary parameters, this commit introduces parameters hand_type and
(palm|prox|mid|tip)_sensor to modularize parameterization.
This allows for more flexible definition of the (tactile) sensors used across the hand.

Using a value of 'none' for those sensors allows to deactivate (Gazebo) sensors.

Backward compatibility for old parameters is maintained via file backward_compat.urdf.xacro,
which translates from old to new parameters.

* Add compatibility test

Cloned all files from robots/*.urdf.xacro prior to this PR into test/robots.old.
Run xacro on all corresponding files and compare their content.

* Fix backward compatibility

- Restore deleted files required by compatibility test
- Fix use of deprecated properties
- Fix use of deprecated parameters
- Undo unrelated changes w.r.t. upstream
- Fix extra_lite hands: it is missing MF not FF

* More simplifications

- Simpify one_finger_unit.urdf.xacro
  There is only one finger. No need to pass *_sensors. A single one is sufficient.
  Also, a fingers parameter doesn't make sense.

- Reduce number of xacro:if in fingers.urdf.xacro

- Plain string default parameters don't need to be quoted

* More specific variable tests

Using `'text' in variable` is a rather sloppy equivalence check.
This commit attempts to harden these checks using the following regexp
replacements:

- More specific test of hand_type
  ('hand.+?') in ([a-z_]+)  ->  $2.startswith($1)

- More specific variable tests
  ('.+') in ([a-z_]+)  ->  $2 == $1

* Simplify if-else clauses

Improve extensibility (adding more sensors) by emloying an exclusive-if-and-final-else
strategy, utilizing a helper variable. This way we avoid augmenting the list in the
'sensor in [...]' tests.

* Issue deprecation warning

Use python's None value as default to know whether old parameters were specified.

* Deprecate specific hand.urdf.xacro files

* More readable hand_types: muscle, muscletrans, motor, motor+

- hand_mt -> muscletrans
- hand_m -> muscle, regexp: (["' ])hand_m -> $1muscle
- hand_e_plus -> motor+
- hand_e -> motor

* Make fingers parameter a string

* Python 2.x compatibility

As xacro returns unicode objects from property evaluations
we cannot apply str.lower to them in Python 2.x
In Python 3.x str and unicode is essentially the same.

* Simplify syntax for sensor specification

Use textual sensor specifications:
- tip_sensors=bio
- tip_sensors='th=bio, ff=bio, mf=std, rf=std, lf=none'
- tip_sensors='bio, bio, std, std, none'

- Rename backward_compat.urdf.xacro -> process_sensor_parameters.xacro
- Introduce macro validate_tokens

* Apply new sensor specification

* Internally use dotified dict for *_sensors

* hand e working with versions and hand type

* distal refactored

* Deleted deprecated changelog

* Replaced std

* Replaced muscletrans with hand_c

* Fixed finger

* Fixed Thumb plus a few issues from finger forearm and palm

* Fixed wrist

* Moved files to legacy folder for now

* Replaced full_hand with hand xacro and updated hand_g

* Fixed hand lite and extra lite

* Removed arm and old meshes

* Moved gazebo and materials to a common folder

* Fixed xacro errors

* Added mucle hand

* Reformated load files

* Refactored meshes to use only components

* Added all robots to legacy folder for now. And left only two robots: unimanual and bimanual

* Adapting test script after xacro refactoring

* Refactoring sr_description: adapted test and added more parameters validation (#124)

* Removing robots.old folder

* Lint fixes

* Fixing CMakeLists

* Removing whitespace

* Applying changes from https://github.com/ubi-agni/sr_common/pull/2

* Adapting tests to refactored sr_description

* Adding validation xacro

* Update process_hand_type_parameter.xacro

* Updated validation xacro and small fixes

* Update test_models.sh

* Fixed validation of parameters

* Fixing formtating and deleted unnecessary files

* Work in progress

* Removed unnecessary files

Co-authored-by: Beatriz Leon <beatriz@shadowrobot.com>

* Update process_hand_type_version_side_parameters.xacro

* refactoring

* cleaning

* according to review

Co-authored-by: Robert Haschke <rhaschke@techfak.uni-bielefeld.de>
Co-authored-by: Guillaume Walck <gwalck@techfak.uni-bielefeld.de>
Co-authored-by: Beatriz Leon <beatriz@shadowrobot.com>
Co-authored-by: maxzieba <max@shadowrobot.com>
Co-authored-by: maxzieba <77073326+maxzieba@users.noreply.github.com>

* Migrating to dae and adding materials (#129)

* testing

* migrating to daes

* removing stl reference

* all changed to dae

* adding material to palm

* Revert "adding material to palm"

This reverts commit 933026584e9373cfa22654a25ca7488c398033e0.

* removing redundant dae elements

* all meshes colored

* fixing hand c colors

* fixing test

* Fixing the color of wrist mesh (#131)

* updating

* testing

* testing

* testing

* fixing

* removing nosetests

* excluding copyright check

* acording to review

Co-authored-by: Robert Haschke <rhaschke@techfak.uni-bielefeld.de>
Co-authored-by: Guillaume Walck <gwalck@techfak.uni-bielefeld.de>
Co-authored-by: Beatriz Leon <beatriz@shadowrobot.com>
Co-authored-by: maxzieba <max@shadowrobot.com>
Co-authored-by: maxzieba <77073326+maxzieba@users.noreply.github.com>

File: sr_description/hand/xacro/finger/distal/distal.urdf.xacro (robot description, xacro)
@@ -1,102 +1,52 @@
 <robot xmlns:xacro="http://www.ros.org/wiki/xacro"
-xmlns:sensor="http://playerstage.sourceforge.net/gazebo/xmlschema/#sensor"
-xmlns:controller="http://playerstage.sourceforge.net/gazebo/xmlschema/#controller"
-xmlns:joint="http://playerstage.sourceforge.net/gazebo/xmlschema/#slider"
-xmlns:interface="http://playerstage.sourceforge.net/gazebo/xmlschema/#interface"
-xmlns:body="http://playerstage.sourceforge.net/gazebo/xmlschema/#body"
-xmlns:geom="http://playerstage.sourceforge.net/gazebo/xmlschema/#geom">
+       xmlns:sensor="http://playerstage.sourceforge.net/gazebo/xmlschema/#sensor"
+       xmlns:controller="http://playerstage.sourceforge.net/gazebo/xmlschema/#controller"
+       xmlns:joint="http://playerstage.sourceforge.net/gazebo/xmlschema/#slider"
+       xmlns:interface="http://playerstage.sourceforge.net/gazebo/xmlschema/#interface"
+       xmlns:body="http://playerstage.sourceforge.net/gazebo/xmlschema/#body"
+       xmlns:geom="http://playerstage.sourceforge.net/gazebo/xmlschema/#geom">
   <xacro:include filename="$(find sr_description)/hand/xacro/finger/distal/distal.gazebo.xacro" />
   <xacro:include filename="$(find sr_description)/hand/xacro/finger/distal/distal.transmission.xacro" />
-  <!-- muscle is true for muscle hand or false for motor hand -->
-  <!-- bio is true for biotac finger or false for standard finger -->
-  <!-- bt_sp is true for BT_SP finger or false for standard finger -->
-  <!-- ubi is true for ubi finger or false for standard finger -->
-  <!-- eli is true for ellipsoid fingertip or false for standard finger -->
-  <!-- prefix can be anything but usually is "r_" or  "l_" for right and left hands distinction -->
-  <!-- link_prefix prepends fingername to the link names -->
-  <!-- joint_prefix prepends fingername to the joint names -->
-  <!-- parent is the parent link for the joint -->
-  <xacro:macro name="distal"
-  params="muscle bio bt_sp ubi eli prefix link_prefix joint_prefix parent">
+  <xacro:macro name="distal" params="prefix:=^ link_prefix:=^ joint_prefix:=^ tip_sensor:=^|pst parent">
     <link name="${prefix}${link_prefix}distal">
       <inertial>
         <mass value="0.012" />
         <origin xyz="0 0 0.012" />
-        <inertia ixx="0.00000094" ixy="0.0" ixz="0.0"
-		 iyy="0.0000011" iyz="0.0" izz="0.00000053" />
+        <inertia ixx="0.00000094" ixy="0.0" ixz="0.0" iyy="0.0000011" iyz="0.0" izz="0.00000053" />
       </inertial>
       <visual>
         <origin xyz="0 0 0" rpy="0 0 0" />
         <geometry name="${prefix}${link_prefix}distal_visual">
-          <xacro:if value="${ubi}">
-            <!-- Ubi distal -->
-            <mesh filename="package://sr_description/meshes/hand/ubi_tactiles/ubi_tip_visual.dae"
-		  scale="0.001 0.001 0.001" />
+          <xacro:if value="${tip_sensor == 'pst'}">
+            <mesh filename="package://sr_description/meshes/components/f_distal/pst/f_distal_pst.dae"
+                  scale="0.001 0.001 0.001" />
           </xacro:if>
-          <xacro:unless value="${ubi}">
-            <xacro:if value="${eli}">
-              <!-- Ellispoid distal  -->
-              <mesh filename="package://sr_description/meshes/hand/ellipsoids/distal_ellipsoid_visual.dae"
-		    scale="0.001 0.001 0.001" />
-            </xacro:if>
-            <xacro:unless value="${eli}">
-              <xacro:if value="${bio}">
-                <!-- biotac distal  -->
-                <mesh filename="package://sr_description/meshes/hand/F1.dae"
-                      scale="0.001 0.001 0.001" />
-              </xacro:if>
-              <xacro:unless value="${bio}">
-		<xacro:if value="${bt_sp}">
-                  <!-- bt_sp distal  -->
-                  <mesh filename="package://sr_description/meshes/hand/biotacs/sp.dae" />
-		</xacro:if>
-		<xacro:unless value="${bt_sp}">
-                  <!-- Standard distal  -->
-                  <mesh filename="package://sr_description/meshes/hand/F1.dae"
-			scale="0.001 0.001 0.001" />
-		</xacro:unless>
-              </xacro:unless>
-            </xacro:unless>
-          </xacro:unless>
+          <xacro:if value="${tip_sensor == 'bt_sp'}">
+            <mesh filename="package://sr_description/meshes/components/f_distal/bt_sp/f_distal_bt_sp.dae"
+                  scale="0.001 0.001 0.001" />
+          </xacro:if>
+          <xacro:if value="${tip_sensor == 'bt_2p'}">
+            <mesh filename="package://sr_description/meshes/components/f_distal/bt_2p/f_distal_bt_2p.dae" />
+          </xacro:if>
         </geometry>
-        <!-- <material name="Grey" /> -->
       </visual>
       <collision>
         <origin xyz="0 0 0" rpy="0 0 0" />
         <geometry name="${prefix}${link_prefix}distal_collision_geom">
-          <xacro:if value="${ubi}">
-            <!-- Ubi distal -->
-            <mesh filename="package://sr_description/meshes/hand/ubi_tactiles/ubi_tip_collision.dae"
-            scale="0.001 0.001 0.001" />
+          <xacro:if value="${tip_sensor == 'pst'}">
+            <mesh filename="package://sr_description/meshes/components/f_distal/pst/f_distal_pst.dae"
+                  scale="0.001 0.001 0.001" />
           </xacro:if>
-          <xacro:unless value="${ubi}">
-            <xacro:if value="${eli}">
-              <!-- Ellispoid distal  -->
-              <mesh filename="package://sr_description/meshes/hand/ellipsoids/distal_ellipsoid.dae"
-              scale="0.001 0.001 0.001" />
-            </xacro:if>
-            <xacro:unless value="${eli}">
-              <xacro:if value="${bio}">
-                <!-- biotac distal  -->
-                <mesh filename="package://sr_description/meshes/hand/F1.dae"
-                scale="0.001 0.001 0.001" />
-              </xacro:if>
-              <xacro:unless value="${bio}">
-		<xacro:if value="${bt_sp}">
-                  <!-- bt_sp distal  -->
-                  <mesh filename="package://sr_description/meshes/hand/biotacs/sp.dae" />
-		</xacro:if>
-		<xacro:unless value="${bt_sp}">
-                  <!-- Standard distal  -->
-                  <mesh filename="package://sr_description/meshes/hand/F1.dae"
-			scale="0.001 0.001 0.001" />
-		</xacro:unless>
-              </xacro:unless>
-            </xacro:unless>
-          </xacro:unless>
+          <xacro:if value="${tip_sensor == 'bt_sp'}">
+            <mesh filename="package://sr_description/meshes/components/f_distal/bt_sp/f_distal_bt_sp.dae"
+                  scale="0.001 0.001 0.001" />
+          </xacro:if>
+          <xacro:if value="${tip_sensor == 'bt_2p'}">
+            <mesh filename="package://sr_description/meshes/components/f_distal/bt_2p/f_distal_bt_2p.dae" />
+          </xacro:if>
         </geometry>
       </collision>
     </link>
-    <xacro:unless value="${bio}">
+    <xacro:unless value="${tip_sensor == 'bt_2p'}">
       <joint name="${prefix}${joint_prefix}J1" type="revolute">
         <parent link="${parent}" />
@@ -104,14 +54,6 @@
         <origin xyz="0 0 0.025" rpy="0 0 0" />
         <axis xyz="1 0 0" />
-        <xacro:if value="${bio}">
-          <!-- biotac fixed distal joint -->
-          <limit lower="${20/180*pi}" upper="${20/180*pi}"
-          effort="10" velocity="2.0" />
-        </xacro:if>
-        <xacro:unless value="${bio}">
-          <!-- standard distal joint -->
-          <limit lower="0" upper="${pi/2}" effort="2"
-          velocity="2.0" />
-        </xacro:unless>
+        <!-- standard distal joint -->
+        <limit lower="0" upper="${pi/2}" effort="2" velocity="2.0" />
         <dynamics damping="0.1" />
       </joint>
@@ -123,6 +65,5 @@
         <inertial>
           <mass value="0.001" />
-          <inertia ixx="0.0" ixy="0.0" ixz="0.0" iyy="0.0"
-          iyz="0.0" izz="0.0" />
+          <inertia ixx="0.0" ixy="0.0" ixz="0.0" iyy="0.0" iyz="0.0" izz="0.0" />
         </inertial>
       </link>
@@ -134,6 +75,5 @@
     </xacro:unless>
     <!-- extensions -->
-    <xacro:distal_gazebo prefix="${prefix}"
-    link_prefix="${link_prefix}" />
+    <xacro:distal_gazebo />
   </xacro:macro>
 </robot>

File: sr_description/hand/xacro/palm/imu.urdf.xacro (robot description, xacro)
@@ -1,4 +1,4 @@
 <robot xmlns:xacro="http://www.ros.org/wiki/xacro" name="shadowhand_motor">
-  <xacro:macro name="imu_sensor" params="prefix">
+  <xacro:macro name="imu_sensor" params="prefix:=^">
     <link name="${prefix}imu"/>
     <joint name="${prefix}palm_to_imu" type="fixed">
@@ -7,9 +7,4 @@
       <origin xyz="0.01785 0.00765 0.049125" rpy="-1.5707963 3.141592 0.0"/>
     </joint>
-    <sensor name="${prefix}imu" update_rate="100">
-      <parent link="${prefix}imu"/>
-      <origin xyz="0 0 0" rpy="0 0 0"/>
-      <imu />
-    </sensor>
   </xacro:macro>
 </robot>
