Commit message: Switching to new xacros (#130)
* F refactoring sr description multi (#126)

* Remove redundant definition of pi

pi is available globally in xacro as python's math.pi

* Delete unused meshes in ubi_tactiles

* Remove use of ubi param

* Remove ubi params

* Replace $(find xacro)/xacro -> xacro

* Remove deprecated --inorder option

* Fix missing xacro namespace prefixes

* Fix typo

* Improved xacro for modularity and to permit sensor selection

Modern xacro allows to automatically forward macro arguments when they are
defined with the arg:=^ syntax. Using this feature simplifies macro calling.

Also, instead of specifying hand attributes with an ever-growing set of
binary parameters, this commit introduces parameters hand_type and
(palm|prox|mid|tip)_sensor to modularize parameterization.
This allows for more flexible definition of the (tactile) sensors used across the hand.

Using a value of 'none' for those sensors allows to deactivate (Gazebo) sensors.

Backward compatibility for old parameters is maintained via file backward_compat.urdf.xacro,
which translates from old to new parameters.

* Add compatibility test

Cloned all files from robots/*.urdf.xacro prior to this PR into test/robots.old.
Run xacro on all corresponding files and compare their content.

* Fix backward compatibility

- Restore deleted files required by compatibility test
- Fix use of deprecated properties
- Fix use of deprecated parameters
- Undo unrelated changes w.r.t. upstream
- Fix extra_lite hands: it is missing MF not FF

* More simplifications

- Simpify one_finger_unit.urdf.xacro
  There is only one finger. No need to pass *_sensors. A single one is sufficient.
  Also, a fingers parameter doesn't make sense.

- Reduce number of xacro:if in fingers.urdf.xacro

- Plain string default parameters don't need to be quoted

* More specific variable tests

Using `'text' in variable` is a rather sloppy equivalence check.
This commit attempts to harden these checks using the following regexp
replacements:

- More specific test of hand_type
  ('hand.+?') in ([a-z_]+)  ->  $2.startswith($1)

- More specific variable tests
  ('.+') in ([a-z_]+)  ->  $2 == $1

* Simplify if-else clauses

Improve extensibility (adding more sensors) by emloying an exclusive-if-and-final-else
strategy, utilizing a helper variable. This way we avoid augmenting the list in the
'sensor in [...]' tests.

* Issue deprecation warning

Use python's None value as default to know whether old parameters were specified.

* Deprecate specific hand.urdf.xacro files

* More readable hand_types: muscle, muscletrans, motor, motor+

- hand_mt -> muscletrans
- hand_m -> muscle, regexp: (["' ])hand_m -> $1muscle
- hand_e_plus -> motor+
- hand_e -> motor

* Make fingers parameter a string

* Python 2.x compatibility

As xacro returns unicode objects from property evaluations
we cannot apply str.lower to them in Python 2.x
In Python 3.x str and unicode is essentially the same.

* Simplify syntax for sensor specification

Use textual sensor specifications:
- tip_sensors=bio
- tip_sensors='th=bio, ff=bio, mf=std, rf=std, lf=none'
- tip_sensors='bio, bio, std, std, none'

- Rename backward_compat.urdf.xacro -> process_sensor_parameters.xacro
- Introduce macro validate_tokens

* Apply new sensor specification

* Internally use dotified dict for *_sensors

* hand e working with versions and hand type

* distal refactored

* Deleted deprecated changelog

* Replaced std

* Replaced muscletrans with hand_c

* Fixed finger

* Fixed Thumb plus a few issues from finger forearm and palm

* Fixed wrist

* Moved files to legacy folder for now

* Replaced full_hand with hand xacro and updated hand_g

* Fixed hand lite and extra lite

* Removed arm and old meshes

* Moved gazebo and materials to a common folder

* Fixed xacro errors

* Added mucle hand

* Reformated load files

* Refactored meshes to use only components

* Added all robots to legacy folder for now. And left only two robots: unimanual and bimanual

* Adapting test script after xacro refactoring

* Refactoring sr_description: adapted test and added more parameters validation (#124)

* Removing robots.old folder

* Lint fixes

* Fixing CMakeLists

* Removing whitespace

* Applying changes from https://github.com/ubi-agni/sr_common/pull/2

* Adapting tests to refactored sr_description

* Adding validation xacro

* Update process_hand_type_parameter.xacro

* Updated validation xacro and small fixes

* Update test_models.sh

* Fixed validation of parameters

* Fixing formtating and deleted unnecessary files

* Work in progress

* Removed unnecessary files

Co-authored-by: Beatriz Leon <beatriz@shadowrobot.com>

* Update process_hand_type_version_side_parameters.xacro

* refactoring

* cleaning

* according to review

Co-authored-by: Robert Haschke <rhaschke@techfak.uni-bielefeld.de>
Co-authored-by: Guillaume Walck <gwalck@techfak.uni-bielefeld.de>
Co-authored-by: Beatriz Leon <beatriz@shadowrobot.com>
Co-authored-by: maxzieba <max@shadowrobot.com>
Co-authored-by: maxzieba <77073326+maxzieba@users.noreply.github.com>

* Migrating to dae and adding materials (#129)

* testing

* migrating to daes

* removing stl reference

* all changed to dae

* adding material to palm

* Revert "adding material to palm"

This reverts commit 933026584e9373cfa22654a25ca7488c398033e0.

* removing redundant dae elements

* all meshes colored

* fixing hand c colors

* fixing test

* Fixing the color of wrist mesh (#131)

* updating

* testing

* testing

* testing

* fixing

* removing nosetests

* excluding copyright check

* acording to review

Co-authored-by: Robert Haschke <rhaschke@techfak.uni-bielefeld.de>
Co-authored-by: Guillaume Walck <gwalck@techfak.uni-bielefeld.de>
Co-authored-by: Beatriz Leon <beatriz@shadowrobot.com>
Co-authored-by: maxzieba <max@shadowrobot.com>
Co-authored-by: maxzieba <77073326+maxzieba@users.noreply.github.com>

File: sr_description/hand/xacro/thumb/thdistal.urdf.xacro (robot description, xacro)
@@ -1,22 +1,13 @@
 <robot xmlns:xacro="http://www.ros.org/wiki/xacro"
-xmlns:sensor="http://playerstage.sourceforge.net/gazebo/xmlschema/#sensor"
-xmlns:controller="http://playerstage.sourceforge.net/gazebo/xmlschema/#controller"
-xmlns:joint="http://playerstage.sourceforge.net/gazebo/xmlschema/#slider"
-xmlns:interface="http://playerstage.sourceforge.net/gazebo/xmlschema/#interface"
-xmlns:body="http://playerstage.sourceforge.net/gazebo/xmlschema/#body"
-xmlns:geom="http://playerstage.sourceforge.net/gazebo/xmlschema/#geom">
+       xmlns:sensor="http://playerstage.sourceforge.net/gazebo/xmlschema/#sensor"
+       xmlns:controller="http://playerstage.sourceforge.net/gazebo/xmlschema/#controller"
+       xmlns:joint="http://playerstage.sourceforge.net/gazebo/xmlschema/#slider"
+       xmlns:interface="http://playerstage.sourceforge.net/gazebo/xmlschema/#interface"
+       xmlns:body="http://playerstage.sourceforge.net/gazebo/xmlschema/#body"
+       xmlns:geom="http://playerstage.sourceforge.net/gazebo/xmlschema/#geom">
   <xacro:include filename="$(find sr_description)/hand/xacro/thumb/thdistal.gazebo.xacro" />
   <xacro:include filename="$(find sr_description)/hand/xacro/thumb/thdistal.transmission.xacro" />
-  <!-- muscle is true for muscle hand or false for motor hand -->
-  <!-- bio is true for biotac finger or false for standard finger -->
-  <!-- bt_sp is true for BT_SP finger or false for standard finger -->
-  <!-- ubi is true for ubi finger or false for standard finger -->
-  <!-- eli is true for ellipsoid fingertip or false for standard finger -->
-  <!-- prefix can be anything but usually is "r_" or  "l_" for right and left hands distinction -->
-  <!-- parent is the parent link for the first joint -->
-  <xacro:macro name="thdistal"
-  params="muscle bio bt_sp ubi eli prefix parent">
-    <xacro:if value="${bio}">
-      <!--    BIOTAC -->
+  <xacro:macro name="thdistal" params="tip_sensor:=^|pst prefix:=^ parent">
+    <xacro:if value="${tip_sensor == 'bt_2p'}">
       <link name="${prefix}thdistal_J1_dummy">
         <inertial>
@@ -32,6 +23,5 @@
         <origin xyz="0 0 0.02" rpy="0 0 ${-pi/2}" />
         <axis xyz="1 0 0" />
-        <limit lower="${20*pi/180}" upper="${20.1*pi/180}"
-        effort="0.0" velocity="2.0" />
+        <limit lower="${20*pi/180}" upper="${20.1*pi/180}" effort="0.0" velocity="2.0" />
         <dynamics damping="0.5" />
       </joint>
@@ -45,12 +35,10 @@
           <!-- approximated only FIXME -->
           <mass value="0.008" />
-          <inertia ixx="0.0000011" ixy="0.0" ixz="0.0"
-          iyy="0.0000011" iyz="0.0" izz="0.0000005" />
+          <inertia ixx="0.0000011" ixy="0.0" ixz="0.0" iyy="0.0000011" iyz="0.0" izz="0.0000005" />
         </inertial>
         <visual>
           <origin xyz="0 0 0" rpy="0 0 0" />
           <geometry name="${prefix}th_distal_visual">
-            <!-- <mesh filename="package://sr_description/meshes/hand/biotacs/biotac.stl" scale="0.0254 0.0254 0.0254" /> -->
-            <mesh filename="package://sr_description/meshes/hand/biotacs/biotac_decimated.dae"
+            <mesh filename="package://sr_description/meshes/components/th_distal/bt_2p/th_distal_bt_2p.dae"
             scale="0.0254 0.0254 0.0254" />
           </geometry>
@@ -59,7 +47,5 @@
         <collision>
           <geometry name="${prefix}th_distal_collision_geom">
-            <!-- <box size="0.001 0.001 0.001" /> -->
-            <!-- <mesh filename="package://sr_description/meshes/hand/biotacs/biotac-v5.stl" scale="0.0254 0.0254 0.0254" /> -->
-            <mesh filename="package://sr_description/meshes/hand/biotacs/biotac_decimated.dae"
+            <mesh filename="package://sr_description/meshes/components/th_distal/bt_2p/th_distal_bt_2p.dae"
             scale="0.0254 0.0254 0.0254" />
           </geometry>
@@ -74,11 +60,9 @@
             <topic>${prefix}thdistal_collision</topic>
           </contact>
-          <plugin name="${prefix}thdistal_gazebo_ros_bumper_controller"
-          filename="libgazebo_ros_bumper.so">
+          <plugin name="${prefix}thdistal_gazebo_ros_bumper_controller" filename="libgazebo_ros_bumper.so">
             <alwaysOn>true</alwaysOn>
             <frameName>${prefix}thdistal</frameName>
             <updateRate>100.0</updateRate>
-            <bumperTopicName>
-            contacts/${prefix}th/distal</bumperTopicName>
+            <bumperTopicName>contacts/${prefix}th/distal</bumperTopicName>
           </plugin>
         </sensor>
@@ -92,17 +76,10 @@
       </joint>
       <!-- extra link to imaginary sphere in fingertip for FK/IK calculations -->
-      <!-- remove visual and collision once the correct position is found -->
       <link name="${prefix}thtip">
         <inertial>
           <mass value="0.001" />
           <origin xyz="0 0 0" rpy="0 0 0" />
-          <inertia ixx="0" ixy="0" ixz="0" iyy="0" iyz="0"
-          izz="0" />
+          <inertia ixx="0" ixy="0" ixz="0" iyy="0" iyz="0" izz="0" />
         </inertial>
-        <!--visual>
-          <geometry>
-            <sphere radius="0.002" />
-          </geometry>
-        </visual-->
       </link>
       <gazebo reference="${prefix}thtip">
@@ -112,10 +89,9 @@
         <parent link="${prefix}thdistal_J1_dummy" />
         <child link="${prefix}thtip" />
-        <origin xyz="0.0 0.004 ${0.032}"
-        rpy="0 0 0" />
+        <origin xyz="0.0 0.004 ${0.032}" rpy="0 0 0" />
         <!-- approximated only FIXME -->
       </joint>
     </xacro:if>
-    <xacro:unless value="${bio}">
+    <xacro:unless value="${tip_sensor == 'bt_2p'}">
       <!-- common -->
       <link name="${prefix}thdistal">
@@ -123,33 +99,21 @@
           <mass value="0.016" />
           <origin xyz="0 0 0.01375" rpy="0 0 0" />
-          <inertia ixx="0.0000021" ixy="0.0" ixz="0.0"
-          iyy="0.0000022" iyz="0.0" izz="0.000001" />
+          <inertia ixx="0.0000021" ixy="0.0" ixz="0.0" iyy="0.0000022" iyz="0.0" izz="0.000001" />
         </inertial>
         <visual>
           <origin xyz="0 0 0" rpy="0 0 0" />
           <geometry name="${prefix}thdistal_visual">
-            <xacro:if value="${eli}">
-              <!-- Ellispoid distal  -->
-              <mesh filename="package://sr_description/meshes/hand/ellipsoids/thdistal_ellipsoid_visual.dae"
-              scale="0.001 0.001 0.001" />
+            <xacro:if value="${tip_sensor == 'pst'}">
+              <mesh filename="package://sr_description/meshes/components/th_distal/pst/th_distal_pst.dae"
+                    scale="0.001 0.001 0.001" />
             </xacro:if>
-            <xacro:unless value="${eli}">
-              <xacro:if value="${ubi}">
-                <!-- Ubi distal -->
-                <mesh filename="package://sr_description/meshes/hand/TH1_z.dae"
-                      scale="0.001 0.001 0.001" />
-              </xacro:if>
-	      <xacro:unless value="${ubi}">
-		<xacro:if value="${bt_sp}">
-		  <!-- bt sp distal  -->
-		  <mesh filename="package://sr_description/meshes/hand/biotacs/sp.dae" />
-		</xacro:if>
-		<xacro:unless value="${bt_sp}">
-		  <!-- Standard distal  -->
-                  <mesh filename="package://sr_description/meshes/hand/TH1_z.dae"
-			scale="0.001 0.001 0.001" />
-		</xacro:unless>
-	      </xacro:unless>
-            </xacro:unless>
+            <xacro:if value="${tip_sensor == 'bt_sp'}">
+              <mesh filename="package://sr_description/meshes/components/th_distal/bt_sp/th_distal_bt_sp.dae"
+                    scale="0.001 0.001 0.001" />
+            </xacro:if>
+            <xacro:if value="${tip_sensor == 'bt_2p'}">
+              <mesh filename="package://sr_description/meshes/components/th_distal/bt_2p/th_distal_bt_2p.dae"
+                    scale="0.001 0.001 0.001" />
+            </xacro:if>
           </geometry>
           <material name="shadow_thmiddle_material">
@@ -160,28 +124,16 @@
           <origin xyz="0 0 0" rpy="0 0 0" />
           <geometry name="${prefix}thmiddle_collision_geom">
-            <xacro:if value="${eli}">
-              <!-- Ellispoid distal  -->
-              <mesh filename="package://sr_description/meshes/hand/ellipsoids/thdistal_ellipsoid.dae"
-              scale="0.001 0.001 0.001" />
+            <xacro:if value="${tip_sensor == 'pst'}">
+              <mesh filename="package://sr_description/meshes/components/th_distal/pst/th_distal_pst.dae"
+                    scale="0.001 0.001 0.001" />
             </xacro:if>
-            <xacro:unless value="${eli}">
-              <xacro:if value="${ubi}">
-                <!-- Ubi distal -->
-                <mesh filename="package://sr_description/meshes/hand/TH1_z.dae"
-                scale="0.001 0.001 0.001" />
-              </xacro:if>
-              <xacro:unless value="${ubi}">
-		<xacro:if value="${bt_sp}">
-		  <!-- bt sp distal  -->
-                  <mesh filename="package://sr_description/meshes/hand/biotacs/sp.dae" />
-		</xacro:if>
-		<xacro:unless value="${bt_sp}">
-                  <!-- Standard distal  -->
-                  <mesh filename="package://sr_description/meshes/hand/TH1_z.dae"
-			scale="0.001 0.001 0.001" />
-		</xacro:unless>
-              </xacro:unless>
-            </xacro:unless>
-            <!--      <box size="0.015 0.015 0.015" /> -->
+            <xacro:if value="${tip_sensor == 'bt_sp'}">
+              <mesh filename="package://sr_description/meshes/components/th_distal/bt_sp/th_distal_bt_sp.dae"
+                    scale="0.001 0.001 0.001" />
+            </xacro:if>
+            <xacro:if value="${tip_sensor == 'bt_2p'}">
+              <mesh filename="package://sr_description/meshes/components/th_distal/bt_2p/th_distal_bt_2p.dae"
+                    scale="0.001 0.001 0.001" />
+            </xacro:if>
           </geometry>
         </collision>
@@ -192,6 +144,5 @@
         <origin xyz="0 0 0.032" rpy="0 0 ${-pi/2}" />
         <axis xyz="1 0 0" />
-        <limit lower="-${15.0*pi/180}" upper="${90.0*pi/180}" effort="1.0"
-        velocity="4.0" />
+        <limit lower="-${15.0*pi/180}" upper="${90.0*pi/180}" effort="1.0" velocity="4.0" />
         <dynamics damping="0.2" />
       </joint>
@@ -203,6 +154,5 @@
         <inertial>
           <mass value="0.001" />
-          <inertia ixx="0.0" ixy="0.0" ixz="0.0" iyy="0.0"
-          iyz="0.0" izz="0.0" />
+          <inertia ixx="0.0" ixy="0.0" ixz="0.0" iyy="0.0" iyz="0.0" izz="0.0" />
         </inertial>
       </link>
@@ -212,9 +162,8 @@
         <origin xyz="0 0 0.0275" rpy="0 0 0" />
       </joint>
-      <xacro:thdistal_gazebo prefix="${prefix}" />
+      <xacro:thdistal_gazebo />
     </xacro:unless>
     <!-- extensions -->
-    <xacro:thdistal_transmission muscletrans="${muscle}"
-    prefix="${prefix}" />
+    <xacro:thdistal_transmission />
   </xacro:macro>
 </robot>

Commit message: Adding finger distal mst

File: sr_description/hand/xacro/finger/distal/distal.urdf.xacro (robot description, xacro)
@@ -54,4 +54,7 @@
             <mesh filename="package://sr_description/meshes/components/f_distal/bt_2p/f_distal_bt_2p.dae" />
           </xacro:if>
+          <xacro:if value="${tip_sensor == 'mst'}">
+            <mesh filename="package://sr_description/meshes/components/f_distal/mst/f_distal_mst.dae" />
+          </xacro:if>
         </geometry>
       </visual>
@@ -69,4 +72,7 @@
           <xacro:if value="${tip_sensor == 'bt_2p'}">
             <mesh filename="package://sr_description/meshes/components/f_distal/bt_2p/f_distal_bt_2p.dae" />
+          </xacro:if>
+          <xacro:if value="${tip_sensor == 'mst'}">
+            <mesh filename="package://sr_description/meshes/components/f_distal/mst/f_distal_mst.dae" />
           </xacro:if>
         </geometry>

File: sr_description/hand/xacro/process_sensor_parameters.xacro (robot description, xacro)
@@ -59,5 +59,5 @@
 	<xacro:macro name="transform_to_type" params="name value default_tactile_sensor:=^|none
 				valid_finger_tokens:=^|${'th ff mf rf lf'.split()}
-				valid_sensor_tokens:=^|${'bt_2p bt_sp pst none'.split()}">
+				valid_sensor_tokens:=^|${'bt_2p bt_sp pst mst none'.split()}">
 		<!-- None acts as marker indicating that we didn't find the correct type specifier yet -->
 		<!-- Finally, _tmp_ should become a list of (finger, sensor) pairs -->

Commit message: Fixing finger distal mst

File: sr_description/hand/xacro/finger/distal/distal.urdf.xacro (robot description, xacro)
@@ -55,5 +55,6 @@
           </xacro:if>
           <xacro:if value="${tip_sensor == 'mst'}">
-            <mesh filename="package://sr_description/meshes/components/f_distal/mst/f_distal_mst.dae" />
+            <mesh filename="package://sr_description/meshes/components/f_distal/mst/f_distal_mst.dae"
+                  scale="0.001 0.001 0.001" />
           </xacro:if>
         </geometry>
@@ -74,5 +75,6 @@
           </xacro:if>
           <xacro:if value="${tip_sensor == 'mst'}">
-            <mesh filename="package://sr_description/meshes/components/f_distal/mst/f_distal_mst.dae" />
+            <mesh filename="package://sr_description/meshes/components/f_distal/mst/f_distal_mst.dae"
+                  scale="0.001 0.001 0.001" />
           </xacro:if>
         </geometry>

Commit message: Changing path

File: sr_description/hand/xacro/finger/distal/distal.urdf.xacro (robot description, xacro)
@@ -55,5 +55,5 @@
           </xacro:if>
           <xacro:if value="${tip_sensor == 'mst'}">
-            <mesh filename="package://sr_description/meshes/components/f_distal/mst/f_distal_mst.dae"
+            <mesh filename="package://sr_mst_description/meshes/f_distal/f_distal_mst.dae"
                   scale="0.001 0.001 0.001" />
           </xacro:if>
@@ -75,5 +75,5 @@
           </xacro:if>
           <xacro:if value="${tip_sensor == 'mst'}">
-            <mesh filename="package://sr_description/meshes/components/f_distal/mst/f_distal_mst.dae"
+            <mesh filename="package://sr_mst_description/meshes/f_distal/f_distal_mst.dae"
                   scale="0.001 0.001 0.001" />
           </xacro:if>

File: sr_description/hand/xacro/thumb/thdistal.urdf.xacro (robot description, xacro)
@@ -133,5 +133,5 @@
             </xacro:if>
             <xacro:if value="${tip_sensor == 'mst'}">
-              <mesh filename="package://sr_description/meshes/components/th_distal/mst/th_distal_mst.dae"
+              <mesh filename="package://sr_mst_description/meshes/th_distal/th_distal_mst.dae"
                     scale="0.001 0.001 0.001" />
             </xacro:if>
@@ -157,5 +157,5 @@
             </xacro:if>
             <xacro:if value="${tip_sensor == 'mst'}">
-              <mesh filename="package://sr_description/meshes/components/th_distal/mst/th_distal_mst.dae"
+              <mesh filename="package://sr_mst_description/meshes/th_distal/th_distal_mst.dae"
                     scale="0.001 0.001 0.001" />
             </xacro:if>

Commit message: Adding meshes

File: sr_description/hand/xacro/finger/distal/distal.urdf.xacro (robot description, xacro)
@@ -55,5 +55,5 @@
           </xacro:if>
           <xacro:if value="${tip_sensor == 'mst'}">
-            <mesh filename="package://sr_mst_description/meshes/f_distal/f_distal_mst.dae"
+            <mesh filename="package://sr_mst/meshes/f_distal/f_distal_mst.dae"
                   scale="0.001 0.001 0.001" />
           </xacro:if>
@@ -75,5 +75,5 @@
           </xacro:if>
           <xacro:if value="${tip_sensor == 'mst'}">
-            <mesh filename="package://sr_mst_description/meshes/f_distal/f_distal_mst.dae"
+            <mesh filename="package://sr_mst/meshes/f_distal/f_distal_mst.dae"
                   scale="0.001 0.001 0.001" />
           </xacro:if>

File: sr_description/hand/xacro/thumb/thdistal.urdf.xacro (robot description, xacro)
@@ -133,5 +133,5 @@
             </xacro:if>
             <xacro:if value="${tip_sensor == 'mst'}">
-              <mesh filename="package://sr_mst_description/meshes/th_distal/th_distal_mst.dae"
+              <mesh filename="package://sr_mst/meshes/th_distal/th_distal_mst.dae"
                     scale="0.001 0.001 0.001" />
             </xacro:if>
@@ -157,5 +157,5 @@
             </xacro:if>
             <xacro:if value="${tip_sensor == 'mst'}">
-              <mesh filename="package://sr_mst_description/meshes/th_distal/th_distal_mst.dae"
+              <mesh filename="package://sr_mst/meshes/th_distal/th_distal_mst.dae"
                     scale="0.001 0.001 0.001" />
             </xacro:if>
