Commit message: wip

File: sr_description/hand/xacro/finger/distal/distal.urdf.xacro (robot description, xacro)
@@ -33,4 +33,5 @@
   <xacro:include filename="$(find sr_description)/hand/xacro/finger/distal/distal.gazebo.xacro" />
   <xacro:include filename="$(find sr_description)/hand/xacro/finger/distal/distal.transmission.xacro" />
+  <xacro:include filename="$(find sr_mst)/xacro/mstXL.urdf.xacro" />
   <xacro:macro name="distal" params="prefix:=^ link_prefix:=^ joint_prefix:=^ tip_sensor:=^|pst parent">
     <link name="${prefix}${link_prefix}distal">
@@ -40,44 +41,44 @@
         <inertia ixx="0.00000094" ixy="0.0" ixz="0.0" iyy="0.0000011" iyz="0.0" izz="0.00000053" />
       </inertial>
-      <visual>
-        <origin xyz="0 0 0" rpy="0 0 0" />
-        <geometry name="${prefix}${link_prefix}distal_visual">
-          <xacro:if value="${tip_sensor == 'pst'}">
-            <mesh filename="package://sr_description/meshes/components/f_distal/pst/f_distal_pst.dae"
-                  scale="0.001 0.001 0.001" />
-          </xacro:if>
-          <xacro:if value="${tip_sensor == 'bt_sp'}">
-            <mesh filename="package://sr_description/meshes/components/f_distal/bt_sp/f_distal_bt_sp.dae"
-                  scale="0.001 0.001 0.001" />
-          </xacro:if>
-          <xacro:if value="${tip_sensor == 'bt_2p'}">
-            <mesh filename="package://sr_description/meshes/components/f_distal/bt_2p/f_distal_bt_2p.dae" />
-          </xacro:if>
-          <xacro:if value="${tip_sensor == 'mst'}">
-            <mesh filename="package://sr_mst/meshes/f_distal/f_distal_mst.dae"
-                  scale="0.001 0.001 0.001" />
-          </xacro:if>
-        </geometry>
-      </visual>
-      <collision>
-        <origin xyz="0 0 0" rpy="0 0 0" />
-        <geometry name="${prefix}${link_prefix}distal_collision_geom">
-          <xacro:if value="${tip_sensor == 'pst'}">
-            <mesh filename="package://sr_description/meshes/components/f_distal/pst/f_distal_pst.dae"
-                  scale="0.001 0.001 0.001" />
-          </xacro:if>
-          <xacro:if value="${tip_sensor == 'bt_sp'}">
-            <mesh filename="package://sr_description/meshes/components/f_distal/bt_sp/f_distal_bt_sp.dae"
-                  scale="0.001 0.001 0.001" />
-          </xacro:if>
-          <xacro:if value="${tip_sensor == 'bt_2p'}">
-            <mesh filename="package://sr_description/meshes/components/f_distal/bt_2p/f_distal_bt_2p.dae" />
-          </xacro:if>
-          <xacro:if value="${tip_sensor == 'mst'}">
-            <mesh filename="package://sr_mst/meshes/f_distal/f_distal_mst.dae"
-                  scale="0.001 0.001 0.001" />
-          </xacro:if>
-        </geometry>
-      </collision>
+      <xacro:unless value="${tip_sensor == 'mst'}">
+        <visual>
+          <origin xyz="0 0 0" rpy="0 0 0" />
+          <geometry name="${prefix}${link_prefix}distal_visual">
+            <xacro:if value="${tip_sensor == 'pst'}">
+              <mesh filename="package://sr_description/meshes/components/f_distal/pst/f_distal_pst.dae"
+                    scale="0.001 0.001 0.001" />
+            </xacro:if>
+            <xacro:if value="${tip_sensor == 'bt_sp'}">
+              <mesh filename="package://sr_description/meshes/components/f_distal/bt_sp/f_distal_bt_sp.dae"
+                    scale="0.001 0.001 0.001" />
+            </xacro:if>
+            <xacro:if value="${tip_sensor == 'bt_2p'}">
+              <mesh filename="package://sr_description/meshes/components/f_distal/bt_2p/f_distal_bt_2p.dae" />
+            </xacro:if>
+            <!-- <xacro:if value="${tip_sensor == 'mst'}">
+              <mesh filename="package://sr_mst/meshes/mstXL/mstXL_skin.stl"/>
+            </xacro:if> -->
+          </geometry>
+        </visual>
+        <collision>
+          <origin xyz="0 0 0" rpy="0 0 0" />
+          <geometry name="${prefix}${link_prefix}distal_collision_geom">
+            <xacro:if value="${tip_sensor == 'pst'}">
+              <mesh filename="package://sr_description/meshes/components/f_distal/pst/f_distal_pst.dae"
+                    scale="0.001 0.001 0.001" />
+            </xacro:if>
+            <xacro:if value="${tip_sensor == 'bt_sp'}">
+              <mesh filename="package://sr_description/meshes/components/f_distal/bt_sp/f_distal_bt_sp.dae"
+                    scale="0.001 0.001 0.001" />
+            </xacro:if>
+            <xacro:if value="${tip_sensor == 'bt_2p'}">
+              <mesh filename="package://sr_description/meshes/components/f_distal/bt_2p/f_distal_bt_2p.dae" />
+            </xacro:if>
+            <xacro:if value="${tip_sensor == 'mst'}">
+              <mesh filename="package://sr_mst/meshes/mstXL/mstXL_skin.stl"/>
+            </xacro:if>
+          </geometry>
+        </collision>
+      </xacro:unless>
     </link>
     <xacro:unless value="${tip_sensor == 'bt_2p'}">
@@ -106,4 +107,7 @@
         <origin xyz="0 0 0.026" rpy="0 0 0" />
       </joint>
+      <xacro:if value="${tip_sensor == 'mst'}">
+        <xacro:mstXL prefix="${prefix}" link_prefix="${link_prefix}" parent="${prefix}${link_prefix}distal" scale="0.001"/>
+      </xacro:if>
     </xacro:unless>
     <!-- extensions -->

Commit message: Currently working with the wrong mesh and taxel tfs positions

File: sr_description/hand/xacro/finger/distal/distal.urdf.xacro (robot description, xacro)
@@ -41,5 +41,4 @@
         <inertia ixx="0.00000094" ixy="0.0" ixz="0.0" iyy="0.0000011" iyz="0.0" izz="0.00000053" />
       </inertial>
-      <xacro:unless value="${tip_sensor == 'mst'}">
         <visual>
           <origin xyz="0 0 0" rpy="0 0 0" />
@@ -56,7 +55,8 @@
               <mesh filename="package://sr_description/meshes/components/f_distal/bt_2p/f_distal_bt_2p.dae" />
             </xacro:if>
-            <!-- <xacro:if value="${tip_sensor == 'mst'}">
-              <mesh filename="package://sr_mst/meshes/mstXL/mstXL_skin.stl"/>
-            </xacro:if> -->
+            <xacro:if value="${tip_sensor == 'mst'}">
+              <mesh filename="package://sr_mst/meshes/f_distal/f_distal_mst.dae"
+                  scale="0.001 0.001 0.001" />
+            </xacro:if>
           </geometry>
         </visual>
@@ -76,9 +76,9 @@
             </xacro:if>
             <xacro:if value="${tip_sensor == 'mst'}">
-              <mesh filename="package://sr_mst/meshes/mstXL/mstXL_skin.stl"/>
+              <mesh filename="package://sr_mst/meshes/f_distal/f_distal_mst.dae"
+                  scale="0.001 0.001 0.001" />
             </xacro:if>
           </geometry>
         </collision>
-      </xacro:unless>
     </link>
     <xacro:unless value="${tip_sensor == 'bt_2p'}">

Commit message: Update MST meshes (and xacro) to MSTXL

File: sr_description/hand/xacro/finger/distal/distal.urdf.xacro (robot description, xacro)
@@ -33,5 +33,5 @@
   <xacro:include filename="$(find sr_description)/hand/xacro/finger/distal/distal.gazebo.xacro" />
   <xacro:include filename="$(find sr_description)/hand/xacro/finger/distal/distal.transmission.xacro" />
-  <xacro:include filename="$(find sr_mst)/xacro/f_distal.urdf.xacro" />
+  <xacro:include filename="$(find sr_mst)/xacro/f_distalXL.urdf.xacro" />
   <xacro:macro name="distal" params="prefix:=^ link_prefix:=^ joint_prefix:=^ tip_sensor:=^|pst parent">
     <link name="${prefix}${link_prefix}distal">
@@ -56,5 +56,5 @@
             </xacro:if>
             <xacro:if value="${tip_sensor == 'mst'}">
-              <mesh filename="package://sr_mst/meshes/f_distal/f_distal_mst.dae"
+              <mesh filename="package://sr_mst/meshes/f_distal_XL/f_distal_mstXL.dae"
                   scale="0.001 0.001 0.001" />
             </xacro:if>
@@ -76,5 +76,5 @@
             </xacro:if>
             <xacro:if value="${tip_sensor == 'mst'}">
-              <mesh filename="package://sr_mst/meshes/f_distal/f_distal_mst.dae"
+              <mesh filename="package://sr_mst/meshes/f_distal_XL/f_distal_mstXL.dae"
                   scale="0.001 0.001 0.001" />
             </xacro:if>
@@ -108,5 +108,5 @@
       </joint>
       <xacro:if value="${tip_sensor == 'mst'}">
-        <xacro:f_mst_distal prefix="${prefix}" link_prefix="${link_prefix}" parent="${prefix}${link_prefix}distal" scale="0.001" show_mesh="false"/>
+        <xacro:f_mstXL_distal prefix="${prefix}" link_prefix="${link_prefix}" parent="${prefix}${link_prefix}distal" scale="0.001" show_mesh="false"/>
       </xacro:if>
     </xacro:unless>
