Commit message: Fixed urdfs with biotacs and dummy palm

File: sr_description/hand/xacro/finger/biotac/biotac.urdf.xacro (robot description, xacro)
@@ -152,9 +152,9 @@
         izz="0.0" />
       </inertial>
-      <visual>
+      <!--visual>
         <geometry>
           <sphere radius="0.002" />
         </geometry>
-      </visual>
+      </visual-->
     </link>
     <gazebo reference="${prefix}${joint_prefix}tip">
@@ -163,7 +163,7 @@
     <joint name="${prefix}${joint_prefix}tip"
     type="fixed">
-      <parent link="${prefix}${link_prefix}middle" />
+      <parent link="${prefix}${link_prefix}_J1_dummy" />
       <child link="${prefix}${link_prefix}tip" />
-      <origin xyz="0.0 -0.009 ${0.008+0.044}" rpy="0 0 -1.571" />
+      <origin xyz="0.0 0.004 0.029" rpy="0 0 0" />
       <!-- approximated only FIXME -->
     </joint>

File: sr_description/hand/xacro/one_finger_unit.urdf.xacro (robot description, xacro)
@@ -19,5 +19,5 @@
     <xacro:forearm muscle="${muscle}" prefix="${prefix}" />
     <!-- Dummy Palm -->
-    <link name="${prefix}dummy_palm">
+    <link name="${prefix}palm">
       <inertial>
         <mass value="0.010" />
@@ -28,5 +28,5 @@
       <visual>
         <origin xyz="0 0 0.0505" rpy="0 0 0" />
-        <geometry name="${prefix}dummy_palm_visual">
+        <geometry name="${prefix}palm_visual">
           <box size="0.015 0.015 0.110" />
         </geometry>
@@ -35,5 +35,5 @@
       <collision>
         <origin xyz="0 0 0.0" rpy="0 0 0" />
-        <geometry name="${prefix}dummy_palm_collision_geom">
+        <geometry name="${prefix}palm_collision_geom">
           <box size="0.015 0.015 0.110" />
         </geometry>
@@ -42,5 +42,5 @@
     <joint name="${prefix}forearm_to_dummy" type="fixed">
       <parent link="${prefix}forearm" />
-      <child link="${prefix}dummy_palm" />
+      <child link="${prefix}palm" />
       <origin xyz="${reflect*0.011} 0.010 0.22"
       rpy="0 0 ${M_PI}" />
@@ -52,5 +52,5 @@
     bio="${bio}" bt_sp="${bt_sp}" ubi="${ubi}" eli="${eli}" prefix="${prefix}"
     reflect="${reflect}" link_prefix="mf" joint_prefix="MF"
-    parent="${prefix}dummy_palm">
+    parent="${prefix}palm">
       <origin xyz="0.0 0 0.116" rpy="0 0 0" />
       <axis xyz="0 ${-1*reflect} 0" />

File: sr_description/hand/xacro/thumb/thdistal.urdf.xacro (robot description, xacro)
@@ -100,9 +100,9 @@
           izz="0" />
         </inertial>
-        <visual>
+        <!--visual>
           <geometry>
             <sphere radius="0.002" />
           </geometry>
-        </visual>
+        </visual-->
       </link>
       <gazebo reference="${prefix}thtip">
@@ -110,8 +110,8 @@
       </gazebo>
       <joint name="${prefix}thtip" type="fixed">
-        <parent link="${prefix}thmiddle" />
+        <parent link="${prefix}thdistal_J1_dummy" />
         <child link="${prefix}thtip" />
-        <origin xyz="-0.009 0.0 ${0.01+0.044}"
-        rpy="0 0 ${-M_PI/2}" />
+        <origin xyz="0.0 0.004 ${0.032}"
+        rpy="0 0 0" />
         <!-- approximated only FIXME -->
       </joint>
