Commit message: Parameterising dexterous hand URDF xacros for simple or complex collision meshes.

File: sr_description/hand/xacro/finger/biotac/biotac.urdf.xacro (robot description, xacro)
@@ -13,5 +13,5 @@
   <!-- parent is the parent link for the joint -->
   <xacro:macro name="biotac_middle"
-  params="muscle prefix link_prefix joint_prefix parent">
+  params="muscle prefix link_prefix joint_prefix parent simple_collisions">
     <link name="${prefix}${link_prefix}middle">
       <inertial>
@@ -29,10 +29,21 @@
         <material name="LightGrey" />
       </visual>
-      <collision>
-        <origin xyz="0 0 0.005" rpy="0 0 0" />
+      <xacro:if value="${simple_collisions}">
+        <collision>
+          <origin xyz="0 0 0.005" rpy="0 0 0" />
+          <geometry name="${prefix}${link_prefix}middle_collision_geom">
+            <box size="0.001 0.001 0.001" />
+          </geometry>
+        </collision>
+      </xacro:if>
+      <xacro:unless value="${simple_collisions}">
+        <collision>
+        <origin xyz="0 0 0" rpy="0 0 1.571" />
         <geometry name="${prefix}${link_prefix}middle_collision_geom">
-          <box size="0.001 0.001 0.001" />
+          <mesh filename="package://sr_description/hand/model/biotacs/biotac_finger_adapter.dae"
+          scale="1 1 1" />
         </geometry>
-      </collision>
+        </collision>
+      </xacro:unless>
     </link>
     <gazebo reference="${prefix}${link_prefix}middle">

File: sr_description/hand/xacro/finger/fingers.urdf.xacro (robot description, xacro)
@@ -18,13 +18,13 @@
   <!-- parent is the parent link for the first joint -->
   <xacro:macro name="finger"
-  params="muscletrans lf bio bt_sp ubi eli reflect prefix link_prefix joint_prefix parent *origin *axis">
+  params="muscletrans lf bio bt_sp ubi eli reflect prefix link_prefix joint_prefix parent *origin *axis simple_collisions" >
     <!-- Little finger special case -->
     <xacro:if value="${lf}">
       <xacro:lfmetacarpal muscle="${muscletrans}"
-      prefix="${prefix}" reflect="${reflect}" parent="${parent}" />
+      prefix="${prefix}" reflect="${reflect}" parent="${parent}" simple_collisions="${simple_collisions}"/>
       <!-- Knuckle -->
       <xacro:knuckle muscle="${muscletrans}" prefix="${prefix}"
       link_prefix="${link_prefix}" joint_prefix="${joint_prefix}"
-      parent="${prefix}lfmetacarpal">
+      parent="${prefix}lfmetacarpal" simple_collisions="${simple_collisions}">
         <xacro:insert_block name="origin" />
       </xacro:knuckle>
@@ -35,5 +35,5 @@
       <xacro:knuckle muscle="${muscletrans}" prefix="${prefix}"
       link_prefix="${link_prefix}" joint_prefix="${joint_prefix}"
-      parent="${parent}">
+      parent="${parent}" simple_collisions="${simple_collisions}">
         <xacro:insert_block name="origin" />
       </xacro:knuckle>
@@ -42,5 +42,5 @@
     <xacro:proximal muscle="${muscletrans}" prefix="${prefix}"
     link_prefix="${link_prefix}" joint_prefix="${joint_prefix}"
-    parent="${prefix}${link_prefix}knuckle"></xacro:proximal>
+    parent="${prefix}${link_prefix}knuckle" simple_collisions="${simple_collisions}"></xacro:proximal>
     <!-- Biotac Middle -->
     <xacro:if value="${bio}">
@@ -48,5 +48,5 @@
       prefix="${prefix}" link_prefix="${link_prefix}"
       joint_prefix="${joint_prefix}"
-      parent="${prefix}${link_prefix}proximal">
+      parent="${prefix}${link_prefix}proximal" simple_collisions="${simple_collisions}">
       </xacro:biotac_middle>
     </xacro:if>
@@ -55,5 +55,5 @@
       <xacro:middle muscle="${muscletrans}" prefix="${prefix}"
       link_prefix="${link_prefix}" joint_prefix="${joint_prefix}"
-      parent="${prefix}${link_prefix}proximal"></xacro:middle>
+      parent="${prefix}${link_prefix}proximal" simple_collisions="${simple_collisions}"></xacro:middle>
     </xacro:unless>
     <!-- Distal  -->

File: sr_description/hand/xacro/finger/knuckle/knuckle.urdf.xacro (robot description, xacro)
@@ -14,5 +14,5 @@
   <!-- parent is the parent link for the joint -->
   <xacro:macro name="knuckle"
-  params="muscle prefix link_prefix joint_prefix parent *origin">
+  params="muscle prefix link_prefix joint_prefix parent *origin simple_collisions">
     <link name="${prefix}${link_prefix}knuckle">
       <inertial>
@@ -30,4 +30,5 @@
         <material name="LightGrey" />
       </visual>
+      <xacro:if value="${simple_collisions}">
       <collision>
         <origin xyz="0 0 0" rpy="0 1.5708 0" />
@@ -36,4 +37,14 @@
         </geometry>
       </collision>
+      </xacro:if>
+      <xacro:unless value="${simple_collisions}">
+        <collision>
+        <origin xyz="0 0 0.0005" rpy="0 0 0" />
+        <geometry name="${prefix}${link_prefix}knuckle_collision_geom">
+          <mesh filename="package://sr_description/hand/model/knuckle.dae"
+          scale="0.001 0.001 0.001" />
+        </geometry>
+        </collision>
+      </xacro:unless>
     </link>
     <joint name="${prefix}${joint_prefix}J4" type="revolute">

File: sr_description/hand/xacro/finger/lfmetacarpal/lfmetacarpal.urdf.xacro (robot description, xacro)
@@ -13,5 +13,5 @@
   <!-- parent is the parent link for the joint -->
   <xacro:macro name="lfmetacarpal"
-  params="muscle prefix reflect parent">
+  params="muscle prefix reflect parent simple_collisions">
     <link name="${prefix}lfmetacarpal">
       <inertial>
@@ -29,4 +29,5 @@
         <material name="Grey" />
       </visual>
+      <xacro:if value="${simple_collisions}">
       <collision>
         <origin xyz="0 0 0.038" rpy="0 0 0" />
@@ -35,4 +36,14 @@
         </geometry>
       </collision>
+      </xacro:if>
+      <xacro:unless value="${simple_collisions}">
+        <collision>
+          <origin xyz="0 0 0" rpy="0 0 0" />
+          <geometry name="${prefix}lfmetacarpal_collision_geom">
+            <mesh filename="package://sr_description/hand/model/lfmetacarpal.dae"
+            scale="${reflect*0.001} 0.001 0.001" />
+          </geometry>
+        </collision>
+      </xacro:unless>
     </link>
     <joint name="${prefix}LFJ5" type="revolute">

File: sr_description/hand/xacro/finger/middle/middle.urdf.xacro (robot description, xacro)
@@ -14,5 +14,5 @@
   <!-- parent is the parent link for the joint -->
   <xacro:macro name="middle"
-  params="muscle prefix link_prefix joint_prefix parent">
+  params="muscle prefix link_prefix joint_prefix parent simple_collisions">
     <link name="${prefix}${link_prefix}middle">
       <inertial>
@@ -30,22 +30,33 @@
         <material name="Grey" />
       </visual>
-      <collision>
-        <origin xyz="0 0 0.0125" rpy="0 0 0" />
+      <xacro:if value="${simple_collisions}">
+        <collision>
+          <origin xyz="0 0 0.0125" rpy="0 0 0" />
+          <geometry name="${prefix}${link_prefix}middle_collision_geom">
+            <cylinder radius="0.007" length="0.025" />
+          </geometry>
+        </collision>
+        <collision>
+          <origin xyz="0 0 0.0" rpy="0 0 0" />
+          <geometry>
+            <sphere radius="0.007" />
+          </geometry>
+        </collision>
+        <collision>
+          <origin xyz="0 0 0.025" rpy="0 0 0" />
+          <geometry>
+            <sphere radius="0.007" />
+          </geometry>
+        </collision>
+      </xacro:if>
+      <xacro:unless value="${simple_collisions}">
+        <collision>
+        <origin xyz="0 0 0" rpy="0 0 0" />
         <geometry name="${prefix}${link_prefix}middle_collision_geom">
-          <cylinder radius="0.007" length="0.025" />
+          <mesh filename="package://sr_description/hand/model/F2.dae"
+          scale="0.001 0.001 0.001" />
         </geometry>
-      </collision>
-      <collision>
-        <origin xyz="0 0 0.0" rpy="0 0 0" />
-        <geometry>
-          <sphere radius="0.007" />
-        </geometry>
-      </collision>
-      <collision>
-        <origin xyz="0 0 0.025" rpy="0 0 0" />
-        <geometry>
-          <sphere radius="0.007" />
-        </geometry>
-      </collision>
+        </collision>
+      </xacro:unless>
     </link>
     <joint name="${prefix}${joint_prefix}J2" type="revolute">

File: sr_description/hand/xacro/finger/proximal/proximal.urdf.xacro (robot description, xacro)
@@ -14,5 +14,5 @@
   <!-- parent is the parent link for the joint -->
   <xacro:macro name="proximal"
-  params="muscle prefix link_prefix joint_prefix parent">
+  params="muscle prefix link_prefix joint_prefix parent simple_collisions">
     <link name="${prefix}${link_prefix}proximal">
       <inertial>
@@ -30,10 +30,21 @@
         <material name="Grey" />
       </visual>
-      <collision>
-        <origin xyz="0 0 0.025" rpy="0 0 0" />
+      <xacro:if value="${simple_collisions}">
+        <collision>
+          <origin xyz="0 0 0.025" rpy="0 0 0" />
+          <geometry name="${prefix}${link_prefix}proximal_collision_geom">
+            <cylinder radius="0.007" length="0.040" />
+          </geometry>
+        </collision>
+      </xacro:if>
+      <xacro:unless value="${simple_collisions}">
+        <collision>
+        <origin xyz="0 0 0" rpy="0 0 0" />
         <geometry name="${prefix}${link_prefix}proximal_collision_geom">
-          <cylinder radius="0.007" length="0.040" />
+          <mesh filename="package://sr_description/hand/model/F3.dae"
+          scale="0.001 0.001 0.001" />
         </geometry>
-      </collision>
+        </collision>
+      </xacro:unless>
     </link>
     <joint name="${prefix}${joint_prefix}J3" type="revolute">

File: sr_description/hand/xacro/forearm/forearm.urdf.xacro (robot description, xacro)
@@ -2,5 +2,5 @@
   <!-- muscle is true for muscle hand or false for motor hand -->
   <!-- prefix can be anything but usually is "r_" or  "l_" for right and left hands distinction -->
-  <xacro:macro name="forearm" params="muscle prefix">
+  <xacro:macro name="forearm" params="muscle prefix simple_collisions">
     <link name="${prefix}forearm">
       <inertial>
@@ -24,33 +24,50 @@
         <material name="Grey" />
       </visual>
-      <collision>
-        <xacro:if value="${muscle}">
-          <origin xyz="0 0 0.185" rpy="0 0 0" />
+      <xacro:if value="${simple_collisions}">
+        <collision>
+          <xacro:if value="${muscle}">
+            <origin xyz="0 0 0.185" rpy="0 0 0" />
+            <geometry name="${prefix}forearm_collision">
+              <cylinder radius="0.075" length="0.37" />
+            </geometry>
+          </xacro:if>
+          <xacro:unless value="${muscle}">
+            <origin xyz="0 0 0.092" rpy="0 0 0" />
+            <geometry name="${prefix}forearm_collision">
+              <cylinder radius="0.07" length="0.184"/>
+            </geometry>
+          </xacro:unless>
+        </collision>
+        <!-- wrist mount -->
+        <collision>
+          <xacro:if value="${muscle}">
+            <origin xyz="0 0 0.395" rpy="0 0 0" />
+            <geometry>
+              <box size="0.03 0.04 0.06" />
+            </geometry>
+          </xacro:if>
+          <xacro:unless value="${muscle}">
+            <origin xyz="0 -0.01 0.181" rpy="0 0.78 0" />
+            <geometry>
+              <box size="0.07 0.07 0.07" />
+            </geometry>
+          </xacro:unless>
+        </collision>
+      </xacro:if>
+      <xacro:unless value="${simple_collisions}">
+        <collision>
+          <origin xyz="0 0 0" rpy="0 0 0" />
           <geometry name="${prefix}forearm_collision">
-            <cylinder radius="0.075" length="0.37" />
+            <xacro:if value="${muscle}">
+              <mesh filename="package://sr_description/hand/model/forearm_muscle.dae"
+              scale="1.0 1.0 1.0" />
+            </xacro:if>
+            <xacro:unless value="${muscle}">
+              <mesh filename="package://sr_description/hand/model/forearm.dae"
+              scale="0.001 0.001 0.001" />
+            </xacro:unless>
           </geometry>
-        </xacro:if>
-        <xacro:unless value="${muscle}">
-          <origin xyz="0 0 0.092" rpy="0 0 0" />
-          <geometry name="${prefix}forearm_collision">
-            <cylinder radius="0.07" length="0.184"/>
-          </geometry>
-        </xacro:unless>
-      </collision>
-      <!-- wrist mount -->
-      <collision>
-        <xacro:if value="${muscle}">
-          <origin xyz="0 0 0.395" rpy="0 0 0" />
-          <geometry>
-            <box size="0.03 0.04 0.06" />
-          </geometry>
-        </xacro:if>
-        <xacro:unless value="${muscle}">
-          <origin xyz="0 -0.01 0.181" rpy="0 0.78 0" />
-          <geometry>
-            <box size="0.07 0.07 0.07" />
-          </geometry>
-        </xacro:unless>
-      </collision>
+        </collision>
+      </xacro:unless>
     </link>
     <gazebo reference="${prefix}forearm">

File: sr_description/hand/xacro/full_hand.urdf.xacro (robot description, xacro)
@@ -19,11 +19,11 @@
   <!-- lf is true if we want a little finger, false otherwise -->
   <xacro:macro name="shadowhand"
-  params="muscletrans muscle bio bt_sp ubi eli reflect prefix lf">
+  params="muscletrans muscle bio bt_sp ubi eli reflect prefix lf simple_collisions">
     <!-- Forearm -->
-    <xacro:forearm muscle="${muscle}" prefix="${prefix}" />
+    <xacro:forearm muscle="${muscle}" prefix="${prefix}" simple_collisions="${simple_collisions}"/>
     <!-- Wrist -->
     <xacro:if value="${muscle}">
       <xacro:wrist muscletrans="${muscletrans}" prefix="${prefix}"
-      reflect="${reflect}" parent="${prefix}forearm">
+      reflect="${reflect}" parent="${prefix}forearm" simple_collisions="${simple_collisions}">
         <origin xyz="0 0 0.4096" rpy="0 0 0" />
       </xacro:wrist>
@@ -31,5 +31,5 @@
     <xacro:unless value="${muscle}">
       <xacro:wrist muscletrans="false" prefix="${prefix}"
-      reflect="${reflect}" parent="${prefix}forearm">
+      reflect="${reflect}" parent="${prefix}forearm" simple_collisions="${simple_collisions}">
         <origin xyz="0 -0.010 0.213" rpy="0 0 0" />
       </xacro:wrist>
@@ -37,10 +37,10 @@
     <!-- Palm -->
     <xacro:palm muscletrans="${muscletrans}" prefix="${prefix}"
-    reflect="${reflect}" parent="${prefix}wrist" />
+    reflect="${reflect}" parent="${prefix}wrist"  simple_collisions="${simple_collisions}"/>
     <!-- First Finger -->
     <xacro:finger muscletrans="${muscletrans}" lf="false"
     bio="${bio}" bt_sp="${bt_sp}" ubi="${ubi}" eli="${eli}" prefix="${prefix}"
     reflect="${reflect}" link_prefix="ff" joint_prefix="FF"
-    parent="${prefix}palm">
+    parent="${prefix}palm" simple_collisions="${simple_collisions}">
       <origin xyz="${reflect*0.033} 0 0.095" rpy="0 0 0" />
       <axis xyz="0 ${-1*reflect} 0" />
@@ -50,5 +50,5 @@
     bio="${bio}" bt_sp="${bt_sp}" ubi="${ubi}" eli="${eli}" prefix="${prefix}"
     reflect="${reflect}" link_prefix="mf" joint_prefix="MF"
-    parent="${prefix}palm">
+    parent="${prefix}palm" simple_collisions="${simple_collisions}">
       <origin xyz="${reflect*0.011} 0 0.099" rpy="0 0 0" />
       <axis xyz="0 ${-1*reflect} 0" />
@@ -58,5 +58,5 @@
     bio="${bio}" bt_sp="${bt_sp}" ubi="${ubi}" eli="${eli}" prefix="${prefix}"
     reflect="${reflect}" link_prefix="rf" joint_prefix="RF"
-    parent="${prefix}palm">
+    parent="${prefix}palm" simple_collisions="${simple_collisions}">
       <origin xyz="${reflect*-0.011} 0 0.095" rpy="0 0 0" />
       <axis xyz="0 ${reflect} 0" />
@@ -67,5 +67,5 @@
       bio="${bio}" bt_sp="${bt_sp}" ubi="${ubi}" eli="${eli}" prefix="${prefix}"
       reflect="${reflect}" link_prefix="lf" joint_prefix="LF"
-      parent="${prefix}palm">
+      parent="${prefix}palm" simple_collisions="${simple_collisions}">
         <origin xyz="0 0 0.06579" rpy="0 0 0" />
         <axis xyz="0 ${reflect} 0" />
@@ -75,5 +75,5 @@
     <xacro:thumb muscletrans="${muscletrans}" bio="${bio}" bt_sp="${bt_sp}"
     ubi="${ubi}" eli="${eli}" prefix="${prefix}"
-    reflect="${reflect}" is_lite="0" parent="${prefix}palm">
+    reflect="${reflect}" is_lite="0" parent="${prefix}palm" simple_collisions="${simple_collisions}">
     </xacro:thumb>
   </xacro:macro>

File: sr_description/hand/xacro/palm/palm.urdf.xacro (robot description, xacro)
@@ -14,5 +14,5 @@
   <!-- parent is the parent link for the joint -->
   <xacro:macro name="palm"
-  params="muscletrans prefix reflect parent">
+  params="muscletrans prefix reflect parent simple_collisions">
     <link name="${prefix}palm">
       <inertial>
@@ -30,61 +30,72 @@
         <material name="Grey" />
       </visual>
-      <collision>
-        <origin xyz="${reflect*0.011} 0.0085 0.038" rpy="0 0 0" />
-        <geometry name="${prefix}palm_collision_geom">
-          <box size="0.062 0.007 0.098" />
-        </geometry>
-      </collision>
-      <collision>
-        <origin xyz="${-reflect*0.002} -0.0035 0.038"
-        rpy="0 0 0" />
-        <geometry>
-          <box size="0.036 0.017 0.098" />
-        </geometry>
-      </collision>
-      <!-- palm complement below first finger -->
-      <collision>
-        <origin xyz="${reflect*0.029} -0.0035 0.082"
-        rpy="0 0 0" />
-        <geometry>
-          <box size="0.026 0.017 0.010" />
-        </geometry>
-      </collision>
-      <collision>
-        <origin xyz="${reflect*0.0265} -0.001 0.070"
-        rpy="0.2 0 ${reflect*0.25}" />
-        <geometry>
-          <box size="0.026 0.014 0.018" />
-        </geometry>
-      </collision>
-      <!-- thumb pulp side -->
-      <collision>
-        <origin xyz="${reflect*0.0315} -0.0085 0.001"
-        rpy="0 0 0" />
-        <geometry>
-          <box size="0.021 0.027 0.024" />
-        </geometry>
-      </collision>
-      <!-- thumb pulp central -->
-      <collision>
-        <origin xyz="${reflect*0.0125} -0.015 0.009" rpy="0 0 ${reflect*-0.48}" />
-        <geometry>
-          <box size="0.022 0.005 0.040" />
-        </geometry>
-      </collision>
-      <!-- above middle finger-->
-      <collision>
-        <origin xyz="${reflect*0.011} 0 0.089" rpy="0 0 0" />
-        <geometry>
-          <box size="0.018 0.024 0.004" />
-        </geometry>
-      </collision>
-      <!-- metacarpal side-->
-      <collision>
-        <origin xyz="${reflect*-0.030} 0 0.009" rpy="0 0 0" />
-        <geometry>
-          <box size="0.020 0.024 0.040" />
-        </geometry>
-      </collision>
+      <xacro:if value="${simple_collisions}">
+        <collision>
+          <origin xyz="${reflect*0.011} 0.0085 0.038" rpy="0 0 0" />
+          <geometry name="${prefix}palm_collision_geom">
+            <box size="0.062 0.007 0.098" />
+          </geometry>
+        </collision>
+        <collision>
+          <origin xyz="${-reflect*0.002} -0.0035 0.038"
+          rpy="0 0 0" />
+          <geometry>
+            <box size="0.036 0.017 0.098" />
+          </geometry>
+        </collision>
+        <!-- palm complement below first finger -->
+        <collision>
+          <origin xyz="${reflect*0.029} -0.0035 0.082"
+          rpy="0 0 0" />
+          <geometry>
+            <box size="0.026 0.017 0.010" />
+          </geometry>
+        </collision>
+        <collision>
+          <origin xyz="${reflect*0.0265} -0.001 0.070"
+          rpy="0.2 0 ${reflect*0.25}" />
+          <geometry>
+            <box size="0.026 0.014 0.018" />
+          </geometry>
+        </collision>
+        <!-- thumb pulp side -->
+        <collision>
+          <origin xyz="${reflect*0.0315} -0.0085 0.001"
+          rpy="0 0 0" />
+          <geometry>
+            <box size="0.021 0.027 0.024" />
+          </geometry>
+        </collision>
+        <!-- thumb pulp central -->
+        <collision>
+          <origin xyz="${reflect*0.0125} -0.015 0.009" rpy="0 0 ${reflect*-0.48}" />
+          <geometry>
+            <box size="0.022 0.005 0.040" />
+          </geometry>
+        </collision>
+        <!-- above middle finger-->
+        <collision>
+          <origin xyz="${reflect*0.011} 0 0.089" rpy="0 0 0" />
+          <geometry>
+            <box size="0.018 0.024 0.004" />
+          </geometry>
+        </collision>
+        <!-- metacarpal side-->
+        <collision>
+          <origin xyz="${reflect*-0.030} 0 0.009" rpy="0 0 0" />
+          <geometry>
+            <box size="0.020 0.024 0.040" />
+          </geometry>
+        </collision>
+      </xacro:if>
+      <xacro:unless value="${simple_collisions}">
+        <collision>
+          <origin xyz="0 0 0" rpy="0 0 0" />
+          <geometry name="${prefix}palm_collision_geom">
+            <mesh filename="package://sr_description/hand/model/palm.dae"
+            scale="${reflect*0.001} 0.001 0.001" />
+          </geometry>
+        </collision>
+      </xacro:unless>
     </link>
     <joint name="${prefix}ee_fixed_joint" type="fixed">

File: sr_description/hand/xacro/thumb/thbase.urdf.xacro (robot description, xacro)
@@ -12,5 +12,5 @@
   <!-- prefix can be anything but usually is "r_" or  "l_" for right and left hands distinction -->
   <!-- parent is the parent link for the first joint -->
-  <xacro:macro name="thbase" params="muscle reflect prefix parent">
+  <xacro:macro name="thbase" params="muscle reflect prefix parent simple_collisions">
     <link name="${prefix}thbase">
       <inertial>
@@ -29,10 +29,20 @@
         </material>
       </visual>
-      <collision>
-        <origin xyz="0 0 0" rpy="0 0 0" />
-        <geometry name="${prefix}thbase_collision_geom">
-          <sphere radius="0.011" />
-        </geometry>
-      </collision>
+      <xacro:if value="${simple_collisions}">
+        <collision>
+          <origin xyz="0 0 0" rpy="0 0 0" />
+          <geometry name="${prefix}thbase_collision_geom">
+            <sphere radius="0.011" />
+          </geometry>
+        </collision>
+      </xacro:if>
+      <xacro:unless value="${simple_collisions}">
+        <collision>
+          <origin xyz="0 0 0" rpy="0 0 0" />
+          <geometry name="${prefix}thbase_collision_geom">
+            <box size="0.001 0.001 0.001" />
+          </geometry>
+        </collision>
+      </xacro:unless>
     </link>
     <joint name="${prefix}THJ5" type="revolute">
