Commit message: Reverting xacro simple coliisions changes. Now stored on F_visual_hand_meshes_as_collision.

File: sr_description/hand/xacro/thumb/thbase.urdf.xacro (robot description, xacro)
@@ -12,5 +12,5 @@
   <!-- prefix can be anything but usually is "r_" or  "l_" for right and left hands distinction -->
   <!-- parent is the parent link for the first joint -->
-  <xacro:macro name="thbase" params="muscle reflect prefix parent simple_collisions">
+  <xacro:macro name="thbase" params="muscle reflect prefix parent">
     <link name="${prefix}thbase">
       <inertial>
@@ -29,20 +29,10 @@
         </material>
       </visual>
-      <xacro:if value="${simple_collisions}">
-        <collision>
-          <origin xyz="0 0 0" rpy="0 0 0" />
-          <geometry name="${prefix}thbase_collision_geom">
-            <sphere radius="0.011" />
-          </geometry>
-        </collision>
-      </xacro:if>
-      <xacro:unless value="${simple_collisions}">
-        <collision>
-          <origin xyz="0 0 0" rpy="0 0 0" />
-          <geometry name="${prefix}thbase_collision_geom">
-            <box size="0.001 0.001 0.001" />
-          </geometry>
-        </collision>
-      </xacro:unless>
+      <collision>
+        <origin xyz="0 0 0" rpy="0 0 0" />
+        <geometry name="${prefix}thbase_collision_geom">
+          <sphere radius="0.011" />
+        </geometry>
+      </collision>
     </link>
     <joint name="${prefix}THJ5" type="revolute">

File: sr_description/hand/xacro/thumb/thhub.urdf.xacro (robot description, xacro)
@@ -13,5 +13,5 @@
   <!-- parent is the parent link for the first joint -->
   <!-- is_lite is this the lite hand, if so lock J3 -->
-  <xacro:macro name="thhub" params="muscle prefix parent is_lite simple_collisions">
+  <xacro:macro name="thhub" params="muscle prefix parent is_lite">
     <link name="${prefix}thhub">
       <inertial>
@@ -30,20 +30,10 @@
         </material>
       </visual>
-      <xacro:if value="${simple_collisions}">
-        <collision>
-          <origin xyz="0 0 0" rpy="0 0 0" />
-          <geometry name="${prefix}thhub_collision_geom">
-            <sphere radius="0.010" />
-          </geometry>
-        </collision>
-      </xacro:if>
-      <xacro:unless value="${simple_collisions}">
-        <collision>
-          <origin xyz="0 0 0" rpy="0 0 0" />
-          <geometry name="${prefix}thhub_collision_geom">
-            <box size="0.001 0.001 0.001" />
-          </geometry>
-        </collision>
-      </xacro:unless>
+      <collision>
+        <origin xyz="0 0 0" rpy="0 0 0" />
+        <geometry name="${prefix}thhub_collision_geom">
+          <sphere radius="0.010" />
+        </geometry>
+      </collision>
     </link>
     <xacro:if value="${is_lite}">

File: sr_description/hand/xacro/thumb/thmiddle.urdf.xacro (robot description, xacro)
@@ -12,5 +12,5 @@
   <!-- prefix can be anything but usually is "r_" or  "l_" for right and left hands distinction -->
   <!-- parent is the parent link for the first joint -->
-  <xacro:macro name="thmiddle" params="muscle bio prefix parent simple_collisions">
+  <xacro:macro name="thmiddle" params="muscle bio prefix parent">
     <link name="${prefix}thmiddle">
       <inertial>
@@ -38,43 +38,24 @@
         </xacro:unless>
       </visual>
-      <xacro:if value="${simple_collisions}">
+      <collision>
+        <xacro:if value="${bio}">
+          <origin xyz="0 0 0.005" rpy="0 0 0" />
+          <geometry name="${prefix}thmiddle_collision_geom">
+            <box size="0.001 0.001 0.001" />
+          </geometry>
+        </xacro:if>
+        <xacro:unless value="${bio}">
+          <origin xyz="0 0 0.012" rpy="0 0 0" />
+          <geometry name="${prefix}thmiddle_collision_geom">
+            <cylinder radius="0.011" length="0.018" />
+          </geometry>
+        </xacro:unless>
+      </collision>
+      <xacro:unless value="${bio}">
         <collision>
-          <xacro:if value="${bio}">
-            <origin xyz="0 0 0.005" rpy="0 0 0" />
-            <geometry name="${prefix}thmiddle_collision_geom">
-              <box size="0.001 0.001 0.001" />
-            </geometry>
-          </xacro:if>
-          <xacro:unless value="${bio}">
-            <origin xyz="0 0 0.012" rpy="0 0 0" />
-            <geometry name="${prefix}thmiddle_collision_geom">
-              <cylinder radius="0.011" length="0.018" />
-            </geometry>
-          </xacro:unless>
-        </collision>
-        <xacro:unless value="${bio}">
-          <collision>
-            <origin xyz="0 0 0.019" rpy="0 0 0" />
-            <geometry>
-              <sphere radius="0.011" />
-            </geometry>
-          </collision>
-        </xacro:unless>
-      </xacro:if>
-      <xacro:unless value="${simple_collisions}">
-        <collision>
-          <origin xyz="0 0 0" rpy="0 0 0" />
-          <xacro:if value="${bio}">
-            <geometry name="${prefix}thmiddle_collision_geom">
-              <mesh filename="package://sr_description/hand/model/biotacs/biotac_thumb_adapter.dae"
-              scale="0.001 0.001 0.001" />
-            </geometry>
-          </xacro:if>
-          <xacro:unless value="${bio}">
-            <geometry name="${prefix}thmiddle_collision_geom">
-              <mesh filename="package://sr_description/hand/model/TH2_z.dae"
-              scale="0.001 0.001 0.001" />
-            </geometry>
-          </xacro:unless>
+          <origin xyz="0 0 0.019" rpy="0 0 0" />
+          <geometry>
+            <sphere radius="0.011" />
+          </geometry>
         </collision>
       </xacro:unless>

File: sr_description/hand/xacro/thumb/thproximal.urdf.xacro (robot description, xacro)
@@ -13,5 +13,5 @@
   <!-- parent is the parent link for the first joint -->
   <xacro:macro name="thproximal"
-  params="muscle reflect prefix parent simple_collisions">
+  params="muscle reflect prefix parent">
     <link name="${prefix}thproximal">
       <inertial>
@@ -31,21 +31,10 @@
         </material>
       </visual>
-      <xacro:if value="${simple_collisions}">
-        <collision>
-          <origin xyz="0 0 0.020" rpy="0 0 0" />
-          <geometry name="${prefix}thproximal_collision_geom">
-            <cylinder radius="0.012" length="0.018" />
-          </geometry>
-        </collision>
-      </xacro:if>
-      <xacro:unless value="${simple_collisions}">
-        <collision>
-          <origin xyz="0 0 0" rpy="0 0 0" />
-          <geometry name="${prefix}thproximal_collision_geom">
-            <mesh filename="package://sr_description/hand/model/TH3_z.dae"
-            scale="0.001 0.001 0.001" />
-          </geometry>
-        </collision>
-      </xacro:unless>
+      <collision>
+        <origin xyz="0 0 0.020" rpy="0 0 0" />
+        <geometry name="${prefix}thproximal_collision_geom">
+          <cylinder radius="0.012" length="0.018" />
+        </geometry>
+      </collision>
     </link>
     <joint name="${prefix}THJ4" type="revolute">

File: sr_description/hand/xacro/thumb/thumb.urdf.xacro (robot description, xacro)
@@ -15,19 +15,19 @@
   <!-- is_lite is this the lite hand, if so lock J3 -->
   <xacro:macro name="thumb"
-  params="muscletrans bio bt_sp ubi eli reflect prefix parent is_lite simple_collisions">
+  params="muscletrans bio bt_sp ubi eli reflect prefix parent is_lite">
     <!-- Base -->
     <xacro:thbase muscle="${muscletrans}" prefix="${prefix}"
-    reflect="${reflect}" parent="${parent}" simple_collisions="${simple_collisions}"></xacro:thbase>
+    reflect="${reflect}" parent="${parent}"></xacro:thbase>
     <!-- Proximal -->
     <xacro:thproximal muscle="${muscletrans}" prefix="${prefix}"
-    reflect="${reflect}" parent="${prefix}thbase" simple_collisions="${simple_collisions}">
+    reflect="${reflect}" parent="${prefix}thbase">
     </xacro:thproximal>
     <!-- Hub -->
     <xacro:thhub muscle="${muscletrans}" prefix="${prefix}"
-    parent="${prefix}thproximal" is_lite="${is_lite}" simple_collisions="${simple_collisions}">
+    parent="${prefix}thproximal" is_lite="${is_lite}">
     &gt;</xacro:thhub>
     <!-- Middle -->
     <xacro:thmiddle muscle="${muscletrans}" bio="${bio}"
-    prefix="${prefix}" parent="${prefix}thhub" simple_collisions="${simple_collisions}"></xacro:thmiddle>
+    prefix="${prefix}" parent="${prefix}thhub"></xacro:thmiddle>
     <!-- Distal -->
     <xacro:thdistal muscle="${muscletrans}" bio="${bio}" bt_sp="${bt_sp}"

File: sr_description/hand/xacro/wrist/wrist.urdf.xacro (robot description, xacro)
@@ -6,5 +6,5 @@
   <!-- parent is the parent joint -->
   <xacro:macro name="wrist"
-  params="muscletrans prefix reflect parent *origin simple_collisions">
+  params="muscletrans prefix reflect parent *origin">
     <link name="${prefix}wrist">
       <inertial>
@@ -22,47 +22,36 @@
         <material name="LightGrey" />
       </visual>
-      <xacro:if value="${simple_collisions}">
-        <collision>
-          <origin xyz="0 0 0" rpy="1.5708 1.5708 0" />
-          <geometry name="${prefix}wrist_collision_geom">
-            <cylinder radius="0.0135" length="0.030" />
-          </geometry>
-        </collision>
-        <collision>
-          <origin xyz="${reflect*-0.026} 0 0.034" rpy="0 1.5708 0" />
-          <geometry>
-            <cylinder radius="0.011" length="0.010" />
-          </geometry>
-        </collision>
-        <collision>
-          <origin xyz="${reflect*0.031} 0 0.034" rpy="0 1.5708 0" />
-          <geometry>
-            <cylinder radius="0.011" length="0.010" />
-          </geometry>
-        </collision>
-        <collision>
-          <origin xyz="${reflect*-0.021} 0 0.011"
-          rpy="0 ${reflect*0.7854} 0" />
-          <geometry>
-            <box size="0.027 0.018 0.010" />
-          </geometry>
-        </collision>
-        <collision>
-          <origin xyz="${reflect*0.026} 0 0.010"
-          rpy="0 ${reflect*-0.7854} 0" />
-          <geometry>
-            <box size="0.027 0.018 0.010" />
-          </geometry>
-        </collision>
-      </xacro:if>
-      <xacro:unless value="${simple_collisions}">
-        <collision>
-          <origin xyz="0 0 0" rpy="0 0 0" />
-          <geometry name="${prefix}wrist_collision_geom">
-            <mesh filename="package://sr_description/hand/model/wrist.dae"
-            scale="${reflect*0.001} 0.001 0.001" />
-          </geometry>
-        </collision>
-      </xacro:unless>
+      <collision>
+        <origin xyz="0 0 0" rpy="1.5708 1.5708 0" />
+        <geometry name="${prefix}wrist_collision_geom">
+          <cylinder radius="0.0135" length="0.030" />
+        </geometry>
+      </collision>
+      <collision>
+        <origin xyz="${reflect*-0.026} 0 0.034" rpy="0 1.5708 0" />
+        <geometry>
+          <cylinder radius="0.011" length="0.010" />
+        </geometry>
+      </collision>
+      <collision>
+        <origin xyz="${reflect*0.031} 0 0.034" rpy="0 1.5708 0" />
+        <geometry>
+          <cylinder radius="0.011" length="0.010" />
+        </geometry>
+      </collision>
+      <collision>
+        <origin xyz="${reflect*-0.021} 0 0.011"
+        rpy="0 ${reflect*0.7854} 0" />
+        <geometry>
+          <box size="0.027 0.018 0.010" />
+        </geometry>
+      </collision>
+      <collision>
+        <origin xyz="${reflect*0.026} 0 0.010"
+        rpy="0 ${reflect*-0.7854} 0" />
+        <geometry>
+          <box size="0.027 0.018 0.010" />
+        </geometry>
+      </collision>
     </link>
     <gazebo reference="${prefix}wrist">

File: sr_description/robots/shadowhand_motor.urdf.xacro (robot description, xacro)
@@ -15,4 +15,4 @@
     </joint>
     <xacro:shadowhand muscletrans="false" muscle="false" hand_type="hand_e" bio="false" bt_sp="false"
-                      ubi="false" eli="false" reflect="1.0" prefix="rh_" lf="true" simple_collisions="true" />
+                      ubi="false" eli="false" reflect="1.0" prefix="rh_" lf="true" />
 </robot>
