Commit message: Moving hand meshes to a more standard path to make gzweb work. Updating xacros accordingly.

File: sr_description/hand/xacro/finger/biotac/biotac.urdf.xacro (robot description, xacro)
@@ -24,5 +24,5 @@
         <origin xyz="0 0 0" rpy="0 0 1.571" />
         <geometry name="${prefix}${link_prefix}middle_visual">
-          <mesh filename="package://sr_description/hand/model/biotacs/biotac_finger_adapter.dae"
+          <mesh filename="package://sr_description/meshes/hand/biotacs/biotac_finger_adapter.dae"
           scale="1 1 1" />
         </geometry>
@@ -104,6 +104,6 @@
         <origin xyz="0 0 0" rpy="0 0 0" />
         <geometry name="${prefix}${link_prefix}distal_visual">
-          <!-- <mesh filename="package://sr_description/hand/model/biotacs/biotac.stl" scale="0.0254 0.0254 0.0254" /> -->
-          <mesh filename="package://sr_description/hand/model/biotacs/biotac_decimated.dae"
+          <!-- <mesh filename="package://sr_description/meshes/hand/biotacs/biotac.stl" scale="0.0254 0.0254 0.0254" /> -->
+          <mesh filename="package://sr_description/meshes/hand/biotacs/biotac_decimated.dae"
           scale="0.0254 0.0254 0.0254" />
         </geometry>
@@ -111,6 +111,6 @@
       <collision>
         <geometry name="${prefix}${link_prefix}distal_collision_geom">
-          <!-- <mesh filename="package://sr_description/hand/model/biotacs/biotac.stl" scale="0.0254 0.0254 0.0254" /> -->
-          <mesh filename="package://sr_description/hand/model/biotacs/biotac_decimated.dae"
+          <!-- <mesh filename="package://sr_description/meshes/hand/biotacs/biotac.stl" scale="0.0254 0.0254 0.0254" /> -->
+          <mesh filename="package://sr_description/meshes/hand/biotacs/biotac_decimated.dae"
           scale="0.0254 0.0254 0.0254" />
         </geometry>

File: sr_description/hand/xacro/finger/distal/distal.urdf.xacro (robot description, xacro)
@@ -31,5 +31,5 @@
           <xacro:if value="${ubi}">
             <!-- Ubi distal -->
-            <mesh filename="package://sr_description/hand/model/ubi_tactiles/ubi_tip_visual.dae"
+            <mesh filename="package://sr_description/meshes/hand/ubi_tactiles/ubi_tip_visual.dae"
 		  scale="0.001 0.001 0.001" />
           </xacro:if>
@@ -37,5 +37,5 @@
             <xacro:if value="${eli}">
               <!-- Ellispoid distal  -->
-              <mesh filename="package://sr_description/hand/model/ellipsoids/distal_ellipsoid_visual.dae"
+              <mesh filename="package://sr_description/meshes/hand/ellipsoids/distal_ellipsoid_visual.dae"
 		    scale="0.001 0.001 0.001" />
             </xacro:if>
@@ -43,5 +43,5 @@
               <xacro:if value="${bio}">
                 <!-- biotac distal  -->
-                <mesh filename="package://sr_description/hand/model/F1.dae"
+                <mesh filename="package://sr_description/meshes/hand/F1.dae"
                       scale="0.001 0.001 0.001" />
               </xacro:if>
@@ -49,9 +49,9 @@
 		<xacro:if value="${bt_sp}">
                   <!-- bt_sp distal  -->
-                  <mesh filename="package://sr_description/hand/model/biotacs/sp.dae" />
+                  <mesh filename="package://sr_description/meshes/hand/biotacs/sp.dae" />
 		</xacro:if>
 		<xacro:unless value="${bt_sp}">
                   <!-- Standard distal  -->
-                  <mesh filename="package://sr_description/hand/model/F1.dae"
+                  <mesh filename="package://sr_description/meshes/hand/F1.dae"
 			scale="0.001 0.001 0.001" />
 		</xacro:unless>
@@ -60,5 +60,5 @@
           </xacro:unless>
         </geometry>
-        <material name="Grey" />
+        <!-- <material name="Grey" /> -->
       </visual>
       <collision>
@@ -67,5 +67,5 @@
           <xacro:if value="${ubi}">
             <!-- Ubi distal -->
-            <mesh filename="package://sr_description/hand/model/ubi_tactiles/ubi_tip_collision.dae"
+            <mesh filename="package://sr_description/meshes/hand/ubi_tactiles/ubi_tip_collision.dae"
             scale="0.001 0.001 0.001" />
           </xacro:if>
@@ -73,5 +73,5 @@
             <xacro:if value="${eli}">
               <!-- Ellispoid distal  -->
-              <mesh filename="package://sr_description/hand/model/ellipsoids/distal_ellipsoid.dae"
+              <mesh filename="package://sr_description/meshes/hand/ellipsoids/distal_ellipsoid.dae"
               scale="0.001 0.001 0.001" />
             </xacro:if>
@@ -79,5 +79,5 @@
               <xacro:if value="${bio}">
                 <!-- biotac distal  -->
-                <mesh filename="package://sr_description/hand/model/F1.dae"
+                <mesh filename="package://sr_description/meshes/hand/F1.dae"
                 scale="0.001 0.001 0.001" />
               </xacro:if>
@@ -85,9 +85,9 @@
 		<xacro:if value="${bt_sp}">
                   <!-- bt_sp distal  -->
-                  <mesh filename="package://sr_description/hand/model/biotacs/sp.dae" />
+                  <mesh filename="package://sr_description/meshes/hand/biotacs/sp.dae" />
 		</xacro:if>
 		<xacro:unless value="${bt_sp}">
                   <!-- Standard distal  -->
-                  <mesh filename="package://sr_description/hand/model/F1.dae"
+                  <mesh filename="package://sr_description/meshes/hand/F1.dae"
 			scale="0.001 0.001 0.001" />
 		</xacro:unless>

File: sr_description/hand/xacro/finger/knuckle/knuckle.urdf.xacro (robot description, xacro)
@@ -25,5 +25,5 @@
         <origin xyz="0 0 0.0005" rpy="0 0 0" />
         <geometry name="${prefix}${link_prefix}knuckle_visual">
-          <mesh filename="package://sr_description/hand/model/knuckle.dae"
+          <mesh filename="package://sr_description/meshes/hand/knuckle.dae"
           scale="0.001 0.001 0.001" />
         </geometry>

File: sr_description/hand/xacro/finger/lfmetacarpal/lfmetacarpal.urdf.xacro (robot description, xacro)
@@ -24,5 +24,5 @@
         <origin xyz="0 0 0" rpy="0 0 0" />
         <geometry name="${prefix}lfmetacarpal_visual">
-          <mesh filename="package://sr_description/hand/model/lfmetacarpal.dae"
+          <mesh filename="package://sr_description/meshes/hand/lfmetacarpal.dae"
           scale="${reflect*0.001} 0.001 0.001" />
         </geometry>

File: sr_description/hand/xacro/finger/middle/middle.urdf.xacro (robot description, xacro)
@@ -25,5 +25,5 @@
         <origin xyz="0 0 0" rpy="0 0 0" />
         <geometry name="${prefix}${link_prefix}middle_visual">
-          <mesh filename="package://sr_description/hand/model/F2.dae"
+          <mesh filename="package://sr_description/meshes/hand/F2.dae"
           scale="0.001 0.001 0.001" />
         </geometry>

File: sr_description/hand/xacro/finger/proximal/proximal.urdf.xacro (robot description, xacro)
@@ -25,5 +25,5 @@
         <origin xyz="0 0 0" rpy="0 0 0" />
         <geometry name="${prefix}${link_prefix}proximal_visual">
-          <mesh filename="package://sr_description/hand/model/F3.dae"
+          <mesh filename="package://sr_description/meshes/hand/F3.dae"
           scale="0.001 0.001 0.001" />
         </geometry>

File: sr_description/hand/xacro/forearm/forearm.urdf.xacro (robot description, xacro)
@@ -26,5 +26,5 @@
           <origin xyz="0 0 0" rpy="0 0 0" />
           <geometry name="${prefix}forearm_visual">
-            <mesh filename="package://sr_description/hand/model/forearm_muscle.dae" scale="1.0 1.0 1.0" />
+            <mesh filename="package://sr_description/meshes/hand/forearm_muscle.dae" scale="1.0 1.0 1.0" />
           </geometry>
           <material name="Grey" />
@@ -36,5 +36,5 @@
             <origin xyz="0 0 0" rpy="0 0 0" />
             <geometry name="${prefix}forearm_visual">
-              <mesh filename="package://sr_description/hand/model/forearm.dae" scale="0.001 0.001 0.001" />
+              <mesh filename="package://sr_description/meshes/hand/forearm.dae" scale="0.001 0.001 0.001" />
             </geometry>
             <material name="light_grey" />
@@ -45,5 +45,5 @@
             <origin xyz="0 0 0" rpy="0 0 0" />
             <geometry name="${prefix}forearm_visual">
-              <mesh filename="package://sr_description/hand/model/forearm_visual_plus.dae" scale="0.001 0.001 0.001" />
+              <mesh filename="package://sr_description/meshes/hand/forearm_visual_plus.dae" scale="0.001 0.001 0.001" />
             </geometry>
             <material name="light_grey" />
@@ -70,5 +70,5 @@
             <origin xyz="0 0 0" rpy="0 0 0" />
             <geometry name="${prefix}forearm_collision">
-              <mesh filename="package://sr_description/hand/model/forearm_collision_plus.stl" scale="0.001 0.001 0.001" />
+              <mesh filename="package://sr_description/meshes/hand/forearm_collision_plus.stl" scale="0.001 0.001 0.001" />
             </geometry>
             <xacro:dark_grey/>
@@ -95,5 +95,5 @@
           <origin rpy="0 -1.57 -1.57" xyz="0.0 0.067 0.0045"/>
           <geometry name="${prefix}cable_extr_visualisation">
-            <mesh filename="package://sr_description/hand/model/cable_collision_mesh.stl" scale="1 1 1" />
+            <mesh filename="package://sr_description/meshes/hand/cable_collision_mesh.stl" scale="1 1 1" />
           </geometry>
         </visual>
@@ -101,5 +101,5 @@
           <origin rpy="0 -1.57 -1.57" xyz="0.0 0.067 0.0045"/>
           <geometry name="${prefix}cable_extr_collision">
-            <mesh filename="package://sr_description/hand/model/cable_collision_mesh.stl" scale="1 1 1" />
+            <mesh filename="package://sr_description/meshes/hand/cable_collision_mesh.stl" scale="1 1 1" />
           </geometry>
         </collision>

File: sr_description/hand/xacro/forearm/forearm_lite.urdf.xacro (robot description, xacro)
@@ -16,9 +16,9 @@
         <geometry name="${prefix}forearm_visual">
           <xacro:if value="${muscle}">
-            <mesh filename="package://sr_description/hand/model/forearm_lite.dae"
+            <mesh filename="package://sr_description/meshes/hand/forearm_lite.dae"
             scale="1.0 1.0 1.0" />
           </xacro:if>
           <xacro:unless value="${muscle}">
-            <mesh filename="package://sr_description/hand/model/forearm_lite.dae"
+            <mesh filename="package://sr_description/meshes/hand/forearm_lite.dae"
             scale="1.0 1.0 1.0" />
           </xacro:unless>
@@ -44,5 +44,5 @@
           <origin rpy="0 -1.57 -1.57" xyz="0.0 0.055 0.0"/>
           <geometry name="${prefix}cable_extr_visualisation">
-            <mesh filename="package://sr_description/hand/model/cable_collision_mesh.stl" scale="1 1 1" />
+            <mesh filename="package://sr_description/meshes/hand/cable_collision_mesh.stl" scale="1 1 1" />
           </geometry>
         </visual>
@@ -50,5 +50,5 @@
           <origin rpy="0 -1.57 -1.57" xyz="0.0 0.055 0.0"/>
           <geometry name="${prefix}cable_extr_collision">
-            <mesh filename="package://sr_description/hand/model/cable_collision_mesh.stl" scale="1 1 1" />
+            <mesh filename="package://sr_description/meshes/hand/cable_collision_mesh.stl" scale="1 1 1" />
           </geometry>
         </collision>

File: sr_description/hand/xacro/palm/palm.urdf.xacro (robot description, xacro)
@@ -25,5 +25,5 @@
         <origin xyz="0 0 0" rpy="0 0 0" />
         <geometry name="${prefix}palm_visual">
-          <mesh filename="package://sr_description/hand/model/palm.dae"
+          <mesh filename="package://sr_description/meshes/hand/palm.dae"
           scale="${reflect*0.001} 0.001 0.001" />
         </geometry>

File: sr_description/hand/xacro/palm/palm_lite.urdf.xacro (robot description, xacro)
@@ -24,5 +24,5 @@
         <origin xyz="0 0 0" rpy="0 0 0" />
         <geometry name="${prefix}palm_visual">
-          <mesh filename="package://sr_description/hand/model/palm.dae"
+          <mesh filename="package://sr_description/meshes/hand/palm.dae"
           scale="${reflect*0.001} 0.001 0.001" />
         </geometry>

File: sr_description/hand/xacro/thumb/thdistal.urdf.xacro (robot description, xacro)
@@ -51,6 +51,6 @@
           <origin xyz="0 0 0" rpy="0 0 0" />
           <geometry name="${prefix}th_distal_visual">
-            <!-- <mesh filename="package://sr_description/hand/model/biotacs/biotac.stl" scale="0.0254 0.0254 0.0254" /> -->
-            <mesh filename="package://sr_description/hand/model/biotacs/biotac_decimated.dae"
+            <!-- <mesh filename="package://sr_description/meshes/hand/biotacs/biotac.stl" scale="0.0254 0.0254 0.0254" /> -->
+            <mesh filename="package://sr_description/meshes/hand/biotacs/biotac_decimated.dae"
             scale="0.0254 0.0254 0.0254" />
           </geometry>
@@ -60,6 +60,6 @@
           <geometry name="${prefix}th_distal_collision_geom">
             <!-- <box size="0.001 0.001 0.001" /> -->
-            <!-- <mesh filename="package://sr_description/hand/model/biotacs/biotac-v5.stl" scale="0.0254 0.0254 0.0254" /> -->
-            <mesh filename="package://sr_description/hand/model/biotacs/biotac_decimated.dae"
+            <!-- <mesh filename="package://sr_description/meshes/hand/biotacs/biotac-v5.stl" scale="0.0254 0.0254 0.0254" /> -->
+            <mesh filename="package://sr_description/meshes/hand/biotacs/biotac_decimated.dae"
             scale="0.0254 0.0254 0.0254" />
           </geometry>
@@ -131,5 +131,5 @@
             <xacro:if value="${eli}">
               <!-- Ellispoid distal  -->
-              <mesh filename="package://sr_description/hand/model/ellipsoids/thdistal_ellipsoid_visual.dae"
+              <mesh filename="package://sr_description/meshes/hand/ellipsoids/thdistal_ellipsoid_visual.dae"
               scale="0.001 0.001 0.001" />
             </xacro:if>
@@ -137,5 +137,5 @@
               <xacro:if value="${ubi}">
                 <!-- Ubi distal -->
-                <mesh filename="package://sr_description/hand/model/TH1_z.dae"
+                <mesh filename="package://sr_description/meshes/hand/TH1_z.dae"
                       scale="0.001 0.001 0.001" />
               </xacro:if>
@@ -143,9 +143,9 @@
 		<xacro:if value="${bt_sp}">
 		  <!-- bt sp distal  -->
-		  <mesh filename="package://sr_description/hand/model/biotacs/sp.dae" />
+		  <mesh filename="package://sr_description/meshes/hand/biotacs/sp.dae" />
 		</xacro:if>
 		<xacro:unless value="${bt_sp}">
 		  <!-- Standard distal  -->
-                  <mesh filename="package://sr_description/hand/model/TH1_z.dae"
+                  <mesh filename="package://sr_description/meshes/hand/TH1_z.dae"
 			scale="0.001 0.001 0.001" />
 		</xacro:unless>
@@ -162,5 +162,5 @@
             <xacro:if value="${eli}">
               <!-- Ellispoid distal  -->
-              <mesh filename="package://sr_description/hand/model/ellipsoids/thdistal_ellipsoid.dae"
+              <mesh filename="package://sr_description/meshes/hand/ellipsoids/thdistal_ellipsoid.dae"
               scale="0.001 0.001 0.001" />
             </xacro:if>
@@ -168,5 +168,5 @@
               <xacro:if value="${ubi}">
                 <!-- Ubi distal -->
-                <mesh filename="package://sr_description/hand/model/TH1_z.dae"
+                <mesh filename="package://sr_description/meshes/hand/TH1_z.dae"
                 scale="0.001 0.001 0.001" />
               </xacro:if>
@@ -174,9 +174,9 @@
 		<xacro:if value="${bt_sp}">
 		  <!-- bt sp distal  -->
-                  <mesh filename="package://sr_description/hand/model/biotacs/sp.dae" />
+                  <mesh filename="package://sr_description/meshes/hand/biotacs/sp.dae" />
 		</xacro:if>
 		<xacro:unless value="${bt_sp}">
                   <!-- Standard distal  -->
-                  <mesh filename="package://sr_description/hand/model/TH1_z.dae"
+                  <mesh filename="package://sr_description/meshes/hand/TH1_z.dae"
 			scale="0.001 0.001 0.001" />
 		</xacro:unless>

File: sr_description/hand/xacro/thumb/thmiddle.urdf.xacro (robot description, xacro)
@@ -24,5 +24,5 @@
         <xacro:if value="${bio}">
           <geometry name="${prefix}thmiddle_visual">
-            <mesh filename="package://sr_description/hand/model/biotacs/biotac_thumb_adapter.dae"
+            <mesh filename="package://sr_description/meshes/hand/biotacs/biotac_thumb_adapter.dae"
             scale="0.001 0.001 0.001" />
           </geometry>
@@ -30,5 +30,5 @@
         <xacro:unless value="${bio}">
           <geometry name="${prefix}thmiddle_visual">
-            <mesh filename="package://sr_description/hand/model/TH2_z.dae"
+            <mesh filename="package://sr_description/meshes/hand/TH2_z.dae"
             scale="0.001 0.001 0.001" />
           </geometry>

File: sr_description/hand/xacro/thumb/thproximal.urdf.xacro (robot description, xacro)
@@ -24,5 +24,5 @@
         <origin xyz="0 0 0" rpy="0 0 0" />
         <geometry name="${prefix}thproximal_visual">
-          <mesh filename="package://sr_description/hand/model/TH3_z.dae"
+          <mesh filename="package://sr_description/meshes/hand/TH3_z.dae"
           scale="0.001 0.001 0.001" />
         </geometry>

File: sr_description/hand/xacro/wrist/wrist.urdf.xacro (robot description, xacro)
@@ -17,5 +17,5 @@
         <origin xyz="0 0 0" rpy="0 0 0" />
         <geometry name="${prefix}wrist_visual">
-          <mesh filename="package://sr_description/hand/model/wrist.dae"
+          <mesh filename="package://sr_description/meshes/hand/wrist.dae"
           scale="${reflect*0.001} 0.001 0.001" />
         </geometry>

File: sr_description/mujoco_models/urdfs/shadowhand_motor.urdf (robot description, URDF)
Before this commit: robot shadowhand_motor, 33 links, 32 joints
Links:
- link rh_ffdistal: geometry collision mesh filename=package://sr_description/meshes/hand/F1.dae scale=0.001 0.001 0.001; visual mesh filename=package://sr_description/meshes/hand/F1.dae scale=0.001 0.001 0.001
- link rh_ffknuckle: geometry collision cylinder length=0.014 radius=0.007; visual mesh filename=package://sr_description/meshes/hand/knuckle.dae scale=0.001 0.001 0.001
- link rh_ffmiddle: geometry collision cylinder length=0.025 radius=0.007; collision sphere radius=0.007
- link rh_ffproximal: geometry collision cylinder length=0.040 radius=0.007; visual mesh filename=package://sr_description/meshes/hand/F3.dae scale=0.001 0.001 0.001
- link rh_forearm: geometry collision box size=0.07 0.07 0.07; collision cylinder length=0.184 radius=0.07
- link rh_lfdistal: geometry collision mesh filename=package://sr_description/meshes/hand/F1.dae scale=0.001 0.001 0.001; visual mesh filename=package://sr_description/meshes/hand/F1.dae scale=0.001 0.001 0.001
- link rh_lfknuckle: geometry collision cylinder length=0.014 radius=0.007; visual mesh filename=package://sr_description/meshes/hand/knuckle.dae scale=0.001 0.001 0.001
- link rh_lfmetacarpal: geometry collision box size=0.018 0.024 0.040; visual mesh filename=package://sr_description/meshes/hand/lfmetacarpal.dae scale=0.001 0.001 0.001
- link rh_lfmiddle: geometry collision cylinder length=0.025 radius=0.007; collision sphere radius=0.007
- link rh_lfproximal: geometry collision cylinder length=0.040 radius=0.007; visual mesh filename=package://sr_description/meshes/hand/F3.dae scale=0.001 0.001 0.001
- link rh_mfdistal: geometry collision mesh filename=package://sr_description/meshes/hand/F1.dae scale=0.001 0.001 0.001; visual mesh filename=package://sr_description/meshes/hand/F1.dae scale=0.001 0.001 0.001
- link rh_mfknuckle: geometry collision cylinder length=0.014 radius=0.007; visual mesh filename=package://sr_description/meshes/hand/knuckle.dae scale=0.001 0.001 0.001
- link rh_mfmiddle: geometry collision cylinder length=0.025 radius=0.007; collision sphere radius=0.007
- link rh_mfproximal: geometry collision cylinder length=0.040 radius=0.007; visual mesh filename=package://sr_description/meshes/hand/F3.dae scale=0.001 0.001 0.001
- link rh_palm: geometry collision box size=0.018 0.024 0.004; collision box size=0.020 0.024 0.040
- link rh_rfdistal: geometry collision mesh filename=package://sr_description/meshes/hand/F1.dae scale=0.001 0.001 0.001; visual mesh filename=package://sr_description/meshes/hand/F1.dae scale=0.001 0.001 0.001
- link rh_rfknuckle: geometry collision cylinder length=0.014 radius=0.007; visual mesh filename=package://sr_description/meshes/hand/knuckle.dae scale=0.001 0.001 0.001
- link rh_rfmiddle: geometry collision cylinder length=0.025 radius=0.007; collision sphere radius=0.007
- link rh_rfproximal: geometry collision cylinder length=0.040 radius=0.007; visual mesh filename=package://sr_description/meshes/hand/F3.dae scale=0.001 0.001 0.001
- link rh_thdistal: geometry collision mesh filename=package://sr_description/meshes/hand/TH1_z.dae scale=0.001 0.001 0.001; visual mesh filename=package://sr_description/meshes/hand/TH1_z.dae scale=0.001 0.001 0.001
- link rh_thmiddle: geometry collision cylinder length=0.018 radius=0.011; collision sphere radius=0.011
- link rh_thproximal: geometry collision cylinder length=0.018 radius=0.012; visual mesh filename=package://sr_description/meshes/hand/TH3_z.dae scale=0.001 0.001 0.001
- link rh_wrist: geometry collision box size=0.027 0.018 0.010; collision box size=0.027 0.018 0.010
