Commit message: Moving hand meshes to a more standard path to make gzweb work. Updating xacros accordingly.

File: sr_description/mujoco_models/urdfs/shadowhand_motor_left.urdf (robot description, URDF)
Before this commit: robot shadowhand_motor, 33 links, 32 joints
Links:
- link lh_ffdistal: geometry collision mesh filename=package://sr_description/meshes/hand/F1.dae scale=0.001 0.001 0.001; visual mesh filename=package://sr_description/meshes/hand/F1.dae scale=0.001 0.001 0.001
- link lh_ffknuckle: geometry collision cylinder length=0.014 radius=0.007; visual mesh filename=package://sr_description/meshes/hand/knuckle.dae scale=0.001 0.001 0.001
- link lh_ffmiddle: geometry collision cylinder length=0.025 radius=0.007; collision sphere radius=0.007
- link lh_ffproximal: geometry collision cylinder length=0.040 radius=0.007; visual mesh filename=package://sr_description/meshes/hand/F3.dae scale=0.001 0.001 0.001
- link lh_forearm: geometry collision box size=0.07 0.07 0.07; collision cylinder length=0.184 radius=0.07
- link lh_lfdistal: geometry collision mesh filename=package://sr_description/meshes/hand/F1.dae scale=0.001 0.001 0.001; visual mesh filename=package://sr_description/meshes/hand/F1.dae scale=0.001 0.001 0.001
- link lh_lfknuckle: geometry collision cylinder length=0.014 radius=0.007; visual mesh filename=package://sr_description/meshes/hand/knuckle.dae scale=0.001 0.001 0.001
- link lh_lfmetacarpal: geometry collision box size=0.018 0.024 0.040; visual mesh filename=package://sr_description/meshes/hand/lfmetacarpal.dae scale=-0.001 0.001 0.001
- link lh_lfmiddle: geometry collision cylinder length=0.025 radius=0.007; collision sphere radius=0.007
- link lh_lfproximal: geometry collision cylinder length=0.040 radius=0.007; visual mesh filename=package://sr_description/meshes/hand/F3.dae scale=0.001 0.001 0.001
- link lh_mfdistal: geometry collision mesh filename=package://sr_description/meshes/hand/F1.dae scale=0.001 0.001 0.001; visual mesh filename=package://sr_description/meshes/hand/F1.dae scale=0.001 0.001 0.001
- link lh_mfknuckle: geometry collision cylinder length=0.014 radius=0.007; visual mesh filename=package://sr_description/meshes/hand/knuckle.dae scale=0.001 0.001 0.001
- link lh_mfmiddle: geometry collision cylinder length=0.025 radius=0.007; collision sphere radius=0.007
- link lh_mfproximal: geometry collision cylinder length=0.040 radius=0.007; visual mesh filename=package://sr_description/meshes/hand/F3.dae scale=0.001 0.001 0.001
- link lh_palm: geometry collision box size=0.018 0.024 0.004; collision box size=0.020 0.024 0.040
- link lh_rfdistal: geometry collision mesh filename=package://sr_description/meshes/hand/F1.dae scale=0.001 0.001 0.001; visual mesh filename=package://sr_description/meshes/hand/F1.dae scale=0.001 0.001 0.001
- link lh_rfknuckle: geometry collision cylinder length=0.014 radius=0.007; visual mesh filename=package://sr_description/meshes/hand/knuckle.dae scale=0.001 0.001 0.001
- link lh_rfmiddle: geometry collision cylinder length=0.025 radius=0.007; collision sphere radius=0.007
- link lh_rfproximal: geometry collision cylinder length=0.040 radius=0.007; visual mesh filename=package://sr_description/meshes/hand/F3.dae scale=0.001 0.001 0.001
- link lh_thdistal: geometry collision mesh filename=package://sr_description/meshes/hand/TH1_z.dae scale=0.001 0.001 0.001; visual mesh filename=package://sr_description/meshes/hand/TH1_z.dae scale=0.001 0.001 0.001
- link lh_thmiddle: geometry collision cylinder length=0.018 radius=0.011; collision sphere radius=0.011
- link lh_thproximal: geometry collision cylinder length=0.018 radius=0.012; visual mesh filename=package://sr_description/meshes/hand/TH3_z.dae scale=0.001 0.001 0.001
- link lh_wrist: geometry collision box size=0.027 0.018 0.010; collision box size=0.027 0.018 0.010

File: sr_description/mujoco_models/urdfs/shadowhand_motor_plus.urdf (robot description, URDF)
Before this commit: robot shadowhand_motor, 33 links, 32 joints
Links:
- link rh_ffdistal: geometry collision mesh filename=package://sr_description/meshes/hand/F1.dae scale=0.001 0.001 0.001; visual mesh filename=package://sr_description/meshes/hand/F1.dae scale=0.001 0.001 0.001
- link rh_ffknuckle: geometry collision cylinder length=0.014 radius=0.007; visual mesh filename=package://sr_description/meshes/hand/knuckle.dae scale=0.001 0.001 0.001
- link rh_ffmiddle: geometry collision cylinder length=0.025 radius=0.007; collision sphere radius=0.007
- link rh_ffproximal: geometry collision cylinder length=0.040 radius=0.007; visual mesh filename=package://sr_description/meshes/hand/F3.dae scale=0.001 0.001 0.001
- link rh_forearm: geometry collision box size=0.07 0.07 0.07; collision mesh filename=package://sr_description/meshes/hand/forearm_collision_plus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 scale=0.001 0.001 0.001
- link rh_lfdistal: geometry collision mesh filename=package://sr_description/meshes/hand/F1.dae scale=0.001 0.001 0.001; visual mesh filename=package://sr_description/meshes/hand/F1.dae scale=0.001 0.001 0.001
- link rh_lfknuckle: geometry collision cylinder length=0.014 radius=0.007; visual mesh filename=package://sr_description/meshes/hand/knuckle.dae scale=0.001 0.001 0.001
- link rh_lfmetacarpal: geometry collision box size=0.018 0.024 0.040; visual mesh filename=package://sr_description/meshes/hand/lfmetacarpal.dae scale=0.001 0.001 0.001
- link rh_lfmiddle: geometry collision cylinder length=0.025 radius=0.007; collision sphere radius=0.007
- link rh_lfproximal: geometry collision cylinder length=0.040 radius=0.007; visual mesh filename=package://sr_description/meshes/hand/F3.dae scale=0.001 0.001 0.001
- link rh_mfdistal: geometry collision mesh filename=package://sr_description/meshes/hand/F1.dae scale=0.001 0.001 0.001; visual mesh filename=package://sr_description/meshes/hand/F1.dae scale=0.001 0.001 0.001
- link rh_mfknuckle: geometry collision cylinder length=0.014 radius=0.007; visual mesh filename=package://sr_description/meshes/hand/knuckle.dae scale=0.001 0.001 0.001
- link rh_mfmiddle: geometry collision cylinder length=0.025 radius=0.007; collision sphere radius=0.007
- link rh_mfproximal: geometry collision cylinder length=0.040 radius=0.007; visual mesh filename=package://sr_description/meshes/hand/F3.dae scale=0.001 0.001 0.001
- link rh_palm: geometry collision box size=0.018 0.024 0.004; collision box size=0.020 0.024 0.040
- link rh_rfdistal: geometry collision mesh filename=package://sr_description/meshes/hand/F1.dae scale=0.001 0.001 0.001; visual mesh filename=package://sr_description/meshes/hand/F1.dae scale=0.001 0.001 0.001
- link rh_rfknuckle: geometry collision cylinder length=0.014 radius=0.007; visual mesh filename=package://sr_description/meshes/hand/knuckle.dae scale=0.001 0.001 0.001
- link rh_rfmiddle: geometry collision cylinder length=0.025 radius=0.007; collision sphere radius=0.007
- link rh_rfproximal: geometry collision cylinder length=0.040 radius=0.007; visual mesh filename=package://sr_description/meshes/hand/F3.dae scale=0.001 0.001 0.001
- link rh_thdistal: geometry collision mesh filename=package://sr_description/meshes/hand/TH1_z.dae scale=0.001 0.001 0.001; visual mesh filename=package://sr_description/meshes/hand/TH1_z.dae scale=0.001 0.001 0.001
- link rh_thmiddle: geometry collision cylinder length=0.018 radius=0.011; collision sphere radius=0.011
- link rh_thproximal: geometry collision cylinder length=0.018 radius=0.012; visual mesh filename=package://sr_description/meshes/hand/TH3_z.dae scale=0.001 0.001 0.001
- link rh_wrist: geometry collision box size=0.027 0.018 0.010; collision box size=0.027 0.018 0.010

File: sr_description/mujoco_models/urdfs/shadowhand_motor_plus_left.urdf (robot description, URDF)
Before this commit: robot shadowhand_motor, 33 links, 32 joints
Links:
- link lh_ffdistal: geometry collision mesh filename=package://sr_description/meshes/hand/F1.dae scale=0.001 0.001 0.001; visual mesh filename=package://sr_description/meshes/hand/F1.dae scale=0.001 0.001 0.001
- link lh_ffknuckle: geometry collision cylinder length=0.014 radius=0.007; visual mesh filename=package://sr_description/meshes/hand/knuckle.dae scale=0.001 0.001 0.001
- link lh_ffmiddle: geometry collision cylinder length=0.025 radius=0.007; collision sphere radius=0.007
- link lh_ffproximal: geometry collision cylinder length=0.040 radius=0.007; visual mesh filename=package://sr_description/meshes/hand/F3.dae scale=0.001 0.001 0.001
- link lh_forearm: geometry collision box size=0.07 0.07 0.07; collision mesh filename=package://sr_description/meshes/hand/forearm_collision_plus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 scale=0.001 0.001 0.001
- link lh_lfdistal: geometry collision mesh filename=package://sr_description/meshes/hand/F1.dae scale=0.001 0.001 0.001; visual mesh filename=package://sr_description/meshes/hand/F1.dae scale=0.001 0.001 0.001
- link lh_lfknuckle: geometry collision cylinder length=0.014 radius=0.007; visual mesh filename=package://sr_description/meshes/hand/knuckle.dae scale=0.001 0.001 0.001
- link lh_lfmetacarpal: geometry collision box size=0.018 0.024 0.040; visual mesh filename=package://sr_description/meshes/hand/lfmetacarpal.dae scale=-0.001 0.001 0.001
- link lh_lfmiddle: geometry collision cylinder length=0.025 radius=0.007; collision sphere radius=0.007
- link lh_lfproximal: geometry collision cylinder length=0.040 radius=0.007; visual mesh filename=package://sr_description/meshes/hand/F3.dae scale=0.001 0.001 0.001
- link lh_mfdistal: geometry collision mesh filename=package://sr_description/meshes/hand/F1.dae scale=0.001 0.001 0.001; visual mesh filename=package://sr_description/meshes/hand/F1.dae scale=0.001 0.001 0.001
- link lh_mfknuckle: geometry collision cylinder length=0.014 radius=0.007; visual mesh filename=package://sr_description/meshes/hand/knuckle.dae scale=0.001 0.001 0.001
- link lh_mfmiddle: geometry collision cylinder length=0.025 radius=0.007; collision sphere radius=0.007
- link lh_mfproximal: geometry collision cylinder length=0.040 radius=0.007; visual mesh filename=package://sr_description/meshes/hand/F3.dae scale=0.001 0.001 0.001
- link lh_palm: geometry collision box size=0.018 0.024 0.004; collision box size=0.020 0.024 0.040
- link lh_rfdistal: geometry collision mesh filename=package://sr_description/meshes/hand/F1.dae scale=0.001 0.001 0.001; visual mesh filename=package://sr_description/meshes/hand/F1.dae scale=0.001 0.001 0.001
- link lh_rfknuckle: geometry collision cylinder length=0.014 radius=0.007; visual mesh filename=package://sr_description/meshes/hand/knuckle.dae scale=0.001 0.001 0.001
- link lh_rfmiddle: geometry collision cylinder length=0.025 radius=0.007; collision sphere radius=0.007
- link lh_rfproximal: geometry collision cylinder length=0.040 radius=0.007; visual mesh filename=package://sr_description/meshes/hand/F3.dae scale=0.001 0.001 0.001
- link lh_thdistal: geometry collision mesh filename=package://sr_description/meshes/hand/TH1_z.dae scale=0.001 0.001 0.001; visual mesh filename=package://sr_description/meshes/hand/TH1_z.dae scale=0.001 0.001 0.001
- link lh_thmiddle: geometry collision cylinder length=0.018 radius=0.011; collision sphere radius=0.011
- link lh_thproximal: geometry collision cylinder length=0.018 radius=0.012; visual mesh filename=package://sr_description/meshes/hand/TH3_z.dae scale=0.001 0.001 0.001
- link lh_wrist: geometry collision box size=0.027 0.018 0.010; collision box size=0.027 0.018 0.010

File: sr_description/robots/shadowhand_edc_muscle.urdf.xacro (robot description, xacro)
@@ -26,5 +26,5 @@
       <origin xyz="0 0 0" rpy="0 0 0" />
       <geometry name="rh_forearm_disk_geom">
-        <mesh filename="package://sr_description/hand/model/forearm_muscle_disk.dae"
+        <mesh filename="package://sr_description/meshes/hand/forearm_muscle_disk.dae"
         scale="1.0 1.0 1.0" />
       </geometry>

File: sr_description/robots/shadowhand_edc_muscle_biotac.urdf.xacro (robot description, xacro)
@@ -29,5 +29,5 @@
       <origin xyz="0 0 0" rpy="0 0 0" />
       <geometry name="rh_forearm_disk_geom">
-        <mesh filename="package://sr_description/hand/model/forearm_muscle_disk.dae"
+        <mesh filename="package://sr_description/meshes/hand/forearm_muscle_disk.dae"
         scale="1.0 1.0 1.0" />
       </geometry>
