Commit message: distal refactored

File: sr_description/hand/xacro/finger/biotac/biotac.urdf.xacro (robot description, xacro)
@@ -1,9 +1,9 @@
 <robot xmlns:xacro="http://www.ros.org/wiki/xacro"
-xmlns:sensor="http://playerstage.sourceforge.net/gazebo/xmlschema/#sensor"
-xmlns:controller="http://playerstage.sourceforge.net/gazebo/xmlschema/#controller"
-xmlns:joint="http://playerstage.sourceforge.net/gazebo/xmlschema/#slider"
-xmlns:interface="http://playerstage.sourceforge.net/gazebo/xmlschema/#interface"
-xmlns:body="http://playerstage.sourceforge.net/gazebo/xmlschema/#body"
-xmlns:geom="http://playerstage.sourceforge.net/gazebo/xmlschema/#geom">
+       xmlns:sensor="http://playerstage.sourceforge.net/gazebo/xmlschema/#sensor"
+       xmlns:controller="http://playerstage.sourceforge.net/gazebo/xmlschema/#controller"
+       xmlns:joint="http://playerstage.sourceforge.net/gazebo/xmlschema/#slider"
+       xmlns:interface="http://playerstage.sourceforge.net/gazebo/xmlschema/#interface"
+       xmlns:body="http://playerstage.sourceforge.net/gazebo/xmlschema/#body"
+       xmlns:geom="http://playerstage.sourceforge.net/gazebo/xmlschema/#geom">
   <xacro:include filename="$(find sr_description)/hand/xacro/finger/middle/middle.transmission.xacro" />
   <!-- prefix can be anything but usually is "r_" or  "l_" for right and left hands distinction -->
@@ -11,18 +11,15 @@
   <!-- joint_prefix prepends fingername to the joint names -->
   <!-- parent is the parent link for the joint -->
-  <xacro:macro name="biotac_middle"
-  params="prefix:=^ link_prefix:=^ joint_prefix:=^ tip_sensor:=^|std mid_sensor:=^|std parent">
+  <xacro:macro name="biotac_middle" params="prefix:=^ link_prefix:=^ joint_prefix:=^ tip_sensor:=^|none mid_sensor:=^|none parent">
     <link name="${prefix}${link_prefix}middle">
       <inertial>
         <origin xyz="0 0 0.0125" rpy="0 0 0" />
         <mass value="0.017" />
-        <inertia ixx="0.0000026" ixy="0.0" ixz="0.0"
-        iyy="0.0000027" iyz="0.0" izz="0.00000087" />
+        <inertia ixx="0.0000026" ixy="0.0" ixz="0.0" iyy="0.0000027" iyz="0.0" izz="0.00000087" />
       </inertial>
       <visual>
         <origin xyz="0 0 0" rpy="0 0 1.571" />
         <geometry name="${prefix}${link_prefix}middle_visual">
-          <mesh filename="package://sr_description/meshes/hand/biotacs/biotac_finger_adapter.dae"
-          scale="1 1 1" />
+          <mesh filename="package://sr_description/meshes/hand/biotacs/biotac_finger_adapter.dae" scale="1 1 1" />
         </geometry>
         <material name="LightGrey" />
@@ -31,5 +28,5 @@
         <origin xyz="0 0 0.005" rpy="0 0 0" />
         <geometry name="${prefix}${link_prefix}middle_collision_geom">
-          <box size="0.001 0.001 0.001" />
+          <box size="0.001 0.001 0.001"/>
         </geometry>
       </collision>
@@ -37,21 +34,17 @@
     <gazebo reference="${prefix}${link_prefix}middle">
       <xacro:unless value="${mid_sensor == 'none'}">
-      <sensor type="contact"
-      name="${prefix}${link_prefix}middle_contact">
-        <always_on>1</always_on>
-        <update_rate>1000.0</update_rate>
-        <contact>
-          <collision>
-          ${prefix}${link_prefix}middle_collision</collision>
-          <topic>${prefix}${link_prefix}middle_collision</topic>
-        </contact>
-        <plugin name="${prefix}${link_prefix}middle_gazebo_ros_bumper_controller"
-        filename="libgazebo_ros_bumper.so">
-          <updateRate>100.0</updateRate>
-          <frameName>${prefix}${link_prefix}middle</frameName>
-          <bumperTopicName>
-          contacts/${prefix}${link_prefix}/middle</bumperTopicName>
-        </plugin>
-      </sensor>
+        <sensor type="contact" name="${prefix}${link_prefix}middle_contact">
+          <always_on>1</always_on>
+          <update_rate>1000.0</update_rate>
+          <contact>
+            <collision>${prefix}${link_prefix}middle_collision</collision>
+            <topic>${prefix}${link_prefix}middle_collision</topic>
+          </contact>
+          <plugin name="${prefix}${link_prefix}middle_gazebo_ros_bumper_controller" filename="libgazebo_ros_bumper.so">
+            <updateRate>100.0</updateRate>
+            <frameName>${prefix}${link_prefix}middle</frameName>
+            <bumperTopicName>contacts/${prefix}${link_prefix}/middle</bumperTopicName>
+          </plugin>
+        </sensor>
       </xacro:unless>
       <material>Gazebo/FlatBlack</material>
@@ -62,6 +55,5 @@
       <origin xyz="0 0 0.045" rpy="0 0 0" />
       <axis xyz="1 0 0" />
-      <limit lower="0" upper="${pi/2}" effort="2.0"
-      velocity="2.0" />
+      <limit lower="0" upper="${pi/2}" effort="2.0" velocity="2.0" />
       <dynamics damping="0.1" />
     </joint>
@@ -74,6 +66,5 @@
         <origin xyz="0 0 0.012" />
         <mass value="0.001" />
-        <inertia ixx="0.00000001" ixy="0.0" ixz="0.0"
-        iyy="0.00000001" iyz="0.0" izz="0.00000001" />
+        <inertia ixx="0.00000001" ixy="0.0" ixz="0.0" iyy="0.00000001" iyz="0.0" izz="0.00000001" />
       </inertial>
     </link>
@@ -83,6 +74,5 @@
       <origin xyz="0 0 0.02" rpy="0 0 0" />
       <axis xyz="1 0 0" />
-      <limit lower="${20*pi/180}" upper="${20.1*pi/180}"
-      effort="0.0" velocity="2.0" />
+      <limit lower="${20*pi/180}" upper="${20.1*pi/180}" effort="0.0" velocity="2.0" />
       <dynamics damping="0.5" />
     </joint>
@@ -97,6 +87,5 @@
         <!-- approximated only FIXME -->
         <mass value="0.012" />
-        <inertia ixx="0.00000094" ixy="0.0" ixz="0.0"
-        iyy="0.0000011" iyz="0.0" izz="0.00000053" />
+        <inertia ixx="0.00000094" ixy="0.0" ixz="0.0" iyy="0.0000011" iyz="0.0" izz="0.00000053" />
       </inertial>
       <visual>
@@ -104,6 +93,5 @@
         <geometry name="${prefix}${link_prefix}distal_visual">
           <!-- <mesh filename="package://sr_description/meshes/hand/biotacs/biotac.stl" scale="0.0254 0.0254 0.0254" /> -->
-          <mesh filename="package://sr_description/meshes/hand/biotacs/biotac_decimated.dae"
-          scale="0.0254 0.0254 0.0254" />
+          <mesh filename="package://sr_description/meshes/hand/biotacs/biotac_decimated.dae" scale="0.0254 0.0254 0.0254" />
         </geometry>
       </visual>
@@ -111,6 +99,5 @@
         <geometry name="${prefix}${link_prefix}distal_collision_geom">
           <!-- <mesh filename="package://sr_description/meshes/hand/biotacs/biotac.stl" scale="0.0254 0.0254 0.0254" /> -->
-          <mesh filename="package://sr_description/meshes/hand/biotacs/biotac_decimated.dae"
-          scale="0.0254 0.0254 0.0254" />
+          <mesh filename="package://sr_description/meshes/hand/biotacs/biotac_decimated.dae" scale="0.0254 0.0254 0.0254" />
         </geometry>
       </collision>
@@ -118,26 +105,21 @@
     <gazebo reference="${prefix}${link_prefix}distal">
       <xacro:unless value="${tip_sensor == 'none'}">
-      <sensor type="contact"
-      name="${prefix}${link_prefix}distal_contact">
-        <always_on>1</always_on>
-        <update_rate>1000.0</update_rate>
-        <contact>
-          <collision>
-          ${prefix}${link_prefix}distal_collision</collision>
-          <topic>${prefix}${link_prefix}distal_collision</topic>
-        </contact>
-        <plugin name="${prefix}${link_prefix}distal_gazebo_ros_bumper_controller"
-        filename="libgazebo_ros_bumper.so">
-          <updateRate>100.0</updateRate>
-          <frameName>${prefix}${link_prefix}distal</frameName>
-          <bumperTopicName>
-          contacts/${prefix}${link_prefix}/distal</bumperTopicName>
-        </plugin>
-      </sensor>
+        <sensor type="contact" name="${prefix}${link_prefix}distal_contact">
+          <always_on>1</always_on>
+          <update_rate>1000.0</update_rate>
+          <contact>
+            <collision>${prefix}${link_prefix}distal_collision</collision>
+            <topic>${prefix}${link_prefix}distal_collision</topic>
+          </contact>
+          <plugin name="${prefix}${link_prefix}distal_gazebo_ros_bumper_controller" filename="libgazebo_ros_bumper.so">
+            <updateRate>100.0</updateRate>
+            <frameName>${prefix}${link_prefix}distal</frameName>
+            <bumperTopicName>contacts/${prefix}${link_prefix}/distal</bumperTopicName>
+          </plugin>
+        </sensor>
       </xacro:unless>
       <selfCollide>true</selfCollide>
     </gazebo>
-    <joint name="${prefix}${joint_prefix}_distal_joint"
-    type="fixed">
+    <joint name="${prefix}${joint_prefix}_distal_joint" type="fixed">
       <parent link="${prefix}${link_prefix}middle" />
       <child link="${prefix}${link_prefix}distal" />
@@ -145,23 +127,15 @@
     </joint>
     <!-- extra link to imaginary sphere in fingertip for FK/IK calculations -->
-    <!-- remove visual and collision once the correct position is found -->
     <link name="${prefix}${link_prefix}tip">
       <inertial>
         <mass value="0.001" />
         <origin xyz="0 0 0" rpy="0 0 0" />
-        <inertia ixx="0.0" ixy="0.0" ixz="0.0" iyy="0.0" iyz="0.0"
-        izz="0.0" />
+        <inertia ixx="0.0" ixy="0.0" ixz="0.0" iyy="0.0" iyz="0.0" izz="0.0" />
       </inertial>
-      <!--visual>
-        <geometry>
-          <sphere radius="0.002" />
-        </geometry>
-      </visual-->
     </link>
     <gazebo reference="${prefix}${joint_prefix}tip">
       <material name="Gazebo/RedGlow" />
     </gazebo>
-    <joint name="${prefix}${joint_prefix}tip"
-    type="fixed">
+    <joint name="${prefix}${joint_prefix}tip" type="fixed">
       <parent link="${prefix}${link_prefix}_J1_dummy" />
       <child link="${prefix}${link_prefix}tip" />

File: sr_description/hand/xacro/finger/distal/distal.gazebo.xacro (robot description, xacro)
@@ -1,6 +1,5 @@
 <?xml version="1.0"?>
 <robot xmlns:xacro="http://www.ros.org/wiki/xacro">
-  <xacro:macro name="distal_gazebo" params="prefix:=^ link_prefix:=^ tip_sensor:=^|std ns:=^|''">
-    <!-- prefix can be anything but usually is "r_" or  "l_" for right and left hands distinction -->
+  <xacro:macro name="distal_gazebo" params="prefix:=^ link_prefix:=^ tip_sensor:=^|none ns:=^|''">
     <gazebo reference="${prefix}${link_prefix}distal">
       <xacro:unless value="${'none' in tip_sensor}" >

File: sr_description/hand/xacro/finger/distal/distal.transmission.xacro (robot description, xacro)
@@ -4,10 +4,7 @@
        xmlns:interface="http://playerstage.sourceforge.net/gazebo/xmlschema/#interface"
        xmlns:xacro="http://www.ros.org/wiki/xacro">
-  <!-- prefix can be anything but usually is "r_" or  "l_" for right and left hands distinction -->
-  <!-- link_prefix prepends fingername to the link names -->
-  <!-- joint_prefix prepends fingername to the joint names -->
   <xacro:macro name="distal_transmission" params="hand_type:=^ prefix:=^ joint_prefix:=^ link_prefix:=^" >
    <!-- muscle hand -->
-    <xacro:if value="${hand_type == 'muscletrans'}">
+    <xacro:if value="${hand_type == 'hand_c'}">
         <transmission name="${prefix}${link_prefix}distal_transmission">
             <type>sr_mechanism_model/SimpleTransmissionForMuscle</type>
@@ -22,5 +19,5 @@
     </xacro:if>
     <!-- motor hand -->
-    <xacro:unless value="${hand_type == 'muscletrans'}">
+    <xacro:unless value="${hand_type == 'hand_c'}">
         <transmission name="${prefix}${link_prefix}distal_transmission">
             <type>sr_mechanism_model/SimpleTransmission</type>

File: sr_description/hand/xacro/finger/distal/distal.urdf.xacro (robot description, xacro)
@@ -13,6 +13,5 @@
   <!-- joint_prefix prepends fingername to the joint names -->
   <!-- parent is the parent link for the joint -->
-  <xacro:macro name="distal"
-  params="prefix:=^ link_prefix:=^ joint_prefix:=^ tip_sensor:=^|std parent">
+  <xacro:macro name="distal" params="prefix:=^ link_prefix:=^ joint_prefix:=^ tip_sensor:=^|std parent">
     <link name="${prefix}${link_prefix}distal">
       <inertial>
@@ -25,44 +24,26 @@
         <origin xyz="0 0 0" rpy="0 0 0" />
         <geometry name="${prefix}${link_prefix}distal_visual">
-          <!-- Do we need to instantiate the standard distal? -->
-          <xacro:property name="standard" value="true" />
-          <xacro:if value="${tip_sensor == 'eli'}">
-            <!-- Ellispoid distal  -->
-            <mesh filename="package://sr_description/meshes/hand/ellipsoids/distal_ellipsoid_visual.dae"
-                  scale="0.001 0.001 0.001" />
-            <xacro:property name="standard" value="false" />
+          <xacro:if value="${tip_sensor == 'pst'}">
+            <mesh filename="package://sr_description/meshes/components/f_distal/pst/f_distal_pst.stl" scale="0.001 0.001 0.001" />
           </xacro:if>
           <xacro:if value="${tip_sensor == 'bt_sp'}">
-            <!-- bt_sp distal  -->
-            <mesh filename="package://sr_description/meshes/hand/biotacs/sp.dae" />
-            <xacro:property name="standard" value="false" />
+            <mesh filename="package://sr_description/meshes/components/f_distal/bt_sp/f_distal_bt_sp.stl" />
           </xacro:if>
-          <xacro:if value="${standard}">
-            <!-- Standard distal  -->
-            <mesh filename="package://sr_description/meshes/hand/F1.dae" scale="0.001 0.001 0.001" />
+          <xacro:if value="${tip_sensor == 'bt_2p'}">
+            <mesh filename="package://sr_description/meshes/components/f_distal/bt_2p/f_distal_bt_2p.dae" />
           </xacro:if>
         </geometry>
-        <!-- <material name="Grey" /> -->
       </visual>
       <collision>
         <origin xyz="0 0 0" rpy="0 0 0" />
         <geometry name="${prefix}${link_prefix}distal_collision_geom">
-          <!-- Do we need to instantiate the standard distal? -->
-          <xacro:property name="standard" value="true" />
-          <xacro:if value="${tip_sensor == 'eli'}">
-            <!-- Ellispoid distal  -->
-            <mesh filename="package://sr_description/meshes/hand/ellipsoids/distal_ellipsoid.dae"
-                  scale="0.001 0.001 0.001" />
-            <xacro:property name="standard" value="false" />
+          <xacro:if value="${tip_sensor == 'pst'}">
+            <mesh filename="package://sr_description/meshes/components/f_distal/pst/f_distal_pst.stl" scale="0.001 0.001 0.001" />
           </xacro:if>
           <xacro:if value="${tip_sensor == 'bt_sp'}">
-            <!-- bt_sp distal  -->
-            <mesh filename="package://sr_description/meshes/hand/biotacs/sp.dae" />
-            <xacro:property name="standard" value="false" />
+            <mesh filename="package://sr_description/meshes/components/f_distal/bt_sp/f_distal_bt_sp.stl" />
           </xacro:if>
-          <xacro:if value="${standard}">
-            <!-- Standard distal  -->
-            <mesh filename="package://sr_description/meshes/hand/F1.dae"
-                  scale="0.001 0.001 0.001" />
+          <xacro:if value="${tip_sensor == 'bt_2p'}">
+            <mesh filename="package://sr_description/meshes/components/f_distal/bt_2p/f_distal_bt_2p.dae" />
           </xacro:if>
         </geometry>

File: sr_description/hand/xacro/finger/fingers.urdf.xacro (robot description, xacro)
@@ -6,15 +6,6 @@
   <xacro:include filename="$(find sr_description)/hand/xacro/finger/lfmetacarpal/lfmetacarpal.urdf.xacro" />
   <xacro:include filename="$(find sr_description)/hand/xacro/finger/biotac/biotac.urdf.xacro" />
-  <!-- lf is true for little finger or false for standard finger -->
-  <!-- tip_sensor describes the sensor none, bt_2p, bt_sp, eli -->
-  <!-- mid_sensor describes the sensor none, bt_2p -->
-  <!-- prox_sensor describes the sensor none, standard -->
-  <!-- reflect is either 1 (for right hand) or -1 (for left hand) -->
-  <!-- prefix can be anything but usually is "r_" or  "l_" for right and left hands distinction -->
-  <!-- link_prefix prepends fingername to the link names -->
-  <!-- joint_prefix prepends fingername to the joint names -->
-  <!-- parent is the parent link for the first joint -->
-  <xacro:macro name="finger"
-  params="tip_sensor:=^|std mid_sensor:=^|std prox_sensor:=^|std reflect:=^ prefix:=^ link_prefix joint_prefix parent *origin *axis">
+  <xacro:macro name="finger" params="tip_sensor:=^|std mid_sensor:=^|std prox_sensor:=^|std reflect:=^ prefix:=^
+                                     link_prefix joint_prefix parent *origin *axis">
     <!-- Little finger special case -->
     <xacro:if value="${link_prefix == 'lf'}">

File: sr_description/hand/xacro/forearm/forearm_g.urdf.xacro (robot description, xacro)
@@ -12,43 +12,27 @@
         <origin xyz="0 0 0" rpy="0 0 ${pi/2}" />
         <geometry name="${prefix}forearm_visual">
-          <xacro:if value="${hand_type == 'muscle'}">
-            <mesh filename="package://sr_description/meshes/hand/forearm_lite.dae"
-            scale="1.0 1.0 1.0" />
-          </xacro:if>
-          <xacro:unless value="${hand_type == 'muscle'}">
-            <mesh filename="package://sr_description/meshes/hand/forearm_lite.dae"
-            scale="1.0 1.0 1.0" />
-          </xacro:unless>
+          <mesh filename="package://sr_description/meshes/products/${hand_type}/${hand_version}/forearm_${hand_version}.dae" scale="1.0 1.0 1.0" />
         </geometry>
         <material name="Grey" />
       </visual>
       <collision>
-        <xacro:if value="${hand_type == 'muscle'}">
-          <origin xyz="0 0 0.185" rpy="0 0 0" />
-          <geometry name="${prefix}forearm_collision">
-            <cylinder radius="0.075" length="0.37" />
-          </geometry>
-        </xacro:if>
-        <xacro:unless value="${hand_type == 'muscle'}">
-          <origin xyz="0 0 0.065" rpy="0 0 0" />
-          <geometry name="${prefix}forearm_collision">
-            <box size="0.120 0.109 0.130" />
-          </geometry>
-        </xacro:unless>
+        <origin xyz="0 0 0.065" rpy="0 0 0" />
+        <geometry name="${prefix}forearm_collision">
+          <box size="0.120 0.109 0.130" />
+        </geometry>
       </collision>
-      <xacro:if value="${cable_mesh}">
-        <visual>
-          <origin rpy="0 -1.57 -1.57" xyz="0.0 0.055 0.0"/>
-          <geometry name="${prefix}cable_extr_visualisation">
-            <mesh filename="package://sr_description/meshes/hand/cable_collision_mesh.stl" scale="1 1 1" />
-          </geometry>
-        </visual>
-        <collision>
-          <origin rpy="0 -1.57 -1.57" xyz="0.0 0.055 0.0"/>
-          <geometry name="${prefix}cable_extr_collision">
-            <mesh filename="package://sr_description/meshes/hand/cable_collision_mesh.stl" scale="1 1 1" />
-          </geometry>
-        </collision>
-      </xacro:if>
+      <!-- cable connector -->
+      <!--visual>
+        <origin rpy="0 -1.57 -1.57" xyz="0.0 0.055 0.0"/>
+        <geometry name="${prefix}cable_extr_visualisation">
+          <mesh filename="package://sr_description/meshes/products/${hand_type}/${hand_version}/cable_connector_base_${hand_version}.stl" scale="1 1 1" />
+        </geometry>
+      </visual>
+      <collision>
+        <origin rpy="0 -1.57 -1.57" xyz="0.0 0.055 0.0"/>
+        <geometry name="${prefix}cable_extr_collision">
+          <mesh filename="package://sr_description/meshes/products/${hand_type}/${hand_version}/cable_connector_base_${hand_version}.stl" scale="1 1 1" />
+        </geometry>
+      </collision-->
     </link>
   </xacro:macro>

File: sr_description/hand/xacro/palm/palm.transmission.xacro (robot description, xacro)
@@ -4,8 +4,7 @@
        xmlns:interface="http://playerstage.sourceforge.net/gazebo/xmlschema/#interface"
        xmlns:xacro="http://www.ros.org/wiki/xacro">
-    <!-- prefix can be anything but usually is "r_" or  "l_" for right and left hands distinction -->
     <xacro:macro name="shadowhand_palm_transmission" params="hand_type:=^ prefix:=^">
         <!-- muscle hand -->
-        <xacro:if value="${hand_type == 'muscletrans'}">
+        <xacro:if value="${hand_type == 'hand_c'}">
             <transmission name="${prefix}palm_transmission">
                 <type>sr_mechanism_model/SimpleTransmissionForMuscle</type>
@@ -20,5 +19,5 @@
         </xacro:if>
         <!-- motor hand -->
-        <xacro:unless value="${hand_type == 'muscletrans'}">
+        <xacro:unless value="${hand_type == 'hand_c'}">
             <transmission name="${prefix}palm_transmission">
                 <type>sr_mechanism_model/SimpleTransmission</type>
