Commit message: distal refactored

File: sr_description/hand/xacro/palm/palm_g.urdf.xacro (robot description, xacro)
@@ -1,27 +1,22 @@
 <robot xmlns:xacro="http://www.ros.org/wiki/xacro"
-xmlns:sensor="http://playerstage.sourceforge.net/gazebo/xmlschema/#sensor"
-xmlns:controller="http://playerstage.sourceforge.net/gazebo/xmlschema/#controller"
-xmlns:joint="http://playerstage.sourceforge.net/gazebo/xmlschema/#slider"
-xmlns:interface="http://playerstage.sourceforge.net/gazebo/xmlschema/#interface"
-xmlns:body="http://playerstage.sourceforge.net/gazebo/xmlschema/#body"
-xmlns:geom="http://playerstage.sourceforge.net/gazebo/xmlschema/#geom">
+       xmlns:sensor="http://playerstage.sourceforge.net/gazebo/xmlschema/#sensor"
+       xmlns:controller="http://playerstage.sourceforge.net/gazebo/xmlschema/#controller"
+       xmlns:joint="http://playerstage.sourceforge.net/gazebo/xmlschema/#slider"
+       xmlns:interface="http://playerstage.sourceforge.net/gazebo/xmlschema/#interface"
+       xmlns:body="http://playerstage.sourceforge.net/gazebo/xmlschema/#body"
+       xmlns:geom="http://playerstage.sourceforge.net/gazebo/xmlschema/#geom">
   <xacro:include filename="$(find sr_description)/hand/xacro/palm/palm.gazebo.xacro" />
   <xacro:include filename="$(find sr_description)/hand/xacro/palm/imu.urdf.xacro" />
-  <!-- prefix can be anything but usually is "r_" or  "l_" for right and left hands distinction -->
-  <!-- reflect is either 1 (for right hand) or -1 (for left hand) -->
-  <!-- parent is the parent link for the joint -->
-  <xacro:macro name="palm"
-  params="prefix:=^ reflect:=^ parent">
+  <xacro:macro name="palm" params="prefix:=^ reflect:=^ parent">
     <link name="${prefix}palm">
       <inertial>
         <origin xyz="0 0 0.035" rpy="0 0 0" />
         <mass value="0.3" />
-        <inertia ixx="0.0003581" ixy="0.0" ixz="0.0"
-        iyy="0.0005287" iyz="0.0" izz="0.000191" />
+        <inertia ixx="0.0003581" ixy="0.0" ixz="0.0" iyy="0.0005287" iyz="0.0" izz="0.000191" />
       </inertial>
       <visual>
         <origin xyz="0 0 0" rpy="0 0 0" />
         <geometry name="${prefix}palm_visual">
-          <mesh filename="package://sr_description/meshes/hand/palm.dae"
+          <mesh filename="package://sr_description/meshes/products/${hand_type}/${hand_version}/palm_${hand_version}.stl"
           scale="${reflect*0.001} 0.001 0.001" />
         </geometry>
@@ -35,6 +30,5 @@
       </collision>
       <collision>
-        <origin xyz="${reflect*0.0005} -0.0035 0.038"
-        rpy="0 0 0" />
+        <origin xyz="${reflect*0.0005} -0.0035 0.038" rpy="0 0 0" />
         <geometry>
           <box size="0.041 0.017 0.098" />
@@ -43,6 +37,5 @@
       <!-- palm complement below first finger -->
       <collision>
-        <origin xyz="${reflect*0.0315} -0.0035 0.073"
-        rpy="0 0 0" />
+        <origin xyz="${reflect*0.0315} -0.0035 0.073" rpy="0 0 0" />
         <geometry>
           <box size="0.021 0.017 0.028" />
@@ -51,6 +44,5 @@
       <!-- thumb pulp side -->
       <collision>
-        <origin xyz="${reflect*0.0315} -0.0085 0.001"
-        rpy="0 0 0" />
+        <origin xyz="${reflect*0.0315} -0.0085 0.001" rpy="0 0 0" />
         <geometry>
           <box size="0.021 0.027 0.024" />

File: sr_description/hand/xacro/thumb/thdistal.urdf.xacro (robot description, xacro)
@@ -8,7 +8,4 @@
   <xacro:include filename="$(find sr_description)/hand/xacro/thumb/thdistal.gazebo.xacro" />
   <xacro:include filename="$(find sr_description)/hand/xacro/thumb/thdistal.transmission.xacro" />
-  <!-- tip_sensor describes the sensor none, bt_2p, bt_sp, eli -->
-  <!-- prefix can be anything but usually is "r_" or  "l_" for right and left hands distinction -->
-  <!-- parent is the parent link for the first joint -->
   <xacro:macro name="thdistal"
     params="tip_sensor:=^|std prefix:=^ parent">

Commit message: Replaced std

File: sr_description/hand/xacro/finger/biotac/biotac.urdf.xacro (robot description, xacro)
@@ -11,5 +11,5 @@
   <!-- joint_prefix prepends fingername to the joint names -->
   <!-- parent is the parent link for the joint -->
-  <xacro:macro name="biotac_middle" params="prefix:=^ link_prefix:=^ joint_prefix:=^ tip_sensor:=^|none mid_sensor:=^|none parent">
+  <xacro:macro name="biotac_middle" params="prefix:=^ link_prefix:=^ joint_prefix:=^ tip_sensor:=^|pst mid_sensor:=^|none parent">
     <link name="${prefix}${link_prefix}middle">
       <inertial>

File: sr_description/hand/xacro/finger/distal/distal.gazebo.xacro (robot description, xacro)
@@ -1,5 +1,5 @@
 <?xml version="1.0"?>
 <robot xmlns:xacro="http://www.ros.org/wiki/xacro">
-  <xacro:macro name="distal_gazebo" params="prefix:=^ link_prefix:=^ tip_sensor:=^|none ns:=^|''">
+  <xacro:macro name="distal_gazebo" params="prefix:=^ link_prefix:=^ tip_sensor:=^|pst ns:=^|''">
     <gazebo reference="${prefix}${link_prefix}distal">
       <xacro:unless value="${'none' in tip_sensor}" >

File: sr_description/hand/xacro/finger/distal/distal.urdf.xacro (robot description, xacro)
@@ -8,10 +8,10 @@
   <xacro:include filename="$(find sr_description)/hand/xacro/finger/distal/distal.gazebo.xacro" />
   <xacro:include filename="$(find sr_description)/hand/xacro/finger/distal/distal.transmission.xacro" />
-  <!-- tip_sensor describes the sensor none, bt_2p, bt_sp, eli -->
+  <!-- tip_sensor describes the sensor bt_2p, bt_sp, pst -->
   <!-- prefix can be anything but usually is "r_" or  "l_" for right and left hands distinction -->
   <!-- link_prefix prepends fingername to the link names -->
   <!-- joint_prefix prepends fingername to the joint names -->
   <!-- parent is the parent link for the joint -->
-  <xacro:macro name="distal" params="prefix:=^ link_prefix:=^ joint_prefix:=^ tip_sensor:=^|std parent">
+  <xacro:macro name="distal" params="prefix:=^ link_prefix:=^ joint_prefix:=^ tip_sensor:=^|pst parent">
     <link name="${prefix}${link_prefix}distal">
       <inertial>

File: sr_description/hand/xacro/finger/fingers.urdf.xacro (robot description, xacro)
@@ -6,5 +6,5 @@
   <xacro:include filename="$(find sr_description)/hand/xacro/finger/lfmetacarpal/lfmetacarpal.urdf.xacro" />
   <xacro:include filename="$(find sr_description)/hand/xacro/finger/biotac/biotac.urdf.xacro" />
-  <xacro:macro name="finger" params="tip_sensor:=^|std mid_sensor:=^|std prox_sensor:=^|std reflect:=^ prefix:=^
+  <xacro:macro name="finger" params="tip_sensor:=^|pst mid_sensor:=^|none prox_sensor:=^|none reflect:=^ prefix:=^
                                      link_prefix joint_prefix parent *origin *axis">
     <!-- Little finger special case -->

File: sr_description/hand/xacro/finger/middle/middle.gazebo.xacro (robot description, xacro)
@@ -1,6 +1,5 @@
 <?xml version="1.0"?>
 <robot xmlns:xacro="http://www.ros.org/wiki/xacro">
-  <xacro:macro name="middle_gazebo" params="prefix:=^ link_prefix:=^ mid_sensor:=^|std">
-    <!-- prefix can be anything but usually is "r_" or  "l_" for right and left hands distinction -->
+  <xacro:macro name="middle_gazebo" params="prefix:=^ link_prefix:=^ mid_sensor:=^|none">
     <gazebo reference="${prefix}${link_prefix}middle">
       <xacro:unless value="${'none' in mid_sensor}">

File: sr_description/hand/xacro/full_hand.urdf.xacro (robot description, xacro)
@@ -10,8 +10,8 @@
   <!-- hand_type can be: E, G, muscle (muscle), muscletrans (muscletrans) -->
   <!-- fingers: list-like string specifying available fingers, default: 'th ff mf rf lf' -->
-  <!-- tip_sensors: plain or dict-like string specifying the fingertip (tactile) sensors: 'th=bt_2p ff=bt_sp mf=eli rf=none, lf=none' -->
+  <!-- tip_sensors: plain or dict-like string specifying the fingertip (tactile) sensors: 'th=bt_2p ff=bt_sp mf=pst rf=pst, lf=pst' -->
   <!-- mid_sensors: plain or dict-like string specifying the middle-phalange (tactile) sensors -->
   <!-- prox_sensors: plain or dict-like string specifying the proximal (tactile) sensors -->
-  <!-- palm_sensor: specifies the palm tactile sensor: std, none -->
+  <!-- palm_sensor: specifies the palm tactile sensor -->
   <!-- reflect is either 1 (for right hand) or -1 (for left hand) -->
   <!-- prefix can be anything but usually is "r_" or  "l_" for right and left hands distinction -->

File: sr_description/hand/xacro/hand_e.urdf.xacro (robot description, xacro)
@@ -6,6 +6,6 @@
   <xacro:include filename="$(find sr_description)/hand/xacro/thumb/thumb.urdf.xacro" />
   <xacro:macro name="sr_hand_e"
-               params="hand_version:=^ reflect:=^ prefix:=^ fingers:=^|all tip_sensors:=^|bt_sp prox_sensors:=^|None
-                      mid_sensors:=^|None palm_sensor:=^|None">
+               params="hand_version:=^ reflect:=^ prefix:=^ fingers:=^|all tip_sensors:=^|bt_sp prox_sensors:=^|none
+                      mid_sensors:=^|none palm_sensor:=^|none">
     <!-- Unify hand type parameter -->
     <xacro:property name="hand_type" value="hand_e" />

File: sr_description/hand/xacro/hand_lite.urdf.xacro (robot description, xacro)
@@ -10,8 +10,8 @@
   <!-- hand_type can be: motor, motor+, muscle (muscle), muscletrans (muscletrans) -->
   <!-- fingers: list-like string specifying available fingers, default: 'th ff mf rf' -->
-  <!-- tip_sensors: plain or dict-like string specifying the fingertip (tactile) sensors: 'th=bt_2p ff=bt_sp mf=eli rf=none, lf=none' -->
+  <!-- tip_sensors: plain or dict-like string specifying the fingertip (tactile) sensors: 'th=bt_2p ff=bt_sp mf=pst rf=pst, lf=pst' -->
   <!-- mid_sensors: plain or dict-like string specifying the middle-phalange (tactile) sensors -->
   <!-- prox_sensors: plain or dict-like string specifying the proximal (tactile) sensors -->
-  <!-- palm_sensor: specifies the palm tactile sensor: none -->
+  <!-- palm_sensor: specifies the palm tactile sensor -->
   <!-- reflect is either 1 (for right hand) or -1 (for left hand) -->
   <!-- prefix can be anything but usually is "r_" or  "l_" for right and left hands distinction -->

File: sr_description/hand/xacro/one_finger_unit.urdf.xacro (robot description, xacro)
@@ -12,6 +12,6 @@
   <!-- bt_sp (deprecated) is true for BT_SP finger or false for standard finger -->
   <!-- eli (deprecated) is true for ellipsoid fingertip or false for standard finger -->
-  <!-- tip_sensor describes the sensor none, bt_2p, bt_sp, eli -->
-  <!-- mid_sensor describes the sensor none, bt_2p -->
+  <!-- tip_sensor describes the sensor bt_2p, bt_sp, pst -->
+  <!-- mid_sensor describes the sensor -->
   <!-- prox_sensor describes the sensor none, bumper -->
   <!-- palm_sensor describes the sensor none, bumper -->
@@ -19,5 +19,5 @@
   <!-- prefix can be anything but usually is "r_" or  "l_" for right and left hands distinction -->
   <xacro:macro name="shadowhand" params="hand_type:='motor' reflect prefix cable_mesh:=False
-          tip_sensor:=std mid_sensor:=std prox_sensor:=std palm_sensor:=std
+          tip_sensor:=pst mid_sensor:=none prox_sensor:=none palm_sensor:=none
           muscletrans:=${None} muscle:=${None} bio:=${None} bt_sp:=${None} eli:=${None}">
     <!-- Unify hand type parameter, also handling deprecated muscletrans, muscle -->

File: sr_description/hand/xacro/palm/palm.gazebo.xacro (robot description, xacro)
@@ -1,5 +1,5 @@
 <?xml version="1.0"?>
 <robot xmlns:xacro="http://www.ros.org/wiki/xacro">
-  <xacro:macro name="shadowhand_palm_gazebo" params="prefix:=^ palm_sensor:=^|std">
+  <xacro:macro name="shadowhand_palm_gazebo" params="prefix:=^ palm_sensor:=^|none">
     <gazebo reference="${prefix}palm">
       <xacro:unless value="${'none' in palm_sensor}" >

File: sr_description/hand/xacro/process_sensor_parameters.xacro (robot description, xacro)
@@ -9,5 +9,5 @@
 	<!---->
 	<!-- Translate deprecated sensor parameters -->
-	<xacro:macro name="translate_from_deprecated" params="name value tip:=${None} mid:=none prox:=none palm:=std">
+	<xacro:macro name="translate_from_deprecated" params="name value tip:=${None} mid:=none prox:=none palm:=none">
 		<xacro:if value="${value}">
 			<xacro:if value="${tip is None}">
@@ -34,7 +34,7 @@
 	<!---->
 	<!-- Transform sensor parameter into proper type -->
-	<xacro:macro name="transform_to_type" params="name value default_tactile_sensor:=^|std
+	<xacro:macro name="transform_to_type" params="name value default_tactile_sensor:=^|none
 				valid_finger_tokens:=^|${'th ff mf rf lf'.split()}
-				valid_sensor_tokens:=^|${'bio bt_sp eli pst std none'.split()}">
+				valid_sensor_tokens:=^|${'bt_2p bt_sp pst none'.split()}">
 		<!-- None acts as marker indicating that we didn't find the correct type specifier yet -->
 		<!-- Finally, _tmp_ should become a list of (finger, sensor) pairs -->
@@ -54,10 +54,10 @@
 			${xacro.warning('Deprecated specifier (dict) used for ' + name + '. Replace with: ' + name + '="' + ' '.join([_fmt_pair_.format(f=k, sensor=v) for k,v in _tmp_]) + '"')}
 		</xacro:if>
-		<!-- Handle dict-like string: 'th=bio, ff=bio, mf=std, rf=std, lf=none' -->
+		<!-- Handle dict-like string: 'th=bio, ff=bio, mf=none, rf=none, lf=none' -->
 		<xacro:if value="${_tmp_ is None and '=' in value}">
 			<!-- Transform into list of finger=sensor pairs -->
 			<xacro:property name="_tmp_" value="${[xacro.tokenize(spec, sep='=') for spec in xacro.tokenize(value)]}" lazy_eval="false" />
 		</xacro:if>
-		<!-- Handle list-like string: 'bio bio std std std' assuming order of valid_finger_tokens -->
+		<!-- Handle list-like string: 'bio bio pst pst pst' assuming order of valid_finger_tokens -->
 		<xacro:if value="${_tmp_ is None and python.any([sep in value for sep in ',; '])}">
 			<xacro:property name="_tmp_" value="${python.zip(valid_finger_tokens, value.split())}" lazy_eval="false" />

File: sr_description/hand/xacro/thumb/thdistal.gazebo.xacro (robot description, xacro)
@@ -1,6 +1,5 @@
 <?xml version="1.0"?>
 <robot xmlns:xacro="http://www.ros.org/wiki/xacro">
-  <xacro:macro name="thdistal_gazebo" params="prefix:=^ tip_sensor:=^|std ns:=^|''">
-    <!-- prefix can be anything but usually is "r_" or  "l_" for right and left hands distinction -->
+  <xacro:macro name="thdistal_gazebo" params="prefix:=^ tip_sensor:=^|pst ns:=^|''">
     <gazebo reference="${prefix}thdistal">
       <xacro:unless value="${'none' in tip_sensor}" >

File: sr_description/hand/xacro/thumb/thdistal.urdf.xacro (robot description, xacro)
@@ -8,6 +8,5 @@
   <xacro:include filename="$(find sr_description)/hand/xacro/thumb/thdistal.gazebo.xacro" />
   <xacro:include filename="$(find sr_description)/hand/xacro/thumb/thdistal.transmission.xacro" />
-  <xacro:macro name="thdistal"
-    params="tip_sensor:=^|std prefix:=^ parent">
+  <xacro:macro name="thdistal" params="tip_sensor:=^|pst prefix:=^ parent">
     <xacro:if value="${tip_sensor == 'bt_2p'}">
       <!--    BIOTAC -->

File: sr_description/hand/xacro/thumb/thmiddle.gazebo.xacro (robot description, xacro)
@@ -1,6 +1,5 @@
 <?xml version="1.0"?>
 <robot xmlns:xacro="http://www.ros.org/wiki/xacro">
-  <xacro:macro name="thmiddle_gazebo" params="prefix:=^ mid_sensor:=^|std">
-    <!-- prefix can be anything but usually is "r_" or  "l_" for right and left hands distinction -->
+  <xacro:macro name="thmiddle_gazebo" params="prefix:=^ mid_sensor:=^|none">
     <gazebo reference="${prefix}thmiddle">
       <xacro:unless value="${'none' in mid_sensor}">

File: sr_description/hand/xacro/thumb/thproximal.gazebo.xacro (robot description, xacro)
@@ -1,5 +1,5 @@
 <?xml version="1.0"?>
 <robot xmlns:xacro="http://www.ros.org/wiki/xacro">
-  <xacro:macro name="thproximal_gazebo" params="prefix:=^ prox_sensor:=^|std">
+  <xacro:macro name="thproximal_gazebo" params="prefix:=^ prox_sensor:=^|none">
     <!-- prefix can be anything but usually is "r_" or  "l_" for right and left hands distinction -->
     <gazebo reference="${prefix}thproximal">

File: sr_description/hand/xacro/thumb/thumb.urdf.xacro (robot description, xacro)
@@ -5,7 +5,7 @@
   <xacro:include filename="$(find sr_description)/hand/xacro/thumb/thmiddle.urdf.xacro" />
   <xacro:include filename="$(find sr_description)/hand/xacro/thumb/thdistal.urdf.xacro" />
-  <!-- tip_sensor describes the sensor none, bt_2p, bt_sp, eli -->
-  <!-- mid_sensor describes the sensor none, bt_2p -->
-  <!-- prox_sensor describes the sensor none, standard -->
+  <!-- tip_sensor describes the sensor -->
+  <!-- mid_sensor describes the sensor -->
+  <!-- prox_sensor describes the sensor -->
   <!-- reflect is either 1 (for right hand) or -1 (for left hand) -->
   <!-- prefix can be anything but usually is "r_" or  "l_" for right and left hands distinction -->
@@ -13,5 +13,5 @@
   <!-- is_lite is this the lite hand, if so lock J3 -->
   <xacro:macro name="thumb"
-  params=" tip_sensor:=^|std mid_sensor:=^|std prox_sensor:=^|std reflect:=^ prefix:=^ parent is_lite">
+  params=" tip_sensor:=^|pst mid_sensor:=^|none prox_sensor:=^|none reflect:=^ prefix:=^ parent is_lite">
     <xacro:if value="${tip_sensor == 'bt_2p'}">
       <xacro:property name="mid_sensor" value="bt_2p" />

File: sr_description/test/test_process_sensor_parameters.xacro (robot description, xacro)
@@ -1,4 +1,4 @@
 <test xmlns:xacro="http://www.ros.org/wiki/xacro">
-	<xacro:macro name="test" params="tip_sensors:=std mid_sensors:=std prox_sensors:=std palm_sensor:=std
+	<xacro:macro name="test" params="tip_sensors:=pst mid_sensors:=none prox_sensors:=none palm_sensor:=none
 	                                 bio:=${None} bt_sp:=${None} eli:=${None}">
 		<xacro:include filename="$(find sr_description)/hand/xacro/process_sensor_parameters.xacro" />
@@ -22,17 +22,17 @@
 		<xacro:test tip_sensors="bio" />
 	</group>
-	<xacro:property name="input" value="bio bio none none none" />
+	<xacro:property name="input" value="bt_2p bt_2p pst pst pst" />
 	<group input="list-like string: ${input}">
 		<xacro:test tip_sensors="${input}" />
 	</group>
-	<xacro:property name="input" value="TH=bio, ff=none, mfx=eli" />
+	<xacro:property name="input" value="TH=bt_2p, ff=pst, mfx=pst" />
 	<group input="dict-like string: ${input}">
 		<xacro:test tip_sensors="${input}" />
 	</group>
-	<xacro:property name="input" value="${['bio', 'eli', 'none']}" />
+	<xacro:property name="input" value="${['bt_2p', 'pst', 'pst']}" />
 	<group input="list: ${input}">
 		<xacro:test tip_sensors="${input}" />
 	</group>
-	<xacro:property name="input" value="${dict(lf='bio', mf='eli', th='none')}" />
+	<xacro:property name="input" value="${dict(lf='bt_2p', mf='pst', th='pst')}" />
 	<group input="dict: ${input}">
 		<xacro:property name="default_sensor" value="none" />
