Commit message: Refactored meshes to use only components

File: sr_description/hand/xacro/finger/knuckle/knuckle.urdf.xacro (robot description, xacro)
@@ -18,5 +18,5 @@
         <origin xyz="0 0 0.0005" rpy="0 0 0" />
         <geometry name="${prefix}${link_prefix}knuckle_visual">
-          <mesh filename="package://sr_description/meshes/products/${hand_type}/${hand_version}/f_knuckle_${hand_version}.dae" scale="0.001 0.001 0.001" />
+          <mesh filename="package://sr_description/meshes/components/f_knuckle/f_knuckle_${hand_version}.dae" scale="0.001 0.001 0.001" />
         </geometry>
         <material name="LightGrey" />

File: sr_description/hand/xacro/finger/lfmetacarpal/lfmetacarpal.urdf.xacro (robot description, xacro)
@@ -23,5 +23,5 @@
         <origin xyz="0 0 0" rpy="0 0 0" />
         <geometry name="${prefix}lfmetacarpal_visual">
-          <mesh filename="package://sr_description/meshes/products/${hand_type}/${hand_version}/lf_metacarpal_${hand_version}.dae"
+          <mesh filename="package://sr_description/meshes/components/lf_metacarpal/lf_metacarpal_${hand_version}.dae"
           scale="${reflect*0.001} 0.001 0.001" />
         </geometry>

File: sr_description/hand/xacro/finger/middle/middle.urdf.xacro (robot description, xacro)
@@ -18,5 +18,5 @@
         <origin xyz="0 0 0" rpy="0 0 0" />
         <geometry name="${prefix}${link_prefix}middle_visual">
-          <mesh filename="package://sr_description/meshes/products/${hand_type}/${hand_version}/f_middle_${hand_version}.dae"
+          <mesh filename="package://sr_description/meshes/components/f_middle/f_middle_${hand_version}.dae"
                 scale="0.001 0.001 0.001" />
         </geometry>

File: sr_description/hand/xacro/finger/proximal/proximal.urdf.xacro (robot description, xacro)
@@ -18,5 +18,5 @@
         <origin xyz="0 0 0" rpy="0 0 0" />
         <geometry name="${prefix}${link_prefix}proximal_visual">
-          <mesh filename="package://sr_description/meshes/products/${hand_type}/${hand_version}/f_proximal_${hand_version}.dae"
+          <mesh filename="package://sr_description/meshes/components/f_proximal/f_proximal_${hand_version}.dae"
                 scale="0.001 0.001 0.001" />
         </geometry>

File: sr_description/hand/xacro/forearm/forearm_c.urdf.xacro (robot description, xacro)
@@ -21,5 +21,5 @@
         <origin xyz="0 0 0" rpy="0 0 0" />
         <geometry name="${prefix}forearm_visual">
-          <mesh filename="package://sr_description/meshes/products/${hand_type}/${hand_version}/forearm_${hand_version}.dae"/>
+          <mesh filename="package://sr_description/meshes/components/forearm/forearm_${hand_version}.dae"/>
         </geometry>
         <material name="Grey" />

File: sr_description/hand/xacro/forearm/forearm_e.urdf.xacro (robot description, xacro)
@@ -21,5 +21,5 @@
         <origin xyz="0 0 0" rpy="0 0 0" />
         <geometry name="${prefix}forearm_visual">
-          <mesh filename="package://sr_description/meshes/products/${hand_type}/${hand_version}/forearm_${hand_version}.dae" scale="0.001 0.001 0.001" />
+          <mesh filename="package://sr_description/meshes/components/forearm/forearm_${hand_version}.dae" scale="0.001 0.001 0.001" />
         </geometry>
         <xacro:light_grey/>
@@ -28,5 +28,5 @@
         <origin xyz="0 0 0" rpy="0 0 0" />
         <geometry name="${prefix}forearm_collision">
-          <mesh filename="package://sr_description/meshes/products/${hand_type}/${hand_version}/forearm_collision_${hand_version}.stl" scale="0.001 0.001 0.001" />
+          <mesh filename="package://sr_description/meshes/components/forearm/forearm_collision_${hand_version}.stl" scale="0.001 0.001 0.001" />
         </geometry>
       </collision>
@@ -42,5 +42,5 @@
         <origin rpy="0 -1.57 -1.57" xyz="0.0 0.067 0.0045"/>
         <geometry name="${prefix}cable_extr_visualisation">
-          <mesh filename="package://sr_description/meshes/products/${hand_type}/${hand_version}/cable_connector_base_${hand_version}.stl" scale="1 1 1" />
+          <mesh filename="package://sr_description/meshes/components/cable_connector/cable_connector_base_${hand_version}.stl" scale="0.001 0.001 0.001" />
         </geometry>
       </visual>
@@ -48,5 +48,5 @@
         <origin rpy="0 -1.57 -1.57" xyz="0.0 0.067 0.0045"/>
         <geometry name="${prefix}cable_extr_collision">
-          <mesh filename="package://sr_description/meshes/products/${hand_type}/${hand_version}/cable_connector_base_${hand_version}.stl" scale="1 1 1" />
+          <mesh filename="package://sr_description/meshes/components/cable_connector/cable_connector_base_${hand_version}.stl" scale="0.001 0.001 0.001" />
         </geometry>
       </collision-->

File: sr_description/hand/xacro/forearm/forearm_g.urdf.xacro (robot description, xacro)
@@ -12,5 +12,5 @@
         <origin xyz="0 0 0" rpy="0 0 ${pi/2}" />
         <geometry name="${prefix}forearm_visual">
-          <mesh filename="package://sr_description/meshes/products/${hand_type}/${hand_version}/forearm_${hand_version}.dae" scale="1.0 1.0 1.0" />
+          <mesh filename="package://sr_description/meshes/components/forearm/forearm_${hand_version}.dae" scale="1.0 1.0 1.0" />
         </geometry>
         <material name="Grey" />
@@ -26,5 +26,5 @@
         <origin rpy="0 -1.57 -1.57" xyz="0.0 0.055 0.0"/>
         <geometry name="${prefix}cable_extr_visualisation">
-          <mesh filename="package://sr_description/meshes/products/${hand_type}/${hand_version}/cable_connector_base_${hand_version}.stl" scale="1 1 1" />
+          <mesh filename="package://sr_description/meshes/components/cable_connector/cable_connector_base_${hand_version}.stl" scale="1 1 1" />
         </geometry>
       </visual>
@@ -32,5 +32,5 @@
         <origin rpy="0 -1.57 -1.57" xyz="0.0 0.055 0.0"/>
         <geometry name="${prefix}cable_extr_collision">
-          <mesh filename="package://sr_description/meshes/products/${hand_type}/${hand_version}/cable_connector_base_${hand_version}.stl" scale="1 1 1" />
+          <mesh filename="package://sr_description/components/cable_connector/cable_connector_base_${hand_version}.stl" scale="1 1 1" />
         </geometry>
       </collision-->

File: sr_description/hand/xacro/palm/palm_e.urdf.xacro (robot description, xacro)
@@ -19,5 +19,5 @@
         <origin xyz="0 0 0" rpy="0 0 0" />
         <geometry name="${prefix}palm_visual">
-          <mesh filename="package://sr_description/meshes/products/${hand_type}/${hand_version}/palm_${hand_version}.stl"
+          <mesh filename="package://sr_description/meshes/components/palm/palm_${hand_version}.stl"
                 scale="${reflect*0.001} 0.001 0.001" />
         </geometry>

File: sr_description/hand/xacro/palm/palm_g.urdf.xacro (robot description, xacro)
@@ -18,5 +18,5 @@
         <origin xyz="0 0 0" rpy="0 0 0" />
         <geometry name="${prefix}palm_visual">
-          <mesh filename="package://sr_description/meshes/products/${hand_type}/${hand_version}/palm_${hand_version}.dae"
+          <mesh filename="package://sr_description/meshes/components/palm/palm_${hand_version}.dae"
           scale="${reflect*0.001} 0.001 0.001" />
         </geometry>

File: sr_description/hand/xacro/thumb/thmiddle.urdf.xacro (robot description, xacro)
@@ -27,5 +27,5 @@
         <xacro:unless value="${mid_sensor == 'bt_2p'}">
           <geometry name="${prefix}thmiddle_visual">
-            <mesh filename="package://sr_description/meshes/products/${hand_type}/${hand_version}/th_middle_${hand_version}.dae"
+            <mesh filename="package://sr_description/meshes/components/th_middle/th_middle_${hand_version}.dae"
             scale="0.001 0.001 0.001" />
           </geometry>

File: sr_description/hand/xacro/thumb/thproximal.urdf.xacro (robot description, xacro)
@@ -18,5 +18,5 @@
         <origin xyz="0 0 0" rpy="0 0 0" />
         <geometry name="${prefix}thproximal_visual">
-          <mesh filename="package://sr_description/meshes/products/${hand_type}/${hand_version}/th_proximal_${hand_version}.dae"
+          <mesh filename="package://sr_description/meshes/components/th_proximal/th_proximal_${hand_version}.dae"
           scale="0.001 0.001 0.001" />
         </geometry>

File: sr_description/hand/xacro/wrist/wrist.urdf.xacro (robot description, xacro)
@@ -11,5 +11,5 @@
         <origin xyz="0 0 0" rpy="0 0 0" />
         <geometry name="${prefix}wrist_visual">
-          <mesh filename="package://sr_description/meshes/products/${hand_type}/${hand_version}/wrist_${hand_version}.dae"
+          <mesh filename="package://sr_description/meshes/components/wrist/wrist_${hand_version}.dae"
           scale="${reflect*0.001} 0.001 0.001" />
         </geometry>
