Commit message: Applying changes from https://github.com/ubi-agni/sr_common/pull/2

File: sr_description/hand/xacro/finger/knuckle/knuckle.gazebo.xacro (robot description, xacro)
@@ -3,18 +3,5 @@
   <xacro:macro name="knuckle_gazebo" params="prefix:=^ link_prefix:=^">
     <gazebo reference="${prefix}${link_prefix}knuckle">
-      <sensor type="contact" name="${prefix}${link_prefix}knuckle_contact">
-        <always_on>1</always_on>
-        <update_rate>1000.0</update_rate>
-        <contact>
-          <collision>${prefix}${link_prefix}knuckle_collision</collision>
-          <topic>${prefix}${link_prefix}knuckle_collision</topic>
-        </contact>
-        <plugin name="${prefix}${link_prefix}knuckle_gazebo_ros_bumper_controller" filename="libgazebo_ros_bumper.so">
-          <alwaysOn>true</alwaysOn>
-          <frameName>${prefix}${link_prefix}knuckle</frameName>
-          <updateRate>100.0</updateRate>
-          <bumperTopicName>contacts/${prefix}${link_prefix}/knuckle</bumperTopicName>
-        </plugin>
-      </sensor>
+      <!-- knuckle is not highly exposed, so bumper is not useful -->
       <material>Gazebo/Grey</material>
     </gazebo>

File: sr_description/hand/xacro/hand.urdf.xacro (robot description, xacro)
@@ -5,4 +5,5 @@
   <xacro:macro name="sr_hand"
                params="hand_type hand_version side fingers tip_sensors prox_sensors mid_sensors palm_sensor">
+  <xacro:include filename="$(find sr_description)/hand/xacro/validate_xacro.xacro" />
     <xacro:if value="${side == 'right'}">
       <xacro:property name="reflect" value="1" />

File: sr_description/hand/xacro/thumb/thbase.gazebo.xacro (robot description, xacro)
@@ -3,18 +3,5 @@
   <xacro:macro name="thbase_gazebo" params="prefix:=^">
     <gazebo reference="${prefix}thbase">
-      <sensor type="contact" name="${prefix}thbase_contact">
-        <always_on>1</always_on>
-        <update_rate>1000.0</update_rate>
-        <contact>
-          <collision>${prefix}thbase_collision</collision>
-          <topic>${prefix}thbase_collision</topic>
-        </contact>
-        <plugin name="${prefix}thbase_gazebo_ros_bumper_controller" filename="libgazebo_ros_bumper.so">
-          <alwaysOn>true</alwaysOn>
-          <frameName>${prefix}thbase</frameName>
-          <updateRate>100.0</updateRate>
-          <bumperTopicName>contacts/${prefix}th/base</bumperTopicName>
-        </plugin>
-      </sensor>
+      <!-- base is inside the proximal and not exposed, so bumper is not needed -->
       <selfCollide>false</selfCollide>
     </gazebo>

File: sr_description/hand/xacro/thumb/thhub.gazebo.xacro (robot description, xacro)
@@ -3,19 +3,6 @@
   <xacro:macro name="thhub_gazebo" params="prefix:=^">
     <gazebo reference="${prefix}thhub">
-      <sensor type="contact" name="${prefix}thhub_contact">
-        <always_on>1</always_on>
-        <update_rate>1000.0</update_rate>
-        <contact>
-          <collision>${prefix}thhub_collision</collision>
-          <topic>${prefix}thhub_collision</topic>
-        </contact>
-        <plugin name="${prefix}thhub_gazebo_ros_bumper_controller" filename="libgazebo_ros_bumper.so">
-          <alwaysOn>true</alwaysOn>
-          <frameName>${prefix}thhub</frameName>
-          <updateRate>100.0</updateRate>
-          <bumperTopicName>contacts/${prefix}th/hub</bumperTopicName>
-        </plugin>
-      </sensor>
-      <selfCollide>true</selfCollide>
+      <!-- hub is inside the proximal and not exposed, so bumper is not needed -->
+      <selfCollide>false</selfCollide>
     </gazebo>
   </xacro:macro>
