Commit message: Update thhub.urdf.xacro

File: sr_description/hand/xacro/thumb/thhub.urdf.xacro (robot description, xacro)
@@ -44,5 +44,5 @@
         <child link="${prefix}thhub" />
         <origin xyz="0 0 0.038" rpy="0 0 0" />
-        <axis xyz="1 0 0" />
+        <axis xyz="${reflect} 0 0" />
         <limit lower="${-12/180*pi}" upper="${12/180*pi}" effort="2.0" velocity="4.0" />
         <dynamics damping="0.2" />
