Commit message: Update sr_description/hand/xacro/thumb/thdistal.urdf.xacro
Co-Authored-By: Beatriz Leon <beatriz@shadowrobot.com>

File: sr_description/hand/xacro/thumb/thdistal.urdf.xacro (robot description, xacro)
@@ -192,5 +192,5 @@
         <origin xyz="0 0 0.032" rpy="0 0 ${-M_PI/2}" />
         <axis xyz="1 0 0" />
-        <limit lower="-0.2618" upper="${90.0*M_PI/180}" effort="1.0"
+        <limit lower="-"${15.0*M_PI/180}"" upper="${90.0*M_PI/180}" effort="1.0"
         velocity="4.0" />
         <dynamics damping="0.2" />

Commit message: Update thdistal.urdf.xacro

File: sr_description/hand/xacro/thumb/thdistal.urdf.xacro (robot description, xacro)
@@ -192,5 +192,5 @@
         <origin xyz="0 0 0.032" rpy="0 0 ${-M_PI/2}" />
         <axis xyz="1 0 0" />
-        <limit lower="-"${15.0*M_PI/180}"" upper="${90.0*M_PI/180}" effort="1.0"
+        <limit lower="-${15.0*M_PI/180}"" upper="${90.0*M_PI/180}" effort="1.0"
         velocity="4.0" />
         <dynamics damping="0.2" />

Commit message: Update thdistal.urdf.xacro

File: sr_description/hand/xacro/thumb/thdistal.urdf.xacro (robot description, xacro)
@@ -192,5 +192,5 @@
         <origin xyz="0 0 0.032" rpy="0 0 ${-M_PI/2}" />
         <axis xyz="1 0 0" />
-        <limit lower="-${15.0*M_PI/180}"" upper="${90.0*M_PI/180}" effort="1.0"
+        <limit lower="-${15.0*M_PI/180}" upper="${90.0*M_PI/180}" effort="1.0"
         velocity="4.0" />
         <dynamics damping="0.2" />

Commit message: Adding thumb distal mst

File: sr_description/hand/xacro/thumb/thdistal.urdf.xacro (robot description, xacro)
@@ -133,4 +133,8 @@
                     scale="0.001 0.001 0.001" />
             </xacro:if>
+            <xacro:if value="${tip_sensor == 'mst'}">
+              <mesh filename="package://sr_description/meshes/components/th_distal/mst/th_distal_mst.dae"
+                    scale="0.001 0.001 0.001" />
+            </xacro:if>
             <xacro:if value="${tip_sensor == 'bt_sp'}">
               <mesh filename="package://sr_description/meshes/components/th_distal/bt_sp/th_distal_bt_sp.dae"
@@ -151,4 +155,8 @@
             <xacro:if value="${tip_sensor == 'pst'}">
               <mesh filename="package://sr_description/meshes/components/th_distal/pst/th_distal_pst.dae"
+                    scale="0.001 0.001 0.001" />
+            </xacro:if>
+            <xacro:if value="${tip_sensor == 'mst'}">
+              <mesh filename="package://sr_description/meshes/components/th_distal/mst/th_distal_mst.dae"
                     scale="0.001 0.001 0.001" />
             </xacro:if>

Commit message: Deleted thumb distal material
The specification of the BiotacGreen material in the thumb distal caused
a warning, that the material was undefined. Since the appearance of the
thumb didn't change without it, I assume that this is an unused line of
code and I deleted it.

File: sr_description/hand/xacro/thumb/thdistal.urdf.xacro (robot description, xacro)
@@ -68,5 +68,4 @@
             scale="0.0254 0.0254 0.0254" />
           </geometry>
-          <material name="BiotacGreen" />
         </visual>
         <collision>

Commit message: Hand model bug fix when using Biotac SP + (version 2) tactile sensors (#161)
* Removing unnecessary rotation on the last thumb link. Correctly alligning thumb meshes with respective thumb links

* Remove changes related to innertia

* Update licences years

File: sr_description/hand/xacro/thumb/thdistal.urdf.xacro (robot description, xacro)
@@ -2,5 +2,5 @@
 <!--
  Software License Agreement (BSD License)
- Copyright © 2022 belongs to Shadow Robot Company Ltd.
+ Copyright © 2022, 2023 belongs to Shadow Robot Company Ltd.
  All rights reserved.
  Redistribution and use in source and binary forms, with or without modification,
@@ -46,5 +46,5 @@
         <parent link="${parent}" />
         <child link="${prefix}thdistal_J1_dummy" />
-        <origin xyz="0 0 0.02" rpy="0 0 ${-pi/2}" />
+        <origin xyz="0 0 0.02" rpy="0 0 0" />
         <axis xyz="1 0 0" />
         <limit lower="${20*pi/180}" upper="${20.1*pi/180}" effort="0.0" velocity="2.0" />
@@ -97,5 +97,5 @@
         <parent link="${prefix}thmiddle" />
         <child link="${prefix}thdistal" />
-        <origin xyz="0 0.0 0.01" rpy="0 0 ${-pi/2}" />
+        <origin xyz="0 0.0 0.01" rpy="0 0 0" />
       </joint>
       <!-- extra link to imaginary sphere in fingertip for FK/IK calculations -->

File: sr_description/hand/xacro/thumb/thproximal.urdf.xacro (robot description, xacro)
@@ -2,5 +2,5 @@
 <!--
  Software License Agreement (BSD License)
- Copyright © 2022 belongs to Shadow Robot Company Ltd.
+ Copyright © 2022, 2023 belongs to Shadow Robot Company Ltd.
  All rights reserved.
  Redistribution and use in source and binary forms, with or without modification,
@@ -41,5 +41,5 @@
       </inertial>
       <visual>
-        <origin xyz="0 0 0" rpy="0 0 0" />
+        <origin xyz="0 0 0" rpy="0 0 ${pi/2}" />
         <geometry name="${prefix}thproximal_visual">
           <mesh filename="package://sr_description/meshes/components/th_proximal/th_proximal_${hand_version}.dae"
