Commit message: Fixed finger

File: sr_description/hand/xacro/finger/fingers.urdf.xacro (robot description, xacro)
@@ -5,6 +5,6 @@
   <xacro:include filename="$(find sr_description)/hand/xacro/finger/distal/distal.urdf.xacro" />
   <xacro:include filename="$(find sr_description)/hand/xacro/finger/lfmetacarpal/lfmetacarpal.urdf.xacro" />
-  <xacro:include filename="$(find sr_description)/hand/xacro/finger/biotac/biotac.urdf.xacro" />
-  <xacro:macro name="finger" params="tip_sensor:=^|pst mid_sensor:=^|none prox_sensor:=^|none reflect:=^ prefix:=^
+  <xacro:include filename="$(find sr_description)/hand/xacro/finger/middle/middle_and_distal_bt_2p.urdf.xacro" />
+  <xacro:macro name="finger" params="hand_type:=^ hand_version:=^ tip_sensor:=^|pst mid_sensor:=^|none prox_sensor:=^|none reflect:=^ prefix:=^
                                      link_prefix joint_prefix parent *origin *axis">
     <!-- Little finger special case -->
@@ -12,5 +12,5 @@
       <xacro:lfmetacarpal parent="${parent}" />
       <!-- Knuckle -->
-      <xacro:knuckle parent="${prefix}lfmetacarpal">
+      <xacro:knuckle hand_type="${hand_type}" hand_version="${hand_version}" parent="${prefix}lfmetacarpal">
         <xacro:insert_block name="origin" />
       </xacro:knuckle>
@@ -19,21 +19,20 @@
     <xacro:unless value="${link_prefix == 'lf'}">
       <!-- Knuckle -->
-      <xacro:knuckle parent="${parent}">
+      <xacro:knuckle hand_type="${hand_type}" hand_version="${hand_version}" parent="${parent}">
         <xacro:insert_block name="origin" />
       </xacro:knuckle>
     </xacro:unless>
     <!-- Proximal -->
-    <xacro:proximal parent="${prefix}${link_prefix}knuckle"></xacro:proximal>
+    <xacro:proximal hand_type="${hand_type}" hand_version="${hand_version}" parent="${prefix}${link_prefix}knuckle"/>
     <!-- BioTac combines Middle + Distal -->
     <xacro:if value="${tip_sensor == 'bt_2p'}">
-      <xacro:biotac_middle parent="${prefix}${link_prefix}proximal">
-      </xacro:biotac_middle>
+      <xacro:middle_and_distal_bt_2p hand_type="${hand_type}" hand_version="${hand_version}" parent="${prefix}${link_prefix}proximal"/>
     </xacro:if>
     <!-- Non-BioTac -->
     <xacro:unless value="${tip_sensor == 'bt_2p'}">
       <!-- Middle -->
-      <xacro:middle parent="${prefix}${link_prefix}proximal"></xacro:middle>
+      <xacro:middle hand_type="${hand_type}" hand_version="${hand_version}" parent="${prefix}${link_prefix}proximal"/>
       <!-- Distal  -->
-      <xacro:distal parent="${prefix}${link_prefix}middle"></xacro:distal>
+      <xacro:distal parent="${prefix}${link_prefix}middle"/>
     </xacro:unless>
   </xacro:macro>

File: sr_description/hand/xacro/finger/knuckle/knuckle.urdf.xacro (robot description, xacro)
@@ -8,5 +8,5 @@
   <xacro:include filename="$(find sr_description)/hand/xacro/finger/knuckle/knuckle.gazebo.xacro" />
   <xacro:include filename="$(find sr_description)/hand/xacro/finger/knuckle/knuckle.transmission.xacro" />
-  <xacro:macro name="knuckle" params="prefix:=^ link_prefix:=^ joint_prefix:=^ parent *origin">
+  <xacro:macro name="knuckle" params="hand_type:=^ hand_version:=^ prefix:=^ link_prefix:=^ joint_prefix:=^ parent *origin">
     <link name="${prefix}${link_prefix}knuckle">
       <inertial>
@@ -18,5 +18,5 @@
         <origin xyz="0 0 0.0005" rpy="0 0 0" />
         <geometry name="${prefix}${link_prefix}knuckle_visual">
-          <mesh filename="package://sr_description/meshes/hand/knuckle.dae" scale="0.001 0.001 0.001" />
+          <mesh filename="package://sr_description/meshes/products/${hand_type}/${hand_version}/f_knuckle_${hand_version}.dae" scale="0.001 0.001 0.001" />
         </geometry>
         <material name="LightGrey" />

File: sr_description/hand/xacro/finger/lfmetacarpal/lfmetacarpal.urdf.xacro (robot description, xacro)
@@ -23,5 +23,5 @@
         <origin xyz="0 0 0" rpy="0 0 0" />
         <geometry name="${prefix}lfmetacarpal_visual">
-          <mesh filename="package://sr_description/meshes/hand/lfmetacarpal.dae"
+          <mesh filename="package://sr_description/meshes/products/${hand_type}/${hand_version}/lf_metacarpal_${hand_version}.dae"
           scale="${reflect*0.001} 0.001 0.001" />
         </geometry>

File: sr_description/hand/xacro/finger/middle/middle_and_distal_bt_2p.urdf.xacro (robot description, xacro)
@@ -7,9 +7,5 @@
        xmlns:geom="http://playerstage.sourceforge.net/gazebo/xmlschema/#geom">
   <xacro:include filename="$(find sr_description)/hand/xacro/finger/middle/middle.transmission.xacro" />
-  <!-- prefix can be anything but usually is "r_" or  "l_" for right and left hands distinction -->
-  <!-- link_prefix prepends fingername to the link names -->
-  <!-- joint_prefix prepends fingername to the joint names -->
-  <!-- parent is the parent link for the joint -->
-  <xacro:macro name="biotac_middle" params="prefix:=^ link_prefix:=^ joint_prefix:=^ tip_sensor:=^|pst mid_sensor:=^|none parent">
+  <xacro:macro name="middle_and_distal_bt_2p" params="hand_type:=^ hand_version:=^ prefix:=^ link_prefix:=^ joint_prefix:=^ tip_sensor:=^|pst mid_sensor:=^|none parent">
     <link name="${prefix}${link_prefix}middle">
       <inertial>
@@ -21,5 +17,5 @@
         <origin xyz="0 0 0" rpy="0 0 1.571" />
         <geometry name="${prefix}${link_prefix}middle_visual">
-          <mesh filename="package://sr_description/meshes/hand/biotacs/biotac_finger_adapter.dae" scale="1 1 1" />
+          <mesh filename="package://sr_description/meshes/components/f_distal/bt_2p/f_distal_bt_2p_adapter.dae" />
         </geometry>
         <material name="LightGrey" />
@@ -92,12 +88,12 @@
         <origin xyz="0 0 0" rpy="0 0 0" />
         <geometry name="${prefix}${link_prefix}distal_visual">
-          <!-- <mesh filename="package://sr_description/meshes/hand/biotacs/biotac.stl" scale="0.0254 0.0254 0.0254" /> -->
-          <mesh filename="package://sr_description/meshes/hand/biotacs/biotac_decimated.dae" scale="0.0254 0.0254 0.0254" />
+          <mesh filename="package://sr_description/meshes/components/f_distal/bt_2p/f_distal_bt_2p.dae"
+                scale="0.0254 0.0254 0.0254" />
         </geometry>
       </visual>
       <collision>
         <geometry name="${prefix}${link_prefix}distal_collision_geom">
-          <!-- <mesh filename="package://sr_description/meshes/hand/biotacs/biotac.stl" scale="0.0254 0.0254 0.0254" /> -->
-          <mesh filename="package://sr_description/meshes/hand/biotacs/biotac_decimated.dae" scale="0.0254 0.0254 0.0254" />
+          <mesh filename="package://sr_description/meshes/components/f_distal/bt_2p/f_distal_bt_2p.dae"
+                scale="0.0254 0.0254 0.0254" />
         </geometry>
       </collision>

File: sr_description/hand/xacro/finger/proximal/proximal.urdf.xacro (robot description, xacro)
@@ -8,22 +8,16 @@
   <xacro:include filename="$(find sr_description)/hand/xacro/finger/proximal/proximal.gazebo.xacro" />
   <xacro:include filename="$(find sr_description)/hand/xacro/finger/proximal/proximal.transmission.xacro" />
-  <!-- prefix can be anything but usually is "r_" or  "l_" for right and left hands distinction -->
-  <!-- link_prefix prepends fingername to the link names -->
-  <!-- joint_prefix prepends fingername to the joint names -->
-  <!-- parent is the parent link for the joint -->
-  <xacro:macro name="proximal"
-  params="prefix:=^ link_prefix:=^ joint_prefix:=^ parent">
+  <xacro:macro name="proximal" params="hand_type:=^ hand_version:=^ prefix:=^ link_prefix:=^ joint_prefix:=^ parent">
     <link name="${prefix}${link_prefix}proximal">
       <inertial>
         <mass value="0.030" />
         <origin xyz="0 0 0.0225" />
-        <inertia ixx="0.0000098" ixy="0.0" ixz="0.0" iyy="0.00001"
-        iyz="0.0" izz="0.0000018" />
+        <inertia ixx="0.0000098" ixy="0.0" ixz="0.0" iyy="0.00001" iyz="0.0" izz="0.0000018" />
       </inertial>
       <visual>
         <origin xyz="0 0 0" rpy="0 0 0" />
         <geometry name="${prefix}${link_prefix}proximal_visual">
-          <mesh filename="package://sr_description/meshes/hand/F3.dae"
-          scale="0.001 0.001 0.001" />
+          <mesh filename="package://sr_description/meshes/products/${hand_type}/${hand_version}/f_proximal_${hand_version}.dae"
+                scale="0.001 0.001 0.001" />
         </geometry>
         <material name="Grey" />
@@ -41,6 +35,5 @@
       <origin xyz="0 0 0" rpy="0 0 0" />
       <axis xyz="1 0 0" />
-      <limit lower="-${15.0*pi/180}" upper="${pi/2}" effort="2"
-      velocity="2.0" />
+      <limit lower="-${15.0*pi/180}" upper="${pi/2}" effort="2" velocity="2.0" />
       <dynamics damping="0.1" />
     </joint>

Commit message: Changing THJ5,4,3,2,1 and LFJ5,4 link origin/axis to conform with remaining fingers convention (with regards to Flex/Ext, Add/Abd joint motions)

File: sr_description/hand/xacro/finger/fingers.urdf.xacro (robot description, xacro)
@@ -13,5 +13,5 @@
       <!-- Knuckle -->
       <xacro:knuckle hand_type="${hand_type}" hand_version="${hand_version}" parent="${prefix}lfmetacarpal">
-        <xacro:insert_block name="origin" />
+        <origin xyz="${reflect*0.05389084} 0 0.03773727" rpy="0 ${reflect*0.9599} 0" />
       </xacro:knuckle>
     </xacro:if>

File: sr_description/hand/xacro/finger/lfmetacarpal/lfmetacarpal.urdf.xacro (robot description, xacro)
@@ -16,5 +16,6 @@
       </inertial>
       <visual>
-        <origin xyz="0 0 0" rpy="0 0 0" />
+        <origin xyz="0 0 0" rpy="0 ${reflect*0.9599} 0" />
+        <axis xyz="0.573576436 0 ${reflect*0.819152044}" />
         <geometry name="${prefix}lfmetacarpal_visual">
           <mesh filename="package://sr_description/meshes/components/lf_metacarpal/lf_metacarpal_${hand_version}.dae"
@@ -33,6 +34,6 @@
       <parent link="${parent}" />
       <child link="${prefix}lfmetacarpal" />
-      <origin xyz="${reflect*-0.033} 0 0.02071" rpy="0 0 0" />
-      <axis xyz="0.573576436 0 ${reflect*0.819152044}" />
+      <origin xyz="${reflect*-0.033} 0 0.02071" rpy="0 ${reflect*-0.9599} 0" />
+      <axis xyz="1 0 0" />
       <limit lower="0" upper="${45/180*pi}" effort="2" velocity="2.0" />
       <dynamics damping="0.1" />

File: sr_description/hand/xacro/thumb/thbase.urdf.xacro (robot description, xacro)
@@ -34,5 +34,5 @@
       <parent link="${parent}" />
       <child link="${prefix}thbase" />
-      <origin xyz="${reflect*0.034} -0.00858 0.029" rpy="0 ${pi/4} ${pi/2-reflect*pi/2}" />
+      <origin xyz="${reflect*0.034} -0.00858 0.029" rpy="${-pi/4} 0 ${-reflect*pi/2}" />
       <axis xyz="0 0 ${reflect*-1}" />
       <limit lower="${-60/180*pi}" upper="${60/180*pi}" effort="5.0" velocity="4.0" />

File: sr_description/hand/xacro/thumb/thdistal.urdf.xacro (robot description, xacro)
@@ -142,5 +142,5 @@
         <parent link="${parent}" />
         <child link="${prefix}thdistal" />
-        <origin xyz="0 0 0.032" rpy="0 0 ${-pi/2}" />
+        <origin xyz="0 0 0.032" rpy="0 0 0" />
         <axis xyz="1 0 0" />
         <limit lower="-${15.0*pi/180}" upper="${90.0*pi/180}" effort="1.0" velocity="4.0" />

File: sr_description/hand/xacro/thumb/thhub.urdf.xacro (robot description, xacro)
@@ -44,5 +44,5 @@
         <child link="${prefix}thhub" />
         <origin xyz="0 0 0.038" rpy="0 0 0" />
-        <axis xyz="${reflect} 0 0" />
+        <axis xyz="0 ${reflect} 0" />
         <limit lower="${-12/180*pi}" upper="${12/180*pi}" effort="2.0" velocity="4.0" />
         <dynamics damping="0.2" />

File: sr_description/hand/xacro/thumb/thmiddle.urdf.xacro (robot description, xacro)
@@ -67,5 +67,5 @@
         <origin xyz="0 0 0" rpy="0 0 0" />
       </xacro:unless>
-      <axis xyz="0 -1 0" />
+      <axis xyz="1 0 0" />
       <limit lower="${-40/180*pi}" upper="${40/180*pi}" effort="2.0" velocity="2.0" />
       <dynamics damping="0.1" />

File: sr_description/hand/xacro/thumb/thproximal.urdf.xacro (robot description, xacro)
@@ -36,5 +36,5 @@
       <child link="${prefix}thproximal" />
       <origin xyz="0 0 0" rpy="0 0 0" />
-      <axis xyz="${reflect} 0 0" />
+      <axis xyz="0 ${reflect} 0" />
       <limit lower="0.0" upper="${70/180*pi}" effort="3" velocity="4.0" />
       <dynamics damping="0.2" />

Commit message: Provide lfknuckle pose in hand_e/hand_c xacro files instead of fingers file, to keep comsistency

File: sr_description/hand/xacro/finger/fingers.urdf.xacro (robot description, xacro)
@@ -38,5 +38,5 @@
       <!-- Knuckle -->
       <xacro:knuckle hand_type="${hand_type}" hand_version="${hand_version}" parent="${prefix}lfmetacarpal">
-        <origin xyz="${reflect*0.05389084} 0 0.03773727" rpy="0 ${reflect*0.9599} 0" />
+        <xacro:insert_block name="origin" />
       </xacro:knuckle>
     </xacro:if>

File: sr_description/hand/xacro/hand_e.urdf.xacro (robot description, xacro)
@@ -80,5 +80,5 @@
       <xacro:finger link_prefix="lf" joint_prefix="LF" tip_sensor="${tip_sensors.lf}" prox_sensor="${prox_sensors.lf}"
                     mid_sensor="${mid_sensors.lf}" parent="${prefix}palm">
-        <origin xyz="0 0 0.06579" rpy="0 0 0" />
+        <origin xyz="${reflect*0.05389084} 0 0.03773727" rpy="0 ${reflect*0.9599} 0" />
         <axis xyz="0 ${reflect} 0" />
       </xacro:finger>
