Commit message: Sp 399 fixing hand e urdf convention (#144)
* Update thhub.urdf.xacro to fix the wrong axis on THJ3 of the Left Hand (#141)

* Changed linter branch from master to lint (#139)

* Update thhub.urdf.xacro

* Update aws.yml

Co-authored-by: maxzieba <77073326+maxzieba@users.noreply.github.com>

* Changing THJ5,4,3,2,1 and LFJ5,4 link origin/axis to conform with remaining fingers convention (with regards to Flex/Ext, Add/Abd joint motions)

* Provide lfknuckle pose in hand_e/hand_c xacro files instead of fingers file, to keep comsistency

* Forgot to add changes to hand_c urdf file

* Remove empty space

Co-authored-by: Beatriz Leon <beatriz@shadowrobot.com>
Co-authored-by: maxzieba <77073326+maxzieba@users.noreply.github.com>

File: sr_description/hand/xacro/finger/lfmetacarpal/lfmetacarpal.urdf.xacro (robot description, xacro)
@@ -41,5 +41,6 @@
       </inertial>
       <visual>
-        <origin xyz="0 0 0" rpy="0 0 0" />
+        <origin xyz="0 0 0" rpy="0 ${reflect*0.9599} 0" />
+        <axis xyz="0.573576436 0 ${reflect*0.819152044}" />
         <geometry name="${prefix}lfmetacarpal_visual">
           <mesh filename="package://sr_description/meshes/components/lf_metacarpal/lf_metacarpal_${hand_version}.dae"
@@ -58,6 +59,6 @@
       <parent link="${parent}" />
       <child link="${prefix}lfmetacarpal" />
-      <origin xyz="${reflect*-0.033} 0 0.02071" rpy="0 0 0" />
-      <axis xyz="0.573576436 0 ${reflect*0.819152044}" />
+      <origin xyz="${reflect*-0.033} 0 0.02071" rpy="0 ${reflect*-0.9599} 0" />
+      <axis xyz="1 0 0" />
       <limit lower="0" upper="${45/180*pi}" effort="2" velocity="2.0" />
       <dynamics damping="0.1" />

File: sr_description/hand/xacro/thumb/thbase.urdf.xacro (robot description, xacro)
@@ -59,5 +59,5 @@
       <parent link="${parent}" />
       <child link="${prefix}thbase" />
-      <origin xyz="${reflect*0.034} -0.00858 0.029" rpy="0 ${pi/4} ${pi/2-reflect*pi/2}" />
+      <origin xyz="${reflect*0.034} -0.00858 0.029" rpy="${-pi/4} 0 ${-reflect*pi/2}" />
       <axis xyz="0 0 ${reflect*-1}" />
       <limit lower="${-60/180*pi}" upper="${60/180*pi}" effort="5.0" velocity="4.0" />

File: sr_description/hand/xacro/thumb/thdistal.urdf.xacro (robot description, xacro)
@@ -167,5 +167,5 @@
         <parent link="${parent}" />
         <child link="${prefix}thdistal" />
-        <origin xyz="0 0 0.032" rpy="0 0 ${-pi/2}" />
+        <origin xyz="0 0 0.032" rpy="0 0 0" />
         <axis xyz="1 0 0" />
         <limit lower="-${15.0*pi/180}" upper="${90.0*pi/180}" effort="1.0" velocity="4.0" />

File: sr_description/hand/xacro/thumb/thhub.urdf.xacro (robot description, xacro)
@@ -69,5 +69,5 @@
         <child link="${prefix}thhub" />
         <origin xyz="0 0 0.038" rpy="0 0 0" />
-        <axis xyz="${reflect} 0 0" />
+        <axis xyz="0 ${reflect} 0" />
         <limit lower="${-12/180*pi}" upper="${12/180*pi}" effort="2.0" velocity="4.0" />
         <dynamics damping="0.2" />

File: sr_description/hand/xacro/thumb/thmiddle.urdf.xacro (robot description, xacro)
@@ -92,5 +92,5 @@
         <origin xyz="0 0 0" rpy="0 0 0" />
       </xacro:unless>
-      <axis xyz="0 -1 0" />
+      <axis xyz="1 0 0" />
       <limit lower="${-40/180*pi}" upper="${40/180*pi}" effort="2.0" velocity="2.0" />
       <dynamics damping="0.1" />

File: sr_description/hand/xacro/thumb/thproximal.urdf.xacro (robot description, xacro)
@@ -61,5 +61,5 @@
       <child link="${prefix}thproximal" />
       <origin xyz="0 0 0" rpy="0 0 0" />
-      <axis xyz="${reflect} 0 0" />
+      <axis xyz="0 ${reflect} 0" />
       <limit lower="0.0" upper="${70/180*pi}" effort="3" velocity="4.0" />
       <dynamics damping="0.2" />

Commit message: fixing collision for lf metacarpal

File: sr_description/hand/xacro/finger/lfmetacarpal/lfmetacarpal.urdf.xacro (robot description, xacro)
@@ -50,5 +50,7 @@
       </visual>
       <collision>
-        <origin xyz="0 0 0.038" rpy="0 0 0" />
+        <!--origin xyz="0 0 0.038" rpy="0 0 0" /-->
+        <origin xyz="0 0 0" rpy="0 ${reflect*0.9599} 0" />
+        <axis xyz="0.573576436 0 ${reflect*0.819152044}" />
         <geometry name="${prefix}lfmetacarpal_collision_geom">
           <box size="0.018 0.024 0.040" />

Commit message: fixing collision for lf metacarpal

File: sr_description/hand/xacro/finger/lfmetacarpal/lfmetacarpal.urdf.xacro (robot description, xacro)
@@ -51,5 +51,5 @@
       <collision>
         <!--origin xyz="0 0 0.038" rpy="0 0 0" /-->
-        <origin xyz="0 0 0" rpy="0 ${reflect*0.9599} 0" />
+        <origin xyz="0 0 0.038" rpy="0 ${reflect*0.9599} 0" />
         <axis xyz="0.573576436 0 ${reflect*0.819152044}" />
         <geometry name="${prefix}lfmetacarpal_collision_geom">

Commit message: Improving meshes

File: sr_description/hand/xacro/finger/lfmetacarpal/lfmetacarpal.urdf.xacro (robot description, xacro)
@@ -50,6 +50,5 @@
       </visual>
       <collision>
-        <!--origin xyz="0 0 0.038" rpy="0 0 0" /-->
-        <origin xyz="0 0 0.038" rpy="0 ${reflect*0.9599} 0" />
+        <origin xyz="${reflect*0.05397275/2.0} 0 ${0.038/2}" rpy="0 ${reflect*0.9599} 0" />
         <axis xyz="0.573576436 0 ${reflect*0.819152044}" />
         <geometry name="${prefix}lfmetacarpal_collision_geom">

File: sr_description/hand/xacro/thumb/thmiddle.urdf.xacro (robot description, xacro)
@@ -59,23 +59,29 @@
         </xacro:unless>
       </visual>
-      <collision>
-        <xacro:if value="${mid_sensor == 'bt_2p'}">
+      <xacro:if value="${mid_sensor == 'bt_2p'}">
+        <collision>
           <origin xyz="0 0 0.005" rpy="0 0 0" />
           <geometry name="${prefix}thmiddle_collision_geom">
             <box size="0.001 0.001 0.001" />
           </geometry>
-        </xacro:if>
-        <xacro:unless value="${mid_sensor == 'bt_2p'}">
+        </collision>
+      </xacro:if>
+      <xacro:unless value="${mid_sensor == 'bt_2p'}">
+        <collision>
           <origin xyz="0 0 0.012" rpy="0 0 0" />
           <geometry name="${prefix}thmiddle_collision_geom">
             <cylinder radius="0.011" length="0.018" />
           </geometry>
-        </xacro:unless>
-      </collision>
-      <xacro:unless value="${mid_sensor == 'bt_2p'}">
+        </collision>
         <collision>
           <origin xyz="0 0 0.019" rpy="0 0 0" />
           <geometry>
             <sphere radius="0.011" />
+          </geometry>
+        </collision>
+        <collision>
+          <origin xyz="0 0 0" rpy="0 1.5708 0" />
+          <geometry name="${prefix}${link_prefix}knuckle_collision_geom">
+            <cylinder radius="0.007" length="0.014" />
           </geometry>
         </collision>

Commit message: New version E4: Includes new meshes for lfmetacarpal and palm (#152)
* Adding lf_metacarpal

* Adding the new meshes for E4 version

* Fixing orientation

* Fixing orientation

* Fixing orientation

* adding E4 new palm meshes

* fixing collision for lf metacarpal

* fixing collision for lf metacarpal

* Improving meshes

* Improving meshes

* Adding palm material

* Adding palm material

* Adding lf metacarpal material

* Fixing lint errors

* Fixing lint errors

* Fixing lint errors

File: sr_description/hand/xacro/finger/lfmetacarpal/lfmetacarpal.urdf.xacro (robot description, xacro)
@@ -2,5 +2,5 @@
 <!--
  Software License Agreement (BSD License)
- Copyright © 2022 belongs to Shadow Robot Company Ltd.
+ Copyright © 2022-2023 belongs to Shadow Robot Company Ltd.
  All rights reserved.
  Redistribution and use in source and binary forms, with or without modification,
@@ -50,5 +50,6 @@
       </visual>
       <collision>
-        <origin xyz="0 0 0.038" rpy="0 0 0" />
+        <origin xyz="${reflect*0.05397275/2.0} 0 ${0.038/2}" rpy="0 ${reflect*0.9599} 0" />
+        <axis xyz="0.573576436 0 ${reflect*0.819152044}" />
         <geometry name="${prefix}lfmetacarpal_collision_geom">
           <box size="0.018 0.024 0.040" />

File: sr_description/hand/xacro/thumb/thmiddle.urdf.xacro (robot description, xacro)
@@ -2,5 +2,5 @@
 <!--
  Software License Agreement (BSD License)
- Copyright © 2022 belongs to Shadow Robot Company Ltd.
+ Copyright © 2022-2023 belongs to Shadow Robot Company Ltd.
  All rights reserved.
  Redistribution and use in source and binary forms, with or without modification,
@@ -59,23 +59,29 @@
         </xacro:unless>
       </visual>
-      <collision>
-        <xacro:if value="${mid_sensor == 'bt_2p'}">
+      <xacro:if value="${mid_sensor == 'bt_2p'}">
+        <collision>
           <origin xyz="0 0 0.005" rpy="0 0 0" />
           <geometry name="${prefix}thmiddle_collision_geom">
             <box size="0.001 0.001 0.001" />
           </geometry>
-        </xacro:if>
-        <xacro:unless value="${mid_sensor == 'bt_2p'}">
+        </collision>
+      </xacro:if>
+      <xacro:unless value="${mid_sensor == 'bt_2p'}">
+        <collision>
           <origin xyz="0 0 0.012" rpy="0 0 0" />
           <geometry name="${prefix}thmiddle_collision_geom">
             <cylinder radius="0.011" length="0.018" />
           </geometry>
-        </xacro:unless>
-      </collision>
-      <xacro:unless value="${mid_sensor == 'bt_2p'}">
+        </collision>
         <collision>
           <origin xyz="0 0 0.019" rpy="0 0 0" />
           <geometry>
             <sphere radius="0.011" />
+          </geometry>
+        </collision>
+        <collision>
+          <origin xyz="0 0 0.032" rpy="0 1.5708 0" />
+          <geometry>
+            <cylinder radius="0.010" length="0.014" />
           </geometry>
         </collision>

Commit message: Removing the axis from the link

File: sr_description/hand/xacro/finger/lfmetacarpal/lfmetacarpal.urdf.xacro (robot description, xacro)
@@ -42,5 +42,4 @@
       <visual>
         <origin xyz="0 0 0" rpy="0 ${reflect*0.9599} 0" />
-        <axis xyz="0.573576436 0 ${reflect*0.819152044}" />
         <geometry name="${prefix}lfmetacarpal_visual">
           <mesh filename="package://sr_description/meshes/components/lf_metacarpal/lf_metacarpal_${hand_version}.dae"
@@ -51,5 +50,4 @@
       <collision>
         <origin xyz="${reflect*0.05397275/2.0} 0 ${0.038/2}" rpy="0 ${reflect*0.9599} 0" />
-        <axis xyz="0.573576436 0 ${reflect*0.819152044}" />
         <geometry name="${prefix}lfmetacarpal_collision_geom">
           <box size="0.018 0.024 0.040" />

Commit message: Removing unnecessary rotation on the last thumb link. Correctly alligning thumb meshes with respective thumb links

File: sr_description/hand/xacro/finger/lfmetacarpal/lfmetacarpal.urdf.xacro (robot description, xacro)
@@ -36,5 +36,5 @@
     <link name="${prefix}lfmetacarpal">
       <inertial>
-        <origin xyz="0 0 0.04" rpy="0 0 0" />
+        <origin xyz="${reflect*0.05397275/1.7} 0 ${0.038/1.7}" rpy="0 ${reflect*0.9599} 0" />
         <mass value="0.030" />
         <inertia ixx="0.0000145" ixy="0.0" ixz="0.0" iyy="0.00001638" iyz="0.0" izz="0.000004272" />

File: sr_description/hand/xacro/thumb/thdistal.urdf.xacro (robot description, xacro)
@@ -46,5 +46,5 @@
         <parent link="${parent}" />
         <child link="${prefix}thdistal_J1_dummy" />
-        <origin xyz="0 0 0.02" rpy="0 0 ${-pi/2}" />
+        <origin xyz="0 0 0.02" rpy="0 0 0" />
         <axis xyz="1 0 0" />
         <limit lower="${20*pi/180}" upper="${20.1*pi/180}" effort="0.0" velocity="2.0" />
@@ -97,5 +97,5 @@
         <parent link="${prefix}thmiddle" />
         <child link="${prefix}thdistal" />
-        <origin xyz="0 0.0 0.01" rpy="0 0 ${-pi/2}" />
+        <origin xyz="0 0.0 0.01" rpy="0 0 0" />
       </joint>
       <!-- extra link to imaginary sphere in fingertip for FK/IK calculations -->

File: sr_description/hand/xacro/thumb/thmiddle.urdf.xacro (robot description, xacro)
@@ -42,5 +42,5 @@
       </inertial>
       <visual>
-        <origin xyz="0 0 0" rpy="0 0 0" />
+        <origin xyz="0 0 0" rpy="0 0 ${pi/2}" />
         <xacro:if value="${mid_sensor == 'bt_2p'}">
           <geometry name="${prefix}thmiddle_visual">

File: sr_description/hand/xacro/thumb/thproximal.urdf.xacro (robot description, xacro)
@@ -41,5 +41,5 @@
       </inertial>
       <visual>
-        <origin xyz="0 0 0" rpy="0 0 0" />
+        <origin xyz="0 0 0" rpy="0 0 ${pi/2}" />
         <geometry name="${prefix}thproximal_visual">
           <mesh filename="package://sr_description/meshes/components/th_proximal/th_proximal_${hand_version}.dae"

Commit message: Remove changes related to innertia

File: sr_description/hand/xacro/finger/lfmetacarpal/lfmetacarpal.urdf.xacro (robot description, xacro)
@@ -36,5 +36,5 @@
     <link name="${prefix}lfmetacarpal">
       <inertial>
-        <origin xyz="${reflect*0.05397275/1.7} 0 ${0.038/1.7}" rpy="0 ${reflect*0.9599} 0" />
+        <origin xyz="0 0 0.04" rpy="0 0 0" />
         <mass value="0.030" />
         <inertia ixx="0.0000145" ixy="0.0" ixz="0.0" iyy="0.00001638" iyz="0.0" izz="0.000004272" />
